File: qspi.sch (KiCad schematic (older format))
At the start: 4 parts

Commit message: SP: actually connect QSPI IO1
KiCad won't connect a bus ripper directly to a pin, it turns out -- this
is the one case where you _must_ have a wire.
Connections:
- wire segments 13 -> 14
Changed lines of the file:
@@
 	4300 3500 4800 3500
 Wire Bus Line
-	4200 2250 6350 2250
+	4200 2250 6450 2250
 Entry Wire Line
-	6250 3100 6350 3200
+	6350 3100 6450 3200
 Wire Bus Line
-	6350 2250 6350 3200
+	6450 2250 6450 3200
 Wire Bus Line
 	4200 2250 4100 2250
-Wire Bus Line
-	4200 2250 4200 3400
 Connection ~ 4200 2250
 Text HLabel 4100 2250 0    50   BiDi ~ 0
@@
 	1    0    0    -1
 $EndComp
+Wire Wire Line
+	6250 3100 6350 3100
+Wire Bus Line
+	4200 2250 4200 3400
 $EndSCHEMATC

Commit message: QSPI: host access buffers and connector
Parts:
- removed R? (x2): 10k, symbol Device:R
- removed U?: AT25SF081-SSHD-X, Package_SO:SOIC-8_3.9x4.9mm_P1.27mm, symbol Memory_Flash:AT25SF081-SSHD-X
- added C? (x2): 0µ1, symbol Device:C_Small
- added D?: 1N4148, symbol Device:D_Small
- added D?: D_TVS, symbol Device:D_TVS
- added J?: IDC, symbol Connector_Generic:Conn_02x08_Odd_Even
- added R?: 10k, symbol Device:R
- added U?: TXB0106PWR, Package_SO:TSSOP-16_4.4x5mm_P0.65mm, symbol txb01xx:TXB0106PWR
- added U?: W25Q256FVFxx, Package_SO:SOIC-16W_7.5x10.3mm_P1.27mm, symbol Memory_Flash:IS25WP256D-xM
Connections:
- net labels added: D0, D1, D2, D3, HOST_D0, HOST_D1, HOST_D2, HOST_D3, HOST_SCK, HOST_VCC, ~HOST_ACCESS, ~HOST_CE, ~RESET
- wire segments 14 -> 55
Other:
- note added: "Avoid backpowering host\n1V8 from SP 3V3"
- note added: "Host Side\nPowered by remote system\n1.2 - 3.6 V"
- note added: "Interleaved\nsignal/ground\non cable for\nintegrity"
- note added: "OE is sampled relative to Vcca;\npull it up when Vcca is powered.\nWhen Vcca unpowered the chip\nignores it. SP access is open drain."
- note added: "SP has excl control of ~RESET"
- moved on the sheet: C?

Commit message: ERC clean.
- Power flags.
- NCs.
- Fixed a few net typos that resulted in disconnects.
Changed lines of the file:
@@
 	1    0    0    -1
 $EndComp
+Text Notes 1700 4950 0    50   ~ 0
+Interleaved\nsignal/ground\non cable for\nintegrity
+Wire Wire Line
+	2850 4500 2850 4200
 Wire Bus Line
 	6350 2550 6350 4900
-Text Notes 1700 4950 0    50   ~ 0
-Interleaved\nsignal/ground\non cable for\nintegrity
+$Comp
+L power:PWR_FLAG #FLG?
+U 1 1 60106F7A
+P 2850 4200
+F 0 "#FLG?" H 2850 4275 50  0001 C CNN
+F 1 "PWR_FLAG" H 2850 4373 50  0000 C CNN
+F 2 "" H 2850 4200 50  0001 C CNN
+F 3 "~" H 2850 4200 50  0001 C CNN
+	1    2850 4200
+	1    0    0    -1
+$EndComp
 $EndSCHEMATC

Commit message: Annotate in preparation for review
Parts:
- gave numbers to parts that had none: 9
Changed lines of the file:
@@
 $EndDescr
 $Comp
-L power:+3V3 #PWR?
+L power:+3V3 #PWR0806
 U 1 1 5F3B01D5
 P 7700 3100
-F 0 "#PWR?" H 7700 2950 50  0001 C CNN
+F 0 "#PWR0806" H 7700 2950 50  0001 C CNN
 F 1 "+3V3" H 7715 3273 50  0000 C CNN
 F 2 "" H 7700 3100 50  0001 C CNN
@@
 $EndComp
 $Comp
-L power:GND #PWR?
+L power:GND #PWR0807
 U 1 1 5F3B036B
 P 7700 4100
-F 0 "#PWR?" H 7700 3850 50  0001 C CNN
+F 0 "#PWR0807" H 7700 3850 50  0001 C CNN
 F 1 "GND" H 7705 3927 50  0000 C CNN
 F 2 "" H 7700 4100 50  0001 C CNN
@@
 D[0..3]
 $Comp
-L Device:C_Small C?
+L Device:C_Small C803
 U 1 1 5F3B7D89
 P 8800 3150
-F 0 "C?" H 8892 3196 50  0000 L CNN
+F 0 "C803" H 8892 3196 50  0000 L CNN
 F 1 "0µ1" H 8892 3105 50  0000 L CNN
 F 2 "" H 8800 3150 50  0001 C CNN
@@
 $EndComp
 $Comp
-L power:+3V3 #PWR?
+L power:+3V3 #PWR0808
 U 1 1 5F3B7FA5
 P 8800 3050
-F 0 "#PWR?" H 8800 2900 50  0001 C CNN
+F 0 "#PWR0808" H 8800 2900 50  0001 C CNN
 F 1 "+3V3" H 8815 3223 50  0000 C CNN
 F 2 "" H 8800 3050 50  0001 C CNN
@@
 $EndComp
 $Comp
-L power:GND #PWR?
+L power:GND #PWR0809
 U 1 1 5F3B8191
 P 8800 3250
-F 0 "#PWR?" H 8800 3000 50  0001 C CNN
+F 0 "#PWR0809" H 8800 3000 50  0001 C CNN
 F 1 "GND" H 8805 3077 50  0000 C CNN
 F 2 "" H 8800 3250 50  0001 C CNN
@@
 D3
 $Comp
-L txb01xx:TXB0106PWR U?
+L txb01xx:TXB0106PWR U801
 U 1 1 5F376223
 P 4800 4800
-F 0 "U?" H 4800 5465 50  0000 C CNN
+F 0 "U801" H 4800 5465 50  0000 C CNN
 F 1 "TXB0106PWR" H 4800 5374 50  0000 C CNN
 F 2 "Package_SO:TSSOP-16_4.4x5mm_P0.65mm" H 4800 4800 50  0001 C CNN
@@
 $EndComp
 $Comp
-L Device:R R?
+L Device:R R801
 U 1 1 5F376F98
 P 4050 5200
-F 0 "R?" V 3950 5200 50  0000 C CNN
+F 0 "R801" V 3950 5200 50  0000 C CNN
 F 1 "10k" V 4050 5200 50  0000 C CNN
 F 2 "" V 3980 5200 50  0001 C CNN
@@
 $EndComp
 $Comp
-L Connector_Generic:Conn_02x08_Odd_Even J?
+L Connector_Generic:Conn_02x08_Odd_Even J801
 U 1 1 5F378801
 P 2600 4800
-F 0 "J?" H 2650 4175 50  0000 C CNN
+F 0 "J801" H 2650 4175 50  0000 C CNN
 F 1 "IDC" H 2650 4266 50  0000 C CNN
 F 2 "" H 2600 4800 50  0001 C CNN
@@
 	2300 5100 2300 5150
 $Comp
-L power:GND #PWR?
+L power:GND #PWR0801
 U 1 1 5F37D4F5
 P 2300 5150
-F 0 "#PWR?" H 2300 4900 50  0001 C CNN
+F 0 "#PWR0801" H 2300 4900 50  0001 C CNN
 F 1 "GND" H 2305 4977 50  0000 C CNN
 F 2 "" H 2300 5150 50  0001 C CNN
@@
 	5400 5100 5400 5600
 $Comp
-L power:GND #PWR?
+L power:GND #PWR0804
 U 1 1 5F385C9A
 P 5400 5850
-F 0 "#PWR?" H 5400 5600 50  0001 C CNN
+F 0 "#PWR0804" H 5400 5600 50  0001 C CNN
 F 1 "GND" H 5405 5677 50  0000 C CNN
 F 2 "" H 5400 5850 50  0001 C CNN
@@
 	5400 4500 5400 3900
 $Comp
-L power:+3V3 #PWR?
+L power:+3V3 #PWR0803
 U 1 1 5F386B12
 P 5400 3900
-F 0 "#PWR?" H 5400 3750 50  0001 C CNN
+F 0 "#PWR0803" H 5400 3750 50  0001 C CNN
 F 1 "+3V3" H 5415 4073 50  0000 C CNN
 F 2 "" H 5400 3900 50  0001 C CNN
@@
 $EndComp
 $Comp
-L Memory_Flash:IS25WP256D-xM U?
+L Memory_Flash:IS25WP256D-xM U802
 U 1 1 5F386ECD
 P 7700 3600
-F 0 "U?" H 7400 4050 50  0000 C CNN
+F 0 "U802" H 7400 4050 50  0000 C CNN
 F 1 "W25Q256FVFxx" H 8000 3150 50  0000 C CNN
 F 2 "Package_SO:SOIC-16W_7.5x10.3mm_P1.27mm" H 7750 4200 50  0001 C CNN
@@
 OE is sampled relative to Vcca;\npull it up when Vcca is powered.\nWhen Vcca unpowered the chip\nignores it. SP access is open drain.
 $Comp
-L Device:D_Small D?
+L Device:D_Small D802
 U 1 1 5F3AC322
 P 6000 5250
-F 0 "D?" H 6000 5043 50  0000 C CNN
+F 0 "D802" H 6000 5043 50  0000 C CNN
 F 1 "1N4148" H 6000 5134 50  0000 C CNN
 F 2 "" V 6000 5250 50  0001 C CNN
@@
 Avoid backpowering host\n1V8 from SP 3V3
 $Comp
-L Device:D_TVS D?
+L Device:D_TVS D801
 U 1 1 5F3AD847
 P 5550 5450
-F 0 "D?" V 5596 5370 50  0000 R CNN
+F 0 "D801" V 5596 5370 50  0000 R CNN
 F 1 "D_TVS" V 5505 5370 50  0000 R CNN
 F 2 "" H 5550 5450 50  0001 C CNN
@@
 SP has excl control of ~RESET
 $Comp
-L Device:C_Small C?
+L Device:C_Small C802
 U 1 1 5F3CC21E
 P 5650 4050
-F 0 "C?" H 5742 4096 50  0000 L CNN
+F 0 "C802" H 5742 4096 50  0000 L CNN
 F 1 "0µ1" H 5742 4005 50  0000 L CNN
 F 2 "" H 5650 4050 50  0001 C CNN
@@
 $EndComp
 $Comp
-L power:GND #PWR?
+L power:GND #PWR0805
 U 1 1 5F3CC22A
 P 5650 4150
-F 0 "#PWR?" H 5650 3900 50  0001 C CNN
+F 0 "#PWR0805" H 5650 3900 50  0001 C CNN
 F 1 "GND" H 5655 3977 50  0000 C CNN
 F 2 "" H 5650 4150 50  0001 C CNN
@@
 Connection ~ 5400 3900
 $Comp
-L Device:C_Small C?
+L Device:C_Small C801
 U 1 1 5F3CEDAC
 P 2850 5200
-F 0 "C?" H 2942 5246 50  0000 L CNN
+F 0 "C801" H 2942 5246 50  0000 L CNN
 F 1 "0µ1" H 2942 5155 50  0000 L CNN
 F 2 "" H 2850 5200 50  0001 C CNN
@@
 Connection ~ 2850 5100
 $Comp
-L power:GND #PWR?
+L power:GND #PWR0802
 U 1 1 5F3D0231
 P 2850 5300
-F 0 "#PWR?" H 2850 5050 50  0001 C CNN
+F 0 "#PWR0802" H 2850 5050 50  0001 C CNN
 F 1 "GND" H 2855 5127 50  0000 C CNN
 F 2 "" H 2850 5300 50  0001 C CNN
@@
 	6350 2550 6350 4900
 $Comp
-L power:PWR_FLAG #FLG?
+L power:PWR_FLAG #FLG0801
 U 1 1 60106F7A
 P 2850 4200
-F 0 "#FLG?" H 2850 4275 50  0001 C CNN
+F 0 "#FLG0801" H 2850 4275 50  0001 C CNN
 F 1 "PWR_FLAG" H 2850 4373 50  0000 C CNN
 F 2 "" H 2850 4200 50  0001 C CNN

Commit message: Fixes from first SP reviews.
- TXB0106 OE is active high; rename nets accordingly.
- STM32H755 is pin-incompatible with the rest of the STM32H7 series, but
  it's not clear that we need its particular features -- switch to
  STM32H753.
Connections:
- net GND: now also R801.2
- net HOST_VCC: no longer R801.2
- net ~HOST_ACCESS renamed HOST_ACCESS
Other:
- note added: "OE is sampled relative to Vcca;\nkeep it pulled down until SP\ndrives it."
- note removed: "OE is sampled relative to Vcca;\npull it up when Vcca is powered.\nWhen Vcca unpowered the chip\nignores it. SP access is open drain."
Changed lines of the file:
@@
-$EndComp
-$Comp
-L Device:R R801
-U 1 1 5F376F98
-P 4050 5200
-F 0 "R801" V 3950 5200 50  0000 C CNN
-F 1 "10k" V 4050 5200 50  0000 C CNN
-F 2 "" V 3980 5200 50  0001 C CNN
-F 3 "~" H 4050 5200 50  0001 C CNN
-	1    4050 5200
-	0    1    1    0
 $EndComp
 $Comp
@@
 	4250 4400 2800 4400
 Wire Wire Line
-	4250 4500 3800 4500
-Wire Wire Line
 	4250 4600 2800 4600
 Wire Wire Line
@@
 	2800 5000 4250 5000
 Wire Wire Line
-	4250 5100 4250 5200
-Wire Wire Line
-	4250 5200 4200 5200
-Wire Wire Line
-	3800 5200 3800 4500
-Wire Wire Line
-	3900 5200 3800 5200
-Connection ~ 3800 4500
-Wire Wire Line
-	3800 4500 2850 4500
-Wire Wire Line
-	4250 5200 4250 5250
-Wire Wire Line
 	4250 5250 5550 5250
-Connection ~ 4250 5200
 Wire Wire Line
 	5350 4600 5700 4600
@@
 	6750 3600 6850 3600
 Text HLabel 6250 5250 2    50   Input ~ 0
-~HOST_ACCESS
+HOST_ACCESS
 Text Notes 4150 4300 2    50   ~ 0
 Host Side\nPowered by remote system\n1.2 - 3.6 V
 Text Notes 3700 5600 0    50   ~ 0
-OE is sampled relative to Vcca;\npull it up when Vcca is powered.\nWhen Vcca unpowered the chip\nignores it. SP access is open drain.
+OE is sampled relative to Vcca;\nkeep it pulled down until SP\ndrives it.
 $Comp
 L Device:D_Small D802
@@
 Wire Wire Line
 	2850 4500 2850 4200
-Wire Bus Line
-	6350 2550 6350 4900
 $Comp
 L power:PWR_FLAG #FLG0801
@@
 	1    0    0    -1
 $EndComp
+Wire Bus Line
+	6350 2550 6350 4900
+Wire Wire Line
+	4250 5200 4250 5250
+Wire Wire Line
+	4250 5100 4250 5200
+Connection ~ 4250 5200
+Wire Wire Line
+	4250 5200 4200 5200
+Wire Wire Line
+	3900 5200 3800 5200
+$Comp
+L Device:R R801
+U 1 1 5F376F98
+P 4050 5200
+F 0 "R801" V 3950 5200 50  0000 C CNN
+F 1 "10k" V 4050 5200 50  0000 C CNN
+F 2 "" V 3980 5200 50  0001 C CNN
+F 3 "~" H 4050 5200 50  0001 C CNN
+	1    4050 5200
+	0    1    1    0
+$EndComp
+Wire Wire Line
+	2850 4500 4250 4500
+$Comp
+L power:GND #PWR0810
+U 1 1 5F41A0A1
+P 3800 5200
+F 0 "#PWR0810" H 3800 4950 50  0001 C CNN
+F 1 "GND" V 3805 5072 50  0000 R CNN
+F 2 "" H 3800 5200 50  0001 C CNN
+F 3 "" H 3800 5200 50  0001 C CNN
+	1    3800 5200
+	0    1    1    0
+$EndComp
 $EndSCHEMATC

Commit message: QSPI: fix issue introduced by my last fix.
Diode and TVS were no longer relevant since the two power nets no longer
meet at OE.
Parts:
- removed D801: D_TVS, symbol Device:D_TVS
- removed D802: 1N4148, symbol Device:D_Small
Connections:
- net HOST_ACCESS: now also R801.1, U801.8 (OE)
Other:
- note added: "OE is sampled relative to Vcca.\nVcca and Vccb share GND.\nPull it down to keep buffer\ndisabled until SP drives high.\nInput appears to be 3V3 tolerant\neven for 1V8 Vcca."
- note removed: "Avoid backpowering host\n1V8 from SP 3V3"
- note removed: "OE is sampled relative to Vcca;\nkeep it pulled down until SP\ndrives it."
Changed lines of the file:
@@
 	2800 5000 4250 5000
 Wire Wire Line
-	4250 5250 5550 5250
-Wire Wire Line
 	5350 4600 5700 4600
 Wire Wire Line
@@
 Wire Wire Line
 	5350 5100 5400 5100
-Wire Wire Line
-	5400 5100 5400 5600
 $Comp
 L power:GND #PWR0804
@@
 Text Notes 4150 4300 2    50   ~ 0
 Host Side\nPowered by remote system\n1.2 - 3.6 V
-Text Notes 3700 5600 0    50   ~ 0
-OE is sampled relative to Vcca;\nkeep it pulled down until SP\ndrives it.
-$Comp
-L Device:D_Small D802
-U 1 1 5F3AC322
-P 6000 5250
-F 0 "D802" H 6000 5043 50  0000 C CNN
-F 1 "1N4148" H 6000 5134 50  0000 C CNN
-F 2 "" V 6000 5250 50  0001 C CNN
-F 3 "~" V 6000 5250 50  0001 C CNN
-	1    6000 5250
-	-1   0    0    1
-$EndComp
-Wire Wire Line
-	6100 5250 6250 5250
-Text Notes 5850 5500 0    50   ~ 0
-Avoid backpowering host\n1V8 from SP 3V3
-$Comp
-L Device:D_TVS D801
-U 1 1 5F3AD847
-P 5550 5450
-F 0 "D801" V 5596 5370 50  0000 R CNN
-F 1 "D_TVS" V 5505 5370 50  0000 R CNN
-F 2 "" H 5550 5450 50  0001 C CNN
-F 3 "~" H 5550 5450 50  0001 C CNN
-	1    5550 5450
-	0    -1   -1   0
-$EndComp
-Wire Wire Line
-	5550 5300 5550 5250
-Connection ~ 5550 5250
-Wire Wire Line
-	5550 5250 5900 5250
-Wire Wire Line
-	5550 5600 5400 5600
-Connection ~ 5400 5600
-Wire Wire Line
-	5400 5600 5400 5850
+Text Notes 3600 5800 0    50   ~ 0
+OE is sampled relative to Vcca.\nVcca and Vccb share GND.\nPull it down to keep buffer\ndisabled until SP drives high.\nInput appears to be 3V3 tolerant\neven for 1V8 Vcca.
 Text Label 2800 4400 0    50   ~ 0
 ~HOST_CE
@@
 	1    0    0    -1
 $EndComp
-Wire Bus Line
-	6350 2550 6350 4900
 Wire Wire Line
 	4250 5200 4250 5250
@@
 	0    1    1    0
 $EndComp
+Wire Wire Line
+	4250 5250 6250 5250
+Wire Wire Line
+	5400 5100 5400 5850
+Wire Bus Line
+	6350 2550 6350 4900
 $EndSCHEMATC

Commit message: Assign noncontroversial footprints.
- For components that only come in one flavor, use it.
- For passives, go with 0603, except for current sense resistors.
- Use the Yamaichi socket footprint for the 'h7
- Delete at least one default but wrong association.
Parts:
- C801, C802: footprint (none) -> Capacitor_SMD:C_0603_1608Metric
- C803: footprint (none) -> LED_SMD:LED_0603_1608Metric_Castellated
- J801: footprint (none) -> Connector_IDC:IDC-Header_2x08_P2.54mm_Vertical
- R801: footprint (none) -> Resistor_SMD:R_0603_1608Metric
Changed lines of the file:
@@
 F 0 "C803" H 8892 3196 50  0000 L CNN
 F 1 "0µ1" H 8892 3105 50  0000 L CNN
-F 2 "" H 8800 3150 50  0001 C CNN
+F 2 "LED_SMD:LED_0603_1608Metric_Castellated" H 8800 3150 50  0001 C CNN
 F 3 "~" H 8800 3150 50  0001 C CNN
 	1    8800 3150
@@
 F 0 "J801" H 2650 4175 50  0000 C CNN
 F 1 "IDC" H 2650 4266 50  0000 C CNN
-F 2 "" H 2600 4800 50  0001 C CNN
+F 2 "Connector_IDC:IDC-Header_2x08_P2.54mm_Vertical" H 2600 4800 50  0001 C CNN
 F 3 "~" H 2600 4800 50  0001 C CNN
 	1    2600 4800
@@
 F 0 "C802" H 5742 4096 50  0000 L CNN
 F 1 "0µ1" H 5742 4005 50  0000 L CNN
-F 2 "" H 5650 4050 50  0001 C CNN
+F 2 "Capacitor_SMD:C_0603_1608Metric" H 5650 4050 50  0001 C CNN
 F 3 "~" H 5650 4050 50  0001 C CNN
 	1    5650 4050
@@
 F 0 "C801" H 2942 5246 50  0000 L CNN
 F 1 "0µ1" H 2942 5155 50  0000 L CNN
-F 2 "" H 2850 5200 50  0001 C CNN
+F 2 "Capacitor_SMD:C_0603_1608Metric" H 2850 5200 50  0001 C CNN
 F 3 "~" H 2850 5200 50  0001 C CNN
 	1    2850 5200
@@
 F 0 "R801" V 3950 5200 50  0000 C CNN
 F 1 "10k" V 4050 5200 50  0000 C CNN
-F 2 "" V 3980 5200 50  0001 C CNN
+F 2 "Resistor_SMD:R_0603_1608Metric" V 3980 5200 50  0001 C CNN
 F 3 "~" H 4050 5200 50  0001 C CNN
 	1    4050 5200
