File: qspi.sch (KiCad schematic (older format))
At the start: 7 parts, among them J801 IDC, U801 TXB0106PWR, U802 W25Q256FVFxx

Commit message: PCB: densification sprint
Most components are now placed in plausible final locations.

About 40% of the board is routed.

Board size is down to about 210x170mm.

Found and fixed a class of errors in the schematic: it turns out that
within one sheet, local labels and hierarchical labels with the same
name are implicitly connected. This caused some of our signals that exit
blocks through e.g. a slew rate control resistor to wind up with both
ends of the resistor connected to the same net!
Parts:
- J801: footprint Connector_IDC:IDC-Header_2x08_P2.54mm_Vertical -> Connector_PinHeader_2.54mm:PinHeader_2x08_P2.54mm_Vertical_SMD
Changed lines of the file:
@@
 F 0 "J801" H 2650 4175 50  0000 C CNN
 F 1 "IDC" H 2650 4266 50  0000 C CNN
-F 2 "Connector_IDC:IDC-Header_2x08_P2.54mm_Vertical" H 2600 4800 50  0001 C CNN
+F 2 "Connector_PinHeader_2.54mm:PinHeader_2x08_P2.54mm_Vertical_SMD" H 2600 4800 50  0001 C CNN
 F 3 "~" H 2600 4800 50  0001 C CNN
 	1    2600 4800

Commit message: PCB: more layout, FPGA expansion, mounting holes
Also fixed a couple of incorrect footprint assignments.
Parts:
- C803: footprint LED_SMD:LED_0603_1608Metric_Castellated -> Capacitor_SMD:C_0603_1608Metric
Changed lines of the file:
@@
 F 0 "C803" H 8892 3196 50  0000 L CNN
 F 1 "0µ1" H 8892 3105 50  0000 L CNN
-F 2 "LED_SMD:LED_0603_1608Metric_Castellated" H 8800 3150 50  0001 C CNN
+F 2 "Capacitor_SMD:C_0603_1608Metric" H 8800 3150 50  0001 C CNN
 F 3 "~" H 8800 3150 50  0001 C CNN
 	1    8800 3150

Commit message: Switch IDC connectors to SMD footprints.
Parts:
- J801: footprint Connector_PinHeader_2.54mm:PinHeader_2x08_P2.54mm_Vertical_SMD -> idc-smd:IDC-Header_02x08_2.54mm_Vertical_SMD
Changed lines of the file:
@@
 F 0 "J801" H 2650 4175 50  0000 C CNN
 F 1 "IDC" H 2650 4266 50  0000 C CNN
-F 2 "Connector_PinHeader_2.54mm:PinHeader_2x08_P2.54mm_Vertical_SMD" H 2600 4800 50  0001 C CNN
+F 2 "idc-smd:IDC-Header_02x08_2.54mm_Vertical_SMD" H 2600 4800 50  0001 C CNN
 F 3 "~" H 2600 4800 50  0001 C CNN
 	1    2600 4800

Commit message: MB: annotate everything with mfg/MPN
Parts:
- C801, C802, C803, R801: Mfg Part Num (none) -> generic
- J801: Mfg (none) -> CNC Tech; Mfg Part Num (none) -> 3020-16-0300-00
- U801: Mfg (none) -> Texas Instruments; Mfg Part Num (none) -> TXB0106PWR
- U802: Mfg (none) -> Winbond; Mfg Part Num (none) -> W25Q256FVFIG
Changed lines of the file:
@@
 F 2 "Capacitor_SMD:C_0603_1608Metric" H 8800 3150 50  0001 C CNN
 F 3 "~" H 8800 3150 50  0001 C CNN
+F 4 "generic" H 8800 3150 50  0001 C CNN "Mfg Part Num"
 	1    8800 3150
 	1    0    0    -1
@@
 F 2 "Package_SO:TSSOP-16_4.4x5mm_P0.65mm" H 4800 4800 50  0001 C CNN
 F 3 "" H 4800 4800 50  0001 C CNN
+F 4 "Texas Instruments" H 4800 4800 50  0001 C CNN "Mfg"
+F 5 "TXB0106PWR" H 4800 4800 50  0001 C CNN "Mfg Part Num"
 	1    4800 4800
 	1    0    0    -1
@@
 F 2 "idc-smd:IDC-Header_02x08_2.54mm_Vertical_SMD" H 2600 4800 50  0001 C CNN
 F 3 "~" H 2600 4800 50  0001 C CNN
+F 4 "CNC Tech" H 2600 4800 50  0001 C CNN "Mfg"
+F 5 "3020-16-0300-00" H 2600 4800 50  0001 C CNN "Mfg Part Num"
 	1    2600 4800
 	-1   0    0    1
@@
 F 2 "Package_SO:SOIC-16W_7.5x10.3mm_P1.27mm" H 7750 4200 50  0001 C CNN
 F 3 "http://www.issi.com/WW/pdf/IS25LP(WP)256D.pdf" H 7750 3100 50  0001 C CNN
+F 4 "Winbond" H 7700 3600 50  0001 C CNN "Mfg"
+F 5 "W25Q256FVFIG" H 7700 3600 50  0001 C CNN "Mfg Part Num"
 	1    7700 3600
 	1    0    0    -1
@@
 F 2 "Capacitor_SMD:C_0603_1608Metric" H 5650 4050 50  0001 C CNN
 F 3 "~" H 5650 4050 50  0001 C CNN
+F 4 "generic" H 5650 4050 50  0001 C CNN "Mfg Part Num"
 	1    5650 4050
 	1    0    0    -1
@@
 F 2 "Capacitor_SMD:C_0603_1608Metric" H 2850 5200 50  0001 C CNN
 F 3 "~" H 2850 5200 50  0001 C CNN
+F 4 "generic" H 2850 5200 50  0001 C CNN "Mfg Part Num"
 	1    2850 5200
 	1    0    0    -1
@@
 F 2 "Resistor_SMD:R_0603_1608Metric" V 3980 5200 50  0001 C CNN
 F 3 "~" H 4050 5200 50  0001 C CNN
+F 4 "generic" H 4050 5200 50  0001 C CNN "Mfg Part Num"
 	1    4050 5200
 	0    1    1    0

Commit message: MB: MPNs for capacitors, adjust some footprints
Can't get a 2kV 10000p cap in 0603 as it turns out
Parts:
- C801, C802, C803: Mfg (none) -> Samsung Electro-Mechanics; Mfg Part Num generic -> CL10B104KB8NNWC
Changed lines of the file:
@@
 F 2 "Capacitor_SMD:C_0603_1608Metric" H 8800 3150 50  0001 C CNN
 F 3 "~" H 8800 3150 50  0001 C CNN
-F 4 "generic" H 8800 3150 50  0001 C CNN "Mfg Part Num"
+F 4 "CL10B104KB8NNWC" H 8800 3150 50  0001 C CNN "Mfg Part Num"
+F 5 "Samsung Electro-Mechanics" H 8800 3150 50  0001 C CNN "Mfg"
 	1    8800 3150
 	1    0    0    -1
@@
 F 2 "Capacitor_SMD:C_0603_1608Metric" H 5650 4050 50  0001 C CNN
 F 3 "~" H 5650 4050 50  0001 C CNN
-F 4 "generic" H 5650 4050 50  0001 C CNN "Mfg Part Num"
+F 4 "CL10B104KB8NNWC" H 5650 4050 50  0001 C CNN "Mfg Part Num"
+F 5 "Samsung Electro-Mechanics" H 5650 4050 50  0001 C CNN "Mfg"
 	1    5650 4050
 	1    0    0    -1
@@
 F 2 "Capacitor_SMD:C_0603_1608Metric" H 2850 5200 50  0001 C CNN
 F 3 "~" H 2850 5200 50  0001 C CNN
-F 4 "generic" H 2850 5200 50  0001 C CNN "Mfg Part Num"
+F 4 "CL10B104KB8NNWC" H 2850 5200 50  0001 C CNN "Mfg Part Num"
+F 5 "Samsung Electro-Mechanics" H 2850 5200 50  0001 C CNN "Mfg"
 	1    2850 5200
 	1    0    0    -1

Commit message: MB: assign single resistors
Parts:
- R801: Mfg (none) -> Bourns; Mfg Part Num generic -> CR0603-JW-103ELF
Changed lines of the file:
@@
 F 2 "Resistor_SMD:R_0603_1608Metric" V 3980 5200 50  0001 C CNN
 F 3 "~" H 4050 5200 50  0001 C CNN
-F 4 "generic" H 4050 5200 50  0001 C CNN "Mfg Part Num"
+F 4 "CR0603-JW-103ELF" H 4050 5200 50  0001 C CNN "Mfg Part Num"
+F 5 "Bourns" H 4050 5200 50  0001 C CNN "Mfg"
 	1    4050 5200
 	0    1    1    0
