File: rot.sch (KiCad schematic (older format))
At the start: 56 parts

Commit message: ERC clean.
- Power flags.
- NCs.
- Fixed a few net typos that resulted in disconnects.
Connections:
- net PIO0_29 is gone; now on net PIO0_21: J?.1 (Pin_1)
- net VDD_PMU is gone; now on net FB: C?.1, C?.1, C?.1, C?.1, J?.12 (Pin_12), L?.2, U?.28 (VDD_PMU), U?.29 (FB)
- net LX: now also L?.1, U?.31 (LX)
- net PIO1_0: now also U?.4 (PIO1_0/ADC0_11)
Changed lines of the file:
@@
 $EndComp
-Wire Wire Line
-	13150 2800 13950 2800
 Wire Wire Line
 	13950 2800 13950 2900
@@
 Connection ~ 4050 1750
 Wire Wire Line
-	4050 1750 4550 1750
+	4050 1750 4450 1750
 Wire Wire Line
 	4050 2100 4050 2150
@@
 Text Label 20150 8000 2    50   ~ 0
 PIO0_20
-Text Label 20150 8250 2    50   ~ 0
-PIO0_29
 Text Label 20150 8350 2    50   ~ 0
 PIO0_22
@@
 Wire Wire Line
 	13500 7050 13500 7100
+$Comp
+L power:PWR_FLAG #FLG?
+U 1 1 60159E34
+P 4450 1750
+F 0 "#FLG?" H 4450 1825 50  0001 C CNN
+F 1 "PWR_FLAG" H 4450 1923 50  0000 C CNN
+F 2 "" H 4450 1750 50  0001 C CNN
+F 3 "~" H 4450 1750 50  0001 C CNN
+	1    4450 1750
+	1    0    0    -1
+$EndComp
+Connection ~ 4450 1750
+Wire Wire Line
+	4450 1750 4550 1750
+$Comp
+L power:PWR_FLAG #FLG?
+U 1 1 6015AAE3
+P 13400 2800
+F 0 "#FLG?" H 13400 2875 50  0001 C CNN
+F 1 "PWR_FLAG" H 13400 2973 50  0000 C CNN
+F 2 "" H 13400 2800 50  0001 C CNN
+F 3 "~" H 13400 2800 50  0001 C CNN
+	1    13400 2800
+	1    0    0    -1
+$EndComp
+Connection ~ 13400 2800
+Wire Wire Line
+	13400 2800 13950 2800
+Wire Wire Line
+	13150 2800 13400 2800
+Text Label 20150 8250 2    50   ~ 0
+PIO0_21
+Text Label 13200 2900 0    50   ~ 0
+LX
+Text Label 13200 2800 0    50   ~ 0
+FB
+Text Label 13150 3450 0    50   ~ 0
+PIO1_0
 $EndSCHEMATC

Commit message: Annotate in preparation for review
Parts:
- gave numbers to parts that had none: 56

Commit message: Assign noncontroversial footprints.
- For components that only come in one flavor, use it.
- For passives, go with 0603, except for current sense resistors.
- Use the Yamaichi socket footprint for the 'h7
- Delete at least one default but wrong association.
Parts:
- C201, C202, C203, C204, C205, C206, C207, C208, C209, C210, C211, C212, C213, C214, C215, C216, C217, C218, C219, C220, C221, C222: footprint (none) -> Capacitor_SMD:C_0603_1608Metric
- D201, D202: footprint (none) -> LED_SMD:LED_0603_1608Metric_Castellated
- FB201, FB202: footprint (none) -> Inductor_SMD:L_0603_1608Metric
- J201: footprint (none) -> Connector_PinHeader_2.54mm:PinHeader_1x04_P2.54mm_Vertical
- J202: footprint (none) -> Connector_PinHeader_1.27mm:PinHeader_2x05_P1.27mm_Vertical_SMD
- J203, J204, J205, J206: footprint (none) -> Connector_PinHeader_2.00mm:PinHeader_1x16_P2.00mm_Vertical
- JP201, JP202, JP203, JP204: footprint (none) -> Jumper:SolderJumper-3_P1.3mm_Bridged12_RoundedPad1.0x1.5mm
- L201, R201, R202, R203, R204, R205, R206, R207, R208, R209, R210, R211, R212, R213, R214: footprint (none) -> Resistor_SMD:R_0603_1608Metric

Commit message: lpc55 htqfp64 footprint
Parts:
- U201: footprint (none) -> lpc55:HTQFP-64-1EP_10x10mm_P0.5mm_EP3.6x3.6mm
Changed lines of the file:
@@
 F 0 "U201" H 11600 5500 50  0000 C CNN
 F 1 "LPC55S28JBD64" H 11600 5400 50  0000 C CNN
-F 2 "" H 11600 5400 50  0001 C CNN
+F 2 "lpc55:HTQFP-64-1EP_10x10mm_P0.5mm_EP3.6x3.6mm" H 11600 5400 50  0001 C CNN
 F 3 "" H 11600 5400 50  0001 C CNN
 	1    11600 5400

Commit message: Button and switch footprint associations.
Parts:
- SW201: footprint (none) -> Button_Switch_SMD:SW_SPDT_CK-JS102011SAQN
- SW202: footprint (none) -> Button_Switch_SMD:SW_Push_1P1T_NO_Vertical_Wuerth_434133025816
Changed lines of the file:
@@
 F 0 "SW202" V 3550 9500 50  0000 L CNN
 F 1 "SW_SPST" V 3600 9500 50  0000 L CNN
-F 2 "" H 3600 9400 50  0001 C CNN
+F 2 "Button_Switch_SMD:SW_Push_1P1T_NO_Vertical_Wuerth_434133025816" H 3600 9400 50  0001 C CNN
 F 3 "~" H 3600 9400 50  0001 C CNN
 	1    3600 9400
@@
 F 0 "SW201" H 3450 11500 50  0000 C CNN
 F 1 "SW_SPDT" H 3450 11400 50  0000 C CNN
-F 2 "" H 3450 11200 50  0001 C CNN
+F 2 "Button_Switch_SMD:SW_SPDT_CK-JS102011SAQN" H 3450 11200 50  0001 C CNN
 F 3 "~" H 3450 11200 50  0001 C CNN
 	1    3450 11200

Commit message: Pick arbitrary but not unreasonable footprints for rest.
Parts:
- Y201, Y202: footprint (none) -> Crystal:Crystal_SMD_Abracon_ABM3-2Pin_5.0x3.2mm
Changed lines of the file:
@@
 F 0 "Y201" H 2300 5050 50  0000 C CNN
 F 1 "16MHz" H 2300 4950 50  0000 C CNN
-F 2 "" H 2300 4750 50  0001 C CNN
+F 2 "Crystal:Crystal_SMD_Abracon_ABM3-2Pin_5.0x3.2mm" H 2300 4750 50  0001 C CNN
 F 3 "~" H 2300 4750 50  0001 C CNN
 	1    2300 4750
@@
 F 0 "Y202" H 2300 6750 50  0000 C CNN
 F 1 "32.768kHz" H 2300 6650 50  0000 C CNN
-F 2 "" H 2300 6450 50  0001 C CNN
+F 2 "Crystal:Crystal_SMD_Abracon_ABM3-2Pin_5.0x3.2mm" H 2300 6450 50  0001 C CNN
 F 3 "~" H 2300 6450 50  0001 C CNN
 	1    2300 6450

Commit message: RoT: Move support circuitry to LPC55 carrier board
Reduces trace lengths between LPC55 and bypass caps, DCDC inductor, and
crystals.  Instead of duplicating a bunch of these components on Gemini
Bringup, plan to always use a carrier with Gemini Bringup.

Reduced qty of signals on carrier connector to allow for additional
ground returns while keeping to a low-ish pin count (50 circuits).
Parts:
- removed C201, C205: 8pF, Capacitor_SMD:C_0603_1608Metric, symbol Device:C
- removed C202, C206: 16pF, Capacitor_SMD:C_0603_1608Metric, symbol Device:C
- removed C203: 4.7uF, Capacitor_SMD:C_0603_1608Metric, symbol Device:C
- removed C204, C219: 47pF, Capacitor_SMD:C_0603_1608Metric, symbol Device:C
- removed C207, C208, C212, C214, C215, C217: 0.1uF, Capacitor_SMD:C_0603_1608Metric, symbol Device:C
- removed C209, C210, C211, C213, C216, C218: 10nF, Capacitor_SMD:C_0603_1608Metric, symbol Device:C
- removed C220: 100nF, Capacitor_SMD:C_0603_1608Metric, symbol Device:C
- removed C221: 2.2uF, Capacitor_SMD:C_0603_1608Metric, symbol Device:C
- removed C222: 22uF, Capacitor_SMD:C_0603_1608Metric, symbol Device:C
- removed D201, D202: LED, LED_SMD:LED_0603_1608Metric_Castellated, symbol Device:LED
- removed FB201, FB202: 600R, Inductor_SMD:L_0603_1608Metric, symbol Device:Ferrite_Bead
- removed J203, J204, J205, J206: Conn_01x16, Connector_PinHeader_2.00mm:PinHeader_1x16_P2.00mm_Vertical, symbol Connector_Generic:Conn_01x16
- removed JP201, JP202, JP203, JP204: SolderJumper_3_Bridged12, Jumper:SolderJumper-3_P1.3mm_Bridged12_RoundedPad1.0x1.5mm, symbol Jumper:SolderJumper_3_Bridged12
- removed L201: 4.7uH, Resistor_SMD:R_0603_1608Metric, symbol Device:L
- removed R201, R202, R203, R204, R211, R213, R214: 100kR, Resistor_SMD:R_0603_1608Metric, symbol Device:R
- removed R205, R206, R207, R208: 100R, Resistor_SMD:R_0603_1608Metric, symbol Device:R
- removed R209, R210: 330R, Resistor_SMD:R_0603_1608Metric, symbol Device:R
- removed U201: LPC55S28JBD64, lpc55:HTQFP-64-1EP_10x10mm_P0.5mm_EP3.6x3.6mm, symbol lpc55:LPC55S28JBD64
- removed Y201: 16MHz, Crystal:Crystal_SMD_Abracon_ABM3-2Pin_5.0x3.2mm, symbol Device:Crystal
- removed Y202: 32.768kHz, Crystal:Crystal_SMD_Abracon_ABM3-2Pin_5.0x3.2mm, symbol Device:Crystal
- added J?: Conn_02x25_Odd_Even, symbol Connector_Generic:Conn_02x25_Odd_Even
- added J?: Conn_01x10, symbol Connector_Generic:Conn_01x10
Connections:
- net +3V3: now also J?.1 (Pin_1), J?.1 (Pin_1), J?.2 (Pin_2), J?.3 (Pin_3), J?.4 (Pin_4), J?.5 (Pin_5), J?.6 (Pin_6), J?.8 (Pin_8); no longer SW201.1 (A)
- net FC0_RXD: now also J?.44 (Pin_44)
- net FC0_TXD: now also J?.48 (Pin_48)
- net GND: now also J?.10 (Pin_10), J?.10 (Pin_10), J?.11 (Pin_11), J?.14 (Pin_14), J?.15 (Pin_15), J?.18 (Pin_18), J?.19 (Pin_19), J?.22 (Pin_22), J?.23 (Pin_23), J?.26 (Pin_26), J?.27 (Pin_27), J?.30 (Pin_30), J?.31 (Pin_31), J?.34 (Pin_34), J?.35 (Pin_35), J?.38 (Pin_38), J?.39 (Pin_39), J?.42 (Pin_42), J?.43 (Pin_43), J?.46 (Pin_46), J?.47 (Pin_47), J?.50 (Pin_50), J?.7 (Pin_7)
- net ISP0: now also J?.25 (Pin_25)
- net PIO0_22: now also J?.20 (Pin_20), J?.4 (Pin_4)
- net PIO0_25: now also J?.24 (Pin_24), J?.5 (Pin_5)
- net PIO0_4: now also J?.36 (Pin_36), J?.8 (Pin_8)
- net SP_MISO: now also J?.33 (Pin_33)
- net SP_MOSI: now also J?.37 (Pin_37)
- net SP_SCK: now also J?.29 (Pin_29)
- net SWD_CLK: now also J202.4 (SWDCLK/TCK), J?.13 (Pin_13)
- net SWD_IO: now also J202.2 (SWDIO/TMS), J?.17 (Pin_17)
- net ~SP_CS: now also J?.41 (Pin_41)
- net ~SP_IRQ: now also J?.45 (Pin_45)
- net ~SP_RESET: now also J?.49 (Pin_49)
- net ~SWD_RESET: now reaches J202.10 (~RESET~), SW202.1 (A)
- net ~SWD_RESET: now also J?.9 (Pin_9)
- net SWD_TRACESWO: now reaches J202.6 (SWO/TDO)
- net SWD_TRACESWO: now also J?.21 (Pin_21)
- new net FC3_CTS_SDAX_SSEL0: J?.12 (Pin_12), J?.2 (Pin_2)
- new net FC3_RTS_SCLX_SSEL1: J?.16 (Pin_16), J?.3 (Pin_3)
- new net FC3_RXD_DSA_MOSI: J?.32 (Pin_32), J?.7 (Pin_7)
- new net FC3_SCK: J?.40 (Pin_40), J?.9 (Pin_9)
- new net FC3_TXD_SCL_MISO: J?.28 (Pin_28), J?.6 (Pin_6)
- no-connect marks 3 -> 2
Other:
- note added: "RoT Aux GPIOs"
- note added: "~SP_RESET~ is open-drain"
- note removed: "1"
- note removed: "1 - 2 Xtal\n2 - 3 No Xtal"
- note removed: "17"
- note removed: "33"
- note removed: "49"
- note removed: "CHECK VALUES\nONCE LED SELECTED"
- note removed: "Crystals"
- note removed: "LPC55 Pin Breakout"
- note removed: "Place 4.7uF near ferrite bead. Others near LPC55 VDD pins."
- note removed: "Place near LPC55 VDDA and VREFP pins"
- note removed: "Power Filtering and Decoupling"
- note removed: "~SP_RESET~ must emulate open-drain by\nbeing either Hi-Z or driving LOW only."
- moved on the sheet: J201, J202, SW201, SW202
