File: rot.sch (KiCad schematic (older format))
At the start: 8 parts, among them J201 Conn_01x04, J202 Conn_ARM_JTAG_SWD_10, J203 Conn_2Rows-51Pins, J204 Conn_01x10, SW201 SW_SPDT, SW202 SW_SPST

Commit message: Change baseboard/carrier connector footprint with Hirose DF9-51x-1V
Parts:
- J203: footprint Connector_PinHeader_2.00mm:PinHeader_2x26_P2.00mm_Vertical_SMD -> hirose-df9:Hirose_DF9-51x-1V(69)_2Rows_51Pin-2MP_P1.0mm_Vertical
Changed lines of the file:
@@
 F 0 "J203" H 11650 7350 50  0000 C CNN
 F 1 "Conn_2Rows-51Pins" H 11650 7250 50  0000 C CNN
-F 2 "Connector_PinHeader_2.00mm:PinHeader_2x26_P2.00mm_Vertical_SMD" H 11600 5900 50  0001 C CNN
+F 2 "hirose-df9:Hirose_DF9-51x-1V(69)_2Rows_51Pin-2MP_P1.0mm_Vertical" H 11600 5900 50  0001 C CNN
 F 3 "~" H 11600 5900 50  0001 C CNN
 F 4 "Hirose" H 11600 5900 50  0001 C CNN "Mfg"

Commit message: MB: switch buttons to cheap, readily available parts
Parts:
- SW202: footprint Button_Switch_SMD:SW_Push_1P1T_NO_Vertical_Wuerth_434133025816 -> c-and-k-pts851:PTS815
Changed lines of the file:
@@
 F 0 "SW202" V 2850 2800 50  0000 L CNN
 F 1 "SW_SPST" V 2900 2800 50  0000 L CNN
-F 2 "Button_Switch_SMD:SW_Push_1P1T_NO_Vertical_Wuerth_434133025816" H 2900 2700 50  0001 C CNN
+F 2 "c-and-k-pts851:PTS815" H 2900 2700 50  0001 C CNN
 F 3 "~" H 2900 2700 50  0001 C CNN
 	1    2900 2700

Commit message: MB: swap remaining through-hole headers for SMD
Parts:
- J201: footprint Connector_PinHeader_2.54mm:PinHeader_1x04_P2.54mm_Vertical -> Connector_PinHeader_2.54mm:PinHeader_1x04_P2.54mm_Vertical_SMD_Pin1Left
- J204: footprint Connector_PinHeader_2.54mm:PinHeader_1x10_P2.54mm_Vertical -> Connector_PinHeader_2.54mm:PinHeader_1x10_P2.54mm_Vertical_SMD_Pin1Left
Changed lines of the file:
@@
 F 0 "J201" H 1250 4700 50  0000 C CNN
 F 1 "Conn_01x04" H 1250 4600 50  0000 C CNN
-F 2 "Connector_PinHeader_2.54mm:PinHeader_1x04_P2.54mm_Vertical" H 1350 4350 50  0001 C CNN
+F 2 "Connector_PinHeader_2.54mm:PinHeader_1x04_P2.54mm_Vertical_SMD_Pin1Left" H 1350 4350 50  0001 C CNN
 F 3 "~" H 1350 4350 50  0001 C CNN
 	1    1350 4350
@@
 F 0 "J204" H 21200 3700 50  0000 L CNN
 F 1 "Conn_01x10" H 21200 3600 50  0000 L CNN
-F 2 "Connector_PinHeader_2.54mm:PinHeader_1x10_P2.54mm_Vertical" H 21100 3700 50  0001 C CNN
+F 2 "Connector_PinHeader_2.54mm:PinHeader_1x10_P2.54mm_Vertical_SMD_Pin1Left" H 21100 3700 50  0001 C CNN
 F 3 "~" H 21100 3700 50  0001 C CNN
 	1    21100 3700

Commit message: MB: annotate everything with mfg/MPN
Parts:
- J201: Mfg (none) -> METZ CONNECT USA; Mfg Part Num (none) -> PM20204VBNN
- J202: Mfg (none) -> Samtec Inc; Mfg Part Num (none) -> FTSH-105-01-F-DV-K
- J204: footprint Connector_PinHeader_2.54mm:PinHeader_1x10_P2.54mm_Vertical_SMD_Pin1Left -> Connector_PinHeader_2.54mm:PinHeader_1x10_P2.54mm_Vertical_SMD_Pin1Right; Mfg (none) -> Amphenol ICC; Mfg Part Num (none) -> 10129380-910001ALF
- R201, R212: Mfg Part Num (none) -> generic
- SW201: Mfg (none) -> C&K; Mfg Part Num (none) -> JS102011SAQN
- SW202: Mfg (none) -> C&K; Mfg Part Num (none) -> PTS815 SJM 250 SMTR LFS
Changed lines of the file:
@@
 F 2 "c-and-k-pts851:PTS815" H 2900 2700 50  0001 C CNN
 F 3 "~" H 2900 2700 50  0001 C CNN
+F 4 "C&K" H 2900 2700 50  0001 C CNN "Mfg"
+F 5 "PTS815 SJM 250 SMTR LFS" H 2900 2700 50  0001 C CNN "Mfg Part Num"
 	1    2900 2700
 	0    1    1    0
@@
 F 2 "Connector_PinHeader_1.27mm:PinHeader_2x05_P1.27mm_Vertical_SMD" H 2300 2000 50  0001 C CNN
 F 3 "http://infocenter.arm.com/help/topic/com.arm.doc.ddi0314h/DDI0314H_coresight_components_trm.pdf" V 1950 750 50  0001 C CNN
+F 4 "Samtec Inc" H 2300 2000 50  0001 C CNN "Mfg"
+F 5 "FTSH-105-01-F-DV-K" H 2300 2000 50  0001 C CNN "Mfg Part Num"
 	1    2300 2000
 	1    0    0    -1
@@
 F 2 "Resistor_SMD:R_0603_1608Metric" V 20130 1600 50  0001 C CNN
 F 3 "~" H 20200 1600 50  0001 C CNN
+F 4 "generic" H 20200 1600 50  0001 C CNN "Mfg Part Num"
 	1    20200 1600
 	1    0    0    -1
@@
 F 2 "Button_Switch_SMD:SW_SPDT_CK-JS102011SAQN" H 3150 4500 50  0001 C CNN
 F 3 "~" H 3150 4500 50  0001 C CNN
+F 4 "C&K" H 3150 4500 50  0001 C CNN "Mfg"
+F 5 "JS102011SAQN" H 3150 4500 50  0001 C CNN "Mfg Part Num"
 	1    3150 4500
 	-1   0    0    -1
@@
 F 2 "Connector_PinHeader_2.54mm:PinHeader_1x04_P2.54mm_Vertical_SMD_Pin1Left" H 1350 4350 50  0001 C CNN
 F 3 "~" H 1350 4350 50  0001 C CNN
+F 4 "METZ CONNECT USA" H 1350 4350 50  0001 C CNN "Mfg"
+F 5 "PM20204VBNN" H 1350 4350 50  0001 C CNN "Mfg Part Num"
 	1    1350 4350
 	-1   0    0    -1
@@
 F 0 "J204" H 21200 3700 50  0000 L CNN
 F 1 "Conn_01x10" H 21200 3600 50  0000 L CNN
-F 2 "Connector_PinHeader_2.54mm:PinHeader_1x10_P2.54mm_Vertical_SMD_Pin1Left" H 21100 3700 50  0001 C CNN
+F 2 "Connector_PinHeader_2.54mm:PinHeader_1x10_P2.54mm_Vertical_SMD_Pin1Right" H 21100 3700 50  0001 C CNN
 F 3 "~" H 21100 3700 50  0001 C CNN
+F 4 "Amphenol ICC" H 21100 3700 50  0001 C CNN "Mfg"
+F 5 "10129380-910001ALF" H 21100 3700 50  0001 C CNN "Mfg Part Num"
 	1    21100 3700
 	1    0    0    -1
@@
 F 2 "Resistor_SMD:R_0603_1608Metric" V 19830 2050 50  0001 C CNN
 F 3 "~" H 19900 2050 50  0001 C CNN
+F 4 "generic" H 19900 2050 50  0001 C CNN "Mfg Part Num"
 	1    19900 2050
 	0    1    1    0

Commit message: MB: assign single resistors
Parts:
- R201: Mfg (none) -> Bourns; Mfg Part Num generic -> CR0603-JW-220ELF
- R212: value 100kR -> 100k; Mfg (none) -> Bourns; Mfg Part Num generic -> CR0603-JW-104ELF
Changed lines of the file:
@@
 P 20200 1600
 F 0 "R212" H 20300 1650 50  0000 L CNN
-F 1 "100kR" H 20300 1600 50  0000 L CNN
+F 1 "100k" H 20300 1600 50  0000 L CNN
 F 2 "Resistor_SMD:R_0603_1608Metric" V 20130 1600 50  0001 C CNN
 F 3 "~" H 20200 1600 50  0001 C CNN
-F 4 "generic" H 20200 1600 50  0001 C CNN "Mfg Part Num"
+F 4 "CR0603-JW-104ELF" H 20200 1600 50  0001 C CNN "Mfg Part Num"
+F 5 "Bourns" H 20200 1600 50  0001 C CNN "Mfg"
 	1    20200 1600
 	1    0    0    -1
@@
 F 2 "Resistor_SMD:R_0603_1608Metric" V 19830 2050 50  0001 C CNN
 F 3 "~" H 19900 2050 50  0001 C CNN
-F 4 "generic" H 19900 2050 50  0001 C CNN "Mfg Part Num"
+F 4 "CR0603-JW-220ELF" H 19900 2050 50  0001 C CNN "Mfg Part Num"
+F 5 "Bourns" H 19900 2050 50  0001 C CNN "Mfg"
 	1    19900 2050
 	0    1    1    0

Commit message: MB: update RoT carrier pinout
Parts:
- added D201: Red, LED_SMD:LED_0603_1608Metric_Castellated, symbol Device:LED
- added D202: Amber, LED_SMD:LED_0603_1608Metric_Castellated, symbol Device:LED
- added R202, R203: 68, Resistor_SMD:R_0603_1608Metric, symbol Device:R
Connections:
- net +3V3: now also J203.47 (Pin_47), J203.49 (Pin_49), J203.51 (Pin_51); no longer J203.1 (Pin_1), J203.2 (Pin_2), J203.3 (Pin_3), J203.4 (Pin_4), J203.5 (Pin_5), J203.6 (Pin_6), J203.8 (Pin_8)
- net FC0_RXD: now also J203.36 (Pin_36); no longer J203.44 (Pin_44)
- net FC0_TXD: now also J203.40 (Pin_40); no longer J203.48 (Pin_48)
- net FC3_CTS_SDAX_SSEL0: now also J203.32 (Pin_32); no longer J203.12 (Pin_12)
- net FC3_RTS_SCLX_SSEL1: now also J203.28 (Pin_28); no longer J203.16 (Pin_16)
- net FC3_RXD_DSA_MOSI: now also J203.12 (Pin_12); no longer J203.32 (Pin_32)
- net FC3_SCK: now also J203.4 (Pin_4); no longer J203.40 (Pin_40)
- net FC3_TXD_SCL_MISO: now also J203.16 (Pin_16); no longer J203.28 (Pin_28)
- net GND: now also J203.1 (Pin_1), J203.13 (Pin_13), J203.17 (Pin_17), J203.2 (Pin_2), J203.21 (Pin_21), J203.25 (Pin_25), J203.29 (Pin_29), J203.45 (Pin_45), J203.5 (Pin_5), J203.6 (Pin_6), J203.9 (Pin_9), R202.1, R203.1; no longer J203.11 (Pin_11), J203.15 (Pin_15), J203.19 (Pin_19), J203.23 (Pin_23), J203.27 (Pin_27), J203.31 (Pin_31), J203.39 (Pin_39), J203.43 (Pin_43), J203.46 (Pin_46), J203.47 (Pin_47), J203.50 (Pin_50), J203.51 (Pin_51), J203.7 (Pin_7)
- net HS_SPI_MISO: now also J203.7 (Pin_7); no longer J203.33 (Pin_33)
- net ISP0: now also J203.3 (Pin_3); no longer J203.25 (Pin_25)
- net PIO0_22: now also J203.24 (Pin_24); no longer J203.20 (Pin_20)
- net PIO0_25: now also J203.20 (Pin_20); no longer J203.24 (Pin_24)
- net PIO0_4: now also J203.8 (Pin_8); no longer J203.36 (Pin_36)
- net SP_MOSI: now also J203.15 (Pin_15); no longer J203.37 (Pin_37)
- net SP_SCK: now also J203.11 (Pin_11); no longer J203.29 (Pin_29)
- net SWD_CLK: now also J203.39 (Pin_39); no longer J203.13 (Pin_13)
- net SWD_IO: now also J203.41 (Pin_41); no longer J203.17 (Pin_17)
- net SWD_TRACESWO: now also J203.37 (Pin_37); no longer J203.21 (Pin_21)
- net ~SP_CS: now also J203.19 (Pin_19); no longer J203.41 (Pin_41)
- net ~SP_IRQ: now also J203.23 (Pin_23); no longer J203.45 (Pin_45)
- net ~SP_RESET: now also J203.27 (Pin_27); no longer J203.49 (Pin_49)
- net ~SWD_RESET: now also J203.43 (Pin_43); no longer J203.9 (Pin_9)
- new net: D201.1 (K), R202.2
- new net: D202.1 (K), R203.2
- new net SCT0_OUT2: D201.2 (A), J203.31 (Pin_31)
- new net SCT0_OUT3: D202.2 (A), J203.33 (Pin_33)

Commit message: Separate footprints for Hirose DF9-51P vs DF9-51S
When mated, pin numbers on DF9-51P will be mirrored around the shorter
axis on DF9-51S.  Separate into two footprints that reflect this such
that pin 1 on DF9-51P connects to pin 1 on DF9-51S.
Parts:
- J203: footprint hirose-df9:Hirose_DF9-51x-1V(69)_2Rows_51Pin-2MP_P1.0mm_Vertical -> hirose-df9:Hirose_DF9-51P-1V(69)_2Rows_51Pin-2MP_P1.0mm_Vertical
Changed lines of the file:
@@
 F 0 "J203" H 11650 7350 50  0000 C CNN
 F 1 "Conn_2Rows-51Pins" H 11650 7250 50  0000 C CNN
-F 2 "hirose-df9:Hirose_DF9-51x-1V(69)_2Rows_51Pin-2MP_P1.0mm_Vertical" H 11600 5900 50  0001 C CNN
+F 2 "hirose-df9:Hirose_DF9-51P-1V(69)_2Rows_51Pin-2MP_P1.0mm_Vertical" H 11600 5900 50  0001 C CNN
 F 3 "~" H 11600 5900 50  0001 C CNN
 F 4 "Hirose" H 11600 5900 50  0001 C CNN "Mfg"

Commit message: gemini-bringup: Add CPNs for all components
Parts:
- D201: CPN (none) -> 224-00005
- D202: CPN (none) -> 224-00006
- J201: CPN (none) -> 215-00021
- J202: CPN (none) -> 215-00022
- J203: CPN (none) -> 215-00023
- J204: CPN (none) -> 215-00024
- R201: CPN (none) -> 232-00019
- R202, R203: CPN (none) -> 232-00020
- R212: CPN (none) -> 232-00021
- SW201: CPN (none) -> 237-00004
- SW202: CPN (none) -> 237-00005
Changed lines of the file:
@@
 F 4 "C&K" H 2900 2700 50  0001 C CNN "Mfg"
 F 5 "PTS815 SJM 250 SMTR LFS" H 2900 2700 50  0001 C CNN "Mfg Part Num"
+F 6 "237-00005" H 2900 2700 50  0001 C CNN "CPN"
 	1    2900 2700
 	0    1    1    0
@@
 F 4 "Samtec Inc" H 2300 2000 50  0001 C CNN "Mfg"
 F 5 "FTSH-105-01-F-DV-K" H 2300 2000 50  0001 C CNN "Mfg Part Num"
+F 6 "215-00022" H 2300 2000 50  0001 C CNN "CPN"
 	1    2300 2000
 	1    0    0    -1
@@
 F 4 "CR0603-JW-104ELF" H 20200 1600 50  0001 C CNN "Mfg Part Num"
 F 5 "Bourns" H 20200 1600 50  0001 C CNN "Mfg"
+F 6 "232-00021" H 20200 1600 50  0001 C CNN "CPN"
 	1    20200 1600
 	1    0    0    -1
@@
 F 4 "C&K" H 3150 4500 50  0001 C CNN "Mfg"
 F 5 "JS102011SAQN" H 3150 4500 50  0001 C CNN "Mfg Part Num"
+F 6 "237-00004" H 3150 4500 50  0001 C CNN "CPN"
 	1    3150 4500
 	-1   0    0    -1
@@
 F 4 "METZ CONNECT USA" H 1350 4350 50  0001 C CNN "Mfg"
 F 5 "PM20204VBNN" H 1350 4350 50  0001 C CNN "Mfg Part Num"
+F 6 "215-00021" H 1350 4350 50  0001 C CNN "CPN"
 	1    1350 4350
 	-1   0    0    -1
@@
 F 4 "Amphenol ICC" H 21100 3700 50  0001 C CNN "Mfg"
 F 5 "10129380-910001ALF" H 21100 3700 50  0001 C CNN "Mfg Part Num"
+F 6 "215-00024" H 21100 3700 50  0001 C CNN "CPN"
 	1    21100 3700
 	1    0    0    -1
@@
 F 4 "CR0603-JW-220ELF" H 19900 2050 50  0001 C CNN "Mfg Part Num"
 F 5 "Bourns" H 19900 2050 50  0001 C CNN "Mfg"
+F 6 "232-00019" H 19900 2050 50  0001 C CNN "CPN"
 	1    19900 2050
 	0    1    1    0
@@
 F 4 "Hirose" H 11600 5900 50  0001 C CNN "Mfg"
 F 5 "DF9-51P-1V(69)" H 11600 5900 50  0001 C CNN "Mfg Part Num"
+F 6 "215-00023" H 11600 5900 50  0001 C CNN "CPN"
 	1    11600 5900
 	1    0    0    -1
@@
 F 4 "150060RS75000" H 2000 5750 50  0001 C CNN "Mfg Part Num"
 F 5 "Würth Elektronik" H 2000 5750 50  0001 C CNN "Mfg"
+F 6 "224-00005" H 2000 5750 50  0001 C CNN "CPN"
 	1    2000 5750
 	-1   0    0    1
@@
 F 4 "CR0603-JW-680ELF" H 2500 5750 50  0001 C CNN "Mfg Part Num"
 F 5 "Bourns" H 2500 5750 50  0001 C CNN "Mfg"
+F 6 "232-00020" H 2500 5750 50  0001 C CNN "CPN"
 	1    2500 5750
 	0    1    1    0
@@
 F 4 "150060AS75000" H 2000 5950 50  0001 C CNN "Mfg Part Num"
 F 5 "Würth Elektronik" H 2000 5950 50  0001 C CNN "Mfg"
+F 6 "224-00006" H 2000 5950 50  0001 C CNN "CPN"
 	1    2000 5950
 	-1   0    0    1
@@
 F 4 "CR0603-JW-680ELF" H 2500 5950 50  0001 C CNN "Mfg Part Num"
 F 5 "Bourns" H 2500 5950 50  0001 C CNN "Mfg"
+F 6 "232-00020" H 2500 5950 50  0001 C CNN "CPN"
 	1    2500 5950
 	0    1    1    0
