File: sp.sch (KiCad schematic (older format))
At the start: 70 parts, among them J301 Conn_ARM_JTAG_SWD_10, J302 HOST_UART, SW301 RESET, SW302 BOOT0, SW303 CLEAR, U301 STM32H753BITx, U302 MAX13235EET, Y301 25MHz, Y302 32.768kHz

Commit message: RoT: Move support circuitry to LPC55 carrier board
Reduces trace lengths between LPC55 and bypass caps, DCDC inductor, and
crystals.  Instead of duplicating a bunch of these components on Gemini
Bringup, plan to always use a carrier with Gemini Bringup.

Reduced qty of signals on carrier connector to allow for additional
ground returns while keeping to a low-ish pin count (50 circuits).
Parts:
- removed C331, C333, C334, C335, C336, C337: 0µ1, Capacitor_SMD:C_0603_1608Metric, symbol Device:C_Small
- removed C332: 1µ, Capacitor_SMD:C_0603_1608Metric, symbol Device:C_Small
- removed R316: 1M, Resistor_SMD:R_0603_1608Metric, symbol Device:R
- removed U302: MAX13235EET, Package_DFN_QFN:TQFN-20-1EP_5x5mm_P0.65mm_EP3.25x3.25mm, symbol max13235:MAX13235EET
- added R? (x4): 100kR, symbol Device:R
Connections:
- net RS232_CTS is gone; now on net USART1_CTS: J302.4 (Pin_4)
- net RS232_RTS is gone; now on net USART1_RTS: J302.6 (Pin_6)
- net RS232_RX is gone; now on net USART1_RX: J302.5 (Pin_5)
- net RS232_TX is gone; now on net USART1_TX: J302.3 (Pin_3)
- net +3V3: now also R?.1, R?.1, R?.1, R?.1
- net GND: no longer J302.9 (Pin_9)
- net ROT_MOSI: now also R?.2
- net ROT_SCK: now also R?.2
- net ~ROT_CS: now also R?.2
- net ~ROT_IRQ: now also R?.2
- net ~RS232_SHDN renamed UART7_RX
Other:
- note removed: "ON/OFF sequencing circuit\nfrom data sheet."
- moved on the sheet: J302

Commit message: Resolve merge conflict from 2020a2de7
2020a2de7 reverted the two previous commits to the SP schematic page. I have taken
a shot at reconstructing it.
Parts:
- removed R? (x4): 100kR, symbol Device:R
- added C331, C333, C334, C335, C336, C337: 0µ1, Capacitor_SMD:C_0603_1608Metric, symbol Device:C_Small
- added C332: 1µ, Capacitor_SMD:C_0603_1608Metric, symbol Device:C_Small
- added R316: 1M, Resistor_SMD:R_0603_1608Metric, symbol Device:R
- added R? (x4): 100k, symbol Device:R
- added U302: MAX13235EET, Package_DFN_QFN:TQFN-20-1EP_5x5mm_P0.65mm_EP3.25x3.25mm, symbol max13235:MAX13235EET
Connections:
- net +3V3: now also C332.1, C333.1, R?.1, R?.1, R?.1, R?.1, U302.17 (VCC), U302.9 (VL)
- net GND: now also J302.9 (Pin_9), C332.2, C333.2, C334.2, C337.2, R316.2, U302.16 (GND), U302.21 (GND)
- net ROT_MOSI: now also R?.2
- net ROT_SCK: now also R?.2
- net USART1_CTS: now also U302.8 (R2OUT); no longer J302.4 (Pin_4)
- net USART1_RTS: now also U302.10 (T2IN); no longer J302.6 (Pin_6)
- net USART1_RX: now also U302.13 (R1OUT); no longer J302.5 (Pin_5)
- net USART1_TX: now also U302.11 (T1IN); no longer J302.3 (Pin_3)
- net ~ROT_CS: now also R?.2
- net ~ROT_IRQ: now also R?.2
- net UART7_RX renamed ~RS232_SHDN
- net ~RS232_SHDN: now also C331.2, U302.18 (~FORCEOFF)
- new net: C335.1, U302.1 (C1+)
- new net: C331.1, R316.1, U302.12 (FORCEON)
- new net: C335.2, U302.2 (C1-)
- new net: C334.1, U302.20 (V+)
- new net: C336.1, U302.3 (C2+)
- new net: C336.2, U302.4 (C2-)
- new net: C337.1, U302.5 (V-)
- new net RS232_CTS: J302.4 (Pin_4), U302.7 (R2IN)
- new net RS232_RTS: J302.6 (Pin_6), U302.6 (T2OUT)
- new net RS232_RX: J302.5 (Pin_5), U302.14 (R1IN)
- new net RS232_TX: J302.3 (Pin_3), U302.15 (T1OUT)
Other:
- note added: "ON/OFF sequencing circuit\nfrom data sheet."
- moved on the sheet: J302

Commit message: Annotate new components.
Parts:
- gave numbers to parts that had none: 4
Changed lines of the file:
@@
 ON/OFF sequencing circuit\nfrom data sheet.
 $Comp
-L power:GND #PWR?
+L power:GND #PWR0334
 U 1 1 5F86CBF0
 P 21350 10100
-F 0 "#PWR?" H 21350 9850 50  0001 C CNN
+F 0 "#PWR0334" H 21350 9850 50  0001 C CNN
 F 1 "GND" V 21355 9972 50  0000 R CNN
 F 2 "" H 21350 10100 50  0001 C CNN
@@
 $EndComp
 $Comp
-L Device:R R?
+L Device:R R317
 U 1 1 5F4C1F41
 P 1950 14750
-F 0 "R?" V 1850 14800 50  0000 L CNN
+F 0 "R317" V 1850 14800 50  0000 L CNN
 F 1 "100k" V 1950 14650 50  0000 L CNN
 F 2 "" V 1880 14750 50  0001 C CNN
@@
 $EndComp
 $Comp
-L Device:R R?
+L Device:R R318
 U 1 1 5F4C217F
 P 2150 14750
-F 0 "R?" V 2050 14800 50  0000 L CNN
+F 0 "R318" V 2050 14800 50  0000 L CNN
 F 1 "100k" V 2150 14650 50  0000 L CNN
 F 2 "" V 2080 14750 50  0001 C CNN
@@
 $EndComp
 $Comp
-L Device:R R?
+L Device:R R319
 U 1 1 5F4C24C5
 P 2350 14750
-F 0 "R?" V 2250 14800 50  0000 L CNN
+F 0 "R319" V 2250 14800 50  0000 L CNN
 F 1 "100k" V 2350 14650 50  0000 L CNN
 F 2 "" V 2280 14750 50  0001 C CNN
@@
 $EndComp
 $Comp
-L Device:R R?
+L Device:R R320
 U 1 1 5F4C26DF
 P 2550 14750
-F 0 "R?" V 2450 14800 50  0000 L CNN
+F 0 "R320" V 2450 14800 50  0000 L CNN
 F 1 "100k" V 2550 14650 50  0000 L CNN
 F 2 "" V 2480 14750 50  0001 C CNN
@@
 	2350 14600 2550 14600
 $Comp
-L power:+3V3 #PWR?
+L power:+3V3 #PWR0333
 U 1 1 5F4DEE4D
 P 2250 14600
-F 0 "#PWR?" H 2250 14450 50  0001 C CNN
+F 0 "#PWR0333" H 2250 14450 50  0001 C CNN
 F 1 "+3V3" H 2265 14773 50  0000 C CNN
 F 2 "" H 2250 14600 50  0001 C CNN

Commit message: Add 1SPI host connector.
fixes #4
Connections:
- net ~SPI_ROM_PROG: now reaches U301.128 (PK2)
- net SPI5_MISO renamed SPI_ROM_MISO
- net SPI5_MOSI renamed SPI_ROM_MOSI
- net SPI5_SCK renamed SPI_ROM_SCK
- net ~SPI5_CS renamed ~SPI_ROM_CS
- no-connect marks 82 -> 77
Other:
- note added: "Host 1SPI ROM egress"
Changed lines of the file:
@@
 $Descr A2 23386 16535
 encoding utf-8
-Sheet 3 13
+Sheet 3 14
 Title "Service Processor"
 Date ""
@@
 Text Notes 3900 15200 0    50   ~ 0
 FPGA SPI egress
-Wire Notes Line
-	3850 15250 3850 14350
-Wire Notes Line
-	3850 14350 5700 14350
-Wire Notes Line
-	5700 14350 5700 15250
-Wire Notes Line
-	5700 15250 3850 15250
 Text HLabel 5100 15050 2    50   Output ~ 0
 ~FPGA_CS1
@@
 Text Label 2500 11250 2    50   ~ 0
 SDMMC1_D[0..3]
-NoConn ~ 10000 5450
-NoConn ~ 10000 5550
-NoConn ~ 10000 5650
 NoConn ~ 10000 6150
 NoConn ~ 10000 6350
@@
 NoConn ~ 10000 7150
 NoConn ~ 10000 7250
-NoConn ~ 10000 7350
-NoConn ~ 10000 7450
 NoConn ~ 10000 7550
 NoConn ~ 10000 7650
@@
 Wire Wire Line
 	2550 14900 2550 15550
+Text HLabel 5000 15550 2    50   Output ~ 0
+SPI_ROM_SCK
+Text HLabel 5000 15650 2    50   Input ~ 0
+SPI_ROM_MISO
+Text HLabel 5000 15750 2    50   Output ~ 0
+SPI_ROM_MOSI
+Text HLabel 5000 15850 2    50   Output ~ 0
+~SPI_ROM_CS
+Text HLabel 5000 15450 2    50   Output ~ 0
+~SPI_ROM_PROG
+Text Label 4450 15450 2    50   ~ 0
+~SPI_ROM_PROG
+Text Label 4450 15550 2    50   ~ 0
+SPI5_SCK
+Text Label 4450 15650 2    50   ~ 0
+SPI5_MISO
+Text Label 4450 15850 2    50   ~ 0
+~SPI5_CS
+Wire Wire Line
+	5000 15850 4450 15850
+Wire Wire Line
+	4450 15750 5000 15750
+Wire Wire Line
+	5000 15650 4450 15650
+Wire Wire Line
+	4450 15550 5000 15550
+Wire Wire Line
+	5000 15450 4450 15450
+Text Notes 3900 16000 0    50   ~ 0
+Host 1SPI ROM egress
+Text Label 4450 15750 2    50   ~ 0
+SPI5_MOSI
+Connection ~ 2550 15550
+Wire Wire Line
+	2550 15550 2750 15550
+Text Label 10000 5650 2    50   ~ 0
+~SPI_ROM_PROG
+Wire Notes Line
+	3850 15250 5700 15250
+Wire Notes Line
+	3850 16050 5700 16050
+Wire Notes Line
+	3850 14350 5700 14350
+Wire Notes Line
+	3850 14350 3850 16050
+Wire Notes Line
+	5700 14350 5700 16050
 Wire Bus Line
 	1900 11250 1900 11650
@@
 Wire Bus Line
 	1900 8500 1900 10100
-Connection ~ 2550 15550
-Wire Wire Line
-	2550 15550 2750 15550
 $EndSCHEMATC

Commit message: Shrink expansion connector pitch, update PCB
Parts:
- R317, R318, R319, R320: footprint (none) -> Resistor_SMD:R_0603_1608Metric
Changed lines of the file:
@@
 F 0 "R317" V 1850 14800 50  0000 L CNN
 F 1 "100k" V 1950 14650 50  0000 L CNN
-F 2 "" V 1880 14750 50  0001 C CNN
+F 2 "Resistor_SMD:R_0603_1608Metric" V 1880 14750 50  0001 C CNN
 F 3 "~" H 1950 14750 50  0001 C CNN
 	1    1950 14750
@@
 F 0 "R318" V 2050 14800 50  0000 L CNN
 F 1 "100k" V 2150 14650 50  0000 L CNN
-F 2 "" V 2080 14750 50  0001 C CNN
+F 2 "Resistor_SMD:R_0603_1608Metric" V 2080 14750 50  0001 C CNN
 F 3 "~" H 2150 14750 50  0001 C CNN
 	1    2150 14750
@@
 F 0 "R319" V 2250 14800 50  0000 L CNN
 F 1 "100k" V 2350 14650 50  0000 L CNN
-F 2 "" V 2280 14750 50  0001 C CNN
+F 2 "Resistor_SMD:R_0603_1608Metric" V 2280 14750 50  0001 C CNN
 F 3 "~" H 2350 14750 50  0001 C CNN
 	1    2350 14750
@@
 F 0 "R320" V 2450 14800 50  0000 L CNN
 F 1 "100k" V 2550 14650 50  0000 L CNN
-F 2 "" V 2480 14750 50  0001 C CNN
+F 2 "Resistor_SMD:R_0603_1608Metric" V 2480 14750 50  0001 C CNN
 F 3 "~" H 2550 14750 50  0001 C CNN
 	1    2550 14750

Commit message: SP: add aux gpio headers.
fixes #2
Parts:
- added J303: AUX_HDR_J, symbol Connector_Generic:Conn_01x07
- added J304: AUX_HDR_G, symbol Connector_Generic:Conn_01x07
- added RN301, RN302: 22, symbol Device:R_Pack05
Connections:
- net +3V3: now also J303.1 (Pin_1), J304.1 (Pin_1)
- net GND: now also J303.7 (Pin_7), J304.7 (Pin_7)
- net at U301.129 (PG2): now also RN302.8 (R3.2)
- net at U301.130 (PG3): now also RN302.7 (R4.2)
- net at U301.131 (PG4): now also RN302.6 (R5.2)
- net at U301.65 (PJ0): now also RN301.10 (R1.2)
- net at U301.66 (PJ1): now also RN301.9 (R2.2)
- net at U301.67 (PJ2): now also RN301.8 (R3.2)
- net at U301.68 (PJ3): now also RN301.7 (R4.2)
- net at U301.69 (PJ4): now also RN301.6 (R5.2)
- net at U301.77 (PG0): now also RN302.10 (R1.2)
- net at U301.78 (PG1): now also RN302.9 (R2.2)
- new net PG0: J304.2 (Pin_2), RN302.1 (R1.1)
- new net PG1: J304.3 (Pin_3), RN302.2 (R2.1)
- new net PG2: J304.4 (Pin_4), RN302.3 (R3.1)
- new net PG3: J304.5 (Pin_5), RN302.4 (R4.1)
- new net PG4: J304.6 (Pin_6), RN302.5 (R5.1)
- new net PJ0: J303.2 (Pin_2), RN301.1 (R1.1)
- new net PJ1: J303.3 (Pin_3), RN301.2 (R2.1)
- new net PJ2: J303.4 (Pin_4), RN301.3 (R3.1)
- new net PJ3: J303.5 (Pin_5), RN301.4 (R4.1)
- new net PJ4: J303.6 (Pin_6), RN301.5 (R5.1)
- no-connect marks 77 -> 67
Changed lines of the file:
@@
 SDMMC1_D[0..3]
 NoConn ~ 10000 6150
-NoConn ~ 10000 6350
-NoConn ~ 10000 6450
-NoConn ~ 10000 6550
-NoConn ~ 10000 6650
-NoConn ~ 10000 6750
 NoConn ~ 10000 6950
 NoConn ~ 10000 7050
@@
 NoConn ~ 10000 10450
 NoConn ~ 10000 10650
-NoConn ~ 10000 11450
-NoConn ~ 10000 11550
-NoConn ~ 10000 11650
-NoConn ~ 10000 11750
-NoConn ~ 10000 11850
 NoConn ~ 10000 11950
 NoConn ~ 10000 12050
@@
 ~RS232_SHDN
 NoConn ~ 18950 9800
-Wire Wire Line
-	11400 13250 11450 13250
-Connection ~ 11400 13250
-Wire Wire Line
-	11300 13250 11400 13250
-Connection ~ 11300 13250
-Wire Wire Line
-	11200 13250 11300 13250
-Connection ~ 11200 13250
-Wire Wire Line
-	11100 13250 11200 13250
-Connection ~ 11100 13250
-Wire Wire Line
-	11000 13250 11100 13250
-Connection ~ 11000 13250
-Wire Wire Line
-	10900 13250 11000 13250
-Wire Wire Line
-	10800 13250 10900 13250
-Connection ~ 10900 13250
-Wire Wire Line
-	12000 13250 12100 13250
-Connection ~ 12000 13250
-Wire Wire Line
-	11900 13250 12000 13250
-Connection ~ 11900 13250
-Wire Wire Line
-	11800 13250 11900 13250
-Connection ~ 11800 13250
-Wire Wire Line
-	11700 13250 11800 13250
-Connection ~ 11700 13250
-Wire Wire Line
-	11600 13250 11700 13250
-Connection ~ 11600 13250
-Wire Wire Line
-	11450 13250 11500 13250
-Wire Wire Line
-	11500 13250 11600 13250
-Connection ~ 11500 13250
-Wire Wire Line
-	11350 2650 11400 2650
-Connection ~ 11400 2650
-Wire Wire Line
-	11300 2650 11350 2650
-Connection ~ 11300 2650
-Wire Wire Line
-	11200 2650 11300 2650
-Connection ~ 11200 2650
-Wire Wire Line
-	11100 2650 11200 2650
-Connection ~ 11100 2650
-Wire Wire Line
-	11000 2650 11100 2650
-Connection ~ 11000 2650
-Wire Wire Line
-	10900 2650 11000 2650
-Connection ~ 10900 2650
-Wire Wire Line
-	10800 2650 10900 2650
-Wire Wire Line
-	10700 2650 10800 2650
-Connection ~ 10800 2650
-Wire Wire Line
-	12200 2650 12300 2650
-Connection ~ 12200 2650
-Wire Wire Line
-	12100 2650 12200 2650
-Connection ~ 12100 2650
-Wire Wire Line
-	12000 2650 12100 2650
-Connection ~ 12000 2650
-Wire Wire Line
-	11900 2650 12000 2650
-Connection ~ 11900 2650
-Wire Wire Line
-	11800 2650 11900 2650
-Connection ~ 11800 2650
-Wire Wire Line
-	11700 2650 11800 2650
-Connection ~ 11700 2650
-Wire Wire Line
-	11600 2650 11700 2650
-Connection ~ 11600 2650
-Wire Wire Line
-	11500 2650 11600 2650
-Wire Wire Line
-	11400 2650 11500 2650
-Connection ~ 11500 2650
-$Comp
-L MCU_ST_STM32H7:STM32H753BITx U301
-U 1 1 5F192C5B
-P 11500 7950
-F 0 "U301" H 11550 3800 50  0000 C CNN
-F 1 "STM32H753BITx" H 11550 3700 50  0000 C CNN
-F 2 "yamaichi-sockets:IC149-208-x61-x5x" H 10200 2850 50  0001 R CNN
-F 3 "http://www.st.com/st-web-ui/static/active/en/resource/technical/document/datasheet/DM00388325.pdf" H 11500 7950 50  0001 C CNN
-	1    11500 7950
-	1    0    0    -1
-$EndComp
 Text Label 13000 3750 0    50   ~ 0
 ~RS232_SHDN
@@
 Wire Notes Line
 	5700 14350 5700 16050
+$Comp
+L Connector_Generic:Conn_01x07 J303
+U 1 1 5F7EA7F4
+P 8450 6550
+F 0 "J303" H 8368 7067 50  0000 C CNN
+F 1 "AUX_HDR_J" H 8368 6976 50  0000 C CNN
+F 2 "" H 8450 6550 50  0001 C CNN
+F 3 "~" H 8450 6550 50  0001 C CNN
+	1    8450 6550
+	-1   0    0    -1
+$EndComp
+Wire Wire Line
+	11400 13250 11450 13250
+Connection ~ 11400 13250
+Wire Wire Line
+	11300 13250 11400 13250
+Connection ~ 11300 13250
+Wire Wire Line
+	11200 13250 11300 13250
+Connection ~ 11200 13250
+Wire Wire Line
+	11100 13250 11200 13250
+Connection ~ 11100 13250
+Wire Wire Line
+	11000 13250 11100 13250
+Connection ~ 11000 13250
+Wire Wire Line
+	10800 13250 10900 13250
+Wire Wire Line
+	10900 13250 11000 13250
+Connection ~ 10900 13250
+Wire Wire Line
+	12000 13250 12100 13250
+Connection ~ 12000 13250
+Wire Wire Line
+	11900 13250 12000 13250
+Connection ~ 11900 13250
+Wire Wire Line
+	11800 13250 11900 13250
+Connection ~ 11800 13250
+Wire Wire Line
+	11700 13250 11800 13250
+Connection ~ 11700 13250
+Wire Wire Line
+	11600 13250 11700 13250
+Connection ~ 11600 13250
+Wire Wire Line
+	11500 13250 11600 13250
+Wire Wire Line
+	11450 13250 11500 13250
+Connection ~ 11500 13250
+Wire Wire Line
+	11350 2650 11400 2650
+Connection ~ 11400 2650
+Wire Wire Line
+	11300 2650 11350 2650
+Connection ~ 11300 2650
+Wire Wire Line
+	11200 2650 11300 2650
+Connection ~ 11200 2650
+Wire Wire Line
+	11100 2650 11200 2650
+Connection ~ 11100 2650
+Wire Wire Line
+	11000 2650 11100 2650
+Connection ~ 11000 2650
+Wire Wire Line
+	10900 2650 11000 2650
+Connection ~ 10900 2650
+Wire Wire Line
+	10700 2650 10800 2650
+Wire Wire Line
+	10800 2650 10900 2650
+Connection ~ 10800 2650
+Wire Wire Line
+	12200 2650 12300 2650
+Connection ~ 12200 2650
+Wire Wire Line
+	12100 2650 12200 2650
+Connection ~ 12100 2650
+Wire Wire Line
+	12000 2650 12100 2650
+Connection ~ 12000 2650
+Wire Wire Line
+	11900 2650 12000 2650
+Connection ~ 11900 2650
+Wire Wire Line
+	11800 2650 11900 2650
+Connection ~ 11800 2650
+Wire Wire Line
+	11700 2650 11800 2650
+Connection ~ 11700 2650
+Wire Wire Line
+	11600 2650 11700 2650
+Connection ~ 11600 2650
+Wire Wire Line
+	11400 2650 11500 2650
+Wire Wire Line
+	11500 2650 11600 2650
+Connection ~ 11500 2650
+$Comp
+L MCU_ST_STM32H7:STM32H753BITx U301
+U 1 1 5F192C5B
+P 11500 7950
+F 0 "U301" H 11550 3800 50  0000 C CNN
+F 1 "STM32H753BITx" H 11550 3700 50  0000 C CNN
+F 2 "yamaichi-sockets:IC149-208-x61-x5x" H 10200 2850 50  0001 R CNN
+F 3 "http://www.st.com/st-web-ui/static/active/en/resource/technical/document/datasheet/DM00388325.pdf" H 11500 7950 50  0001 C CNN
+	1    11500 7950
+	1    0    0    -1
+$EndComp
+$Comp
+L power:GND #PWR0336
+U 1 1 5F8AF632
+P 8650 6850
+F 0 "#PWR0336" H 8650 6600 50  0001 C CNN
+F 1 "GND" H 8655 6677 50  0000 C CNN
+F 2 "" H 8650 6850 50  0001 C CNN
+F 3 "" H 8650 6850 50  0001 C CNN
+	1    8650 6850
+	1    0    0    -1
+$EndComp
+Text Label 8700 6350 0    50   ~ 0
+PJ0
+Text Label 8700 6450 0    50   ~ 0
+PJ1
+Text Label 8700 6550 0    50   ~ 0
+PJ2
+Text Label 8700 6650 0    50   ~ 0
+PJ3
+Text Label 8700 6750 0    50   ~ 0
+PJ4
+$Comp
+L Device:R_Pack05 RN301
+U 1 1 5F950D28
+P 9100 6550
+F 0 "RN301" V 8683 6550 50  0000 C CNN
+F 1 "22" V 8774 6550 50  0000 C CNN
+F 2 "" V 9475 6550 50  0001 C CNN
+F 3 "~" H 9100 6550 50  0001 C CNN
+	1    9100 6550
+	0    1    1    0
+$EndComp
+Wire Wire Line
+	9300 6350 10000 6350
+Wire Wire Line
+	9300 6450 10000 6450
+Wire Wire Line
+	9300 6550 10000 6550
+Wire Wire Line
+	9300 6650 10000 6650
+Wire Wire Line
+	9300 6750 10000 6750
+$Comp
+L power:+3V3 #PWR0335
+U 1 1 5F88DFFB
+P 8650 6050
+F 0 "#PWR0335" H 8650 5900 50  0001 C CNN
+F 1 "+3V3" H 8665 6223 50  0000 C CNN
+F 2 "" H 8650 6050 50  0001 C CNN
+F 3 "" H 8650 6050 50  0001 C CNN
+	1    8650 6050
+	1    0    0    -1
+$EndComp
+Wire Wire Line
+	8650 6050 8650 6250
+Wire Wire Line
+	8650 6350 8900 6350
+Wire Wire Line
+	8650 6450 8900 6450
+Wire Wire Line
+	8650 6550 8900 6550
+Wire Wire Line
+	8650 6650 8900 6650
+Wire Wire Line
+	8650 6750 8900 6750
+$Comp
+L Connector_Generic:Conn_01x07 J304
+U 1 1 5FBE11F6
+P 8550 11650
+F 0 "J304" H 8468 12167 50  0000 C CNN
+F 1 "AUX_HDR_G" H 8468 12076 50  0000 C CNN
+F 2 "" H 8550 11650 50  0001 C CNN
+F 3 "~" H 8550 11650 50  0001 C CNN
+	1    8550 11650
+	-1   0    0    -1
+$EndComp
+$Comp
+L Device:R_Pack05 RN302
+U 1 1 5FBE40AE
+P 9150 11650
+F 0 "RN302" V 8733 11650 50  0000 C CNN
+F 1 "22" V 8824 11650 50  0000 C CNN
+F 2 "" V 9525 11650 50  0001 C CNN
+F 3 "~" H 9150 11650 50  0001 C CNN
+	1    9150 11650
+	0    1    1    0
+$EndComp
+Wire Wire Line
+	9350 11450 10000 11450
+Wire Wire Line
+	9350 11550 10000 11550
+Wire Wire Line
+	9350 11650 10000 11650
+Wire Wire Line
+	9350 11750 10000 11750
+Wire Wire Line
+	9350 11850 10000 11850
+Wire Wire Line
+	8750 11450 8950 11450
+Wire Wire Line
+	8750 11550 8950 11550
+Wire Wire Line
+	8750 11650 8950 11650
+Wire Wire Line
+	8750 11750 8950 11750
+Wire Wire Line
+	8750 11850 8950 11850
+Text Label 8750 11450 0    50   ~ 0
+PG0
+Text Label 8750 11550 0    50   ~ 0
+PG1
+Text Label 8750 11650 0    50   ~ 0
+PG2
+Text Label 8750 11750 0    50   ~ 0
+PG3
+Text Label 8750 11850 0    50   ~ 0
+PG4
+Wire Wire Line
+	8750 11350 8750 11100
 Wire Bus Line
 	1900 11250 1900 11650
@@
 Wire Bus Line
 	1900 8500 1900 10100
+$Comp
+L power:+3V3 #PWR0337
+U 1 1 5FE1D1B6
+P 8750 11100
+F 0 "#PWR0337" H 8750 10950 50  0001 C CNN
+F 1 "+3V3" H 8765 11273 50  0000 C CNN
+F 2 "" H 8750 11100 50  0001 C CNN
+F 3 "" H 8750 11100 50  0001 C CNN
+	1    8750 11100
+	1    0    0    -1
+$EndComp
+$Comp
+L power:GND #PWR0338
+U 1 1 5FE1DD44
+P 8750 11950
+F 0 "#PWR0338" H 8750 11700 50  0001 C CNN
+F 1 "GND" H 8755 11777 50  0000 C CNN
+F 2 "" H 8750 11950 50  0001 C CNN
+F 3 "" H 8750 11950 50  0001 C CNN
+	1    8750 11950
+	1    0    0    -1
+$EndComp
 $EndSCHEMATC

Commit message: Series resistors on high-speed signals.
fixes #7
Parts:
- added R321, R322, R323, R324, R325, R326, R327, R328, R329: 22, Resistor_SMD:R_0603_1608Metric, symbol Device:R
- J303, J304: footprint (none) -> Connector_PinHeader_2.54mm:PinHeader_1x07_P2.54mm_Vertical
- RN301, RN302: footprint (none) -> Resistor_SMD:R_Array_Convex_5x0603
Connections:
- net FPGA_CLK: now also R324.1, R324.2
- net FPGA_MOSI: now also R327.2; no longer U301.157 (PI3)
- net FPGA_SCK: now also R326.2; no longer U301.155 (PI1)
- net QSPI_CLK: now also R325.1, R325.2
- net ROT_MOSI: now also R322.2; no longer U301.5 (PE6)
- net ROT_SCK: now also R321.2; no longer U301.1 (PE2)
- net SDMMC1_CLK: now also R323.1, R323.2
- net SPI_ROM_MOSI: now also R329.2; no longer U301.122 (PJ10)
- net SPI_ROM_SCK: now also R328.2; no longer U301.126 (PK0)
- new net ROT_SPI4_MOSI: R322.1, U301.5 (PE6)
- new net ROT_SPI4_SCK: R321.1, U301.1 (PE2)
- new net SPI2_MOSI: R327.1, U301.157 (PI3)
- new net SPI2_SCK: R326.1, U301.155 (PI1)
- new net SPI5_MOSI: R329.1, U301.122 (PJ10)
- new net SPI5_SCK: R328.1, U301.126 (PK0)
Other:
- moved on the sheet: R317, R318, R319, R320

Commit message: SP: diode to drain reset cap at powerdown
fixes #11
Parts:
- added D305: D_Small, Diode_SMD:D_0603_1608Metric, symbol Device:D_Small
Connections:
- net +3V3: now also D305.1 (K)
- net ~RESET: now also D305.2 (A)
Other:
- note added: "Diode promptly drains reset cap at powerdown."
Changed lines of the file:
@@
 Wire Wire Line
 	2700 11550 2750 11550
+$Comp
+L Device:D_Small D305
+U 1 1 5F95D875
+P 3000 1900
+F 0 "D305" V 2954 1970 50  0000 L CNN
+F 1 "D_Small" V 3045 1970 50  0000 L CNN
+F 2 "Diode_SMD:D_0603_1608Metric" V 3000 1900 50  0001 C CNN
+F 3 "~" V 3000 1900 50  0001 C CNN
+	1    3000 1900
+	0    1    1    0
+$EndComp
+Wire Wire Line
+	3000 2100 3000 2000
 Wire Bus Line
 	1900 11250 1900 11650
@@
 Wire Bus Line
 	1900 8500 1900 10100
+$Comp
+L power:+3V3 #PWR0339
+U 1 1 5F988B5A
+P 3000 1800
+F 0 "#PWR0339" H 3000 1650 50  0001 C CNN
+F 1 "+3V3" H 3015 1973 50  0000 C CNN
+F 2 "" H 3000 1800 50  0001 C CNN
+F 3 "" H 3000 1800 50  0001 C CNN
+	1    3000 1800
+	1    0    0    -1
+$EndComp
+Text Notes 3100 1800 0    50   ~ 0
+Diode promptly drains reset cap at powerdown.
 $EndSCHEMATC
