File: sp.sch (KiCad schematic (older format))
At the start: 90 parts, among them J301 Conn_ARM_JTAG_SWD_10, J302 HOST_UART, J303 AUX_HDR_J, J304 AUX_HDR_G, SW301 RESET, SW302 BOOT0, U301 STM32H753BITx, U302 MAX13235EET, Y301 8 MHz / H130A-8.000-8-2030, Y302 32.768kHz / FC-135 32.7680KA-A

Commit message: sp: recalculate and document crystal load capacitor constraints
Parts:
- added R339: 0R, symbol Device:R
- C319, C327: value 12p -> 11pF 3.3Vpp
- C320, C323: value 12p -> 20pF 3.3Vpp
- Y301: value 8 MHz / H130A-8.000-8-2030 -> 8 MHz 8pF
- Y302: value 32.768kHz / FC-135 32.7680KA-A -> 32.768kHz
Connections:
- net OSC_OUT: now also R339.2; no longer C319.1, Y301.1
- new net: C319.1, R339.1, Y301.1
Other:
- note added: "Cl1 = Cl2 = 2*Cl - Cpin\nCl1 = Cl2 = 11pF\n\nRext = 0\n\nGm_crit = 4*(ESR+Rext)*(2*pi*F)^2*(C0+Cl)^2\nGm_crit = 0.145180 mA/V"
- note added: "Cl1 = Cl2 = 2*Cl - Cpin\nCl1 = Cl2 = 20pF\n\nGm_crit = 4*(ESR+Rext)*(2*pi*F)^2*(C0+Cl)^2\nGm_crit = 2.163 uA/V"
- note added: "HSE Xtal:\nF = 8MHz\nC0 = 5pF\nCl = 8pF\nESR = 85R\n\nHSE STM32:\nCpin = 5pF\nGm_crit_max = 1.5 mA/V"
- note added: "LSE Xtal:\nF = 32.768kHz\nC0 = 1pF\nCl = 12.5pF\nESR = 70kR\n\nLSE STM32:\nCpin = 5pF\nGm_crit_max:\n LSEDRV[1:0] = 00: 0.5 uA/V\n LSEDRV[1:0] = 01: 0.75 uA/V\n LSEDRV[1:0] = 10: 1.7 uA/V\n LSEDRV[1:0] = 11: 2.7 uA/V\n"
- moved on the sheet: C319, C320, C323, C327, Y301, Y302

Commit message: gemini-bringup: custom fields for rating constraints on passives
Instead of packing tons of detail into a single "Value" field, limit
"Value" to the primary characteristic of the device (i.e. capacitance
for capacitors, resistance for resistors, current for fuses, impedence
at frequency for ferrite beads). For all other rating constraints, use
custom fields of the form <component-refdes-prefix>_<constraint>. For
example, R_P contains the power a resistor must dissipate.  Use
calculated values when possible rather than standard values as the
intent is to capture the constraint, not a specific device choice.
Parts:
- C301, C305, C306, C307, C308, C309, C310, C311, C312, C313, C314, C315, C317, C318, C321, C322, C325, C330, C331, C333: value 0µ1 -> 0.1uF; C_Vbias (none) -> 3.3V
- C302, C303: value 2µ2 100mR -> 2.2uF; C_ESR (none) -> 100mR; C_Vbias (none) -> 1.35V
- C304: value 4µ7 -> 4.7uF; C_Vbias (none) -> 3.3V
- C319, C327: value 11pF 3.3Vpp -> 11pF; C_Vpp (none) -> 3.3V
- C320, C323: value 20pF 3.3Vpp -> 20pF; C_Vpp (none) -> 3.3V
- C326, C332: value 1µ -> 1uF; C_Vbias (none) -> 3.3V
- C334, C337: value 0µ1 -> 0.1uF; C_Vbias (none) -> 5V
- C335, C336: value 0µ1 -> 0.1uF; C_Vpp (none) -> 5V
- D301: D_If (none) -> 20mA; D_Iv (none) -> 250mcd; D_Vf (none) -> 2V
- D302: D_If (none) -> 20mA; D_Iv (none) -> 130mcd; D_Vf (none) -> 2V
- D303: D_If (none) -> 10mA; D_Iv (none) -> 280mcd; D_Vf (none) -> 3.2V
- D304: D_If (none) -> 18mA; D_Iv (none) -> 130mcd; D_Vf (none) -> 3.2V
- D305: D_Vr (none) -> 3.3V
- R301, R302: value 68 -> 68R
- R303: value 10 -> 10R
- R304: value 5R6 -> 5.6R
- R305, R306, R307, R311, R312, R313, R314, R315, R321, R322, R323, R324, R325, R326, R327, R328, R329, R330, R331, R332, R333, R334, R335, R336, R337, R338: value 22 -> 22R
- R308, R309: value 10k -> 10kR
- R310: value 0 -> 0R
- R316: value 1M -> 1MR
- R317, R318, R319, R320: value 100k -> 100kR
- SW301, SW302: SW_Icontact (none) -> 110uA
- Y301: value 8 MHz 8pF -> 8 MHz; Y_C0 (none) -> 5pF; Y_Cl (none) -> 8pF; Y_ESR (none) -> 85R; Y_Gm_crit_max (none) -> 1.5mA/V
- Y302: Y_C0 (none) -> 1pF; Y_Cl (none) -> 12.5pF; Y_ESR (none) -> 70kR; Y_Gm_crit_max (none) -> 2.7uA/V
Other:
- moved on the sheet: C304, C305, C306, C307, C308, C309, C310, C311, C312, C313, C314, C315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

Commit message: sp: specify footprint for R339
Parts:
- R339: footprint (none) -> Resistor_SMD:R_0603_1608Metric
Changed lines of the file:
@@
 F 0 "R339" V 20950 3600 50  0000 C CNN
 F 1 "0R" V 21050 3600 50  0000 C CNN
-F 2 "" V 21130 3600 50  0001 C CNN
+F 2 "Resistor_SMD:R_0603_1608Metric" V 21130 3600 50  0001 C CNN
 F 3 "~" H 21200 3600 50  0001 C CNN
 	1    21200 3600

Commit message: gemini-bringup: resistor power rating constraints
Parts:
- R301, R302: R_P (none) -> 27mW
- R303: R_P (none) -> 1mW
- R304: R_P (none) -> 2mW
- R308: R_P (none) -> 100uW
- R309: R_P (none) -> 300uW
- R316: R_P (none) -> 3.3uW
- R317, R318, R319, R320: R_P (none) -> 33uW
Changed lines of the file:
@@
 F 5 "Bourns" H 4500 2950 50  0001 C CNN "Mfg"
 F 6 "232-00024" H 4500 2950 50  0001 C CNN "CPN"
+F 7 "100uW" H 4500 2950 50  0001 C CNN "R_P"
 	1    4500 2950
 	0    1    1    0
@@
 F 5 "Bourns" H 9650 3050 50  0001 C CNN "Mfg"
 F 6 "232-00024" H 9650 3050 50  0001 C CNN "CPN"
+F 7 "300uW" H 9650 3050 50  0001 C CNN "R_P"
 	1    9650 3050
 	0    1    1    0
@@
 F 5 "Bourns" H 3150 4000 50  0001 C CNN "Mfg"
 F 6 "232-00020" H 3150 4000 50  0001 C CNN "CPN"
+F 7 "27mW" H 3150 4000 50  0001 C CNN "R_P"
 	1    3150 4000
 	0    1    1    0
@@
 F 5 "Bourns" H 3150 4200 50  0001 C CNN "Mfg"
 F 6 "232-00020" H 3150 4200 50  0001 C CNN "CPN"
+F 7 "27mW" H 3150 4200 50  0001 C CNN "R_P"
 	1    3150 4200
 	0    1    1    0
@@
 F 5 "Bourns" H 3150 4400 50  0001 C CNN "Mfg"
 F 6 "232-00022" H 3150 4400 50  0001 C CNN "CPN"
+F 7 "1mW" V 3150 4400 50  0001 C CNN "R_P"
 	1    3150 4400
 	0    1    1    0
@@
 F 5 "KOA Speer Electronics" H 3150 4600 50  0001 C CNN "Mfg"
 F 6 "232-00023" H 3150 4600 50  0001 C CNN "CPN"
+F 7 "2mW" V 3150 4600 50  0001 C CNN "R_P"
 	1    3150 4600
 	0    1    1    0
@@
 F 5 "Bourns" H 2500 14750 50  0001 C CNN "Mfg"
 F 6 "232-00021" H 2500 14750 50  0001 C CNN "CPN"
+F 7 "33uW" H 2500 14750 50  0001 C CNN "R_P"
 	1    2500 14750
 	1    0    0    -1
@@
 F 5 "Bourns" H 2700 14750 50  0001 C CNN "Mfg"
 F 6 "232-00021" H 2700 14750 50  0001 C CNN "CPN"
+F 7 "33uW" H 2700 14750 50  0001 C CNN "R_P"
 	1    2700 14750
 	1    0    0    -1
@@
 F 5 "Bourns" H 2900 14750 50  0001 C CNN "Mfg"
 F 6 "232-00021" H 2900 14750 50  0001 C CNN "CPN"
+F 7 "33uW" H 2900 14750 50  0001 C CNN "R_P"
 	1    2900 14750
 	1    0    0    -1
@@
 F 5 "Bourns" H 3100 14750 50  0001 C CNN "Mfg"
 F 6 "232-00021" H 3100 14750 50  0001 C CNN "CPN"
+F 7 "33uW" H 3100 14750 50  0001 C CNN "R_P"
 	1    3100 14750
 	1    0    0    -1
@@
 F 5 "Bourns" H 17750 9550 50  0001 C CNN "Mfg"
 F 6 "232-00026" H 17750 9550 50  0001 C CNN "CPN"
+F 7 "3.3uW" H 17750 9550 50  0001 C CNN "R_P"
 	1    17750 9550
 	0    1    1    0

Commit message: sp: add CPN to zero-ohm jumper
Parts:
- R339: CPN (none) -> 232-00025
Changed lines of the file:
@@
 F 2 "Resistor_SMD:R_0603_1608Metric" V 21130 3600 50  0001 C CNN
 F 3 "~" H 21200 3600 50  0001 C CNN
+F 4 "232-00025" H 21200 3600 50  0001 C CNN "CPN"
 	1    21200 3600
 	0    1    1    0

Commit message: gemini-bringup: reselect all caps respecting C/V derating
Parts:
- C301, C305, C306, C307, C308, C309, C310, C311, C312, C313, C314, C315, C317, C318, C321, C322, C325, C330, C331, C333, C334, C335, C336, C337: Mfg Samsung Electro-Mechanics -> Kemet; Mfg Part Num CL10B104KB8NNWC -> C0603C104M4RACTU
- C302, C303: Mfg Yageo -> Kemet; Mfg Part Num CC0603KRX7R6BB184 -> C0603C225K4PACTU
- C304: footprint Capacitor_SMD:C_0603_1608Metric -> Capacitor_SMD:C_0805_2012Metric; Mfg Samsung Electro-Mechanics -> Kemet; Mfg Part Num CL10A475KQ8NNNC -> C0805C475K4PACTU
- C319, C327: CPN 212-00014 -> 212-00026; Mfg Walsin Technology Corporation -> Kemet; Mfg Part Num 0603N120J500CT -> C0603C110J5GACTU
- C320, C323: CPN 212-00014 -> 212-00027; Mfg Walsin Technology Corporation -> Kemet; Mfg Part Num 0603N120J500CT -> C0603C200J5GACTU
- C326, C332: footprint Capacitor_SMD:C_0603_1608Metric -> Capacitor_SMD:C_0805_2012Metric; Mfg Samsung Electro-Mechanics -> Kemet; Mfg Part Num CL10B105KP8NFNC -> C0805C105K3RACTU

Commit message: gemini-bringup: update resistor MPNs to match Bourns part numbers associated with CPN
Parts:
- R304: Mfg KOA Speer Electronics -> Bourns; Mfg Part Num RK73B1JTTD5R6J -> CR0603-J/-5R6ELF
- R339: Mfg (none) -> Bourns; Mfg Part Num (none) -> CR0603-J/-000ELF
Changed lines of the file:
@@
 F 2 "Resistor_SMD:R_0603_1608Metric" V 3080 4600 50  0001 C CNN
 F 3 "~" H 3150 4600 50  0001 C CNN
-F 4 "RK73B1JTTD5R6J" H 3150 4600 50  0001 C CNN "Mfg Part Num"
-F 5 "KOA Speer Electronics" H 3150 4600 50  0001 C CNN "Mfg"
+F 4 "CR0603-J/-5R6ELF" H 3150 4600 50  0001 C CNN "Mfg Part Num"
+F 5 "Bourns" H 3150 4600 50  0001 C CNN "Mfg"
 F 6 "232-00023" H 3150 4600 50  0001 C CNN "CPN"
 F 7 "2mW" V 3150 4600 50  0001 C CNN "R_P"
@@
 F 3 "~" H 21200 3600 50  0001 C CNN
 F 4 "232-00025" H 21200 3600 50  0001 C CNN "CPN"
+F 5 "Bourns" H 21200 3600 50  0001 C CNN "Mfg"
+F 6 "CR0603-J/-000ELF" H 21200 3600 50  0001 C CNN "Mfg Part Num"
 	1    21200 3600
 	0    1    1    0

Commit message: sp: remove labels from STM32H753 pins that are marked no-connect
Connections:
- net I2C2_B_SCL: no longer names the net of U301.90 (PB10)
- net I2C2_B_SDA: no longer names the net of U301.91 (PB11)
- net I2C2_H_SCL: no longer names the net of U301.48 (PH4)
- net I2C2_H_SDA: no longer names the net of U301.49 (PH5)
- net UART4_RX: no longer names the net of U301.152 (PH14)
- net UART4_TX: no longer names the net of U301.151 (PH13)
- net UART7_TX: no longer names the net of U301.160 (PA15)
- net UART8_RX: no longer names the net of U301.121 (PJ9)
- net UART8_TX: no longer names the net of U301.120 (PJ8)
- net USART6_RX: no longer names the net of U301.139 (PC7)
- net USART6_TX: no longer names the net of U301.138 (PC6)
- net ~I2C2_B_SMBA: no longer names the net of U301.104 (PB12)
- net ~I2C2_H_SMBA: no longer names the net of U301.96 (PH6)
Changed lines of the file:
@@
 Text Label 13000 5550 0    50   ~ 0
 I2C1_B_SDA
-Text Label 13000 5650 0    50   ~ 0
-I2C2_B_SCL
-Text Label 13000 5750 0    50   ~ 0
-I2C2_B_SDA
 Text HLabel 2250 12950 2    50   BiDi ~ 0
 I2C2_F_SCL
@@
 Text Label 3350 12950 2    50   ~ 0
 I2C4_F_SCL
-Text Label 10000 10150 2    50   ~ 0
-I2C2_H_SCL
 Text HLabel 3900 12850 2    50   BiDi ~ 0
 I2C_MUX_SDA
 Text Label 3350 12850 2    50   ~ 0
 I2C4_F_SDA
-Text Label 10000 10250 2    50   ~ 0
-I2C2_H_SDA
 Text HLabel 4000 12150 2    50   BiDi ~ 0
 I2C3_H_SCL
@@
 Text Notes 21400 10650 0    50   ~ 0
 This is a DCE-side version of the old\nPC internal serial port connector,\nwhich is still used on EthanolX. We\nimplement the DCE side so that the\ntwo machines can be connected by\na 10-pin ribbon cable.
-Text Label 10000 11150 2    50   ~ 0
-UART4_RX
-Text Label 10000 11050 2    50   ~ 0
-UART4_TX
-Text Label 13000 4450 0    50   ~ 0
-UART7_TX
-Text Label 10000 7250 2    50   ~ 0
-UART8_RX
-Text Label 10000 7150 2    50   ~ 0
-UART8_TX
 Text Label 13000 4050 0    50   ~ 0
 USART1_CTS
@@
 Text Label 18950 9000 2    50   ~ 0
 USART1_TX
-Text Label 13000 7050 0    50   ~ 0
-USART6_RX
-Text Label 13000 6950 0    50   ~ 0
-USART6_TX
 Text Notes 8850 2100 0    50   ~ 0
 Use MOMENTARY NC\nMust be closed when\npower is on!
@@
 Text Label 13000 5150 0    50   ~ 0
 ~I2C1_B_SMBA
-Text Label 13000 5850 0    50   ~ 0
-~I2C2_B_SMBA
 Text HLabel 2250 13050 2    50   BiDi ~ 0
 ~I2C2_F_SMBA
@@
 Text Label 3350 13050 2    50   ~ 0
 ~I2C4_F_SMBA
-Text Label 10000 10350 2    50   ~ 0
-~I2C2_H_SMBA
 Text HLabel 4000 12250 2    50   BiDi ~ 0
 ~I2C3_H_SMBA
