File: fpga_ext.sch (KiCad schematic (older format))
At the start: 1 part

Commit message: Annotate in preparation for review
Parts:
- gave numbers to parts that had none: 1
Changed lines of the file:
@@
 $EndDescr
 $Comp
-L Connector_Generic:Conn_02x24_Odd_Even J?
+L Connector_Generic:Conn_02x24_Odd_Even J1001
 U 1 1 5F327423
 P 6100 3350
-F 0 "J?" H 6150 4667 50  0000 C CNN
+F 0 "J1001" H 6150 4667 50  0000 C CNN
 F 1 "EXPANSION" H 6150 4576 50  0000 C CNN
 F 2 "" H 6100 3350 50  0001 C CNN
@@
 ~BL1
 $Comp
-L power:GND #PWR?
+L power:GND #PWR01008
 U 1 1 5F33063B
 P 5900 4550
-F 0 "#PWR?" H 5900 4300 50  0001 C CNN
+F 0 "#PWR01008" H 5900 4300 50  0001 C CNN
 F 1 "GND" V 5905 4422 50  0000 R CNN
 F 2 "" H 5900 4550 50  0001 C CNN
@@
 $EndComp
 $Comp
-L power:+3V3 #PWR?
+L power:+3V3 #PWR01007
 U 1 1 5F3308F6
 P 5900 4250
-F 0 "#PWR?" H 5900 4100 50  0001 C CNN
+F 0 "#PWR01007" H 5900 4100 50  0001 C CNN
 F 1 "+3V3" V 5915 4378 50  0000 L CNN
 F 2 "" H 5900 4250 50  0001 C CNN
@@
 $EndComp
 $Comp
-L power:+3V3 #PWR?
+L power:+3V3 #PWR01005
 U 1 1 5F330AA5
 P 5900 3650
-F 0 "#PWR?" H 5900 3500 50  0001 C CNN
+F 0 "#PWR01005" H 5900 3500 50  0001 C CNN
 F 1 "+3V3" V 5915 3778 50  0000 L CNN
 F 2 "" H 5900 3650 50  0001 C CNN
@@
 $EndComp
 $Comp
-L power:+3V3 #PWR?
+L power:+3V3 #PWR01003
 U 1 1 5F3310BE
 P 5900 3050
-F 0 "#PWR?" H 5900 2900 50  0001 C CNN
+F 0 "#PWR01003" H 5900 2900 50  0001 C CNN
 F 1 "+3V3" V 5915 3178 50  0000 L CNN
 F 2 "" H 5900 3050 50  0001 C CNN
@@
 $EndComp
 $Comp
-L power:GND #PWR?
+L power:GND #PWR01006
 U 1 1 5F331418
 P 5900 3950
-F 0 "#PWR?" H 5900 3700 50  0001 C CNN
+F 0 "#PWR01006" H 5900 3700 50  0001 C CNN
 F 1 "GND" V 5905 3822 50  0000 R CNN
 F 2 "" H 5900 3950 50  0001 C CNN
@@
 $EndComp
 $Comp
-L power:GND #PWR?
+L power:GND #PWR01004
 U 1 1 5F3317E3
 P 5900 3350
-F 0 "#PWR?" H 5900 3100 50  0001 C CNN
+F 0 "#PWR01004" H 5900 3100 50  0001 C CNN
 F 1 "GND" V 5905 3222 50  0000 R CNN
 F 2 "" H 5900 3350 50  0001 C CNN
@@
 $EndComp
 $Comp
-L power:+3V3 #PWR?
+L power:+3V3 #PWR01016
 U 1 1 5F331C70
 P 6400 4350
-F 0 "#PWR?" H 6400 4200 50  0001 C CNN
+F 0 "#PWR01016" H 6400 4200 50  0001 C CNN
 F 1 "+3V3" V 6415 4478 50  0000 L CNN
 F 2 "" H 6400 4350 50  0001 C CNN
@@
 $EndComp
 $Comp
-L power:+3V3 #PWR?
+L power:+3V3 #PWR01014
 U 1 1 5F3323FB
 P 6400 3750
-F 0 "#PWR?" H 6400 3600 50  0001 C CNN
+F 0 "#PWR01014" H 6400 3600 50  0001 C CNN
 F 1 "+3V3" V 6415 3878 50  0000 L CNN
 F 2 "" H 6400 3750 50  0001 C CNN
@@
 $EndComp
 $Comp
-L power:+3V3 #PWR?
+L power:+3V3 #PWR01012
 U 1 1 5F332974
 P 6400 3250
-F 0 "#PWR?" H 6400 3100 50  0001 C CNN
+F 0 "#PWR01012" H 6400 3100 50  0001 C CNN
 F 1 "+3V3" V 6415 3378 50  0000 L CNN
 F 2 "" H 6400 3250 50  0001 C CNN
@@
 $EndComp
 $Comp
-L power:GND #PWR?
+L power:GND #PWR01015
 U 1 1 5F333841
 P 6400 4050
-F 0 "#PWR?" H 6400 3800 50  0001 C CNN
+F 0 "#PWR01015" H 6400 3800 50  0001 C CNN
 F 1 "GND" V 6405 3922 50  0000 R CNN
 F 2 "" H 6400 4050 50  0001 C CNN
@@
 $EndComp
 $Comp
-L power:GND #PWR?
+L power:GND #PWR01013
 U 1 1 5F333E54
 P 6400 3450
-F 0 "#PWR?" H 6400 3200 50  0001 C CNN
+F 0 "#PWR01013" H 6400 3200 50  0001 C CNN
 F 1 "GND" V 6405 3322 50  0000 R CNN
 F 2 "" H 6400 3450 50  0001 C CNN
@@
 $EndComp
 $Comp
-L power:GND #PWR?
+L power:GND #PWR01011
 U 1 1 5F334346
 P 6400 2950
-F 0 "#PWR?" H 6400 2700 50  0001 C CNN
+F 0 "#PWR01011" H 6400 2700 50  0001 C CNN
 F 1 "GND" V 6405 2822 50  0000 R CNN
 F 2 "" H 6400 2950 50  0001 C CNN
@@
 $EndComp
 $Comp
-L power:GND #PWR?
+L power:GND #PWR01002
 U 1 1 5F335D9F
 P 5900 2750
-F 0 "#PWR?" H 5900 2500 50  0001 C CNN
+F 0 "#PWR01002" H 5900 2500 50  0001 C CNN
 F 1 "GND" V 5905 2622 50  0000 R CNN
 F 2 "" H 5900 2750 50  0001 C CNN
@@
 SPI_MISO
 $Comp
-L power:GND #PWR?
+L power:GND #PWR01009
 U 1 1 5F357D29
 P 6400 2350
-F 0 "#PWR?" H 6400 2100 50  0001 C CNN
+F 0 "#PWR01009" H 6400 2100 50  0001 C CNN
 F 1 "GND" V 6405 2222 50  0000 R CNN
 F 2 "" H 6400 2350 50  0001 C CNN
@@
 SPI_MOSI
 $Comp
-L power:+3V3 #PWR?
+L power:+3V3 #PWR01010
 U 1 1 5F3588DB
 P 6400 2650
-F 0 "#PWR?" H 6400 2500 50  0001 C CNN
+F 0 "#PWR01010" H 6400 2500 50  0001 C CNN
 F 1 "+3V3" V 6415 2778 50  0000 L CNN
 F 2 "" H 6400 2650 50  0001 C CNN
@@
 ~RESET
 $Comp
-L power:+12V #PWR?
+L power:+12V #PWR01001
 U 1 1 5F3C0A1E
 P 5900 2450
-F 0 "#PWR?" H 5900 2300 50  0001 C CNN
+F 0 "#PWR01001" H 5900 2300 50  0001 C CNN
 F 1 "+12V" V 5915 2578 50  0000 L CNN
 F 2 "" H 5900 2450 50  0001 C CNN

Commit message: More footprint associations
Parts:
- J1001: footprint (none) -> Connector_PinSocket_2.54mm:PinSocket_2x24_P2.54mm_Vertical
Changed lines of the file:
@@
 F 0 "J1001" H 6150 4667 50  0000 C CNN
 F 1 "EXPANSION" H 6150 4576 50  0000 C CNN
-F 2 "" H 6100 3350 50  0001 C CNN
+F 2 "Connector_PinSocket_2.54mm:PinSocket_2x24_P2.54mm_Vertical" H 6100 3350 50  0001 C CNN
 F 3 "~" H 6100 3350 50  0001 C CNN
 	1    6100 3350

Commit message: Shrink expansion connector pitch, update PCB
Parts:
- J1001: footprint Connector_PinSocket_2.54mm:PinSocket_2x24_P2.54mm_Vertical -> Connector_PinSocket_2.00mm:PinSocket_2x24_P2.00mm_Vertical_SMD
Changed lines of the file:
@@
 F 0 "J1001" H 6150 4667 50  0000 C CNN
 F 1 "EXPANSION" H 6150 4576 50  0000 C CNN
-F 2 "Connector_PinSocket_2.54mm:PinSocket_2x24_P2.54mm_Vertical" H 6100 3350 50  0001 C CNN
+F 2 "Connector_PinSocket_2.00mm:PinSocket_2x24_P2.00mm_Vertical_SMD" H 6100 3350 50  0001 C CNN
 F 3 "~" H 6100 3350 50  0001 C CNN
 	1    6100 3350

Commit message: Series resistors on high-speed signals.
fixes #7
Parts:
- added R1001: 22, Resistor_SMD:R_0603_1608Metric, symbol Device:R
Connections:
- net SPI_MISO: now also R1001.1; no longer J1001.12 (Pin_12)
- new net: J1001.12 (Pin_12), R1001.2
Changed lines of the file:
@@
 Text HLabel 5900 2650 0    50   Input ~ 0
 SPI_CLK
-Text HLabel 6400 2750 2    50   Output ~ 0
+Text HLabel 6900 2750 2    50   Output ~ 0
 SPI_MISO
 $Comp
@@
 Text Notes 4950 5150 0    50   ~ 0
 Notes:\n- Return paths near all fast signals (which is nearly everything).\n- 12V available in case we need 5V or something\n- A/D muxed because demuxing in FPGA is free\n- Two SPI selects to address (e.g.) both FPGA and bitstream ROM\n- I2C because why not\n- Only one CE routed (of 2 avail) because what is CE1 for anyway
+$Comp
+L Device:R R1001
+U 1 1 5F68AF0C
+P 6650 2750
+F 0 "R1001" V 6600 2900 50  0000 C CNN
+F 1 "22" V 6650 2750 50  0000 C CNN
+F 2 "Resistor_SMD:R_0603_1608Metric" V 6580 2750 50  0001 C CNN
+F 3 "~" H 6650 2750 50  0001 C CNN
+	1    6650 2750
+	0    1    1    0
+$EndComp
+Wire Wire Line
+	6500 2750 6400 2750
+Wire Wire Line
+	6800 2750 6900 2750
 Wire Bus Line
 	7850 2800 7850 4300
