File: fpga_ext.sch (KiCad schematic (older format))
At the start: 2 parts, among them J1001 EXPANSION

Commit message: MB: annotate everything with mfg/MPN
Parts:
- J1001: Mfg (none) -> Samtec; Mfg Part Num (none) -> TMM-124-01-L-D-SM
- R1001: Mfg Part Num (none) -> generic
Changed lines of the file:
@@
 F 2 "Connector_PinSocket_2.00mm:PinSocket_2x24_P2.00mm_Vertical_SMD" H 6100 3350 50  0001 C CNN
 F 3 "~" H 6100 3350 50  0001 C CNN
+F 4 "Samtec" H 6100 3350 50  0001 C CNN "Mfg"
+F 5 "TMM-124-01-L-D-SM" H 6100 3350 50  0001 C CNN "Mfg Part Num"
 	1    6100 3350
 	1    0    0    -1
@@
 F 2 "Resistor_SMD:R_0603_1608Metric" V 6580 2750 50  0001 C CNN
 F 3 "~" H 6650 2750 50  0001 C CNN
+F 4 "generic" H 6650 2750 50  0001 C CNN "Mfg Part Num"
 	1    6650 2750
 	0    1    1    0

Commit message: MB: assign single resistors
Parts:
- R1001: Mfg (none) -> Bourns; Mfg Part Num generic -> CR0603-JW-220ELF
Changed lines of the file:
@@
 F 2 "Resistor_SMD:R_0603_1608Metric" V 6580 2750 50  0001 C CNN
 F 3 "~" H 6650 2750 50  0001 C CNN
-F 4 "generic" H 6650 2750 50  0001 C CNN "Mfg Part Num"
+F 4 "CR0603-JW-220ELF" H 6650 2750 50  0001 C CNN "Mfg Part Num"
+F 5 "Bourns" H 6650 2750 50  0001 C CNN "Mfg"
 	1    6650 2750
 	0    1    1    0

Commit message: MB: add caps suggested in review
Parts:
- added C1001, C1002: 0µ1, Capacitor_SMD:C_0603_1608Metric, symbol Device:C_Small
Connections:
- net +3V3: now also C1001.1, C1002.1
- net GND: now also C1001.2, C1002.2
Changed lines of the file:
@@
 Wire Wire Line
 	6800 2750 6900 2750
+$Comp
+L Device:C_Small C?
+U 1 1 5F682351
+P 5050 3050
+AR Path="/5F1928E5/5F682351" Ref="C?"  Part="1"
+AR Path="/5F326BAF/5F682351" Ref="C1002"  Part="1"
+F 0 "C1002" H 5142 3096 50  0000 L CNN
+F 1 "0µ1" H 5142 3005 50  0000 L CNN
+F 2 "Capacitor_SMD:C_0603_1608Metric" H 5050 3050 50  0001 C CNN
+F 3 "~" H 5050 3050 50  0001 C CNN
+F 4 "CL10B104KB8NNWC" H 5050 3050 50  0001 C CNN "Mfg Part Num"
+F 5 "Samsung Electro-Mechanics" H 5050 3050 50  0001 C CNN "Mfg"
+	1    5050 3050
+	1    0    0    -1
+$EndComp
+$Comp
+L Device:C_Small C?
+U 1 1 5F68370A
+P 4600 3050
+AR Path="/5F1928E5/5F68370A" Ref="C?"  Part="1"
+AR Path="/5F326BAF/5F68370A" Ref="C1001"  Part="1"
+F 0 "C1001" H 4692 3096 50  0000 L CNN
+F 1 "0µ1" H 4692 3005 50  0000 L CNN
+F 2 "Capacitor_SMD:C_0603_1608Metric" H 4600 3050 50  0001 C CNN
+F 3 "~" H 4600 3050 50  0001 C CNN
+F 4 "CL10B104KB8NNWC" H 4600 3050 50  0001 C CNN "Mfg Part Num"
+F 5 "Samsung Electro-Mechanics" H 4600 3050 50  0001 C CNN "Mfg"
+	1    4600 3050
+	1    0    0    -1
+$EndComp
+Wire Wire Line
+	4600 2950 4850 2950
+Wire Wire Line
+	4600 3150 4850 3150
 Wire Bus Line
 	7850 2800 7850 4300
+$Comp
+L power:GND #PWR01018
+U 1 1 5F68432D
+P 4850 3150
+F 0 "#PWR01018" H 4850 2900 50  0001 C CNN
+F 1 "GND" V 4855 3022 50  0000 R CNN
+F 2 "" H 4850 3150 50  0001 C CNN
+F 3 "" H 4850 3150 50  0001 C CNN
+	1    4850 3150
+	1    0    0    -1
+$EndComp
+Connection ~ 4850 3150
+Wire Wire Line
+	4850 3150 5050 3150
+$Comp
+L power:+3V3 #PWR01017
+U 1 1 5F684B82
+P 4850 2950
+F 0 "#PWR01017" H 4850 2800 50  0001 C CNN
+F 1 "+3V3" V 4865 3078 50  0000 L CNN
+F 2 "" H 4850 2950 50  0001 C CNN
+F 3 "" H 4850 2950 50  0001 C CNN
+	1    4850 2950
+	1    0    0    -1
+$EndComp
+Connection ~ 4850 2950
+Wire Wire Line
+	4850 2950 5050 2950
 $EndSCHEMATC

Commit message: gemini-bringup: Add CPNs for all components
Parts:
- C1001, C1002: CPN (none) -> 212-00011
- J1001: CPN (none) -> 215-00033
- R1001: CPN (none) -> 232-00019
Changed lines of the file:
@@
 F 4 "Samtec" H 6100 3350 50  0001 C CNN "Mfg"
 F 5 "TMM-124-01-L-D-SM" H 6100 3350 50  0001 C CNN "Mfg Part Num"
+F 6 "215-00033" H 6100 3350 50  0001 C CNN "CPN"
 	1    6100 3350
 	1    0    0    -1
@@
 F 4 "CR0603-JW-220ELF" H 6650 2750 50  0001 C CNN "Mfg Part Num"
 F 5 "Bourns" H 6650 2750 50  0001 C CNN "Mfg"
+F 6 "232-00019" H 6650 2750 50  0001 C CNN "CPN"
 	1    6650 2750
 	0    1    1    0
@@
 F 4 "CL10B104KB8NNWC" H 5050 3050 50  0001 C CNN "Mfg Part Num"
 F 5 "Samsung Electro-Mechanics" H 5050 3050 50  0001 C CNN "Mfg"
+F 6 "212-00011" H 5050 3050 50  0001 C CNN "CPN"
 	1    5050 3050
 	1    0    0    -1
@@
 F 4 "CL10B104KB8NNWC" H 4600 3050 50  0001 C CNN "Mfg Part Num"
 F 5 "Samsung Electro-Mechanics" H 4600 3050 50  0001 C CNN "Mfg"
+F 6 "212-00011" H 4600 3050 50  0001 C CNN "CPN"
 	1    4600 3050
 	1    0    0    -1

Commit message: fpga_ext: specify rating constraints on passives
Parts:
- C1001, C1002: value 0µ1 -> 0.1uF 3.3VDCbias
- R1001: value 22 -> 22R
Other:
- moved on the sheet: C1001, C1002, R1001
Changed lines of the file:
@@
 Text HLabel 5900 2650 0    50   Input ~ 0
 SPI_CLK
-Text HLabel 6900 2750 2    50   Output ~ 0
+Text HLabel 7200 2750 2    50   Output ~ 0
 SPI_MISO
 $Comp
@@
 Text Label 5900 3450 2    50   ~ 0
 DA15
-Text Label 7700 2700 2    50   ~ 0
+Text Label 8200 2700 2    50   ~ 0
 DA0
-Text Label 7700 2800 2    50   ~ 0
+Text Label 8200 2800 2    50   ~ 0
 DA1
-Text Label 7700 2900 2    50   ~ 0
+Text Label 8200 2900 2    50   ~ 0
 DA2
-Text Label 7700 3000 2    50   ~ 0
+Text Label 8200 3000 2    50   ~ 0
 DA3
-Text Label 7700 3100 2    50   ~ 0
+Text Label 8200 3100 2    50   ~ 0
 DA4
-Text Label 7700 3200 2    50   ~ 0
+Text Label 8200 3200 2    50   ~ 0
 DA5
-Text Label 7700 3300 2    50   ~ 0
+Text Label 8200 3300 2    50   ~ 0
 DA6
-Text Label 7700 3400 2    50   ~ 0
+Text Label 8200 3400 2    50   ~ 0
 DA7
-Text Label 7700 3500 2    50   ~ 0
+Text Label 8200 3500 2    50   ~ 0
 DA8
-Text Label 7700 3600 2    50   ~ 0
+Text Label 8200 3600 2    50   ~ 0
 DA9
-Text Label 7700 3700 2    50   ~ 0
+Text Label 8200 3700 2    50   ~ 0
 DA10
-Text Label 7700 3800 2    50   ~ 0
+Text Label 8200 3800 2    50   ~ 0
 DA11
-Text Label 7700 3900 2    50   ~ 0
+Text Label 8200 3900 2    50   ~ 0
 DA12
-Text Label 7700 4000 2    50   ~ 0
+Text Label 8200 4000 2    50   ~ 0
 DA13
-Text Label 7700 4100 2    50   ~ 0
+Text Label 8200 4100 2    50   ~ 0
 DA14
-Text Label 7700 4200 2    50   ~ 0
+Text Label 8200 4200 2    50   ~ 0
 DA15
 Wire Wire Line
-	7700 2700 7750 2700
-Wire Wire Line
-	7700 2800 7750 2800
-Wire Wire Line
-	7700 2900 7750 2900
-Wire Wire Line
-	7700 3000 7750 3000
-Wire Wire Line
-	7700 3100 7750 3100
-Wire Wire Line
-	7700 3200 7750 3200
-Wire Wire Line
-	7700 3300 7750 3300
-Wire Wire Line
-	7700 3400 7750 3400
-Wire Wire Line
-	7700 3500 7750 3500
-Wire Wire Line
-	7700 3600 7750 3600
-Wire Wire Line
-	7700 3700 7750 3700
-Wire Wire Line
-	7700 3800 7750 3800
-Wire Wire Line
-	7700 3900 7750 3900
-Wire Wire Line
-	7700 4000 7750 4000
-Wire Wire Line
-	7700 4100 7750 4100
-Wire Wire Line
-	7700 4200 7750 4200
-Entry Wire Line
-	7750 2700 7850 2800
-Entry Wire Line
-	7750 2800 7850 2900
-Entry Wire Line
-	7750 2900 7850 3000
-Entry Wire Line
-	7750 3000 7850 3100
-Entry Wire Line
-	7750 3100 7850 3200
-Entry Wire Line
-	7750 3200 7850 3300
-Entry Wire Line
-	7750 3300 7850 3400
-Entry Wire Line
-	7750 3400 7850 3500
-Entry Wire Line
-	7750 3500 7850 3600
-Entry Wire Line
-	7750 3600 7850 3700
-Entry Wire Line
-	7750 3700 7850 3800
-Entry Wire Line
-	7750 3800 7850 3900
-Entry Wire Line
-	7750 3900 7850 4000
-Entry Wire Line
-	7750 4000 7850 4100
-Entry Wire Line
-	7750 4100 7850 4200
-Entry Wire Line
-	7750 4200 7850 4300
-Text Label 7900 4300 0    50   ~ 0
+	8200 2700 8250 2700
+Wire Wire Line
+	8200 2800 8250 2800
+Wire Wire Line
+	8200 2900 8250 2900
+Wire Wire Line
+	8200 3000 8250 3000
+Wire Wire Line
+	8200 3100 8250 3100
+Wire Wire Line
+	8200 3200 8250 3200
+Wire Wire Line
+	8200 3300 8250 3300
+Wire Wire Line
+	8200 3400 8250 3400
+Wire Wire Line
+	8200 3500 8250 3500
+Wire Wire Line
+	8200 3600 8250 3600
+Wire Wire Line
+	8200 3700 8250 3700
+Wire Wire Line
+	8200 3800 8250 3800
+Wire Wire Line
+	8200 3900 8250 3900
+Wire Wire Line
+	8200 4000 8250 4000
+Wire Wire Line
+	8200 4100 8250 4100
+Wire Wire Line
+	8200 4200 8250 4200
+Entry Wire Line
+	8250 2700 8350 2800
+Entry Wire Line
+	8250 2800 8350 2900
+Entry Wire Line
+	8250 2900 8350 3000
+Entry Wire Line
+	8250 3000 8350 3100
+Entry Wire Line
+	8250 3100 8350 3200
+Entry Wire Line
+	8250 3200 8350 3300
+Entry Wire Line
+	8250 3300 8350 3400
+Entry Wire Line
+	8250 3400 8350 3500
+Entry Wire Line
+	8250 3500 8350 3600
+Entry Wire Line
+	8250 3600 8350 3700
+Entry Wire Line
+	8250 3700 8350 3800
+Entry Wire Line
+	8250 3800 8350 3900
+Entry Wire Line
+	8250 3900 8350 4000
+Entry Wire Line
+	8250 4000 8350 4100
+Entry Wire Line
+	8250 4100 8350 4200
+Entry Wire Line
+	8250 4200 8350 4300
+Text Label 8400 4300 0    50   ~ 0
 DA[0..15]
 Wire Bus Line
-	7850 4300 8300 4300
-Text HLabel 8300 4300 2    50   BiDi ~ 0
+	8350 4300 8800 4300
+Text HLabel 8800 4300 2    50   BiDi ~ 0
 DA[0..15]
 Text HLabel 5900 2250 0    50   Input ~ 0
@@
 L Device:R R1001
 U 1 1 5F68AF0C
-P 6650 2750
-F 0 "R1001" V 6600 2900 50  0000 C CNN
-F 1 "22" V 6650 2750 50  0000 C CNN
-F 2 "Resistor_SMD:R_0603_1608Metric" V 6580 2750 50  0001 C CNN
-F 3 "~" H 6650 2750 50  0001 C CNN
-F 4 "CR0603-JW-220ELF" H 6650 2750 50  0001 C CNN "Mfg Part Num"
-F 5 "Bourns" H 6650 2750 50  0001 C CNN "Mfg"
-F 6 "232-00019" H 6650 2750 50  0001 C CNN "CPN"
-	1    6650 2750
+P 6950 2750
+F 0 "R1001" V 6850 2750 50  0000 C CNN
+F 1 "22R" V 7050 2750 50  0000 C CNN
+F 2 "Resistor_SMD:R_0603_1608Metric" V 6880 2750 50  0001 C CNN
+F 3 "~" H 6950 2750 50  0001 C CNN
+F 4 "CR0603-JW-220ELF" H 6950 2750 50  0001 C CNN "Mfg Part Num"
+F 5 "Bourns" H 6950 2750 50  0001 C CNN "Mfg"
+F 6 "232-00019" H 6950 2750 50  0001 C CNN "CPN"
+	1    6950 2750
 	0    1    1    0
 $EndComp
 Wire Wire Line
-	6500 2750 6400 2750
-Wire Wire Line
-	6800 2750 6900 2750
+	6800 2750 6400 2750
+Wire Wire Line
+	7100 2750 7200 2750
 $Comp
 L Device:C_Small C?
 U 1 1 5F682351
-P 5050 3050
+P 4550 3050
 AR Path="/5F1928E5/5F682351" Ref="C?"  Part="1"
 AR Path="/5F326BAF/5F682351" Ref="C1002"  Part="1"
-F 0 "C1002" H 5142 3096 50  0000 L CNN
-F 1 "0µ1" H 5142 3005 50  0000 L CNN
-F 2 "Capacitor_SMD:C_0603_1608Metric" H 5050 3050 50  0001 C CNN
-F 3 "~" H 5050 3050 50  0001 C CNN
-F 4 "CL10B104KB8NNWC" H 5050 3050 50  0001 C CNN "Mfg Part Num"
-F 5 "Samsung Electro-Mechanics" H 5050 3050 50  0001 C CNN "Mfg"
-F 6 "212-00011" H 5050 3050 50  0001 C CNN "CPN"
-	1    5050 3050
+F 0 "C1002" H 4650 3100 50  0000 L CNN
+F 1 "0.1uF 3.3VDCbias" H 4650 3000 50  0000 L CNN
+F 2 "Capacitor_SMD:C_0603_1608Metric" H 4550 3050 50  0001 C CNN
+F 3 "~" H 4550 3050 50  0001 C CNN
+F 4 "CL10B104KB8NNWC" H 4550 3050 50  0001 C CNN "Mfg Part Num"
+F 5 "Samsung Electro-Mechanics" H 4550 3050 50  0001 C CNN "Mfg"
+F 6 "212-00011" H 4550 3050 50  0001 C CNN "CPN"
+	1    4550 3050
 	1    0    0    -1
 $EndComp
@@
 L Device:C_Small C?
 U 1 1 5F68370A
-P 4600 3050
+P 4100 3050
 AR Path="/5F1928E5/5F68370A" Ref="C?"  Part="1"
 AR Path="/5F326BAF/5F68370A" Ref="C1001"  Part="1"
-F 0 "C1001" H 4692 3096 50  0000 L CNN
-F 1 "0µ1" H 4692 3005 50  0000 L CNN
-F 2 "Capacitor_SMD:C_0603_1608Metric" H 4600 3050 50  0001 C CNN
-F 3 "~" H 4600 3050 50  0001 C CNN
-F 4 "CL10B104KB8NNWC" H 4600 3050 50  0001 C CNN "Mfg Part Num"
-F 5 "Samsung Electro-Mechanics" H 4600 3050 50  0001 C CNN "Mfg"
-F 6 "212-00011" H 4600 3050 50  0001 C CNN "CPN"
-	1    4600 3050
-	1    0    0    -1
-$EndComp
-Wire Wire Line
-	4600 2950 4850 2950
-Wire Wire Line
-	4600 3150 4850 3150
-Wire Bus Line
-	7850 2800 7850 4300
+F 0 "C1001" H 4000 3100 50  0000 R CNN
+F 1 "0.1uF 3.3VDCbias" H 4000 3000 50  0000 R CNN
+F 2 "Capacitor_SMD:C_0603_1608Metric" H 4100 3050 50  0001 C CNN
+F 3 "~" H 4100 3050 50  0001 C CNN
+F 4 "CL10B104KB8NNWC" H 4100 3050 50  0001 C CNN "Mfg Part Num"
+F 5 "Samsung Electro-Mechanics" H 4100 3050 50  0001 C CNN "Mfg"
+F 6 "212-00011" H 4100 3050 50  0001 C CNN "CPN"
+	1    4100 3050
+	1    0    0    -1
+$EndComp
+Wire Wire Line
+	4100 2950 4350 2950
+Wire Wire Line
+	4100 3150 4350 3150
 $Comp
 L power:GND #PWR01018
 U 1 1 5F68432D
-P 4850 3150
-F 0 "#PWR01018" H 4850 2900 50  0001 C CNN
-F 1 "GND" V 4855 3022 50  0000 R CNN
-F 2 "" H 4850 3150 50  0001 C CNN
-F 3 "" H 4850 3150 50  0001 C CNN
-	1    4850 3150
-	1    0    0    -1
-$EndComp
-Connection ~ 4850 3150
-Wire Wire Line
-	4850 3150 5050 3150
+P 4350 3150
+F 0 "#PWR01018" H 4350 2900 50  0001 C CNN
+F 1 "GND" V 4355 3022 50  0000 R CNN
+F 2 "" H 4350 3150 50  0001 C CNN
+F 3 "" H 4350 3150 50  0001 C CNN
+	1    4350 3150
+	1    0    0    -1
+$EndComp
+Connection ~ 4350 3150
+Wire Wire Line
+	4350 3150 4550 3150
 $Comp
 L power:+3V3 #PWR01017
 U 1 1 5F684B82
-P 4850 2950
-F 0 "#PWR01017" H 4850 2800 50  0001 C CNN
-F 1 "+3V3" V 4865 3078 50  0000 L CNN
-F 2 "" H 4850 2950 50  0001 C CNN
-F 3 "" H 4850 2950 50  0001 C CNN
-	1    4850 2950
-	1    0    0    -1
-$EndComp
-Connection ~ 4850 2950
-Wire Wire Line
-	4850 2950 5050 2950
+P 4350 2950
+F 0 "#PWR01017" H 4350 2800 50  0001 C CNN
+F 1 "+3V3" V 4365 3078 50  0000 L CNN
+F 2 "" H 4350 2950 50  0001 C CNN
+F 3 "" H 4350 2950 50  0001 C CNN
+	1    4350 2950
+	1    0    0    -1
+$EndComp
+Connection ~ 4350 2950
+Wire Wire Line
+	4350 2950 4550 2950
+Wire Bus Line
+	8350 2800 8350 4300
 $EndSCHEMATC

Commit message: gemini-bringup: custom fields for rating constraints on passives
Instead of packing tons of detail into a single "Value" field, limit
"Value" to the primary characteristic of the device (i.e. capacitance
for capacitors, resistance for resistors, current for fuses, impedence
at frequency for ferrite beads). For all other rating constraints, use
custom fields of the form <component-refdes-prefix>_<constraint>. For
example, R_P contains the power a resistor must dissipate.  Use
calculated values when possible rather than standard values as the
intent is to capture the constraint, not a specific device choice.
Parts:
- C1001, C1002: value 0.1uF 3.3VDCbias -> 0.1uF; C_Vbias (none) -> 3.3V
Other:
- moved on the sheet: C1001, C1002, R1001
Changed lines of the file:
@@
 Text HLabel 5900 2650 0    50   Input ~ 0
 SPI_CLK
-Text HLabel 7200 2750 2    50   Output ~ 0
+Text HLabel 6900 2750 2    50   Output ~ 0
 SPI_MISO
 $Comp
@@
 Text Label 5900 3450 2    50   ~ 0
 DA15
-Text Label 8200 2700 2    50   ~ 0
+Text Label 7700 2700 2    50   ~ 0
 DA0
-Text Label 8200 2800 2    50   ~ 0
+Text Label 7700 2800 2    50   ~ 0
 DA1
-Text Label 8200 2900 2    50   ~ 0
+Text Label 7700 2900 2    50   ~ 0
 DA2
-Text Label 8200 3000 2    50   ~ 0
+Text Label 7700 3000 2    50   ~ 0
 DA3
-Text Label 8200 3100 2    50   ~ 0
+Text Label 7700 3100 2    50   ~ 0
 DA4
-Text Label 8200 3200 2    50   ~ 0
+Text Label 7700 3200 2    50   ~ 0
 DA5
-Text Label 8200 3300 2    50   ~ 0
+Text Label 7700 3300 2    50   ~ 0
 DA6
-Text Label 8200 3400 2    50   ~ 0
+Text Label 7700 3400 2    50   ~ 0
 DA7
-Text Label 8200 3500 2    50   ~ 0
+Text Label 7700 3500 2    50   ~ 0
 DA8
-Text Label 8200 3600 2    50   ~ 0
+Text Label 7700 3600 2    50   ~ 0
 DA9
-Text Label 8200 3700 2    50   ~ 0
+Text Label 7700 3700 2    50   ~ 0
 DA10
-Text Label 8200 3800 2    50   ~ 0
+Text Label 7700 3800 2    50   ~ 0
 DA11
-Text Label 8200 3900 2    50   ~ 0
+Text Label 7700 3900 2    50   ~ 0
 DA12
-Text Label 8200 4000 2    50   ~ 0
+Text Label 7700 4000 2    50   ~ 0
 DA13
-Text Label 8200 4100 2    50   ~ 0
+Text Label 7700 4100 2    50   ~ 0
 DA14
-Text Label 8200 4200 2    50   ~ 0
+Text Label 7700 4200 2    50   ~ 0
 DA15
 Wire Wire Line
-	8200 2700 8250 2700
-Wire Wire Line
-	8200 2800 8250 2800
-Wire Wire Line
-	8200 2900 8250 2900
-Wire Wire Line
-	8200 3000 8250 3000
-Wire Wire Line
-	8200 3100 8250 3100
-Wire Wire Line
-	8200 3200 8250 3200
-Wire Wire Line
-	8200 3300 8250 3300
-Wire Wire Line
-	8200 3400 8250 3400
-Wire Wire Line
-	8200 3500 8250 3500
-Wire Wire Line
-	8200 3600 8250 3600
-Wire Wire Line
-	8200 3700 8250 3700
-Wire Wire Line
-	8200 3800 8250 3800
-Wire Wire Line
-	8200 3900 8250 3900
-Wire Wire Line
-	8200 4000 8250 4000
-Wire Wire Line
-	8200 4100 8250 4100
-Wire Wire Line
-	8200 4200 8250 4200
-Entry Wire Line
-	8250 2700 8350 2800
-Entry Wire Line
-	8250 2800 8350 2900
-Entry Wire Line
-	8250 2900 8350 3000
-Entry Wire Line
-	8250 3000 8350 3100
-Entry Wire Line
-	8250 3100 8350 3200
-Entry Wire Line
-	8250 3200 8350 3300
-Entry Wire Line
-	8250 3300 8350 3400
-Entry Wire Line
-	8250 3400 8350 3500
-Entry Wire Line
-	8250 3500 8350 3600
-Entry Wire Line
-	8250 3600 8350 3700
-Entry Wire Line
-	8250 3700 8350 3800
-Entry Wire Line
-	8250 3800 8350 3900
-Entry Wire Line
-	8250 3900 8350 4000
-Entry Wire Line
-	8250 4000 8350 4100
-Entry Wire Line
-	8250 4100 8350 4200
-Entry Wire Line
-	8250 4200 8350 4300
-Text Label 8400 4300 0    50   ~ 0
+	7700 2700 7750 2700
+Wire Wire Line
+	7700 2800 7750 2800
+Wire Wire Line
+	7700 2900 7750 2900
+Wire Wire Line
+	7700 3000 7750 3000
+Wire Wire Line
+	7700 3100 7750 3100
+Wire Wire Line
+	7700 3200 7750 3200
+Wire Wire Line
+	7700 3300 7750 3300
+Wire Wire Line
+	7700 3400 7750 3400
+Wire Wire Line
+	7700 3500 7750 3500
+Wire Wire Line
+	7700 3600 7750 3600
+Wire Wire Line
+	7700 3700 7750 3700
+Wire Wire Line
+	7700 3800 7750 3800
+Wire Wire Line
+	7700 3900 7750 3900
+Wire Wire Line
+	7700 4000 7750 4000
+Wire Wire Line
+	7700 4100 7750 4100
+Wire Wire Line
+	7700 4200 7750 4200
+Entry Wire Line
+	7750 2700 7850 2800
+Entry Wire Line
+	7750 2800 7850 2900
+Entry Wire Line
+	7750 2900 7850 3000
+Entry Wire Line
+	7750 3000 7850 3100
+Entry Wire Line
+	7750 3100 7850 3200
+Entry Wire Line
+	7750 3200 7850 3300
+Entry Wire Line
+	7750 3300 7850 3400
+Entry Wire Line
+	7750 3400 7850 3500
+Entry Wire Line
+	7750 3500 7850 3600
+Entry Wire Line
+	7750 3600 7850 3700
+Entry Wire Line
+	7750 3700 7850 3800
+Entry Wire Line
+	7750 3800 7850 3900
+Entry Wire Line
+	7750 3900 7850 4000
+Entry Wire Line
+	7750 4000 7850 4100
+Entry Wire Line
+	7750 4100 7850 4200
+Entry Wire Line
+	7750 4200 7850 4300
+Text Label 7900 4300 0    50   ~ 0
 DA[0..15]
 Wire Bus Line
-	8350 4300 8800 4300
-Text HLabel 8800 4300 2    50   BiDi ~ 0
+	7850 4300 8300 4300
+Text HLabel 8300 4300 2    50   BiDi ~ 0
 DA[0..15]
 Text HLabel 5900 2250 0    50   Input ~ 0
@@
 L Device:R R1001
 U 1 1 5F68AF0C
-P 6950 2750
-F 0 "R1001" V 6850 2750 50  0000 C CNN
-F 1 "22R" V 7050 2750 50  0000 C CNN
-F 2 "Resistor_SMD:R_0603_1608Metric" V 6880 2750 50  0001 C CNN
-F 3 "~" H 6950 2750 50  0001 C CNN
-F 4 "CR0603-JW-220ELF" H 6950 2750 50  0001 C CNN "Mfg Part Num"
-F 5 "Bourns" H 6950 2750 50  0001 C CNN "Mfg"
-F 6 "232-00019" H 6950 2750 50  0001 C CNN "CPN"
-	1    6950 2750
+P 6650 2750
+F 0 "R1001" V 6600 2900 50  0000 C CNN
+F 1 "22R" V 6650 2750 50  0000 C CNN
+F 2 "Resistor_SMD:R_0603_1608Metric" V 6580 2750 50  0001 C CNN
+F 3 "~" H 6650 2750 50  0001 C CNN
+F 4 "CR0603-JW-220ELF" H 6650 2750 50  0001 C CNN "Mfg Part Num"
+F 5 "Bourns" H 6650 2750 50  0001 C CNN "Mfg"
+F 6 "232-00019" H 6650 2750 50  0001 C CNN "CPN"
+	1    6650 2750
 	0    1    1    0
 $EndComp
 Wire Wire Line
-	6800 2750 6400 2750
-Wire Wire Line
-	7100 2750 7200 2750
+	6500 2750 6400 2750
+Wire Wire Line
+	6800 2750 6900 2750
 $Comp
 L Device:C_Small C?
 U 1 1 5F682351
-P 4550 3050
+P 5050 3050
 AR Path="/5F1928E5/5F682351" Ref="C?"  Part="1"
 AR Path="/5F326BAF/5F682351" Ref="C1002"  Part="1"
-F 0 "C1002" H 4650 3100 50  0000 L CNN
-F 1 "0.1uF 3.3VDCbias" H 4650 3000 50  0000 L CNN
-F 2 "Capacitor_SMD:C_0603_1608Metric" H 4550 3050 50  0001 C CNN
-F 3 "~" H 4550 3050 50  0001 C CNN
-F 4 "CL10B104KB8NNWC" H 4550 3050 50  0001 C CNN "Mfg Part Num"
-F 5 "Samsung Electro-Mechanics" H 4550 3050 50  0001 C CNN "Mfg"
-F 6 "212-00011" H 4550 3050 50  0001 C CNN "CPN"
-	1    4550 3050
+F 0 "C1002" H 5142 3096 50  0000 L CNN
+F 1 "0.1uF" H 5142 3005 50  0000 L CNN
+F 2 "Capacitor_SMD:C_0603_1608Metric" H 5050 3050 50  0001 C CNN
+F 3 "~" H 5050 3050 50  0001 C CNN
+F 4 "CL10B104KB8NNWC" H 5050 3050 50  0001 C CNN "Mfg Part Num"
+F 5 "Samsung Electro-Mechanics" H 5050 3050 50  0001 C CNN "Mfg"
+F 6 "212-00011" H 5050 3050 50  0001 C CNN "CPN"
+F 7 "3.3V" H 5050 3050 50  0001 C CNN "C_Vbias"
+	1    5050 3050
 	1    0    0    -1
 $EndComp
@@
 L Device:C_Small C?
 U 1 1 5F68370A
-P 4100 3050
+P 4600 3050
 AR Path="/5F1928E5/5F68370A" Ref="C?"  Part="1"
 AR Path="/5F326BAF/5F68370A" Ref="C1001"  Part="1"
-F 0 "C1001" H 4000 3100 50  0000 R CNN
-F 1 "0.1uF 3.3VDCbias" H 4000 3000 50  0000 R CNN
-F 2 "Capacitor_SMD:C_0603_1608Metric" H 4100 3050 50  0001 C CNN
-F 3 "~" H 4100 3050 50  0001 C CNN
-F 4 "CL10B104KB8NNWC" H 4100 3050 50  0001 C CNN "Mfg Part Num"
-F 5 "Samsung Electro-Mechanics" H 4100 3050 50  0001 C CNN "Mfg"
-F 6 "212-00011" H 4100 3050 50  0001 C CNN "CPN"
-	1    4100 3050
-	1    0    0    -1
-$EndComp
-Wire Wire Line
-	4100 2950 4350 2950
-Wire Wire Line
-	4100 3150 4350 3150
+F 0 "C1001" H 4692 3096 50  0000 L CNN
+F 1 "0.1uF" H 4692 3005 50  0000 L CNN
+F 2 "Capacitor_SMD:C_0603_1608Metric" H 4600 3050 50  0001 C CNN
+F 3 "~" H 4600 3050 50  0001 C CNN
+F 4 "CL10B104KB8NNWC" H 4600 3050 50  0001 C CNN "Mfg Part Num"
+F 5 "Samsung Electro-Mechanics" H 4600 3050 50  0001 C CNN "Mfg"
+F 6 "212-00011" H 4600 3050 50  0001 C CNN "CPN"
+F 7 "3.3V" H 4600 3050 50  0001 C CNN "C_Vbias"
+	1    4600 3050
+	1    0    0    -1
+$EndComp
+Wire Wire Line
+	4600 2950 4850 2950
+Wire Wire Line
+	4600 3150 4850 3150
 $Comp
 L power:GND #PWR01018
 U 1 1 5F68432D
-P 4350 3150
-F 0 "#PWR01018" H 4350 2900 50  0001 C CNN
-F 1 "GND" V 4355 3022 50  0000 R CNN
-F 2 "" H 4350 3150 50  0001 C CNN
-F 3 "" H 4350 3150 50  0001 C CNN
-	1    4350 3150
-	1    0    0    -1
-$EndComp
-Connection ~ 4350 3150
-Wire Wire Line
-	4350 3150 4550 3150
+P 4850 3150
+F 0 "#PWR01018" H 4850 2900 50  0001 C CNN
+F 1 "GND" V 4855 3022 50  0000 R CNN
+F 2 "" H 4850 3150 50  0001 C CNN
+F 3 "" H 4850 3150 50  0001 C CNN
+	1    4850 3150
+	1    0    0    -1
+$EndComp
+Connection ~ 4850 3150
+Wire Wire Line
+	4850 3150 5050 3150
 $Comp
 L power:+3V3 #PWR01017
 U 1 1 5F684B82
-P 4350 2950
-F 0 "#PWR01017" H 4350 2800 50  0001 C CNN
-F 1 "+3V3" V 4365 3078 50  0000 L CNN
-F 2 "" H 4350 2950 50  0001 C CNN
-F 3 "" H 4350 2950 50  0001 C CNN
-	1    4350 2950
-	1    0    0    -1
-$EndComp
-Connection ~ 4350 2950
-Wire Wire Line
-	4350 2950 4550 2950
+P 4850 2950
+F 0 "#PWR01017" H 4850 2800 50  0001 C CNN
+F 1 "+3V3" V 4865 3078 50  0000 L CNN
+F 2 "" H 4850 2950 50  0001 C CNN
+F 3 "" H 4850 2950 50  0001 C CNN
+	1    4850 2950
+	1    0    0    -1
+$EndComp
+Connection ~ 4850 2950
+Wire Wire Line
+	4850 2950 5050 2950
 Wire Bus Line
-	8350 2800 8350 4300
+	7850 2800 7850 4300
 $EndSCHEMATC
