File: fpga_ext.sch (KiCad schematic (older format))
At the start: 4 parts, among them J1001 EXPANSION

Commit message: gemini-bringup: reselect all caps respecting C/V derating
Parts:
- C1001, C1002: Mfg Samsung Electro-Mechanics -> Kemet; Mfg Part Num CL10B104KB8NNWC -> C0603C104M4RACTU
Changed lines of the file:
@@
 F 2 "Capacitor_SMD:C_0603_1608Metric" H 5050 3050 50  0001 C CNN
 F 3 "~" H 5050 3050 50  0001 C CNN
-F 4 "CL10B104KB8NNWC" H 5050 3050 50  0001 C CNN "Mfg Part Num"
-F 5 "Samsung Electro-Mechanics" H 5050 3050 50  0001 C CNN "Mfg"
+F 4 "C0603C104M4RACTU" H 5050 3050 50  0001 C CNN "Mfg Part Num"
+F 5 "Kemet" H 5050 3050 50  0001 C CNN "Mfg"
 F 6 "212-00011" H 5050 3050 50  0001 C CNN "CPN"
 F 7 "3.3V" H 5050 3050 50  0001 C CNN "C_Vbias"
@@
 F 2 "Capacitor_SMD:C_0603_1608Metric" H 4600 3050 50  0001 C CNN
 F 3 "~" H 4600 3050 50  0001 C CNN
-F 4 "CL10B104KB8NNWC" H 4600 3050 50  0001 C CNN "Mfg Part Num"
-F 5 "Samsung Electro-Mechanics" H 4600 3050 50  0001 C CNN "Mfg"
+F 4 "C0603C104M4RACTU" H 4600 3050 50  0001 C CNN "Mfg Part Num"
+F 5 "Kemet" H 4600 3050 50  0001 C CNN "Mfg"
 F 6 "212-00011" H 4600 3050 50  0001 C CNN "CPN"
 F 7 "3.3V" H 4600 3050 50  0001 C CNN "C_Vbias"
