File: fpga_ext.sch (KiCad schematic (older format))
At the start: 4 parts, among them J1001 EXPANSION

Commit message: Change column "Mfg Part Num" to "MPN" to align with manufacturer guidelines
Parts:
- C1001, C1002: MPN (none) -> C0603C104M4RACTU; Mfg Part Num C0603C104M4RACTU -> (none)
- J1001: MPN (none) -> TMM-124-01-L-D-SM; Mfg Part Num TMM-124-01-L-D-SM -> (none)
- R1001: MPN (none) -> CR0603-JW-220ELF; Mfg Part Num CR0603-JW-220ELF -> (none)
Changed lines of the file:
@@
 F 3 "~" H 6100 3350 50  0001 C CNN
 F 4 "Samtec" H 6100 3350 50  0001 C CNN "Mfg"
-F 5 "TMM-124-01-L-D-SM" H 6100 3350 50  0001 C CNN "Mfg Part Num"
+F 5 "TMM-124-01-L-D-SM" H 6100 3350 50  0001 C CNN "MPN"
 F 6 "215-00033" H 6100 3350 50  0001 C CNN "CPN"
 	1    6100 3350
@@
 F 2 "Resistor_SMD:R_0603_1608Metric" V 6580 2750 50  0001 C CNN
 F 3 "~" H 6650 2750 50  0001 C CNN
-F 4 "CR0603-JW-220ELF" H 6650 2750 50  0001 C CNN "Mfg Part Num"
+F 4 "CR0603-JW-220ELF" H 6650 2750 50  0001 C CNN "MPN"
 F 5 "Bourns" H 6650 2750 50  0001 C CNN "Mfg"
 F 6 "232-00019" H 6650 2750 50  0001 C CNN "CPN"
@@
 F 2 "Capacitor_SMD:C_0603_1608Metric" H 5050 3050 50  0001 C CNN
 F 3 "~" H 5050 3050 50  0001 C CNN
-F 4 "C0603C104M4RACTU" H 5050 3050 50  0001 C CNN "Mfg Part Num"
+F 4 "C0603C104M4RACTU" H 5050 3050 50  0001 C CNN "MPN"
 F 5 "Kemet" H 5050 3050 50  0001 C CNN "Mfg"
 F 6 "212-00011" H 5050 3050 50  0001 C CNN "CPN"
@@
 F 2 "Capacitor_SMD:C_0603_1608Metric" H 4600 3050 50  0001 C CNN
 F 3 "~" H 4600 3050 50  0001 C CNN
-F 4 "C0603C104M4RACTU" H 4600 3050 50  0001 C CNN "Mfg Part Num"
+F 4 "C0603C104M4RACTU" H 4600 3050 50  0001 C CNN "MPN"
 F 5 "Kemet" H 4600 3050 50  0001 C CNN "Mfg"
 F 6 "212-00011" H 4600 3050 50  0001 C CNN "CPN"
