File: gemini-bringup.kicad_pcb (KiCad board)
At the start: 4 copper layers, 260 x 160 mm, 221 parts, among them J1001 EXPANSION, J1101 SMBUS, J1201 SMBUS, J1301 SMBUS, J1401 IDC_BOX_HDR, J201 Conn_01x04, J202 Conn_ARM_JTAG_SWD_10, J203 Conn_02x25_Odd_Even, J204 Conn_01x10, J301 Conn_ARM_JTAG_SWD_10, J302 HOST_UART, J303 AUX_HDR_J, J304 AUX_HDR_G, J401 RJ45_Amphenol_RJMG1BD3B8K1ANR, J402 RJ45_Amphenol_RJMG1BD3B8K1ANR, J501 SMBUS, J502 SMBUS, J503 SMBUS, J504 SMBUS, J601 Barrel_Jack, J701 Conn_01x04_Male, J702 Conn_01x04_Male, J703 Conn_01x04_Male, J704 Conn_01x04_Male, J705 Conn_01x04_Male, J706 Conn_01x04_Male, J801 IDC, J901 Micro_SD_Card, SW201 SW_SPDT, SW202 SW_SPST, SW301 RESET, SW302 BOOT0, SW303 CLEAR, U1101 TCA9802, U1201 TCA9802, U1301 TCA9802, U1401 TXB0106PWR, U301 STM32H753BITx, U302 MAX13235EET, U401 KSZ8863RLL, U501 LTC4306CGN, U601 OKI-78SR-3.3_1.5-W36-C, U602 INA219AxDCN, U603 INA219AxDCN, U701 MAX31790, U801 TXB0106PWR, U802 W25Q256FVFxx, U901 EMIF06-MSD02N16, Y301 25MHz, Y302 32.768kHz, Y401 25MHz ±50ppm

Commit message: SP: add pullup on switch SPISN per manual.
fixes #16
Parts:
- added R423: 10k, Resistor_SMD:R_0603_1608Metric, F.Cu at (62.4, 43.0)

Commit message: SP: dedicated I2C bus to FPGA EXP socket
fixes #20
Parts:
- added R104: 3k, Resistor_SMD:R_0603_1608Metric, F.Cu at (156.1, 101.1)
- added R105: 3k, Resistor_SMD:R_0603_1608Metric, F.Cu at (160.1, 101.1)
Connections:
- J1001 pad 2: /SP_I2C1_B_SCL -> /FPGA_SCL
- J1001 pad 3: /SP_I2C1_B_SDA -> /FPGA_SDA
- U301 pad 97: /sp/I2C3_H_SCL -> /FPGA_SCL
- U301 pad 98: /sp/I2C3_H_SDA -> /FPGA_SDA

Commit message: SP: GPIO control of Eth Switch reset
fixes #22
Connections:
- C401 pad 1: /sp/~RESET -> /sp/~ETH_RESET
- R406 pad 2: /sp/~RESET -> /sp/~ETH_RESET
- U301 pad 37: Net-(U301-Pad37) -> /sp/~ETH_RESET
- U401 pad 47: /sp/~RESET -> /sp/~ETH_RESET

Commit message: Add uncommitted 16-line GPIO expander.
fixes #26
Parts:
- added J1501: I2CGPIO1, Connector_PinHeader_2.54mm:PinHeader_1x10_P2.54mm_Vertical, F.Cu at (214.0, 169.7)
- added J1502: I2CGPIO0, Connector_PinHeader_2.54mm:PinHeader_1x10_P2.54mm_Vertical, F.Cu at (194.0, 147.1)
- added U1501: PCA9555PW, Package_SO:TSSOP-24_4.4x7.8mm_P0.65mm, F.Cu at (203.4, 156.2)

Commit message: Eth Switch: remove REFCLKO pullup
fixes #24
Parts:
- removed R409: 10k, Resistor_SMD:R_0603_1608Metric
Changed lines of the file:
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@@
     (tracks 0)
     (zones 0)
-    (modules 227)
+    (modules 226)
     (nets 410)
   )
@@
     (model ${KISYS3DMOD}/Resistor_SMD.3dshapes/R_0603_1608Metric.wrl
       (at (xyz 0 0 0))
-      (scale (xyz 1 1 1))
-      (rotate (xyz 0 0 0))
-    )
-  )
-  (module Resistor_SMD:R_0603_1608Metric (layer F.Cu)
-    (at 27.81 74.91 270)
-    (descr "Resistor SMD 0603 (1608 Metric), square (rectangular) end terminal, IPC_7351 nominal, (Body size source: http://www.tortai-tech.com/upload/download/2011102023233369053.pdf), generated with kicad-footprint-generator")
-    (tags resistor)
-    (attr smd)
-    (fp_text reference R409 (at 0 -1.43 90) (layer F.SilkS)
-      (effects (font (size 1 1) (thickness 0.15)))
-    )
-    (fp_text value 10k (at 0 1.43 90) (layer F.Fab)
-      (effects (font (size 1 1) (thickness 0.15)))
-    )
-    (fp_line (start -0.8 0.4) (end -0.8 -0.4) (layer F.Fab) (width 0.1))
-    (fp_line (start -0.8 -0.4) (end 0.8 -0.4) (layer F.Fab) (width 0.1))
-    (fp_line (start 0.8 -0.4) (end 0.8 0.4) (layer F.Fab) (width 0.1))
-    (fp_line (start 0.8 0.4) (end -0.8 0.4) (layer F.Fab) (width 0.1))
-    (fp_line (start -0.162779 -0.51) (end 0.162779 -0.51) (layer F.SilkS) (width 0.12))
-    (fp_line (start -0.162779 0.51) (end 0.162779 0.51) (layer F.SilkS) (width 0.12))
-    (fp_line (start -1.48 0.73) (end -1.48 -0.73) (layer F.CrtYd) (width 0.05))
-    (fp_line (start -1.48 -0.73) (end 1.48 -0.73) (layer F.CrtYd) (width 0.05))
-    (fp_line (start 1.48 -0.73) (end 1.48 0.73) (layer F.CrtYd) (width 0.05))
-    (fp_line (start 1.48 0.73) (end -1.48 0.73) (layer F.CrtYd) (width 0.05))
-    (fp_text user %R (at 0 0 90) (layer F.Fab)
-      (effects (font (size 0.4 0.4) (thickness 0.06)))
-    )
-    (pad 2 smd roundrect (at 0.7875 0 270) (size 0.875 0.95) (layers F.Cu F.Paste F.Mask) (roundrect_rratio 0.25)
-      (net 181 "Net-(R402-Pad1)"))
-    (pad 1 smd roundrect (at -0.7875 0 270) (size 0.875 0.95) (layers F.Cu F.Paste F.Mask) (roundrect_rratio 0.25)
-      (net 6 +3V3))
-    (model ${KISYS3DMOD}/Resistor_SMD.3dshapes/R_0603_1608Metric.wrl
-      (at (xyz 0 0 0))

Commit message: Eth Switch: reset diode and pullup.
fixes #23
Parts:
- added D401: 1N4148, Diode_SMD:D_0603_1608Metric, F.Cu at (35.4, 30.3)
- added R409: 10k, Resistor_SMD:R_0603_1608Metric, F.Cu at (39.4, 30.3)
Changed lines of the file:
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@@
     (tracks 0)
     (zones 0)
-    (modules 226)
+    (modules 228)
     (nets 410)
   )
@@
     (add_net VDDA)
   )
+  (module Resistor_SMD:R_0603_1608Metric (layer F.Cu)
+    (at 39.41 30.26)
+    (descr "Resistor SMD 0603 (1608 Metric), square (rectangular) end terminal, IPC_7351 nominal, (Body size source: http://www.tortai-tech.com/upload/download/2011102023233369053.pdf), generated with kicad-footprint-generator")
+    (tags resistor)
+    (attr smd)
+    (fp_text reference R409 (at 0 -1.43) (layer F.SilkS)
+      (effects (font (size 1 1) (thickness 0.15)))
+    )
+    (fp_text value 10k (at 0 1.43) (layer F.Fab)
+      (effects (font (size 1 1) (thickness 0.15)))
+    )
+    (fp_text user %R (at 0 0) (layer F.Fab)
+      (effects (font (size 0.4 0.4) (thickness 0.06)))
+    )
+    (fp_line (start -0.8 0.4) (end -0.8 -0.4) (layer F.Fab) (width 0.1))
+    (fp_line (start -0.8 -0.4) (end 0.8 -0.4) (layer F.Fab) (width 0.1))
+    (fp_line (start 0.8 -0.4) (end 0.8 0.4) (layer F.Fab) (width 0.1))
+    (fp_line (start 0.8 0.4) (end -0.8 0.4) (layer F.Fab) (width 0.1))
+    (fp_line (start -0.162779 -0.51) (end 0.162779 -0.51) (layer F.SilkS) (width 0.12))
+    (fp_line (start -0.162779 0.51) (end 0.162779 0.51) (layer F.SilkS) (width 0.12))
+    (fp_line (start -1.48 0.73) (end -1.48 -0.73) (layer F.CrtYd) (width 0.05))
+    (fp_line (start -1.48 -0.73) (end 1.48 -0.73) (layer F.CrtYd) (width 0.05))
+    (fp_line (start 1.48 -0.73) (end 1.48 0.73) (layer F.CrtYd) (width 0.05))
+    (fp_line (start 1.48 0.73) (end -1.48 0.73) (layer F.CrtYd) (width 0.05))
+    (pad 2 smd roundrect (at 0.7875 0) (size 0.875 0.95) (layers F.Cu F.Paste F.Mask) (roundrect_rratio 0.25)
+      (net 6 +3V3))
+    (pad 1 smd roundrect (at -0.7875 0) (size 0.875 0.95) (layers F.Cu F.Paste F.Mask) (roundrect_rratio 0.25)
+      (net 392 /sp/~ETH_RESET))
+    (model ${KISYS3DMOD}/Resistor_SMD.3dshapes/R_0603_1608Metric.wrl
+      (at (xyz 0 0 0))
+      (scale (xyz 1 1 1))
+      (rotate (xyz 0 0 0))
+    )
+  )
+  (module Diode_SMD:D_0603_1608Metric (layer F.Cu)
+    (at 35.4 30.3)
+    (descr "Diode SMD 0603 (1608 Metric), square (rectangular) end terminal, IPC_7351 nominal, (Body size source: http://www.tortai-tech.com/upload/download/2011102023233369053.pdf), generated with kicad-footprint-generator")
+    (tags diode)
+    (attr smd)
+    (fp_text reference D401 (at 0 -1.43) (layer F.SilkS)
+      (effects (font (size 1 1) (thickness 0.15)))
+    )
+    (fp_text value 1N4148 (at 0 1.43) (layer F.Fab)
+      (effects (font (size 1 1) (thickness 0.15)))
+    )
+    (fp_text user %R (at 0 0) (layer F.Fab)
+      (effects (font (size 0.4 0.4) (thickness 0.06)))
+    )
+    (fp_line (start 0.8 -0.4) (end -0.5 -0.4) (layer F.Fab) (width 0.1))
+    (fp_line (start -0.5 -0.4) (end -0.8 -0.1) (layer F.Fab) (width 0.1))
+    (fp_line (start -0.8 -0.1) (end -0.8 0.4) (layer F.Fab) (width 0.1))
+    (fp_line (start -0.8 0.4) (end 0.8 0.4) (layer F.Fab) (width 0.1))
+    (fp_line (start 0.8 0.4) (end 0.8 -0.4) (layer F.Fab) (width 0.1))
+    (fp_line (start 0.8 -0.735) (end -1.485 -0.735) (layer F.SilkS) (width 0.12))
+    (fp_line (start -1.485 -0.735) (end -1.485 0.735) (layer F.SilkS) (width 0.12))
+    (fp_line (start -1.485 0.735) (end 0.8 0.735) (layer F.SilkS) (width 0.12))
+    (fp_line (start -1.48 0.73) (end -1.48 -0.73) (layer F.CrtYd) (width 0.05))
+    (fp_line (start -1.48 -0.73) (end 1.48 -0.73) (layer F.CrtYd) (width 0.05))
+    (fp_line (start 1.48 -0.73) (end 1.48 0.73) (layer F.CrtYd) (width 0.05))
+    (fp_line (start 1.48 0.73) (end -1.48 0.73) (layer F.CrtYd) (width 0.05))
+    (pad 2 smd roundrect (at 0.7875 0) (size 0.875 0.95) (layers F.Cu F.Paste F.Mask) (roundrect_rratio 0.25)
+      (net 392 /sp/~ETH_RESET))
+    (pad 1 smd roundrect (at -0.7875 0) (size 0.875 0.95) (layers F.Cu F.Paste F.Mask) (roundrect_rratio 0.25)
+      (net 6 +3V3))
+    (model ${KISYS3DMOD}/Diode_SMD.3dshapes/D_0603_1608Metric.wrl
+      (at (xyz 0 0 0))
+      (scale (xyz 1 1 1))
+      (rotate (xyz 0 0 0))
+    )
+  )
   (module Package_SO:TSSOP-24_4.4x7.8mm_P0.65mm (layer F.Cu)

Commit message: Adjust all crystal load capacitances.
fixes #8
Parts:
- C319, C327: value 3p9 -> 12p
- C320, C323: value 0p5 -> 12p5
- C410, C411: value 18p -> 12p
- Y301: value 25MHz -> 25MHz ±50ppm / SXTHM212ASA174-25.000M; footprint Crystal:Crystal_SMD_Abracon_ABM3B-4Pin_5.0x3.2mm -> Crystal:Crystal_SMD_HC49-SD
- Y302: value 32.768kHz -> 32.768kHz / FC-135 32.7680KA-A; footprint Crystal:Crystal_SMD_Abracon_ABM3-2Pin_5.0x3.2mm -> Crystal:Crystal_SMD_3215-2Pin_3.2x1.5mm
- Y401: value 25MHz ±50ppm -> 25MHz ±50ppm / SXTHM212ASA174-25.000M; footprint Crystal:Crystal_SMD_Abracon_ABM3B-4Pin_5.0x3.2mm -> Crystal:Crystal_SMD_HC49-SD
Connections:
- Y301 pad 2: GND -> /sp/OSC_IN
- Y401 pad 2: GND -> Net-(C411-Pad2)

Commit message: PCB: rearrange fan layout, simplify nets
Parts:
- J701: value Conn_01x04_Male -> FAN6
- J702: value Conn_01x04_Male -> FAN5
- J703: value Conn_01x04_Male -> FAN4
- J704: value Conn_01x04_Male -> FAN3
- J705: value Conn_01x04_Male -> FAN2
- J706: value Conn_01x04_Male -> FAN1
- moved RN702 101.1 mm to (265.0, 126.0), turned to 180 degrees
- moved RN703 95.3 mm to (253.0, 119.0), turned to 270 degrees
- moved J703 94.0 mm to (269.0, 139.0), turned to 0 degrees
- moved J705 85.6 mm to (264.0, 113.0)
- moved J702 82.3 mm to (256.0, 139.0), turned to 0 degrees
- moved J704 82.3 mm to (277.0, 113.0)
- moved U701 81.2 mm to (249.0, 126.0)
- moved J706 80.6 mm to (251.0, 113.0)
- moved RN701 76.2 mm to (253.0, 133.0), turned to 90 degrees
- moved J701 73.2 mm to (243.0, 139.0), turned to 0 degrees
- moved J1101 8.06 mm to (262.0, 75.0)
- moved J1201 8.06 mm to (262.0, 85.0)
- moved J1301 8.06 mm to (262.0, 95.0)
- moved R1101 8.06 mm to (247.0, 73.0)
- moved R1102 8.06 mm to (247.0, 77.0)
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Connections:
- RN701 pad 1: Net-(J701-Pad4) -> Net-(J701-Pad3)
- RN701 pad 2: Net-(J701-Pad3) -> Net-(J701-Pad4)
- RN701 pad 3: Net-(J702-Pad4) -> Net-(J702-Pad3)
- RN701 pad 4: Net-(J702-Pad3) -> Net-(J702-Pad4)
- RN702 pad 1: Net-(J703-Pad4) -> Net-(J703-Pad3)
- RN702 pad 2: Net-(J703-Pad3) -> Net-(J703-Pad4)
- RN702 pad 3: Net-(J704-Pad4) -> Net-(J704-Pad3)
- RN702 pad 4: Net-(J704-Pad3) -> Net-(J704-Pad4)
- RN703 pad 1: Net-(J705-Pad4) -> Net-(J705-Pad3)
- RN703 pad 2: Net-(J705-Pad3) -> Net-(J705-Pad4)
- RN703 pad 3: Net-(J706-Pad4) -> Net-(J706-Pad3)
- RN703 pad 4: Net-(J706-Pad3) -> Net-(J706-Pad4)
