File: gemini-bringup.kicad_pcb (KiCad board)
At the start: 4 copper layers, 187.2 x 112 mm, 282 parts, among them J1001 EXPANSION, J1101 SMBUS, J1201 SMBUS, J1301 SMBUS, J1401 IDC_BOX_HDR, J1501 I2CGPIO1, J1502 I2CGPIO0, J201 Conn_01x04, J202 Conn_ARM_JTAG_SWD_10, J203 Conn_2Rows-51Pins, J204 Conn_01x10, J301 Conn_ARM_JTAG_SWD_10, J302 HOST_UART, J303 AUX_HDR_J, J304 AUX_HDR_G, J401 RJ45_Würth_74980111211, J402 RJ45_Würth_74980111211, J501 SMBUS, J502 SMBUS, J503 SMBUS, J504 SMBUS, J601 Barrel_Jack, J701 FAN6, J702 FAN5, J703 FAN4, J704 FAN3, J705 FAN2, J706 FAN1, J801 IDC, J901 Micro_SD_Card, SW201 SW_SPDT, SW202 SW_SPST, SW301 RESET, SW302 BOOT0, U1101 TCA9802, U1201 TCA9802, U1301 TCA9802, U1401 TXB0106PWR, U1501 PCA9555PW, U301 STM32H753BITx, U302 MAX13235EET, U401 KSZ8863RLL, U501 LTC4306CGN, U601 OKI-78SR-3.3_1.5-W36-C, U602 INA219AxDCN, U603 INA219AxDCN, U701 MAX31790, U702 MCP1703A-5002_SOT89, U703 PCA9306DP1, U801 TXB0106PWR, U802 W25Q256FVFxx, U901 EMIF06-MSD02N16, Y301 8 MHz, Y302 32.768kHz, Y401 25MHz ±50ppm

Commit message: gemini-bringup: integrate zero-ohm resistor in ethernet switch crystal layout
Parts:
- moved R409 175.9 mm to (89.8, 101.3)
- moved Y401 1.77 mm to (88.8, 104.1)
- moved C410 1.77 mm to (90.4, 106.9)
- moved C411 1.77 mm to (87.2, 106.9)
- moved R405 1.02 mm to (92.8, 101.2)
Routing:
- net Net-(R409-Pad1): track 0.00 -> 5.24 mm
- net Net-(C410-Pad2): track 9.72 -> 5.72 mm
- net Net-(C411-Pad2): track 9.73 -> 11.6 mm
Changed lines of the file:
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@@
     (thickness 1.6)
     (drawings 58)
-    (tracks 4039)
+    (tracks 4044)
     (zones 0)
     (modules 282)
@@
   )
   (module Resistor_SMD:R_0603_1608Metric (layer F.Cu)
-    (at 264.866 84.13)
+    (at 89.8275 101.346)
     (descr "Resistor SMD 0603 (1608 Metric), square (rectangular) end terminal, IPC_7351 nominal, (Body size source: http://www.tortai-tech.com/upload/download/2011102023233369053.pdf), generated with kicad-footprint-generator")
     (tags resistor)
     (attr smd)
-    (fp_text reference R409 (at 0 -1.43) (layer F.SilkS)
-      (effects (font (size 1 1) (thickness 0.15)))
+    (fp_text reference R409 (at -1.3085 -1.27 180) (layer F.SilkS)
+      (effects (font (size 0.75 0.75) (thickness 0.15)))
     )
     (fp_text value 0R (at 0 1.43) (layer F.Fab)
@@
   )
   (module Capacitor_SMD:C_0603_1608Metric (layer F.Cu)
-    (at 90.9875 105.2)
+    (at 90.3525 106.851)
     (descr "Capacitor SMD 0603 (1608 Metric), square (rectangular) end terminal, IPC_7351 nominal, (Body size source: http://www.tortai-tech.com/upload/download/2011102023233369053.pdf), generated with kicad-footprint-generator")
     (tags capacitor)
@@
   )
   (module Crystal:Crystal_SMD_5032-2Pin_5.0x3.2mm (layer F.Cu)
-    (at 89.4 102.4 180)
+    (at 88.765 104.051 180)
     (descr "SMD Crystal SERIES SMD2520/2 http://www.icbase.com/File/PDF/HKC/HKC00061008.pdf, 5.0x3.2mm^2 package")
     (tags "SMD SMT crystal")
     (attr smd)
-    (fp_text reference Y401 (at 0 2.6) (layer F.SilkS)
+    (fp_text reference Y401 (at 3.675 -0.089 90) (layer F.SilkS)
       (effects (font (size 0.75 0.75) (thickness 0.15)))
     )
@@
   )
   (module Resistor_SMD:R_0603_1608Metric (layer F.Cu)
-    (at 93.8 101.2 270)
+    (at 92.784 101.2 270)
     (descr "Resistor SMD 0603 (1608 Metric), square (rectangular) end terminal, IPC_7351 nominal, (Body size source: http://www.tortai-tech.com/upload/download/2011102023233369053.pdf), generated with kicad-footprint-generator")
     (tags resistor)
@@
   )
   (module Capacitor_SMD:C_0603_1608Metric (layer F.Cu)
-    (at 87.7875 105.2 180)
+    (at 87.1525 106.851 180)
     (descr "Capacitor SMD 0603 (1608 Metric), square (rectangular) end terminal, IPC_7351 nominal, (Body size source: http://www.tortai-tech.com/upload/download/2011102023233369053.pdf), generated with kicad-footprint-generator")
     (tags capacitor)
@@
   (segment (start 66.2 80.7875) (end 66.2 81.6) (width 0.2) (layer B.Cu) (net 1) (status 10))
   (segment (start 66.2 81.6) (end 66.2 82.4) (width 0.2) (layer B.Cu) (net 1) (status 20))
-  (via (at 89.4 105.2) (size 0.8) (drill 0.4) (layers F.Cu B.Cu) (net 1))
-  (segment (start 88.575 105.2) (end 89.4 105.2) (width 0.2) (layer F.Cu) (net 1) (status 10))
-  (segment (start 89.4 105.2) (end 90.2 105.2) (width 0.2) (layer F.Cu) (net 1) (status 20))
+  (via (at 88.765 106.851) (size 0.8) (drill 0.4) (layers F.Cu B.Cu) (net 1))
+  (segment (start 87.94 106.851) (end 88.765 106.851) (width 0.2) (layer F.Cu) (net 1) (status 10))
+  (segment (start 88.765 106.851) (end 89.565 106.851) (width 0.2) (layer F.Cu) (net 1) (status 20))
   (via (at 94.2 92.6) (size 0.8) (drill 0.4) (layers F.Cu B.Cu) (net 1))
   (segment (start 94.2125 92.5875) (end 94.2 92.6) (width 0.2) (layer B.Cu) (net 1))
@@
   (segment (start 66.2 83.975) (end 67.9875 83.975) (width 0.2) (layer B.Cu) (net 14) (status 30))
   (segment (start 68.0125 84) (end 68.0125 82.4) (width 0.2) (layer B.Cu) (net 14) (status 30))
-  (segment (start 91.25 104.675) (end 91.775 105.2) (width 0.2) (layer F.Cu) (net 15) (status 20))
-  (segment (start 91.25 102.4) (end 91.25 104.675) (width 0.2) (layer F.Cu) (net 15) (status 10))
-  (segment (start 89.65 100.8) (end 91.25 102.4) (width 0.2) (layer F.Cu) (net 15) (status 20))
-  (segment (start 89.65 96.3625) (end 89.65 100.8) (width 0.2) (layer F.Cu) (net 15) (status 10))
-  (segment (start 87.55 104.65) (end 87 105.2) (width 0.2) (layer F.Cu) (net 16) (status 20))
-  (segment (start 87.55 102.4) (end 87.55 104.65) (width 0.2) (layer F.Cu) (net 16) (status 10))
-  (segment (start 89.15 100.8) (end 87.55 102.4) (width 0.2) (layer F.Cu) (net 16) (status 20))
-  (segment (start 89.15 96.3625) (end 89.15 100.8) (width 0.2) (layer F.Cu) (net 16) (status 10))
+  (segment (start 90.615 106.326) (end 91.14 106.851) (width 0.2) (layer F.Cu) (net 15) (status 20))
+  (segment (start 90.615 104.051) (end 90.615 106.326) (width 0.2) (layer F.Cu) (net 15) (status 10))
+  (segment (start 90.615 101.346) (end 90.615 104.051) (width 0.2) (layer F.Cu) (net 15))
+  (segment (start 86.915 106.301) (end 86.365 106.851) (width 0.2) (layer F.Cu) (net 16) (status 20))
+  (segment (start 86.915 104.051) (end 86.915 106.301) (width 0.2) (layer F.Cu) (net 16) (status 10))
+  (segment (start 86.915 99.365204) (end 86.915 104.051) (width 0.2) (layer F.Cu) (net 16))
+  (segment (start 89.15 97.130204) (end 86.915 99.365204) (width 0.2) (layer F.Cu) (net 16))
+  (segment (start 89.15 96.3625) (end 89.15 97.130204) (width 0.2) (layer F.Cu) (net 16))
   (segment (start 68 79.2125) (end 68.0125 79.2) (width 0.2) (layer B.Cu) (net 17) (status 30))
   (segment (start 66.2 79.2125) (end 68 79.2125) (width 0.2) (layer B.Cu) (net 17) (status 30))
@@
   (segment (start 66.0625 54.7375) (end 67.435099 56.110099) (width 0.2) (layer F.Cu) (net 308))
   (segment (start 65.5 54.175) (end 66.0625 54.7375) (width 0.2) (layer F.Cu) (net 308))
+  (segment (start 89.59991 97.34409) (end 89.04 97.904) (width 0.2) (layer F.Cu) (net 310))
+  (segment (start 89.59991 96.83609) (end 89.59991 97.34409) (width 0.2) (layer F.Cu) (net 310))
+  (segment (start 89.04 97.904) (end 89.04 101.346) (width 0.2) (layer F.Cu) (net 310))
+  (segment (start 89.65 96.786) (end 89.59991 96.83609) (width 0.2) (layer F.Cu) (net 310))
+  (segment (start 89.65 96.3625) (end 89.65 96.786) (width 0.2) (layer F.Cu) (net 310))
   (zone (net 1) (net_name GND) (layer In2.Cu) (hatch edge 0.508)
     (connect_pads (clearance 0.2))

Commit message: gemini-bringup: incorporate zero-ohm link in STM32H753 high-speed crystal
Parts:
- moved R339 134.6 mm to (118.5, 73.7)
Routing:
- net /sp/OSC_OUT: track 14.4 -> 6.19 mm
- net Net-(C319-Pad1): track 0.00 -> 6.61 mm
Changed lines of the file:
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@@
     (thickness 1.6)
     (drawings 58)
-    (tracks 4044)
+    (tracks 4045)
     (zones 0)
     (modules 282)
@@
   )
   (module Resistor_SMD:R_0603_1608Metric (layer F.Cu)
-    (at 252.476 86.36)
+    (at 118.5165 73.66)
     (descr "Resistor SMD 0603 (1608 Metric), square (rectangular) end terminal, IPC_7351 nominal, (Body size source: http://www.tortai-tech.com/upload/download/2011102023233369053.pdf), generated with kicad-footprint-generator")
     (tags resistor)
     (attr smd)
-    (fp_text reference R339 (at 0 -1.43) (layer F.SilkS)
-      (effects (font (size 1 1) (thickness 0.15)))
+    (fp_text reference R339 (at -0.0255 -3.048) (layer F.SilkS)
+      (effects (font (size 0.75 0.75) (thickness 0.15)))
     )
     (fp_text value 0R (at 0 1.43) (layer F.Fab)
@@
     (tags resistor)
     (attr smd)
-    (fp_text reference R325 (at 0 -1.43) (layer F.SilkS)
+    (fp_text reference R325 (at 0.1965 -3.157) (layer F.SilkS)
       (effects (font (size 0.75 0.75) (thickness 0.15)))
     )
@@
   (via (at 59.584 37.986) (size 0.8) (drill 0.4) (layers F.Cu B.Cu) (net 6))
   (segment (start 60.734 37.986) (end 59.584 37.986) (width 0.4) (layer F.Cu) (net 6))
-  (segment (start 112.9375 74.85) (end 112 75.7875) (width 0.2) (layer F.Cu) (net 7) (status 20))
-  (segment (start 115 74.85) (end 112.9375 74.85) (width 0.2) (layer F.Cu) (net 7) (status 10))
-  (segment (start 116.6 73.25) (end 115 74.85) (width 0.2) (layer F.Cu) (net 7) (status 20))
-  (segment (start 125.325 73.25) (end 116.6 73.25) (width 0.2) (layer F.Cu) (net 7) (status 10))
+  (segment (start 119.714 73.25) (end 119.304 73.66) (width 0.2) (layer F.Cu) (net 7))
+  (segment (start 125.325 73.25) (end 119.714 73.25) (width 0.2) (layer F.Cu) (net 7))
+  (segment (start 112.9375 74.85) (end 112 75.7875) (width 0.2) (layer F.Cu) (net 309) (status 20))
+  (segment (start 115 74.85) (end 112.9375 74.85) (width 0.2) (layer F.Cu) (net 309) (status 10))
   (segment (start 116 61.75) (end 115 62.75) (width 0.2) (layer F.Cu) (net 8) (status 20))
   (segment (start 125.325 61.75) (end 116 61.75) (width 0.2) (layer F.Cu) (net 8) (status 10))
@@
   (segment (start 95.9 84) (end 94.8125 84) (width 0.2) (layer F.Cu) (net 140) (status 20))
   (segment (start 112.8 81.7) (end 111.6 81.7) (width 0.2) (layer F.Cu) (net 140) (status 10))
-  (segment (start 115.8 79.5) (end 114.4 79.5) (width 0.2) (layer F.Cu) (net 141) (status 20))
-  (segment (start 120.5375 74.7625) (end 115.8 79.5) (width 0.2) (layer F.Cu) (net 141))
-  (segment (start 120.5375 74.75) (end 120.5375 74.7625) (width 0.2) (layer F.Cu) (net 141))
-  (segment (start 125.325 74.75) (end 120.5375 74.75) (width 0.2) (layer F.Cu) (net 141) (status 10))
+  (segment (start 116.207 79.5) (end 114.4 79.5) (width 0.2) (layer F.Cu) (net 141))
+  (segment (start 120.957 74.75) (end 116.207 79.5) (width 0.2) (layer F.Cu) (net 141))
+  (segment (start 125.325 74.75) (end 120.957 74.75) (width 0.2) (layer F.Cu) (net 141))
   (segment (start 105.5125 79.5) (end 95.5625 89.45) (width 0.2) (layer F.Cu) (net 142) (status 20))
   (segment (start 112.825 79.5) (end 105.5125 79.5) (width 0.2) (layer F.Cu) (net 142) (status 10))
@@
   (segment (start 99.9625 89.95) (end 100.0125 90) (width 0.2) (layer F.Cu) (net 152) (status 30))
   (segment (start 95.5625 89.95) (end 99.9625 89.95) (width 0.2) (layer F.Cu) (net 152) (status 30))
+  (segment (start 100.0125 88.2875) (end 100.0125 90) (width 0.2) (layer F.Cu) (net 152))
   (segment (start 107.89991 80.40009) (end 100.0125 88.2875) (width 0.2) (layer F.Cu) (net 152))
-  (segment (start 113.56241 80.23759) (end 113.39991 80.40009) (width 0.2) (layer F.Cu) (net 152))
   (segment (start 113.39991 80.40009) (end 107.89991 80.40009) (width 0.2) (layer F.Cu) (net 152))
+  (segment (start 113.56241 80.23759) (end 113.39991 80.40009) (width 0.2) (layer F.Cu) (net 152))
   (segment (start 114.791502 77.9) (end 113.56241 79.129092) (width 0.2) (layer F.Cu) (net 152))
   (segment (start 113.56241 79.129092) (end 113.56241 80.23759) (width 0.2) (layer F.Cu) (net 152))
-  (segment (start 116.2 77.9) (end 114.791502 77.9) (width 0.2) (layer F.Cu) (net 152))
-  (segment (start 100.0125 88.2875) (end 100.0125 90) (width 0.2) (layer F.Cu) (net 152) (status 20))
-  (segment (start 119.85 74.25) (end 116.2 77.9) (width 0.2) (layer F.Cu) (net 152))
-  (segment (start 125.325 74.25) (end 119.85 74.25) (width 0.2) (layer F.Cu) (net 152) (status 10))
+  (segment (start 116.918 77.9) (end 114.791502 77.9) (width 0.2) (layer F.Cu) (net 152))
+  (segment (start 120.568 74.25) (end 116.918 77.9) (width 0.2) (layer F.Cu) (net 152))
+  (segment (start 125.325 74.25) (end 120.568 74.25) (width 0.2) (layer F.Cu) (net 152))
   (segment (start 84.05 91.95) (end 81.8 94.2) (width 0.2) (layer F.Cu) (net 153) (status 20))
   (segment (start 87.2375 91.95) (end 84.05 91.95) (width 0.2) (layer F.Cu) (net 153) (status 10))
@@
   (segment (start 90.7875 83.975) (end 90.8 83.9875) (width 0.2) (layer F.Cu) (net 240) (status 30))
   (segment (start 87.6 83.975) (end 90.7875 83.975) (width 0.2) (layer F.Cu) (net 240) (status 30))
-  (segment (start 121.25 75.25) (end 115.7 80.8) (width 0.2) (layer F.Cu) (net 240))
-  (segment (start 125.325 75.25) (end 121.25 75.25) (width 0.2) (layer F.Cu) (net 240) (status 10))
-  (segment (start 115.7 80.8) (end 111.4 80.8) (width 0.2) (layer F.Cu) (net 240))
   (via (at 107.7 84.5) (size 0.8) (drill 0.4) (layers F.Cu B.Cu) (net 240))
-  (segment (start 111.4 80.8) (end 107.7 84.5) (width 0.2) (layer F.Cu) (net 240))
   (via (at 91.7 85.1) (size 0.8) (drill 0.4) (layers F.Cu B.Cu) (net 240))
   (segment (start 107.1 85.1) (end 91.7 85.1) (width 0.2) (layer B.Cu) (net 240))
@@
   (segment (start 87.425 84.15) (end 87.6 83.975) (width 0.2) (layer F.Cu) (net 240))
   (segment (start 87.425 84.225) (end 87.425 84.15) (width 0.2) (layer F.Cu) (net 240))
+  (segment (start 111.4 80.8) (end 107.7 84.5) (width 0.2) (layer F.Cu) (net 240))
+  (segment (start 115.923 80.8) (end 111.4 80.8) (width 0.2) (layer F.Cu) (net 240))
+  (segment (start 121.473 75.25) (end 115.923 80.8) (width 0.2) (layer F.Cu) (net 240))
+  (segment (start 125.325 75.25) (end 121.473 75.25) (width 0.2) (layer F.Cu) (net 240))
   (segment (start 210.0625 72.825) (end 214.025 72.825) (width 0.2) (layer F.Cu) (net 241))
   (segment (start 222.280099 88.450099) (end 223.08 89.25) (width 0.2) (layer F.Cu) (net 241))
@@
   (segment (start 66.0625 54.7375) (end 67.435099 56.110099) (width 0.2) (layer F.Cu) (net 308))
   (segment (start 65.5 54.175) (end 66.0625 54.7375) (width 0.2) (layer F.Cu) (net 308))
+  (segment (start 116.19 73.66) (end 115 74.85) (width 0.2) (layer F.Cu) (net 309))
+  (segment (start 117.729 73.66) (end 116.19 73.66) (width 0.2) (layer F.Cu) (net 309))
   (segment (start 89.59991 97.34409) (end 89.04 97.904) (width 0.2) (layer F.Cu) (net 310))
   (segment (start 89.59991 96.83609) (end 89.59991 97.34409) (width 0.2) (layer F.Cu) (net 310))

Commit message: gemini-bringup: rework STM32H753 VDDA bypass caps
Parts:
- moved C326 4.28 mm to (128.4, 79.6), turned to 270 degrees
- moved C330 0.06 mm to (129.5, 76.4)
Routing:
- net VDDA: track 7.69 -> 1.74 mm
- net GND: track 336.3 -> 338.0 mm
- added copper zone on B.Cu, net VDDA
Changed lines of the file:
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@@
     (thickness 1.6)
     (drawings 58)
-    (tracks 4045)
+    (tracks 4041)
     (zones 0)
     (modules 282)
@@
   )
   (module Capacitor_SMD:C_0805_2012Metric (layer B.Cu)
-    (at 131.2 76.4 90)
+    (at 128.397 79.629 270)
     (descr "Capacitor SMD 0805 (2012 Metric), square (rectangular) end terminal, IPC_7351 nominal, (Body size source: https://docs.google.com/spreadsheets/d/1BsfQQcO9C6DZCsRaXUlFlo91Tg2WpOkGARC1WS5S8t0/edit?usp=sharing), generated with kicad-footprint-generator")
     (tags capacitor)
@@
       (effects (font (size 0.5 0.5) (thickness 0.08)) (justify mirror))
     )
-    (pad 2 smd roundrect (at 0.9375 0 90) (size 0.975 1.4) (layers B.Cu B.Paste B.Mask) (roundrect_rratio 0.25)
+    (pad 2 smd roundrect (at 0.9375 0 270) (size 0.975 1.4) (layers B.Cu B.Paste B.Mask) (roundrect_rratio 0.25)
       (net 1 GND))
-    (pad 1 smd roundrect (at -0.9375 0 90) (size 0.975 1.4) (layers B.Cu B.Paste B.Mask) (roundrect_rratio 0.25)
+    (pad 1 smd roundrect (at -0.9375 0 270) (size 0.975 1.4) (layers B.Cu B.Paste B.Mask) (roundrect_rratio 0.25)
       (net 3 VDDA))
     (model ${KISYS3DMOD}/Capacitor_SMD.3dshapes/C_0805_2012Metric.wrl
@@
   )
   (module Capacitor_SMD:C_0603_1608Metric (layer B.Cu)
-    (at 129.6 76.4 90)
+    (at 129.54 76.4 90)
     (descr "Capacitor SMD 0603 (1608 Metric), square (rectangular) end terminal, IPC_7351 nominal, (Body size source: http://www.tortai-tech.com/upload/download/2011102023233369053.pdf), generated with kicad-footprint-generator")
     (tags capacitor)
@@
   (segment (start 126.239931 69.25) (end 126.800315 68.689616) (width 0.2) (layer F.Cu) (net 1))
   (segment (start 125.325 69.25) (end 126.239931 69.25) (width 0.2) (layer F.Cu) (net 1) (status 10))
-  (segment (start 126.55 76.75) (end 126.8 77) (width 0.2) (layer F.Cu) (net 1))
-  (via (at 126.8 77) (size 0.8) (drill 0.4) (layers F.Cu B.Cu) (net 1))
-  (segment (start 125.325 76.75) (end 126.55 76.75) (width 0.2) (layer F.Cu) (net 1) (status 10))
   (via (at 126.8 81.8) (size 0.8) (drill 0.4) (layers F.Cu B.Cu) (net 1))
   (segment (start 126.35 82.25) (end 126.8 81.8) (width 0.2) (layer F.Cu) (net 1))
@@
   (segment (start 126.6125 81.6125) (end 126.8 81.8) (width 0.2) (layer B.Cu) (net 1))
   (segment (start 125.6 81.6125) (end 126.6125 81.6125) (width 0.2) (layer B.Cu) (net 1) (status 10))
-  (segment (start 126.6125 77.1875) (end 126.8 77) (width 0.2) (layer B.Cu) (net 1))
-  (segment (start 125.6 77.1875) (end 126.6125 77.1875) (width 0.2) (layer B.Cu) (net 1) (status 10))
   (segment (start 126.477431 69.0125) (end 126.800315 68.689616) (width 0.2) (layer B.Cu) (net 1))
   (segment (start 125.6 69.0125) (end 126.477431 69.0125) (width 0.2) (layer B.Cu) (net 1) (status 10))
   (segment (start 126.665431 63.2125) (end 126.779487 63.326556) (width 0.2) (layer B.Cu) (net 1))
   (segment (start 125.6 63.2125) (end 126.665431 63.2125) (width 0.2) (layer B.Cu) (net 1) (status 10))
-  (via (at 130.4 75.6) (size 0.8) (drill 0.4) (layers F.Cu B.Cu) (net 1))
-  (segment (start 130.3875 75.6125) (end 130.4 75.6) (width 0.2) (layer B.Cu) (net 1))
-  (segment (start 131.2 75.6125) (end 130.3875 75.6125) (width 0.2) (layer B.Cu) (net 1) (status 10))
-  (segment (start 130.3875 75.6125) (end 129.6 75.6125) (width 0.2) (layer B.Cu) (net 1) (status 20))
+  (via (at 130.683 75.6125) (size 0.8) (drill 0.4) (layers F.Cu B.Cu) (net 1))
   (segment (start 74.53 98.6) (end 74.7 98.43) (width 0.3) (layer F.Cu) (net 1) (status 30))
   (via (at 66.2 103) (size 0.8) (drill 0.4) (layers F.Cu B.Cu) (net 1))
@@
   (segment (start 94.2 93.255) (end 94.2 92.6) (width 0.2) (layer B.Cu) (net 1))
   (segment (start 93.094 94.361) (end 94.2 93.255) (width 0.2) (layer B.Cu) (net 1))
+  (segment (start 126.538297 77.1875) (end 126.79114 76.934657) (width 0.2) (layer B.Cu) (net 1))
+  (segment (start 126.606483 76.75) (end 126.79114 76.934657) (width 0.2) (layer F.Cu) (net 1))
+  (segment (start 125.6 77.1875) (end 126.538297 77.1875) (width 0.2) (layer B.Cu) (net 1))
+  (via (at 126.79114 76.934657) (size 0.8) (drill 0.4) (layers F.Cu B.Cu) (net 1))
+  (segment (start 125.325 76.75) (end 126.606483 76.75) (width 0.2) (layer F.Cu) (net 1))
+  (segment (start 129.54 75.6125) (end 130.683 75.6125) (width 0.2) (layer B.Cu) (net 1))
+  (segment (start 128.0335 80.5665) (end 128.397 80.5665) (width 0.2) (layer B.Cu) (net 1))
+  (segment (start 126.8 81.8) (end 128.0335 80.5665) (width 0.2) (layer B.Cu) (net 1))
   (segment (start 187.699901 21.699901) (end 182.3 16.3) (width 0.2) (layer F.Cu) (net 2))
   (segment (start 198.1 18.15) (end 194.550099 21.699901) (width 0.2) (layer F.Cu) (net 2))
@@
   (segment (start 186.7 40.3) (end 186.7 22.699802) (width 0.2) (layer F.Cu) (net 2))
   (segment (start 184.5 42.5) (end 186.7 40.3) (width 0.2) (layer F.Cu) (net 2))
-  (segment (start 126.75 77.75) (end 127 78) (width 0.2) (layer F.Cu) (net 3))
-  (via (at 127 78) (size 0.8) (drill 0.4) (layers F.Cu B.Cu) (net 3))
-  (segment (start 125.325 77.75) (end 126.75 77.75) (width 0.2) (layer F.Cu) (net 3) (status 10))
-  (segment (start 127.1875 78) (end 128 77.1875) (width 0.2) (layer B.Cu) (net 3) (status 20))
-  (segment (start 127 78) (end 127.1875 78) (width 0.2) (layer B.Cu) (net 3))
-  (segment (start 128 77.1875) (end 131.2 77.1875) (width 0.2) (layer B.Cu) (net 3) (status 30))
-  (segment (start 127 78.7875) (end 126.5875 79.2) (width 0.2) (layer B.Cu) (net 3) (status 20))
-  (segment (start 127 78) (end 127 78.7875) (width 0.2) (layer B.Cu) (net 3))
+  (segment (start 126.5875 78.1365) (end 126.746 77.978) (width 0.2) (layer B.Cu) (net 3))
+  (segment (start 126.518 77.75) (end 126.746 77.978) (width 0.2) (layer F.Cu) (net 3))
+  (segment (start 125.325 77.75) (end 126.518 77.75) (width 0.2) (layer F.Cu) (net 3))
+  (via (at 126.746 77.978) (size 0.8) (drill 0.4) (layers F.Cu B.Cu) (net 3))
   (via (at 126.9 73.8) (size 0.8) (drill 0.4) (layers F.Cu B.Cu) (net 4))
   (segment (start 126.85 73.75) (end 126.9 73.8) (width 0.2) (layer F.Cu) (net 4))
@@
       )
     )
+  )
+  (zone (net 3) (net_name VDDA) (layer B.Cu) (hatch edge 0.508)
+    (connect_pads yes (clearance 0.2))
+    (min_thickness 0.254)
+    (fill yes (arc_segments 32) (thermal_gap 0.3) (thermal_bridge_width 0.3))
+    (polygon
+      (pts
+        (xy 130.302 78.232) (xy 129.159 79.883) (xy 125.984 79.883) (xy 125.984 77.851) (xy 127.254 76.454)
+        (xy 130.302 76.454)
+      )
+    )
