File: i2c-ext.sch (KiCad schematic (older format))
At the start: 4 parts

Commit message: ERC clean.
- Power flags.
- NCs.
- Fixed a few net typos that resulted in disconnects.
Parts:
- added R?: 10k, symbol Device:R
Connections:
- net +3V3: now also R?.1
- net at U?.5 (EN): now also R?.2
Changed lines of the file:
@@
 $Descr A4 11693 8268
 encoding utf-8
-Sheet 11 13
+Sheet 13 13
 Title "Offboard I2C connector (one bus)"
 Date ""
@@
 	7150 3400 7150 3150
 Wire Wire Line
-	7150 3150 5700 3150
+	7150 3150 6300 3150
 Wire Wire Line
 	7150 3600 7050 3600
@@
 Text Notes 6050 3400 0    50   ~ 0
 NO PULLUPS THIS SIDE\nTCA9802 handles it
+$Comp
+L Device:R R?
+U 1 1 600BC5DC
+P 5050 3750
+AR Path="/5F2F1B47/600BC5DC" Ref="R?"  Part="1"
+AR Path="/5F2F7878/600BC5DC" Ref="R?"  Part="1"
+AR Path="/5F2FE5B6/600BC5DC" Ref="R?"  Part="1"
+AR Path="/5F3042B8/600BC5DC" Ref="R?"  Part="1"
+F 0 "R?" V 5000 3850 50  0000 L CNN
+F 1 "10k" V 5050 3700 50  0000 L CNN
+F 2 "" V 4980 3750 50  0001 C CNN
+F 3 "~" H 5050 3750 50  0001 C CNN
+	1    5050 3750
+	0    -1   -1   0
+$EndComp
+$Comp
+L power:+3V3 #PWR?
+U 1 1 600BD49C
+P 4900 3750
+F 0 "#PWR?" H 4900 3600 50  0001 C CNN
+F 1 "+3V3" V 4915 3878 50  0000 L CNN
+F 2 "" H 4900 3750 50  0001 C CNN
+F 3 "" H 4900 3750 50  0001 C CNN
+	1    4900 3750
+	0    -1   -1   0
+$EndComp
+$Comp
+L power:PWR_FLAG #FLG?
+U 1 1 60108223
+P 6300 3150
+F 0 "#FLG?" H 6300 3225 50  0001 C CNN
+F 1 "PWR_FLAG" H 6300 3323 50  0000 C CNN
+F 2 "" H 6300 3150 50  0001 C CNN
+F 3 "~" H 6300 3150 50  0001 C CNN
+	1    6300 3150
+	1    0    0    -1
+$EndComp
+Connection ~ 6300 3150
+Wire Wire Line
+	6300 3150 5700 3150
 $EndSCHEMATC

Commit message: Annotate in preparation for review
Parts:
- gave numbers to parts that had none: 5
Changed lines of the file:
@@
 $EndDescr
 $Comp
-L Interface:TCA9802 U?
+L Interface:TCA9802 U1101
 U 1 1 5F2F1DD6
 P 5600 3650
-AR Path="/5F2F1B47/5F2F1DD6" Ref="U?"  Part="1"
+AR Path="/5F2F1B47/5F2F1DD6" Ref="U1101"  Part="1"
 AR Path="/5F2F7878/5F2F1DD6" Ref="U?"  Part="1"
-AR Path="/5F2FE5B6/5F2F1DD6" Ref="U?"  Part="1"
-AR Path="/5F3042B8/5F2F1DD6" Ref="U?"  Part="1"
-F 0 "U?" H 5600 3550 50  0000 C CNN
+AR Path="/5F2FE5B6/5F2F1DD6" Ref="U1201"  Part="1"
+AR Path="/5F3042B8/5F2F1DD6" Ref="U1301"  Part="1"
+F 0 "U1301" H 5600 3550 50  0000 C CNN
 F 1 "TCA9802" H 5800 3200 50  0000 C CNN
 F 2 "Package_SO:VSSOP-8_3.0x3.0mm_P0.65mm" H 6500 3200 50  0001 C CNN
@@
 $EndComp
 $Comp
-L power:+3V3 #PWR?
+L power:+3V3 #PWR01103
 U 1 1 5F2F21C9
 P 5500 3150
-AR Path="/5F2F1B47/5F2F21C9" Ref="#PWR?"  Part="1"
+AR Path="/5F2F1B47/5F2F21C9" Ref="#PWR01103"  Part="1"
 AR Path="/5F2F7878/5F2F21C9" Ref="#PWR?"  Part="1"
-AR Path="/5F2FE5B6/5F2F21C9" Ref="#PWR?"  Part="1"
-AR Path="/5F3042B8/5F2F21C9" Ref="#PWR?"  Part="1"
-F 0 "#PWR?" H 5500 3000 50  0001 C CNN
+AR Path="/5F2FE5B6/5F2F21C9" Ref="#PWR01203"  Part="1"
+AR Path="/5F3042B8/5F2F21C9" Ref="#PWR01303"  Part="1"
+F 0 "#PWR01303" H 5500 3000 50  0001 C CNN
 F 1 "+3V3" H 5515 3323 50  0000 C CNN
 F 2 "" H 5500 3150 50  0001 C CNN
@@
 $EndComp
 $Comp
-L power:GND #PWR?
+L power:GND #PWR01104
 U 1 1 5F2F2367
 P 5600 4150
-AR Path="/5F2F1B47/5F2F2367" Ref="#PWR?"  Part="1"
+AR Path="/5F2F1B47/5F2F2367" Ref="#PWR01104"  Part="1"
 AR Path="/5F2F7878/5F2F2367" Ref="#PWR?"  Part="1"
-AR Path="/5F2FE5B6/5F2F2367" Ref="#PWR?"  Part="1"
-AR Path="/5F3042B8/5F2F2367" Ref="#PWR?"  Part="1"
-F 0 "#PWR?" H 5600 3900 50  0001 C CNN
+AR Path="/5F2FE5B6/5F2F2367" Ref="#PWR01204"  Part="1"
+AR Path="/5F3042B8/5F2F2367" Ref="#PWR01304"  Part="1"
+F 0 "#PWR01304" H 5600 3900 50  0001 C CNN
 F 1 "GND" H 5605 3977 50  0000 C CNN
 F 2 "" H 5600 4150 50  0001 C CNN
@@
 $EndComp
 $Comp
-L Connector_Generic:Conn_01x05 J?
+L Connector_Generic:Conn_01x05 J1101
 U 1 1 5F2F26BC
 P 7350 3600
-AR Path="/5F2F1B47/5F2F26BC" Ref="J?"  Part="1"
+AR Path="/5F2F1B47/5F2F26BC" Ref="J1101"  Part="1"
 AR Path="/5F2F7878/5F2F26BC" Ref="J?"  Part="1"
-AR Path="/5F2FE5B6/5F2F26BC" Ref="J?"  Part="1"
-AR Path="/5F3042B8/5F2F26BC" Ref="J?"  Part="1"
-F 0 "J?" H 7430 3642 50  0000 L CNN
+AR Path="/5F2FE5B6/5F2F26BC" Ref="J1201"  Part="1"
+AR Path="/5F3042B8/5F2F26BC" Ref="J1301"  Part="1"
+F 0 "J1301" H 7430 3642 50  0000 L CNN
 F 1 "SMBUS" H 7430 3551 50  0000 L CNN
 F 2 "" H 7350 3600 50  0001 C CNN
@@
 	7050 3600 7050 4100
 $Comp
-L power:GND #PWR?
+L power:GND #PWR01105
 U 1 1 5F2F3249
 P 7050 4100
-AR Path="/5F2F1B47/5F2F3249" Ref="#PWR?"  Part="1"
+AR Path="/5F2F1B47/5F2F3249" Ref="#PWR01105"  Part="1"
 AR Path="/5F2F7878/5F2F3249" Ref="#PWR?"  Part="1"
-AR Path="/5F2FE5B6/5F2F3249" Ref="#PWR?"  Part="1"
-AR Path="/5F3042B8/5F2F3249" Ref="#PWR?"  Part="1"
-F 0 "#PWR?" H 7050 3850 50  0001 C CNN
+AR Path="/5F2FE5B6/5F2F3249" Ref="#PWR01205"  Part="1"
+AR Path="/5F3042B8/5F2F3249" Ref="#PWR01305"  Part="1"
+F 0 "#PWR01305" H 7050 3850 50  0001 C CNN
 F 1 "GND" H 7055 3927 50  0000 C CNN
 F 2 "" H 7050 4100 50  0001 C CNN
@@
 	4700 3650 5050 3650
 $Comp
-L Device:R R?
+L Device:R R1101
 U 1 1 5F2F4AED
 P 4900 3200
-AR Path="/5F2F1B47/5F2F4AED" Ref="R?"  Part="1"
+AR Path="/5F2F1B47/5F2F4AED" Ref="R1101"  Part="1"
 AR Path="/5F2F7878/5F2F4AED" Ref="R?"  Part="1"
-AR Path="/5F2FE5B6/5F2F4AED" Ref="R?"  Part="1"
-AR Path="/5F3042B8/5F2F4AED" Ref="R?"  Part="1"
-F 0 "R?" V 4850 3300 50  0000 L CNN
+AR Path="/5F2FE5B6/5F2F4AED" Ref="R1201"  Part="1"
+AR Path="/5F3042B8/5F2F4AED" Ref="R1301"  Part="1"
+F 0 "R1301" V 4850 3300 50  0000 L CNN
 F 1 "3k" V 4900 3150 50  0000 L CNN
 F 2 "" V 4830 3200 50  0001 C CNN
@@
 	4900 3550 5200 3550
 $Comp
-L Device:R R?
+L Device:R R1102
 U 1 1 5F2F511D
 P 5050 3200
-AR Path="/5F2F1B47/5F2F511D" Ref="R?"  Part="1"
+AR Path="/5F2F1B47/5F2F511D" Ref="R1102"  Part="1"
 AR Path="/5F2F7878/5F2F511D" Ref="R?"  Part="1"
-AR Path="/5F2FE5B6/5F2F511D" Ref="R?"  Part="1"
-AR Path="/5F3042B8/5F2F511D" Ref="R?"  Part="1"
-F 0 "R?" V 5000 3300 50  0000 L CNN
+AR Path="/5F2FE5B6/5F2F511D" Ref="R1202"  Part="1"
+AR Path="/5F3042B8/5F2F511D" Ref="R1302"  Part="1"
+F 0 "R1302" V 5000 3300 50  0000 L CNN
 F 1 "3k" V 5050 3150 50  0000 L CNN
 F 2 "" V 4980 3200 50  0001 C CNN
@@
 	4900 2950 4900 3050
 $Comp
-L power:+3V3 #PWR?
+L power:+3V3 #PWR01102
 U 1 1 5F2F5A4A
 P 5000 2950
-AR Path="/5F2F1B47/5F2F5A4A" Ref="#PWR?"  Part="1"
+AR Path="/5F2F1B47/5F2F5A4A" Ref="#PWR01102"  Part="1"
 AR Path="/5F2F7878/5F2F5A4A" Ref="#PWR?"  Part="1"
-AR Path="/5F2FE5B6/5F2F5A4A" Ref="#PWR?"  Part="1"
-AR Path="/5F3042B8/5F2F5A4A" Ref="#PWR?"  Part="1"
-F 0 "#PWR?" H 5000 2800 50  0001 C CNN
+AR Path="/5F2FE5B6/5F2F5A4A" Ref="#PWR01202"  Part="1"
+AR Path="/5F3042B8/5F2F5A4A" Ref="#PWR01302"  Part="1"
+F 0 "#PWR01302" H 5000 2800 50  0001 C CNN
 F 1 "+3V3" H 5015 3123 50  0000 C CNN
 F 2 "" H 5000 2950 50  0001 C CNN
@@
 NO PULLUPS THIS SIDE\nTCA9802 handles it
 $Comp
-L Device:R R?
+L Device:R R1103
 U 1 1 600BC5DC
 P 5050 3750
-AR Path="/5F2F1B47/600BC5DC" Ref="R?"  Part="1"
+AR Path="/5F2F1B47/600BC5DC" Ref="R1103"  Part="1"
 AR Path="/5F2F7878/600BC5DC" Ref="R?"  Part="1"
-AR Path="/5F2FE5B6/600BC5DC" Ref="R?"  Part="1"
-AR Path="/5F3042B8/600BC5DC" Ref="R?"  Part="1"
-F 0 "R?" V 5000 3850 50  0000 L CNN
+AR Path="/5F2FE5B6/600BC5DC" Ref="R1203"  Part="1"
+AR Path="/5F3042B8/600BC5DC" Ref="R1303"  Part="1"
+F 0 "R1303" V 5000 3850 50  0000 L CNN
 F 1 "10k" V 5050 3700 50  0000 L CNN
 F 2 "" V 4980 3750 50  0001 C CNN
@@
 $EndComp
 $Comp
-L power:+3V3 #PWR?
+L power:+3V3 #PWR01101
 U 1 1 600BD49C
 P 4900 3750
-F 0 "#PWR?" H 4900 3600 50  0001 C CNN
+AR Path="/5F2F1B47/600BD49C" Ref="#PWR01101"  Part="1"
+AR Path="/5F2FE5B6/600BD49C" Ref="#PWR01201"  Part="1"
+AR Path="/5F3042B8/600BD49C" Ref="#PWR01301"  Part="1"
+F 0 "#PWR01301" H 4900 3600 50  0001 C CNN
 F 1 "+3V3" V 4915 3878 50  0000 L CNN
 F 2 "" H 4900 3750 50  0001 C CNN
@@
 $EndComp
 $Comp
-L power:PWR_FLAG #FLG?
+L power:PWR_FLAG #FLG01101
 U 1 1 60108223
 P 6300 3150
-F 0 "#FLG?" H 6300 3225 50  0001 C CNN
+AR Path="/5F2F1B47/60108223" Ref="#FLG01101"  Part="1"
+AR Path="/5F2FE5B6/60108223" Ref="#FLG01201"  Part="1"
+AR Path="/5F3042B8/60108223" Ref="#FLG01301"  Part="1"
+F 0 "#FLG01301" H 6300 3225 50  0001 C CNN
 F 1 "PWR_FLAG" H 6300 3323 50  0000 C CNN
 F 2 "" H 6300 3150 50  0001 C CNN

Commit message: Assign noncontroversial footprints.
- For components that only come in one flavor, use it.
- For passives, go with 0603, except for current sense resistors.
- Use the Yamaichi socket footprint for the 'h7
- Delete at least one default but wrong association.
Parts:
- J1101: footprint (none) -> Connector_PinHeader_2.54mm:PinHeader_1x05_P2.54mm_Vertical
- R1101, R1102, R1103: footprint (none) -> Resistor_SMD:R_0603_1608Metric
Changed lines of the file:
@@
 $Descr A4 11693 8268
 encoding utf-8
-Sheet 13 13
+Sheet 11 13
 Title "Offboard I2C connector (one bus)"
 Date ""
@@
 AR Path="/5F2FE5B6/5F2F1DD6" Ref="U1201"  Part="1"
 AR Path="/5F3042B8/5F2F1DD6" Ref="U1301"  Part="1"
-F 0 "U1301" H 5600 3550 50  0000 C CNN
+F 0 "U1101" H 5600 3550 50  0000 C CNN
 F 1 "TCA9802" H 5800 3200 50  0000 C CNN
 F 2 "Package_SO:VSSOP-8_3.0x3.0mm_P0.65mm" H 6500 3200 50  0001 C CNN
@@
 AR Path="/5F2FE5B6/5F2F26BC" Ref="J1201"  Part="1"
 AR Path="/5F3042B8/5F2F26BC" Ref="J1301"  Part="1"
-F 0 "J1301" H 7430 3642 50  0000 L CNN
+F 0 "J1101" H 7430 3642 50  0000 L CNN
 F 1 "SMBUS" H 7430 3551 50  0000 L CNN
-F 2 "" H 7350 3600 50  0001 C CNN
+F 2 "Connector_PinHeader_2.54mm:PinHeader_1x05_P2.54mm_Vertical" H 7350 3600 50  0001 C CNN
 F 3 "~" H 7350 3600 50  0001 C CNN
 	1    7350 3600
@@
 AR Path="/5F2FE5B6/5F2F4AED" Ref="R1201"  Part="1"
 AR Path="/5F3042B8/5F2F4AED" Ref="R1301"  Part="1"
-F 0 "R1301" V 4850 3300 50  0000 L CNN
+F 0 "R1101" V 4850 3300 50  0000 L CNN
 F 1 "3k" V 4900 3150 50  0000 L CNN
-F 2 "" V 4830 3200 50  0001 C CNN
+F 2 "Resistor_SMD:R_0603_1608Metric" V 4830 3200 50  0001 C CNN
 F 3 "~" H 4900 3200 50  0001 C CNN
 	1    4900 3200
@@
 AR Path="/5F2FE5B6/5F2F511D" Ref="R1202"  Part="1"
 AR Path="/5F3042B8/5F2F511D" Ref="R1302"  Part="1"
-F 0 "R1302" V 5000 3300 50  0000 L CNN
+F 0 "R1102" V 5000 3300 50  0000 L CNN
 F 1 "3k" V 5050 3150 50  0000 L CNN
-F 2 "" V 4980 3200 50  0001 C CNN
+F 2 "Resistor_SMD:R_0603_1608Metric" V 4980 3200 50  0001 C CNN
 F 3 "~" H 5050 3200 50  0001 C CNN
 	1    5050 3200
@@
 AR Path="/5F2FE5B6/600BC5DC" Ref="R1203"  Part="1"
 AR Path="/5F3042B8/600BC5DC" Ref="R1303"  Part="1"
-F 0 "R1303" V 5000 3850 50  0000 L CNN
+F 0 "R1103" V 5000 3850 50  0000 L CNN
 F 1 "10k" V 5050 3700 50  0000 L CNN
-F 2 "" V 4980 3750 50  0001 C CNN
+F 2 "Resistor_SMD:R_0603_1608Metric" V 4980 3750 50  0001 C CNN
 F 3 "~" H 5050 3750 50  0001 C CNN
 	1    5050 3750

Commit message: SMD resistor packs @ fan controller, i2c mux
Changed lines of the file:
@@
 AR Path="/5F2FE5B6/5F2F1DD6" Ref="U1201"  Part="1"
 AR Path="/5F3042B8/5F2F1DD6" Ref="U1301"  Part="1"
-F 0 "U1101" H 5600 3550 50  0000 C CNN
+F 0 "U1301" H 5600 3550 50  0000 C CNN
 F 1 "TCA9802" H 5800 3200 50  0000 C CNN
 F 2 "Package_SO:VSSOP-8_3.0x3.0mm_P0.65mm" H 6500 3200 50  0001 C CNN
@@
 AR Path="/5F2FE5B6/5F2F26BC" Ref="J1201"  Part="1"
 AR Path="/5F3042B8/5F2F26BC" Ref="J1301"  Part="1"
-F 0 "J1101" H 7430 3642 50  0000 L CNN
+F 0 "J1301" H 7430 3642 50  0000 L CNN
 F 1 "SMBUS" H 7430 3551 50  0000 L CNN
 F 2 "Connector_PinHeader_2.54mm:PinHeader_1x05_P2.54mm_Vertical" H 7350 3600 50  0001 C CNN
@@
 AR Path="/5F2FE5B6/5F2F4AED" Ref="R1201"  Part="1"
 AR Path="/5F3042B8/5F2F4AED" Ref="R1301"  Part="1"
-F 0 "R1101" V 4850 3300 50  0000 L CNN
+F 0 "R1301" V 4850 3300 50  0000 L CNN
 F 1 "3k" V 4900 3150 50  0000 L CNN
 F 2 "Resistor_SMD:R_0603_1608Metric" V 4830 3200 50  0001 C CNN
@@
 AR Path="/5F2FE5B6/5F2F511D" Ref="R1202"  Part="1"
 AR Path="/5F3042B8/5F2F511D" Ref="R1302"  Part="1"
-F 0 "R1102" V 5000 3300 50  0000 L CNN
+F 0 "R1302" V 5000 3300 50  0000 L CNN
 F 1 "3k" V 5050 3150 50  0000 L CNN
 F 2 "Resistor_SMD:R_0603_1608Metric" V 4980 3200 50  0001 C CNN
@@
 AR Path="/5F2FE5B6/600BC5DC" Ref="R1203"  Part="1"
 AR Path="/5F3042B8/600BC5DC" Ref="R1303"  Part="1"
-F 0 "R1103" V 5000 3850 50  0000 L CNN
+F 0 "R1303" V 5000 3850 50  0000 L CNN
 F 1 "10k" V 5050 3700 50  0000 L CNN
 F 2 "Resistor_SMD:R_0603_1608Metric" V 4980 3750 50  0001 C CNN

Commit message: Switch SMBus to 6-pin SMD Molex SL
Parts:
- J1101: footprint Connector_PinHeader_2.54mm:PinHeader_1x05_P2.54mm_Vertical -> molex-sl:SL_1x06_Vertical_SMD; symbol Connector_Generic:Conn_01x05 -> Connector_Generic:Conn_01x06
Connections:
- net GND: now also J1101.6 (Pin_6)
Changed lines of the file:
@@
 $Descr A4 11693 8268
 encoding utf-8
-Sheet 12 15
+Sheet 11 15
 Title "Offboard I2C connector (one bus)"
 Date ""
@@
 AR Path="/5F2FE5B6/5F2F1DD6" Ref="U1201"  Part="1"
 AR Path="/5F3042B8/5F2F1DD6" Ref="U1301"  Part="1"
-F 0 "U1301" H 5600 3550 50  0000 C CNN
+F 0 "U1101" H 5600 3550 50  0000 C CNN
 F 1 "TCA9802" H 5800 3200 50  0000 C CNN
 F 2 "Package_SO:VSSOP-8_3.0x3.0mm_P0.65mm" H 6500 3200 50  0001 C CNN
@@
 AR Path="/5F2FE5B6/5F2F21C9" Ref="#PWR01203"  Part="1"
 AR Path="/5F3042B8/5F2F21C9" Ref="#PWR01303"  Part="1"
-F 0 "#PWR01303" H 5500 3000 50  0001 C CNN
+F 0 "#PWR01103" H 5500 3000 50  0001 C CNN
 F 1 "+3V3" H 5515 3323 50  0000 C CNN
 F 2 "" H 5500 3150 50  0001 C CNN
@@
 AR Path="/5F2FE5B6/5F2F2367" Ref="#PWR01204"  Part="1"
 AR Path="/5F3042B8/5F2F2367" Ref="#PWR01304"  Part="1"
-F 0 "#PWR01304" H 5600 3900 50  0001 C CNN
+F 0 "#PWR01104" H 5600 3900 50  0001 C CNN
 F 1 "GND" H 5605 3977 50  0000 C CNN
 F 2 "" H 5600 4150 50  0001 C CNN
@@
 $EndComp
 $Comp
-L Connector_Generic:Conn_01x05 J1101
+L Connector_Generic:Conn_01x06 J1101
 U 1 1 5F2F26BC
 P 7350 3600
@@
 AR Path="/5F2FE5B6/5F2F26BC" Ref="J1201"  Part="1"
 AR Path="/5F3042B8/5F2F26BC" Ref="J1301"  Part="1"
-F 0 "J1301" H 7430 3642 50  0000 L CNN
+F 0 "J1101" H 7430 3642 50  0000 L CNN
 F 1 "SMBUS" H 7430 3551 50  0000 L CNN
-F 2 "Connector_PinHeader_2.54mm:PinHeader_1x05_P2.54mm_Vertical" H 7350 3600 50  0001 C CNN
+F 2 "molex-sl:SL_1x06_Vertical_SMD" H 7350 3600 50  0001 C CNN
 F 3 "~" H 7350 3600 50  0001 C CNN
 	1    7350 3600
@@
 	7150 3600 7050 3600
 Wire Wire Line
-	7050 3600 7050 4100
+	7050 3600 7050 3900
 $Comp
 L power:GND #PWR01105
@@
 AR Path="/5F2FE5B6/5F2F3249" Ref="#PWR01205"  Part="1"
 AR Path="/5F3042B8/5F2F3249" Ref="#PWR01305"  Part="1"
-F 0 "#PWR01305" H 7050 3850 50  0001 C CNN
+F 0 "#PWR01105" H 7050 3850 50  0001 C CNN
 F 1 "GND" H 7055 3927 50  0000 C CNN
 F 2 "" H 7050 4100 50  0001 C CNN
@@
 AR Path="/5F2FE5B6/5F2F4AED" Ref="R1201"  Part="1"
 AR Path="/5F3042B8/5F2F4AED" Ref="R1301"  Part="1"
-F 0 "R1301" V 4850 3300 50  0000 L CNN
+F 0 "R1101" V 4850 3300 50  0000 L CNN
 F 1 "3k" V 4900 3150 50  0000 L CNN
 F 2 "Resistor_SMD:R_0603_1608Metric" V 4830 3200 50  0001 C CNN
@@
 AR Path="/5F2FE5B6/5F2F511D" Ref="R1202"  Part="1"
 AR Path="/5F3042B8/5F2F511D" Ref="R1302"  Part="1"
-F 0 "R1302" V 5000 3300 50  0000 L CNN
+F 0 "R1102" V 5000 3300 50  0000 L CNN
 F 1 "3k" V 5050 3150 50  0000 L CNN
 F 2 "Resistor_SMD:R_0603_1608Metric" V 4980 3200 50  0001 C CNN
@@
 AR Path="/5F2FE5B6/5F2F5A4A" Ref="#PWR01202"  Part="1"
 AR Path="/5F3042B8/5F2F5A4A" Ref="#PWR01302"  Part="1"
-F 0 "#PWR01302" H 5000 2800 50  0001 C CNN
+F 0 "#PWR01102" H 5000 2800 50  0001 C CNN
 F 1 "+3V3" H 5015 3123 50  0000 C CNN
 F 2 "" H 5000 2950 50  0001 C CNN
@@
 AR Path="/5F2FE5B6/600BC5DC" Ref="R1203"  Part="1"
 AR Path="/5F3042B8/600BC5DC" Ref="R1303"  Part="1"
-F 0 "R1303" V 5000 3850 50  0000 L CNN
+F 0 "R1103" V 5000 3850 50  0000 L CNN
 F 1 "10k" V 5050 3700 50  0000 L CNN
 F 2 "Resistor_SMD:R_0603_1608Metric" V 4980 3750 50  0001 C CNN
@@
 AR Path="/5F2FE5B6/600BD49C" Ref="#PWR01201"  Part="1"
 AR Path="/5F3042B8/600BD49C" Ref="#PWR01301"  Part="1"
-F 0 "#PWR01301" H 4900 3600 50  0001 C CNN
+F 0 "#PWR01101" H 4900 3600 50  0001 C CNN
 F 1 "+3V3" V 4915 3878 50  0000 L CNN
 F 2 "" H 4900 3750 50  0001 C CNN
@@
 AR Path="/5F2FE5B6/60108223" Ref="#FLG01201"  Part="1"
 AR Path="/5F3042B8/60108223" Ref="#FLG01301"  Part="1"
-F 0 "#FLG01301" H 6300 3225 50  0001 C CNN
+F 0 "#FLG01101" H 6300 3225 50  0001 C CNN
 F 1 "PWR_FLAG" H 6300 3323 50  0000 C CNN
 F 2 "" H 6300 3150 50  0001 C CNN
@@
 Wire Wire Line
 	6300 3150 5700 3150
+Wire Wire Line
+	7150 3900 7050 3900
+Connection ~ 7050 3900
+Wire Wire Line
+	7050 3900 7050 4100
 $EndSCHEMATC
