File: i2c-ext.sch (KiCad schematic (older format))
At the start: 7 parts, among them J1101 SMBUS, U1101 TCA9802

Commit message: i2c-ext: specify rating constraints on passives
Parts:
- C1101: value 0µ1 -> 0.1uF 3.3VDCbias
- C1102: value 0µ1 -> 0.1uF 3.6VDCbias
- R1101, R1102: value 3k3 -> 3.3kR
- R1103: value 10k -> 10kR
Other:
- moved on the sheet: R1301, R1302
Changed lines of the file:
@@
 Text HLabel 6850 3800 0    50   Input ~ 0
 ~SMBA
-Text HLabel 4700 3550 0    50   Input ~ 0
+Text HLabel 4500 3550 0    50   Input ~ 0
 SCL
-Text HLabel 4700 3650 0    50   Input ~ 0
+Text HLabel 4500 3650 0    50   Input ~ 0
 SDA
 Wire Wire Line
-	4700 3550 4900 3550
+	4500 3550 4700 3550
 Wire Wire Line
-	4700 3650 5050 3650
+	4500 3650 4850 3650
 $Comp
 L Device:R R1101
 U 1 1 5F2F4AED
-P 4900 3200
+P 4700 3200
 AR Path="/5F2F1B47/5F2F4AED" Ref="R1101"  Part="1"
 AR Path="/5F2F7878/5F2F4AED" Ref="R?"  Part="1"
 AR Path="/5F2FE5B6/5F2F4AED" Ref="R1201"  Part="1"
 AR Path="/5F3042B8/5F2F4AED" Ref="R1301"  Part="1"
-F 0 "R1301" V 4850 3300 50  0000 L CNN
-F 1 "3k3" V 4900 3150 50  0000 L CNN
-F 2 "Resistor_SMD:R_0603_1608Metric" V 4830 3200 50  0001 C CNN
-F 3 "~" H 4900 3200 50  0001 C CNN
-F 4 "CR0603-JW-332ELF" H 4900 3200 50  0001 C CNN "Mfg Part Num"
-F 5 "Bourns" H 4900 3200 50  0001 C CNN "Mfg"
-F 6 "232-00018" H 4900 3200 50  0001 C CNN "CPN"
-	1    4900 3200
+F 0 "R1301" H 4400 3250 50  0000 L CNN
+F 1 "3.3kR" H 4400 3150 50  0000 L CNN
+F 2 "Resistor_SMD:R_0603_1608Metric" V 4630 3200 50  0001 C CNN
+F 3 "~" H 4700 3200 50  0001 C CNN
+F 4 "CR0603-JW-332ELF" H 4700 3200 50  0001 C CNN "Mfg Part Num"
+F 5 "Bourns" H 4700 3200 50  0001 C CNN "Mfg"
+F 6 "232-00018" H 4700 3200 50  0001 C CNN "CPN"
+	1    4700 3200
 	1    0    0    -1
 $EndComp
 Wire Wire Line
-	4900 3350 4900 3550
-Connection ~ 4900 3550
+	4700 3350 4700 3550
+Connection ~ 4700 3550
 Wire Wire Line
-	4900 3550 5200 3550
+	4700 3550 5200 3550
 $Comp
 L Device:R R1102
 U 1 1 5F2F511D
-P 5050 3200
+P 4850 3200
 AR Path="/5F2F1B47/5F2F511D" Ref="R1102"  Part="1"
 AR Path="/5F2F7878/5F2F511D" Ref="R?"  Part="1"
 AR Path="/5F2FE5B6/5F2F511D" Ref="R1202"  Part="1"
 AR Path="/5F3042B8/5F2F511D" Ref="R1302"  Part="1"
-F 0 "R1302" V 5000 3300 50  0000 L CNN
-F 1 "3k3" V 5050 3150 50  0000 L CNN
-F 2 "Resistor_SMD:R_0603_1608Metric" V 4980 3200 50  0001 C CNN
-F 3 "~" H 5050 3200 50  0001 C CNN
-F 4 "CR0603-JW-332ELF" H 5050 3200 50  0001 C CNN "Mfg Part Num"
-F 5 "Bourns" H 5050 3200 50  0001 C CNN "Mfg"
-F 6 "232-00018" H 5050 3200 50  0001 C CNN "CPN"
-	1    5050 3200
+F 0 "R1302" H 4950 3250 50  0000 L CNN
+F 1 "3.3kR" H 4950 3150 50  0000 L CNN
+F 2 "Resistor_SMD:R_0603_1608Metric" V 4780 3200 50  0001 C CNN
+F 3 "~" H 4850 3200 50  0001 C CNN
+F 4 "CR0603-JW-332ELF" H 4850 3200 50  0001 C CNN "Mfg Part Num"
+F 5 "Bourns" H 4850 3200 50  0001 C CNN "Mfg"
+F 6 "232-00018" H 4850 3200 50  0001 C CNN "CPN"
+	1    4850 3200
 	1    0    0    -1
 $EndComp
 Wire Wire Line
-	5050 3350 5050 3650
-Connection ~ 5050 3650
+	4850 3350 4850 3650
+Connection ~ 4850 3650
 Wire Wire Line
-	5050 3650 5200 3650
+	4850 3650 5200 3650
 Wire Wire Line
-	5050 3050 5050 2950
+	4850 3050 4850 2950
 Wire Wire Line
-	5050 2950 5000 2950
+	4850 2950 4800 2950
 Wire Wire Line
-	4900 2950 4900 3050
+	4700 2950 4700 3050
 $Comp
 L power:+3V3 #PWR01102
 U 1 1 5F2F5A4A
-P 5000 2950
+P 4800 2950
 AR Path="/5F2F1B47/5F2F5A4A" Ref="#PWR01102"  Part="1"
 AR Path="/5F2F7878/5F2F5A4A" Ref="#PWR?"  Part="1"
 AR Path="/5F2FE5B6/5F2F5A4A" Ref="#PWR01202"  Part="1"
 AR Path="/5F3042B8/5F2F5A4A" Ref="#PWR01302"  Part="1"
-F 0 "#PWR01302" H 5000 2800 50  0001 C CNN
-F 1 "+3V3" H 5015 3123 50  0000 C CNN
-F 2 "" H 5000 2950 50  0001 C CNN
-F 3 "" H 5000 2950 50  0001 C CNN
-	1    5000 2950
+F 0 "#PWR01302" H 4800 2800 50  0001 C CNN
+F 1 "+3V3" H 4815 3123 50  0000 C CNN
+F 2 "" H 4800 2950 50  0001 C CNN
+F 3 "" H 4800 2950 50  0001 C CNN
+	1    4800 2950
 	1    0    0    -1
 $EndComp
-Connection ~ 5000 2950
+Connection ~ 4800 2950
 Wire Wire Line
-	5000 2950 4900 2950
+	4800 2950 4700 2950
 Text Notes 6050 3400 0    50   ~ 0
 NO PULLUPS THIS SIDE\nTCA9802 handles it
@@
 AR Path="/5F2FE5B6/600BC5DC" Ref="R1203"  Part="1"
 AR Path="/5F3042B8/600BC5DC" Ref="R1303"  Part="1"
-F 0 "R1303" V 5000 3850 50  0000 L CNN
-F 1 "10k" V 5050 3700 50  0000 L CNN
+F 0 "R1303" V 4950 3650 50  0000 L CNN
+F 1 "10kR" V 5050 3650 50  0000 L CNN
 F 2 "Resistor_SMD:R_0603_1608Metric" V 4980 3750 50  0001 C CNN
 F 3 "~" H 5050 3750 50  0001 C CNN
@@
 AR Path="/5F3042B8/5F6C7B85" Ref="C1302"  Part="1"
 F 0 "C1302" H 7992 3396 50  0000 L CNN
-F 1 "0µ1" H 7992 3305 50  0000 L CNN
+F 1 "0.1uF 3.6VDCbias" H 7992 3305 50  0000 L CNN
 F 2 "Capacitor_SMD:C_0603_1608Metric" H 7900 3350 50  0001 C CNN
 F 3 "~" H 7900 3350 50  0001 C CNN
@@
 AR Path="/5F3042B8/5F6C8975" Ref="C1301"  Part="1"
 F 0 "C1301" H 4992 4546 50  0000 L CNN
-F 1 "0µ1" H 4992 4455 50  0000 L CNN
+F 1 "0.1uF 3.3VDCbias" H 4992 4455 50  0000 L CNN
 F 2 "Capacitor_SMD:C_0603_1608Metric" H 4900 4500 50  0001 C CNN
 F 3 "~" H 4900 4500 50  0001 C CNN

Commit message: gemini-bringup: custom fields for rating constraints on passives
Instead of packing tons of detail into a single "Value" field, limit
"Value" to the primary characteristic of the device (i.e. capacitance
for capacitors, resistance for resistors, current for fuses, impedence
at frequency for ferrite beads). For all other rating constraints, use
custom fields of the form <component-refdes-prefix>_<constraint>. For
example, R_P contains the power a resistor must dissipate.  Use
calculated values when possible rather than standard values as the
intent is to capture the constraint, not a specific device choice.
Parts:
- C1101: value 0.1uF 3.3VDCbias -> 0.1uF; C_Vbias (none) -> 3.3V
- C1102: value 0.1uF 3.6VDCbias -> 0.1uF; C_Vbias (none) -> 3.6V
Other:
- moved on the sheet: R1301, R1302
Changed lines of the file:
@@
 Text HLabel 6850 3800 0    50   Input ~ 0
 ~SMBA
-Text HLabel 4500 3550 0    50   Input ~ 0
+Text HLabel 4700 3550 0    50   Input ~ 0
 SCL
-Text HLabel 4500 3650 0    50   Input ~ 0
+Text HLabel 4700 3650 0    50   Input ~ 0
 SDA
 Wire Wire Line
-	4500 3550 4700 3550
+	4700 3550 4900 3550
 Wire Wire Line
-	4500 3650 4850 3650
+	4700 3650 5050 3650
 $Comp
 L Device:R R1101
 U 1 1 5F2F4AED
-P 4700 3200
+P 4900 3200
 AR Path="/5F2F1B47/5F2F4AED" Ref="R1101"  Part="1"
 AR Path="/5F2F7878/5F2F4AED" Ref="R?"  Part="1"
 AR Path="/5F2FE5B6/5F2F4AED" Ref="R1201"  Part="1"
 AR Path="/5F3042B8/5F2F4AED" Ref="R1301"  Part="1"
-F 0 "R1301" H 4400 3250 50  0000 L CNN
-F 1 "3.3kR" H 4400 3150 50  0000 L CNN
-F 2 "Resistor_SMD:R_0603_1608Metric" V 4630 3200 50  0001 C CNN
-F 3 "~" H 4700 3200 50  0001 C CNN
-F 4 "CR0603-JW-332ELF" H 4700 3200 50  0001 C CNN "Mfg Part Num"
-F 5 "Bourns" H 4700 3200 50  0001 C CNN "Mfg"
-F 6 "232-00018" H 4700 3200 50  0001 C CNN "CPN"
-	1    4700 3200
+F 0 "R1301" V 4850 3300 50  0000 L CNN
+F 1 "3.3kR" V 4900 3150 50  0000 L CNN
+F 2 "Resistor_SMD:R_0603_1608Metric" V 4830 3200 50  0001 C CNN
+F 3 "~" H 4900 3200 50  0001 C CNN
+F 4 "CR0603-JW-332ELF" H 4900 3200 50  0001 C CNN "Mfg Part Num"
+F 5 "Bourns" H 4900 3200 50  0001 C CNN "Mfg"
+F 6 "232-00018" H 4900 3200 50  0001 C CNN "CPN"
+	1    4900 3200
 	1    0    0    -1
 $EndComp
 Wire Wire Line
-	4700 3350 4700 3550
-Connection ~ 4700 3550
+	4900 3350 4900 3550
+Connection ~ 4900 3550
 Wire Wire Line
-	4700 3550 5200 3550
+	4900 3550 5200 3550
 $Comp
 L Device:R R1102
 U 1 1 5F2F511D
-P 4850 3200
+P 5050 3200
 AR Path="/5F2F1B47/5F2F511D" Ref="R1102"  Part="1"
 AR Path="/5F2F7878/5F2F511D" Ref="R?"  Part="1"
 AR Path="/5F2FE5B6/5F2F511D" Ref="R1202"  Part="1"
 AR Path="/5F3042B8/5F2F511D" Ref="R1302"  Part="1"
-F 0 "R1302" H 4950 3250 50  0000 L CNN
-F 1 "3.3kR" H 4950 3150 50  0000 L CNN
-F 2 "Resistor_SMD:R_0603_1608Metric" V 4780 3200 50  0001 C CNN
-F 3 "~" H 4850 3200 50  0001 C CNN
-F 4 "CR0603-JW-332ELF" H 4850 3200 50  0001 C CNN "Mfg Part Num"
-F 5 "Bourns" H 4850 3200 50  0001 C CNN "Mfg"
-F 6 "232-00018" H 4850 3200 50  0001 C CNN "CPN"
-	1    4850 3200
+F 0 "R1302" V 5000 3300 50  0000 L CNN
+F 1 "3.3kR" V 5050 3150 50  0000 L CNN
+F 2 "Resistor_SMD:R_0603_1608Metric" V 4980 3200 50  0001 C CNN
+F 3 "~" H 5050 3200 50  0001 C CNN
+F 4 "CR0603-JW-332ELF" H 5050 3200 50  0001 C CNN "Mfg Part Num"
+F 5 "Bourns" H 5050 3200 50  0001 C CNN "Mfg"
+F 6 "232-00018" H 5050 3200 50  0001 C CNN "CPN"
+	1    5050 3200
 	1    0    0    -1
 $EndComp
 Wire Wire Line
-	4850 3350 4850 3650
-Connection ~ 4850 3650
+	5050 3350 5050 3650
+Connection ~ 5050 3650
 Wire Wire Line
-	4850 3650 5200 3650
+	5050 3650 5200 3650
 Wire Wire Line
-	4850 3050 4850 2950
+	5050 3050 5050 2950
 Wire Wire Line
-	4850 2950 4800 2950
+	5050 2950 5000 2950
 Wire Wire Line
-	4700 2950 4700 3050
+	4900 2950 4900 3050
 $Comp
 L power:+3V3 #PWR01102
 U 1 1 5F2F5A4A
-P 4800 2950
+P 5000 2950
 AR Path="/5F2F1B47/5F2F5A4A" Ref="#PWR01102"  Part="1"
 AR Path="/5F2F7878/5F2F5A4A" Ref="#PWR?"  Part="1"
 AR Path="/5F2FE5B6/5F2F5A4A" Ref="#PWR01202"  Part="1"
 AR Path="/5F3042B8/5F2F5A4A" Ref="#PWR01302"  Part="1"
-F 0 "#PWR01302" H 4800 2800 50  0001 C CNN
-F 1 "+3V3" H 4815 3123 50  0000 C CNN
-F 2 "" H 4800 2950 50  0001 C CNN
-F 3 "" H 4800 2950 50  0001 C CNN
-	1    4800 2950
+F 0 "#PWR01302" H 5000 2800 50  0001 C CNN
+F 1 "+3V3" H 5015 3123 50  0000 C CNN
+F 2 "" H 5000 2950 50  0001 C CNN
+F 3 "" H 5000 2950 50  0001 C CNN
+	1    5000 2950
 	1    0    0    -1
 $EndComp
-Connection ~ 4800 2950
+Connection ~ 5000 2950
 Wire Wire Line
-	4800 2950 4700 2950
+	5000 2950 4900 2950
 Text Notes 6050 3400 0    50   ~ 0
 NO PULLUPS THIS SIDE\nTCA9802 handles it
@@
 AR Path="/5F2FE5B6/600BC5DC" Ref="R1203"  Part="1"
 AR Path="/5F3042B8/600BC5DC" Ref="R1303"  Part="1"
-F 0 "R1303" V 4950 3650 50  0000 L CNN
-F 1 "10kR" V 5050 3650 50  0000 L CNN
+F 0 "R1303" V 5000 3850 50  0000 L CNN
+F 1 "10kR" V 5050 3700 50  0000 L CNN
 F 2 "Resistor_SMD:R_0603_1608Metric" V 4980 3750 50  0001 C CNN
 F 3 "~" H 5050 3750 50  0001 C CNN
@@
 AR Path="/5F3042B8/5F6C7B85" Ref="C1302"  Part="1"
 F 0 "C1302" H 7992 3396 50  0000 L CNN
-F 1 "0.1uF 3.6VDCbias" H 7992 3305 50  0000 L CNN
+F 1 "0.1uF" H 7992 3305 50  0000 L CNN
 F 2 "Capacitor_SMD:C_0603_1608Metric" H 7900 3350 50  0001 C CNN
 F 3 "~" H 7900 3350 50  0001 C CNN
@@
 F 5 "Samsung Electro-Mechanics" H 7900 3350 50  0001 C CNN "Mfg"
 F 6 "212-00011" H 7900 3350 50  0001 C CNN "CPN"
+F 7 "3.6V" H 7900 3350 50  0001 C CNN "C_Vbias"
 	1    7900 3350
 	1    0    0    -1
@@
 AR Path="/5F3042B8/5F6C8975" Ref="C1301"  Part="1"
 F 0 "C1301" H 4992 4546 50  0000 L CNN
-F 1 "0.1uF 3.3VDCbias" H 4992 4455 50  0000 L CNN
+F 1 "0.1uF" H 4992 4455 50  0000 L CNN
 F 2 "Capacitor_SMD:C_0603_1608Metric" H 4900 4500 50  0001 C CNN
 F 3 "~" H 4900 4500 50  0001 C CNN
@@
 F 5 "Samsung Electro-Mechanics" H 4900 4500 50  0001 C CNN "Mfg"
 F 6 "212-00011" H 4900 4500 50  0001 C CNN "CPN"
+F 7 "3.3V" H 4900 4500 50  0001 C CNN "C_Vbias"
 	1    4900 4500
 	1    0    0    -1

Commit message: gemini-bringup: resistor power rating constraints
Parts:
- R1101, R1102: R_P (none) -> 1mW
- R1103: R_P (none) -> 300uW
Changed lines of the file:
@@
 F 5 "Bourns" H 4900 3200 50  0001 C CNN "Mfg"
 F 6 "232-00018" H 4900 3200 50  0001 C CNN "CPN"
+F 7 "1mW" H 4900 3200 50  0001 C CNN "R_P"
 	1    4900 3200
 	1    0    0    -1
@@
 F 5 "Bourns" H 5050 3200 50  0001 C CNN "Mfg"
 F 6 "232-00018" H 5050 3200 50  0001 C CNN "CPN"
+F 7 "1mW" H 5050 3200 50  0001 C CNN "R_P"
 	1    5050 3200
 	1    0    0    -1
@@
 F 5 "Bourns" H 5050 3750 50  0001 C CNN "Mfg"
 F 6 "232-00024" H 5050 3750 50  0001 C CNN "CPN"
+F 7 "300uW" H 5050 3750 50  0001 C CNN "R_P"
 	1    5050 3750
 	0    -1   -1   0

Commit message: gemini-bringup: reselect all caps respecting C/V derating
Parts:
- C1101, C1102: Mfg Samsung Electro-Mechanics -> Kemet; Mfg Part Num CL10B104KB8NNWC -> C0603C104M4RACTU
Changed lines of the file:
@@
 F 2 "Capacitor_SMD:C_0603_1608Metric" H 7900 3350 50  0001 C CNN
 F 3 "~" H 7900 3350 50  0001 C CNN
-F 4 "CL10B104KB8NNWC" H 7900 3350 50  0001 C CNN "Mfg Part Num"
-F 5 "Samsung Electro-Mechanics" H 7900 3350 50  0001 C CNN "Mfg"
+F 4 "C0603C104M4RACTU" H 7900 3350 50  0001 C CNN "Mfg Part Num"
+F 5 "Kemet" H 7900 3350 50  0001 C CNN "Mfg"
 F 6 "212-00011" H 7900 3350 50  0001 C CNN "CPN"
 F 7 "3.6V" H 7900 3350 50  0001 C CNN "C_Vbias"
@@
 F 2 "Capacitor_SMD:C_0603_1608Metric" H 4900 4500 50  0001 C CNN
 F 3 "~" H 4900 4500 50  0001 C CNN
-F 4 "CL10B104KB8NNWC" H 4900 4500 50  0001 C CNN "Mfg Part Num"
-F 5 "Samsung Electro-Mechanics" H 4900 4500 50  0001 C CNN "Mfg"
+F 4 "C0603C104M4RACTU" H 4900 4500 50  0001 C CNN "Mfg Part Num"
+F 5 "Kemet" H 4900 4500 50  0001 C CNN "Mfg"
 F 6 "212-00011" H 4900 4500 50  0001 C CNN "CPN"
 F 7 "3.3V" H 4900 4500 50  0001 C CNN "C_Vbias"
