File: power.sch (KiCad schematic (older format))
At the start: 15 parts, among them J601 Barrel_Jack, U601 OKI-78SR-3.3_1.5-W36-C, U602 INA219AxDCN, U603 INA219AxDCN

Commit message: 22uF bulk caps on power outputs.
fixes #9
Parts:
- added C605, C606: 22µ 16V, Capacitor_SMD:C_0805_2012Metric, symbol Device:C_Small
Connections:
- net GND: now also C605.2, C606.2
- net at F601.1, R603.4: now also C606.1
- net at R604.4, U601.3 (OUT): now also C605.1
Other:
- moved on the sheet: U601
Changed lines of the file:
@@
 L power:+12V #PWR0604
 U 1 1 5F3CD544
-P 3500 2100
-F 0 "#PWR0604" H 3500 1950 50  0001 C CNN
-F 1 "+12V" H 3515 2273 50  0000 C CNN
-F 2 "" H 3500 2100 50  0001 C CNN
-F 3 "" H 3500 2100 50  0001 C CNN
-	1    3500 2100
+P 3800 2100
+F 0 "#PWR0604" H 3800 1950 50  0001 C CNN
+F 1 "+12V" H 3815 2273 50  0000 C CNN
+F 2 "" H 3800 2100 50  0001 C CNN
+F 3 "" H 3800 2100 50  0001 C CNN
+	1    3800 2100
 	1    0    0    -1
 $EndComp
@@
 L Converter_DCDC:OKI-78SR-3.3_1.5-W36-C U601
 U 1 1 5F3CE73F
-P 2250 3850
-F 0 "U601" H 2250 4092 50  0000 C CNN
-F 1 "OKI-78SR-3.3_1.5-W36-C" H 2250 4001 50  0000 C CNN
-F 2 "Converter_DCDC:Converter_DCDC_muRata_OKI-78SR_Vertical" H 2300 3600 50  0001 L CIN
-F 3 "https://power.murata.com/data/power/oki-78sr.pdf" H 2250 3850 50  0001 C CNN
-	1    2250 3850
+P 1900 3850
+F 0 "U601" H 1900 4092 50  0000 C CNN
+F 1 "OKI-78SR-3.3_1.5-W36-C" H 1900 4001 50  0000 C CNN
+F 2 "Converter_DCDC:Converter_DCDC_muRata_OKI-78SR_Vertical" H 1950 3600 50  0001 L CIN
+F 3 "https://power.murata.com/data/power/oki-78sr.pdf" H 1900 3850 50  0001 C CNN
+	1    1900 3850
 	1    0    0    -1
 $EndComp
@@
 L power:+12V #PWR0602
 U 1 1 5F3CF10D
-P 1950 3850
-F 0 "#PWR0602" H 1950 3700 50  0001 C CNN
-F 1 "+12V" V 1965 3978 50  0000 L CNN
-F 2 "" H 1950 3850 50  0001 C CNN
-F 3 "" H 1950 3850 50  0001 C CNN
-	1    1950 3850
+P 1600 3850
+F 0 "#PWR0602" H 1600 3700 50  0001 C CNN
+F 1 "+12V" V 1615 3978 50  0000 L CNN
+F 2 "" H 1600 3850 50  0001 C CNN
+F 3 "" H 1600 3850 50  0001 C CNN
+	1    1600 3850
 	0    -1   -1   0
 $EndComp
@@
 L power:+3V3 #PWR0605
 U 1 1 5F3CF3DE
-P 3500 3850
-F 0 "#PWR0605" H 3500 3700 50  0001 C CNN
-F 1 "+3V3" V 3515 3978 50  0000 L CNN
-F 2 "" H 3500 3850 50  0001 C CNN
-F 3 "" H 3500 3850 50  0001 C CNN
-	1    3500 3850
+P 4300 3850
+F 0 "#PWR0605" H 4300 3700 50  0001 C CNN
+F 1 "+3V3" V 4315 3978 50  0000 L CNN
+F 2 "" H 4300 3850 50  0001 C CNN
+F 3 "" H 4300 3850 50  0001 C CNN
+	1    4300 3850
 	0    1    1    0
 $EndComp
@@
 L power:GND #PWR0603
 U 1 1 5F3CF71D
-P 2250 4150
-F 0 "#PWR0603" H 2250 3900 50  0001 C CNN
-F 1 "GND" H 2255 3977 50  0000 C CNN
-F 2 "" H 2250 4150 50  0001 C CNN
-F 3 "" H 2250 4150 50  0001 C CNN
-	1    2250 4150
+P 1900 4150
+F 0 "#PWR0603" H 1900 3900 50  0001 C CNN
+F 1 "GND" H 1905 3977 50  0000 C CNN
+F 2 "" H 1900 4150 50  0001 C CNN
+F 3 "" H 1900 4150 50  0001 C CNN
+	1    1900 4150
 	1    0    0    -1
 $EndComp
@@
 L power:PWR_FLAG #FLG0602
 U 1 1 600BF38A
-P 3500 2100
-F 0 "#FLG0602" H 3500 2175 50  0001 C CNN
-F 1 "PWR_FLAG" V 3500 2228 50  0000 L CNN
-F 2 "" H 3500 2100 50  0001 C CNN
-F 3 "~" H 3500 2100 50  0001 C CNN
-	1    3500 2100
+P 3800 2100
+F 0 "#FLG0602" H 3800 2175 50  0001 C CNN
+F 1 "PWR_FLAG" V 3800 2228 50  0000 L CNN
+F 2 "" H 3800 2100 50  0001 C CNN
+F 3 "~" H 3800 2100 50  0001 C CNN
+	1    3800 2100
 	0    1    1    0
 $EndComp
@@
 L power:PWR_FLAG #FLG0603
 U 1 1 600BF66D
-P 3500 3850
-F 0 "#FLG0603" H 3500 3925 50  0001 C CNN
-F 1 "PWR_FLAG" H 3500 4023 50  0000 C CNN
-F 2 "" H 3500 3850 50  0001 C CNN
-F 3 "~" H 3500 3850 50  0001 C CNN
-	1    3500 3850
-	1    0    0    -1
-$EndComp
-Connection ~ 3500 3850
+P 4300 3850
+F 0 "#FLG0603" H 4300 3925 50  0001 C CNN
+F 1 "PWR_FLAG" H 4300 4023 50  0000 C CNN
+F 2 "" H 4300 3850 50  0001 C CNN
+F 3 "~" H 4300 3850 50  0001 C CNN
+	1    4300 3850
+	1    0    0    -1
+$EndComp
+Connection ~ 4300 3850
 $Comp
 L power:PWR_FLAG #FLG0601
@@
 Connection ~ 1900 2300
 Wire Wire Line
-	2950 2100 2350 2100
+	2950 2100 2450 2100
 Wire Wire Line
 	3050 2250 2900 2250
-Wire Wire Line
-	3350 2100 3500 2100
-Connection ~ 3500 2100
+Connection ~ 3800 2100
 Wire Wire Line
 	3250 2250 3400 2250
@@
 $EndComp
 Wire Wire Line
-	2550 3850 2950 3850
-Wire Wire Line
-	3350 3850 3500 3850
+	2200 3850 2300 3850
 Wire Wire Line
 	3400 4000 3250 4000
@@
 Connection ~ 3400 4400
 NoConn ~ 1650 2200
+$Comp
+L Device:C_Small C606
+U 1 1 5F918180
+P 2450 2200
+F 0 "C606" H 2542 2246 50  0000 L CNN
+F 1 "22µ 16V" H 2542 2155 50  0000 L CNN
+F 2 "Capacitor_SMD:C_0805_2012Metric" H 2450 2200 50  0001 C CNN
+F 3 "~" H 2450 2200 50  0001 C CNN
+	1    2450 2200
+	1    0    0    -1
+$EndComp
+$Comp
+L power:GND #PWR0612
+U 1 1 5F918467
+P 2450 2300
+F 0 "#PWR0612" H 2450 2050 50  0001 C CNN
+F 1 "GND" H 2455 2127 50  0000 C CNN
+F 2 "" H 2450 2300 50  0001 C CNN
+F 3 "" H 2450 2300 50  0001 C CNN
+	1    2450 2300
+	1    0    0    -1
+$EndComp
+$Comp
+L Device:C_Small C605
+U 1 1 5F91AE04
+P 2300 3950
+F 0 "C605" H 2392 3996 50  0000 L CNN
+F 1 "22µ 16V" H 2392 3905 50  0000 L CNN
+F 2 "Capacitor_SMD:C_0805_2012Metric" H 2300 3950 50  0001 C CNN
+F 3 "~" H 2300 3950 50  0001 C CNN
+	1    2300 3950
+	1    0    0    -1
+$EndComp
+$Comp
+L power:GND #PWR0611
+U 1 1 5F91AE0A
+P 2300 4050
+F 0 "#PWR0611" H 2300 3800 50  0001 C CNN
+F 1 "GND" H 2305 3877 50  0000 C CNN
+F 2 "" H 2300 4050 50  0001 C CNN
+F 3 "" H 2300 4050 50  0001 C CNN
+	1    2300 4050
+	1    0    0    -1
+$EndComp
+Connection ~ 2300 3850
+Wire Wire Line
+	2300 3850 2950 3850
+Wire Wire Line
+	3350 3850 4300 3850
+Connection ~ 2450 2100
+Wire Wire Line
+	2450 2100 2350 2100
+Wire Wire Line
+	3350 2100 3800 2100
 $EndSCHEMATC

Commit message: PCB: route power area
Parts:
- F601: footprint Fuse:Fuse_0603_1608Metric -> Fuse:Fuse_1812_4532Metric
- R603, R604: footprint Resistor_SMD:R_Shunt_Ohmite_LVK12 -> passives:R_Shunt_Ohmite_LVK12_CW_Pinout
Connections:
- net +12V: now also R603.4; no longer R603.1
- net +3V3: now also R604.4; no longer R604.1
- net at R603.2: now also R601.1; no longer R605.1
- net at R603.3: now also R605.1; no longer R601.1
- net at C606.1, F601.1: now also R603.1; no longer R603.4
- net at C605.1, U601.3 (OUT): now also R604.1; no longer R604.4
- net at R604.2: now also R602.1; no longer R606.1
- net at R604.3: now also R606.1; no longer R602.1
Changed lines of the file:
@@
 F 0 "R603" V 2943 2100 50  0000 C CNN
 F 1 "20m 1% 1/8W" V 3034 2100 50  0000 C CNN
-F 2 "Resistor_SMD:R_Shunt_Ohmite_LVK12" V 3080 2100 50  0001 C CNN
+F 2 "passives:R_Shunt_Ohmite_LVK12_CW_Pinout" V 3080 2100 50  0001 C CNN
 F 3 "~" H 3150 2100 50  0001 C CNN
 	1    3150 2100
-	0    1    1    0
+	0    -1   1    0
 $EndComp
 Wire Wire Line
@@
 F 0 "R604" V 2943 3850 50  0000 C CNN
 F 1 "40m 1% 1/8W" V 3034 3850 50  0000 C CNN
-F 2 "Resistor_SMD:R_Shunt_Ohmite_LVK12" V 3080 3850 50  0001 C CNN
+F 2 "passives:R_Shunt_Ohmite_LVK12_CW_Pinout" V 3080 3850 50  0001 C CNN
 F 3 "~" H 3150 3850 50  0001 C CNN
 	1    3150 3850
-	0    1    1    0
+	0    -1   1    0
 $EndComp
 $Comp
@@
 F 0 "F601" V 2045 2100 50  0000 C CNN
 F 1 "Polyfuse_Small" V 2136 2100 50  0000 C CNN
-F 2 "Fuse:Fuse_0603_1608Metric" H 2300 1900 50  0001 L CNN
+F 2 "Fuse:Fuse_1812_4532Metric" H 2300 1900 50  0001 L CNN
 F 3 "~" H 2250 2100 50  0001 C CNN
 	1    2250 2100

Commit message: MB: annotate everything with mfg/MPN
Parts:
- C601, C602, C603, C604, C605, C606, R601, R602, R605, R606: Mfg Part Num (none) -> generic
- F601: value Polyfuse_Small -> TBD; Mfg Part Num (none) -> generic
- J601: Mfg (none) -> Cliff Electronic Components; Mfg Part Num (none) -> FC681465S
- R603: Mfg (none) -> Ohmite; Mfg Part Num (none) -> LVK12R020FER
- R604: Mfg (none) -> Ohmite; Mfg Part Num (none) -> LVK12R040FER
- U601: Mfg (none) -> Murata; Mfg Part Num (none) -> OKI-78SR-3.3_1.5-W36-C
- U602, U603: Mfg (none) -> Texas Instruments; Mfg Part Num (none) -> INA219AIDCNT
Changed lines of the file:
@@
 F 2 "Connector_BarrelJack:BarrelJack_CLIFF_FC681465S_SMT_Horizontal" H 1400 2160 50  0001 C CNN
 F 3 "~" H 1400 2160 50  0001 C CNN
+F 4 "Cliff Electronic Components" H 1350 2200 50  0001 C CNN "Mfg"
+F 5 "FC681465S" H 1350 2200 50  0001 C CNN "Mfg Part Num"
 	1    1350 2200
 	1    0    0    -1
@@
 F 2 "passives:R_Shunt_Ohmite_LVK12_CW_Pinout" V 3080 2100 50  0001 C CNN
 F 3 "~" H 3150 2100 50  0001 C CNN
+F 4 "Ohmite" H 3150 2100 50  0001 C CNN "Mfg"
+F 5 "LVK12R020FER" H 3150 2100 50  0001 C CNN "Mfg Part Num"
 	1    3150 2100
 	0    -1   1    0
@@
 F 2 "Package_TO_SOT_SMD:SOT-23-8" H 4600 2750 50  0001 C CNN
 F 3 "http://www.ti.com/lit/ds/symlink/ina219.pdf" H 4300 3000 50  0001 C CNN
+F 4 "Texas Instruments" H 3950 3100 50  0001 C CNN "Mfg"
+F 5 "INA219AIDCNT" H 3950 3100 50  0001 C CNN "Mfg Part Num"
 	1    3950 3100
 	1    0    0    -1
@@
 F 2 "Resistor_SMD:R_0603_1608Metric" V 2830 2400 50  0001 C CNN
 F 3 "~" H 2900 2400 50  0001 C CNN
+F 4 "generic" H 2900 2400 50  0001 C CNN "Mfg Part Num"
 	1    2900 2400
 	1    0    0    -1
@@
 F 2 "Resistor_SMD:R_0603_1608Metric" V 3330 2400 50  0001 C CNN
 F 3 "~" H 3400 2400 50  0001 C CNN
+F 4 "generic" H 3400 2400 50  0001 C CNN "Mfg Part Num"
 	1    3400 2400
 	1    0    0    -1
@@
 F 2 "Capacitor_SMD:C_0603_1608Metric" H 3150 2650 50  0001 C CNN
 F 3 "~" H 3150 2650 50  0001 C CNN
+F 4 "generic" H 3150 2650 50  0001 C CNN "Mfg Part Num"
 	1    3150 2650
 	0    1    1    0
@@
 F 2 "Capacitor_SMD:C_0603_1608Metric" H 4450 2700 50  0001 C CNN
 F 3 "~" H 4450 2700 50  0001 C CNN
+F 4 "generic" H 4450 2700 50  0001 C CNN "Mfg Part Num"
 	1    4450 2700
 	-1   0    0    1
@@
 F 2 "Converter_DCDC:Converter_DCDC_muRata_OKI-78SR_Vertical" H 1950 3600 50  0001 L CIN
 F 3 "https://power.murata.com/data/power/oki-78sr.pdf" H 1900 3850 50  0001 C CNN
+F 4 "Murata" H 1900 3850 50  0001 C CNN "Mfg"
+F 5 "OKI-78SR-3.3_1.5-W36-C" H 1900 3850 50  0001 C CNN "Mfg Part Num"
 	1    1900 3850
 	1    0    0    -1
@@
 F 2 "passives:R_Shunt_Ohmite_LVK12_CW_Pinout" V 3080 3850 50  0001 C CNN
 F 3 "~" H 3150 3850 50  0001 C CNN
+F 4 "Ohmite" H 3150 3850 50  0001 C CNN "Mfg"
+F 5 "LVK12R040FER" H 3150 3850 50  0001 C CNN "Mfg Part Num"
 	1    3150 3850
 	0    -1   1    0
@@
 F 2 "Package_TO_SOT_SMD:SOT-23-8" H 4600 4500 50  0001 C CNN
 F 3 "http://www.ti.com/lit/ds/symlink/ina219.pdf" H 4300 4750 50  0001 C CNN
+F 4 "Texas Instruments" H 3950 4850 50  0001 C CNN "Mfg"
+F 5 "INA219AIDCNT" H 3950 4850 50  0001 C CNN "Mfg Part Num"
 	1    3950 4850
 	1    0    0    -1
@@
 F 2 "Resistor_SMD:R_0603_1608Metric" V 2830 4150 50  0001 C CNN
 F 3 "~" H 2900 4150 50  0001 C CNN
+F 4 "generic" H 2900 4150 50  0001 C CNN "Mfg Part Num"
 	1    2900 4150
 	1    0    0    -1
@@
 F 2 "Resistor_SMD:R_0603_1608Metric" V 3330 4150 50  0001 C CNN
 F 3 "~" H 3400 4150 50  0001 C CNN
+F 4 "generic" H 3400 4150 50  0001 C CNN "Mfg Part Num"
 	1    3400 4150
 	1    0    0    -1
@@
 F 2 "Capacitor_SMD:C_0603_1608Metric" H 4450 4450 50  0001 C CNN
 F 3 "~" H 4450 4450 50  0001 C CNN
+F 4 "generic" H 4450 4450 50  0001 C CNN "Mfg Part Num"
 	1    4450 4450
 	-1   0    0    1
@@
 P 2250 2100
 F 0 "F601" V 2045 2100 50  0000 C CNN
-F 1 "Polyfuse_Small" V 2136 2100 50  0000 C CNN
+F 1 "TBD" V 2136 2100 50  0000 C CNN
 F 2 "Fuse:Fuse_1812_4532Metric" H 2300 1900 50  0001 L CNN
 F 3 "~" H 2250 2100 50  0001 C CNN
+F 4 "generic" H 2250 2100 50  0001 C CNN "Mfg Part Num"
 	1    2250 2100
 	0    1    1    0
@@
 F 2 "Capacitor_SMD:C_0603_1608Metric" H 3150 4400 50  0001 C CNN
 F 3 "~" H 3150 4400 50  0001 C CNN
+F 4 "generic" H 3150 4400 50  0001 C CNN "Mfg Part Num"
 	1    3150 4400
 	0    1    1    0
@@
 F 2 "Capacitor_SMD:C_0805_2012Metric" H 2450 2200 50  0001 C CNN
 F 3 "~" H 2450 2200 50  0001 C CNN
+F 4 "generic" H 2450 2200 50  0001 C CNN "Mfg Part Num"
 	1    2450 2200
 	1    0    0    -1
@@
 F 2 "Capacitor_SMD:C_0805_2012Metric" H 2300 3950 50  0001 C CNN
 F 3 "~" H 2300 3950 50  0001 C CNN
+F 4 "generic" H 2300 3950 50  0001 C CNN "Mfg Part Num"
 	1    2300 3950
 	1    0    0    -1

Commit message: MB: MPNs for capacitors, adjust some footprints
Can't get a 2kV 10000p cap in 0603 as it turns out
Parts:
- C603, C604: Mfg (none) -> Samsung Electro-Mechanics; Mfg Part Num generic -> CL10B104KB8NNWC
- C605, C606: Mfg (none) -> Samsung Electro-Mechanics; Mfg Part Num generic -> CL10A226MO7JZNC
Changed lines of the file:
@@
 F 2 "Capacitor_SMD:C_0603_1608Metric" H 4450 2700 50  0001 C CNN
 F 3 "~" H 4450 2700 50  0001 C CNN
-F 4 "generic" H 4450 2700 50  0001 C CNN "Mfg Part Num"
+F 4 "CL10B104KB8NNWC" H 4450 2700 50  0001 C CNN "Mfg Part Num"
+F 5 "Samsung Electro-Mechanics" H 4450 2700 50  0001 C CNN "Mfg"
 	1    4450 2700
 	-1   0    0    1
@@
 F 2 "Capacitor_SMD:C_0603_1608Metric" H 4450 4450 50  0001 C CNN
 F 3 "~" H 4450 4450 50  0001 C CNN
-F 4 "generic" H 4450 4450 50  0001 C CNN "Mfg Part Num"
+F 4 "CL10B104KB8NNWC" H 4450 4450 50  0001 C CNN "Mfg Part Num"
+F 5 "Samsung Electro-Mechanics" H 4450 4450 50  0001 C CNN "Mfg"
 	1    4450 4450
 	-1   0    0    1
@@
 F 2 "Capacitor_SMD:C_0805_2012Metric" H 2450 2200 50  0001 C CNN
 F 3 "~" H 2450 2200 50  0001 C CNN
-F 4 "generic" H 2450 2200 50  0001 C CNN "Mfg Part Num"
+F 4 "CL10A226MO7JZNC" H 2450 2200 50  0001 C CNN "Mfg Part Num"
+F 5 "Samsung Electro-Mechanics" H 2450 2200 50  0001 C CNN "Mfg"
 	1    2450 2200
 	1    0    0    -1
@@
 F 2 "Capacitor_SMD:C_0805_2012Metric" H 2300 3950 50  0001 C CNN
 F 3 "~" H 2300 3950 50  0001 C CNN
-F 4 "generic" H 2300 3950 50  0001 C CNN "Mfg Part Num"
+F 4 "CL10A226MO7JZNC" H 2300 3950 50  0001 C CNN "Mfg Part Num"
+F 5 "Samsung Electro-Mechanics" H 2300 3950 50  0001 C CNN "Mfg"
 	1    2300 3950
 	1    0    0    -1

Commit message: MB: assign ferrites'n'fuses
Parts:
- F601: value TBD -> 16V 2A PTC; Mfg (none) -> Littelfuse Inc; Mfg Part Num generic -> 1812L200/16DR
Changed lines of the file:
@@
 P 2250 2100
 F 0 "F601" V 2045 2100 50  0000 C CNN
-F 1 "TBD" V 2136 2100 50  0000 C CNN
+F 1 "16V 2A PTC" V 2136 2100 50  0000 C CNN
 F 2 "Fuse:Fuse_1812_4532Metric" H 2300 1900 50  0001 L CNN
 F 3 "~" H 2250 2100 50  0001 C CNN
-F 4 "generic" H 2250 2100 50  0001 C CNN "Mfg Part Num"
+F 4 "1812L200/16DR" H 2250 2100 50  0001 C CNN "Mfg Part Num"
+F 5 "Littelfuse Inc" H 2250 2100 50  0001 C CNN "Mfg"
 	1    2250 2100
 	0    1    1    0

Commit message: MB: assign single resistors
Parts:
- R601, R602, R605, R606: Mfg (none) -> Bourns; Mfg Part Num generic -> CR0603-J/-000ELF
Changed lines of the file:
@@
 F 2 "Resistor_SMD:R_0603_1608Metric" V 2830 2400 50  0001 C CNN
 F 3 "~" H 2900 2400 50  0001 C CNN
-F 4 "generic" H 2900 2400 50  0001 C CNN "Mfg Part Num"
+F 4 "CR0603-J/-000ELF" H 2900 2400 50  0001 C CNN "Mfg Part Num"
+F 5 "Bourns" H 2900 2400 50  0001 C CNN "Mfg"
 	1    2900 2400
 	1    0    0    -1
@@
 F 2 "Resistor_SMD:R_0603_1608Metric" V 3330 2400 50  0001 C CNN
 F 3 "~" H 3400 2400 50  0001 C CNN
-F 4 "generic" H 3400 2400 50  0001 C CNN "Mfg Part Num"
+F 4 "CR0603-J/-000ELF" H 3400 2400 50  0001 C CNN "Mfg Part Num"
+F 5 "Bourns" H 3400 2400 50  0001 C CNN "Mfg"
 	1    3400 2400
 	1    0    0    -1
@@
 F 2 "Resistor_SMD:R_0603_1608Metric" V 2830 4150 50  0001 C CNN
 F 3 "~" H 2900 4150 50  0001 C CNN
-F 4 "generic" H 2900 4150 50  0001 C CNN "Mfg Part Num"
+F 4 "CR0603-J/-000ELF" H 2900 4150 50  0001 C CNN "Mfg Part Num"
+F 5 "Bourns" H 2900 4150 50  0001 C CNN "Mfg"
 	1    2900 4150
 	1    0    0    -1
@@
 F 2 "Resistor_SMD:R_0603_1608Metric" V 3330 4150 50  0001 C CNN
 F 3 "~" H 3400 4150 50  0001 C CNN
-F 4 "generic" H 3400 4150 50  0001 C CNN "Mfg Part Num"
+F 4 "CR0603-J/-000ELF" H 3400 4150 50  0001 C CNN "Mfg Part Num"
+F 5 "Bourns" H 3400 4150 50  0001 C CNN "Mfg"
 	1    3400 4150
 	1    0    0    -1
