File: power.sch (KiCad schematic (older format))
At the start: 17 parts, among them J601 Barrel_Jack, U601 OKI-78SR-3.3_1.5-W36-C, U602 INA219AxDCN, U603 INA219AxDCN

Commit message: MB: improve 3v3 and INA219 routing.
Per review comments from Mark.
Connections:
- net +3V3: now also R604.1; no longer R604.4
- net at C605.1, U601.3 (OUT): now also R604.4; no longer R604.1
- net at R604.2: now also R606.1; no longer R602.1
- net at R604.3: now also R602.1; no longer R606.1
Changed lines of the file:
@@
 F 5 "LVK12R040FER" H 3150 3850 50  0001 C CNN "Mfg Part Num"
 	1    3150 3850
-	0    -1   1    0
+	0    1    1    0
 $EndComp
 $Comp

Commit message: power: replace 40mOhm shunt with 47mOhm as former doesn't exist in LVK12R series
Parts:
- R604: value 40m 1% 1/8W -> 47m 1% 1/8W; Mfg Part Num LVK12R040FER -> LVK12R047FER
Changed lines of the file:
@@
 P 3150 3850
 F 0 "R604" V 2943 3850 50  0000 C CNN
-F 1 "40m 1% 1/8W" V 3034 3850 50  0000 C CNN
+F 1 "47m 1% 1/8W" V 3034 3850 50  0000 C CNN
 F 2 "passives:R_Shunt_Ohmite_LVK12_CW_Pinout" V 3080 3850 50  0001 C CNN
 F 3 "~" H 3150 3850 50  0001 C CNN
 F 4 "Ohmite" H 3150 3850 50  0001 C CNN "Mfg"
-F 5 "LVK12R040FER" H 3150 3850 50  0001 C CNN "Mfg Part Num"
+F 5 "LVK12R047FER" H 3150 3850 50  0001 C CNN "Mfg Part Num"
 	1    3150 3850
 	0    1    1    0

Commit message: MB: replace power jack with one we can, like, buy
Parts:
- J601: footprint Connector_BarrelJack:BarrelJack_CLIFF_FC681465S_SMT_Horizontal -> Connector_BarrelJack:BarrelJack_CUI_PJ-036AH-SMT_Horizontal; Mfg Cliff Electronic Components -> CUI Devices; Mfg Part Num FC681465S -> PJ-036AH-SMT-TR
Changed lines of the file:
@@
 F 0 "J601" H 1407 2525 50  0000 C CNN
 F 1 "Barrel_Jack" H 1407 2434 50  0000 C CNN
-F 2 "Connector_BarrelJack:BarrelJack_CLIFF_FC681465S_SMT_Horizontal" H 1400 2160 50  0001 C CNN
+F 2 "Connector_BarrelJack:BarrelJack_CUI_PJ-036AH-SMT_Horizontal" H 1400 2160 50  0001 C CNN
 F 3 "~" H 1400 2160 50  0001 C CNN
-F 4 "Cliff Electronic Components" H 1350 2200 50  0001 C CNN "Mfg"
-F 5 "FC681465S" H 1350 2200 50  0001 C CNN "Mfg Part Num"
+F 4 "CUI Devices" H 1350 2200 50  0001 C CNN "Mfg"
+F 5 "PJ-036AH-SMT-TR" H 1350 2200 50  0001 C CNN "Mfg Part Num"
 	1    1350 2200
 	1    0    0    -1

Commit message: gemini-bringup: Add CPNs for all components
Parts:
- C603, C604: CPN (none) -> 212-00011
- C605, C606: CPN (none) -> 212-00020
- F601: CPN (none) -> 219-00002
- J601: CPN (none) -> 215-00037
- R601, R602, R605, R606: CPN (none) -> 232-00025
- R603: CPN (none) -> 232-00031
- R604: CPN (none) -> 232-00032
- U601: CPN (none) -> 229-00003
- U602, U603: CPN (none) -> 221-00015
Changed lines of the file:
@@
 F 4 "CUI Devices" H 1350 2200 50  0001 C CNN "Mfg"
 F 5 "PJ-036AH-SMT-TR" H 1350 2200 50  0001 C CNN "Mfg Part Num"
+F 6 "215-00037" H 1350 2200 50  0001 C CNN "CPN"
 	1    1350 2200
 	1    0    0    -1
@@
 F 4 "Ohmite" H 3150 2100 50  0001 C CNN "Mfg"
 F 5 "LVK12R020FER" H 3150 2100 50  0001 C CNN "Mfg Part Num"
+F 6 "232-00031" H 3150 2100 50  0001 C CNN "CPN"
 	1    3150 2100
 	0    -1   1    0
@@
 F 4 "Texas Instruments" H 3950 3100 50  0001 C CNN "Mfg"
 F 5 "INA219AIDCNT" H 3950 3100 50  0001 C CNN "Mfg Part Num"
+F 6 "221-00015" H 3950 3100 50  0001 C CNN "CPN"
 	1    3950 3100
 	1    0    0    -1
@@
 F 4 "CR0603-J/-000ELF" H 2900 2400 50  0001 C CNN "Mfg Part Num"
 F 5 "Bourns" H 2900 2400 50  0001 C CNN "Mfg"
+F 6 "232-00025" H 2900 2400 50  0001 C CNN "CPN"
 	1    2900 2400
 	1    0    0    -1
@@
 F 4 "CR0603-J/-000ELF" H 3400 2400 50  0001 C CNN "Mfg Part Num"
 F 5 "Bourns" H 3400 2400 50  0001 C CNN "Mfg"
+F 6 "232-00025" H 3400 2400 50  0001 C CNN "CPN"
 	1    3400 2400
 	1    0    0    -1
@@
 F 4 "CL10B104KB8NNWC" H 4450 2700 50  0001 C CNN "Mfg Part Num"
 F 5 "Samsung Electro-Mechanics" H 4450 2700 50  0001 C CNN "Mfg"
+F 6 "212-00011" H 4450 2700 50  0001 C CNN "CPN"
 	1    4450 2700
 	-1   0    0    1
@@
 F 4 "Murata" H 1900 3850 50  0001 C CNN "Mfg"
 F 5 "OKI-78SR-3.3_1.5-W36-C" H 1900 3850 50  0001 C CNN "Mfg Part Num"
+F 6 "229-00003" H 1900 3850 50  0001 C CNN "CPN"
 	1    1900 3850
 	1    0    0    -1
@@
 F 4 "Ohmite" H 3150 3850 50  0001 C CNN "Mfg"
 F 5 "LVK12R047FER" H 3150 3850 50  0001 C CNN "Mfg Part Num"
+F 6 "232-00032" H 3150 3850 50  0001 C CNN "CPN"
 	1    3150 3850
 	0    1    1    0
@@
 F 4 "Texas Instruments" H 3950 4850 50  0001 C CNN "Mfg"
 F 5 "INA219AIDCNT" H 3950 4850 50  0001 C CNN "Mfg Part Num"
+F 6 "221-00015" H 3950 4850 50  0001 C CNN "CPN"
 	1    3950 4850
 	1    0    0    -1
@@
 F 4 "CR0603-J/-000ELF" H 2900 4150 50  0001 C CNN "Mfg Part Num"
 F 5 "Bourns" H 2900 4150 50  0001 C CNN "Mfg"
+F 6 "232-00025" H 2900 4150 50  0001 C CNN "CPN"
 	1    2900 4150
 	1    0    0    -1
@@
 F 4 "CR0603-J/-000ELF" H 3400 4150 50  0001 C CNN "Mfg Part Num"
 F 5 "Bourns" H 3400 4150 50  0001 C CNN "Mfg"
+F 6 "232-00025" H 3400 4150 50  0001 C CNN "CPN"
 	1    3400 4150
 	1    0    0    -1
@@
 F 4 "CL10B104KB8NNWC" H 4450 4450 50  0001 C CNN "Mfg Part Num"
 F 5 "Samsung Electro-Mechanics" H 4450 4450 50  0001 C CNN "Mfg"
+F 6 "212-00011" H 4450 4450 50  0001 C CNN "CPN"
 	1    4450 4450
 	-1   0    0    1
@@
 F 4 "1812L200/16DR" H 2250 2100 50  0001 C CNN "Mfg Part Num"
 F 5 "Littelfuse Inc" H 2250 2100 50  0001 C CNN "Mfg"
+F 6 "219-00002" H 2250 2100 50  0001 C CNN "CPN"
 	1    2250 2100
 	0    1    1    0
@@
 F 4 "CL10A226MO7JZNC" H 2450 2200 50  0001 C CNN "Mfg Part Num"
 F 5 "Samsung Electro-Mechanics" H 2450 2200 50  0001 C CNN "Mfg"
+F 6 "212-00020" H 2450 2200 50  0001 C CNN "CPN"
 	1    2450 2200
 	1    0    0    -1
@@
 F 4 "CL10A226MO7JZNC" H 2300 3950 50  0001 C CNN "Mfg Part Num"
 F 5 "Samsung Electro-Mechanics" H 2300 3950 50  0001 C CNN "Mfg"
+F 6 "212-00020" H 2300 3950 50  0001 C CNN "CPN"
 	1    2300 3950
 	1    0    0    -1

Commit message: gemini-bringup: Mark DNP (do not populate) in a Config field rather than value to match KiBOM expectations
Parts:
- C601, C602: Config (none) -> DNP
Changed lines of the file:
@@
 F 3 "~" H 3150 2650 50  0001 C CNN
 F 4 "generic" H 3150 2650 50  0001 C CNN "Mfg Part Num"
+F 5 "DNP" H 3150 2650 50  0001 C CNN "Config"
 	1    3150 2650
 	0    1    1    0
@@
 F 3 "~" H 3150 4400 50  0001 C CNN
 F 4 "generic" H 3150 4400 50  0001 C CNN "Mfg Part Num"
+F 5 "DNP" H 3150 4400 50  0001 C CNN "Config"
 	1    3150 4400
 	0    1    1    0

Commit message: power: Use correct pinout for CUI PJ-036AH-SMT barrel jack
Per datasheet, pin 2 is ring.
Parts:
- J601: symbol Connector:Barrel_Jack_Switch_Pin3Ring -> Connector:Barrel_Jack_Switch
Connections:
- net GND: now also J601.2; no longer J601.3
Changed lines of the file:
@@
 $EndDescr
 $Comp
-L Connector:Barrel_Jack_Switch_Pin3Ring J601
+L Connector:Barrel_Jack_Switch J601
 U 1 1 5F3C5136
 P 1350 2200

Commit message: power: specify rating constraints on passives
Parts:
- C603, C604: value 0µ1 -> 0.1uF 3.3VDCbias
- C605: value 22µ 16V -> 22uF 3.3VDCbias
- C606: value 22µ 16V -> 22µ 12VDCbias
- R603: value 20m 1% 1/8W -> 20mR 1% 80mW
- R604: value 47m 1% 1/8W -> 47mR 1% 50mW
Other:
- note added: "Nominal load: 100mA\nMax load: 1A\nVshunt @ nominal load: 4.7mV\nVshunt @ max load: 47mV\nCurrent LSB: 250µA"
- note added: "Nominal load: 1A\nMax load: 2A\nVshunt @ nominal load: 20mV\nVshunt @ max load: 40mV\nCurrent LSB: 500µA"
- note removed: "Nominal load: 100mA\nMax load: 1A\nVshunt: 40mV\nCurrent LSB: 250µA"
- note removed: "Nominal load: 1A\nMax load: 2A\nVshunt: 40mV\nCurrent LSB: 500µA"
- moved on the sheet: C605, C606, F601, J601, U601

Commit message: gemini-bringup: custom fields for rating constraints on passives
Instead of packing tons of detail into a single "Value" field, limit
"Value" to the primary characteristic of the device (i.e. capacitance
for capacitors, resistance for resistors, current for fuses, impedence
at frequency for ferrite beads). For all other rating constraints, use
custom fields of the form <component-refdes-prefix>_<constraint>. For
example, R_P contains the power a resistor must dissipate.  Use
calculated values when possible rather than standard values as the
intent is to capture the constraint, not a specific device choice.
Parts:
- C603, C604: value 0.1uF 3.3VDCbias -> 0.1uF; C_Vbias (none) -> 3.3V
- C605: value 22uF 3.3VDCbias -> 22uF; C_Vbias (none) -> 12V
- C606: value 22µ 12VDCbias -> 22uF; C_Vbias (none) -> 12V
- F601: value 16V 2A PTC -> 2A; F_Vdc (none) -> 12V
- R601, R602, R605, R606: value 0 -> 0R
- R603: value 20mR 1% 80mW -> 20mR 1%; R_P (none) -> 80mW
- R604: value 47mR 1% 50mW -> 47mR 1%; R_P (none) -> 47mW
Other:
- note added: "Nominal load: 100mA\nMax load: 1A\nVshunt: 40mV\nCurrent LSB: 250µA"
- note added: "Nominal load: 1A\nMax load: 2A\nVshunt: 40mV\nCurrent LSB: 500µA"
- note removed: "Nominal load: 100mA\nMax load: 1A\nVshunt @ nominal load: 4.7mV\nVshunt @ max load: 47mV\nCurrent LSB: 250µA"
- note removed: "Nominal load: 1A\nMax load: 2A\nVshunt @ nominal load: 20mV\nVshunt @ max load: 40mV\nCurrent LSB: 500µA"
- moved on the sheet: C605, C606, F601, J601, U601
