File: i2c-mux.sch (KiCad schematic (older format))
At the start: 20 parts, among them J501 SMBUS, J502 SMBUS, J503 SMBUS, J504 SMBUS, U501 LTC4306CGN

Commit message: SMD resistor packs @ fan controller, i2c mux
Parts:
- removed R504, R505, R506, R507, R508, R509, R510, R511, R512, R513, R514, R515: 3k, Resistor_SMD:R_0603_1608Metric, symbol Device:R
- added RN501, RN502, RN503, RN504: 3k3, Resistor_SMD:R_Array_Convex_4x1206, symbol Device:R_Pack04
Connections:
- net RSCL: now also RN501.1 (R1.1)
- net RSDA: now also RN501.3 (R3.1)
- net RVCC: now also RN501.5 (R4.2), RN501.6 (R3.2), RN501.7 (R2.2), RN501.8 (R1.2)
- net ~RSMBA: now also RN501.4 (R4.1)
- net at J502.1 (Pin_1): now also RN502.5 (R4.2), RN502.6 (R3.2), RN502.7 (R2.2), RN502.8 (R1.2)
- net at J502.2 (Pin_2), U501.23 (SCL2): now also RN502.1 (R1.1)
- net at J502.4 (Pin_4), U501.22 (SDA2): now also RN502.3 (R3.1)
- net at J502.5 (Pin_5), U501.24 (NALERT2): now also RN502.4 (R4.1)
- net at J503.1 (Pin_1): now also RN503.5 (R4.2), RN503.6 (R3.2), RN503.7 (R2.2), RN503.8 (R1.2)
- net at J503.2 (Pin_2), U501.1 (SCL3): now also RN503.1 (R1.1)
- net at J503.4 (Pin_4), U501.2 (SDA3): now also RN503.3 (R3.1)
- net at J503.5 (Pin_5), U501.21 (NALERT3): now also RN503.4 (R4.1)
- net at J504.1 (Pin_1): now also RN504.5 (R4.2), RN504.6 (R3.2), RN504.7 (R2.2), RN504.8 (R1.2)
- net at J504.2 (Pin_2), U501.17 (SCL4): now also RN504.1 (R1.1)
- net at J504.4 (Pin_4), U501.16 (SDA4): now also RN504.3 (R3.1)
- net at J504.5 (Pin_5), U501.9 (NALERT4): now also RN504.4 (R4.1)

Commit message: Add 1SPI host connector.
fixes #4
Connections:
- no-connect marks 3 -> 7
Changed lines of the file:
@@
 $Descr A4 11693 8268
 encoding utf-8
-Sheet 5 13
+Sheet 5 14
 Title ""
 Date ""
@@
 Wire Wire Line
 	4900 5100 7100 5100
+NoConn ~ 7700 4900
+NoConn ~ 7700 4200
+NoConn ~ 7700 3500
+NoConn ~ 7700 2800
 $EndSCHEMATC

Commit message: Swap more connectors to SMT, route UART and SPI
Parts:
- RN501, RN502, RN503, RN504: footprint Resistor_SMD:R_Array_Convex_4x1206 -> Resistor_SMD:R_Array_Convex_4x0603
Changed lines of the file:
@@
 F 0 "RN501" V 7483 2900 50  0000 C CNN
 F 1 "3k3" V 7574 2900 50  0000 C CNN
-F 2 "Resistor_SMD:R_Array_Convex_4x1206" V 8175 2900 50  0001 C CNN
+F 2 "Resistor_SMD:R_Array_Convex_4x0603" V 8175 2900 50  0001 C CNN
 F 3 "~" H 7900 2900 50  0001 C CNN
 	1    7900 2900
@@
 F 0 "RN502" V 7483 3600 50  0000 C CNN
 F 1 "3k3" V 7574 3600 50  0000 C CNN
-F 2 "Resistor_SMD:R_Array_Convex_4x1206" V 8175 3600 50  0001 C CNN
+F 2 "Resistor_SMD:R_Array_Convex_4x0603" V 8175 3600 50  0001 C CNN
 F 3 "~" H 7900 3600 50  0001 C CNN
 	1    7900 3600
@@
 F 0 "RN503" V 7483 4300 50  0000 C CNN
 F 1 "3k3" V 7574 4300 50  0000 C CNN
-F 2 "Resistor_SMD:R_Array_Convex_4x1206" V 8175 4300 50  0001 C CNN
+F 2 "Resistor_SMD:R_Array_Convex_4x0603" V 8175 4300 50  0001 C CNN
 F 3 "~" H 7900 4300 50  0001 C CNN
 	1    7900 4300
@@
 F 0 "RN504" V 7483 5000 50  0000 C CNN
 F 1 "3k3" V 7574 5000 50  0000 C CNN
-F 2 "Resistor_SMD:R_Array_Convex_4x1206" V 8175 5000 50  0001 C CNN
+F 2 "Resistor_SMD:R_Array_Convex_4x0603" V 8175 5000 50  0001 C CNN
 F 3 "~" H 7900 5000 50  0001 C CNN
 	1    7900 5000

Commit message: Switch SMBus to 6-pin SMD Molex SL
Parts:
- J501, J502, J503, J504: footprint Connector_PinHeader_2.54mm:PinHeader_1x05_P2.54mm_Vertical -> molex-sl:SL_1x06_Vertical_SMD; symbol Connector_Generic:Conn_01x05 -> Connector_Generic:Conn_01x06
Connections:
- net GND: now also J501.6 (Pin_6), J502.6 (Pin_6), J503.6 (Pin_6), J504.6 (Pin_6)
Changed lines of the file:
@@
 Notes:\n- PUs provided\n- 2.2V-5.5V OK\n- NOT ISOLATED - common ground req'd
 $Comp
-L Connector_Generic:Conn_01x05 J501
+L Connector_Generic:Conn_01x06 J501
 U 1 1 5F30BFFF
 P 7300 2800
 F 0 "J501" H 7380 2842 50  0000 L CNN
 F 1 "SMBUS" H 7380 2751 50  0000 L CNN
-F 2 "Connector_PinHeader_2.54mm:PinHeader_1x05_P2.54mm_Vertical" H 7300 2800 50  0001 C CNN
+F 2 "molex-sl:SL_1x06_Vertical_SMD" H 7300 2800 50  0001 C CNN
 F 3 "~" H 7300 2800 50  0001 C CNN
 	1    7300 2800
@@
 	5100 3000 5100 3400
 $Comp
-L Connector_Generic:Conn_01x05 J502
+L Connector_Generic:Conn_01x06 J502
 U 1 1 5F31ACF0
 P 7300 3500
 F 0 "J502" H 7380 3542 50  0000 L CNN
 F 1 "SMBUS" H 7380 3451 50  0000 L CNN
-F 2 "Connector_PinHeader_2.54mm:PinHeader_1x05_P2.54mm_Vertical" H 7300 3500 50  0001 C CNN
+F 2 "molex-sl:SL_1x06_Vertical_SMD" H 7300 3500 50  0001 C CNN
 F 3 "~" H 7300 3500 50  0001 C CNN
 	1    7300 3500
@@
 	7100 3500 6950 3500
 $Comp
-L Connector_Generic:Conn_01x05 J503
+L Connector_Generic:Conn_01x06 J503
 U 1 1 5F31DFF7
 P 7300 4200
 F 0 "J503" H 7380 4242 50  0000 L CNN
 F 1 "SMBUS" H 7380 4151 50  0000 L CNN
-F 2 "Connector_PinHeader_2.54mm:PinHeader_1x05_P2.54mm_Vertical" H 7300 4200 50  0001 C CNN
+F 2 "molex-sl:SL_1x06_Vertical_SMD" H 7300 4200 50  0001 C CNN
 F 3 "~" H 7300 4200 50  0001 C CNN
 	1    7300 4200
@@
 	6550 4300 6550 4200
 $Comp
-L Connector_Generic:Conn_01x05 J504
+L Connector_Generic:Conn_01x06 J504
 U 1 1 5F3236BF
 P 7300 4900
 F 0 "J504" H 7380 4942 50  0000 L CNN
 F 1 "SMBUS" H 7380 4851 50  0000 L CNN
-F 2 "Connector_PinHeader_2.54mm:PinHeader_1x05_P2.54mm_Vertical" H 7300 4900 50  0001 C CNN
+F 2 "molex-sl:SL_1x06_Vertical_SMD" H 7300 4900 50  0001 C CNN
 F 3 "~" H 7300 4900 50  0001 C CNN
 	1    7300 4900
@@
 	5450 3900 4900 3900
 Wire Wire Line
-	6950 2800 6950 3500
+	6950 2800 6950 3100
 Connection ~ 6950 3500
 Wire Wire Line
-	6950 3500 6950 4200
+	6950 3500 6950 3800
 Connection ~ 6950 4200
 Wire Wire Line
-	6950 4200 6950 4900
-Wire Wire Line
-	6950 4900 6950 5250
+	6950 4200 6950 4500
+Wire Wire Line
+	6950 4900 6950 5200
 Connection ~ 6950 4900
 $Comp
@@
 NoConn ~ 7700 3500
 NoConn ~ 7700 2800
+Wire Wire Line
+	7100 3100 6950 3100
+Connection ~ 6950 3100
+Wire Wire Line
+	6950 3100 6950 3500
+Wire Wire Line
+	7100 3800 6950 3800
+Connection ~ 6950 3800
+Wire Wire Line
+	6950 3800 6950 4200
+Wire Wire Line
+	7100 4500 6950 4500
+Connection ~ 6950 4500
+Wire Wire Line
+	6950 4500 6950 4900
+Wire Wire Line
+	7100 5200 6950 5200
+Connection ~ 6950 5200
+Wire Wire Line
+	6950 5200 6950 5250
 $EndSCHEMATC

Commit message: MB: annotate everything with mfg/MPN
Parts:
- J501, J502, J503, J504: Mfg (none) -> Molex; Mfg Part Num (none) -> 0740991006
- R501, R502, R503, RN501, RN502, RN503, RN504: Mfg Part Num (none) -> generic
- U501: Mfg (none) -> Analog; Mfg Part Num (none) -> LTC4306CGN
Changed lines of the file:
@@
 F 2 "Package_SO:SSOP-24_3.9x8.7mm_P0.635mm" H 4250 3850 50  0001 C CNN
 F 3 "" H 4250 3850 50  0001 C CNN
+F 4 "Analog" H 4250 3850 50  0001 C CNN "Mfg"
+F 5 "LTC4306CGN" H 4250 3850 50  0001 C CNN "Mfg Part Num"
 	1    4250 3850
 	1    0    0    -1
@@
 F 2 "molex-sl:SL_1x06_Vertical_SMD" H 7300 2800 50  0001 C CNN
 F 3 "~" H 7300 2800 50  0001 C CNN
+F 4 "Molex" H 7300 2800 50  0001 C CNN "Mfg"
+F 5 "0740991006" H 7300 2800 50  0001 C CNN "Mfg Part Num"
 	1    7300 2800
 	1    0    0    -1
@@
 F 2 "molex-sl:SL_1x06_Vertical_SMD" H 7300 3500 50  0001 C CNN
 F 3 "~" H 7300 3500 50  0001 C CNN
+F 4 "Molex" H 7300 3500 50  0001 C CNN "Mfg"
+F 5 "0740991006" H 7300 3500 50  0001 C CNN "Mfg Part Num"
 	1    7300 3500
 	1    0    0    -1
@@
 F 2 "molex-sl:SL_1x06_Vertical_SMD" H 7300 4200 50  0001 C CNN
 F 3 "~" H 7300 4200 50  0001 C CNN
+F 4 "Molex" H 7300 4200 50  0001 C CNN "Mfg"
+F 5 "0740991006" H 7300 4200 50  0001 C CNN "Mfg Part Num"
 	1    7300 4200
 	1    0    0    -1
@@
 F 2 "molex-sl:SL_1x06_Vertical_SMD" H 7300 4900 50  0001 C CNN
 F 3 "~" H 7300 4900 50  0001 C CNN
+F 4 "Molex" H 7300 4900 50  0001 C CNN "Mfg"
+F 5 "0740991006" H 7300 4900 50  0001 C CNN "Mfg Part Num"
 	1    7300 4900
 	1    0    0    -1
@@
 F 2 "Resistor_SMD:R_0603_1608Metric" V 3480 2850 50  0001 C CNN
 F 3 "~" H 3550 2850 50  0001 C CNN
+F 4 "generic" H 3550 2850 50  0001 C CNN "Mfg Part Num"
 	1    3550 2850
 	-1   0    0    1
@@
 F 2 "Resistor_SMD:R_0603_1608Metric" V 3280 2850 50  0001 C CNN
 F 3 "~" H 3350 2850 50  0001 C CNN
+F 4 "generic" H 3350 2850 50  0001 C CNN "Mfg Part Num"
 	1    3350 2850
 	-1   0    0    1
@@
 F 2 "Resistor_SMD:R_0603_1608Metric" V 3080 2850 50  0001 C CNN
 F 3 "~" H 3150 2850 50  0001 C CNN
+F 4 "generic" H 3150 2850 50  0001 C CNN "Mfg Part Num"
 	1    3150 2850
 	-1   0    0    1
@@
 F 2 "Resistor_SMD:R_Array_Convex_4x0603" V 8175 2900 50  0001 C CNN
 F 3 "~" H 7900 2900 50  0001 C CNN
+F 4 "generic" H 7900 2900 50  0001 C CNN "Mfg Part Num"
 	1    7900 2900
 	0    1    1    0
@@
 F 2 "Resistor_SMD:R_Array_Convex_4x0603" V 8175 3600 50  0001 C CNN
 F 3 "~" H 7900 3600 50  0001 C CNN
+F 4 "generic" H 7900 3600 50  0001 C CNN "Mfg Part Num"
 	1    7900 3600
 	0    1    1    0
@@
 F 2 "Resistor_SMD:R_Array_Convex_4x0603" V 8175 4300 50  0001 C CNN
 F 3 "~" H 7900 4300 50  0001 C CNN
+F 4 "generic" H 7900 4300 50  0001 C CNN "Mfg Part Num"
 	1    7900 4300
 	0    1    1    0
@@
 F 2 "Resistor_SMD:R_Array_Convex_4x0603" V 8175 5000 50  0001 C CNN
 F 3 "~" H 7900 5000 50  0001 C CNN
+F 4 "generic" H 7900 5000 50  0001 C CNN "Mfg Part Num"
 	1    7900 5000
 	0    1    1    0

Commit message: MB: assign single resistors
Parts:
- R501, R502, R503: value 3k -> 3k3; Mfg (none) -> Bourns; Mfg Part Num generic -> CR0603-JW-332ELF
Changed lines of the file:
@@
 P 3550 2850
 F 0 "R503" V 3450 2850 50  0000 C CNN
-F 1 "3k" V 3550 2850 50  0000 C CNN
+F 1 "3k3" V 3550 2850 50  0000 C CNN
 F 2 "Resistor_SMD:R_0603_1608Metric" V 3480 2850 50  0001 C CNN
 F 3 "~" H 3550 2850 50  0001 C CNN
-F 4 "generic" H 3550 2850 50  0001 C CNN "Mfg Part Num"
+F 4 "CR0603-JW-332ELF" H 3550 2850 50  0001 C CNN "Mfg Part Num"
+F 5 "Bourns" H 3550 2850 50  0001 C CNN "Mfg"
 	1    3550 2850
 	-1   0    0    1
@@
 P 3350 2850
 F 0 "R502" V 3250 2850 50  0000 C CNN
-F 1 "3k" V 3350 2850 50  0000 C CNN
+F 1 "3k3" V 3350 2850 50  0000 C CNN
 F 2 "Resistor_SMD:R_0603_1608Metric" V 3280 2850 50  0001 C CNN
 F 3 "~" H 3350 2850 50  0001 C CNN
-F 4 "generic" H 3350 2850 50  0001 C CNN "Mfg Part Num"
+F 4 "CR0603-JW-332ELF" H 3350 2850 50  0001 C CNN "Mfg Part Num"
+F 5 "Bourns" H 3350 2850 50  0001 C CNN "Mfg"
 	1    3350 2850
 	-1   0    0    1
@@
 P 3150 2850
 F 0 "R501" V 3050 2850 50  0000 C CNN
-F 1 "3k" V 3150 2850 50  0000 C CNN
+F 1 "3k3" V 3150 2850 50  0000 C CNN
 F 2 "Resistor_SMD:R_0603_1608Metric" V 3080 2850 50  0001 C CNN
 F 3 "~" H 3150 2850 50  0001 C CNN
-F 4 "generic" H 3150 2850 50  0001 C CNN "Mfg Part Num"
+F 4 "CR0603-JW-332ELF" H 3150 2850 50  0001 C CNN "Mfg Part Num"
+F 5 "Bourns" H 3150 2850 50  0001 C CNN "Mfg"
 	1    3150 2850
 	-1   0    0    1

Commit message: MB: assign resistor networks
...and replace the x5 networks with discretes because they don't exist.
Parts:
- RN501, RN502, RN503, RN504: Mfg (none) -> Bourns; Mfg Part Num generic -> CAY16-3301F4LF
Changed lines of the file:
@@
 F 2 "Resistor_SMD:R_Array_Convex_4x0603" V 8175 2900 50  0001 C CNN
 F 3 "~" H 7900 2900 50  0001 C CNN
-F 4 "generic" H 7900 2900 50  0001 C CNN "Mfg Part Num"
+F 4 "CAY16-3301F4LF" H 7900 2900 50  0001 C CNN "Mfg Part Num"
+F 5 "Bourns" H 7900 2900 50  0001 C CNN "Mfg"
 	1    7900 2900
 	0    1    1    0
@@
 F 2 "Resistor_SMD:R_Array_Convex_4x0603" V 8175 3600 50  0001 C CNN
 F 3 "~" H 7900 3600 50  0001 C CNN
-F 4 "generic" H 7900 3600 50  0001 C CNN "Mfg Part Num"
+F 4 "CAY16-3301F4LF" H 7900 3600 50  0001 C CNN "Mfg Part Num"
+F 5 "Bourns" H 7900 3600 50  0001 C CNN "Mfg"
 	1    7900 3600
 	0    1    1    0
@@
 F 2 "Resistor_SMD:R_Array_Convex_4x0603" V 8175 4300 50  0001 C CNN
 F 3 "~" H 7900 4300 50  0001 C CNN
-F 4 "generic" H 7900 4300 50  0001 C CNN "Mfg Part Num"
+F 4 "CAY16-3301F4LF" H 7900 4300 50  0001 C CNN "Mfg Part Num"
+F 5 "Bourns" H 7900 4300 50  0001 C CNN "Mfg"
 	1    7900 4300
 	0    1    1    0
@@
 F 2 "Resistor_SMD:R_Array_Convex_4x0603" V 8175 5000 50  0001 C CNN
 F 3 "~" H 7900 5000 50  0001 C CNN
-F 4 "generic" H 7900 5000 50  0001 C CNN "Mfg Part Num"
+F 4 "CAY16-3301F4LF" H 7900 5000 50  0001 C CNN "Mfg Part Num"
+F 5 "Bourns" H 7900 5000 50  0001 C CNN "Mfg"
 	1    7900 5000
 	0    1    1    0
