File: i2c-mux.sch (KiCad schematic (older format))
At the start: 12 parts, among them J501 SMBUS, J502 SMBUS, J503 SMBUS, J504 SMBUS, U501 LTC4306CGN

Commit message: MB: add caps suggested in review
Parts:
- added C501: 0µ1, Capacitor_SMD:C_0603_1608Metric, symbol Device:C_Small
Connections:
- net +3V3: now also C501.1
- net GND: now also C501.2
Changed lines of the file:
@@
 Wire Wire Line
 	6950 5200 6950 5250
+$Comp
+L Device:C_Small C?
+U 1 1 5F6D05E3
+P 2800 4350
+AR Path="/5F1928E5/5F29584B/5F6D05E3" Ref="C?"  Part="1"
+AR Path="/5F3B585A/5F6D05E3" Ref="C501"  Part="1"
+F 0 "C501" H 2892 4396 50  0000 L CNN
+F 1 "0µ1" H 2892 4305 50  0000 L CNN
+F 2 "Capacitor_SMD:C_0603_1608Metric" H 2800 4350 50  0001 C CNN
+F 3 "~" H 2800 4350 50  0001 C CNN
+F 4 "CL10B104KB8NNWC" H 2800 4350 50  0001 C CNN "Mfg Part Num"
+F 5 "Samsung Electro-Mechanics" H 2800 4350 50  0001 C CNN "Mfg"
+	1    2800 4350
+	1    0    0    -1
+$EndComp
+$Comp
+L power:+3V3 #PWR0506
+U 1 1 5F6D2D19
+P 2800 4250
+F 0 "#PWR0506" H 2800 4100 50  0001 C CNN
+F 1 "+3V3" H 2815 4423 50  0000 C CNN
+F 2 "" H 2800 4250 50  0001 C CNN
+F 3 "" H 2800 4250 50  0001 C CNN
+	1    2800 4250
+	1    0    0    -1
+$EndComp
+$Comp
+L power:GND #PWR0507
+U 1 1 5F6D30E2
+P 2800 4450
+F 0 "#PWR0507" H 2800 4200 50  0001 C CNN
+F 1 "GND" H 2805 4277 50  0000 C CNN
+F 2 "" H 2800 4450 50  0001 C CNN
+F 3 "" H 2800 4450 50  0001 C CNN
+	1    2800 4450
+	1    0    0    -1
+$EndComp
 $EndSCHEMATC

Commit message: gemini-bringup: Add CPNs for all components
Parts:
- C501: CPN (none) -> 212-00011
- J501, J502, J503, J504: CPN (none) -> 215-00028
- R501, R502, R503: CPN (none) -> 232-00018
- RN501, RN502, RN503, RN504: CPN (none) -> 232-00034
- U501: CPN (none) -> 221-00014
Changed lines of the file:
@@
 F 4 "Analog" H 4250 3850 50  0001 C CNN "Mfg"
 F 5 "LTC4306CGN" H 4250 3850 50  0001 C CNN "Mfg Part Num"
+F 6 "221-00014" H 4250 3850 50  0001 C CNN "CPN"
 	1    4250 3850
 	1    0    0    -1
@@
 F 4 "Molex" H 7300 2800 50  0001 C CNN "Mfg"
 F 5 "0740991006" H 7300 2800 50  0001 C CNN "Mfg Part Num"
+F 6 "215-00028" H 7300 2800 50  0001 C CNN "CPN"
 	1    7300 2800
 	1    0    0    -1
@@
 F 4 "Molex" H 7300 3500 50  0001 C CNN "Mfg"
 F 5 "0740991006" H 7300 3500 50  0001 C CNN "Mfg Part Num"
+F 6 "215-00028" H 7300 3500 50  0001 C CNN "CPN"
 	1    7300 3500
 	1    0    0    -1
@@
 F 4 "Molex" H 7300 4200 50  0001 C CNN "Mfg"
 F 5 "0740991006" H 7300 4200 50  0001 C CNN "Mfg Part Num"
+F 6 "215-00028" H 7300 4200 50  0001 C CNN "CPN"
 	1    7300 4200
 	1    0    0    -1
@@
 F 4 "Molex" H 7300 4900 50  0001 C CNN "Mfg"
 F 5 "0740991006" H 7300 4900 50  0001 C CNN "Mfg Part Num"
+F 6 "215-00028" H 7300 4900 50  0001 C CNN "CPN"
 	1    7300 4900
 	1    0    0    -1
@@
 F 4 "CR0603-JW-332ELF" H 3550 2850 50  0001 C CNN "Mfg Part Num"
 F 5 "Bourns" H 3550 2850 50  0001 C CNN "Mfg"
+F 6 "232-00018" H 3550 2850 50  0001 C CNN "CPN"
 	1    3550 2850
 	-1   0    0    1
@@
 F 4 "CR0603-JW-332ELF" H 3350 2850 50  0001 C CNN "Mfg Part Num"
 F 5 "Bourns" H 3350 2850 50  0001 C CNN "Mfg"
+F 6 "232-00018" H 3350 2850 50  0001 C CNN "CPN"
 	1    3350 2850
 	-1   0    0    1
@@
 F 4 "CR0603-JW-332ELF" H 3150 2850 50  0001 C CNN "Mfg Part Num"
 F 5 "Bourns" H 3150 2850 50  0001 C CNN "Mfg"
+F 6 "232-00018" H 3150 2850 50  0001 C CNN "CPN"
 	1    3150 2850
 	-1   0    0    1
@@
 F 4 "CAY16-3301F4LF" H 7900 2900 50  0001 C CNN "Mfg Part Num"
 F 5 "Bourns" H 7900 2900 50  0001 C CNN "Mfg"
+F 6 "232-00034" H 7900 2900 50  0001 C CNN "CPN"
 	1    7900 2900
 	0    1    1    0
@@
 F 4 "CAY16-3301F4LF" H 7900 3600 50  0001 C CNN "Mfg Part Num"
 F 5 "Bourns" H 7900 3600 50  0001 C CNN "Mfg"
+F 6 "232-00034" H 7900 3600 50  0001 C CNN "CPN"
 	1    7900 3600
 	0    1    1    0
@@
 F 4 "CAY16-3301F4LF" H 7900 4300 50  0001 C CNN "Mfg Part Num"
 F 5 "Bourns" H 7900 4300 50  0001 C CNN "Mfg"
+F 6 "232-00034" H 7900 4300 50  0001 C CNN "CPN"
 	1    7900 4300
 	0    1    1    0
@@
 F 4 "CAY16-3301F4LF" H 7900 5000 50  0001 C CNN "Mfg Part Num"
 F 5 "Bourns" H 7900 5000 50  0001 C CNN "Mfg"
+F 6 "232-00034" H 7900 5000 50  0001 C CNN "CPN"
 	1    7900 5000
 	0    1    1    0
@@
 F 4 "CL10B104KB8NNWC" H 2800 4350 50  0001 C CNN "Mfg Part Num"
 F 5 "Samsung Electro-Mechanics" H 2800 4350 50  0001 C CNN "Mfg"
+F 6 "212-00011" H 2800 4350 50  0001 C CNN "CPN"
 	1    2800 4350
 	1    0    0    -1

Commit message: i2c-mux: specify rating constraints on passives
Parts:
- C501: value 0µ1 -> 0.1uF 3.3VDCbias
- R501, R502, R503, RN501, RN502, RN503, RN504: value 3k3 -> 3.3kR
Other:
- moved on the sheet: C501
Changed lines of the file:
@@
 P 3550 2850
 F 0 "R503" V 3450 2850 50  0000 C CNN
-F 1 "3k3" V 3550 2850 50  0000 C CNN
+F 1 "3.3kR" V 3550 2850 50  0000 C CNN
 F 2 "Resistor_SMD:R_0603_1608Metric" V 3480 2850 50  0001 C CNN
 F 3 "~" H 3550 2850 50  0001 C CNN
@@
 P 3350 2850
 F 0 "R502" V 3250 2850 50  0000 C CNN
-F 1 "3k3" V 3350 2850 50  0000 C CNN
+F 1 "3.3kR" V 3350 2850 50  0000 C CNN
 F 2 "Resistor_SMD:R_0603_1608Metric" V 3280 2850 50  0001 C CNN
 F 3 "~" H 3350 2850 50  0001 C CNN
@@
 P 3150 2850
 F 0 "R501" V 3050 2850 50  0000 C CNN
-F 1 "3k3" V 3150 2850 50  0000 C CNN
+F 1 "3.3kR" V 3150 2850 50  0000 C CNN
 F 2 "Resistor_SMD:R_0603_1608Metric" V 3080 2850 50  0001 C CNN
 F 3 "~" H 3150 2850 50  0001 C CNN
@@
 P 7900 2900
 F 0 "RN501" V 7483 2900 50  0000 C CNN
-F 1 "3k3" V 7574 2900 50  0000 C CNN
+F 1 "3.3kR" V 7574 2900 50  0000 C CNN
 F 2 "Resistor_SMD:R_Array_Convex_4x0603" V 8175 2900 50  0001 C CNN
 F 3 "~" H 7900 2900 50  0001 C CNN
@@
 P 7900 3600
 F 0 "RN502" V 7483 3600 50  0000 C CNN
-F 1 "3k3" V 7574 3600 50  0000 C CNN
+F 1 "3.3kR" V 7574 3600 50  0000 C CNN
 F 2 "Resistor_SMD:R_Array_Convex_4x0603" V 8175 3600 50  0001 C CNN
 F 3 "~" H 7900 3600 50  0001 C CNN
@@
 P 7900 4300
 F 0 "RN503" V 7483 4300 50  0000 C CNN
-F 1 "3k3" V 7574 4300 50  0000 C CNN
+F 1 "3.3kR" V 7574 4300 50  0000 C CNN
 F 2 "Resistor_SMD:R_Array_Convex_4x0603" V 8175 4300 50  0001 C CNN
 F 3 "~" H 7900 4300 50  0001 C CNN
@@
 P 7900 5000
 F 0 "RN504" V 7483 5000 50  0000 C CNN
-F 1 "3k3" V 7574 5000 50  0000 C CNN
+F 1 "3.3kR" V 7574 5000 50  0000 C CNN
 F 2 "Resistor_SMD:R_Array_Convex_4x0603" V 8175 5000 50  0001 C CNN
 F 3 "~" H 7900 5000 50  0001 C CNN
@@
 L Device:C_Small C?
 U 1 1 5F6D05E3
-P 2800 4350
+P 2450 4350
 AR Path="/5F1928E5/5F29584B/5F6D05E3" Ref="C?"  Part="1"
 AR Path="/5F3B585A/5F6D05E3" Ref="C501"  Part="1"
-F 0 "C501" H 2892 4396 50  0000 L CNN
-F 1 "0µ1" H 2892 4305 50  0000 L CNN
-F 2 "Capacitor_SMD:C_0603_1608Metric" H 2800 4350 50  0001 C CNN
-F 3 "~" H 2800 4350 50  0001 C CNN
-F 4 "CL10B104KB8NNWC" H 2800 4350 50  0001 C CNN "Mfg Part Num"
-F 5 "Samsung Electro-Mechanics" H 2800 4350 50  0001 C CNN "Mfg"
-F 6 "212-00011" H 2800 4350 50  0001 C CNN "CPN"
-	1    2800 4350
+F 0 "C501" H 2542 4396 50  0000 L CNN
+F 1 "0.1uF 3.3VDCbias" H 2542 4305 50  0000 L CNN
+F 2 "Capacitor_SMD:C_0603_1608Metric" H 2450 4350 50  0001 C CNN
+F 3 "~" H 2450 4350 50  0001 C CNN
+F 4 "CL10B104KB8NNWC" H 2450 4350 50  0001 C CNN "Mfg Part Num"
+F 5 "Samsung Electro-Mechanics" H 2450 4350 50  0001 C CNN "Mfg"
+F 6 "212-00011" H 2450 4350 50  0001 C CNN "CPN"
+	1    2450 4350
 	1    0    0    -1
 $EndComp
@@
 L power:+3V3 #PWR0506
 U 1 1 5F6D2D19
-P 2800 4250
-F 0 "#PWR0506" H 2800 4100 50  0001 C CNN
-F 1 "+3V3" H 2815 4423 50  0000 C CNN
-F 2 "" H 2800 4250 50  0001 C CNN
-F 3 "" H 2800 4250 50  0001 C CNN
-	1    2800 4250
+P 2450 4250
+F 0 "#PWR0506" H 2450 4100 50  0001 C CNN
+F 1 "+3V3" H 2465 4423 50  0000 C CNN
+F 2 "" H 2450 4250 50  0001 C CNN
+F 3 "" H 2450 4250 50  0001 C CNN
+	1    2450 4250
 	1    0    0    -1
 $EndComp
@@
 L power:GND #PWR0507
 U 1 1 5F6D30E2
-P 2800 4450
-F 0 "#PWR0507" H 2800 4200 50  0001 C CNN
-F 1 "GND" H 2805 4277 50  0000 C CNN
-F 2 "" H 2800 4450 50  0001 C CNN
-F 3 "" H 2800 4450 50  0001 C CNN
-	1    2800 4450
+P 2450 4450
+F 0 "#PWR0507" H 2450 4200 50  0001 C CNN
+F 1 "GND" H 2455 4277 50  0000 C CNN
+F 2 "" H 2450 4450 50  0001 C CNN
+F 3 "" H 2450 4450 50  0001 C CNN
+	1    2450 4450
 	1    0    0    -1
 $EndComp

Commit message: gemini-bringup: custom fields for rating constraints on passives
Instead of packing tons of detail into a single "Value" field, limit
"Value" to the primary characteristic of the device (i.e. capacitance
for capacitors, resistance for resistors, current for fuses, impedence
at frequency for ferrite beads). For all other rating constraints, use
custom fields of the form <component-refdes-prefix>_<constraint>. For
example, R_P contains the power a resistor must dissipate.  Use
calculated values when possible rather than standard values as the
intent is to capture the constraint, not a specific device choice.
Parts:
- C501: value 0.1uF 3.3VDCbias -> 0.1uF; C_Vbias (none) -> 3.3V
Other:
- moved on the sheet: C501
Changed lines of the file:
@@
 L Device:C_Small C?
 U 1 1 5F6D05E3
-P 2450 4350
+P 2800 4350
 AR Path="/5F1928E5/5F29584B/5F6D05E3" Ref="C?"  Part="1"
 AR Path="/5F3B585A/5F6D05E3" Ref="C501"  Part="1"
-F 0 "C501" H 2542 4396 50  0000 L CNN
-F 1 "0.1uF 3.3VDCbias" H 2542 4305 50  0000 L CNN
-F 2 "Capacitor_SMD:C_0603_1608Metric" H 2450 4350 50  0001 C CNN
-F 3 "~" H 2450 4350 50  0001 C CNN
-F 4 "CL10B104KB8NNWC" H 2450 4350 50  0001 C CNN "Mfg Part Num"
-F 5 "Samsung Electro-Mechanics" H 2450 4350 50  0001 C CNN "Mfg"
-F 6 "212-00011" H 2450 4350 50  0001 C CNN "CPN"
-	1    2450 4350
+F 0 "C501" H 2892 4396 50  0000 L CNN
+F 1 "0.1uF" H 2892 4305 50  0000 L CNN
+F 2 "Capacitor_SMD:C_0603_1608Metric" H 2800 4350 50  0001 C CNN
+F 3 "~" H 2800 4350 50  0001 C CNN
+F 4 "CL10B104KB8NNWC" H 2800 4350 50  0001 C CNN "Mfg Part Num"
+F 5 "Samsung Electro-Mechanics" H 2800 4350 50  0001 C CNN "Mfg"
+F 6 "212-00011" H 2800 4350 50  0001 C CNN "CPN"
+F 7 "3.3V" H 2800 4350 50  0001 C CNN "C_Vbias"
+	1    2800 4350
 	1    0    0    -1
 $EndComp
@@
 L power:+3V3 #PWR0506
 U 1 1 5F6D2D19
-P 2450 4250
-F 0 "#PWR0506" H 2450 4100 50  0001 C CNN
-F 1 "+3V3" H 2465 4423 50  0000 C CNN
-F 2 "" H 2450 4250 50  0001 C CNN
-F 3 "" H 2450 4250 50  0001 C CNN
-	1    2450 4250
+P 2800 4250
+F 0 "#PWR0506" H 2800 4100 50  0001 C CNN
+F 1 "+3V3" H 2815 4423 50  0000 C CNN
+F 2 "" H 2800 4250 50  0001 C CNN
+F 3 "" H 2800 4250 50  0001 C CNN
+	1    2800 4250
 	1    0    0    -1
 $EndComp
@@
 L power:GND #PWR0507
 U 1 1 5F6D30E2
-P 2450 4450
-F 0 "#PWR0507" H 2450 4200 50  0001 C CNN
-F 1 "GND" H 2455 4277 50  0000 C CNN
-F 2 "" H 2450 4450 50  0001 C CNN
-F 3 "" H 2450 4450 50  0001 C CNN
-	1    2450 4450
+P 2800 4450
+F 0 "#PWR0507" H 2800 4200 50  0001 C CNN
+F 1 "GND" H 2805 4277 50  0000 C CNN
+F 2 "" H 2800 4450 50  0001 C CNN
+F 3 "" H 2800 4450 50  0001 C CNN
+	1    2800 4450
 	1    0    0    -1
 $EndComp

Commit message: gemini-bringup: resistor power rating constraints
Parts:
- R501, R502, R503: R_P (none) -> 1mW
- RN501, RN502, RN503, RN504: RN_Ppkg (none) -> 5mW; RN_Pres (none) -> 1.7mW
Changed lines of the file:
@@
 F 5 "Bourns" H 3550 2850 50  0001 C CNN "Mfg"
 F 6 "232-00018" H 3550 2850 50  0001 C CNN "CPN"
+F 7 "1mW" H 3550 2850 50  0001 C CNN "R_P"
 	1    3550 2850
 	-1   0    0    1
@@
 F 5 "Bourns" H 3350 2850 50  0001 C CNN "Mfg"
 F 6 "232-00018" H 3350 2850 50  0001 C CNN "CPN"
+F 7 "1mW" H 3350 2850 50  0001 C CNN "R_P"
 	1    3350 2850
 	-1   0    0    1
@@
 F 5 "Bourns" H 3150 2850 50  0001 C CNN "Mfg"
 F 6 "232-00018" H 3150 2850 50  0001 C CNN "CPN"
+F 7 "1mW" H 3150 2850 50  0001 C CNN "R_P"
 	1    3150 2850
 	-1   0    0    1
@@
 F 5 "Bourns" H 7900 2900 50  0001 C CNN "Mfg"
 F 6 "232-00034" H 7900 2900 50  0001 C CNN "CPN"
+F 7 "1.7mW" V 7900 2900 50  0001 C CNN "RN_Pres"
+F 8 "5mW" V 7900 2900 50  0001 C CNN "RN_Ppkg"
 	1    7900 2900
 	0    1    1    0
@@
 F 5 "Bourns" H 7900 3600 50  0001 C CNN "Mfg"
 F 6 "232-00034" H 7900 3600 50  0001 C CNN "CPN"
+F 7 "5mW" H 7900 3600 50  0001 C CNN "RN_Ppkg"
+F 8 "1.7mW" H 7900 3600 50  0001 C CNN "RN_Pres"
 	1    7900 3600
 	0    1    1    0
@@
 F 5 "Bourns" H 7900 4300 50  0001 C CNN "Mfg"
 F 6 "232-00034" H 7900 4300 50  0001 C CNN "CPN"
+F 7 "5mW" H 7900 4300 50  0001 C CNN "RN_Ppkg"
+F 8 "1.7mW" H 7900 4300 50  0001 C CNN "RN_Pres"
 	1    7900 4300
 	0    1    1    0
@@
 F 5 "Bourns" H 7900 5000 50  0001 C CNN "Mfg"
 F 6 "232-00034" H 7900 5000 50  0001 C CNN "CPN"
+F 7 "5mW" H 7900 5000 50  0001 C CNN "RN_Ppkg"
+F 8 "1.7mW" H 7900 5000 50  0001 C CNN "RN_Pres"
 	1    7900 5000
 	0    1    1    0

Commit message: gemini-bringup: reselect all caps respecting C/V derating
Parts:
- C501: Mfg Samsung Electro-Mechanics -> Kemet; Mfg Part Num CL10B104KB8NNWC -> C0603C104M4RACTU
Changed lines of the file:
@@
 F 2 "Capacitor_SMD:C_0603_1608Metric" H 2800 4350 50  0001 C CNN
 F 3 "~" H 2800 4350 50  0001 C CNN
-F 4 "CL10B104KB8NNWC" H 2800 4350 50  0001 C CNN "Mfg Part Num"
-F 5 "Samsung Electro-Mechanics" H 2800 4350 50  0001 C CNN "Mfg"
+F 4 "C0603C104M4RACTU" H 2800 4350 50  0001 C CNN "Mfg Part Num"
+F 5 "Kemet" H 2800 4350 50  0001 C CNN "Mfg"
 F 6 "212-00011" H 2800 4350 50  0001 C CNN "CPN"
 F 7 "3.3V" H 2800 4350 50  0001 C CNN "C_Vbias"
