File: sdcard.sch (KiCad schematic (older format))
At the start: 2 parts

Commit message: Annotate in preparation for review
Parts:
- gave numbers to parts that had none: 2
Changed lines of the file:
@@
 	7050 3650 7050 4200
 $Comp
-L emif06-msdn02-n16:EMIF06-MSD02N16 U?
+L emif06-msdn02-n16:EMIF06-MSD02N16 U901
 U 1 1 5F2CB8E1
 P 5550 3500
-F 0 "U?" H 5575 4115 50  0000 C CNN
+F 0 "U901" H 5575 4115 50  0000 C CNN
 F 1 "EMIF06-MSD02N16" H 5575 4024 50  0000 C CNN
 F 2 "" H 5650 3500 50  0001 C CNN
@@
 $EndComp
 $Comp
-L Connector:Micro_SD_Card J?
+L Connector:Micro_SD_Card J901
 U 1 1 5F2CD2A2
 P 8100 3450
-F 0 "J?" H 8050 4167 50  0000 C CNN
+F 0 "J901" H 8050 4167 50  0000 C CNN
 F 1 "Micro_SD_Card" H 8050 4076 50  0000 C CNN
 F 2 "" H 9250 3750 50  0001 C CNN
@@
 $EndComp
 $Comp
-L power:GND #PWR?
+L power:GND #PWR0901
 U 1 1 5F2CE322
 P 4950 3250
-F 0 "#PWR?" H 4950 3000 50  0001 C CNN
+F 0 "#PWR0901" H 4950 3000 50  0001 C CNN
 F 1 "GND" V 4955 3122 50  0000 R CNN
 F 2 "" H 4950 3250 50  0001 C CNN
@@
 	7200 3850 6200 3850
 $Comp
-L power:GND #PWR?
+L power:GND #PWR0902
 U 1 1 5F2CF76B
 P 5550 4050
-F 0 "#PWR?" H 5550 3800 50  0001 C CNN
+F 0 "#PWR0902" H 5550 3800 50  0001 C CNN
 F 1 "GND" H 5555 3877 50  0000 C CNN
 F 2 "" H 5550 4050 50  0001 C CNN
@@
 $EndComp
 $Comp
-L power:GND #PWR?
+L power:GND #PWR0905
 U 1 1 5F2CF93F
 P 7050 4200
-F 0 "#PWR?" H 7050 3950 50  0001 C CNN
+F 0 "#PWR0905" H 7050 3950 50  0001 C CNN
 F 1 "GND" H 7055 4027 50  0000 C CNN
 F 2 "" H 7050 4200 50  0001 C CNN
@@
 $EndComp
 $Comp
-L power:+3V3 #PWR?
+L power:+3V3 #PWR0904
 U 1 1 5F2CFAEE
 P 7050 2950
-F 0 "#PWR?" H 7050 2800 50  0001 C CNN
+F 0 "#PWR0904" H 7050 2800 50  0001 C CNN
 F 1 "+3V3" H 7065 3123 50  0000 C CNN
 F 2 "" H 7050 2950 50  0001 C CNN
@@
 $EndComp
 $Comp
-L power:+3V3 #PWR?
+L power:+3V3 #PWR0903
 U 1 1 5F2CFB57
 P 6300 2950
-F 0 "#PWR?" H 6300 2800 50  0001 C CNN
+F 0 "#PWR0903" H 6300 2800 50  0001 C CNN
 F 1 "+3V3" H 6315 3123 50  0000 C CNN
 F 2 "" H 6300 2950 50  0001 C CNN
@@
 Socket is wired for card detect with\ninternal pullup resistor, but card\nhot swapping not really expected.
 $Comp
-L power:GND #PWR?
+L power:GND #PWR0906
 U 1 1 5F2D96B2
 P 8900 4050
-F 0 "#PWR?" H 8900 3800 50  0001 C CNN
+F 0 "#PWR0906" H 8900 3800 50  0001 C CNN
 F 1 "GND" H 8905 3877 50  0000 C CNN
 F 2 "" H 8900 4050 50  0001 C CNN

Commit message: Assign noncontroversial footprints.
- For components that only come in one flavor, use it.
- For passives, go with 0603, except for current sense resistors.
- Use the Yamaichi socket footprint for the 'h7
- Delete at least one default but wrong association.
Parts:
- U901: footprint (none) -> micro-qfn16-narrow:DFN-16-1EP_1.2x3.5mm_P0.4mm_EP0.3x2.8mm
Changed lines of the file:
@@
 F 0 "U901" H 5575 4115 50  0000 C CNN
 F 1 "EMIF06-MSD02N16" H 5575 4024 50  0000 C CNN
-F 2 "" H 5650 3500 50  0001 C CNN
+F 2 "micro-qfn16-narrow:DFN-16-1EP_1.2x3.5mm_P0.4mm_EP0.3x2.8mm" H 5650 3500 50  0001 C CNN
 F 3 "" H 5650 3500 50  0001 C CNN
 	1    5550 3500
@@
 Wire Bus Line
 	4000 3200 4250 3200
-Wire Bus Line
-	4250 3200 4250 3750
 Text Label 4000 3200 0    50   ~ 0
 D[0..3]
@@
 	1    0    0    -1
 $EndComp
+Wire Bus Line
+	4250 3200 4250 3750
 $EndSCHEMATC

Commit message: More footprint associations
Parts:
- J901: footprint (none) -> Connector_Card:microSD_HC_Wuerth_693072010801
Changed lines of the file:
@@
 F 0 "J901" H 8050 4167 50  0000 C CNN
 F 1 "Micro_SD_Card" H 8050 4076 50  0000 C CNN
-F 2 "" H 9250 3750 50  0001 C CNN
+F 2 "Connector_Card:microSD_HC_Wuerth_693072010801" H 9250 3750 50  0001 C CNN
 F 3 "http://katalog.we-online.de/em/datasheet/693072010801.pdf" H 8100 3450 50  0001 C CNN
 	1    8100 3450

Commit message: MB: annotate everything with mfg/MPN
Parts:
- J901: Mfg (none) -> Würth Elektronik; Mfg Part Num (none) -> 693072010801
- U901: Mfg (none) -> ST; Mfg Part Num (none) -> EMIF06-MSD02N16
Changed lines of the file:
@@
 F 2 "micro-qfn16-narrow:DFN-16-1EP_1.2x3.5mm_P0.4mm_EP0.3x2.8mm" H 5650 3500 50  0001 C CNN
 F 3 "" H 5650 3500 50  0001 C CNN
+F 4 "ST" H 5550 3500 50  0001 C CNN "Mfg"
+F 5 "EMIF06-MSD02N16" H 5550 3500 50  0001 C CNN "Mfg Part Num"
 	1    5550 3500
 	1    0    0    -1
@@
 F 2 "Connector_Card:microSD_HC_Wuerth_693072010801" H 9250 3750 50  0001 C CNN
 F 3 "http://katalog.we-online.de/em/datasheet/693072010801.pdf" H 8100 3450 50  0001 C CNN
+F 4 "Würth Elektronik" H 8100 3450 50  0001 C CNN "Mfg"
+F 5 "693072010801" H 8100 3450 50  0001 C CNN "Mfg Part Num"
 	1    8100 3450
 	1    0    0    -1

Commit message: MB: add caps suggested in review
Parts:
- added C901: 0µ1, Capacitor_SMD:C_0603_1608Metric, symbol Device:C_Small
Connections:
- net +3V3: now also C901.1
- net GND: now also C901.2
Changed lines of the file:
@@
+	1    0    0    -1
+$EndComp
+$Comp
+L Device:C_Small C?
+U 1 1 5F68D900
+P 6050 4800
+AR Path="/5F1928E5/5F68D900" Ref="C?"  Part="1"
+AR Path="/5F2C887E/5F68D900" Ref="C901"  Part="1"
+F 0 "C901" H 6142 4846 50  0000 L CNN
+F 1 "0µ1" H 6142 4755 50  0000 L CNN
+F 2 "Capacitor_SMD:C_0603_1608Metric" H 6050 4800 50  0001 C CNN
+F 3 "~" H 6050 4800 50  0001 C CNN
+F 4 "CL10B104KB8NNWC" H 6050 4800 50  0001 C CNN "Mfg Part Num"
+F 5 "Samsung Electro-Mechanics" H 6050 4800 50  0001 C CNN "Mfg"
+	1    6050 4800
 	1    0    0    -1
 $EndComp
 Wire Bus Line
 	4250 3200 4250 3750
+$Comp
+L power:+3V3 #PWR0907
+U 1 1 5F68DC3A
+P 6050 4700
+F 0 "#PWR0907" H 6050 4550 50  0001 C CNN
+F 1 "+3V3" H 6065 4873 50  0000 C CNN
+F 2 "" H 6050 4700 50  0001 C CNN
+F 3 "" H 6050 4700 50  0001 C CNN
+	1    6050 4700
+	1    0    0    -1
+$EndComp
+$Comp
+L power:GND #PWR0908
+U 1 1 5F68E3C5
+P 6050 4900
+F 0 "#PWR0908" H 6050 4650 50  0001 C CNN
+F 1 "GND" H 6055 4727 50  0000 C CNN
+F 2 "" H 6050 4900 50  0001 C CNN
+F 3 "" H 6050 4900 50  0001 C CNN
+	1    6050 4900
+	1    0    0    -1
+$EndComp
 $EndSCHEMATC
