File: sdcard.sch (KiCad schematic (older format))
At the start: 3 parts, among them J901 Micro_SD_Card, U901 EMIF06-MSD02N16

Commit message: gemini-bringup: Add CPNs for all components
Parts:
- C901: CPN (none) -> 212-00011
- J901: CPN (none) -> 215-00032
- U901: CPN (none) -> 221-00021
Changed lines of the file:
@@
 F 4 "ST" H 5550 3500 50  0001 C CNN "Mfg"
 F 5 "EMIF06-MSD02N16" H 5550 3500 50  0001 C CNN "Mfg Part Num"
+F 6 "221-00021" H 5550 3500 50  0001 C CNN "CPN"
 	1    5550 3500
 	1    0    0    -1
@@
 F 4 "Würth Elektronik" H 8100 3450 50  0001 C CNN "Mfg"
 F 5 "693072010801" H 8100 3450 50  0001 C CNN "Mfg Part Num"
+F 6 "215-00032" H 8100 3450 50  0001 C CNN "CPN"
 	1    8100 3450
 	1    0    0    -1
@@
 F 4 "CL10B104KB8NNWC" H 6050 4800 50  0001 C CNN "Mfg Part Num"
 F 5 "Samsung Electro-Mechanics" H 6050 4800 50  0001 C CNN "Mfg"
+F 6 "212-00011" H 6050 4800 50  0001 C CNN "CPN"
 	1    6050 4800
 	1    0    0    -1

Commit message: sdcard: specify rating constraints on passives
Parts:
- C901: value 0µ1 -> 0.1uF 3.3VDCbias
Changed lines of the file:
@@
 AR Path="/5F2C887E/5F68D900" Ref="C901"  Part="1"
 F 0 "C901" H 6142 4846 50  0000 L CNN
-F 1 "0µ1" H 6142 4755 50  0000 L CNN
+F 1 "0.1uF 3.3VDCbias" H 6142 4755 50  0000 L CNN
 F 2 "Capacitor_SMD:C_0603_1608Metric" H 6050 4800 50  0001 C CNN
 F 3 "~" H 6050 4800 50  0001 C CNN

Commit message: gemini-bringup: custom fields for rating constraints on passives
Instead of packing tons of detail into a single "Value" field, limit
"Value" to the primary characteristic of the device (i.e. capacitance
for capacitors, resistance for resistors, current for fuses, impedence
at frequency for ferrite beads). For all other rating constraints, use
custom fields of the form <component-refdes-prefix>_<constraint>. For
example, R_P contains the power a resistor must dissipate.  Use
calculated values when possible rather than standard values as the
intent is to capture the constraint, not a specific device choice.
Parts:
- C901: value 0.1uF 3.3VDCbias -> 0.1uF; C_Vbias (none) -> 3.3V
Changed lines of the file:
@@
 AR Path="/5F2C887E/5F68D900" Ref="C901"  Part="1"
 F 0 "C901" H 6142 4846 50  0000 L CNN
-F 1 "0.1uF 3.3VDCbias" H 6142 4755 50  0000 L CNN
+F 1 "0.1uF" H 6142 4755 50  0000 L CNN
 F 2 "Capacitor_SMD:C_0603_1608Metric" H 6050 4800 50  0001 C CNN
 F 3 "~" H 6050 4800 50  0001 C CNN
@@
 F 5 "Samsung Electro-Mechanics" H 6050 4800 50  0001 C CNN "Mfg"
 F 6 "212-00011" H 6050 4800 50  0001 C CNN "CPN"
+F 7 "3.3V" H 6050 4800 50  0001 C CNN "C_Vbias"
 	1    6050 4800
 	1    0    0    -1

Commit message: gemini-bringup: reselect all caps respecting C/V derating
Parts:
- C901: Mfg Samsung Electro-Mechanics -> Kemet; Mfg Part Num CL10B104KB8NNWC -> C0603C104M4RACTU
Changed lines of the file:
@@
 F 2 "Capacitor_SMD:C_0603_1608Metric" H 6050 4800 50  0001 C CNN
 F 3 "~" H 6050 4800 50  0001 C CNN
-F 4 "CL10B104KB8NNWC" H 6050 4800 50  0001 C CNN "Mfg Part Num"
-F 5 "Samsung Electro-Mechanics" H 6050 4800 50  0001 C CNN "Mfg"
+F 4 "C0603C104M4RACTU" H 6050 4800 50  0001 C CNN "Mfg Part Num"
+F 5 "Kemet" H 6050 4800 50  0001 C CNN "Mfg"
 F 6 "212-00011" H 6050 4800 50  0001 C CNN "CPN"
 F 7 "3.3V" H 6050 4800 50  0001 C CNN "C_Vbias"
