File: lpc55_carrier.sch (KiCad schematic (older format))
At the start: 48 parts, among them J101 Conn_2Rows-51Pins, U101 LPC55S28JBD64, Y101 16MHz, Y102 32.768kHz

Commit message: lpc55_carrier: Power/voltage/tolerance/etc ratings for passives
Update footprints accordingly.
Parts:
- C101, C113: value 4.7uF -> 4.7uF 16V; footprint Capacitor_SMD:C_0603_1608Metric -> Capacitor_SMD:C_0805_2012Metric
- C102, C104, C106, C108, C111, C115, C118: value 0.1uF -> 0.1uF 16V
- C103, C105, C107, C109, C116, C125: value 10nF -> 10000pF 16V
- C110, C114, C119: value 47pF -> 47pF 16V
- C112: value 2.2uF -> 2.2uF 6.3V; footprint Capacitor_SMD:C_0603_1608Metric -> Capacitor_SMD:C_0805_2012Metric
- C117, C120: value 22uF -> 22uF 16V; footprint Capacitor_SMD:C_0805_2012Metric -> Capacitor_SMD:C_1210_3225Metric
- C121, C122: value 18pF -> 18pF 16V
- C123, C124: value 12pF -> 12pF 16V
- D103: value D -> 1.25Vf 150mA
- FB101, FB102: value 600R -> 600R @ 100MHz 10mA
- L101: value 4.7uH -> 4.7uH 400mA 290mR
- Y101: value 16MHz -> 16MHz 18pF
- Y102: value 32.768kHz -> 32.768kHz 12.5pF
Changed lines of the file:
@@
 P 2300 4750
 F 0 "Y101" H 2300 5150 50  0000 C CNN
-F 1 "16MHz" H 2300 5050 50  0000 C CNN
+F 1 "16MHz 18pF" H 2300 5050 50  0000 C CNN
 F 2 "Crystal:Crystal_SMD_5032-4Pin_5.0x3.2mm" H 2300 4750 50  0001 C CNN
 F 3 "~" H 2300 4750 50  0001 C CNN
@@
 P 1950 5000
 F 0 "C121" H 1800 5050 50  0000 R CNN
-F 1 "18pF" H 1800 5000 50  0000 R CNN
+F 1 "18pF 16V" H 1800 5000 50  0000 R CNN
 F 2 "Capacitor_SMD:C_0603_1608Metric" H 1988 4850 50  0001 C CNN
 F 3 "~" H 1950 5000 50  0001 C CNN
@@
 P 2600 5000
 F 0 "C122" H 2750 5050 50  0000 L CNN
-F 1 "18pF" H 2750 5000 50  0000 L CNN
+F 1 "18pF 16V" H 2750 5000 50  0000 L CNN
 F 2 "Capacitor_SMD:C_0603_1608Metric" H 2638 4850 50  0001 C CNN
 F 3 "~" H 2600 5000 50  0001 C CNN
@@
 P 2300 6450
 F 0 "Y102" H 2300 6750 50  0000 C CNN
-F 1 "32.768kHz" H 2300 6650 50  0000 C CNN
+F 1 "32.768kHz 12.5pF" H 2300 6650 50  0000 C CNN
 F 2 "Crystal:Crystal_SMD_3215-2Pin_3.2x1.5mm" H 2300 6450 50  0001 C CNN
 F 3 "~" H 2300 6450 50  0001 C CNN
@@
 P 1950 6700
 F 0 "C123" H 2100 6750 50  0000 L CNN
-F 1 "12pF" H 2100 6700 50  0000 L CNN
+F 1 "12pF 16V" H 2100 6700 50  0000 L CNN
 F 2 "Capacitor_SMD:C_0603_1608Metric" H 1988 6550 50  0001 C CNN
 F 3 "~" H 1950 6700 50  0001 C CNN
@@
 P 2600 6700
 F 0 "C124" H 2750 6750 50  0000 L CNN
-F 1 "12pF" H 2750 6700 50  0000 L CNN
+F 1 "12pF 16V" H 2750 6700 50  0000 L CNN
 F 2 "Capacitor_SMD:C_0603_1608Metric" H 2638 6550 50  0001 C CNN
 F 3 "~" H 2600 6700 50  0001 C CNN
@@
 P 4550 8550
 F 0 "C125" H 4700 8600 50  0000 L CNN
-F 1 "10nF" H 4700 8550 50  0000 L CNN
+F 1 "10000pF 16V" H 4700 8550 50  0000 L CNN
 F 2 "Capacitor_SMD:C_0603_1608Metric" H 4588 8400 50  0001 C CNN
 F 3 "~" H 4550 8550 50  0001 C CNN
@@
 P 13500 2900
 F 0 "L101" V 13400 2900 50  0000 C CNN
-F 1 "4.7uH" V 13300 2900 50  0000 C CNN
+F 1 "4.7uH 400mA 290mR" V 13300 2900 50  0000 C CNN
 F 2 "Inductor_SMD:L_0805_2012Metric" H 13500 2900 50  0001 C CNN
 F 3 "~" H 13500 2900 50  0001 C CNN
@@
 P 13950 3100
 F 0 "C120" H 14100 3150 50  0000 L CNN
-F 1 "22uF" H 14100 3100 50  0000 L CNN
-F 2 "Capacitor_SMD:C_0805_2012Metric" H 13988 2950 50  0001 C CNN
+F 1 "22uF 16V" H 14100 3100 50  0000 L CNN
+F 2 "Capacitor_SMD:C_1210_3225Metric" H 13988 2950 50  0001 C CNN
 F 3 "~" H 13950 3100 50  0001 C CNN
 F 4 "212-00016" H 13950 3100 50  0001 C CNN "CPN"
@@
 P 12600 2250
 F 0 "C110" H 12750 2300 50  0000 L CNN
-F 1 "47pF" H 12750 2250 50  0000 L CNN
+F 1 "47pF 16V" H 12750 2250 50  0000 L CNN
 F 2 "Capacitor_SMD:C_0603_1608Metric" H 12638 2100 50  0001 C CNN
 F 3 "~" H 12600 2250 50  0001 C CNN
@@
 P 13050 2250
 F 0 "C111" H 13200 2300 50  0000 L CNN
-F 1 "0.1uF" H 13200 2250 50  0000 L CNN
+F 1 "0.1uF 16V" H 13200 2250 50  0000 L CNN
 F 2 "Capacitor_SMD:C_0603_1608Metric" H 13088 2100 50  0001 C CNN
 F 3 "~" H 13050 2250 50  0001 C CNN
@@
 P 13550 2250
 F 0 "C112" H 13700 2300 50  0000 L CNN
-F 1 "2.2uF" H 13700 2250 50  0000 L CNN
-F 2 "Capacitor_SMD:C_0603_1608Metric" H 13588 2100 50  0001 C CNN
+F 1 "2.2uF 6.3V" H 13700 2250 50  0000 L CNN
+F 2 "Capacitor_SMD:C_0805_2012Metric" H 13588 2100 50  0001 C CNN
 F 3 "~" H 13550 2250 50  0001 C CNN
 F 4 "212-00023" H 13550 2250 50  0001 C CNN "CPN"
@@
 P 2300 1750
 F 0 "FB101" V 2000 1750 50  0000 C CNN
-F 1 "600R" V 2100 1750 50  0000 C CNN
+F 1 "600R @ 100MHz 10mA" V 2100 1750 50  0000 C CNN
 F 2 "Inductor_SMD:L_0603_1608Metric" V 2230 1750 50  0001 C CNN
 F 3 "~" H 2300 1750 50  0001 C CNN
@@
 P 2900 1950
 F 0 "C101" H 3050 2000 50  0000 L CNN
-F 1 "4.7uF" H 3050 1950 50  0000 L CNN
-F 2 "Capacitor_SMD:C_0603_1608Metric" H 2938 1800 50  0001 C CNN
+F 1 "4.7uF 16V" H 3050 1950 50  0000 L CNN
+F 2 "Capacitor_SMD:C_0805_2012Metric" H 2938 1800 50  0001 C CNN
 F 3 "~" H 2900 1950 50  0001 C CNN
 F 4 "212-00013" H 2900 1950 50  0001 C CNN "CPN"
@@
 P 3350 1950
 F 0 "C102" H 3500 2000 50  0000 L CNN
-F 1 "0.1uF" H 3500 1950 50  0000 L CNN
+F 1 "0.1uF 16V" H 3500 1950 50  0000 L CNN
 F 2 "Capacitor_SMD:C_0603_1608Metric" H 3388 1800 50  0001 C CNN
 F 3 "~" H 3350 1950 50  0001 C CNN
@@
 P 3800 1950
 F 0 "C103" H 3950 2000 50  0000 L CNN
-F 1 "10nF" H 3950 1950 50  0000 L CNN
+F 1 "10000pF 16V" H 3950 1950 50  0000 L CNN
 F 2 "Capacitor_SMD:C_0603_1608Metric" H 3838 1800 50  0001 C CNN
 F 3 "~" H 3800 1950 50  0001 C CNN
@@
 P 4250 1950
 F 0 "C104" H 4400 2000 50  0000 L CNN
-F 1 "0.1uF" H 4400 1950 50  0000 L CNN
+F 1 "0.1uF 16V" H 4400 1950 50  0000 L CNN
 F 2 "Capacitor_SMD:C_0603_1608Metric" H 4288 1800 50  0001 C CNN
 F 3 "~" H 4250 1950 50  0001 C CNN
@@
 P 4700 1950
 F 0 "C105" H 4850 2000 50  0000 L CNN
-F 1 "10nF" H 4850 1950 50  0000 L CNN
+F 1 "10000pF 16V" H 4850 1950 50  0000 L CNN
 F 2 "Capacitor_SMD:C_0603_1608Metric" H 4738 1800 50  0001 C CNN
 F 3 "~" H 4700 1950 50  0001 C CNN
@@
 P 5200 1950
 F 0 "C106" H 5350 2000 50  0000 L CNN
-F 1 "0.1uF" H 5350 1950 50  0000 L CNN
+F 1 "0.1uF 16V" H 5350 1950 50  0000 L CNN
 F 2 "Capacitor_SMD:C_0603_1608Metric" H 5238 1800 50  0001 C CNN
 F 3 "~" H 5200 1950 50  0001 C CNN
@@
 P 5700 1950
 F 0 "C107" H 5850 2000 50  0000 L CNN
-F 1 "10nF" H 5850 1950 50  0000 L CNN
+F 1 "10000pF 16V" H 5850 1950 50  0000 L CNN
 F 2 "Capacitor_SMD:C_0603_1608Metric" H 5738 1800 50  0001 C CNN
 F 3 "~" H 5700 1950 50  0001 C CNN
@@
 P 6250 1950
 F 0 "C108" H 6400 2000 50  0000 L CNN
-F 1 "0.1uF" H 6400 1950 50  0000 L CNN
+F 1 "0.1uF 16V" H 6400 1950 50  0000 L CNN
 F 2 "Capacitor_SMD:C_0603_1608Metric" H 6288 1800 50  0001 C CNN
 F 3 "~" H 6250 1950 50  0001 C CNN
@@
 P 6800 1950
 F 0 "C109" H 6950 2000 50  0000 L CNN
-F 1 "10nF" H 6950 1950 50  0000 L CNN
+F 1 "10000pF 16V" H 6950 1950 50  0000 L CNN
 F 2 "Capacitor_SMD:C_0603_1608Metric" H 6838 1800 50  0001 C CNN
 F 3 "~" H 6800 1950 50  0001 C CNN
@@
 P 2300 2550
 F 0 "FB102" V 2000 2550 50  0000 C CNN
-F 1 "600R" V 2100 2550 50  0000 C CNN
+F 1 "600R @ 100MHz 10mA" V 2100 2550 50  0000 C CNN
 F 2 "Inductor_SMD:L_0603_1608Metric" V 2230 2550 50  0001 C CNN
 F 3 "~" H 2300 2550 50  0001 C CNN
@@
 P 3350 2750
 F 0 "C114" H 3500 2800 50  0000 L CNN
-F 1 "47pF" H 3500 2750 50  0000 L CNN
+F 1 "47pF 16V" H 3500 2750 50  0000 L CNN
 F 2 "Capacitor_SMD:C_0603_1608Metric" H 3388 2600 50  0001 C CNN
 F 3 "~" H 3350 2750 50  0001 C CNN
@@
 P 3800 2750
 F 0 "C115" H 3950 2800 50  0000 L CNN
-F 1 "0.1uF" H 3950 2750 50  0000 L CNN
+F 1 "0.1uF 16V" H 3950 2750 50  0000 L CNN
 F 2 "Capacitor_SMD:C_0603_1608Metric" H 3838 2600 50  0001 C CNN
 F 3 "~" H 3800 2750 50  0001 C CNN
@@
 P 4300 2750
 F 0 "C116" H 4450 2800 50  0000 L CNN
-F 1 "10nF" H 4450 2750 50  0000 L CNN
+F 1 "10000pF 16V" H 4450 2750 50  0000 L CNN
 F 2 "Capacitor_SMD:C_0603_1608Metric" H 4338 2600 50  0001 C CNN
 F 3 "~" H 4300 2750 50  0001 C CNN
@@
 P 4300 8150
 F 0 "D103" V 4250 8250 50  0000 L CNN
-F 1 "D" V 4300 8250 50  0000 L CNN
+F 1 "1.25Vf 150mA" V 4300 8250 50  0000 L CNN
 F 2 "Diode_SMD:D_SOD-323" H 4300 8150 50  0001 C CNN
 F 3 "~" H 4300 8150 50  0001 C CNN
@@
 P 4800 2750
 F 0 "C117" H 4950 2800 50  0000 L CNN
-F 1 "22uF" H 4950 2750 50  0000 L CNN
-F 2 "Capacitor_SMD:C_0805_2012Metric" H 4838 2600 50  0001 C CNN
+F 1 "22uF 16V" H 4950 2750 50  0000 L CNN
+F 2 "Capacitor_SMD:C_1210_3225Metric" H 4838 2600 50  0001 C CNN
 F 3 "~" H 4800 2750 50  0001 C CNN
 F 4 "212-00016" H 4800 2750 50  0001 C CNN "CPN"
@@
 P 5300 2750
 F 0 "C118" H 5450 2800 50  0000 L CNN
-F 1 "0.1uF" H 5450 2750 50  0000 L CNN
+F 1 "0.1uF 16V" H 5450 2750 50  0000 L CNN
 F 2 "Capacitor_SMD:C_0603_1608Metric" H 5338 2600 50  0001 C CNN
 F 3 "~" H 5300 2750 50  0001 C CNN
@@
 P 5850 2750
 F 0 "C119" H 6000 2800 50  0000 L CNN
-F 1 "47pF" H 6000 2750 50  0000 L CNN
+F 1 "47pF 16V" H 6000 2750 50  0000 L CNN
 F 2 "Capacitor_SMD:C_0603_1608Metric" H 5888 2600 50  0001 C CNN
 F 3 "~" H 5850 2750 50  0001 C CNN
@@
 P 2900 2750
 F 0 "C113" H 3050 2800 50  0000 L CNN
-F 1 "4.7uF" H 3050 2750 50  0000 L CNN
-F 2 "Capacitor_SMD:C_0603_1608Metric" H 2938 2600 50  0001 C CNN
+F 1 "4.7uF 16V" H 3050 2750 50  0000 L CNN
+F 2 "Capacitor_SMD:C_0805_2012Metric" H 2938 2600 50  0001 C CNN
 F 3 "~" H 2900 2750 50  0001 C CNN
 F 4 "212-00013" H 2900 2750 50  0001 C CNN "CPN"

Commit message: lpc55_carrier: document POR pin modes
Other:
- note added: "-\nPD\nPU\nPD\nPU"
- note added: "Default\nPIO0_2\nPIO0_5\nPIO0_11\nPIO0_12"
- note added: "Input/Output/Hi-Z"
- note added: "POR Pin Mode"
- note added: "Pin"
- note added: "Pull up/down"
- note added: "Z\nI\nI\nI\nI"
Changed lines of the file:
@@
 Wire Wire Line
 	1850 1750 2000 1750
+Text Notes 9000 1850 0    50   ~ 0
+Default\nPIO0_2\nPIO0_5\nPIO0_11\nPIO0_12
+Text Notes 9700 1850 0    50   ~ 0
+-\nPD\nPU\nPD\nPU
+Text Notes 10550 1850 0    50   ~ 0
+Z\nI\nI\nI\nI
+Text Notes 9050 1400 0    50   Italic 0
+Pin
+Text Notes 9500 1400 0    50   Italic 0
+Pull up/down
+Text Notes 10200 1400 0    50   Italic 0
+Input/Output/Hi-Z
+Text Notes 9600 1250 0    50   ~ 10
+POR Pin Mode
+Wire Notes Line
+	8950 1150 11000 1150
+Wire Notes Line
+	11000 1900 8950 1900
+Wire Notes Line
+	8950 1900 8950 1150
+Wire Notes Line
+	8950 1300 11000 1300
+Wire Notes Line
+	11000 1150 11000 1900
+Wire Notes Line
+	8950 1450 11000 1450
 $EndSCHEMATC

Commit message: lpc55_carrier: remove external ISP0 pull-up as internal is enabled by default
Parts:
- removed R111: 100kR, Resistor_SMD:R_0603_1608Metric, symbol Device:R
Connections:
- wire segments 250 -> 247
Other:
- note added: "ISP0"
- note removed: "Recovery"
Changed lines of the file:
@@
 Text Label 10050 3950 2    50   ~ 0
 ISP0
-Text Label 3050 11350 0    50   ~ 0
-ISP0
-Text Notes 2750 11600 0    50   ~ 0
+Text Notes 8200 4150 0    50   ~ 0
 Default to Passive Boot.\nPull LOW for ISP boot.
-Text Notes 1350 11800 0    50   ~ 10
-Recovery
-Wire Notes Line
-	1250 11950 3900 11950
-Wire Notes Line
-	3900 11950 3900 10550
-Wire Notes Line
-	3900 10550 1250 10550
-Wire Notes Line
-	1250 10550 1250 11950
 Text Label 10050 3650 2    50   ~ 0
 FC3_TXD_SCL_MISO
@@
 Text Label 13200 2800 0    50   ~ 0
 FB
-$Comp
-L Device:R R111
-U 1 1 5F3C1231
-P 2400 11100
-F 0 "R111" H 2500 11150 50  0000 L CNN
-F 1 "100kR" H 2500 11100 50  0000 L CNN
-F 2 "Resistor_SMD:R_0603_1608Metric" V 2330 11100 50  0001 C CNN
-F 3 "~" H 2400 11100 50  0001 C CNN
-F 4 "232-00021" H 2400 11100 50  0001 C CNN "CPN"
-	1    2400 11100
-	1    0    0    -1
-$EndComp
-Wire Wire Line
-	2400 11250 2400 11350
-Wire Wire Line
-	2400 10950 2400 10900
-Wire Wire Line
-	2400 11350 3050 11350
 $Comp
 L Device:D D103
@@
 Text Label 3950 8900 1    50   ~ 0
 VDD
-Text Label 2400 10900 1    50   ~ 0
-VDD
 $Comp
 L Device:C C113
@@
 Wire Notes Line
 	8950 1450 11000 1450
+Text Notes 8200 3900 0    50   ~ 10
+ISP0
+Wire Notes Line
+	8150 3750 9200 3750
+Wire Notes Line
+	9200 3750 9200 4200
+Wire Notes Line
+	9200 4200 8150 4200
+Wire Notes Line
+	8150 4200 8150 3750
 $EndSCHEMATC

Commit message: lpc55_carrier: remove external pullups on SWD as internal pull-up/down are enabled at POR
Parts:
- removed R105, R106, R107: 100kR, Resistor_SMD:R_0603_1608Metric, symbol Device:R
Connections:
- wire segments 247 -> 235
Changed lines of the file:
@@
 $EndComp
-$Comp
-L Device:R R105
-U 1 1 5F7E38EA
-P 3550 9200
-F 0 "R105" H 3650 9250 50  0000 L CNN
-F 1 "100kR" H 3650 9200 50  0000 L CNN
-F 2 "Resistor_SMD:R_0603_1608Metric" V 3480 9200 50  0001 C CNN
-F 3 "~" H 3550 9200 50  0001 C CNN
-F 4 "232-00021" H 3550 9200 50  0001 C CNN "CPN"
-	1    3550 9200
-	1    0    0    -1
-$EndComp
-$Comp
-L Device:R R106
-U 1 1 5F7E3EBA
-P 3950 9200
-F 0 "R106" H 4050 9250 50  0000 L CNN
-F 1 "100kR" H 4050 9200 50  0000 L CNN
-F 2 "Resistor_SMD:R_0603_1608Metric" V 3880 9200 50  0001 C CNN
-F 3 "~" H 3950 9200 50  0001 C CNN
-F 4 "232-00021" H 3950 9200 50  0001 C CNN "CPN"
-	1    3950 9200
-	1    0    0    -1
-$EndComp
-$Comp
-L Device:R R107
-U 1 1 5F7E437C
-P 4350 9200
-F 0 "R107" H 4450 9250 50  0000 L CNN
-F 1 "100kR" H 4450 9200 50  0000 L CNN
-F 2 "Resistor_SMD:R_0603_1608Metric" V 4280 9200 50  0001 C CNN
-F 3 "~" H 4350 9200 50  0001 C CNN
-F 4 "232-00021" H 4350 9200 50  0001 C CNN "CPN"
-	1    4350 9200
-	1    0    0    -1
-$EndComp
-Wire Wire Line
-	3550 9350 3550 9400
-Wire Wire Line
-	3950 9350 3950 9750
-Wire Wire Line
-	4350 9350 4350 10100
-Wire Wire Line
-	3550 9050 3550 8950
-Wire Wire Line
-	3950 9050 3950 8950
-Wire Wire Line
-	3950 8950 3550 8950
-Wire Wire Line
-	4350 9050 4350 8950
-Wire Wire Line
-	4350 8950 3950 8950
-Connection ~ 3950 8950
 $Comp
 L Device:R R104
@@
 	4300 7900 4550 7900
 Wire Wire Line
-	3950 8950 3950 8900
-Wire Wire Line
 	3250 8350 4300 8350
-Wire Wire Line
-	3250 9400 3550 9400
-Wire Wire Line
-	3250 9750 3950 9750
-Wire Wire Line
-	3250 10100 4350 10100
 Text Label 5200 10100 0    50   ~ 0
 PIO0_10
@@
 Wire Wire Line
 	2600 10100 2950 10100
-Connection ~ 3550 9400
-Wire Wire Line
-	3550 9400 5200 9400
-Connection ~ 3950 9750
-Wire Wire Line
-	3950 9750 5200 9750
-Connection ~ 4350 10100
-Wire Wire Line
-	4350 10100 5200 10100
 Text Label 13250 6750 0    50   ~ 0
 VDDA
@@
 	13250 7400 13250 7250
 Text Label 4550 7800 1    50   ~ 0
-VDD
-Text Label 3950 8900 1    50   ~ 0
 VDD
 $Comp
@@
 Wire Notes Line
 	8150 4200 8150 3750
+Wire Wire Line
+	3250 9400 5200 9400
+Wire Wire Line
+	3250 9750 5200 9750
+Wire Wire Line
+	3250 10100 5200 10100
 $EndSCHEMATC

Commit message: lpc55_carrier: document capacitor DC bias rather than voltage rating required due to derating
Parts:
- C101, C113: value 4.7uF 16V -> 4.7uF 3.3VDCbias
- C102, C104, C106, C108, C115, C118: value 0.1uF 16V -> 0.1uF 3.3VDCbias
- C103, C105, C107, C109, C116, C125: value 10000pF 16V -> 10000pF 3.3VDCbias
- C110: value 47pF 16V -> 47pF 1.2VDCbias
- C111: value 0.1uF 16V -> 0.1uF 1.2VDCbias
- C112: value 2.2uF 6.3V -> 2.2uF 1.2VDCbias
- C114, C119: value 47pF 16V -> 47pF 3.3VDCbias
- C117: value 22uF 16V -> 22uF 3.3VDCbias
- C120: value 22uF 16V -> 22uF 1.2VDCbias
- C121, C122: value 18pF 16V -> 18pF 6.3V
- C123, C124: value 12pF 16V -> 12pF 6.3V
Changed lines of the file:
@@
 P 1950 5000
 F 0 "C121" H 1800 5050 50  0000 R CNN
-F 1 "18pF 16V" H 1800 5000 50  0000 R CNN
+F 1 "18pF 6.3V" H 1800 5000 50  0000 R CNN
 F 2 "Capacitor_SMD:C_0603_1608Metric" H 1988 4850 50  0001 C CNN
 F 3 "~" H 1950 5000 50  0001 C CNN
@@
 P 2600 5000
 F 0 "C122" H 2750 5050 50  0000 L CNN
-F 1 "18pF 16V" H 2750 5000 50  0000 L CNN
+F 1 "18pF 6.3V" H 2750 5000 50  0000 L CNN
 F 2 "Capacitor_SMD:C_0603_1608Metric" H 2638 4850 50  0001 C CNN
 F 3 "~" H 2600 5000 50  0001 C CNN
@@
 P 1950 6700
 F 0 "C123" H 2100 6750 50  0000 L CNN
-F 1 "12pF 16V" H 2100 6700 50  0000 L CNN
+F 1 "12pF 6.3V" H 2100 6700 50  0000 L CNN
 F 2 "Capacitor_SMD:C_0603_1608Metric" H 1988 6550 50  0001 C CNN
 F 3 "~" H 1950 6700 50  0001 C CNN
@@
 P 2600 6700
 F 0 "C124" H 2750 6750 50  0000 L CNN
-F 1 "12pF 16V" H 2750 6700 50  0000 L CNN
+F 1 "12pF 6.3V" H 2750 6700 50  0000 L CNN
 F 2 "Capacitor_SMD:C_0603_1608Metric" H 2638 6550 50  0001 C CNN
 F 3 "~" H 2600 6700 50  0001 C CNN
@@
 P 4550 8550
 F 0 "C125" H 4700 8600 50  0000 L CNN
-F 1 "10000pF 16V" H 4700 8550 50  0000 L CNN
+F 1 "10000pF 3.3VDCbias" H 4700 8550 50  0000 L CNN
 F 2 "Capacitor_SMD:C_0603_1608Metric" H 4588 8400 50  0001 C CNN
 F 3 "~" H 4550 8550 50  0001 C CNN
@@
 P 13950 3100
 F 0 "C120" H 14100 3150 50  0000 L CNN
-F 1 "22uF 16V" H 14100 3100 50  0000 L CNN
+F 1 "22uF 1.2VDCbias" H 14100 3100 50  0000 L CNN
 F 2 "Capacitor_SMD:C_1210_3225Metric" H 13988 2950 50  0001 C CNN
 F 3 "~" H 13950 3100 50  0001 C CNN
@@
 P 12600 2250
 F 0 "C110" H 12750 2300 50  0000 L CNN
-F 1 "47pF 16V" H 12750 2250 50  0000 L CNN
+F 1 "47pF 1.2VDCbias" H 12750 2250 50  0000 L CNN
 F 2 "Capacitor_SMD:C_0603_1608Metric" H 12638 2100 50  0001 C CNN
 F 3 "~" H 12600 2250 50  0001 C CNN
@@
 P 13050 2250
 F 0 "C111" H 13200 2300 50  0000 L CNN
-F 1 "0.1uF 16V" H 13200 2250 50  0000 L CNN
+F 1 "0.1uF 1.2VDCbias" H 13200 2250 50  0000 L CNN
 F 2 "Capacitor_SMD:C_0603_1608Metric" H 13088 2100 50  0001 C CNN
 F 3 "~" H 13050 2250 50  0001 C CNN
@@
 P 13550 2250
 F 0 "C112" H 13700 2300 50  0000 L CNN
-F 1 "2.2uF 6.3V" H 13700 2250 50  0000 L CNN
+F 1 "2.2uF 1.2VDCbias" H 13700 2250 50  0000 L CNN
 F 2 "Capacitor_SMD:C_0805_2012Metric" H 13588 2100 50  0001 C CNN
 F 3 "~" H 13550 2250 50  0001 C CNN
@@
 P 2900 1950
 F 0 "C101" H 3050 2000 50  0000 L CNN
-F 1 "4.7uF 16V" H 3050 1950 50  0000 L CNN
+F 1 "4.7uF 3.3VDCbias" H 3050 1950 50  0000 L CNN
 F 2 "Capacitor_SMD:C_0805_2012Metric" H 2938 1800 50  0001 C CNN
 F 3 "~" H 2900 1950 50  0001 C CNN
@@
 P 3350 1950
 F 0 "C102" H 3500 2000 50  0000 L CNN
-F 1 "0.1uF 16V" H 3500 1950 50  0000 L CNN
+F 1 "0.1uF 3.3VDCbias" H 3500 1950 50  0000 L CNN
 F 2 "Capacitor_SMD:C_0603_1608Metric" H 3388 1800 50  0001 C CNN
 F 3 "~" H 3350 1950 50  0001 C CNN
@@
 P 3800 1950
 F 0 "C103" H 3950 2000 50  0000 L CNN
-F 1 "10000pF 16V" H 3950 1950 50  0000 L CNN
+F 1 "10000pF 3.3VDCbias" H 3950 1950 50  0000 L CNN
 F 2 "Capacitor_SMD:C_0603_1608Metric" H 3838 1800 50  0001 C CNN
 F 3 "~" H 3800 1950 50  0001 C CNN
@@
 P 4250 1950
 F 0 "C104" H 4400 2000 50  0000 L CNN
-F 1 "0.1uF 16V" H 4400 1950 50  0000 L CNN
+F 1 "0.1uF 3.3VDCbias" H 4400 1950 50  0000 L CNN
 F 2 "Capacitor_SMD:C_0603_1608Metric" H 4288 1800 50  0001 C CNN
 F 3 "~" H 4250 1950 50  0001 C CNN
@@
 P 4700 1950
 F 0 "C105" H 4850 2000 50  0000 L CNN
-F 1 "10000pF 16V" H 4850 1950 50  0000 L CNN
+F 1 "10000pF 3.3VDCbias" H 4850 1950 50  0000 L CNN
 F 2 "Capacitor_SMD:C_0603_1608Metric" H 4738 1800 50  0001 C CNN
 F 3 "~" H 4700 1950 50  0001 C CNN
@@
 P 5200 1950
 F 0 "C106" H 5350 2000 50  0000 L CNN
-F 1 "0.1uF 16V" H 5350 1950 50  0000 L CNN
+F 1 "0.1uF 3.3VDCbias" H 5350 1950 50  0000 L CNN
 F 2 "Capacitor_SMD:C_0603_1608Metric" H 5238 1800 50  0001 C CNN
 F 3 "~" H 5200 1950 50  0001 C CNN
@@
 P 5700 1950
 F 0 "C107" H 5850 2000 50  0000 L CNN
-F 1 "10000pF 16V" H 5850 1950 50  0000 L CNN
+F 1 "10000pF 3.3VDCbias" H 5850 1950 50  0000 L CNN
 F 2 "Capacitor_SMD:C_0603_1608Metric" H 5738 1800 50  0001 C CNN
 F 3 "~" H 5700 1950 50  0001 C CNN
@@
 P 6250 1950
 F 0 "C108" H 6400 2000 50  0000 L CNN
-F 1 "0.1uF 16V" H 6400 1950 50  0000 L CNN
+F 1 "0.1uF 3.3VDCbias" H 6400 1950 50  0000 L CNN
 F 2 "Capacitor_SMD:C_0603_1608Metric" H 6288 1800 50  0001 C CNN
 F 3 "~" H 6250 1950 50  0001 C CNN
@@
 P 6800 1950
 F 0 "C109" H 6950 2000 50  0000 L CNN
-F 1 "10000pF 16V" H 6950 1950 50  0000 L CNN
+F 1 "10000pF 3.3VDCbias" H 6950 1950 50  0000 L CNN
 F 2 "Capacitor_SMD:C_0603_1608Metric" H 6838 1800 50  0001 C CNN
 F 3 "~" H 6800 1950 50  0001 C CNN
@@
 P 3350 2750
 F 0 "C114" H 3500 2800 50  0000 L CNN
-F 1 "47pF 16V" H 3500 2750 50  0000 L CNN
+F 1 "47pF 3.3VDCbias" H 3500 2750 50  0000 L CNN
 F 2 "Capacitor_SMD:C_0603_1608Metric" H 3388 2600 50  0001 C CNN
 F 3 "~" H 3350 2750 50  0001 C CNN
@@
 P 3800 2750
 F 0 "C115" H 3950 2800 50  0000 L CNN
-F 1 "0.1uF 16V" H 3950 2750 50  0000 L CNN
+F 1 "0.1uF 3.3VDCbias" H 3950 2750 50  0000 L CNN
 F 2 "Capacitor_SMD:C_0603_1608Metric" H 3838 2600 50  0001 C CNN
 F 3 "~" H 3800 2750 50  0001 C CNN
@@
 P 4300 2750
 F 0 "C116" H 4450 2800 50  0000 L CNN
-F 1 "10000pF 16V" H 4450 2750 50  0000 L CNN
+F 1 "10000pF 3.3VDCbias" H 4450 2750 50  0000 L CNN
 F 2 "Capacitor_SMD:C_0603_1608Metric" H 4338 2600 50  0001 C CNN
 F 3 "~" H 4300 2750 50  0001 C CNN
@@
 P 4800 2750
 F 0 "C117" H 4950 2800 50  0000 L CNN
-F 1 "22uF 16V" H 4950 2750 50  0000 L CNN
+F 1 "22uF 3.3VDCbias" H 4950 2750 50  0000 L CNN
 F 2 "Capacitor_SMD:C_1210_3225Metric" H 4838 2600 50  0001 C CNN
 F 3 "~" H 4800 2750 50  0001 C CNN
@@
 P 5300 2750
 F 0 "C118" H 5450 2800 50  0000 L CNN
-F 1 "0.1uF 16V" H 5450 2750 50  0000 L CNN
+F 1 "0.1uF 3.3VDCbias" H 5450 2750 50  0000 L CNN
 F 2 "Capacitor_SMD:C_0603_1608Metric" H 5338 2600 50  0001 C CNN
 F 3 "~" H 5300 2750 50  0001 C CNN
@@
 P 5850 2750
 F 0 "C119" H 6000 2800 50  0000 L CNN
-F 1 "47pF 16V" H 6000 2750 50  0000 L CNN
+F 1 "47pF 3.3VDCbias" H 6000 2750 50  0000 L CNN
 F 2 "Capacitor_SMD:C_0603_1608Metric" H 5888 2600 50  0001 C CNN
 F 3 "~" H 5850 2750 50  0001 C CNN
@@
 P 2900 2750
 F 0 "C113" H 3050 2800 50  0000 L CNN
-F 1 "4.7uF 16V" H 3050 2750 50  0000 L CNN
+F 1 "4.7uF 3.3VDCbias" H 3050 2750 50  0000 L CNN
 F 2 "Capacitor_SMD:C_0805_2012Metric" H 2938 2600 50  0001 C CNN
 F 3 "~" H 2900 2750 50  0001 C CNN
