File: lpc55_carrier.sch (KiCad schematic (older format))
At the start: 44 parts, among them J101 Conn_2Rows-51Pins, U101 LPC55S28JBD64, Y101 16MHz 18pF, Y102 32.768kHz 12.5pF

Commit message: lpc55_carrier: series terminate SP->RoT SPI drivers (MISO)
Parts:
- added R101: 22R, Resistor_SMD:R_0603_1608Metric, symbol Device:R
Connections:
- net labels added: PIO0_18, PIO0_26, PIO1_1, PIO1_2, PIO1_3
- wire segments 235 -> 241
Other:
- note added: "SP->RoT SPI"
- moved on the sheet: H101, H102
Changed lines of the file:
@@
 Wire Notes Line
 	1200 3750 1200 7300
-Text Label 10050 6050 2    50   ~ 0
-HS_SPI_MOSI
 Text Label 13150 3650 0    50   ~ 0
-HS_SPI_SCK
+PIO1_2
 Text Label 13150 3750 0    50   ~ 0
-HS_SPI_MISO
+PIO1_3
 Text Label 13150 3550 0    50   ~ 0
-~HS_SPI_SSEL1
+PIO1_1
 Text Label 10050 5250 2    50   ~ 0
-~HS_SPI_IRQ
+PIO0_18
 $Comp
 L Device:R R108
@@
 L Mechanical:MountingHole H101
 U 1 1 5F8EE4E5
-P 1600 12650
-F 0 "H101" H 1700 12700 50  0000 L CNN
-F 1 "M3" H 1700 12650 50  0000 L CNN
-F 2 "MountingHole:MountingHole_3.2mm_M3" H 1600 12650 50  0001 C CNN
-F 3 "~" H 1600 12650 50  0001 C CNN
-	1    1600 12650
+P 1550 13200
+F 0 "H101" H 1650 13250 50  0000 L CNN
+F 1 "M3" H 1650 13200 50  0000 L CNN
+F 2 "MountingHole:MountingHole_3.2mm_M3" H 1550 13200 50  0001 C CNN
+F 3 "~" H 1550 13200 50  0001 C CNN
+	1    1550 13200
 	1    0    0    -1
 $EndComp
@@
 L Mechanical:MountingHole H102
 U 1 1 5F8EF079
-P 2000 12650
-F 0 "H102" H 2100 12700 50  0000 L CNN
-F 1 "M3" H 2100 12650 50  0000 L CNN
-F 2 "MountingHole:MountingHole_3.2mm_M3" H 2000 12650 50  0001 C CNN
-F 3 "~" H 2000 12650 50  0001 C CNN
-	1    2000 12650
-	1    0    0    -1
-$EndComp
-Wire Notes Line
-	1250 12400 3900 12400
-Wire Notes Line
-	3900 12400 3900 13050
-Wire Notes Line
-	3900 13050 1250 13050
-Wire Notes Line
-	1250 13050 1250 12400
-Text Notes 1350 12950 0    50   ~ 10
+P 1950 13200
+F 0 "H102" H 2050 13250 50  0000 L CNN
+F 1 "M3" H 2050 13200 50  0000 L CNN
+F 2 "MountingHole:MountingHole_3.2mm_M3" H 1950 13200 50  0001 C CNN
+F 3 "~" H 1950 13200 50  0001 C CNN
+	1    1950 13200
+	1    0    0    -1
+$EndComp
+Wire Notes Line
+	1200 12950 3850 12950
+Wire Notes Line
+	3850 12950 3850 13600
+Wire Notes Line
+	3850 13600 1200 13600
+Wire Notes Line
+	1200 13600 1200 12950
+Text Notes 1300 13500 0    50   ~ 10
 Mounting
 Connection ~ 2700 1750
@@
 Wire Wire Line
 	3250 10100 5200 10100
+Text Label 2750 10800 2    50   ~ 0
+~HS_SPI_SSEL1
+Text Label 3500 10800 0    50   ~ 0
+PIO1_1
+Wire Wire Line
+	3500 10800 2750 10800
+Text Label 2750 11200 2    50   ~ 0
+HS_SPI_SCK
+Text Label 3500 11200 0    50   ~ 0
+PIO1_2
+Wire Wire Line
+	3500 11200 2750 11200
+Text Label 3500 11600 0    50   ~ 0
+PIO1_3
+$Comp
+L Device:R R101
+U 1 1 5FA9ABD5
+P 3100 11600
+F 0 "R101" V 2850 11600 50  0000 C CNN
+F 1 "22R" V 2950 11600 50  0000 C CNN
+F 2 "Resistor_SMD:R_0603_1608Metric" V 3030 11600 50  0001 C CNN
+F 3 "~" H 3100 11600 50  0001 C CNN
+	1    3100 11600
+	0    -1   1    0
+$EndComp
+Wire Wire Line
+	3500 11600 3250 11600
+Wire Wire Line
+	2950 11600 2750 11600
+Text Label 2750 11600 2    50   ~ 0
+HS_SPI_MISO
+Text Label 3500 12400 0    50   ~ 0
+PIO0_18
+Wire Wire Line
+	3500 12400 2750 12400
+Text Label 2750 12400 2    50   ~ 0
+~HS_SPI_IRQ
+Text Label 3500 12000 0    50   ~ 0
+PIO0_26
+Wire Wire Line
+	3500 12000 2750 12000
+Text Label 10050 6050 2    50   ~ 0
+PIO0_26
+Text Label 2750 12000 2    50   ~ 0
+HS_SPI_MOSI
+Text Notes 1300 12650 0    50   ~ 10
+SP->RoT SPI
+Wire Notes Line
+	1200 10400 5800 10400
+Wire Notes Line
+	5800 10400 5800 12700
+Wire Notes Line
+	5800 12700 1200 12700
+Wire Notes Line
+	1200 12700 1200 10400
 $EndSCHEMATC

Commit message: lpc55_carrier: document use of internal pull-ups on SP->RoT SPI
Other:
- note added: "~HS_SPI_SSEL1~ and ~HS_SPI_IRQ~\nmust have internal pull-ups enabled"
Changed lines of the file:
@@
 Wire Notes Line
 	1200 12700 1200 10400
+Text Notes 4200 10900 0    50   ~ 0
+~HS_SPI_SSEL1~ and ~HS_SPI_IRQ~\nmust have internal pull-ups enabled
 $EndSCHEMATC

Commit message: lpc55_carrier: change SWD current limit resistors to 22R
This is sole use of 100R while 22R is used for series termination in
many places.

3.3V / 22R = 0.150A
Parts:
- R104, R108, R109, R110: value 100R -> 22R
Changed lines of the file:
@@
 P 3100 9400
 F 0 "R108" V 2850 9400 50  0000 C CNN
-F 1 "100R" V 2950 9400 50  0000 C CNN
+F 1 "22R" V 2950 9400 50  0000 C CNN
 F 2 "Resistor_SMD:R_0603_1608Metric" V 3030 9400 50  0001 C CNN
 F 3 "~" H 3100 9400 50  0001 C CNN
@@
 P 3100 8350
 F 0 "R104" V 2850 8350 50  0000 C CNN
-F 1 "100R" V 2950 8350 50  0000 C CNN
+F 1 "22R" V 2950 8350 50  0000 C CNN
 F 2 "Resistor_SMD:R_0603_1608Metric" V 3030 8350 50  0001 C CNN
 F 3 "~" H 3100 8350 50  0001 C CNN
@@
 P 3100 9750
 F 0 "R109" V 2850 9750 50  0000 C CNN
-F 1 "100R" V 2950 9750 50  0000 C CNN
+F 1 "22R" V 2950 9750 50  0000 C CNN
 F 2 "Resistor_SMD:R_0603_1608Metric" V 3030 9750 50  0001 C CNN
 F 3 "~" H 3100 9750 50  0001 C CNN
@@
 P 3100 10100
 F 0 "R110" V 2850 10100 50  0000 C CNN
-F 1 "100R" V 2950 10100 50  0000 C CNN
+F 1 "22R" V 2950 10100 50  0000 C CNN
 F 2 "Resistor_SMD:R_0603_1608Metric" V 3030 10100 50  0001 C CNN
 F 3 "~" H 3100 10100 50  0001 C CNN
