File: lpc55_carrier.kicad_pcb (KiCad board)
At the start: 4 copper layers, 50 parts, among them J101 Conn_2Rows-51Pins, U101 LPC55S28JBD64, Y101 16MHz, Y102 32.768kHz

Commit message: lpc55_carrier: all nets routed
Parts:
- removed D101, D102: LED, LED_SMD:LED_0603_1608Metric
- removed R101, R102: 330R, Resistor_SMD:R_0603_1608Metric
- moved J101 83.4 mm to (110.7, 68.3), turned to 0 degrees
- moved R104 72.6 mm to (106.2, 78.0), turned to 90 degrees
- moved R109 71.5 mm to (104.6, 78.0), turned to 90 degrees
- moved R108 69.8 mm to (103.1, 78.0), turned to 90 degrees
- moved R110 68.8 mm to (101.6, 78.0), turned to 90 degrees
- moved FB102 56.0 mm to (89.9, 80.5), turned to 270 degrees
- moved FB101 54.3 mm to (87.4, 85.0), turned to 0 degrees
- moved C113 49.6 mm to (88.1, 80.5), turned to 270 degrees
- moved C101 48.5 mm to (86.6, 82.1), turned to 90 degrees
- moved R106 39.3 mm to (104.6, 82.0), turned to 90 degrees
- moved R105 37.1 mm to (103.1, 82.0), turned to 90 degrees
- moved R107 29.8 mm to (101.6, 82.0), turned to 90 degrees
- moved C121 13.1 mm to (69.7, 83.1), turned to 180 degrees
- moved C124 11.9 mm to (104.6, 71.6), turned to 90 degrees
- moved C122 9.24 mm to (69.7, 74.5), turned to 180 degrees
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Connections:
- J101 pad 1: +3V3 -> GND
- J101 pad 11: GND -> /HS_SPI_SCK
- J101 pad 12: /FC3_CTS_SDAX_SSEL0 -> /FC3_RXD_DSA_MOSI
- J101 pad 13: /SWD_CLK -> GND
- J101 pad 15: GND -> /HS_SPI_MOSI
- J101 pad 16: /FC3_RTS_SCLX_SSEL1 -> /FC3_TXD_SCL_MISO
- J101 pad 17: /SWD_IO -> GND
- J101 pad 19: GND -> /~HS_SPI_SSEL1
- J101 pad 2: +3V3 -> GND
- J101 pad 20: /PIO0_22 -> /PIO0_25
- J101 pad 21: /SWD_TRACESWO -> GND
- J101 pad 23: GND -> /~HS_SPI_IRQ
- J101 pad 24: /PIO0_25 -> /PIO0_22
- J101 pad 25: /ISP0 -> GND
- J101 pad 27: GND -> /~SP_RESET
- J101 pad 28: /FC3_TXD_SCL_MISO -> /FC3_RTS_SCLX_SSEL1
- J101 pad 29: /HS_SPI_SCK -> GND
- J101 pad 3: +3V3 -> /ISP0
- J101 pad 31: GND -> /SCT0_OUT2
- J101 pad 32: /FC3_RXD_DSA_MOSI -> /FC3_CTS_SDAX_SSEL0
- J101 pad 33: /HS_SPI_MISO -> /SCT0_OUT3
- J101 pad 36: /PIO0_4 -> /FC0_RXD
- J101 pad 37: /HS_SPI_MOSI -> /SWD_TRACESWO
- J101 pad 39: GND -> /SWD_CLK
- J101 pad 4: +3V3 -> /FC3_SCK
- J101 pad 40: /FC3_SCK -> /FC0_TXD
- J101 pad 41: /~HS_SPI_SSEL1 -> /SWD_IO
- J101 pad 43: GND -> /~SWD_RESET
- J101 pad 44: /FC0_RXD -> +3V3
- J101 pad 45: /~HS_SPI_IRQ -> GND
- J101 pad 46: GND -> +3V3
- J101 pad 47: GND -> +3V3
- J101 pad 48: /FC0_TXD -> +3V3
- J101 pad 49: /~SP_RESET -> +3V3
- J101 pad 5: +3V3 -> GND
- J101 pad 50: GND -> +3V3
- J101 pad 51: GND -> +3V3
- J101 pad 6: +3V3 -> GND
- J101 pad 7: GND -> /HS_SPI_MISO
- J101 pad 8: +3V3 -> /PIO0_4
- J101 pad 9: /~SWD_RESET -> GND
- JP101 pad 2: (no net) -> /OSC_IN
- JP102 pad 2: (no net) -> /OSC_OUT
- JP103 pad 2: (no net) -> /OSC_RTC_IN
- JP104 pad 2: (no net) -> /OSC_RTC_OUT
Routing:
- net /PIO0_10: track 0.00 -> 56.7 mm, vias 0 -> 2
- net /PIO0_11: track 0.00 -> 56.6 mm, vias 0 -> 2
- net /PIO0_12: track 0.00 -> 56.6 mm, vias 0 -> 2
- net /~RESET: track 0.00 -> 54.0 mm, vias 0 -> 2
- net /SCT0_OUT2: track 0.00 -> 43.5 mm, vias 1 -> 2
- net /SCT0_OUT3: track 0.00 -> 43.0 mm, vias 1 -> 2
- net /FC0_RXD: track 0.00 -> 42.9 mm, vias 0 -> 2
- net /FC0_TXD: track 0.00 -> 42.8 mm, vias 0 -> 2
- net /FC3_RXD_DSA_MOSI: track 0.00 -> 41.4 mm, vias 0 -> 2
- net /FC3_CTS_SDAX_SSEL0: track 0.00 -> 41.4 mm, vias 0 -> 2
- net /FC3_SCK: track 0.00 -> 41.3 mm, vias 0 -> 2
- net /FC3_TXD_SCL_MISO: track 0.00 -> 41.3 mm, vias 0 -> 2
- net /PIO0_4: track 0.00 -> 41.3 mm, vias 0 -> 2
- net /FC3_RTS_SCLX_SSEL1: track 0.00 -> 39.6 mm, vias 0 -> 2
- net /PIO0_22: track 0.00 -> 39.5 mm, vias 0 -> 2
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- added copper zone on F.Cu, net +3V3
- added copper zone on F.Cu, net /FB
- added copper zone on B.Cu, net /VDD
- added copper zone on F.Cu, net /VDD
- added copper zone on B.Cu, net /VDDA
- added copper zone on F.Cu, net /VDDA
- added copper zone on F.Cu, net GND

Commit message: lpc55_carrier: switch to 2 layer, front component only
Other:
- board outline added: 51.4 x 37.1 mm
- copper layers 4 -> 2
Changed lines of the file:
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@@
   (general
     (thickness 1.6)
-    (drawings 0)
+    (drawings 4)
     (tracks 2563)
     (zones 0)
@@
   (layers
     (0 F.Cu signal)
-    (1 In1.Cu power hide)
-    (2 In2.Cu power hide)
-    (31 B.Cu signal)
-    (32 B.Adhes user hide)
+    (31 B.Cu signal hide)
     (33 F.Adhes user hide)
-    (34 B.Paste user hide)
     (35 F.Paste user)
-    (36 B.SilkS user hide)
     (37 F.SilkS user)
     (38 B.Mask user hide)
@@
     (46 B.CrtYd user hide)
     (47 F.CrtYd user)
-    (48 B.Fab user hide)
-    (49 F.Fab user hide)
+    (49 F.Fab user)
   )
   (setup
-    (last_trace_width 0.2)
+    (last_trace_width 0.3)
     (user_trace_width 0.3)
     (user_trace_width 0.4)
@@
     )
   )
+  (gr_line (start 65.405 50.038) (end 116.84 50.038) (layer Edge.Cuts) (width 0.12))
+  (gr_line (start 65.405 87.122) (end 65.405 50.038) (layer Edge.Cuts) (width 0.12))
+  (gr_line (start 116.84 87.122) (end 65.405 87.122) (layer Edge.Cuts) (width 0.12))
+  (gr_line (start 116.84 50.038) (end 116.84 87.122) (layer Edge.Cuts) (width 0.12))
   (segment (start 84.5565 70.1635) (end 84.5565 74.93) (width 0.2) (layer F.Cu) (net 1))
   (segment (start 84.57 70.15) (end 84.5565 70.1635) (width 0.2) (layer F.Cu) (net 1))

Commit message: lpc55_carrier: move to 4-layer with 2 inner ground planes
Reduces potential problems where signals passed over reference plane
voids or crossed between reference planes.
Routing:
- net GND: vias 0 -> 23
- added copper zone on In1.Cu, net GND
- added copper zone on In2.Cu, net GND
Other:
- copper layers 2 -> 4

Commit message: lpc55_carrier: Incorporate layout review feedback
- Sprinkle more ground vias near high speed signals
- Sprinkle more ground vias in sparse areas
- Remove meander on HS_SPI_SCK to provide shortest length and improve
setup/hold time
- Add more vias to VDD layer change after filter
Routing:
- net /HS_SPI_SCK: track 20.6 -> 20.0 mm
- net GND: vias 23 -> 32
- net /VDD: vias 9 -> 11

Commit message: lpc55_carrier: layout feedback, no really
Routing:
- net GND: vias 32 -> 34
Changed lines of the file:
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@@
     (thickness 1.6)
     (drawings 4)
-    (tracks 2567)
+    (tracks 2569)
     (zones 0)
     (modules 46)
@@
   (layers
     (0 F.Cu signal)
-    (1 In1.Cu power hide)
+    (1 In1.Cu power)
     (2 In2.Cu power hide)
     (31 B.Cu signal)
@@
   (via (at 96.52 75.184) (size 0.8) (drill 0.4) (layers F.Cu B.Cu) (net 1))
   (via (at 93.726 75.692) (size 0.8) (drill 0.4) (layers F.Cu B.Cu) (net 1))
-  (via (at 95.885 78.613) (size 0.8) (drill 0.4) (layers F.Cu B.Cu) (net 1))
+  (via (at 94.996 78.74) (size 0.8) (drill 0.4) (layers F.Cu B.Cu) (net 1))
   (via (at 96.647 58.547) (size 0.8) (drill 0.4) (layers F.Cu B.Cu) (net 1))
   (via (at 67.818 78.867) (size 0.8) (drill 0.4) (layers F.Cu B.Cu) (net 1))
@@
   (via (at 103.759 59.563) (size 0.8) (drill 0.4) (layers F.Cu B.Cu) (net 1))
   (via (at 99.06 58.928) (size 0.8) (drill 0.4) (layers F.Cu B.Cu) (net 1))
+  (via (at 100.33 69.85) (size 0.8) (drill 0.4) (layers F.Cu B.Cu) (net 1))
+  (via (at 95.631 67.564) (size 0.8) (drill 0.4) (layers F.Cu B.Cu) (net 1))
   (segment (start 70.485 80.8535) (end 70.485 83.1215) (width 0.2) (layer F.Cu) (net 2))
   (segment (start 81.57 73.116) (end 81.57 72.354) (width 0.2) (layer F.Cu) (net 2))

Commit message: lpc55_carrier: specify exact crystals, update footprints and load caps
Parts:
- C121, C122: value 8pF -> 18pF
- C123, C124: value 16pF -> 12pF
- Y101: footprint Crystal:Crystal_SMD_Abracon_ABM3-2Pin_5.0x3.2mm -> Crystal:Crystal_SMD_5032-2Pin_5.0x3.2mm
- Y102: footprint Crystal:Crystal_SMD_Abracon_ABM3-2Pin_5.0x3.2mm -> Crystal:Crystal_SMD_3215-2Pin_3.2x1.5mm
- moved C124 1.27 mm to (103.4, 71.6)
- moved C123 0.64 mm to (96.6, 71.6)
- turned Y102 to 180 degrees
Routing:
- net /OSC_RTC_OUT: track 22.8 -> 22.0 mm

Commit message: lpc55_carrier: update connector footprint to DF9-51S
Parts:
- J101: footprint hirose-df9:Hirose_DF9-51x-1V(69)_2Rows_51Pin-2MP_P1.0mm_Vertical -> hirose-df9:Hirose_DF9-51S-1V(69)_2Rows_51Pin-2MP_P1.0mm_Vertical
Changed lines of the file:
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@@
     )
   )
-  (module "hirose-df9:Hirose_DF9-51x-1V(69)_2Rows_51Pin-2MP_P1.0mm_Vertical" (layer F.Cu)
+  (module "hirose-df9:Hirose_DF9-51S-1V(69)_2Rows_51Pin-2MP_P1.0mm_Vertical" (layer F.Cu)
     (at 110.744 68.326)
     (attr smd)

Commit message: lpc55_carrier: fix package for H130B-16.000 crystal
Parts:
- Y101: footprint Crystal:Crystal_SMD_5032-2Pin_5.0x3.2mm -> Crystal:Crystal_SMD_5032-4Pin_5.0x3.2mm
- moved C121 1.15 mm to (70.7, 82.5)
- moved C122 0.30 mm to (69.5, 74.3), turned to 90 degrees
Connections:
- JP103 pad 2: /OSC_RTC_IN -> (no net)
- JP104 pad 2: /OSC_RTC_OUT -> (no net)
- Y101 pad 2: /OSC_OUT -> (no net)
Routing:
- net /OSC_OUT: track 25.6 -> 27.6 mm
- net /OSC_IN: track 25.6 -> 24.2 mm
- net GND: vias 34 -> 35
