File: lpc55_carrier.kicad_pcb (KiCad board)
At the start: 4 copper layers, 51.4 x 37.1 mm, 48 parts, among them J101 Conn_2Rows-51Pins, U101 LPC55S28JBD64, Y101 16MHz, Y102 32.768kHz

Commit message: lpc55_carrier: add board identifier
Parts:
- added G***: 913-00002, grumpy:Oxide_Board_Identifier_22x6mm, B.Cu at (97.0, 71.8)

Commit message: lpc55_carrier: update PCB from schematic
Parts:
- removed the G*** at (97.0, 71.8)
- removed R105, R106, R107, R111: 100kR, Resistor_SMD:R_0603_1608Metric
- added G***: LOGO, grumpy:logo-4mm-mask, F.Cu at (100.4, 53.8)
- added G***: 913-00002, grumpy:Oxide_Board_Identifier_16x6mm, F.Cu at (96.1, 83.8)
- added R101: 22R, Resistor_SMD:R_0603_1608Metric, F.Cu at (99.2, 62.2)
- added TP101: GND, TestPoint:TestPoint_Pad_2.0x2.0mm, B.Cu at (89.3, 65.0)
- added TP102: VDD, TestPoint:TestPoint_Pad_D2.0mm, B.Cu at (71.0, 59.4)
- added TP103: XTAL_RTC, test-point:TestPoint_2Pads_Pitch8mm_D2.0mm, B.Cu at (98.7, 68.0)
- added TP104: VDDA, TestPoint:TestPoint_Pad_D2.0mm, B.Cu at (90.4, 72.6)
- added TP105: VDD_PMU, TestPoint:TestPoint_Pad_D2.0mm, B.Cu at (88.1, 75.4)
- added TP106: XTAL_32M, test-point:TestPoint_2Pads_Pitch8mm_D2.0mm, B.Cu at (75.9, 75.4)
- added TP107: ~RESET, TestPoint:TestPoint_Pad_D2.0mm, B.Cu at (108.3, 78.9)
- added TP108: ISP0, TestPoint:TestPoint_Pad_D2.0mm, B.Cu at (86.4, 56.8)
- added TP109: SWO, TestPoint:TestPoint_Pad_D2.0mm, B.Cu at (105.7, 75.9)
- C101, C113: value 4.7uF -> 4.7uF 3.3VDCbias; footprint Capacitor_SMD:C_0603_1608Metric -> Capacitor_SMD:C_0805_2012Metric
- C102, C104, C106, C108, C115, C118: value 0.1uF -> 0.1uF 3.3VDCbias
- C103, C105, C107, C109, C116, C125: value 10nF -> 10000pF 3.3VDCbias
- C110: value 47pF -> 47pF 1.2VDCbias
- C111: value 0.1uF -> 0.1uF 1.2VDCbias
- C112: value 2.2uF -> 2.2uF 1.2VDCbias; footprint Capacitor_SMD:C_0603_1608Metric -> Capacitor_SMD:C_0805_2012Metric
- C114, C119: value 47pF -> 47pF 3.3VDCbias
- C117: value 22uF -> 22uF 3.3VDCbias; footprint Capacitor_SMD:C_0805_2012Metric -> Capacitor_SMD:C_1210_3225Metric
- C120: value 22uF -> 22uF 1.2VDCbias; footprint Capacitor_SMD:C_0805_2012Metric -> Capacitor_SMD:C_1210_3225Metric
- C121, C122: value 18pF -> 33pF 1.2VAC
- C123, C124: value 12pF -> 22pF 3.3VAC
- D103: value D -> 1.25Vf 150mA
- FB101, FB102: value 600R -> 600R @ 100MHz 10mA
- L101: value 4.7uH -> 4.7uH 400mA 290mR
- R104, R108, R109, R110: value 100R -> 22R
- Y101: value 16MHz -> 16MHz 18pF
- Y102: value 32.768kHz -> 32.768kHz 12.5pF
- moved C118 1.02 mm to (93.5, 71.0)
- moved C101 0.55 mm to (86.0, 82.1)
- moved L101 0.47 mm to (88.6, 72.4), turned to 180 degrees
- moved C124 0.40 mm to (103.8, 71.6)
- moved Y102 0.40 mm to (100.7, 72.4)
- moved C123 0.40 mm to (97.0, 71.6)
- moved JP103 0.40 mm to (98.2, 68.8)
- moved JP104 0.40 mm to (103.3, 68.8)
- moved C117 0.20 mm to (93.4, 68.4)
- moved C110 0.20 mm to (85.1, 73.2)
- moved C111 0.20 mm to (85.1, 74.9)
- moved C112 0.20 mm to (85.1, 71.4)
Connections:
- net /~HS_SPI_IRQ renamed /PIO0_18
- net /~HS_SPI_SSEL1 renamed /PIO1_1
- JP101 pad 2: /OSC_IN -> /XTAL32M_P
- JP102 pad 2: /OSC_OUT -> /XTAL32M_N
- JP103 pad 2: /OSC_RTC_IN -> /XTAL32K_P
- JP104 pad 2: /OSC_RTC_OUT -> /XTAL32K_N
- U101 pad 19: /OSC_OUT -> /XTAL32M_N
- U101 pad 20: /OSC_IN -> /XTAL32M_P
- U101 pad 34: /OSC_RTC_IN -> /XTAL32K_P
- U101 pad 35: /OSC_RTC_OUT -> /XTAL32K_N
- U101 pad 42: /HS_SPI_MISO -> /PIO1_3
Routing:
- net /XTAL32K_P: track 0.00 -> 20.1 mm, vias 0 -> 1
- net /OSC_RTC_IN: track 22.6 -> 5.68 mm
- net /OSC_RTC_OUT: track 22.0 -> 5.36 mm
- net /XTAL32K_N: track 0.00 -> 15.3 mm
- net /OSC_OUT: track 19.2 -> 4.58 mm
- net /XTAL32M_N: track 0.00 -> 12.9 mm
- net /XTAL32M_P: track 0.00 -> 12.8 mm, vias 0 -> 1
- net /OSC_IN: track 21.9 -> 9.81 mm
- net /HS_SPI_MISO: track 20.6 -> 10.1 mm
- net /PIO1_3: track 0.00 -> 9.12 mm
- net GND: track 5.74 -> 13.2 mm, vias 34 -> 35
- net /ISP0: track 32.1 -> 35.3 mm
- net /FB: track 0.00 -> 2.62 mm, vias 0 -> 1
- net /~RESET: track 54.0 -> 56.6 mm
- net /SWD_TRACESWO: track 8.29 -> 10.8 mm, vias 0 -> 1
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
Commit message: lpc55_carrier: layout ready for CAM
Parts:
- added REF**: Fiducial_0.5mm_Mask1.5mm, Fiducial:Fiducial_0.5mm_Mask1.5mm, B.Cu at (75.8, 54.1)
- added REF**: Fiducial_0.5mm_Mask1.5mm, Fiducial:Fiducial_0.5mm_Mask1.5mm, F.Cu at (75.8, 54.1)
Other:
- rule pad_to_mask_clearance: 0.05 -> 0

Commit message: lpc55_carrier: shrink silkscreen to 0.75mm width and height
Parts:
- removed the G*** at (96.1, 83.8)
- added G***: 913-XXXXX, grumpy:Oxide_Board_Identifier_18x5mm, F.Cu at (91.8, 84.5)

Commit message: lpc55_carrier: fix board P/N
Parts:
- G***: value 913-XXXXX -> 913-00002
