File: sp-ethernet.sch (KiCad schematic (older format))
At the start: 52 parts, among them J401 RJ45_Amphenol_RJMG1BD3B8K1ANR, J402 RJ45_Amphenol_RJMG1BD3B8K1ANR, U401 KSZ8863RLL, Y401 25MHz ±50ppm / H130A-25.000-1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

Commit message: Eth: fix mistakes, route switch layout
I've switched the Magjacks from an Amphenol through-hole part with an
awful pin order, to a Wuerth surface-mount part with a much more
reasonable pinout.

I found a few mistakes in the schematic.

- LED anodes were tied to transistor center taps; moved to 3v3.
- Reset line was doubly pulled up; removed one of two pullups.
Parts:
- removed R409: 10k, Resistor_SMD:R_0603_1608Metric, symbol Device:R
- J401, J402: value RJ45_Amphenol_RJMG1BD3B8K1ANR -> RJ45_Würth_74980111211; footprint Connector_RJ:RJ45_Amphenol_RJMG1BD3B8K1ANR -> magjack:Würth_100BT_Magjack; symbol Connector:RJ45_Amphenol_RJMG1BD3B8K1ANR -> magjack:RJ45_Würth_74980111211
Connections:
- wire segments 161 -> 158
Changed lines of the file:
@@
 Connection ~ 7800 3150
 $Comp
-L Connector:RJ45_Amphenol_RJMG1BD3B8K1ANR J401
+L magjack:RJ45_Würth_74980111211 J401
 U 1 1 5F2FACCC
 P 10200 2400
 F 0 "J401" H 10200 3125 50  0000 C CNN
-F 1 "RJ45_Amphenol_RJMG1BD3B8K1ANR" H 10200 3034 50  0000 C CNN
-F 2 "Connector_RJ:RJ45_Amphenol_RJMG1BD3B8K1ANR" H 10200 3100 50  0001 C CNN
-F 3 "https://www.amphenolcanada.com/ProductSearch/Drawings/AC/RJMG1BD3B8K1ANR.PDF" H 10200 3200 50  0001 C CNN
+F 1 "RJ45_Würth_74980111211" H 10200 3034 50  0000 C CNN
+F 2 "magjack:Würth_100BT_Magjack" H 10200 3100 50  0001 C CNN
+F 3 "https://www.we-online.de/katalog/datasheet/74980111211.pdf" H 10200 3200 50  0001 C CNN
 	1    10200 2400
 	1    0    0    -1
@@
 	9300 2800 9200 2800
 Wire Wire Line
-	9200 2800 9200 2600
-Wire Wire Line
 	9200 2600 9300 2600
-Wire Wire Line
-	9200 2600 9200 2300
-Connection ~ 9200 2600
-Connection ~ 9200 2300
 Text Label 8750 2700 2    50   ~ 0
 P1LEDS
@@
 P1LEDA
 $Comp
-L Connector:RJ45_Amphenol_RJMG1BD3B8K1ANR J402
+L magjack:RJ45_Würth_74980111211 J402
 U 1 1 5F78C158
 P 10200 5100
 F 0 "J402" H 10200 5825 50  0000 C CNN
-F 1 "RJ45_Amphenol_RJMG1BD3B8K1ANR" H 10200 5734 50  0000 C CNN
-F 2 "Connector_RJ:RJ45_Amphenol_RJMG1BD3B8K1ANR" H 10200 5800 50  0001 C CNN
-F 3 "https://www.amphenolcanada.com/ProductSearch/Drawings/AC/RJMG1BD3B8K1ANR.PDF" H 10200 5900 50  0001 C CNN
+F 1 "RJ45_Würth_74980111211" H 10200 5734 50  0000 C CNN
+F 2 "magjack:Würth_100BT_Magjack" H 10200 5800 50  0001 C CNN
+F 3 "https://www.we-online.de/katalog/datasheet/74980111211.pdf" H 10200 5900 50  0001 C CNN
 	1    10200 5100
 	1    0    0    -1
@@
 	9300 5500 9200 5500
 Wire Wire Line
-	9200 5500 9200 5300
-Wire Wire Line
 	9200 5300 9300 5300
-Wire Wire Line
-	9200 5300 9200 5000
-Connection ~ 9200 5300
-Connection ~ 9200 5000
 Text Label 8750 5400 2    50   ~ 0
 P2LEDS
 Text Label 8750 5600 2    50   ~ 0
 P2LEDA
-Wire Wire Line
-	9200 4300 9200 2800
-Connection ~ 9200 4300
-Connection ~ 9200 2800
 Wire Wire Line
 	9200 4300 9200 4700
@@
 This PU req'd for\nour clock mode\n("mode 5")
 Wire Wire Line
-	6300 1750 9200 1750
+	6300 1750 9100 1750
 Wire Wire Line
 	4750 1750 5000 1750
@@
 	2100 1550 2500 1550
 $Comp
-L Device:R R409
-U 1 1 5F492454
-P 1150 3550
-F 0 "R409" V 1050 3500 50  0000 L CNN
-F 1 "10k" V 1150 3500 50  0000 L CNN
-F 2 "Resistor_SMD:R_0603_1608Metric" V 1080 3550 50  0001 C CNN
-F 3 "~" H 1150 3550 50  0001 C CNN
-	1    1150 3550
-	1    0    0    -1
-$EndComp
-Connection ~ 1150 3400
-Wire Wire Line
-	1150 3400 1000 3400
-$Comp
 L Device:D_Small D401
 U 1 1 5F4936FF
@@
 Connection ~ 1300 3400
 Wire Wire Line
-	1300 3400 1150 3400
-Wire Wire Line
 	1300 3650 1300 3700
-Wire Wire Line
-	1300 3700 1250 3700
 $Comp
 L power:+3V3 #PWR0429
 U 1 1 5F4A41AA
-P 1250 3700
-F 0 "#PWR0429" H 1250 3550 50  0001 C CNN
-F 1 "+3V3" H 1265 3873 50  0000 C CNN
-F 2 "" H 1250 3700 50  0001 C CNN
-F 3 "" H 1250 3700 50  0001 C CNN
-	1    1250 3700
+P 1300 3700
+F 0 "#PWR0429" H 1300 3550 50  0001 C CNN
+F 1 "+3V3" H 1315 3873 50  0000 C CNN
+F 2 "" H 1300 3700 50  0001 C CNN
+F 3 "" H 1300 3700 50  0001 C CNN
+	1    1300 3700
 	-1   0    0    1
 $EndComp
-Connection ~ 1250 3700
-Wire Wire Line
-	1250 3700 1150 3700
 Text Label 5100 2300 0    50   ~ 0
 TX1+
@@
 Text Label 5100 3150 0    50   ~ 0
 RX2-
+Wire Wire Line
+	9200 5500 9200 5300
+$Comp
+L power:+3V3 #PWR0108
+U 1 1 5F54BD6B
+P 9200 5300
+F 0 "#PWR0108" H 9200 5150 50  0001 C CNN
+F 1 "+3V3" H 9215 5473 50  0000 C CNN
+F 2 "" H 9200 5300 50  0001 C CNN
+F 3 "" H 9200 5300 50  0001 C CNN
+	1    9200 5300
+	1    0    0    -1
+$EndComp
+Connection ~ 9200 5300
+Wire Wire Line
+	9200 2600 9200 2800
+$Comp
+L power:+3V3 #PWR0109
+U 1 1 5F5544DB
+P 9200 2600
+F 0 "#PWR0109" H 9200 2450 50  0001 C CNN
+F 1 "+3V3" H 9215 2773 50  0000 C CNN
+F 2 "" H 9200 2600 50  0001 C CNN
+F 3 "" H 9200 2600 50  0001 C CNN
+	1    9200 2600
+	1    0    0    -1
+$EndComp
+Connection ~ 9200 2600
+Wire Wire Line
+	9100 1750 9100 4300
+Wire Wire Line
+	9100 4300 9200 4300
+Connection ~ 9100 1750
+Wire Wire Line
+	9100 1750 9200 1750
+Connection ~ 9200 4300
+Wire Wire Line
+	1000 3400 1300 3400
 $EndSCHEMATC

Commit message: MB: annotate everything with mfg/MPN
Parts:
- C401, C402, C403, C404, C405, C406, C407, C408, C409, C410, C411, C412, C413, C414, C415, C416, C417, C418, C419, C420, C421, C422, D401, FB401, FB402, R401, R402, R403, R404, R405, R406, R407, R408, R410, R411, R412, R413, R414, R415, R416, R417, R418, R419, R420, R421, R422, R423: Mfg Part Num (none) -> generic
- J401, J402: Mfg (none) -> Würth Elektronik; Mfg Part Num (none) -> 74980111211
- U401: Mfg (none) -> Microchip; Mfg Part Num (none) -> KSZ8863RLL
- Y401: Mfg (none) -> Raltron Electronics; Mfg Part Num (none) -> H130A-25.000-18-F-2030

Commit message: MB: MPNs for capacitors, adjust some footprints
Can't get a 2kV 10000p cap in 0603 as it turns out
Parts:
- C401, C418, C419: Mfg (none) -> Samsung Electro-Mechanics; Mfg Part Num generic -> CL10A106MQ8NNNC
- C402, C403, C405, C407, C409, C412, C413, C414, C415, C417: Mfg (none) -> Samsung Electro-Mechanics; Mfg Part Num generic -> CL10B104KB8NNWC
- C404, C406, C408, C416: Mfg (none) -> Samsung Electro-Mechanics; Mfg Part Num generic -> CL10A226MP8NUNE
- C410, C411: Mfg (none) -> Walsin Technology Corporation; Mfg Part Num generic -> 0603N180J500CT
- C420, C421: footprint Capacitor_SMD:C_0603_1608Metric -> Capacitor_SMD:C_1206_3216Metric; Mfg (none) -> Kemet; Mfg Part Num generic -> C1206C102KGRACTU
- C422: value 0 -> DNP; Mfg Part Num generic -> (none)
Changed lines of the file:
@@
 F 2 "Capacitor_SMD:C_0603_1608Metric" H 5950 1850 50  0001 C CNN
 F 3 "~" H 5950 1850 50  0001 C CNN
-F 4 "generic" H 5950 1850 50  0001 C CNN "Mfg Part Num"
+F 4 "CL10B104KB8NNWC" H 5950 1850 50  0001 C CNN "Mfg Part Num"
+F 5 "Samsung Electro-Mechanics" H 5950 1850 50  0001 C CNN "Mfg"
 	1    5950 1850
 	1    0    0    -1
@@
 F 2 "Capacitor_SMD:C_0603_1608Metric" H 6300 1850 50  0001 C CNN
 F 3 "~" H 6300 1850 50  0001 C CNN
-F 4 "generic" H 6300 1850 50  0001 C CNN "Mfg Part Num"
+F 4 "CL10A226MP8NUNE" H 6300 1850 50  0001 C CNN "Mfg Part Num"
+F 5 "Samsung Electro-Mechanics" H 6300 1850 50  0001 C CNN "Mfg"
 	1    6300 1850
 	1    0    0    -1
@@
 F 2 "Capacitor_SMD:C_0603_1608Metric" H 4750 1200 50  0001 C CNN
 F 3 "~" H 4750 1200 50  0001 C CNN
-F 4 "generic" H 4750 1200 50  0001 C CNN "Mfg Part Num"
+F 4 "CL10B104KB8NNWC" H 4750 1200 50  0001 C CNN "Mfg Part Num"
+F 5 "Samsung Electro-Mechanics" H 4750 1200 50  0001 C CNN "Mfg"
 	1    4750 1200
 	1    0    0    -1
@@
 F 2 "Capacitor_SMD:C_0603_1608Metric" H 5100 1200 50  0001 C CNN
 F 3 "~" H 5100 1200 50  0001 C CNN
-F 4 "generic" H 5100 1200 50  0001 C CNN "Mfg Part Num"
+F 4 "CL10A226MP8NUNE" H 5100 1200 50  0001 C CNN "Mfg Part Num"
+F 5 "Samsung Electro-Mechanics" H 5100 1200 50  0001 C CNN "Mfg"
 	1    5100 1200
 	1    0    0    -1
@@
 F 2 "Capacitor_SMD:C_0603_1608Metric" H 3950 1150 50  0001 C CNN
 F 3 "~" H 3950 1150 50  0001 C CNN
-F 4 "generic" H 3950 1150 50  0001 C CNN "Mfg Part Num"
+F 4 "CL10A226MP8NUNE" H 3950 1150 50  0001 C CNN "Mfg Part Num"
+F 5 "Samsung Electro-Mechanics" H 3950 1150 50  0001 C CNN "Mfg"
 	1    3950 1150
 	1    0    0    -1
@@
 F 2 "Capacitor_SMD:C_0603_1608Metric" H 3650 1150 50  0001 C CNN
 F 3 "~" H 3650 1150 50  0001 C CNN
-F 4 "generic" H 3650 1150 50  0001 C CNN "Mfg Part Num"
+F 4 "CL10B104KB8NNWC" H 3650 1150 50  0001 C CNN "Mfg Part Num"
+F 5 "Samsung Electro-Mechanics" H 3650 1150 50  0001 C CNN "Mfg"
 	1    3650 1150
 	1    0    0    -1
@@
 F 2 "Capacitor_SMD:C_0603_1608Metric" H 3350 1150 50  0001 C CNN
 F 3 "~" H 3350 1150 50  0001 C CNN
-F 4 "generic" H 3350 1150 50  0001 C CNN "Mfg Part Num"
+F 4 "CL10B104KB8NNWC" H 3350 1150 50  0001 C CNN "Mfg Part Num"
+F 5 "Samsung Electro-Mechanics" H 3350 1150 50  0001 C CNN "Mfg"
 	1    3350 1150
 	1    0    0    -1
@@
 F 2 "Capacitor_SMD:C_0603_1608Metric" H 7200 1300 50  0001 C CNN
 F 3 "~" H 7200 1300 50  0001 C CNN
-F 4 "generic" H 7200 1300 50  0001 C CNN "Mfg Part Num"
+F 4 "CL10A226MP8NUNE" H 7200 1300 50  0001 C CNN "Mfg Part Num"
+F 5 "Samsung Electro-Mechanics" H 7200 1300 50  0001 C CNN "Mfg"
 	1    7200 1300
 	1    0    0    -1
@@
 F 2 "Capacitor_SMD:C_0603_1608Metric" H 6900 1300 50  0001 C CNN
 F 3 "~" H 6900 1300 50  0001 C CNN
-F 4 "generic" H 6900 1300 50  0001 C CNN "Mfg Part Num"
+F 4 "CL10B104KB8NNWC" H 6900 1300 50  0001 C CNN "Mfg Part Num"
+F 5 "Samsung Electro-Mechanics" H 6900 1300 50  0001 C CNN "Mfg"
 	1    6900 1300
 	1    0    0    -1
@@
 F 2 "Capacitor_SMD:C_0603_1608Metric" H 6600 1300 50  0001 C CNN
 F 3 "~" H 6600 1300 50  0001 C CNN
-F 4 "generic" H 6600 1300 50  0001 C CNN "Mfg Part Num"
+F 4 "CL10B104KB8NNWC" H 6600 1300 50  0001 C CNN "Mfg Part Num"
+F 5 "Samsung Electro-Mechanics" H 6600 1300 50  0001 C CNN "Mfg"
 	1    6600 1300
 	1    0    0    -1
@@
 F 2 "Capacitor_SMD:C_0603_1608Metric" H 5850 3850 50  0001 C CNN
 F 3 "~" H 5850 3850 50  0001 C CNN
-F 4 "generic" H 5850 3850 50  0001 C CNN "Mfg Part Num"
+F 4 "CL10B104KB8NNWC" H 5850 3850 50  0001 C CNN "Mfg Part Num"
+F 5 "Samsung Electro-Mechanics" H 5850 3850 50  0001 C CNN "Mfg"
 	1    5850 3850
 	1    0    0    -1
@@
 F 2 "Capacitor_SMD:C_0603_1608Metric" H 6450 3850 50  0001 C CNN
 F 3 "~" H 6450 3850 50  0001 C CNN
-F 4 "generic" H 6450 3850 50  0001 C CNN "Mfg Part Num"
+F 4 "CL10B104KB8NNWC" H 6450 3850 50  0001 C CNN "Mfg Part Num"
+F 5 "Samsung Electro-Mechanics" H 6450 3850 50  0001 C CNN "Mfg"
 	1    6450 3850
 	1    0    0    -1
@@
 F 2 "Capacitor_SMD:C_0603_1608Metric" H 7050 3850 50  0001 C CNN
 F 3 "~" H 7050 3850 50  0001 C CNN
-F 4 "generic" H 7050 3850 50  0001 C CNN "Mfg Part Num"
+F 4 "CL10B104KB8NNWC" H 7050 3850 50  0001 C CNN "Mfg Part Num"
+F 5 "Samsung Electro-Mechanics" H 7050 3850 50  0001 C CNN "Mfg"
 	1    7050 3850
 	1    0    0    -1
@@
 F 2 "Capacitor_SMD:C_0603_1608Metric" H 7650 3850 50  0001 C CNN
 F 3 "~" H 7650 3850 50  0001 C CNN
-F 4 "generic" H 7650 3850 50  0001 C CNN "Mfg Part Num"
+F 4 "CL10B104KB8NNWC" H 7650 3850 50  0001 C CNN "Mfg Part Num"
+F 5 "Samsung Electro-Mechanics" H 7650 3850 50  0001 C CNN "Mfg"
 	1    7650 3850
 	1    0    0    -1
@@
 F 2 "Capacitor_SMD:C_0603_1608Metric" H 9300 1600 50  0001 C CNN
 F 3 "~" H 9300 1600 50  0001 C CNN
-F 4 "generic" H 9300 1600 50  0001 C CNN "Mfg Part Num"
+F 4 "CL10A106MQ8NNNC" H 9300 1600 50  0001 C CNN "Mfg Part Num"
+F 5 "Samsung Electro-Mechanics" H 9300 1600 50  0001 C CNN "Mfg"
 	1    9300 1600
 	0    1    1    0
@@
 F 0 "C420" V 10471 3250 50  0000 C CNN
 F 1 "1000p 2kV" V 10562 3250 50  0000 C CNN
-F 2 "Capacitor_SMD:C_0603_1608Metric" H 10700 3250 50  0001 C CNN
+F 2 "Capacitor_SMD:C_1206_3216Metric" H 10700 3250 50  0001 C CNN
 F 3 "~" H 10700 3250 50  0001 C CNN
-F 4 "generic" H 10700 3250 50  0001 C CNN "Mfg Part Num"
+F 4 "C1206C102KGRACTU" H 10700 3250 50  0001 C CNN "Mfg Part Num"
+F 5 "Kemet" H 10700 3250 50  0001 C CNN "Mfg"
 	1    10700 3250
 	0    1    1    0
@@
 F 2 "Capacitor_SMD:C_0603_1608Metric" H 5900 5900 50  0001 C CNN
 F 3 "~" H 5900 5900 50  0001 C CNN
-F 4 "generic" H 5900 5900 50  0001 C CNN "Mfg Part Num"
+F 4 "0603N180J500CT" H 5900 5900 50  0001 C CNN "Mfg Part Num"
+F 5 "Walsin Technology Corporation" H 5900 5900 50  0001 C CNN "Mfg"
 	1    5900 5900
 	-1   0    0    1
@@
 F 2 "Capacitor_SMD:C_0603_1608Metric" H 6400 5900 50  0001 C CNN
 F 3 "~" H 6400 5900 50  0001 C CNN
-F 4 "generic" H 6400 5900 50  0001 C CNN "Mfg Part Num"
+F 4 "0603N180J500CT" H 6400 5900 50  0001 C CNN "Mfg Part Num"
+F 5 "Walsin Technology Corporation" H 6400 5900 50  0001 C CNN "Mfg"
 	1    6400 5900
 	-1   0    0    1
@@
 F 2 "Capacitor_SMD:C_0603_1608Metric" H 1550 3500 50  0001 C CNN
 F 3 "~" H 1550 3500 50  0001 C CNN
-F 4 "generic" H 1550 3500 50  0001 C CNN "Mfg Part Num"
+F 4 "CL10A106MQ8NNNC" H 1550 3500 50  0001 C CNN "Mfg Part Num"
+F 5 "Samsung Electro-Mechanics" H 1550 3500 50  0001 C CNN "Mfg"
 	1    1550 3500
 	1    0    0    -1
@@
 F 2 "Capacitor_SMD:C_0603_1608Metric" H 9300 4300 50  0001 C CNN
 F 3 "~" H 9300 4300 50  0001 C CNN
-F 4 "generic" H 9300 4300 50  0001 C CNN "Mfg Part Num"
+F 4 "CL10A106MQ8NNNC" H 9300 4300 50  0001 C CNN "Mfg Part Num"
+F 5 "Samsung Electro-Mechanics" H 9300 4300 50  0001 C CNN "Mfg"
 	1    9300 4300
 	0    1    1    0
@@
 F 0 "C421" V 10471 5950 50  0000 C CNN
 F 1 "1000p 2kV" V 10562 5950 50  0000 C CNN
-F 2 "Capacitor_SMD:C_0603_1608Metric" H 10700 5950 50  0001 C CNN
+F 2 "Capacitor_SMD:C_1206_3216Metric" H 10700 5950 50  0001 C CNN
 F 3 "~" H 10700 5950 50  0001 C CNN
-F 4 "generic" H 10700 5950 50  0001 C CNN "Mfg Part Num"
+F 4 "C1206C102KGRACTU" H 10700 5950 50  0001 C CNN "Mfg Part Num"
+F 5 "Kemet" H 10700 5950 50  0001 C CNN "Mfg"
 	1    10700 5950
 	0    1    1    0
@@
 P 5500 1750
 F 0 "C422" V 5271 1750 50  0000 C CNN
-F 1 "0" V 5362 1750 50  0000 C CNN
+F 1 "DNP" V 5362 1750 50  0000 C CNN
 F 2 "Capacitor_SMD:C_0603_1608Metric" H 5500 1750 50  0001 C CNN
 F 3 "~" H 5500 1750 50  0001 C CNN
-F 4 "generic" H 5500 1750 50  0001 C CNN "Mfg Part Num"
+F 4 "" H 5500 1750 50  0001 C CNN "Mfg Part Num"
 	1    5500 1750
 	0    1    1    0

Commit message: MB: diode selection
Switched 0603 diodes to SOD-323 due to availability
Adjusted H7 debug LED current limit resistors for Vf
Parts:
- D401: footprint Diode_SMD:D_0603_1608Metric -> Diode_SMD:D_SOD-323; Mfg (none) -> Taiwan Semiconductor Corporation; Mfg Part Num generic -> 1N4148WS-G RVG
Changed lines of the file:
@@
 F 0 "D401" V 1346 3480 50  0000 R CNN
 F 1 "1N4148" V 1255 3480 50  0000 R CNN
-F 2 "Diode_SMD:D_0603_1608Metric" V 1300 3550 50  0001 C CNN
+F 2 "Diode_SMD:D_SOD-323" V 1300 3550 50  0001 C CNN
 F 3 "~" V 1300 3550 50  0001 C CNN
-F 4 "generic" H 1300 3550 50  0001 C CNN "Mfg Part Num"
+F 4 "1N4148WS-G RVG" H 1300 3550 50  0001 C CNN "Mfg Part Num"
+F 5 "Taiwan Semiconductor Corporation" H 1300 3550 50  0001 C CNN "Mfg"
 	1    1300 3550
 	0    -1   -1   0

Commit message: MB: assign ferrites'n'fuses
Parts:
- FB401, FB402: value tbd -> 33R @ 100MHz; Mfg (none) -> Murata Electronics; Mfg Part Num generic -> BLM18PG330SN1D
Changed lines of the file:
@@
 P 4600 1000
 F 0 "FB401" H 4700 1046 50  0000 L CNN
-F 1 "tbd" H 4700 955 50  0000 L CNN
+F 1 "33R @ 100MHz" H 4700 955 50  0000 L CNN
 F 2 "Inductor_SMD:L_0603_1608Metric" V 4530 1000 50  0001 C CNN
 F 3 "~" H 4600 1000 50  0001 C CNN
-F 4 "generic" H 4600 1000 50  0001 C CNN "Mfg Part Num"
+F 4 "BLM18PG330SN1D" H 4600 1000 50  0001 C CNN "Mfg Part Num"
+F 5 "Murata Electronics" H 4600 1000 50  0001 C CNN "Mfg"
 	1    4600 1000
 	1    0    0    -1
@@
 P 5950 1650
 F 0 "FB402" H 6050 1696 50  0000 L CNN
-F 1 "tbd" H 6050 1605 50  0000 L CNN
+F 1 "33R @ 100MHz" H 6050 1605 50  0000 L CNN
 F 2 "Inductor_SMD:L_0603_1608Metric" V 5880 1650 50  0001 C CNN
 F 3 "~" H 5950 1650 50  0001 C CNN
-F 4 "generic" H 5950 1650 50  0001 C CNN "Mfg Part Num"
+F 4 "BLM18PG330SN1D" H 5950 1650 50  0001 C CNN "Mfg Part Num"
+F 5 "Murata Electronics" H 5950 1650 50  0001 C CNN "Mfg"
 	1    5950 1650
 	1    0    0    -1
