File: sp-ethernet.sch (KiCad schematic (older format))
At the start: 51 parts, among them J401 RJ45_Würth_74980111211, J402 RJ45_Würth_74980111211, U401 KSZ8863RLL, Y401 25MHz ±50ppm / H130A-25.000-1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

Commit message: MB: assign single resistors
Parts:
- R401, R402, R403, R404: Mfg (none) -> Bourns; Mfg Part Num generic -> CR0603-JW-220ELF
- R405, R406, R423: Mfg (none) -> Bourns; Mfg Part Num generic -> CR0603-JW-103ELF
- R407, R408: Mfg (none) -> Bourns; Mfg Part Num generic -> CR0603-JW-472ELF
- R410: Mfg (none) -> Stackpole Electronics; Mfg Part Num generic -> RMCF0603FT11K8
- R411, R412, R413, R414, R415, R416, R417, R418: Mfg (none) -> Stackpole Electronics; Mfg Part Num generic -> RMCF0603FT49R9
- R419, R420, R421, R422: Mfg (none) -> KOA Speer Electronics; Mfg Part Num generic -> RK73B1JTTD181J
Changed lines of the file:
@@
 F 2 "Resistor_SMD:R_0603_1608Metric" V 5630 3500 50  0001 C CNN
 F 3 "~" H 5700 3500 50  0001 C CNN
-F 4 "generic" H 5700 3500 50  0001 C CNN "Mfg Part Num"
+F 4 "RMCF0603FT49R9" H 5700 3500 50  0001 C CNN "Mfg Part Num"
+F 5 "Stackpole Electronics" H 5700 3500 50  0001 C CNN "Mfg"
 	1    5700 3500
 	1    0    0    -1
@@
 F 2 "Resistor_SMD:R_0603_1608Metric" V 5930 3500 50  0001 C CNN
 F 3 "~" H 6000 3500 50  0001 C CNN
-F 4 "generic" H 6000 3500 50  0001 C CNN "Mfg Part Num"
+F 4 "RMCF0603FT49R9" H 6000 3500 50  0001 C CNN "Mfg Part Num"
+F 5 "Stackpole Electronics" H 6000 3500 50  0001 C CNN "Mfg"
 	1    6000 3500
 	1    0    0    -1
@@
 F 2 "Resistor_SMD:R_0603_1608Metric" V 6230 3500 50  0001 C CNN
 F 3 "~" H 6300 3500 50  0001 C CNN
-F 4 "generic" H 6300 3500 50  0001 C CNN "Mfg Part Num"
+F 4 "RMCF0603FT49R9" H 6300 3500 50  0001 C CNN "Mfg Part Num"
+F 5 "Stackpole Electronics" H 6300 3500 50  0001 C CNN "Mfg"
 	1    6300 3500
 	1    0    0    -1
@@
 F 2 "Resistor_SMD:R_0603_1608Metric" V 6530 3500 50  0001 C CNN
 F 3 "~" H 6600 3500 50  0001 C CNN
-F 4 "generic" H 6600 3500 50  0001 C CNN "Mfg Part Num"
+F 4 "RMCF0603FT49R9" H 6600 3500 50  0001 C CNN "Mfg Part Num"
+F 5 "Stackpole Electronics" H 6600 3500 50  0001 C CNN "Mfg"
 	1    6600 3500
 	1    0    0    -1
@@
 F 2 "Resistor_SMD:R_0603_1608Metric" V 6830 3500 50  0001 C CNN
 F 3 "~" H 6900 3500 50  0001 C CNN
-F 4 "generic" H 6900 3500 50  0001 C CNN "Mfg Part Num"
+F 4 "RMCF0603FT49R9" H 6900 3500 50  0001 C CNN "Mfg Part Num"
+F 5 "Stackpole Electronics" H 6900 3500 50  0001 C CNN "Mfg"
 	1    6900 3500
 	1    0    0    -1
@@
 F 2 "Resistor_SMD:R_0603_1608Metric" V 7130 3500 50  0001 C CNN
 F 3 "~" H 7200 3500 50  0001 C CNN
-F 4 "generic" H 7200 3500 50  0001 C CNN "Mfg Part Num"
+F 4 "RMCF0603FT49R9" H 7200 3500 50  0001 C CNN "Mfg Part Num"
+F 5 "Stackpole Electronics" H 7200 3500 50  0001 C CNN "Mfg"
 	1    7200 3500
 	1    0    0    -1
@@
 F 2 "Resistor_SMD:R_0603_1608Metric" V 7430 3500 50  0001 C CNN
 F 3 "~" H 7500 3500 50  0001 C CNN
-F 4 "generic" H 7500 3500 50  0001 C CNN "Mfg Part Num"
+F 4 "RMCF0603FT49R9" H 7500 3500 50  0001 C CNN "Mfg Part Num"
+F 5 "Stackpole Electronics" H 7500 3500 50  0001 C CNN "Mfg"
 	1    7500 3500
 	1    0    0    -1
@@
 F 2 "Resistor_SMD:R_0603_1608Metric" V 7730 3500 50  0001 C CNN
 F 3 "~" H 7800 3500 50  0001 C CNN
-F 4 "generic" H 7800 3500 50  0001 C CNN "Mfg Part Num"
+F 4 "RMCF0603FT49R9" H 7800 3500 50  0001 C CNN "Mfg Part Num"
+F 5 "Stackpole Electronics" H 7800 3500 50  0001 C CNN "Mfg"
 	1    7800 3500
 	1    0    0    -1
@@
 F 2 "Resistor_SMD:R_0603_1608Metric" V 1180 2600 50  0001 C CNN
 F 3 "~" H 1250 2600 50  0001 C CNN
-F 4 "generic" H 1250 2600 50  0001 C CNN "Mfg Part Num"
+F 4 "CR0603-JW-220ELF" H 1250 2600 50  0001 C CNN "Mfg Part Num"
+F 5 "Bourns" H 1250 2600 50  0001 C CNN "Mfg"
 	1    1250 2600
 	0    1    1    0
@@
 F 2 "Resistor_SMD:R_0603_1608Metric" V 2030 1700 50  0001 C CNN
 F 3 "~" H 2100 1700 50  0001 C CNN
-F 4 "generic" H 2100 1700 50  0001 C CNN "Mfg Part Num"
+F 4 "CR0603-JW-472ELF" H 2100 1700 50  0001 C CNN "Mfg Part Num"
+F 5 "Bourns" H 2100 1700 50  0001 C CNN "Mfg"
 	1    2100 1700
 	1    0    0    -1
@@
 F 2 "Resistor_SMD:R_0603_1608Metric" V 1830 1700 50  0001 C CNN
 F 3 "~" H 1900 1700 50  0001 C CNN
-F 4 "generic" H 1900 1700 50  0001 C CNN "Mfg Part Num"
+F 4 "CR0603-JW-472ELF" H 1900 1700 50  0001 C CNN "Mfg Part Num"
+F 5 "Bourns" H 1900 1700 50  0001 C CNN "Mfg"
 	1    1900 1700
 	1    0    0    -1
@@
 F 2 "Resistor_SMD:R_0603_1608Metric" V 1430 4100 50  0001 C CNN
 F 3 "~" H 1500 4100 50  0001 C CNN
-F 4 "generic" H 1500 4100 50  0001 C CNN "Mfg Part Num"
+F 4 "CR0603-JW-103ELF" H 1500 4100 50  0001 C CNN "Mfg Part Num"
+F 5 "Bourns" H 1500 4100 50  0001 C CNN "Mfg"
 	1    1500 4100
 	0    1    1    0
@@
 F 2 "Resistor_SMD:R_0603_1608Metric" V 1380 2400 50  0001 C CNN
 F 3 "~" H 1450 2400 50  0001 C CNN
-F 4 "generic" H 1450 2400 50  0001 C CNN "Mfg Part Num"
+F 4 "CR0603-JW-220ELF" H 1450 2400 50  0001 C CNN "Mfg Part Num"
+F 5 "Bourns" H 1450 2400 50  0001 C CNN "Mfg"
 	1    1450 2400
 	0    1    1    0
@@
 F 2 "Resistor_SMD:R_0603_1608Metric" V 1180 2250 50  0001 C CNN
 F 3 "~" H 1250 2250 50  0001 C CNN
-F 4 "generic" H 1250 2250 50  0001 C CNN "Mfg Part Num"
+F 4 "CR0603-JW-220ELF" H 1250 2250 50  0001 C CNN "Mfg Part Num"
+F 5 "Bourns" H 1250 2250 50  0001 C CNN "Mfg"
 	1    1250 2250
 	0    1    1    0
@@
 F 2 "Resistor_SMD:R_0603_1608Metric" V 1380 2150 50  0001 C CNN
 F 3 "~" H 1450 2150 50  0001 C CNN
-F 4 "generic" H 1450 2150 50  0001 C CNN "Mfg Part Num"
+F 4 "CR0603-JW-220ELF" H 1450 2150 50  0001 C CNN "Mfg Part Num"
+F 5 "Bourns" H 1450 2150 50  0001 C CNN "Mfg"
 	1    1450 2150
 	0    1    1    0
@@
 F 2 "Resistor_SMD:R_0603_1608Metric" V 1630 1700 50  0001 C CNN
 F 3 "~" H 1700 1700 50  0001 C CNN
-F 4 "generic" H 1700 1700 50  0001 C CNN "Mfg Part Num"
+F 4 "CR0603-JW-103ELF" H 1700 1700 50  0001 C CNN "Mfg Part Num"
+F 5 "Bourns" H 1700 1700 50  0001 C CNN "Mfg"
 	1    1700 1700
 	1    0    0    -1
@@
 F 2 "Resistor_SMD:R_0603_1608Metric" V 5180 4750 50  0001 C CNN
 F 3 "~" H 5250 4750 50  0001 C CNN
-F 4 "generic" H 5250 4750 50  0001 C CNN "Mfg Part Num"
+F 4 "RMCF0603FT11K8" H 5250 4750 50  0001 C CNN "Mfg Part Num"
+F 5 "Stackpole Electronics" H 5250 4750 50  0001 C CNN "Mfg"
 	1    5250 4750
 	1    0    0    -1
@@
 F 2 "Resistor_SMD:R_0603_1608Metric" V 8830 2700 50  0001 C CNN
 F 3 "~" H 8900 2700 50  0001 C CNN
-F 4 "generic" H 8900 2700 50  0001 C CNN "Mfg Part Num"
+F 4 "RK73B1JTTD181J" H 8900 2700 50  0001 C CNN "Mfg Part Num"
+F 5 "KOA Speer Electronics" H 8900 2700 50  0001 C CNN "Mfg"
 	1    8900 2700
 	0    1    1    0
@@
 F 2 "Resistor_SMD:R_0603_1608Metric" V 8830 2900 50  0001 C CNN
 F 3 "~" H 8900 2900 50  0001 C CNN
-F 4 "generic" H 8900 2900 50  0001 C CNN "Mfg Part Num"
+F 4 "RK73B1JTTD181J" H 8900 2900 50  0001 C CNN "Mfg Part Num"
+F 5 "KOA Speer Electronics" H 8900 2900 50  0001 C CNN "Mfg"
 	1    8900 2900
 	0    1    1    0
@@
 F 2 "Resistor_SMD:R_0603_1608Metric" V 8830 5400 50  0001 C CNN
 F 3 "~" H 8900 5400 50  0001 C CNN
-F 4 "generic" H 8900 5400 50  0001 C CNN "Mfg Part Num"
+F 4 "RK73B1JTTD181J" H 8900 5400 50  0001 C CNN "Mfg Part Num"
+F 5 "KOA Speer Electronics" H 8900 5400 50  0001 C CNN "Mfg"
 	1    8900 5400
 	0    1    1    0
@@
 F 2 "Resistor_SMD:R_0603_1608Metric" V 8830 5600 50  0001 C CNN
 F 3 "~" H 8900 5600 50  0001 C CNN
-F 4 "generic" H 8900 5600 50  0001 C CNN "Mfg Part Num"
+F 4 "RK73B1JTTD181J" H 8900 5600 50  0001 C CNN "Mfg Part Num"
+F 5 "KOA Speer Electronics" H 8900 5600 50  0001 C CNN "Mfg"
 	1    8900 5600
 	0    1    1    0
@@
 F 2 "Resistor_SMD:R_0603_1608Metric" V 2430 1700 50  0001 C CNN
 F 3 "~" H 2500 1700 50  0001 C CNN
-F 4 "generic" H 2500 1700 50  0001 C CNN "Mfg Part Num"
+F 4 "CR0603-JW-103ELF" H 2500 1700 50  0001 C CNN "Mfg Part Num"
+F 5 "Bourns" H 2500 1700 50  0001 C CNN "Mfg"
 	1    2500 1700
 	-1   0    0    1

Commit message: MB: add caps suggested in review
Parts:
- added C423, C424: 0µ1, Capacitor_SMD:C_0603_1608Metric, symbol Device:C_Small
Connections:
- net +3V3: now also C423.1, C424.1
- net GND: now also C423.2, C424.2
Changed lines of the file:
@@
 Wire Wire Line
 	1000 3400 1300 3400
+$Comp
+L Device:C_Small C423
+U 1 1 5F698C36
+P 1850 5300
+F 0 "C423" H 1942 5346 50  0000 L CNN
+F 1 "0µ1" H 1942 5255 50  0000 L CNN
+F 2 "Capacitor_SMD:C_0603_1608Metric" H 1850 5300 50  0001 C CNN
+F 3 "~" H 1850 5300 50  0001 C CNN
+F 4 "CL10B104KB8NNWC" H 1850 5300 50  0001 C CNN "Mfg Part Num"
+F 5 "Samsung Electro-Mechanics" H 1850 5300 50  0001 C CNN "Mfg"
+	1    1850 5300
+	1    0    0    -1
+$EndComp
+$Comp
+L Device:C_Small C424
+U 1 1 5F6A02F3
+P 2250 5300
+F 0 "C424" H 2342 5346 50  0000 L CNN
+F 1 "0µ1" H 2342 5255 50  0000 L CNN
+F 2 "Capacitor_SMD:C_0603_1608Metric" H 2250 5300 50  0001 C CNN
+F 3 "~" H 2250 5300 50  0001 C CNN
+F 4 "CL10B104KB8NNWC" H 2250 5300 50  0001 C CNN "Mfg Part Num"
+F 5 "Samsung Electro-Mechanics" H 2250 5300 50  0001 C CNN "Mfg"
+	1    2250 5300
+	1    0    0    -1
+$EndComp
+Wire Wire Line
+	1850 5200 2050 5200
+Wire Wire Line
+	1850 5400 2050 5400
+$Comp
+L power:+3V3 #PWR0417
+U 1 1 5F6B77D9
+P 2050 5200
+F 0 "#PWR0417" H 2050 5050 50  0001 C CNN
+F 1 "+3V3" H 2065 5373 50  0000 C CNN
+F 2 "" H 2050 5200 50  0001 C CNN
+F 3 "" H 2050 5200 50  0001 C CNN
+	1    2050 5200
+	1    0    0    -1
+$EndComp
+Connection ~ 2050 5200
+Wire Wire Line
+	2050 5200 2250 5200
+$Comp
+L power:GND #PWR0418
+U 1 1 5F6B7FFC
+P 2050 5400
+F 0 "#PWR0418" H 2050 5150 50  0001 C CNN
+F 1 "GND" H 2055 5227 50  0000 C CNN
+F 2 "" H 2050 5400 50  0001 C CNN
+F 3 "" H 2050 5400 50  0001 C CNN
+	1    2050 5400
+	1    0    0    -1
+$EndComp
+Connection ~ 2050 5400
+Wire Wire Line
+	2050 5400 2250 5400
 $EndSCHEMATC

Commit message: Update MPNs to full, orderable, normally-stocked MPNs
Parts:
- Y401: Mfg Part Num H130A-25.000-18-F-2030 -> H130A-25.000-18-F-3030
Changed lines of the file:
@@
 F 3 "~" H 6200 5500 50  0001 C CNN
 F 4 "Raltron Electronics" H 6200 5500 50  0001 C CNN "Mfg"
-F 5 "H130A-25.000-18-F-2030" H 6200 5500 50  0001 C CNN "Mfg Part Num"
+F 5 "H130A-25.000-18-F-3030" H 6200 5500 50  0001 C CNN "Mfg Part Num"
 	1    6200 5500
 	1    0    0    -1
