File: sp-ethernet.sch (KiCad schematic (older format))
At the start: 53 parts, among them J401 RJ45_Würth_74980111211, J402 RJ45_Würth_74980111211, U401 KSZ8863RLL, Y401 25MHz ±50ppm / H130A-25.000-1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

Commit message: gemini-bringup: Add CPNs for all components
Parts:
- C401, C418, C419: CPN (none) -> 212-00018
- C402, C403, C405, C407, C409, C412, C413, C414, C415, C417, C423, C424: CPN (none) -> 212-00011
- C404, C406, C408, C416: CPN (none) -> 212-00016
- C410, C411: CPN (none) -> 212-00017
- C420, C421: CPN (none) -> 212-00019
- D401: CPN (none) -> 217-00002
- FB401, FB402: CPN (none) -> 242-00017
- J401, J402: CPN (none) -> 215-00027
- R401, R402, R403, R404: CPN (none) -> 232-00019
- R405, R406, R423: CPN (none) -> 232-00024
- R407, R408: CPN (none) -> 232-00027
- R410: CPN (none) -> 232-00028
- R411, R412, R413, R414, R415, R416, R417, R418: CPN (none) -> 232-00029
- R419, R420, R421, R422: CPN (none) -> 232-00030
- U401: CPN (none) -> 221-00013
- Y401: CPN (none) -> 216-00005

Commit message: gemini-bringup: Mark DNP (do not populate) in a Config field rather than value to match KiBOM expectations
Parts:
- C422: Config (none) -> DNP
Changed lines of the file:
@@
 F 3 "~" H 5500 1750 50  0001 C CNN
 F 4 "" H 5500 1750 50  0001 C CNN "Mfg Part Num"
+F 5 "DNP" H 5500 1750 50  0001 C CNN "Config"
 	1    5500 1750
 	0    1    1    0

Commit message: gemini-bringup: custom fields for rating constraints on passives
Instead of packing tons of detail into a single "Value" field, limit
"Value" to the primary characteristic of the device (i.e. capacitance
for capacitors, resistance for resistors, current for fuses, impedence
at frequency for ferrite beads). For all other rating constraints, use
custom fields of the form <component-refdes-prefix>_<constraint>. For
example, R_P contains the power a resistor must dissipate.  Use
calculated values when possible rather than standard values as the
intent is to capture the constraint, not a specific device choice.
Parts:
- C401, C418, C419: value 10µ -> 10uF; C_Vbias (none) -> 3.3V
- C402, C403, C405: value 0µ1 -> 0.1uF; C_Vbias (none) -> 1.8V
- C404, C406: value 22µ -> 22uF; C_Vbias (none) -> 1.8V
- C407, C413, C414, C423, C424: value 0µ1 -> 0.1uF; C_Vbias (none) -> 3.3V
- C408, C416: value 22µ -> 22uF; C_Vbias (none) -> 3.3V
- C409, C412, C415, C417: value 0µ1 -> 0.1uF; C_Vpp (none) -> 3.3V
- C410, C411: value 18p -> 18pF; C_Vpp (none) -> 3.3V
- C420, C421: value 1000p 2kV -> 1000pF 2kV
- D401: D_Vr (none) -> 3.3V
- R401, R402, R403, R404: value 22 -> 22R
- R405, R406, R423: value 10k -> 10kR
- R407, R408: value 4k7 -> 4.7kR
- R410: value 11k8 1% -> 11.8kR 1%
- R411, R412, R413, R414, R415, R416, R417, R418: value 49R9 1% -> 49.9R 1%
- R419, R420, R421, R422: value 180 -> 180R
- Y401: value 25MHz ±50ppm / H130A-25.000-18-F-2030 -> 25MHz ±50ppm; Y_Cl (none) -> 18pF

Commit message: sp-ethernet: adjust RJ45 LED resistors
LEDs inside Wurth 74980111211 RJ45 have Vf between 1.8V and 2.8V.
Assuming Vf=2.3V is normal, 180R would only provide ~5mA for LEDs
spec'd for 20mA.  56R would be ideal but it'd be the only use of that
value. We use 68R for other LEDs and in this case would provide ~15mA
which is a little low but should be fine for status LEDs.
Parts:
- R419, R420, R421, R422: value 180R -> 68R
Changed lines of the file:
@@
 P 8900 2700
 F 0 "R419" V 8800 2700 50  0000 C CNN
-F 1 "180R" V 8900 2700 50  0000 C CNN
+F 1 "68R" V 8900 2700 50  0000 C CNN
 F 2 "Resistor_SMD:R_0603_1608Metric" V 8830 2700 50  0001 C CNN
 F 3 "~" H 8900 2700 50  0001 C CNN
@@
 P 8900 2900
 F 0 "R420" V 8800 2900 50  0000 C CNN
-F 1 "180R" V 8900 2900 50  0000 C CNN
+F 1 "68R" V 8900 2900 50  0000 C CNN
 F 2 "Resistor_SMD:R_0603_1608Metric" V 8830 2900 50  0001 C CNN
 F 3 "~" H 8900 2900 50  0001 C CNN
@@
 P 8900 5400
 F 0 "R421" V 8800 5400 50  0000 C CNN
-F 1 "180R" V 8900 5400 50  0000 C CNN
+F 1 "68R" V 8900 5400 50  0000 C CNN
 F 2 "Resistor_SMD:R_0603_1608Metric" V 8830 5400 50  0001 C CNN
 F 3 "~" H 8900 5400 50  0001 C CNN
@@
 P 8900 5600
 F 0 "R422" V 8800 5600 50  0000 C CNN
-F 1 "180R" V 8900 5600 50  0000 C CNN
+F 1 "68R" V 8900 5600 50  0000 C CNN
 F 2 "Resistor_SMD:R_0603_1608Metric" V 8830 5600 50  0001 C CNN
 F 3 "~" H 8900 5600 50  0001 C CNN

Commit message: gemini-bringup: resistor power rating constraints
Parts:
- R405, R406, R423: R_P (none) -> 300uW
- R407, R408: R_P (none) -> 700uW
- R419, R420, R421, R422: R_P (none) -> 15mW
Changed lines of the file:
@@
 F 5 "Stackpole Electronics" H 5700 3500 50  0001 C CNN "Mfg"
 F 6 "232-00029" H 5700 3500 50  0001 C CNN "CPN"
+F 7 "" H 5700 3500 50  0001 C CNN "R_P"
 	1    5700 3500
 	1    0    0    -1
@@
 F 5 "Stackpole Electronics" H 6000 3500 50  0001 C CNN "Mfg"
 F 6 "232-00029" H 6000 3500 50  0001 C CNN "CPN"
+F 7 "" H 6000 3500 50  0001 C CNN "R_P"
 	1    6000 3500
 	1    0    0    -1
@@
 F 5 "Stackpole Electronics" H 6300 3500 50  0001 C CNN "Mfg"
 F 6 "232-00029" H 6300 3500 50  0001 C CNN "CPN"
+F 7 "" H 6300 3500 50  0001 C CNN "R_P"
 	1    6300 3500
 	1    0    0    -1
@@
 F 5 "Stackpole Electronics" H 6600 3500 50  0001 C CNN "Mfg"
 F 6 "232-00029" H 6600 3500 50  0001 C CNN "CPN"
+F 7 "" H 6600 3500 50  0001 C CNN "R_P"
 	1    6600 3500
 	1    0    0    -1
@@
 F 5 "Stackpole Electronics" H 6900 3500 50  0001 C CNN "Mfg"
 F 6 "232-00029" H 6900 3500 50  0001 C CNN "CPN"
+F 7 "" H 6900 3500 50  0001 C CNN "R_P"
 	1    6900 3500
 	1    0    0    -1
@@
 F 5 "Stackpole Electronics" H 7200 3500 50  0001 C CNN "Mfg"
 F 6 "232-00029" H 7200 3500 50  0001 C CNN "CPN"
+F 7 "" H 7200 3500 50  0001 C CNN "R_P"
 	1    7200 3500
 	1    0    0    -1
@@
 F 5 "Stackpole Electronics" H 7500 3500 50  0001 C CNN "Mfg"
 F 6 "232-00029" H 7500 3500 50  0001 C CNN "CPN"
+F 7 "" H 7500 3500 50  0001 C CNN "R_P"
 	1    7500 3500
 	1    0    0    -1
@@
 F 5 "Stackpole Electronics" H 7800 3500 50  0001 C CNN "Mfg"
 F 6 "232-00029" H 7800 3500 50  0001 C CNN "CPN"
+F 7 "" H 7800 3500 50  0001 C CNN "R_P"
 	1    7800 3500
 	1    0    0    -1
@@
 F 5 "Bourns" H 2100 1700 50  0001 C CNN "Mfg"
 F 6 "232-00027" H 2100 1700 50  0001 C CNN "CPN"
+F 7 "700uW" H 2100 1700 50  0001 C CNN "R_P"
 	1    2100 1700
 	1    0    0    -1
@@
 F 5 "Bourns" H 1900 1700 50  0001 C CNN "Mfg"
 F 6 "232-00027" H 1900 1700 50  0001 C CNN "CPN"
+F 7 "700uW" H 1900 1700 50  0001 C CNN "R_P"
 	1    1900 1700
 	1    0    0    -1
@@
 F 5 "Bourns" H 1500 4100 50  0001 C CNN "Mfg"
 F 6 "232-00024" H 1500 4100 50  0001 C CNN "CPN"
+F 7 "300uW" H 1500 4100 50  0001 C CNN "R_P"
 	1    1500 4100
 	0    1    1    0
@@
 F 5 "Bourns" H 1700 1700 50  0001 C CNN "Mfg"
 F 6 "232-00024" H 1700 1700 50  0001 C CNN "CPN"
+F 7 "300uW" H 1700 1700 50  0001 C CNN "R_P"
 	1    1700 1700
 	1    0    0    -1
@@
 F 5 "KOA Speer Electronics" H 8900 2700 50  0001 C CNN "Mfg"
 F 6 "232-00030" H 8900 2700 50  0001 C CNN "CPN"
+F 7 "15mW" V 8900 2700 50  0001 C CNN "R_P"
 	1    8900 2700
 	0    1    1    0
@@
 F 5 "KOA Speer Electronics" H 8900 2900 50  0001 C CNN "Mfg"
 F 6 "232-00030" H 8900 2900 50  0001 C CNN "CPN"
+F 7 "15mW" H 8900 2900 50  0001 C CNN "R_P"
 	1    8900 2900
 	0    1    1    0
@@
 F 5 "KOA Speer Electronics" H 8900 5400 50  0001 C CNN "Mfg"
 F 6 "232-00030" H 8900 5400 50  0001 C CNN "CPN"
+F 7 "15mW" H 8900 5400 50  0001 C CNN "R_P"
 	1    8900 5400
 	0    1    1    0
@@
 F 5 "KOA Speer Electronics" H 8900 5600 50  0001 C CNN "Mfg"
 F 6 "232-00030" H 8900 5600 50  0001 C CNN "CPN"
+F 7 "15mW" H 8900 5600 50  0001 C CNN "R_P"
 	1    8900 5600
 	0    1    1    0
@@
 F 5 "Bourns" H 2500 1700 50  0001 C CNN "Mfg"
 F 6 "232-00024" H 2500 1700 50  0001 C CNN "CPN"
+F 7 "300uW" H 2500 1700 50  0001 C CNN "R_P"
 	1    2500 1700
 	-1   0    0    1

Commit message: sp-ethernet: recalculate and document crystal load caps
Parts:
- added R409: 0R, symbol Device:R
- C410, C411: value 18pF -> 30pF
Connections:
- net at C410.2, Y401.1: now also R409.2; no longer U401.15 (X2)
- new net: R409.1, U401.15 (X2)
Other:
- note added: "Cl1 = Cl2 = 2*Cl - Cpin\nCl1 = Cl2 = 31pF\n\nRext = 0\n\nGm_crit = 4*(ESR+Rext)*(2*pi*F)^2*(C0+Cl)^2\nGm_crit = 1.044 mA/V"
- note added: "Xtal:\nF = 25MHz\nC0 = 5pF\nCl = 18pF\nESR = 20R\n\nOscillator:\nCpin = unspecified, assume 5pF\nGm_crit_max = unspecified"
- moved on the sheet: C410, C411, Y401
Changed lines of the file:
@@
 $EndComp
 Connection ~ 10200 3250
-Wire Wire Line
-	6100 5500 6100 4500
-Wire Wire Line
-	6300 4400 6300 5500
 $Comp
 L Device:C_Small C410
 U 1 1 5F3C7DBF
-P 5900 5900
-F 0 "C410" H 5808 5854 50  0000 R CNN
-F 1 "18pF" H 5808 5945 50  0000 R CNN
-F 2 "Capacitor_SMD:C_0603_1608Metric" H 5900 5900 50  0001 C CNN
-F 3 "~" H 5900 5900 50  0001 C CNN
-F 4 "0603N180J500CT" H 5900 5900 50  0001 C CNN "Mfg Part Num"
-F 5 "Walsin Technology Corporation" H 5900 5900 50  0001 C CNN "Mfg"
-F 6 "212-00017" H 5900 5900 50  0001 C CNN "CPN"
-F 7 "3.3V" H 5900 5900 50  0001 C CNN "C_Vpp"
-	1    5900 5900
+P 5900 5600
+F 0 "C410" H 5808 5554 50  0000 R CNN
+F 1 "30pF" H 5808 5645 50  0000 R CNN
+F 2 "Capacitor_SMD:C_0603_1608Metric" H 5900 5600 50  0001 C CNN
+F 3 "~" H 5900 5600 50  0001 C CNN
+F 4 "0603N180J500CT" H 5900 5600 50  0001 C CNN "Mfg Part Num"
+F 5 "Walsin Technology Corporation" H 5900 5600 50  0001 C CNN "Mfg"
+F 6 "212-00017" H 5900 5600 50  0001 C CNN "CPN"
+F 7 "3.3V" H 5900 5600 50  0001 C CNN "C_Vpp"
+	1    5900 5600
 	-1   0    0    1
 $EndComp
@@
 L Device:C_Small C411
 U 1 1 5F3C8B0B
-P 6400 5900
-F 0 "C411" H 6308 5854 50  0000 R CNN
-F 1 "18pF" H 6308 5945 50  0000 R CNN
-F 2 "Capacitor_SMD:C_0603_1608Metric" H 6400 5900 50  0001 C CNN
-F 3 "~" H 6400 5900 50  0001 C CNN
-F 4 "0603N180J500CT" H 6400 5900 50  0001 C CNN "Mfg Part Num"
-F 5 "Walsin Technology Corporation" H 6400 5900 50  0001 C CNN "Mfg"
-F 6 "212-00017" H 6400 5900 50  0001 C CNN "CPN"
-F 7 "3.3V" H 6400 5900 50  0001 C CNN "C_Vpp"
-	1    6400 5900
+P 6750 5600
+F 0 "C411" H 6658 5554 50  0000 R CNN
+F 1 "30pF" H 6658 5645 50  0000 R CNN
+F 2 "Capacitor_SMD:C_0603_1608Metric" H 6750 5600 50  0001 C CNN
+F 3 "~" H 6750 5600 50  0001 C CNN
+F 4 "0603N180J500CT" H 6750 5600 50  0001 C CNN "Mfg Part Num"
+F 5 "Walsin Technology Corporation" H 6750 5600 50  0001 C CNN "Mfg"
+F 6 "212-00017" H 6750 5600 50  0001 C CNN "CPN"
+F 7 "3.3V" H 6750 5600 50  0001 C CNN "C_Vpp"
+	1    6750 5600
 	-1   0    0    1
 $EndComp
 Wire Wire Line
-	6100 5500 5900 5500
-Wire Wire Line
-	5900 5500 5900 5800
-Connection ~ 6100 5500
-Wire Wire Line
-	6300 5500 6400 5500
-Wire Wire Line
-	6400 5500 6400 5800
-Connection ~ 6300 5500
+	6450 5200 6750 5200
+Wire Wire Line
+	6750 5200 6750 5500
 $Comp
 L power:GND #PWR0416
 U 1 1 5F3DE90A
-P 5900 6000
-F 0 "#PWR0416" H 5900 5750 50  0001 C CNN
-F 1 "GND" H 5905 5827 50  0000 C CNN
-F 2 "" H 5900 6000 50  0001 C CNN
-F 3 "" H 5900 6000 50  0001 C CNN
-	1    5900 6000
+P 5900 5700
+F 0 "#PWR0416" H 5900 5450 50  0001 C CNN
+F 1 "GND" H 5905 5527 50  0000 C CNN
+F 2 "" H 5900 5700 50  0001 C CNN
+F 3 "" H 5900 5700 50  0001 C CNN
+	1    5900 5700
 	1    0    0    -1
 $EndComp
@@
 L power:GND #PWR0419
 U 1 1 5F3DEC98
-P 6400 6000
-F 0 "#PWR0419" H 6400 5750 50  0001 C CNN
-F 1 "GND" H 6405 5827 50  0000 C CNN
-F 2 "" H 6400 6000 50  0001 C CNN
-F 3 "" H 6400 6000 50  0001 C CNN
-	1    6400 6000
+P 6750 5700
+F 0 "#PWR0419" H 6750 5450 50  0001 C CNN
+F 1 "GND" H 6755 5527 50  0000 C CNN
+F 2 "" H 6750 5700 50  0001 C CNN
+F 3 "" H 6750 5700 50  0001 C CNN
+	1    6750 5700
 	1    0    0    -1
 $EndComp
@@
 	5500 3900 5500 4500
 Wire Wire Line
-	5500 4500 6100 4500
+	5500 4500 5900 4500
 Wire Wire Line
 	5050 3900 5500 3900
 Wire Wire Line
 	5600 3800 5600 4400
-Wire Wire Line
-	5600 4400 6300 4400
 Wire Wire Line
 	5050 3800 5600 3800
@@
 L Device:Crystal_Small Y401
 U 1 1 5F3B0977
-P 6200 5500
-F 0 "Y401" H 6344 5546 50  0000 L CNN
-F 1 "25MHz ±50ppm" H 6344 5455 50  0000 L CNN
-F 2 "Crystal:Crystal_SMD_5032-2Pin_5.0x3.2mm" H 6200 5500 50  0001 C CNN
-F 3 "~" H 6200 5500 50  0001 C CNN
-F 4 "Raltron Electronics" H 6200 5500 50  0001 C CNN "Mfg"
-F 5 "H130A-25.000-18-F-3030" H 6200 5500 50  0001 C CNN "Mfg Part Num"
-F 6 "216-00005" H 6200 5500 50  0001 C CNN "CPN"
-F 7 "" H 6200 5500 50  0001 C CNN "Config"
-F 8 "18pF" H 6200 5500 50  0001 C CNN "Y_Cl"
-	1    6200 5500
-	1    0    0    -1
-$EndComp
+P 6350 5200
+F 0 "Y401" H 6350 5450 50  0000 C CNN
+F 1 "25MHz ±50ppm" H 6350 5350 50  0000 C CNN
+F 2 "Crystal:Crystal_SMD_5032-2Pin_5.0x3.2mm" H 6350 5200 50  0001 C CNN
+F 3 "~" H 6350 5200 50  0001 C CNN
+F 4 "Raltron Electronics" H 6350 5200 50  0001 C CNN "Mfg"
+F 5 "H130A-25.000-18-F-3030" H 6350 5200 50  0001 C CNN "Mfg Part Num"
+F 6 "216-00005" H 6350 5200 50  0001 C CNN "CPN"
+F 7 "" H 6350 5200 50  0001 C CNN "Config"
+F 8 "18pF" H 6350 5200 50  0001 C CNN "Y_Cl"
+	1    6350 5200
+	1    0    0    -1
+$EndComp
+Text Notes 3050 6250 0    50   ~ 0
+Xtal:\nF = 25MHz\nC0 = 5pF\nCl = 18pF\nESR = 20R\n\nOscillator:\nCpin = unspecified, assume 5pF\nGm_crit_max = unspecified
+Text Notes 4450 6250 0    50   ~ 0
+Cl1 = Cl2 = 2*Cl - Cpin\nCl1 = Cl2 = 31pF\n\nRext = 0\n\nGm_crit = 4*(ESR+Rext)*(2*pi*F)^2*(C0+Cl)^2\nGm_crit = 1.044 mA/V
+Wire Wire Line
+	6750 4400 6750 5200
+Wire Wire Line
+	5600 4400 6750 4400
+Connection ~ 6750 5200
+Wire Wire Line
+	5900 5200 5900 5500
+Wire Wire Line
+	6250 5200 5900 5200
+Wire Wire Line
+	5900 4500 5900 4600
+$Comp
+L Device:R R409
+U 1 1 6011A892
+P 5900 4750
+F 0 "R409" H 6000 4800 50  0000 L CNN
+F 1 "0R" H 6000 4750 50  0000 L CNN
+F 2 "" V 5830 4750 50  0001 C CNN
+F 3 "~" H 5900 4750 50  0001 C CNN
+	1    5900 4750
+	1    0    0    -1
+$EndComp
+Wire Wire Line
+	5900 4900 5900 5200
+Connection ~ 5900 5200
 $EndSCHEMATC

Commit message: sp-ethernet: remove DNP capacitor between +3.3V and VDDA_3.3
May have been intended as an optional filter but as-is leaves VDDA_3.3
disconnected. If populated, VDDA_3.3 would be AC-coupled which also
doesn't work. Just remove entirely.
Parts:
- removed C422: DNP, Capacitor_SMD:C_0603_1608Metric, symbol Device:C_Small
Connections:
- net at U401.5 (VDDA_3.3): now also C407.1, C408.1, C418.2, C419.2, FB402.2, J401.4 (TCT), J401.7 (RCT), J402.4 (TCT), J402.7 (RCT)
Changed lines of the file:
@@
 	1    0    0    -1
 $EndComp
-$Comp
-L Device:C_Small C422
-U 1 1 5F3FCDA3
-P 5500 1750
-F 0 "C422" V 5271 1750 50  0000 C CNN
-F 1 "DNP" V 5362 1750 50  0000 C CNN
-F 2 "Capacitor_SMD:C_0603_1608Metric" H 5500 1750 50  0001 C CNN
-F 3 "~" H 5500 1750 50  0001 C CNN
-F 4 "" H 5500 1750 50  0001 C CNN "Mfg Part Num"
-F 5 "DNP" H 5500 1750 50  0001 C CNN "Config"
-	1    5500 1750
-	0    1    1    0
-$EndComp
-Wire Wire Line
-	5000 1750 5400 1750
 Connection ~ 5000 1750
-Wire Wire Line
-	5600 1750 5950 1750
 $Comp
 L Device:R R423
@@
 	5900 4900 5900 5200
 Connection ~ 5900 5200
+Wire Wire Line
+	5000 1750 5950 1750
 $EndSCHEMATC

Commit message: sp-ethernet: use correct CPN for 68R resistors
Parts:
- R419, R420, R421, R422: CPN 232-00030 -> 232-00020
Changed lines of the file:
@@
 F 4 "RK73B1JTTD181J" H 8900 2700 50  0001 C CNN "Mfg Part Num"
 F 5 "KOA Speer Electronics" H 8900 2700 50  0001 C CNN "Mfg"
-F 6 "232-00030" H 8900 2700 50  0001 C CNN "CPN"
+F 6 "232-00020" H 8900 2700 50  0001 C CNN "CPN"
 F 7 "15mW" V 8900 2700 50  0001 C CNN "R_P"
 	1    8900 2700
@@
 F 4 "RK73B1JTTD181J" H 8900 2900 50  0001 C CNN "Mfg Part Num"
 F 5 "KOA Speer Electronics" H 8900 2900 50  0001 C CNN "Mfg"
-F 6 "232-00030" H 8900 2900 50  0001 C CNN "CPN"
+F 6 "232-00020" H 8900 2900 50  0001 C CNN "CPN"
 F 7 "15mW" H 8900 2900 50  0001 C CNN "R_P"
 	1    8900 2900
@@
 F 4 "RK73B1JTTD181J" H 8900 5400 50  0001 C CNN "Mfg Part Num"
 F 5 "KOA Speer Electronics" H 8900 5400 50  0001 C CNN "Mfg"
-F 6 "232-00030" H 8900 5400 50  0001 C CNN "CPN"
+F 6 "232-00020" H 8900 5400 50  0001 C CNN "CPN"
 F 7 "15mW" H 8900 5400 50  0001 C CNN "R_P"
 	1    8900 5400
@@
 F 4 "RK73B1JTTD181J" H 8900 5600 50  0001 C CNN "Mfg Part Num"
 F 5 "KOA Speer Electronics" H 8900 5600 50  0001 C CNN "Mfg"
-F 6 "232-00030" H 8900 5600 50  0001 C CNN "CPN"
+F 6 "232-00020" H 8900 5600 50  0001 C CNN "CPN"
 F 7 "15mW" H 8900 5600 50  0001 C CNN "R_P"
 	1    8900 5600
