File: fans.sch (KiCad schematic (older format))
At the start: 26 parts, among them J701 FAN6, J702 FAN5, J703 FAN4, J704 FAN3, J705 FAN2, J706 FAN1, U701 MAX31790, U702 MCP1703A-5002_SOT89, U703 PCA9306DP

Commit message: MB: MPNs for capacitors, adjust some footprints
Can't get a 2kV 10000p cap in 0603 as it turns out
Parts:
- C701, C702: Mfg (none) -> Samsung Electro-Mechanics; Mfg Part Num generic -> CL10B105KP8NFNC
Changed lines of the file:
@@
 F 2 "Capacitor_SMD:C_0603_1608Metric" H 2450 1600 50  0001 C CNN
 F 3 "~" H 2450 1600 50  0001 C CNN
-F 4 "generic" H 2450 1600 50  0001 C CNN "Mfg Part Num"
+F 4 "CL10B105KP8NFNC" H 2450 1600 50  0001 C CNN "Mfg Part Num"
+F 5 "Samsung Electro-Mechanics" H 2450 1600 50  0001 C CNN "Mfg"
 	1    2450 1600
 	1    0    0    -1
@@
 F 2 "Capacitor_SMD:C_0603_1608Metric" H 3600 1600 50  0001 C CNN
 F 3 "~" H 3600 1600 50  0001 C CNN
-F 4 "generic" H 3600 1600 50  0001 C CNN "Mfg Part Num"
+F 4 "CL10B105KP8NFNC" H 3600 1600 50  0001 C CNN "Mfg Part Num"
+F 5 "Samsung Electro-Mechanics" H 3600 1600 50  0001 C CNN "Mfg"
 	1    3600 1600
 	1    0    0    -1

Commit message: MB: assign single resistors
Parts:
- R701: Mfg (none) -> KOA Speer Electronics; Mfg Part Num generic -> RK73B1JTTD204J
- R702, R703, R704, R705, R706, R707, R708, R709, R710, R711, R712, R713, R714, R715: Mfg (none) -> Bourns; Mfg Part Num generic -> CR0603-JW-332ELF
Changed lines of the file:
@@
 F 2 "Resistor_SMD:R_0603_1608Metric" V 2130 2000 50  0001 C CNN
 F 3 "~" H 2200 2000 50  0001 C CNN
-F 4 "generic" H 2200 2000 50  0001 C CNN "Mfg Part Num"
+F 4 "RK73B1JTTD204J" H 2200 2000 50  0001 C CNN "Mfg Part Num"
+F 5 "KOA Speer Electronics" H 2200 2000 50  0001 C CNN "Mfg"
 	1    2200 2000
 	1    0    0    -1
@@
 F 2 "Resistor_SMD:R_0603_1608Metric" V 2680 2400 50  0001 C CNN
 F 3 "~" H 2750 2400 50  0001 C CNN
-F 4 "generic" H 2750 2400 50  0001 C CNN "Mfg Part Num"
+F 4 "CR0603-JW-332ELF" H 2750 2400 50  0001 C CNN "Mfg Part Num"
+F 5 "Bourns" H 2750 2400 50  0001 C CNN "Mfg"
 	1    2750 2400
 	1    0    0    -1
@@
 F 2 "Resistor_SMD:R_0603_1608Metric" V 2930 2400 50  0001 C CNN
 F 3 "~" H 3000 2400 50  0001 C CNN
-F 4 "generic" H 3000 2400 50  0001 C CNN "Mfg Part Num"
+F 4 "CR0603-JW-332ELF" H 3000 2400 50  0001 C CNN "Mfg Part Num"
+F 5 "Bourns" H 3000 2400 50  0001 C CNN "Mfg"
 	1    3000 2400
 	1    0    0    -1
@@
 F 2 "Resistor_SMD:R_0603_1608Metric" V 5880 1450 50  0001 C CNN
 F 3 "~" H 5950 1450 50  0001 C CNN
-F 4 "generic" H 5950 1450 50  0001 C CNN "Mfg Part Num"
+F 4 "CR0603-JW-332ELF" H 5950 1450 50  0001 C CNN "Mfg Part Num"
+F 5 "Bourns" H 5950 1450 50  0001 C CNN "Mfg"
 	1    5950 1450
 	1    0    0    -1
@@
 F 2 "Resistor_SMD:R_0603_1608Metric" V 5980 1450 50  0001 C CNN
 F 3 "~" H 6050 1450 50  0001 C CNN
-F 4 "generic" H 6050 1450 50  0001 C CNN "Mfg Part Num"
+F 4 "CR0603-JW-332ELF" H 6050 1450 50  0001 C CNN "Mfg Part Num"
+F 5 "Bourns" H 6050 1450 50  0001 C CNN "Mfg"
 	1    6050 1450
 	1    0    0    -1
@@
 F 2 "Resistor_SMD:R_0603_1608Metric" V 6080 1450 50  0001 C CNN
 F 3 "~" H 6150 1450 50  0001 C CNN
-F 4 "generic" H 6150 1450 50  0001 C CNN "Mfg Part Num"
+F 4 "CR0603-JW-332ELF" H 6150 1450 50  0001 C CNN "Mfg Part Num"
+F 5 "Bourns" H 6150 1450 50  0001 C CNN "Mfg"
 	1    6150 1450
 	1    0    0    -1
@@
 F 2 "Resistor_SMD:R_0603_1608Metric" V 6180 1450 50  0001 C CNN
 F 3 "~" H 6250 1450 50  0001 C CNN
-F 4 "generic" H 6250 1450 50  0001 C CNN "Mfg Part Num"
+F 4 "CR0603-JW-332ELF" H 6250 1450 50  0001 C CNN "Mfg Part Num"
+F 5 "Bourns" H 6250 1450 50  0001 C CNN "Mfg"
 	1    6250 1450
 	1    0    0    -1
@@
 F 2 "Resistor_SMD:R_0603_1608Metric" V 6430 1450 50  0001 C CNN
 F 3 "~" H 6500 1450 50  0001 C CNN
-F 4 "generic" H 6500 1450 50  0001 C CNN "Mfg Part Num"
+F 4 "CR0603-JW-332ELF" H 6500 1450 50  0001 C CNN "Mfg Part Num"
+F 5 "Bourns" H 6500 1450 50  0001 C CNN "Mfg"
 	1    6500 1450
 	1    0    0    -1
@@
 F 2 "Resistor_SMD:R_0603_1608Metric" V 6530 1450 50  0001 C CNN
 F 3 "~" H 6600 1450 50  0001 C CNN
-F 4 "generic" H 6600 1450 50  0001 C CNN "Mfg Part Num"
+F 4 "CR0603-JW-332ELF" H 6600 1450 50  0001 C CNN "Mfg Part Num"
+F 5 "Bourns" H 6600 1450 50  0001 C CNN "Mfg"
 	1    6600 1450
 	1    0    0    -1
@@
 F 2 "Resistor_SMD:R_0603_1608Metric" V 6630 1450 50  0001 C CNN
 F 3 "~" H 6700 1450 50  0001 C CNN
-F 4 "generic" H 6700 1450 50  0001 C CNN "Mfg Part Num"
+F 4 "CR0603-JW-332ELF" H 6700 1450 50  0001 C CNN "Mfg Part Num"
+F 5 "Bourns" H 6700 1450 50  0001 C CNN "Mfg"
 	1    6700 1450
 	1    0    0    -1
@@
 F 2 "Resistor_SMD:R_0603_1608Metric" V 6730 1450 50  0001 C CNN
 F 3 "~" H 6800 1450 50  0001 C CNN
-F 4 "generic" H 6800 1450 50  0001 C CNN "Mfg Part Num"
+F 4 "CR0603-JW-332ELF" H 6800 1450 50  0001 C CNN "Mfg Part Num"
+F 5 "Bourns" H 6800 1450 50  0001 C CNN "Mfg"
 	1    6800 1450
 	1    0    0    -1
@@
 F 2 "Resistor_SMD:R_0603_1608Metric" V 6930 1450 50  0001 C CNN
 F 3 "~" H 7000 1450 50  0001 C CNN
-F 4 "generic" H 7000 1450 50  0001 C CNN "Mfg Part Num"
+F 4 "CR0603-JW-332ELF" H 7000 1450 50  0001 C CNN "Mfg Part Num"
+F 5 "Bourns" H 7000 1450 50  0001 C CNN "Mfg"
 	1    7000 1450
 	1    0    0    -1
@@
 F 2 "Resistor_SMD:R_0603_1608Metric" V 7030 1450 50  0001 C CNN
 F 3 "~" H 7100 1450 50  0001 C CNN
-F 4 "generic" H 7100 1450 50  0001 C CNN "Mfg Part Num"
+F 4 "CR0603-JW-332ELF" H 7100 1450 50  0001 C CNN "Mfg Part Num"
+F 5 "Bourns" H 7100 1450 50  0001 C CNN "Mfg"
 	1    7100 1450
 	1    0    0    -1
@@
 F 2 "Resistor_SMD:R_0603_1608Metric" V 7130 1450 50  0001 C CNN
 F 3 "~" H 7200 1450 50  0001 C CNN
-F 4 "generic" H 7200 1450 50  0001 C CNN "Mfg Part Num"
+F 4 "CR0603-JW-332ELF" H 7200 1450 50  0001 C CNN "Mfg Part Num"
+F 5 "Bourns" H 7200 1450 50  0001 C CNN "Mfg"
 	1    7200 1450
 	1    0    0    -1
@@
 F 2 "Resistor_SMD:R_0603_1608Metric" V 7230 1450 50  0001 C CNN
 F 3 "~" H 7300 1450 50  0001 C CNN
-F 4 "generic" H 7300 1450 50  0001 C CNN "Mfg Part Num"
+F 4 "CR0603-JW-332ELF" H 7300 1450 50  0001 C CNN "Mfg Part Num"
+F 5 "Bourns" H 7300 1450 50  0001 C CNN "Mfg"
 	1    7300 1450
 	1    0    0    -1

Commit message: MB: add caps suggested in review
Parts:
- added C703, C704: 0µ1, Capacitor_SMD:C_0603_1608Metric, symbol Device:C_Small
Connections:
- net +3V3: now also C703.1
- net FAN5V: now also C704.1
- net GND: now also C703.2, C704.2
Changed lines of the file:
@@
 Text Label 3950 1400 0    50   ~ 0
 FAN5V
-Text Label 5750 1300 2    50   ~ 0
+Text Label 4750 1300 2    50   ~ 0
 FAN5V
 Text Label 4550 2450 1    50   ~ 0
@@
 $EndComp
 Wire Wire Line
-	5750 1300 5950 1300
+	4750 1300 4900 1300
 Connection ~ 5950 1300
 Wire Wire Line
@@
 Wire Wire Line
 	7200 1300 7300 1300
+$Comp
+L Device:C_Small C?
+U 1 1 5F6D6DB8
+P 4900 1400
+AR Path="/5F1928E5/5F29584B/5F6D6DB8" Ref="C?"  Part="1"
+AR Path="/5F24B563/5F6D6DB8" Ref="C704"  Part="1"
+F 0 "C704" H 4992 1446 50  0000 L CNN
+F 1 "0µ1" H 4992 1355 50  0000 L CNN
+F 2 "Capacitor_SMD:C_0603_1608Metric" H 4900 1400 50  0001 C CNN
+F 3 "~" H 4900 1400 50  0001 C CNN
+F 4 "CL10B104KB8NNWC" H 4900 1400 50  0001 C CNN "Mfg Part Num"
+F 5 "Samsung Electro-Mechanics" H 4900 1400 50  0001 C CNN "Mfg"
+	1    4900 1400
+	1    0    0    -1
+$EndComp
+Connection ~ 4900 1300
+Wire Wire Line
+	4900 1300 5950 1300
+$Comp
+L power:GND #PWR0710
+U 1 1 5F6D94F0
+P 4900 1500
+F 0 "#PWR0710" H 4900 1250 50  0001 C CNN
+F 1 "GND" H 4905 1327 50  0000 C CNN
+F 2 "" H 4900 1500 50  0001 C CNN
+F 3 "" H 4900 1500 50  0001 C CNN
+	1    4900 1500
+	1    0    0    -1
+$EndComp
+$Comp
+L Device:C_Small C?
+U 1 1 5F6D9DA4
+P 1300 3650
+AR Path="/5F1928E5/5F29584B/5F6D9DA4" Ref="C?"  Part="1"
+AR Path="/5F24B563/5F6D9DA4" Ref="C703"  Part="1"
+F 0 "C703" H 1392 3696 50  0000 L CNN
+F 1 "0µ1" H 1392 3605 50  0000 L CNN
+F 2 "Capacitor_SMD:C_0603_1608Metric" H 1300 3650 50  0001 C CNN
+F 3 "~" H 1300 3650 50  0001 C CNN
+F 4 "CL10B104KB8NNWC" H 1300 3650 50  0001 C CNN "Mfg Part Num"
+F 5 "Samsung Electro-Mechanics" H 1300 3650 50  0001 C CNN "Mfg"
+	1    1300 3650
+	1    0    0    -1
+$EndComp
+$Comp
+L power:+3V3 #PWR0705
+U 1 1 5F6DAF5B
+P 1300 3550
+F 0 "#PWR0705" H 1300 3400 50  0001 C CNN
+F 1 "+3V3" H 1315 3723 50  0000 C CNN
+F 2 "" H 1300 3550 50  0001 C CNN
+F 3 "" H 1300 3550 50  0001 C CNN
+	1    1300 3550
+	1    0    0    -1
+$EndComp
+$Comp
+L power:GND #PWR0709
+U 1 1 5F6DB2FB
+P 1300 3750
+F 0 "#PWR0709" H 1300 3500 50  0001 C CNN
+F 1 "GND" H 1305 3577 50  0000 C CNN
+F 2 "" H 1300 3750 50  0001 C CNN
+F 3 "" H 1300 3750 50  0001 C CNN
+	1    1300 3750
+	1    0    0    -1
+$EndComp
 $EndSCHEMATC

Commit message: fans: include package code in MCP1703A-5002 MPN
Resolves #36
Parts:
- U702: Mfg Part Num MCP1703A-5002 -> MCP1703AT-5002E/MB
Changed lines of the file:
@@
 F 3 "http://ww1.microchip.com/downloads/en/DeviceDoc/20005122B.pdf" H 3150 1350 50  0001 C CNN
 F 4 "Microchip" H 3150 1400 50  0001 C CNN "Mfg"
-F 5 "MCP1703A-5002" H 3150 1400 50  0001 C CNN "Mfg Part Num"
+F 5 "MCP1703AT-5002E/MB" H 3150 1400 50  0001 C CNN "Mfg Part Num"
 	1    3150 1400
 	1    0    0    -1

Commit message: fans: expand PCA9306DP to full, orderable MPN
Parts:
- U703: value PCA9306DP -> PCA9306DP1; Mfg Part Num PCA9306DP -> PCA9306DP1,125
Changed lines of the file:
@@
 P 1800 2750
 F 0 "U703" H 2000 3200 50  0000 C CNN
-F 1 "PCA9306DP" H 2050 2300 50  0000 C CNN
+F 1 "PCA9306DP1" H 2050 2300 50  0000 C CNN
 F 2 "Package_SO:TSSOP-8_3x3mm_P0.65mm" H 1800 2300 50  0001 C CNN
 F 3 "https://www.nxp.com/docs/en/data-sheet/PCA9306.pdf" H 1500 3200 50  0001 C CNN
 F 4 "NXP" H 1800 2750 50  0001 C CNN "Mfg"
-F 5 "PCA9306DP" H 1800 2750 50  0001 C CNN "Mfg Part Num"
+F 5 "PCA9306DP1,125" H 1800 2750 50  0001 C CNN "Mfg Part Num"
 	1    1800 2750
 	1    0    0    -1

Commit message: fans: expand MAX31790 to full, orderable MPN
Parts:
- U701: Mfg Part Num MAX31790 -> MAX31790ATI+
Changed lines of the file:
@@
 F 3 "" H 4550 3350 50  0001 C CNN
 F 4 "Maxim" H 4550 3350 50  0001 C CNN "Mfg"
-F 5 "MAX31790" H 4550 3350 50  0001 C CNN "Mfg Part Num"
+F 5 "MAX31790ATI+" H 4550 3350 50  0001 C CNN "Mfg Part Num"
 	1    4550 3350
 	1    0    0    -1

Commit message: gemini-bringup: Add CPNs for all components
Parts:
- C701, C702: CPN (none) -> 212-00015
- C703, C704: CPN (none) -> 212-00011
- J701, J702, J703, J704, J705, J706: CPN (none) -> 215-00029
- R701: CPN (none) -> 232-00033
- R702, R703, R704, R705, R706, R707, R708, R709, R710, R711, R712, R713, R714, R715: CPN (none) -> 232-00018
- U701: CPN (none) -> 221-00016
- U702: CPN (none) -> 229-00004
- U703: CPN (none) -> 221-00018
Changed lines of the file:
@@
 F 4 "Molex" H 9450 4200 50  0001 C CNN "Mfg"
 F 5 "0740991005" H 9450 4200 50  0001 C CNN "Mfg Part Num"
+F 6 "215-00029" H 9450 4200 50  0001 C CNN "CPN"
 	1    9450 4200
 	1    0    0    -1
@@
 F 4 "Molex" H 9450 3550 50  0001 C CNN "Mfg"
 F 5 "0740991005" H 9450 3550 50  0001 C CNN "Mfg Part Num"
+F 6 "215-00029" H 9450 3550 50  0001 C CNN "CPN"
 	1    9450 3550
 	1    0    0    -1
@@
 F 4 "Molex" H 9450 2900 50  0001 C CNN "Mfg"
 F 5 "0740991005" H 9450 2900 50  0001 C CNN "Mfg Part Num"
+F 6 "215-00029" H 9450 2900 50  0001 C CNN "CPN"
 	1    9450 2900
 	1    0    0    -1
@@
 F 4 "Molex" H 8150 4200 50  0001 C CNN "Mfg"
 F 5 "0740991005" H 8150 4200 50  0001 C CNN "Mfg Part Num"
+F 6 "215-00029" H 8150 4200 50  0001 C CNN "CPN"
 	1    8150 4200
 	1    0    0    -1
@@
 F 4 "Molex" H 8150 3550 50  0001 C CNN "Mfg"
 F 5 "0740991005" H 8150 3550 50  0001 C CNN "Mfg Part Num"
+F 6 "215-00029" H 8150 3550 50  0001 C CNN "CPN"
 	1    8150 3550
 	1    0    0    -1
@@
 F 4 "Molex" H 8150 2900 50  0001 C CNN "Mfg"
 F 5 "0740991005" H 8150 2900 50  0001 C CNN "Mfg Part Num"
+F 6 "215-00029" H 8150 2900 50  0001 C CNN "CPN"
 	1    8150 2900
 	1    0    0    -1
@@
 F 4 "Maxim" H 4550 3350 50  0001 C CNN "Mfg"
 F 5 "MAX31790ATI+" H 4550 3350 50  0001 C CNN "Mfg Part Num"
+F 6 "221-00016" H 4550 3350 50  0001 C CNN "CPN"
 	1    4550 3350
 	1    0    0    -1
@@
 F 4 "Microchip" H 3150 1400 50  0001 C CNN "Mfg"
 F 5 "MCP1703AT-5002E/MB" H 3150 1400 50  0001 C CNN "Mfg Part Num"
+F 6 "229-00004" H 3150 1400 50  0001 C CNN "CPN"
 	1    3150 1400
 	1    0    0    -1
@@
 F 4 "CL10B105KP8NFNC" H 2450 1600 50  0001 C CNN "Mfg Part Num"
 F 5 "Samsung Electro-Mechanics" H 2450 1600 50  0001 C CNN "Mfg"
+F 6 "212-00015" H 2450 1600 50  0001 C CNN "CPN"
 	1    2450 1600
 	1    0    0    -1
@@
 F 4 "CL10B105KP8NFNC" H 3600 1600 50  0001 C CNN "Mfg Part Num"
 F 5 "Samsung Electro-Mechanics" H 3600 1600 50  0001 C CNN "Mfg"
+F 6 "212-00015" H 3600 1600 50  0001 C CNN "CPN"
 	1    3600 1600
 	1    0    0    -1
@@
 F 4 "NXP" H 1800 2750 50  0001 C CNN "Mfg"
 F 5 "PCA9306DP1,125" H 1800 2750 50  0001 C CNN "Mfg Part Num"
+F 6 "221-00018" H 1800 2750 50  0001 C CNN "CPN"
 	1    1800 2750
 	1    0    0    -1
@@
 F 4 "RK73B1JTTD204J" H 2200 2000 50  0001 C CNN "Mfg Part Num"
 F 5 "KOA Speer Electronics" H 2200 2000 50  0001 C CNN "Mfg"
+F 6 "232-00033" H 2200 2000 50  0001 C CNN "CPN"
 	1    2200 2000
 	1    0    0    -1
@@
 F 4 "CR0603-JW-332ELF" H 2750 2400 50  0001 C CNN "Mfg Part Num"
 F 5 "Bourns" H 2750 2400 50  0001 C CNN "Mfg"
+F 6 "232-00018" H 2750 2400 50  0001 C CNN "CPN"
 	1    2750 2400
 	1    0    0    -1
@@
 F 4 "CR0603-JW-332ELF" H 3000 2400 50  0001 C CNN "Mfg Part Num"
 F 5 "Bourns" H 3000 2400 50  0001 C CNN "Mfg"
+F 6 "232-00018" H 3000 2400 50  0001 C CNN "CPN"
 	1    3000 2400
 	1    0    0    -1
@@
 F 4 "CR0603-JW-332ELF" H 5950 1450 50  0001 C CNN "Mfg Part Num"
 F 5 "Bourns" H 5950 1450 50  0001 C CNN "Mfg"
+F 6 "232-00018" H 5950 1450 50  0001 C CNN "CPN"
 	1    5950 1450
 	1    0    0    -1
@@
 F 4 "CR0603-JW-332ELF" H 6050 1450 50  0001 C CNN "Mfg Part Num"
 F 5 "Bourns" H 6050 1450 50  0001 C CNN "Mfg"
+F 6 "232-00018" H 6050 1450 50  0001 C CNN "CPN"
 	1    6050 1450
 	1    0    0    -1
@@
 F 4 "CR0603-JW-332ELF" H 6150 1450 50  0001 C CNN "Mfg Part Num"
 F 5 "Bourns" H 6150 1450 50  0001 C CNN "Mfg"
+F 6 "232-00018" H 6150 1450 50  0001 C CNN "CPN"
 	1    6150 1450
 	1    0    0    -1
@@
 F 4 "CR0603-JW-332ELF" H 6250 1450 50  0001 C CNN "Mfg Part Num"
 F 5 "Bourns" H 6250 1450 50  0001 C CNN "Mfg"
+F 6 "232-00018" H 6250 1450 50  0001 C CNN "CPN"
 	1    6250 1450
 	1    0    0    -1
@@
 F 4 "CR0603-JW-332ELF" H 6500 1450 50  0001 C CNN "Mfg Part Num"
 F 5 "Bourns" H 6500 1450 50  0001 C CNN "Mfg"
+F 6 "232-00018" H 6500 1450 50  0001 C CNN "CPN"
 	1    6500 1450
 	1    0    0    -1
@@
 F 4 "CR0603-JW-332ELF" H 6600 1450 50  0001 C CNN "Mfg Part Num"
 F 5 "Bourns" H 6600 1450 50  0001 C CNN "Mfg"
+F 6 "232-00018" H 6600 1450 50  0001 C CNN "CPN"
 	1    6600 1450
 	1    0    0    -1
@@
 F 4 "CR0603-JW-332ELF" H 6700 1450 50  0001 C CNN "Mfg Part Num"
 F 5 "Bourns" H 6700 1450 50  0001 C CNN "Mfg"
+F 6 "232-00018" H 6700 1450 50  0001 C CNN "CPN"
 	1    6700 1450
 	1    0    0    -1
@@
 F 4 "CR0603-JW-332ELF" H 6800 1450 50  0001 C CNN "Mfg Part Num"
 F 5 "Bourns" H 6800 1450 50  0001 C CNN "Mfg"
+F 6 "232-00018" H 6800 1450 50  0001 C CNN "CPN"
 	1    6800 1450
 	1    0    0    -1
@@
 F 4 "CR0603-JW-332ELF" H 7000 1450 50  0001 C CNN "Mfg Part Num"
 F 5 "Bourns" H 7000 1450 50  0001 C CNN "Mfg"
+F 6 "232-00018" H 7000 1450 50  0001 C CNN "CPN"
 	1    7000 1450
 	1    0    0    -1
@@
 F 4 "CR0603-JW-332ELF" H 7100 1450 50  0001 C CNN "Mfg Part Num"
 F 5 "Bourns" H 7100 1450 50  0001 C CNN "Mfg"
+F 6 "232-00018" H 7100 1450 50  0001 C CNN "CPN"
 	1    7100 1450
 	1    0    0    -1
@@
 F 4 "CR0603-JW-332ELF" H 7200 1450 50  0001 C CNN "Mfg Part Num"
 F 5 "Bourns" H 7200 1450 50  0001 C CNN "Mfg"
+F 6 "232-00018" H 7200 1450 50  0001 C CNN "CPN"
 	1    7200 1450
 	1    0    0    -1
@@
 F 4 "CR0603-JW-332ELF" H 7300 1450 50  0001 C CNN "Mfg Part Num"
 F 5 "Bourns" H 7300 1450 50  0001 C CNN "Mfg"
+F 6 "232-00018" H 7300 1450 50  0001 C CNN "CPN"
 	1    7300 1450
 	1    0    0    -1
@@
 F 4 "CL10B104KB8NNWC" H 4900 1400 50  0001 C CNN "Mfg Part Num"
 F 5 "Samsung Electro-Mechanics" H 4900 1400 50  0001 C CNN "Mfg"
+F 6 "212-00011" H 4900 1400 50  0001 C CNN "CPN"
 	1    4900 1400
 	1    0    0    -1
@@
 F 4 "CL10B104KB8NNWC" H 1300 3650 50  0001 C CNN "Mfg Part Num"
 F 5 "Samsung Electro-Mechanics" H 1300 3650 50  0001 C CNN "Mfg"
+F 6 "212-00011" H 1300 3650 50  0001 C CNN "CPN"
 	1    1300 3650
 	1    0    0    -1
