File: fans.sch (KiCad schematic (older format))
At the start: 28 parts, among them J701 FAN6, J702 FAN5, J703 FAN4, J704 FAN3, J705 FAN2, J706 FAN1, U701 MAX31790, U702 MCP1703A-5002_SOT89, U703 PCA9306DP1

Commit message: fans: specify rating constraints on passives
Parts:
- C701: value 1µ -> 1uF 12VDCbias
- C702: value 1µ -> 1uF 5VDCbias
- C703: value 0µ1 -> 0.1uF 3.3VDCbias
- C704: value 0µ1 -> 0.1uF 5VDCbias
- R701: value 200k -> 200kR
- R702, R703, R704, R705, R706, R707, R708, R709, R710, R711, R712, R713, R714, R715: value 3k3 -> 3.3kR
Other:
- moved on the sheet: C701
Changed lines of the file:
@@
 L Device:C_Small C701
 U 1 1 5F48A9CC
-P 2450 1600
-F 0 "C701" H 2542 1646 50  0000 L CNN
-F 1 "1µ" H 2542 1555 50  0000 L CNN
-F 2 "Capacitor_SMD:C_0603_1608Metric" H 2450 1600 50  0001 C CNN
-F 3 "~" H 2450 1600 50  0001 C CNN
-F 4 "CL10B105KP8NFNC" H 2450 1600 50  0001 C CNN "Mfg Part Num"
-F 5 "Samsung Electro-Mechanics" H 2450 1600 50  0001 C CNN "Mfg"
-F 6 "212-00015" H 2450 1600 50  0001 C CNN "CPN"
-	1    2450 1600
+P 2200 1600
+F 0 "C701" H 2292 1646 50  0000 L CNN
+F 1 "1uF 12VDCbias" H 2292 1555 50  0000 L CNN
+F 2 "Capacitor_SMD:C_0603_1608Metric" H 2200 1600 50  0001 C CNN
+F 3 "~" H 2200 1600 50  0001 C CNN
+F 4 "CL10B105KP8NFNC" H 2200 1600 50  0001 C CNN "Mfg Part Num"
+F 5 "Samsung Electro-Mechanics" H 2200 1600 50  0001 C CNN "Mfg"
+F 6 "212-00015" H 2200 1600 50  0001 C CNN "CPN"
+	1    2200 1600
 	1    0    0    -1
 $EndComp
@@
 P 3600 1600
 F 0 "C702" H 3692 1646 50  0000 L CNN
-F 1 "1µ" H 3692 1555 50  0000 L CNN
+F 1 "1uF 5VDCbias" H 3692 1555 50  0000 L CNN
 F 2 "Capacitor_SMD:C_0603_1608Metric" H 3600 1600 50  0001 C CNN
 F 3 "~" H 3600 1600 50  0001 C CNN
@@
 Connection ~ 3150 1700
 Wire Wire Line
-	3150 1700 2450 1700
-Wire Wire Line
-	2450 1500 2450 1400
-Wire Wire Line
-	2450 1400 2850 1400
+	3150 1700 2200 1700
+Wire Wire Line
+	2200 1500 2200 1400
+Wire Wire Line
+	2200 1400 2850 1400
 $Comp
 L power:+12V #PWR0706
 U 1 1 5F495AE2
-P 2450 1400
-F 0 "#PWR0706" H 2450 1250 50  0001 C CNN
-F 1 "+12V" H 2465 1573 50  0000 C CNN
-F 2 "" H 2450 1400 50  0001 C CNN
-F 3 "" H 2450 1400 50  0001 C CNN
-	1    2450 1400
-	1    0    0    -1
-$EndComp
-Connection ~ 2450 1400
+P 2200 1400
+F 0 "#PWR0706" H 2200 1250 50  0001 C CNN
+F 1 "+12V" H 2215 1573 50  0000 C CNN
+F 2 "" H 2200 1400 50  0001 C CNN
+F 3 "" H 2200 1400 50  0001 C CNN
+	1    2200 1400
+	1    0    0    -1
+$EndComp
+Connection ~ 2200 1400
 Wire Wire Line
 	3600 1400 3950 1400
@@
 	1    0    0    -1
 $EndComp
-$Comp
-L Device:R R701
-U 1 1 5F4BDB11
-P 2200 2000
-F 0 "R701" H 2270 2046 50  0000 L CNN
-F 1 "200k" V 2200 1900 50  0000 L CNN
-F 2 "Resistor_SMD:R_0603_1608Metric" V 2130 2000 50  0001 C CNN
-F 3 "~" H 2200 2000 50  0001 C CNN
-F 4 "RK73B1JTTD204J" H 2200 2000 50  0001 C CNN "Mfg Part Num"
-F 5 "KOA Speer Electronics" H 2200 2000 50  0001 C CNN "Mfg"
-F 6 "232-00033" H 2200 2000 50  0001 C CNN "CPN"
-	1    2200 2000
-	1    0    0    -1
-$EndComp
 Wire Wire Line
 	1900 2250 1900 2150
@@
 U 1 1 5F4E01D9
 P 2750 2400
-F 0 "R702" H 2820 2446 50  0000 L CNN
-F 1 "3k3" V 2750 2300 50  0000 L CNN
+F 0 "R702" H 2450 2450 50  0000 L CNN
+F 1 "3.3kR" H 2450 2350 50  0000 L CNN
 F 2 "Resistor_SMD:R_0603_1608Metric" V 2680 2400 50  0001 C CNN
 F 3 "~" H 2750 2400 50  0001 C CNN
@@
 U 1 1 5F4E073B
 P 3000 2400
-F 0 "R703" H 3070 2446 50  0000 L CNN
-F 1 "3k3" V 3000 2300 50  0000 L CNN
+F 0 "R703" H 3100 2450 50  0000 L CNN
+F 1 "3.3kR" H 3100 2350 50  0000 L CNN
 F 2 "Resistor_SMD:R_0603_1608Metric" V 2930 2400 50  0001 C CNN
 F 3 "~" H 3000 2400 50  0001 C CNN
@@
 U 1 1 5F596D71
 P 5950 1450
-F 0 "R704" V 5900 1550 50  0000 L CNN
-F 1 "3k3" V 5950 1400 50  0000 L CNN
+F 0 "R704" V 5950 1650 50  0000 L CNN
+F 1 "3.3kR" V 5950 1900 50  0000 L CNN
 F 2 "Resistor_SMD:R_0603_1608Metric" V 5880 1450 50  0001 C CNN
 F 3 "~" H 5950 1450 50  0001 C CNN
@@
 U 1 1 5F597263
 P 6050 1450
-F 0 "R705" V 6000 1550 50  0000 L CNN
-F 1 "3k3" V 6050 1400 50  0000 L CNN
+F 0 "R705" V 6050 1650 50  0000 L CNN
+F 1 "3.3kR" V 6050 1900 50  0000 L CNN
 F 2 "Resistor_SMD:R_0603_1608Metric" V 5980 1450 50  0001 C CNN
 F 3 "~" H 6050 1450 50  0001 C CNN
@@
 U 1 1 5F597494
 P 6150 1450
-F 0 "R706" V 6100 1550 50  0000 L CNN
-F 1 "3k3" V 6150 1400 50  0000 L CNN
+F 0 "R706" V 6150 1650 50  0000 L CNN
+F 1 "3.3kR" V 6150 1900 50  0000 L CNN
 F 2 "Resistor_SMD:R_0603_1608Metric" V 6080 1450 50  0001 C CNN
 F 3 "~" H 6150 1450 50  0001 C CNN
@@
 U 1 1 5F597612
 P 6250 1450
-F 0 "R707" V 6200 1550 50  0000 L CNN
-F 1 "3k3" V 6250 1400 50  0000 L CNN
+F 0 "R707" V 6250 1650 50  0000 L CNN
+F 1 "3.3kR" V 6250 1900 50  0000 L CNN
 F 2 "Resistor_SMD:R_0603_1608Metric" V 6180 1450 50  0001 C CNN
 F 3 "~" H 6250 1450 50  0001 C CNN
@@
 U 1 1 5F5986DF
 P 6500 1450
-F 0 "R708" V 6450 1550 50  0000 L CNN
-F 1 "3k3" V 6500 1400 50  0000 L CNN
+F 0 "R708" V 6500 1650 50  0000 L CNN
+F 1 "3.3kR" V 6500 1900 50  0000 L CNN
 F 2 "Resistor_SMD:R_0603_1608Metric" V 6430 1450 50  0001 C CNN
 F 3 "~" H 6500 1450 50  0001 C CNN
@@
 U 1 1 5F5986E5
 P 6600 1450
-F 0 "R709" V 6550 1550 50  0000 L CNN
-F 1 "3k3" V 6600 1400 50  0000 L CNN
+F 0 "R709" V 6600 1650 50  0000 L CNN
+F 1 "3.3kR" V 6600 1900 50  0000 L CNN
 F 2 "Resistor_SMD:R_0603_1608Metric" V 6530 1450 50  0001 C CNN
 F 3 "~" H 6600 1450 50  0001 C CNN
@@
 U 1 1 5F5986EB
 P 6700 1450
-F 0 "R710" V 6650 1550 50  0000 L CNN
-F 1 "3k3" V 6700 1400 50  0000 L CNN
+F 0 "R710" V 6700 1650 50  0000 L CNN
+F 1 "3.3kR" V 6700 1900 50  0000 L CNN
 F 2 "Resistor_SMD:R_0603_1608Metric" V 6630 1450 50  0001 C CNN
 F 3 "~" H 6700 1450 50  0001 C CNN
@@
 U 1 1 5F5986F1
 P 6800 1450
-F 0 "R711" V 6750 1550 50  0000 L CNN
-F 1 "3k3" V 6800 1400 50  0000 L CNN
+F 0 "R711" V 6800 1650 50  0000 L CNN
+F 1 "3.3kR" V 6800 1900 50  0000 L CNN
 F 2 "Resistor_SMD:R_0603_1608Metric" V 6730 1450 50  0001 C CNN
 F 3 "~" H 6800 1450 50  0001 C CNN
@@
 U 1 1 5F599DD6
 P 7000 1450
-F 0 "R712" V 6950 1550 50  0000 L CNN
-F 1 "3k3" V 7000 1400 50  0000 L CNN
+F 0 "R712" V 7000 1650 50  0000 L CNN
+F 1 "3.3kR" V 7000 1900 50  0000 L CNN
 F 2 "Resistor_SMD:R_0603_1608Metric" V 6930 1450 50  0001 C CNN
 F 3 "~" H 7000 1450 50  0001 C CNN
@@
 U 1 1 5F599DDC
 P 7100 1450
-F 0 "R713" V 7050 1550 50  0000 L CNN
-F 1 "3k3" V 7100 1400 50  0000 L CNN
+F 0 "R713" V 7100 1650 50  0000 L CNN
+F 1 "3.3kR" V 7100 1900 50  0000 L CNN
 F 2 "Resistor_SMD:R_0603_1608Metric" V 7030 1450 50  0001 C CNN
 F 3 "~" H 7100 1450 50  0001 C CNN
@@
 U 1 1 5F599DE2
 P 7200 1450
-F 0 "R714" V 7150 1550 50  0000 L CNN
-F 1 "3k3" V 7200 1400 50  0000 L CNN
+F 0 "R714" V 7200 1650 50  0000 L CNN
+F 1 "3.3kR" V 7200 1900 50  0000 L CNN
 F 2 "Resistor_SMD:R_0603_1608Metric" V 7130 1450 50  0001 C CNN
 F 3 "~" H 7200 1450 50  0001 C CNN
@@
 U 1 1 5F599DE8
 P 7300 1450
-F 0 "R715" V 7250 1550 50  0000 L CNN
-F 1 "3k3" V 7300 1400 50  0000 L CNN
+F 0 "R715" V 7300 1650 50  0000 L CNN
+F 1 "3.3kR" V 7300 1900 50  0000 L CNN
 F 2 "Resistor_SMD:R_0603_1608Metric" V 7230 1450 50  0001 C CNN
 F 3 "~" H 7300 1450 50  0001 C CNN
@@
 AR Path="/5F24B563/5F6D6DB8" Ref="C704"  Part="1"
 F 0 "C704" H 4992 1446 50  0000 L CNN
-F 1 "0µ1" H 4992 1355 50  0000 L CNN
+F 1 "0.1uF 5VDCbias" H 4992 1355 50  0000 L CNN
 F 2 "Capacitor_SMD:C_0603_1608Metric" H 4900 1400 50  0001 C CNN
 F 3 "~" H 4900 1400 50  0001 C CNN
@@
 AR Path="/5F24B563/5F6D9DA4" Ref="C703"  Part="1"
 F 0 "C703" H 1392 3696 50  0000 L CNN
-F 1 "0µ1" H 1392 3605 50  0000 L CNN
+F 1 "0.1uF 3.3VDCbias" H 1392 3605 50  0000 L CNN
 F 2 "Capacitor_SMD:C_0603_1608Metric" H 1300 3650 50  0001 C CNN
 F 3 "~" H 1300 3650 50  0001 C CNN
@@
 Text Label 3800 2950 2    50   ~ 0
 FAN5V
+$Comp
+L Device:R R701
+U 1 1 5F4BDB11
+P 2200 2000
+F 0 "R701" H 2300 2050 50  0000 L CNN
+F 1 "200kR" H 2300 1950 50  0000 L CNN
+F 2 "Resistor_SMD:R_0603_1608Metric" V 2130 2000 50  0001 C CNN
+F 3 "~" H 2200 2000 50  0001 C CNN
+F 4 "RK73B1JTTD204J" H 2200 2000 50  0001 C CNN "Mfg Part Num"
+F 5 "KOA Speer Electronics" H 2200 2000 50  0001 C CNN "Mfg"
+F 6 "232-00033" H 2200 2000 50  0001 C CNN "CPN"
+	1    2200 2000
+	1    0    0    -1
+$EndComp
 $EndSCHEMATC

Commit message: gemini-bringup: custom fields for rating constraints on passives
Instead of packing tons of detail into a single "Value" field, limit
"Value" to the primary characteristic of the device (i.e. capacitance
for capacitors, resistance for resistors, current for fuses, impedence
at frequency for ferrite beads). For all other rating constraints, use
custom fields of the form <component-refdes-prefix>_<constraint>. For
example, R_P contains the power a resistor must dissipate.  Use
calculated values when possible rather than standard values as the
intent is to capture the constraint, not a specific device choice.
Parts:
- C701: value 1uF 12VDCbias -> 1uF; C_Vbias (none) -> 12V
- C702: value 1uF 5VDCbias -> 1uF; C_Vbias (none) -> 5V
- C703: value 0.1uF 3.3VDCbias -> 0.1uF; C_Vbias (none) -> 3.3V
- C704: value 0.1uF 5VDCbias -> 0.1uF; C_Vbias (none) -> 5V
- R701: value 200kR -> 200k
Other:
- moved on the sheet: C701
Changed lines of the file:
@@
 L Device:C_Small C701
 U 1 1 5F48A9CC
-P 2200 1600
-F 0 "C701" H 2292 1646 50  0000 L CNN
-F 1 "1uF 12VDCbias" H 2292 1555 50  0000 L CNN
-F 2 "Capacitor_SMD:C_0603_1608Metric" H 2200 1600 50  0001 C CNN
-F 3 "~" H 2200 1600 50  0001 C CNN
-F 4 "CL10B105KP8NFNC" H 2200 1600 50  0001 C CNN "Mfg Part Num"
-F 5 "Samsung Electro-Mechanics" H 2200 1600 50  0001 C CNN "Mfg"
-F 6 "212-00015" H 2200 1600 50  0001 C CNN "CPN"
-	1    2200 1600
+P 2450 1600
+F 0 "C701" H 2542 1646 50  0000 L CNN
+F 1 "1uF" H 2542 1555 50  0000 L CNN
+F 2 "Capacitor_SMD:C_0603_1608Metric" H 2450 1600 50  0001 C CNN
+F 3 "~" H 2450 1600 50  0001 C CNN
+F 4 "CL10B105KP8NFNC" H 2450 1600 50  0001 C CNN "Mfg Part Num"
+F 5 "Samsung Electro-Mechanics" H 2450 1600 50  0001 C CNN "Mfg"
+F 6 "212-00015" H 2450 1600 50  0001 C CNN "CPN"
+F 7 "12V" H 2450 1600 50  0001 C CNN "C_Vbias"
+	1    2450 1600
 	1    0    0    -1
 $EndComp
@@
 P 3600 1600
 F 0 "C702" H 3692 1646 50  0000 L CNN
-F 1 "1uF 5VDCbias" H 3692 1555 50  0000 L CNN
+F 1 "1uF" H 3692 1555 50  0000 L CNN
 F 2 "Capacitor_SMD:C_0603_1608Metric" H 3600 1600 50  0001 C CNN
 F 3 "~" H 3600 1600 50  0001 C CNN
@@
 F 5 "Samsung Electro-Mechanics" H 3600 1600 50  0001 C CNN "Mfg"
 F 6 "212-00015" H 3600 1600 50  0001 C CNN "CPN"
+F 7 "5V" H 3600 1600 50  0001 C CNN "C_Vbias"
 	1    3600 1600
 	1    0    0    -1
@@
 Connection ~ 3150 1700
 Wire Wire Line
-	3150 1700 2200 1700
-Wire Wire Line
-	2200 1500 2200 1400
-Wire Wire Line
-	2200 1400 2850 1400
+	3150 1700 2450 1700
+Wire Wire Line
+	2450 1500 2450 1400
+Wire Wire Line
+	2450 1400 2850 1400
 $Comp
 L power:+12V #PWR0706
 U 1 1 5F495AE2
-P 2200 1400
-F 0 "#PWR0706" H 2200 1250 50  0001 C CNN
-F 1 "+12V" H 2215 1573 50  0000 C CNN
-F 2 "" H 2200 1400 50  0001 C CNN
-F 3 "" H 2200 1400 50  0001 C CNN
-	1    2200 1400
-	1    0    0    -1
-$EndComp
-Connection ~ 2200 1400
+P 2450 1400
+F 0 "#PWR0706" H 2450 1250 50  0001 C CNN
+F 1 "+12V" H 2465 1573 50  0000 C CNN
+F 2 "" H 2450 1400 50  0001 C CNN
+F 3 "" H 2450 1400 50  0001 C CNN
+	1    2450 1400
+	1    0    0    -1
+$EndComp
+Connection ~ 2450 1400
 Wire Wire Line
 	3600 1400 3950 1400
@@
 	1    0    0    -1
 $EndComp
+$Comp
+L Device:R R701
+U 1 1 5F4BDB11
+P 2200 2000
+F 0 "R701" H 2270 2046 50  0000 L CNN
+F 1 "200k" V 2200 1900 50  0000 L CNN
+F 2 "Resistor_SMD:R_0603_1608Metric" V 2130 2000 50  0001 C CNN
+F 3 "~" H 2200 2000 50  0001 C CNN
+F 4 "RK73B1JTTD204J" H 2200 2000 50  0001 C CNN "Mfg Part Num"
+F 5 "KOA Speer Electronics" H 2200 2000 50  0001 C CNN "Mfg"
+F 6 "232-00033" H 2200 2000 50  0001 C CNN "CPN"
+	1    2200 2000
+	1    0    0    -1
+$EndComp
 Wire Wire Line
 	1900 2250 1900 2150
@@
 U 1 1 5F4E01D9
 P 2750 2400
-F 0 "R702" H 2450 2450 50  0000 L CNN
-F 1 "3.3kR" H 2450 2350 50  0000 L CNN
+F 0 "R702" H 2820 2446 50  0000 L CNN
+F 1 "3.3kR" V 2750 2300 50  0000 L CNN
 F 2 "Resistor_SMD:R_0603_1608Metric" V 2680 2400 50  0001 C CNN
 F 3 "~" H 2750 2400 50  0001 C CNN
@@
 U 1 1 5F4E073B
 P 3000 2400
-F 0 "R703" H 3100 2450 50  0000 L CNN
-F 1 "3.3kR" H 3100 2350 50  0000 L CNN
+F 0 "R703" H 3070 2446 50  0000 L CNN
+F 1 "3.3kR" V 3000 2300 50  0000 L CNN
 F 2 "Resistor_SMD:R_0603_1608Metric" V 2930 2400 50  0001 C CNN
 F 3 "~" H 3000 2400 50  0001 C CNN
@@
 U 1 1 5F596D71
 P 5950 1450
-F 0 "R704" V 5950 1650 50  0000 L CNN
-F 1 "3.3kR" V 5950 1900 50  0000 L CNN
+F 0 "R704" V 5900 1550 50  0000 L CNN
+F 1 "3.3kR" V 5950 1400 50  0000 L CNN
 F 2 "Resistor_SMD:R_0603_1608Metric" V 5880 1450 50  0001 C CNN
 F 3 "~" H 5950 1450 50  0001 C CNN
@@
 U 1 1 5F597263
 P 6050 1450
-F 0 "R705" V 6050 1650 50  0000 L CNN
-F 1 "3.3kR" V 6050 1900 50  0000 L CNN
+F 0 "R705" V 6000 1550 50  0000 L CNN
+F 1 "3.3kR" V 6050 1400 50  0000 L CNN
 F 2 "Resistor_SMD:R_0603_1608Metric" V 5980 1450 50  0001 C CNN
 F 3 "~" H 6050 1450 50  0001 C CNN
@@
 U 1 1 5F597494
 P 6150 1450
-F 0 "R706" V 6150 1650 50  0000 L CNN
-F 1 "3.3kR" V 6150 1900 50  0000 L CNN
+F 0 "R706" V 6100 1550 50  0000 L CNN
+F 1 "3.3kR" V 6150 1400 50  0000 L CNN
 F 2 "Resistor_SMD:R_0603_1608Metric" V 6080 1450 50  0001 C CNN
 F 3 "~" H 6150 1450 50  0001 C CNN
@@
 U 1 1 5F597612
 P 6250 1450
-F 0 "R707" V 6250 1650 50  0000 L CNN
-F 1 "3.3kR" V 6250 1900 50  0000 L CNN
+F 0 "R707" V 6200 1550 50  0000 L CNN
+F 1 "3.3kR" V 6250 1400 50  0000 L CNN
 F 2 "Resistor_SMD:R_0603_1608Metric" V 6180 1450 50  0001 C CNN
 F 3 "~" H 6250 1450 50  0001 C CNN
@@
 U 1 1 5F5986DF
 P 6500 1450
-F 0 "R708" V 6500 1650 50  0000 L CNN
-F 1 "3.3kR" V 6500 1900 50  0000 L CNN
+F 0 "R708" V 6450 1550 50  0000 L CNN
+F 1 "3.3kR" V 6500 1400 50  0000 L CNN
 F 2 "Resistor_SMD:R_0603_1608Metric" V 6430 1450 50  0001 C CNN
 F 3 "~" H 6500 1450 50  0001 C CNN
@@
 U 1 1 5F5986E5
 P 6600 1450
-F 0 "R709" V 6600 1650 50  0000 L CNN
-F 1 "3.3kR" V 6600 1900 50  0000 L CNN
+F 0 "R709" V 6550 1550 50  0000 L CNN
+F 1 "3.3kR" V 6600 1400 50  0000 L CNN
 F 2 "Resistor_SMD:R_0603_1608Metric" V 6530 1450 50  0001 C CNN
 F 3 "~" H 6600 1450 50  0001 C CNN
@@
 U 1 1 5F5986EB
 P 6700 1450
-F 0 "R710" V 6700 1650 50  0000 L CNN
-F 1 "3.3kR" V 6700 1900 50  0000 L CNN
+F 0 "R710" V 6650 1550 50  0000 L CNN
+F 1 "3.3kR" V 6700 1400 50  0000 L CNN
 F 2 "Resistor_SMD:R_0603_1608Metric" V 6630 1450 50  0001 C CNN
 F 3 "~" H 6700 1450 50  0001 C CNN
@@
 U 1 1 5F5986F1
 P 6800 1450
-F 0 "R711" V 6800 1650 50  0000 L CNN
-F 1 "3.3kR" V 6800 1900 50  0000 L CNN
+F 0 "R711" V 6750 1550 50  0000 L CNN
+F 1 "3.3kR" V 6800 1400 50  0000 L CNN
 F 2 "Resistor_SMD:R_0603_1608Metric" V 6730 1450 50  0001 C CNN
 F 3 "~" H 6800 1450 50  0001 C CNN
@@
 U 1 1 5F599DD6
 P 7000 1450
-F 0 "R712" V 7000 1650 50  0000 L CNN
-F 1 "3.3kR" V 7000 1900 50  0000 L CNN
+F 0 "R712" V 6950 1550 50  0000 L CNN
+F 1 "3.3kR" V 7000 1400 50  0000 L CNN
 F 2 "Resistor_SMD:R_0603_1608Metric" V 6930 1450 50  0001 C CNN
 F 3 "~" H 7000 1450 50  0001 C CNN
@@
 U 1 1 5F599DDC
 P 7100 1450
-F 0 "R713" V 7100 1650 50  0000 L CNN
-F 1 "3.3kR" V 7100 1900 50  0000 L CNN
+F 0 "R713" V 7050 1550 50  0000 L CNN
+F 1 "3.3kR" V 7100 1400 50  0000 L CNN
 F 2 "Resistor_SMD:R_0603_1608Metric" V 7030 1450 50  0001 C CNN
 F 3 "~" H 7100 1450 50  0001 C CNN
@@
 U 1 1 5F599DE2
 P 7200 1450
-F 0 "R714" V 7200 1650 50  0000 L CNN
-F 1 "3.3kR" V 7200 1900 50  0000 L CNN
+F 0 "R714" V 7150 1550 50  0000 L CNN
+F 1 "3.3kR" V 7200 1400 50  0000 L CNN
 F 2 "Resistor_SMD:R_0603_1608Metric" V 7130 1450 50  0001 C CNN
 F 3 "~" H 7200 1450 50  0001 C CNN
@@
 U 1 1 5F599DE8
 P 7300 1450
-F 0 "R715" V 7300 1650 50  0000 L CNN
-F 1 "3.3kR" V 7300 1900 50  0000 L CNN
+F 0 "R715" V 7250 1550 50  0000 L CNN
+F 1 "3.3kR" V 7300 1400 50  0000 L CNN
 F 2 "Resistor_SMD:R_0603_1608Metric" V 7230 1450 50  0001 C CNN
 F 3 "~" H 7300 1450 50  0001 C CNN
@@
 AR Path="/5F24B563/5F6D6DB8" Ref="C704"  Part="1"
 F 0 "C704" H 4992 1446 50  0000 L CNN
-F 1 "0.1uF 5VDCbias" H 4992 1355 50  0000 L CNN
+F 1 "0.1uF" H 4992 1355 50  0000 L CNN
 F 2 "Capacitor_SMD:C_0603_1608Metric" H 4900 1400 50  0001 C CNN
 F 3 "~" H 4900 1400 50  0001 C CNN
@@
 F 5 "Samsung Electro-Mechanics" H 4900 1400 50  0001 C CNN "Mfg"
 F 6 "212-00011" H 4900 1400 50  0001 C CNN "CPN"
+F 7 "5V" H 4900 1400 50  0001 C CNN "C_Vbias"
 	1    4900 1400
 	1    0    0    -1
@@
 AR Path="/5F24B563/5F6D9DA4" Ref="C703"  Part="1"
 F 0 "C703" H 1392 3696 50  0000 L CNN
-F 1 "0.1uF 3.3VDCbias" H 1392 3605 50  0000 L CNN
+F 1 "0.1uF" H 1392 3605 50  0000 L CNN
 F 2 "Capacitor_SMD:C_0603_1608Metric" H 1300 3650 50  0001 C CNN
 F 3 "~" H 1300 3650 50  0001 C CNN
@@
 F 5 "Samsung Electro-Mechanics" H 1300 3650 50  0001 C CNN "Mfg"
 F 6 "212-00011" H 1300 3650 50  0001 C CNN "CPN"
+F 7 "3.3V" H 1300 3650 50  0001 C CNN "C_Vbias"
 	1    1300 3650
 	1    0    0    -1
@@
 Text Label 3800 2950 2    50   ~ 0
 FAN5V
-$Comp
-L Device:R R701
-U 1 1 5F4BDB11
-P 2200 2000
-F 0 "R701" H 2300 2050 50  0000 L CNN
-F 1 "200kR" H 2300 1950 50  0000 L CNN
-F 2 "Resistor_SMD:R_0603_1608Metric" V 2130 2000 50  0001 C CNN
-F 3 "~" H 2200 2000 50  0001 C CNN
-F 4 "RK73B1JTTD204J" H 2200 2000 50  0001 C CNN "Mfg Part Num"
-F 5 "KOA Speer Electronics" H 2200 2000 50  0001 C CNN "Mfg"
-F 6 "232-00033" H 2200 2000 50  0001 C CNN "CPN"
-	1    2200 2000
-	1    0    0    -1
-$EndComp
 $EndSCHEMATC

Commit message: gemini-bringup: resistor power rating constraints
Parts:
- R701: R_P (none) -> 25uW
- R702, R703, R704, R705, R706, R707, R708, R709, R710, R711, R712, R713, R714, R715: R_P (none) -> 1.5mW
Changed lines of the file:
@@
 F 5 "KOA Speer Electronics" H 2200 2000 50  0001 C CNN "Mfg"
 F 6 "232-00033" H 2200 2000 50  0001 C CNN "CPN"
+F 7 "25uW" H 2200 2000 50  0001 C CNN "R_P"
 	1    2200 2000
 	1    0    0    -1
@@
 F 5 "Bourns" H 2750 2400 50  0001 C CNN "Mfg"
 F 6 "232-00018" H 2750 2400 50  0001 C CNN "CPN"
+F 7 "1.5mW" H 2750 2400 50  0001 C CNN "R_P"
 	1    2750 2400
 	1    0    0    -1
@@
 F 5 "Bourns" H 3000 2400 50  0001 C CNN "Mfg"
 F 6 "232-00018" H 3000 2400 50  0001 C CNN "CPN"
+F 7 "1.5mW" H 3000 2400 50  0001 C CNN "R_P"
 	1    3000 2400
 	1    0    0    -1
@@
 F 5 "Bourns" H 5950 1450 50  0001 C CNN "Mfg"
 F 6 "232-00018" H 5950 1450 50  0001 C CNN "CPN"
+F 7 "1.5mW" H 5950 1450 50  0001 C CNN "R_P"
 	1    5950 1450
 	1    0    0    -1
@@
 F 5 "Bourns" H 6050 1450 50  0001 C CNN "Mfg"
 F 6 "232-00018" H 6050 1450 50  0001 C CNN "CPN"
+F 7 "1.5mW" H 6050 1450 50  0001 C CNN "R_P"
 	1    6050 1450
 	1    0    0    -1
@@
 F 5 "Bourns" H 6150 1450 50  0001 C CNN "Mfg"
 F 6 "232-00018" H 6150 1450 50  0001 C CNN "CPN"
+F 7 "1.5mW" H 6150 1450 50  0001 C CNN "R_P"
 	1    6150 1450
 	1    0    0    -1
@@
 F 5 "Bourns" H 6250 1450 50  0001 C CNN "Mfg"
 F 6 "232-00018" H 6250 1450 50  0001 C CNN "CPN"
+F 7 "1.5mW" H 6250 1450 50  0001 C CNN "R_P"
 	1    6250 1450
 	1    0    0    -1
@@
 F 5 "Bourns" H 6500 1450 50  0001 C CNN "Mfg"
 F 6 "232-00018" H 6500 1450 50  0001 C CNN "CPN"
+F 7 "1.5mW" H 6500 1450 50  0001 C CNN "R_P"
 	1    6500 1450
 	1    0    0    -1
@@
 F 5 "Bourns" H 6600 1450 50  0001 C CNN "Mfg"
 F 6 "232-00018" H 6600 1450 50  0001 C CNN "CPN"
+F 7 "1.5mW" H 6600 1450 50  0001 C CNN "R_P"
 	1    6600 1450
 	1    0    0    -1
@@
 F 5 "Bourns" H 6700 1450 50  0001 C CNN "Mfg"
 F 6 "232-00018" H 6700 1450 50  0001 C CNN "CPN"
+F 7 "1.5mW" H 6700 1450 50  0001 C CNN "R_P"
 	1    6700 1450
 	1    0    0    -1
@@
 F 5 "Bourns" H 6800 1450 50  0001 C CNN "Mfg"
 F 6 "232-00018" H 6800 1450 50  0001 C CNN "CPN"
+F 7 "1.5mW" H 6800 1450 50  0001 C CNN "R_P"
 	1    6800 1450
 	1    0    0    -1
@@
 F 5 "Bourns" H 7000 1450 50  0001 C CNN "Mfg"
 F 6 "232-00018" H 7000 1450 50  0001 C CNN "CPN"
+F 7 "1.5mW" H 7000 1450 50  0001 C CNN "R_P"
 	1    7000 1450
 	1    0    0    -1
@@
 F 5 "Bourns" H 7100 1450 50  0001 C CNN "Mfg"
 F 6 "232-00018" H 7100 1450 50  0001 C CNN "CPN"
+F 7 "1.5mW" H 7100 1450 50  0001 C CNN "R_P"
 	1    7100 1450
 	1    0    0    -1
@@
 F 5 "Bourns" H 7200 1450 50  0001 C CNN "Mfg"
 F 6 "232-00018" H 7200 1450 50  0001 C CNN "CPN"
+F 7 "1.5mW" H 7200 1450 50  0001 C CNN "R_P"
 	1    7200 1450
 	1    0    0    -1
@@
 F 5 "Bourns" H 7300 1450 50  0001 C CNN "Mfg"
 F 6 "232-00018" H 7300 1450 50  0001 C CNN "CPN"
+F 7 "1.5mW" H 7300 1450 50  0001 C CNN "R_P"
 	1    7300 1450
 	1    0    0    -1

Commit message: gemini-bringup: Test points on major power rails
Parts:
- added TP701: FAN5V, symbol Connector:TestPoint
Connections:
- net FAN5V: now also TP701.1
Changed lines of the file:
@@
 Connection ~ 2450 1400
 Wire Wire Line
-	3600 1400 3950 1400
+	3600 1400 3800 1400
 Connection ~ 3600 1400
 Text Label 3950 1400 0    50   ~ 0
@@
 Text Label 3800 2950 2    50   ~ 0
 FAN5V
+$Comp
+L Connector:TestPoint TP701
+U 1 1 5FCF47A1
+P 3800 1400
+F 0 "TP701" H 3800 1750 50  0000 C CNN
+F 1 "FAN5V" H 3800 1650 50  0000 C CNN
+F 2 "" H 4000 1400 50  0001 C CNN
+F 3 "~" H 4000 1400 50  0001 C CNN
+	1    3800 1400
+	1    0    0    -1
+$EndComp
+Connection ~ 3800 1400
+Wire Wire Line
+	3800 1400 3950 1400
 $EndSCHEMATC
