File: fans.sch (KiCad schematic (older format))
At the start: 29 parts, among them J701 FAN6, J702 FAN5, J703 FAN4, J704 FAN3, J705 FAN2, J706 FAN1, U701 MAX31790, U702 MCP1703A-5002_SOT89, U703 PCA9306DP1

Commit message: gemini-bringup: reselect all caps respecting C/V derating
Parts:
- C701, C702: footprint Capacitor_SMD:C_0603_1608Metric -> Capacitor_SMD:C_0805_2012Metric; Mfg Samsung Electro-Mechanics -> Kemet; Mfg Part Num CL10B105KP8NFNC -> C0805C105K3RACTU
- C703, C704: Mfg Samsung Electro-Mechanics -> Kemet; Mfg Part Num CL10B104KB8NNWC -> C0603C104M4RACTU
Changed lines of the file:
@@
 F 0 "C701" H 2542 1646 50  0000 L CNN
 F 1 "1uF" H 2542 1555 50  0000 L CNN
-F 2 "Capacitor_SMD:C_0603_1608Metric" H 2450 1600 50  0001 C CNN
+F 2 "Capacitor_SMD:C_0805_2012Metric" H 2450 1600 50  0001 C CNN
 F 3 "~" H 2450 1600 50  0001 C CNN
-F 4 "CL10B105KP8NFNC" H 2450 1600 50  0001 C CNN "Mfg Part Num"
-F 5 "Samsung Electro-Mechanics" H 2450 1600 50  0001 C CNN "Mfg"
+F 4 "C0805C105K3RACTU" H 2450 1600 50  0001 C CNN "Mfg Part Num"
+F 5 "Kemet" H 2450 1600 50  0001 C CNN "Mfg"
 F 6 "212-00015" H 2450 1600 50  0001 C CNN "CPN"
 F 7 "12V" H 2450 1600 50  0001 C CNN "C_Vbias"
@@
 F 0 "C702" H 3692 1646 50  0000 L CNN
 F 1 "1uF" H 3692 1555 50  0000 L CNN
-F 2 "Capacitor_SMD:C_0603_1608Metric" H 3600 1600 50  0001 C CNN
+F 2 "Capacitor_SMD:C_0805_2012Metric" H 3600 1600 50  0001 C CNN
 F 3 "~" H 3600 1600 50  0001 C CNN
-F 4 "CL10B105KP8NFNC" H 3600 1600 50  0001 C CNN "Mfg Part Num"
-F 5 "Samsung Electro-Mechanics" H 3600 1600 50  0001 C CNN "Mfg"
+F 4 "C0805C105K3RACTU" H 3600 1600 50  0001 C CNN "Mfg Part Num"
+F 5 "Kemet" H 3600 1600 50  0001 C CNN "Mfg"
 F 6 "212-00015" H 3600 1600 50  0001 C CNN "CPN"
 F 7 "5V" H 3600 1600 50  0001 C CNN "C_Vbias"
@@
 F 2 "Capacitor_SMD:C_0603_1608Metric" H 4900 1400 50  0001 C CNN
 F 3 "~" H 4900 1400 50  0001 C CNN
-F 4 "CL10B104KB8NNWC" H 4900 1400 50  0001 C CNN "Mfg Part Num"
-F 5 "Samsung Electro-Mechanics" H 4900 1400 50  0001 C CNN "Mfg"
+F 4 "C0603C104M4RACTU" H 4900 1400 50  0001 C CNN "Mfg Part Num"
+F 5 "Kemet" H 4900 1400 50  0001 C CNN "Mfg"
 F 6 "212-00011" H 4900 1400 50  0001 C CNN "CPN"
 F 7 "5V" H 4900 1400 50  0001 C CNN "C_Vbias"
@@
 F 2 "Capacitor_SMD:C_0603_1608Metric" H 1300 3650 50  0001 C CNN
 F 3 "~" H 1300 3650 50  0001 C CNN
-F 4 "CL10B104KB8NNWC" H 1300 3650 50  0001 C CNN "Mfg Part Num"
-F 5 "Samsung Electro-Mechanics" H 1300 3650 50  0001 C CNN "Mfg"
+F 4 "C0603C104M4RACTU" H 1300 3650 50  0001 C CNN "Mfg Part Num"
+F 5 "Kemet" H 1300 3650 50  0001 C CNN "Mfg"
 F 6 "212-00011" H 1300 3650 50  0001 C CNN "CPN"
 F 7 "3.3V" H 1300 3650 50  0001 C CNN "C_Vbias"

Commit message: gemini-bringup: update resistor MPNs to match Bourns part numbers associated with CPN
Parts:
- R701: Mfg KOA Speer Electronics -> Bourns; Mfg Part Num RK73B1JTTD204J -> CR0603-JW-204ELF
Changed lines of the file:
@@
 F 2 "Resistor_SMD:R_0603_1608Metric" V 2130 2000 50  0001 C CNN
 F 3 "~" H 2200 2000 50  0001 C CNN
-F 4 "RK73B1JTTD204J" H 2200 2000 50  0001 C CNN "Mfg Part Num"
-F 5 "KOA Speer Electronics" H 2200 2000 50  0001 C CNN "Mfg"
+F 4 "CR0603-JW-204ELF" H 2200 2000 50  0001 C CNN "Mfg Part Num"
+F 5 "Bourns" H 2200 2000 50  0001 C CNN "Mfg"
 F 6 "232-00033" H 2200 2000 50  0001 C CNN "CPN"
 F 7 "25uW" H 2200 2000 50  0001 C CNN "R_P"

Commit message: gemini-bringup: assign footprints for test points
Parts:
- TP701: footprint (none) -> TestPoint:TestPoint_Pad_D1.0mm
Changed lines of the file:
@@
 F 0 "TP701" H 3800 1750 50  0000 C CNN
 F 1 "FAN5V" H 3800 1650 50  0000 C CNN
-F 2 "" H 4000 1400 50  0001 C CNN
+F 2 "TestPoint:TestPoint_Pad_D1.0mm" H 4000 1400 50  0001 C CNN
 F 3 "~" H 4000 1400 50  0001 C CNN
 	1    3800 1400

Commit message: fans: update for U701 footprint name change
Parts:
- U701: footprint tqfn28:QFN-28_EP_4x4_Pitch0.4mm -> tqfn28:TQFN-28_1EP_4x4mm_P0.4mm_EP2.7x2.7mm
Changed lines of the file:
@@
 F 0 "U701" H 4500 3450 50  0000 L CNN
 F 1 "MAX31790" H 4400 3350 50  0000 L CNN
-F 2 "tqfn28:QFN-28_EP_4x4_Pitch0.4mm" H 4550 3350 50  0001 C CNN
+F 2 "tqfn28:TQFN-28_1EP_4x4mm_P0.4mm_EP2.7x2.7mm" H 4550 3350 50  0001 C CNN
 F 3 "" H 4550 3350 50  0001 C CNN
 F 4 "Maxim" H 4550 3350 50  0001 C CNN "Mfg"
