File: gemini-bringup.sch (KiCad schematic (older format))
At the start: 5 parts

Commit message: PCB: more layout, FPGA expansion, mounting holes
Also fixed a couple of incorrect footprint assignments.
Parts:
- added H101, H102, H103, H104, H105, H106, H107, H108, H109, H110: M3, MountingHole:MountingHole_3.2mm_M3, symbol Mechanical:MountingHole
Changed lines of the file:
@@
 	2550 7350 2350 7350
 Connection ~ 2550 6500
+$Comp
+L Mechanical:MountingHole H101
+U 1 1 5F8B5846
+P 1300 950
+F 0 "H101" H 1400 996 50  0000 L CNN
+F 1 "M3" H 1400 905 50  0000 L CNN
+F 2 "MountingHole:MountingHole_3.2mm_M3" H 1300 950 50  0001 C CNN
+F 3 "~" H 1300 950 50  0001 C CNN
+	1    1300 950
+	1    0    0    -1
+$EndComp
+$Comp
+L Mechanical:MountingHole H104
+U 1 1 5F8B599D
+P 1650 950
+F 0 "H104" H 1750 996 50  0000 L CNN
+F 1 "M3" H 1750 905 50  0000 L CNN
+F 2 "MountingHole:MountingHole_3.2mm_M3" H 1650 950 50  0001 C CNN
+F 3 "~" H 1650 950 50  0001 C CNN
+	1    1650 950
+	1    0    0    -1
+$EndComp
+$Comp
+L Mechanical:MountingHole H107
+U 1 1 5F8B5C3B
+P 2000 950
+F 0 "H107" H 2100 996 50  0000 L CNN
+F 1 "M3" H 2100 905 50  0000 L CNN
+F 2 "MountingHole:MountingHole_3.2mm_M3" H 2000 950 50  0001 C CNN
+F 3 "~" H 2000 950 50  0001 C CNN
+	1    2000 950
+	1    0    0    -1
+$EndComp
+$Comp
+L Mechanical:MountingHole H109
+U 1 1 5F8B5ECC
+P 2350 950
+F 0 "H109" H 2450 996 50  0000 L CNN
+F 1 "M3" H 2450 905 50  0000 L CNN
+F 2 "MountingHole:MountingHole_3.2mm_M3" H 2350 950 50  0001 C CNN
+F 3 "~" H 2350 950 50  0001 C CNN
+	1    2350 950
+	1    0    0    -1
+$EndComp
+$Comp
+L Mechanical:MountingHole H102
+U 1 1 5F8B6164
+P 1300 1200
+F 0 "H102" H 1400 1246 50  0000 L CNN
+F 1 "M3" H 1400 1155 50  0000 L CNN
+F 2 "MountingHole:MountingHole_3.2mm_M3" H 1300 1200 50  0001 C CNN
+F 3 "~" H 1300 1200 50  0001 C CNN
+	1    1300 1200
+	1    0    0    -1
+$EndComp
+$Comp
+L Mechanical:MountingHole H105
+U 1 1 5F8B6547
+P 1650 1200
+F 0 "H105" H 1750 1246 50  0000 L CNN
+F 1 "M3" H 1750 1155 50  0000 L CNN
+F 2 "MountingHole:MountingHole_3.2mm_M3" H 1650 1200 50  0001 C CNN
+F 3 "~" H 1650 1200 50  0001 C CNN
+	1    1650 1200
+	1    0    0    -1
+$EndComp
+$Comp
+L Mechanical:MountingHole H108
+U 1 1 5F8B6759
+P 2000 1200
+F 0 "H108" H 2100 1246 50  0000 L CNN
+F 1 "M3" H 2100 1155 50  0000 L CNN
+F 2 "MountingHole:MountingHole_3.2mm_M3" H 2000 1200 50  0001 C CNN
+F 3 "~" H 2000 1200 50  0001 C CNN
+	1    2000 1200
+	1    0    0    -1
+$EndComp
+$Comp
+L Mechanical:MountingHole H110
+U 1 1 5F8B691D
+P 2350 1200
+F 0 "H110" H 2450 1246 50  0000 L CNN
+F 1 "M3" H 2450 1155 50  0000 L CNN
+F 2 "MountingHole:MountingHole_3.2mm_M3" H 2350 1200 50  0001 C CNN
+F 3 "~" H 2350 1200 50  0001 C CNN
+	1    2350 1200
+	1    0    0    -1
+$EndComp
+$Comp
+L Mechanical:MountingHole H103
+U 1 1 5F8B6B59
+P 1300 1450
+F 0 "H103" H 1400 1496 50  0000 L CNN
+F 1 "M3" H 1400 1405 50  0000 L CNN
+F 2 "MountingHole:MountingHole_3.2mm_M3" H 1300 1450 50  0001 C CNN
+F 3 "~" H 1300 1450 50  0001 C CNN
+	1    1300 1450
+	1    0    0    -1
+$EndComp
+$Comp
+L Mechanical:MountingHole H106
+U 1 1 5F8B6E32
+P 1650 1450
+F 0 "H106" H 1750 1496 50  0000 L CNN
+F 1 "M3" H 1750 1405 50  0000 L CNN
+F 2 "MountingHole:MountingHole_3.2mm_M3" H 1650 1450 50  0001 C CNN
+F 3 "~" H 1650 1450 50  0001 C CNN
+	1    1650 1450
+	1    0    0    -1
+$EndComp
 $EndSCHEMATC

Commit message: MB: annotate everything with mfg/MPN
Parts:
- R101, R102, R103, R104, R105: Mfg Part Num (none) -> generic
Changed lines of the file:
@@
 F 2 "Resistor_SMD:R_0603_1608Metric" V 9130 1900 50  0001 C CNN
 F 3 "~" H 9200 1900 50  0001 C CNN
+F 4 "generic" H 9200 1900 50  0001 C CNN "Mfg Part Num"
 	1    9200 1900
 	1    0    0    -1
@@
 F 2 "Resistor_SMD:R_0603_1608Metric" V 9280 1900 50  0001 C CNN
 F 3 "~" H 9350 1900 50  0001 C CNN
+F 4 "generic" H 9350 1900 50  0001 C CNN "Mfg Part Num"
 	1    9350 1900
 	1    0    0    -1
@@
 F 2 "Resistor_SMD:R_0603_1608Metric" V 9430 1900 50  0001 C CNN
 F 3 "~" H 9500 1900 50  0001 C CNN
+F 4 "generic" H 9500 1900 50  0001 C CNN "Mfg Part Num"
 	1    9500 1900
 	1    0    0    -1
@@
 F 2 "Resistor_SMD:R_0603_1608Metric" V 4180 3150 50  0001 C CNN
 F 3 "~" H 4250 3150 50  0001 C CNN
+F 4 "generic" H 4250 3150 50  0001 C CNN "Mfg Part Num"
 	1    4250 3150
 	1    0    0    -1
@@
 F 2 "Resistor_SMD:R_0603_1608Metric" V 4330 3150 50  0001 C CNN
 F 3 "~" H 4400 3150 50  0001 C CNN
+F 4 "generic" H 4400 3150 50  0001 C CNN "Mfg Part Num"
 	1    4400 3150
 	1    0    0    -1

Commit message: MB: assign single resistors
Parts:
- R101, R102, R103, R104, R105: value 3k -> 3k3; Mfg (none) -> Bourns; Mfg Part Num generic -> CR0603-JW-332ELF
Changed lines of the file:
@@
 P 9200 1900
 F 0 "R101" V 9150 2000 50  0000 L CNN
-F 1 "3k" V 9200 1850 50  0000 L CNN
+F 1 "3k3" V 9200 1850 50  0000 L CNN
 F 2 "Resistor_SMD:R_0603_1608Metric" V 9130 1900 50  0001 C CNN
 F 3 "~" H 9200 1900 50  0001 C CNN
-F 4 "generic" H 9200 1900 50  0001 C CNN "Mfg Part Num"
+F 4 "CR0603-JW-332ELF" H 9200 1900 50  0001 C CNN "Mfg Part Num"
+F 5 "Bourns" H 9200 1900 50  0001 C CNN "Mfg"
 	1    9200 1900
 	1    0    0    -1
@@
 P 9350 1900
 F 0 "R102" V 9300 2000 50  0000 L CNN
-F 1 "3k" V 9350 1850 50  0000 L CNN
+F 1 "3k3" V 9350 1850 50  0000 L CNN
 F 2 "Resistor_SMD:R_0603_1608Metric" V 9280 1900 50  0001 C CNN
 F 3 "~" H 9350 1900 50  0001 C CNN
-F 4 "generic" H 9350 1900 50  0001 C CNN "Mfg Part Num"
+F 4 "CR0603-JW-332ELF" H 9350 1900 50  0001 C CNN "Mfg Part Num"
+F 5 "Bourns" H 9350 1900 50  0001 C CNN "Mfg"
 	1    9350 1900
 	1    0    0    -1
@@
 P 9500 1900
 F 0 "R103" V 9450 2000 50  0000 L CNN
-F 1 "3k" V 9500 1850 50  0000 L CNN
+F 1 "3k3" V 9500 1850 50  0000 L CNN
 F 2 "Resistor_SMD:R_0603_1608Metric" V 9430 1900 50  0001 C CNN
 F 3 "~" H 9500 1900 50  0001 C CNN
-F 4 "generic" H 9500 1900 50  0001 C CNN "Mfg Part Num"
+F 4 "CR0603-JW-332ELF" H 9500 1900 50  0001 C CNN "Mfg Part Num"
+F 5 "Bourns" H 9500 1900 50  0001 C CNN "Mfg"
 	1    9500 1900
 	1    0    0    -1
@@
 P 4250 3150
 F 0 "R104" V 4200 3250 50  0000 L CNN
-F 1 "3k" V 4250 3100 50  0000 L CNN
+F 1 "3k3" V 4250 3100 50  0000 L CNN
 F 2 "Resistor_SMD:R_0603_1608Metric" V 4180 3150 50  0001 C CNN
 F 3 "~" H 4250 3150 50  0001 C CNN
-F 4 "generic" H 4250 3150 50  0001 C CNN "Mfg Part Num"
+F 4 "CR0603-JW-332ELF" H 4250 3150 50  0001 C CNN "Mfg Part Num"
+F 5 "Bourns" H 4250 3150 50  0001 C CNN "Mfg"
 	1    4250 3150
 	1    0    0    -1
@@
 P 4400 3150
 F 0 "R105" V 4350 3250 50  0000 L CNN
-F 1 "3k" V 4400 3100 50  0000 L CNN
+F 1 "3k3" V 4400 3100 50  0000 L CNN
 F 2 "Resistor_SMD:R_0603_1608Metric" V 4330 3150 50  0001 C CNN
 F 3 "~" H 4400 3150 50  0001 C CNN
-F 4 "generic" H 4400 3150 50  0001 C CNN "Mfg Part Num"
+F 4 "CR0603-JW-332ELF" H 4400 3150 50  0001 C CNN "Mfg Part Num"
+F 5 "Bourns" H 4400 3150 50  0001 C CNN "Mfg"
 	1    4400 3150
 	1    0    0    -1

Commit message: MB: re-lay-out RoT for revised connector and mechanicals
Parts:
- removed H106, H107: M3, MountingHole:MountingHole_3.2mm_M3, symbol Mechanical:MountingHole
Changed lines of the file:
@@
-$EndComp
-$Comp
-L Mechanical:MountingHole H107
-U 1 1 5F8B5C3B
-P 2000 950
-F 0 "H107" H 2100 996 50  0000 L CNN
-F 1 "M3" H 2100 905 50  0000 L CNN
-F 2 "MountingHole:MountingHole_3.2mm_M3" H 2000 950 50  0001 C CNN
-F 3 "~" H 2000 950 50  0001 C CNN
-	1    2000 950
-	1    0    0    -1
 $EndComp
 $Comp
@@
 	1    0    0    -1
 $EndComp
-$Comp
-L Mechanical:MountingHole H106
-U 1 1 5F8B6E32
-P 1650 1450
-F 0 "H106" H 1750 1496 50  0000 L CNN
-F 1 "M3" H 1750 1405 50  0000 L CNN
-F 2 "MountingHole:MountingHole_3.2mm_M3" H 1650 1450 50  0001 C CNN
-F 3 "~" H 1650 1450 50  0001 C CNN
-	1    1650 1450
-	1    0    0    -1
-$EndComp

Commit message: MB: power area fixes, start snarking
Parts:
- added H106: GRAPHIC PLACEHOLDER, grumpy:grumpy, symbol Mechanical:MountingHole
- added H107: M3, MountingHole:MountingHole_3.2mm_M3, symbol Mechanical:MountingHole
Changed lines of the file:
@@
+	1    0    0    -1
+$EndComp
+$Comp
+L Mechanical:MountingHole H106
+U 1 1 5F7CAC07
+P 3200 900
+F 0 "H106" H 3300 946 50  0000 L CNN
+F 1 "GRAPHIC PLACEHOLDER" H 3300 855 50  0000 L CNN
+F 2 "grumpy:grumpy" H 3200 900 50  0001 C CNN
+F 3 "~" H 3200 900 50  0001 C CNN
+	1    3200 900
+	1    0    0    -1
+$EndComp
+$Comp
+L Mechanical:MountingHole H107
+U 1 1 5F7F0EA3
+P 2000 950
+F 0 "H107" H 2100 996 50  0000 L CNN
+F 1 "M3" H 2100 905 50  0000 L CNN
+F 2 "MountingHole:MountingHole_3.2mm_M3" H 2000 950 50  0001 C CNN
+F 3 "~" H 2000 950 50  0001 C CNN
+	1    2000 950
 	1    0    0    -1
 $EndComp

Commit message: MB: logos etc
Parts:
- added H111: GRAPHIC PLACEHOLDER, grumpy:newt_of_trust, symbol Mechanical:MountingHole
Changed lines of the file:
@@
+	1    0    0    -1
+$EndComp
+$Comp
+L Mechanical:MountingHole H111
+U 1 1 5F84B4F9
+P 3200 1100
+F 0 "H111" H 3300 1146 50  0000 L CNN
+F 1 "GRAPHIC PLACEHOLDER" H 3300 1055 50  0000 L CNN
+F 2 "grumpy:newt_of_trust" H 3200 1100 50  0001 C CNN
+F 3 "~" H 3200 1100 50  0001 C CNN
+	1    3200 1100
 	1    0    0    -1
 $EndComp

Commit message: MB: whoops, update sch
Parts:
- added H112: GRAPHIC PLACEHOLDER, grumpy:logo-4mm-mask, symbol Mechanical:MountingHole
Changed lines of the file:
@@
+	1    0    0    -1
+$EndComp
+$Comp
+L Mechanical:MountingHole H112
+U 1 1 5F768622
+P 3200 1300
+F 0 "H112" H 3300 1346 50  0000 L CNN
+F 1 "GRAPHIC PLACEHOLDER" H 3300 1255 50  0000 L CNN
+F 2 "grumpy:logo-4mm-mask" H 3200 1300 50  0001 C CNN
+F 3 "~" H 3200 1300 50  0001 C CNN
+	1    3200 1300
 	1    0    0    -1
 $EndComp

Commit message: gemini-bringup: Add CPNs for all components
Parts:
- R101, R102, R103, R104, R105: CPN (none) -> 232-00018
Changed lines of the file:
@@
 F 4 "CR0603-JW-332ELF" H 9200 1900 50  0001 C CNN "Mfg Part Num"
 F 5 "Bourns" H 9200 1900 50  0001 C CNN "Mfg"
+F 6 "232-00018" H 9200 1900 50  0001 C CNN "CPN"
 	1    9200 1900
 	1    0    0    -1
@@
 F 4 "CR0603-JW-332ELF" H 9350 1900 50  0001 C CNN "Mfg Part Num"
 F 5 "Bourns" H 9350 1900 50  0001 C CNN "Mfg"
+F 6 "232-00018" H 9350 1900 50  0001 C CNN "CPN"
 	1    9350 1900
 	1    0    0    -1
@@
 F 4 "CR0603-JW-332ELF" H 9500 1900 50  0001 C CNN "Mfg Part Num"
 F 5 "Bourns" H 9500 1900 50  0001 C CNN "Mfg"
+F 6 "232-00018" H 9500 1900 50  0001 C CNN "CPN"
 	1    9500 1900
 	1    0    0    -1
@@
 F 4 "CR0603-JW-332ELF" H 4250 3150 50  0001 C CNN "Mfg Part Num"
 F 5 "Bourns" H 4250 3150 50  0001 C CNN "Mfg"
+F 6 "232-00018" H 4250 3150 50  0001 C CNN "CPN"
 	1    4250 3150
 	1    0    0    -1
@@
 F 4 "CR0603-JW-332ELF" H 4400 3150 50  0001 C CNN "Mfg Part Num"
 F 5 "Bourns" H 4400 3150 50  0001 C CNN "Mfg"
+F 6 "232-00018" H 4400 3150 50  0001 C CNN "CPN"
 	1    4400 3150
 	1    0    0    -1
