File: gemini-bringup.sch (KiCad schematic (older format))
At the start: 17 parts

Commit message: gemini-bringup: custom fields for rating constraints on passives
Instead of packing tons of detail into a single "Value" field, limit
"Value" to the primary characteristic of the device (i.e. capacitance
for capacitors, resistance for resistors, current for fuses, impedence
at frequency for ferrite beads). For all other rating constraints, use
custom fields of the form <component-refdes-prefix>_<constraint>. For
example, R_P contains the power a resistor must dissipate.  Use
calculated values when possible rather than standard values as the
intent is to capture the constraint, not a specific device choice.
Parts:
- R101, R102, R103, R104, R105: value 3k3 -> 3.3kR
Changed lines of the file:
@@
 P 9200 1900
 F 0 "R101" V 9150 2000 50  0000 L CNN
-F 1 "3k3" V 9200 1850 50  0000 L CNN
+F 1 "3.3kR" V 9200 1850 50  0000 L CNN
 F 2 "Resistor_SMD:R_0603_1608Metric" V 9130 1900 50  0001 C CNN
 F 3 "~" H 9200 1900 50  0001 C CNN
@@
 P 9350 1900
 F 0 "R102" V 9300 2000 50  0000 L CNN
-F 1 "3k3" V 9350 1850 50  0000 L CNN
+F 1 "3.3kR" V 9350 1850 50  0000 L CNN
 F 2 "Resistor_SMD:R_0603_1608Metric" V 9280 1900 50  0001 C CNN
 F 3 "~" H 9350 1900 50  0001 C CNN
@@
 P 9500 1900
 F 0 "R103" V 9450 2000 50  0000 L CNN
-F 1 "3k3" V 9500 1850 50  0000 L CNN
+F 1 "3.3kR" V 9500 1850 50  0000 L CNN
 F 2 "Resistor_SMD:R_0603_1608Metric" V 9430 1900 50  0001 C CNN
 F 3 "~" H 9500 1900 50  0001 C CNN
@@
 P 4250 3150
 F 0 "R104" V 4200 3250 50  0000 L CNN
-F 1 "3k3" V 4250 3100 50  0000 L CNN
+F 1 "3.3kR" V 4250 3100 50  0000 L CNN
 F 2 "Resistor_SMD:R_0603_1608Metric" V 4180 3150 50  0001 C CNN
 F 3 "~" H 4250 3150 50  0001 C CNN
@@
 P 4400 3150
 F 0 "R105" V 4350 3250 50  0000 L CNN
-F 1 "3k3" V 4400 3100 50  0000 L CNN
+F 1 "3.3kR" V 4400 3100 50  0000 L CNN
 F 2 "Resistor_SMD:R_0603_1608Metric" V 4330 3150 50  0001 C CNN
 F 3 "~" H 4400 3150 50  0001 C CNN

Commit message: gemini-bringup: resistor power rating constraints
Parts:
- R101, R102, R103, R104, R105: R_P (none) -> 1mW
Changed lines of the file:
@@
 F 5 "Bourns" H 9200 1900 50  0001 C CNN "Mfg"
 F 6 "232-00018" H 9200 1900 50  0001 C CNN "CPN"
+F 7 "1mW" H 9200 1900 50  0001 C CNN "R_P"
 	1    9200 1900
 	1    0    0    -1
@@
 F 5 "Bourns" H 9350 1900 50  0001 C CNN "Mfg"
 F 6 "232-00018" H 9350 1900 50  0001 C CNN "CPN"
+F 7 "1mW" H 9350 1900 50  0001 C CNN "R_P"
 	1    9350 1900
 	1    0    0    -1
@@
 F 5 "Bourns" H 9500 1900 50  0001 C CNN "Mfg"
 F 6 "232-00018" H 9500 1900 50  0001 C CNN "CPN"
+F 7 "1mW" H 9500 1900 50  0001 C CNN "R_P"
 	1    9500 1900
 	1    0    0    -1
@@
 F 5 "Bourns" H 4250 3150 50  0001 C CNN "Mfg"
 F 6 "232-00018" H 4250 3150 50  0001 C CNN "CPN"
+F 7 "1mW" H 4250 3150 50  0001 C CNN "R_P"
 	1    4250 3150
 	1    0    0    -1
@@
 F 5 "Bourns" H 4400 3150 50  0001 C CNN "Mfg"
 F 6 "232-00018" H 4400 3150 50  0001 C CNN "CPN"
+F 7 "1mW" H 4400 3150 50  0001 C CNN "R_P"
 	1    4400 3150
 	1    0    0    -1

Commit message: gemini-bringup: Test points on major power rails
Parts:
- added TP101: +12V, symbol Connector:TestPoint
- added TP103: +3.3V, symbol Connector:TestPoint
- added TP104: GND, symbol Connector:TestPoint
Connections:
- net +3V3: now also TP103.1
- new net +12V: TP101.1
- new net GND: TP104.1
Changed lines of the file:
@@
 	1    0    0    -1
 $EndComp
+$Comp
+L Connector:TestPoint TP101
+U 1 1 5FC8EAFF
+P 5850 950
+F 0 "TP101" V 5800 1150 50  0000 L CNN
+F 1 "+12V" V 5850 1150 50  0000 L CNN
+F 2 "" H 6050 950 50  0001 C CNN
+F 3 "~" H 6050 950 50  0001 C CNN
+	1    5850 950
+	0    1    1    0
+$EndComp
+Text Label 5850 950  2    50   ~ 0
++12V
+$Comp
+L Connector:TestPoint TP103
+U 1 1 5FC8F323
+P 5850 1100
+F 0 "TP103" V 5800 1300 50  0000 L CNN
+F 1 "+3.3V" V 5850 1300 50  0000 L CNN
+F 2 "" H 6050 1100 50  0001 C CNN
+F 3 "~" H 6050 1100 50  0001 C CNN
+	1    5850 1100
+	0    1    1    0
+$EndComp
+Text Label 5850 1100 2    50   ~ 0
++3V3
+$Comp
+L Connector:TestPoint TP104
+U 1 1 5FC95488
+P 5850 1250
+F 0 "TP104" V 5800 1450 50  0000 L CNN
+F 1 "GND" V 5850 1450 50  0000 L CNN
+F 2 "" H 6050 1250 50  0001 C CNN
+F 3 "~" H 6050 1250 50  0001 C CNN
+	1    5850 1250
+	0    1    1    0
+$EndComp
+Text Label 5850 1250 2    50   ~ 0
+GND
 $EndSCHEMATC

Commit message: gemini-bringup: assign footprints for test points
Parts:
- TP101, TP103: footprint (none) -> TestPoint:TestPoint_Pad_D1.0mm
- TP104: footprint (none) -> TestPoint:TestPoint_Pad_1.0x1.0mm
Changed lines of the file:
@@
 F 0 "TP101" V 5800 1150 50  0000 L CNN
 F 1 "+12V" V 5850 1150 50  0000 L CNN
-F 2 "" H 6050 950 50  0001 C CNN
+F 2 "TestPoint:TestPoint_Pad_D1.0mm" H 6050 950 50  0001 C CNN
 F 3 "~" H 6050 950 50  0001 C CNN
 	1    5850 950
@@
 F 0 "TP103" V 5800 1300 50  0000 L CNN
 F 1 "+3.3V" V 5850 1300 50  0000 L CNN
-F 2 "" H 6050 1100 50  0001 C CNN
+F 2 "TestPoint:TestPoint_Pad_D1.0mm" H 6050 1100 50  0001 C CNN
 F 3 "~" H 6050 1100 50  0001 C CNN
 	1    5850 1100
@@
 F 0 "TP104" V 5800 1450 50  0000 L CNN
 F 1 "GND" V 5850 1450 50  0000 L CNN
-F 2 "" H 6050 1250 50  0001 C CNN
+F 2 "TestPoint:TestPoint_Pad_1.0x1.0mm" H 6050 1250 50  0001 C CNN
 F 3 "~" H 6050 1250 50  0001 C CNN
 	1    5850 1250

Commit message: gemini-bringup: add Oxide board identifier
Parts:
- H112: value GRAPHIC PLACEHOLDER -> 913-00001; footprint grumpy:logo-4mm-mask -> grumpy:Oxide_Board_Identifier_30.5x9mm
Changed lines of the file:
@@
 U 1 1 5F768622
 P 3200 1300
-F 0 "H112" H 3300 1346 50  0000 L CNN
-F 1 "GRAPHIC PLACEHOLDER" H 3300 1255 50  0000 L CNN
-F 2 "grumpy:logo-4mm-mask" H 3200 1300 50  0001 C CNN
+F 0 "H112" H 3200 1150 50  0000 C CNN
+F 1 "913-00001" H 3200 1050 50  0000 C CNN
+F 2 "grumpy:Oxide_Board_Identifier_30.5x9mm" H 3200 950 50  0000 C CNN
 F 3 "~" H 3200 1300 50  0001 C CNN
 	1    3200 1300

Commit message: gemini-bringup: add bypass caps near I2C2_F_x reference plane changes
Parts:
- added C101, C102: 0.1uF, Capacitor_SMD:C_0603_1608Metric, symbol Device:C_Small
Connections:
- net +3V3: now also C101.1, C102.1
- net GND: now also C101.2, C102.2
Changed lines of the file:
@@
 Text Label 5850 1250 2    50   ~ 0
 GND
+$Comp
+L Device:C_Small C101
+U 1 1 5FD0A6EF
+P 8400 1100
+F 0 "C101" H 8500 1150 50  0000 L CNN
+F 1 "0.1uF" H 8500 1100 50  0000 L CNN
+F 2 "Capacitor_SMD:C_0603_1608Metric" H 8400 1100 50  0001 C CNN
+F 3 "~" H 8400 1100 50  0001 C CNN
+F 4 "212-00011" H 8400 1100 50  0001 C CNN "CPN"
+F 5 "3.3V" H 8400 1100 50  0001 C CNN "C_Vbias"
+F 6 "Kemet" H 8400 1100 50  0001 C CNN "Mfg"
+F 7 "C0603C104M4RACTU" H 8400 1100 50  0001 C CNN "Mfg Part Num"
+	1    8400 1100
+	1    0    0    -1
+$EndComp
+$Comp
+L power:GND #PWR0125
+U 1 1 5FD0AE90
+P 8600 1250
+F 0 "#PWR0125" H 8600 1000 50  0001 C CNN
+F 1 "GND" H 8650 1050 50  0000 C CNN
+F 2 "" H 8600 1250 50  0001 C CNN
+F 3 "" H 8600 1250 50  0001 C CNN
+	1    8600 1250
+	1    0    0    -1
+$EndComp
+$Comp
+L power:+3V3 #PWR0124
+U 1 1 5FD0B0E2
+P 8600 950
+F 0 "#PWR0124" H 8600 800 50  0001 C CNN
+F 1 "+3V3" H 8615 1123 50  0000 C CNN
+F 2 "" H 8600 950 50  0001 C CNN
+F 3 "" H 8600 950 50  0001 C CNN
+	1    8600 950
+	1    0    0    -1
+$EndComp
+$Comp
+L Device:C_Small C102
+U 1 1 5FD0FA33
+P 8800 1100
+F 0 "C102" H 8900 1150 50  0000 L CNN
+F 1 "0.1uF" H 8900 1100 50  0000 L CNN
+F 2 "Capacitor_SMD:C_0603_1608Metric" H 8800 1100 50  0001 C CNN
+F 3 "~" H 8800 1100 50  0001 C CNN
+F 4 "212-00011" H 8800 1100 50  0001 C CNN "CPN"
+F 5 "3.3V" H 8800 1100 50  0001 C CNN "C_Vbias"
+F 6 "Kemet" H 8800 1100 50  0001 C CNN "Mfg"
+F 7 "C0603C104M4RACTU" H 8800 1100 50  0001 C CNN "Mfg Part Num"
+	1    8800 1100
+	1    0    0    -1
+$EndComp
+Wire Wire Line
+	8400 1000 8600 1000
+Wire Wire Line
+	8600 950  8600 1000
+Connection ~ 8600 1000
+Wire Wire Line
+	8600 1000 8800 1000
+Wire Wire Line
+	8400 1200 8600 1200
+Wire Wire Line
+	8600 1200 8600 1250
+Wire Wire Line
+	8600 1200 8800 1200
+Connection ~ 8600 1200
 $EndSCHEMATC

Commit message: gemini-bringup: add bypass caps near SPI6_x reference plane changes
Parts:
- added C?: 0.1uF, Capacitor_SMD:C_0603_1608Metric, symbol Device:C_Small
Connections:
- net +3V3: now also C?.1
- net GND: now also C?.2
Changed lines of the file:
@@
 	8600 1200 8800 1200
 Connection ~ 8600 1200
+$Comp
+L Device:C_Small C?
+U 1 1 5FD39084
+P 9200 1100
+F 0 "C?" H 9300 1150 50  0000 L CNN
+F 1 "0.1uF" H 9300 1100 50  0000 L CNN
+F 2 "Capacitor_SMD:C_0603_1608Metric" H 9200 1100 50  0001 C CNN
+F 3 "~" H 9200 1100 50  0001 C CNN
+F 4 "212-00011" H 9200 1100 50  0001 C CNN "CPN"
+F 5 "3.3V" H 9200 1100 50  0001 C CNN "C_Vbias"
+F 6 "Kemet" H 9200 1100 50  0001 C CNN "Mfg"
+F 7 "C0603C104M4RACTU" H 9200 1100 50  0001 C CNN "Mfg Part Num"
+	1    9200 1100
+	1    0    0    -1
+$EndComp
+Wire Wire Line
+	8800 1000 9200 1000
+Connection ~ 8800 1000
+Wire Wire Line
+	8800 1200 9200 1200
+Connection ~ 8800 1200
 $EndSCHEMATC

Commit message: gemini-bringup: add bypass caps near DA0-DA3 reference plane changes
Parts:
- added C104: 0.1uF, Capacitor_SMD:C_0603_1608Metric, symbol Device:C_Small
- gave numbers to parts that had none: 1
Connections:
- net +3V3: now also C104.1
- net GND: now also C104.2
Changed lines of the file:
@@
 Connection ~ 8600 1200
 $Comp
-L Device:C_Small C?
+L Device:C_Small C103
 U 1 1 5FD39084
 P 9200 1100
-F 0 "C?" H 9300 1150 50  0000 L CNN
+F 0 "C103" H 9300 1150 50  0000 L CNN
 F 1 "0.1uF" H 9300 1100 50  0000 L CNN
 F 2 "Capacitor_SMD:C_0603_1608Metric" H 9200 1100 50  0001 C CNN
@@
 	8800 1200 9200 1200
 Connection ~ 8800 1200
+$Comp
+L Device:C_Small C104
+U 1 1 5FD40D1A
+P 9600 1100
+F 0 "C104" H 9700 1150 50  0000 L CNN
+F 1 "0.1uF" H 9700 1100 50  0000 L CNN
+F 2 "Capacitor_SMD:C_0603_1608Metric" H 9600 1100 50  0001 C CNN
+F 3 "~" H 9600 1100 50  0001 C CNN
+F 4 "212-00011" H 9600 1100 50  0001 C CNN "CPN"
+F 5 "3.3V" H 9600 1100 50  0001 C CNN "C_Vbias"
+F 6 "Kemet" H 9600 1100 50  0001 C CNN "Mfg"
+F 7 "C0603C104M4RACTU" H 9600 1100 50  0001 C CNN "Mfg Part Num"
+	1    9600 1100
+	1    0    0    -1
+$EndComp
+Wire Wire Line
+	9200 1000 9600 1000
+Connection ~ 9200 1000
+Wire Wire Line
+	9200 1200 9600 1200
+Connection ~ 9200 1200
 $EndSCHEMATC
