File: spi-to-ethanol.sch (KiCad schematic (older format))
At the start: 4 parts, among them J1401 IDC_BOX_HDR, U1401 TXB0106PWR

Commit message: Series resistors on high-speed signals.
fixes #7
Parts:
- added R1403, R1404, R1405: 22, Resistor_SMD:R_0603_1608Metric, symbol Device:R
Connections:
- net P0_ROM_SPI_CLK: now also R1404.1; no longer U1401.4 (A3)
- net P0_ROM_SPI_MOSI: now also R1405.1; no longer U1401.5 (A4)
- net SPI_ROM_MISO: now also R1403.2; no longer U1401.14 (B2)
- new net: R1403.1, U1401.14 (B2)
- new net: R1404.2, U1401.4 (A3)
- new net: R1405.2, U1401.5 (A4)
Changed lines of the file:
@@
 	4900 3950 4900 3600
-Wire Wire Line
-	4900 3600 4200 3600
-Wire Wire Line
-	4200 3700 4800 3700
 Wire Wire Line
 	4800 3700 4800 4050
@@
 Wire Wire Line
 	3000 3400 3100 3400
-Text HLabel 2550 3300 0    50   Input ~ 0
+Text HLabel 2250 3300 0    50   Input ~ 0
 ~SPI_ROM_CS
-Text HLabel 2550 3500 0    50   Output ~ 0
+Text HLabel 2250 3500 0    50   Output ~ 0
 SPI_ROM_MISO
-Text HLabel 2550 3600 0    50   Input ~ 0
+Text HLabel 2250 3600 0    50   Input ~ 0
 SPI_ROM_MOSI
-Text HLabel 2550 3700 0    50   Input ~ 0
+Text HLabel 2250 3700 0    50   Input ~ 0
 SPI_ROM_SCK
-Text HLabel 2550 3800 0    50   Input ~ 0
+Text HLabel 2250 3800 0    50   Input ~ 0
 ~SPI_ROM_PROG
 NoConn ~ 3100 3900
 Wire Wire Line
 	3100 3300 2650 3300
-Wire Wire Line
-	2550 3500 3100 3500
-Wire Wire Line
-	2550 3600 3100 3600
-Wire Wire Line
-	2550 3700 3100 3700
-Wire Wire Line
-	2550 3800 2850 3800
 Wire Wire Line
 	3100 4000 3100 4200
@@
 Connection ~ 2650 3300
 Wire Wire Line
-	2650 3300 2550 3300
-Wire Wire Line
 	2850 3000 2850 3800
 Connection ~ 2850 3800
@@
 $EndComp
 Connection ~ 5450 3400
+Wire Wire Line
+	2250 3300 2650 3300
+Wire Wire Line
+	2250 3600 3100 3600
+Wire Wire Line
+	2250 3700 3100 3700
+Wire Wire Line
+	2250 3800 2850 3800
+$Comp
+L Device:R R1403
+U 1 1 5F683FBE
+P 2650 3500
+F 0 "R1403" V 2600 3650 50  0000 C CNN
+F 1 "22" V 2650 3500 50  0000 C CNN
+F 2 "Resistor_SMD:R_0603_1608Metric" V 2580 3500 50  0001 C CNN
+F 3 "~" H 2650 3500 50  0001 C CNN
+	1    2650 3500
+	0    1    1    0
+$EndComp
+Wire Wire Line
+	3100 3500 2800 3500
+Wire Wire Line
+	2500 3500 2250 3500
+$Comp
+L Device:R R1404
+U 1 1 5F686598
+P 4550 3600
+F 0 "R1404" V 4500 3750 50  0000 C CNN
+F 1 "22" V 4550 3600 50  0000 C CNN
+F 2 "Resistor_SMD:R_0603_1608Metric" V 4480 3600 50  0001 C CNN
+F 3 "~" H 4550 3600 50  0001 C CNN
+	1    4550 3600
+	0    1    1    0
+$EndComp
+$Comp
+L Device:R R1405
+U 1 1 5F686B24
+P 4550 3700
+F 0 "R1405" V 4500 3850 50  0000 C CNN
+F 1 "22" V 4550 3700 50  0000 C CNN
+F 2 "Resistor_SMD:R_0603_1608Metric" V 4480 3700 50  0001 C CNN
+F 3 "~" H 4550 3700 50  0001 C CNN
+	1    4550 3700
+	0    1    1    0
+$EndComp
+Wire Wire Line
+	4400 3600 4200 3600
+Wire Wire Line
+	4400 3700 4200 3700
+Wire Wire Line
+	4700 3600 4900 3600
+Wire Wire Line
+	4800 3700 4700 3700
 $EndSCHEMATC

Commit message: Switch IDC connectors to SMD footprints.
Parts:
- J1401: footprint Connector_IDC:IDC-Header_2x04_P2.54mm_Vertical -> idc-smd:IDC-Header_02x04_2.54mm_Vertical_SMD
Changed lines of the file:
@@
 F 0 "J1401" H 5900 3967 50  0000 C CNN
 F 1 "IDC_BOX_HDR" H 5900 3876 50  0000 C CNN
-F 2 "Connector_IDC:IDC-Header_2x04_P2.54mm_Vertical" H 5850 3650 50  0001 C CNN
+F 2 "idc-smd:IDC-Header_02x04_2.54mm_Vertical_SMD" H 5850 3650 50  0001 C CNN
 F 3 "~" H 5850 3650 50  0001 C CNN
 	1    5850 3650

Commit message: MB: annotate everything with mfg/MPN
Parts:
- J1401: Mfg (none) -> Würth Elektronik; Mfg Part Num (none) -> 61200820621
- R1401, R1402, R1403, R1404, R1405: Mfg Part Num (none) -> generic
- U1401: Mfg (none) -> Texas Instruments; Mfg Part Num (none) -> TXB0106PWR
Changed lines of the file:
@@
 F 2 "idc-smd:IDC-Header_02x04_2.54mm_Vertical_SMD" H 5850 3650 50  0001 C CNN
 F 3 "~" H 5850 3650 50  0001 C CNN
+F 4 "Würth Elektronik" H 5850 3650 50  0001 C CNN "Mfg"
+F 5 "61200820621" H 5850 3650 50  0001 C CNN "Mfg Part Num"
 	1    5850 3650
 	1    0    0    -1
@@
 F 2 "Package_SO:TSSOP-16_4.4x5mm_P0.65mm" H 3650 3700 50  0001 C CNN
 F 3 "" H 3650 3700 50  0001 C CNN
+F 4 "Texas Instruments" H 3650 3700 50  0001 C CNN "Mfg"
+F 5 "TXB0106PWR" H 3650 3700 50  0001 C CNN "Mfg Part Num"
 	1    3650 3700
 	-1   0    0    -1
@@
 F 2 "Resistor_SMD:R_0603_1608Metric" V 2780 2850 50  0001 C CNN
 F 3 "~" H 2850 2850 50  0001 C CNN
+F 4 "generic" H 2850 2850 50  0001 C CNN "Mfg Part Num"
 	1    2850 2850
 	1    0    0    -1
@@
 F 2 "Resistor_SMD:R_0603_1608Metric" V 2580 2850 50  0001 C CNN
 F 3 "~" H 2650 2850 50  0001 C CNN
+F 4 "generic" H 2650 2850 50  0001 C CNN "Mfg Part Num"
 	1    2650 2850
 	1    0    0    -1
@@
 F 2 "Resistor_SMD:R_0603_1608Metric" V 2580 3500 50  0001 C CNN
 F 3 "~" H 2650 3500 50  0001 C CNN
+F 4 "generic" H 2650 3500 50  0001 C CNN "Mfg Part Num"
 	1    2650 3500
 	0    1    1    0
@@
 F 2 "Resistor_SMD:R_0603_1608Metric" V 4480 3600 50  0001 C CNN
 F 3 "~" H 4550 3600 50  0001 C CNN
+F 4 "generic" H 4550 3600 50  0001 C CNN "Mfg Part Num"
 	1    4550 3600
 	0    1    1    0
@@
 F 2 "Resistor_SMD:R_0603_1608Metric" V 4480 3700 50  0001 C CNN
 F 3 "~" H 4550 3700 50  0001 C CNN
+F 4 "generic" H 4550 3700 50  0001 C CNN "Mfg Part Num"
 	1    4550 3700
 	0    1    1    0

Commit message: MB: assign single resistors
Parts:
- R1401, R1402: Mfg (none) -> Bourns; Mfg Part Num generic -> CR0603-JW-103ELF
- R1403, R1404, R1405: Mfg (none) -> Bourns; Mfg Part Num generic -> CR0603-JW-220ELF
Changed lines of the file:
@@
 F 2 "Resistor_SMD:R_0603_1608Metric" V 2780 2850 50  0001 C CNN
 F 3 "~" H 2850 2850 50  0001 C CNN
-F 4 "generic" H 2850 2850 50  0001 C CNN "Mfg Part Num"
+F 4 "CR0603-JW-103ELF" H 2850 2850 50  0001 C CNN "Mfg Part Num"
+F 5 "Bourns" H 2850 2850 50  0001 C CNN "Mfg"
 	1    2850 2850
 	1    0    0    -1
@@
 F 2 "Resistor_SMD:R_0603_1608Metric" V 2580 2850 50  0001 C CNN
 F 3 "~" H 2650 2850 50  0001 C CNN
-F 4 "generic" H 2650 2850 50  0001 C CNN "Mfg Part Num"
+F 4 "CR0603-JW-103ELF" H 2650 2850 50  0001 C CNN "Mfg Part Num"
+F 5 "Bourns" H 2650 2850 50  0001 C CNN "Mfg"
 	1    2650 2850
 	1    0    0    -1
@@
 F 2 "Resistor_SMD:R_0603_1608Metric" V 2580 3500 50  0001 C CNN
 F 3 "~" H 2650 3500 50  0001 C CNN
-F 4 "generic" H 2650 3500 50  0001 C CNN "Mfg Part Num"
+F 4 "CR0603-JW-220ELF" H 2650 3500 50  0001 C CNN "Mfg Part Num"
+F 5 "Bourns" H 2650 3500 50  0001 C CNN "Mfg"
 	1    2650 3500
 	0    1    1    0
@@
 F 2 "Resistor_SMD:R_0603_1608Metric" V 4480 3600 50  0001 C CNN
 F 3 "~" H 4550 3600 50  0001 C CNN
-F 4 "generic" H 4550 3600 50  0001 C CNN "Mfg Part Num"
+F 4 "CR0603-JW-220ELF" H 4550 3600 50  0001 C CNN "Mfg Part Num"
+F 5 "Bourns" H 4550 3600 50  0001 C CNN "Mfg"
 	1    4550 3600
 	0    1    1    0
@@
 F 2 "Resistor_SMD:R_0603_1608Metric" V 4480 3700 50  0001 C CNN
 F 3 "~" H 4550 3700 50  0001 C CNN
-F 4 "generic" H 4550 3700 50  0001 C CNN "Mfg Part Num"
+F 4 "CR0603-JW-220ELF" H 4550 3700 50  0001 C CNN "Mfg Part Num"
+F 5 "Bourns" H 4550 3700 50  0001 C CNN "Mfg"
 	1    4550 3700
 	0    1    1    0

Commit message: MB: add caps suggested in review
Parts:
- added C1401, C1402: 0µ1, Capacitor_SMD:C_0603_1608Metric, symbol Device:C_Small
Connections:
- net +3V3: now also C1401.1
- net 1v8: now also C1402.1
- net GND: now also C1401.2, C1402.2
Changed lines of the file:
@@
 L power:+3V3 #PWR0104
 U 1 1 5F4199CC
-P 3000 2900
-F 0 "#PWR0104" H 3000 2750 50  0001 C CNN
-F 1 "+3V3" H 3015 3073 50  0000 C CNN
-F 2 "" H 3000 2900 50  0001 C CNN
-F 3 "" H 3000 2900 50  0001 C CNN
-	1    3000 2900
-	1    0    0    -1
-$EndComp
-Wire Wire Line
-	3000 2900 3000 3400
+P 3000 2700
+F 0 "#PWR0104" H 3000 2550 50  0001 C CNN
+F 1 "+3V3" H 3015 2873 50  0000 C CNN
+F 2 "" H 3000 2700 50  0001 C CNN
+F 3 "" H 3000 2700 50  0001 C CNN
+	1    3000 2700
+	1    0    0    -1
+$EndComp
+Wire Wire Line
+	3000 2700 3000 2850
 Wire Wire Line
 	3000 3400 3100 3400
@@
 Wire Wire Line
 	4800 3700 4700 3700
+$Comp
+L Device:C_Small C?
+U 1 1 5F6C03A9
+P 4300 4250
+AR Path="/5F1928E5/5F29584B/5F6C03A9" Ref="C?"  Part="1"
+AR Path="/5F40F867/5F6C03A9" Ref="C1402"  Part="1"
+F 0 "C1402" H 4392 4296 50  0000 L CNN
+F 1 "0µ1" H 4392 4205 50  0000 L CNN
+F 2 "Capacitor_SMD:C_0603_1608Metric" H 4300 4250 50  0001 C CNN
+F 3 "~" H 4300 4250 50  0001 C CNN
+F 4 "CL10B104KB8NNWC" H 4300 4250 50  0001 C CNN "Mfg Part Num"
+F 5 "Samsung Electro-Mechanics" H 4300 4250 50  0001 C CNN "Mfg"
+	1    4300 4250
+	1    0    0    -1
+$EndComp
+Wire Wire Line
+	4300 4150 4300 4000
+Connection ~ 4300 4000
+$Comp
+L power:GND #PWR01402
+U 1 1 5F6C1B1B
+P 4300 4350
+F 0 "#PWR01402" H 4300 4100 50  0001 C CNN
+F 1 "GND" H 4305 4177 50  0000 C CNN
+F 2 "" H 4300 4350 50  0001 C CNN
+F 3 "" H 4300 4350 50  0001 C CNN
+	1    4300 4350
+	1    0    0    -1
+$EndComp
+$Comp
+L Device:C_Small C?
+U 1 1 5F6C1DD4
+P 3150 2950
+AR Path="/5F1928E5/5F29584B/5F6C1DD4" Ref="C?"  Part="1"
+AR Path="/5F40F867/5F6C1DD4" Ref="C1401"  Part="1"
+F 0 "C1401" H 3242 2996 50  0000 L CNN
+F 1 "0µ1" H 3242 2905 50  0000 L CNN
+F 2 "Capacitor_SMD:C_0603_1608Metric" H 3150 2950 50  0001 C CNN
+F 3 "~" H 3150 2950 50  0001 C CNN
+F 4 "CL10B104KB8NNWC" H 3150 2950 50  0001 C CNN "Mfg Part Num"
+F 5 "Samsung Electro-Mechanics" H 3150 2950 50  0001 C CNN "Mfg"
+	1    3150 2950
+	1    0    0    -1
+$EndComp
+Wire Wire Line
+	3150 2850 3000 2850
+Connection ~ 3000 2850
+Wire Wire Line
+	3000 2850 3000 3400
+$Comp
+L power:GND #PWR01401
+U 1 1 5F6C4559
+P 3150 3050
+F 0 "#PWR01401" H 3150 2800 50  0001 C CNN
+F 1 "GND" H 3155 2877 50  0000 C CNN
+F 2 "" H 3150 3050 50  0001 C CNN
+F 3 "" H 3150 3050 50  0001 C CNN
+	1    3150 3050
+	1    0    0    -1
+$EndComp
 $EndSCHEMATC

Commit message: gemini-bringup: Add CPNs for all components
Parts:
- C1401, C1402: CPN (none) -> 212-00011
- J1401: CPN (none) -> 215-00034
- R1401, R1402: CPN (none) -> 232-00024
- R1403, R1404, R1405: CPN (none) -> 232-00019
- U1401: CPN (none) -> 221-00019
Changed lines of the file:
@@
 F 4 "Würth Elektronik" H 5850 3650 50  0001 C CNN "Mfg"
 F 5 "61200820621" H 5850 3650 50  0001 C CNN "Mfg Part Num"
+F 6 "215-00034" H 5850 3650 50  0001 C CNN "CPN"
 	1    5850 3650
 	1    0    0    -1
@@
 F 4 "Texas Instruments" H 3650 3700 50  0001 C CNN "Mfg"
 F 5 "TXB0106PWR" H 3650 3700 50  0001 C CNN "Mfg Part Num"
+F 6 "221-00019" H 3650 3700 50  0001 C CNN "CPN"
 	1    3650 3700
 	-1   0    0    -1
@@
 F 4 "CR0603-JW-103ELF" H 2850 2850 50  0001 C CNN "Mfg Part Num"
 F 5 "Bourns" H 2850 2850 50  0001 C CNN "Mfg"
+F 6 "232-00024" H 2850 2850 50  0001 C CNN "CPN"
 	1    2850 2850
 	1    0    0    -1
@@
 F 4 "CR0603-JW-103ELF" H 2650 2850 50  0001 C CNN "Mfg Part Num"
 F 5 "Bourns" H 2650 2850 50  0001 C CNN "Mfg"
+F 6 "232-00024" H 2650 2850 50  0001 C CNN "CPN"
 	1    2650 2850
 	1    0    0    -1
@@
 F 4 "CR0603-JW-220ELF" H 2650 3500 50  0001 C CNN "Mfg Part Num"
 F 5 "Bourns" H 2650 3500 50  0001 C CNN "Mfg"
+F 6 "232-00019" H 2650 3500 50  0001 C CNN "CPN"
 	1    2650 3500
 	0    1    1    0
@@
 F 4 "CR0603-JW-220ELF" H 4550 3600 50  0001 C CNN "Mfg Part Num"
 F 5 "Bourns" H 4550 3600 50  0001 C CNN "Mfg"
+F 6 "232-00019" H 4550 3600 50  0001 C CNN "CPN"
 	1    4550 3600
 	0    1    1    0
@@
 F 4 "CR0603-JW-220ELF" H 4550 3700 50  0001 C CNN "Mfg Part Num"
 F 5 "Bourns" H 4550 3700 50  0001 C CNN "Mfg"
+F 6 "232-00019" H 4550 3700 50  0001 C CNN "CPN"
 	1    4550 3700
 	0    1    1    0
@@
 F 4 "CL10B104KB8NNWC" H 4300 4250 50  0001 C CNN "Mfg Part Num"
 F 5 "Samsung Electro-Mechanics" H 4300 4250 50  0001 C CNN "Mfg"
+F 6 "212-00011" H 4300 4250 50  0001 C CNN "CPN"
 	1    4300 4250
 	1    0    0    -1
@@
 F 4 "CL10B104KB8NNWC" H 3150 2950 50  0001 C CNN "Mfg Part Num"
 F 5 "Samsung Electro-Mechanics" H 3150 2950 50  0001 C CNN "Mfg"
+F 6 "212-00011" H 3150 2950 50  0001 C CNN "CPN"
 	1    3150 2950
 	1    0    0    -1

Commit message: spi-to-ethanol: specify rating constraints on passives
Parts:
- C1401: value 0µ1 -> 0.1uF 3.3VDCbias
- C1402: value 0µ1 -> 01.uF 1.8VDCbias
- R1401, R1402: value 10k -> 10kR
- R1403, R1404, R1405: value 22 -> 22R
Connections:
- net ~SPI_ROM_PROG is gone; now on net SPI_ROM_MISO: R1402.2, U1401.11 (B5)
Other:
- moved on the sheet: C1401, R1401, R1402, R1403
Changed lines of the file:
@@
 	6250 3550 6250 3950
 Wire Wire Line
-	6250 3950 4900 3950
-Wire Wire Line
-	4900 3950 4900 3600
+	6250 3950 4950 3950
+Wire Wire Line
+	4950 3950 4950 3600
 Wire Wire Line
 	4800 3700 4800 4050
@@
 $EndComp
 Wire Wire Line
-	3000 2700 3000 2850
-Wire Wire Line
 	3000 3400 3100 3400
 Text HLabel 2250 3300 0    50   Input ~ 0
@@
 NoConn ~ 3100 3900
 Wire Wire Line
-	3100 3300 2650 3300
+	3100 3300 2400 3300
 Wire Wire Line
 	3100 4000 3100 4200
@@
 L Device:R R1402
 U 1 1 5F41FBDE
-P 2850 2850
-F 0 "R1402" V 2750 2750 50  0000 L CNN
-F 1 "10k" V 2850 2800 50  0000 L CNN
-F 2 "Resistor_SMD:R_0603_1608Metric" V 2780 2850 50  0001 C CNN
-F 3 "~" H 2850 2850 50  0001 C CNN
-F 4 "CR0603-JW-103ELF" H 2850 2850 50  0001 C CNN "Mfg Part Num"
-F 5 "Bourns" H 2850 2850 50  0001 C CNN "Mfg"
-F 6 "232-00024" H 2850 2850 50  0001 C CNN "CPN"
-	1    2850 2850
+P 2600 2850
+F 0 "R1402" H 2700 2900 50  0000 L CNN
+F 1 "10kR" H 2700 2850 50  0000 L CNN
+F 2 "Resistor_SMD:R_0603_1608Metric" V 2530 2850 50  0001 C CNN
+F 3 "~" H 2600 2850 50  0001 C CNN
+F 4 "CR0603-JW-103ELF" H 2600 2850 50  0001 C CNN "Mfg Part Num"
+F 5 "Bourns" H 2600 2850 50  0001 C CNN "Mfg"
+F 6 "232-00024" H 2600 2850 50  0001 C CNN "CPN"
+	1    2600 2850
 	1    0    0    -1
 $EndComp
@@
 L Device:R R1401
 U 1 1 5F420CA2
-P 2650 2850
-F 0 "R1401" V 2550 2750 50  0000 L CNN
-F 1 "10k" V 2650 2800 50  0000 L CNN
-F 2 "Resistor_SMD:R_0603_1608Metric" V 2580 2850 50  0001 C CNN
-F 3 "~" H 2650 2850 50  0001 C CNN
-F 4 "CR0603-JW-103ELF" H 2650 2850 50  0001 C CNN "Mfg Part Num"
-F 5 "Bourns" H 2650 2850 50  0001 C CNN "Mfg"
-F 6 "232-00024" H 2650 2850 50  0001 C CNN "CPN"
-	1    2650 2850
-	1    0    0    -1
-$EndComp
-Wire Wire Line
-	2650 3000 2650 3300
-Connection ~ 2650 3300
-Wire Wire Line
-	2850 3000 2850 3800
-Connection ~ 2850 3800
-Wire Wire Line
-	2850 3800 3100 3800
-Wire Wire Line
-	2650 2700 2750 2700
+P 2400 2850
+F 0 "R1401" H 2300 2900 50  0000 R CNN
+F 1 "10kR" H 2300 2850 50  0000 R CNN
+F 2 "Resistor_SMD:R_0603_1608Metric" V 2330 2850 50  0001 C CNN
+F 3 "~" H 2400 2850 50  0001 C CNN
+F 4 "CR0603-JW-103ELF" H 2400 2850 50  0001 C CNN "Mfg Part Num"
+F 5 "Bourns" H 2400 2850 50  0001 C CNN "Mfg"
+F 6 "232-00024" H 2400 2850 50  0001 C CNN "CPN"
+	1    2400 2850
+	1    0    0    -1
+$EndComp
+Wire Wire Line
+	2400 3000 2400 3300
+Connection ~ 2400 3300
+Wire Wire Line
+	2600 3000 2600 3500
+Connection ~ 2600 3800
+Wire Wire Line
+	2600 3800 3100 3800
+Wire Wire Line
+	2400 2700 2500 2700
 $Comp
 L power:+3V3 #PWR0106
 U 1 1 5F422974
-P 2750 2700
-F 0 "#PWR0106" H 2750 2550 50  0001 C CNN
-F 1 "+3V3" H 2765 2873 50  0000 C CNN
-F 2 "" H 2750 2700 50  0001 C CNN
-F 3 "" H 2750 2700 50  0001 C CNN
-	1    2750 2700
-	1    0    0    -1
-$EndComp
-Connection ~ 2750 2700
-Wire Wire Line
-	2750 2700 2850 2700
+P 2500 2700
+F 0 "#PWR0106" H 2500 2550 50  0001 C CNN
+F 1 "+3V3" H 2515 2873 50  0000 C CNN
+F 2 "" H 2500 2700 50  0001 C CNN
+F 3 "" H 2500 2700 50  0001 C CNN
+	1    2500 2700
+	1    0    0    -1
+$EndComp
+Connection ~ 2500 2700
+Wire Wire Line
+	2500 2700 2600 2700
 $Comp
 L power:PWR_FLAG #FLG0101
@@
 Connection ~ 5450 3400
 Wire Wire Line
-	2250 3300 2650 3300
+	2250 3300 2400 3300
 Wire Wire Line
 	2250 3600 3100 3600
@@
 	2250 3700 3100 3700
 Wire Wire Line
-	2250 3800 2850 3800
-$Comp
-L Device:R R1403
-U 1 1 5F683FBE
-P 2650 3500
-F 0 "R1403" V 2600 3650 50  0000 C CNN
-F 1 "22" V 2650 3500 50  0000 C CNN
-F 2 "Resistor_SMD:R_0603_1608Metric" V 2580 3500 50  0001 C CNN
-F 3 "~" H 2650 3500 50  0001 C CNN
-F 4 "CR0603-JW-220ELF" H 2650 3500 50  0001 C CNN "Mfg Part Num"
-F 5 "Bourns" H 2650 3500 50  0001 C CNN "Mfg"
-F 6 "232-00019" H 2650 3500 50  0001 C CNN "CPN"
-	1    2650 3500
-	0    1    1    0
-$EndComp
-Wire Wire Line
-	3100 3500 2800 3500
-Wire Wire Line
-	2500 3500 2250 3500
+	2250 3800 2600 3800
+Wire Wire Line
+	3100 3500 2900 3500
+Wire Wire Line
+	2600 3500 2250 3500
 $Comp
 L Device:R R1404
 U 1 1 5F686598
 P 4550 3600
-F 0 "R1404" V 4500 3750 50  0000 C CNN
-F 1 "22" V 4550 3600 50  0000 C CNN
+F 0 "R1404" V 4500 3850 50  0000 C CNN
+F 1 "22R" V 4550 3600 50  0000 C CNN
 F 2 "Resistor_SMD:R_0603_1608Metric" V 4480 3600 50  0001 C CNN
 F 3 "~" H 4550 3600 50  0001 C CNN
@@
 U 1 1 5F686B24
 P 4550 3700
-F 0 "R1405" V 4500 3850 50  0000 C CNN
-F 1 "22" V 4550 3700 50  0000 C CNN
+F 0 "R1405" V 4500 3950 50  0000 C CNN
+F 1 "22R" V 4550 3700 50  0000 C CNN
 F 2 "Resistor_SMD:R_0603_1608Metric" V 4480 3700 50  0001 C CNN
 F 3 "~" H 4550 3700 50  0001 C CNN
@@
 	4400 3700 4200 3700
 Wire Wire Line
-	4700 3600 4900 3600
+	4700 3600 4950 3600
 Wire Wire Line
 	4800 3700 4700 3700
@@
 AR Path="/5F40F867/5F6C03A9" Ref="C1402"  Part="1"
 F 0 "C1402" H 4392 4296 50  0000 L CNN
-F 1 "0µ1" H 4392 4205 50  0000 L CNN
+F 1 "01.uF 1.8VDCbias" H 4392 4205 50  0000 L CNN
 F 2 "Capacitor_SMD:C_0603_1608Metric" H 4300 4250 50  0001 C CNN
 F 3 "~" H 4300 4250 50  0001 C CNN
@@
 L Device:C_Small C?
 U 1 1 5F6C1DD4
-P 3150 2950
+P 3150 2800
 AR Path="/5F1928E5/5F29584B/5F6C1DD4" Ref="C?"  Part="1"
 AR Path="/5F40F867/5F6C1DD4" Ref="C1401"  Part="1"
-F 0 "C1401" H 3242 2996 50  0000 L CNN
-F 1 "0µ1" H 3242 2905 50  0000 L CNN
-F 2 "Capacitor_SMD:C_0603_1608Metric" H 3150 2950 50  0001 C CNN
-F 3 "~" H 3150 2950 50  0001 C CNN
-F 4 "CL10B104KB8NNWC" H 3150 2950 50  0001 C CNN "Mfg Part Num"
-F 5 "Samsung Electro-Mechanics" H 3150 2950 50  0001 C CNN "Mfg"
-F 6 "212-00011" H 3150 2950 50  0001 C CNN "CPN"
-	1    3150 2950
-	1    0    0    -1
-$EndComp
-Wire Wire Line
-	3150 2850 3000 2850
-Connection ~ 3000 2850
-Wire Wire Line
-	3000 2850 3000 3400
+F 0 "C1401" H 3242 2846 50  0000 L CNN
+F 1 "0.1uF 3.3VDCbias" H 3242 2755 50  0000 L CNN
+F 2 "Capacitor_SMD:C_0603_1608Metric" H 3150 2800 50  0001 C CNN
+F 3 "~" H 3150 2800 50  0001 C CNN
+F 4 "CL10B104KB8NNWC" H 3150 2800 50  0001 C CNN "Mfg Part Num"
+F 5 "Samsung Electro-Mechanics" H 3150 2800 50  0001 C CNN "Mfg"
+F 6 "212-00011" H 3150 2800 50  0001 C CNN "CPN"
+	1    3150 2800
+	1    0    0    -1
+$EndComp
+Wire Wire Line
+	3150 2700 3000 2700
+Connection ~ 3000 2700
+Wire Wire Line
+	3000 2700 3000 3400
 $Comp
 L power:GND #PWR01401
 U 1 1 5F6C4559
-P 3150 3050
-F 0 "#PWR01401" H 3150 2800 50  0001 C CNN
-F 1 "GND" H 3155 2877 50  0000 C CNN
-F 2 "" H 3150 3050 50  0001 C CNN
-F 3 "" H 3150 3050 50  0001 C CNN
-	1    3150 3050
-	1    0    0    -1
+P 3150 2900
+F 0 "#PWR01401" H 3150 2650 50  0001 C CNN
+F 1 "GND" H 3155 2727 50  0000 C CNN
+F 2 "" H 3150 2900 50  0001 C CNN
+F 3 "" H 3150 2900 50  0001 C CNN
+	1    3150 2900
+	1    0    0    -1
+$EndComp
+Connection ~ 2600 3500
+Wire Wire Line
+	2600 3500 2600 3800
+$Comp
+L Device:R R1403
+U 1 1 5F683FBE
+P 2750 3500
+F 0 "R1403" V 2650 3500 50  0000 C CNN
+F 1 "22R" V 2750 3500 50  0000 C CNN
+F 2 "Resistor_SMD:R_0603_1608Metric" V 2680 3500 50  0001 C CNN
+F 3 "~" H 2750 3500 50  0001 C CNN
+F 4 "CR0603-JW-220ELF" H 2750 3500 50  0001 C CNN "Mfg Part Num"
+F 5 "Bourns" H 2750 3500 50  0001 C CNN "Mfg"
+F 6 "232-00019" H 2750 3500 50  0001 C CNN "CPN"
+	1    2750 3500
+	0    1    1    0
 $EndComp
 $EndSCHEMATC
