File: spi-to-ethanol.sch (KiCad schematic (older format))
At the start: 9 parts, among them J1401 IDC_BOX_HDR, U1401 TXB0106PWR

Commit message: gemini-bringup: custom fields for rating constraints on passives
Instead of packing tons of detail into a single "Value" field, limit
"Value" to the primary characteristic of the device (i.e. capacitance
for capacitors, resistance for resistors, current for fuses, impedence
at frequency for ferrite beads). For all other rating constraints, use
custom fields of the form <component-refdes-prefix>_<constraint>. For
example, R_P contains the power a resistor must dissipate.  Use
calculated values when possible rather than standard values as the
intent is to capture the constraint, not a specific device choice.
Parts:
- C1401: value 0.1uF 3.3VDCbias -> 0.1uF; C_Vbias (none) -> 3.3V
- C1402: value 01.uF 1.8VDCbias -> 01.uF; C_Vbias (none) -> 1.8V
Changed lines of the file:
@@
 AR Path="/5F40F867/5F6C03A9" Ref="C1402"  Part="1"
 F 0 "C1402" H 4392 4296 50  0000 L CNN
-F 1 "01.uF 1.8VDCbias" H 4392 4205 50  0000 L CNN
+F 1 "01.uF" H 4392 4205 50  0000 L CNN
 F 2 "Capacitor_SMD:C_0603_1608Metric" H 4300 4250 50  0001 C CNN
 F 3 "~" H 4300 4250 50  0001 C CNN
@@
 F 5 "Samsung Electro-Mechanics" H 4300 4250 50  0001 C CNN "Mfg"
 F 6 "212-00011" H 4300 4250 50  0001 C CNN "CPN"
+F 7 "1.8V" H 4300 4250 50  0001 C CNN "C_Vbias"
 	1    4300 4250
 	1    0    0    -1
@@
 AR Path="/5F40F867/5F6C1DD4" Ref="C1401"  Part="1"
 F 0 "C1401" H 3242 2846 50  0000 L CNN
-F 1 "0.1uF 3.3VDCbias" H 3242 2755 50  0000 L CNN
+F 1 "0.1uF" H 3242 2755 50  0000 L CNN
 F 2 "Capacitor_SMD:C_0603_1608Metric" H 3150 2800 50  0001 C CNN
 F 3 "~" H 3150 2800 50  0001 C CNN
@@
 F 5 "Samsung Electro-Mechanics" H 3150 2800 50  0001 C CNN "Mfg"
 F 6 "212-00011" H 3150 2800 50  0001 C CNN "CPN"
+F 7 "3.3V" H 3150 2800 50  0001 C CNN "C_Vbias"
 	1    3150 2800
 	1    0    0    -1

Commit message: gemini-bringup: resistor power rating constraints
Parts:
- R1401, R1402: R_P (none) -> 300uW
Changed lines of the file:
@@
 F 5 "Bourns" H 2600 2850 50  0001 C CNN "Mfg"
 F 6 "232-00024" H 2600 2850 50  0001 C CNN "CPN"
+F 7 "300uW" H 2600 2850 50  0001 C CNN "R_P"
 	1    2600 2850
 	1    0    0    -1
@@
 F 5 "Bourns" H 2400 2850 50  0001 C CNN "Mfg"
 F 6 "232-00024" H 2400 2850 50  0001 C CNN "CPN"
+F 7 "300uW" H 2400 2850 50  0001 C CNN "R_P"
 	1    2400 2850
 	1    0    0    -1

Commit message: spi-to-ethanol: fix capacitor value typo
Parts:
- C1402: value 01.uF -> 0.1uF
Changed lines of the file:
@@
 AR Path="/5F40F867/5F6C03A9" Ref="C1402"  Part="1"
 F 0 "C1402" H 4392 4296 50  0000 L CNN
-F 1 "01.uF" H 4392 4205 50  0000 L CNN
+F 1 "0.1uF" H 4392 4205 50  0000 L CNN
 F 2 "Capacitor_SMD:C_0603_1608Metric" H 4300 4250 50  0001 C CNN
 F 3 "~" H 4300 4250 50  0001 C CNN

Commit message: gemini-bringup: reselect all caps respecting C/V derating
Parts:
- C1401, C1402: Mfg Samsung Electro-Mechanics -> Kemet; Mfg Part Num CL10B104KB8NNWC -> C0603C104M4RACTU
Changed lines of the file:
@@
 F 2 "Capacitor_SMD:C_0603_1608Metric" H 4300 4250 50  0001 C CNN
 F 3 "~" H 4300 4250 50  0001 C CNN
-F 4 "CL10B104KB8NNWC" H 4300 4250 50  0001 C CNN "Mfg Part Num"
-F 5 "Samsung Electro-Mechanics" H 4300 4250 50  0001 C CNN "Mfg"
+F 4 "C0603C104M4RACTU" H 4300 4250 50  0001 C CNN "Mfg Part Num"
+F 5 "Kemet" H 4300 4250 50  0001 C CNN "Mfg"
 F 6 "212-00011" H 4300 4250 50  0001 C CNN "CPN"
 F 7 "1.8V" H 4300 4250 50  0001 C CNN "C_Vbias"
@@
 F 2 "Capacitor_SMD:C_0603_1608Metric" H 3150 2800 50  0001 C CNN
 F 3 "~" H 3150 2800 50  0001 C CNN
-F 4 "CL10B104KB8NNWC" H 3150 2800 50  0001 C CNN "Mfg Part Num"
-F 5 "Samsung Electro-Mechanics" H 3150 2800 50  0001 C CNN "Mfg"
+F 4 "C0603C104M4RACTU" H 3150 2800 50  0001 C CNN "Mfg Part Num"
+F 5 "Kemet" H 3150 2800 50  0001 C CNN "Mfg"
 F 6 "212-00011" H 3150 2800 50  0001 C CNN "CPN"
 F 7 "3.3V" H 3150 2800 50  0001 C CNN "C_Vbias"

Commit message: spi-to-ethanol: remove accidental connection between ~SPI_ROM_PROG and SPI_ROM_MISO
Connections:
- net SPI_ROM_MISO: no longer R1402.2, U1401.11 (B5)
- new net ~SPI_ROM_PROG: R1402.2, U1401.11 (B5)
Other:
- moved on the sheet: R1401, R1402, R1403
Changed lines of the file:
@@
 Wire Wire Line
 	3000 3400 3100 3400
-Text HLabel 2250 3300 0    50   Input ~ 0
+Text HLabel 2150 3300 0    50   Input ~ 0
 ~SPI_ROM_CS
-Text HLabel 2250 3500 0    50   Output ~ 0
+Text HLabel 2150 3500 0    50   Output ~ 0
 SPI_ROM_MISO
-Text HLabel 2250 3600 0    50   Input ~ 0
+Text HLabel 2150 3600 0    50   Input ~ 0
 SPI_ROM_MOSI
-Text HLabel 2250 3700 0    50   Input ~ 0
+Text HLabel 2150 3700 0    50   Input ~ 0
 SPI_ROM_SCK
-Text HLabel 2250 3800 0    50   Input ~ 0
+Text HLabel 2150 3800 0    50   Input ~ 0
 ~SPI_ROM_PROG
 NoConn ~ 3100 3900
 Wire Wire Line
-	3100 3300 2400 3300
+	3100 3300 2300 3300
 Wire Wire Line
 	3100 4000 3100 4200
@@
 L Device:R R1402
 U 1 1 5F41FBDE
-P 2600 2850
-F 0 "R1402" H 2700 2900 50  0000 L CNN
-F 1 "10kR" H 2700 2850 50  0000 L CNN
-F 2 "Resistor_SMD:R_0603_1608Metric" V 2530 2850 50  0001 C CNN
-F 3 "~" H 2600 2850 50  0001 C CNN
-F 4 "CR0603-JW-103ELF" H 2600 2850 50  0001 C CNN "Mfg Part Num"
-F 5 "Bourns" H 2600 2850 50  0001 C CNN "Mfg"
-F 6 "232-00024" H 2600 2850 50  0001 C CNN "CPN"
-F 7 "300uW" H 2600 2850 50  0001 C CNN "R_P"
-	1    2600 2850
+P 2500 2850
+F 0 "R1402" H 2600 2900 50  0000 L CNN
+F 1 "10kR" H 2600 2850 50  0000 L CNN
+F 2 "Resistor_SMD:R_0603_1608Metric" V 2430 2850 50  0001 C CNN
+F 3 "~" H 2500 2850 50  0001 C CNN
+F 4 "CR0603-JW-103ELF" H 2500 2850 50  0001 C CNN "Mfg Part Num"
+F 5 "Bourns" H 2500 2850 50  0001 C CNN "Mfg"
+F 6 "232-00024" H 2500 2850 50  0001 C CNN "CPN"
+F 7 "300uW" H 2500 2850 50  0001 C CNN "R_P"
+	1    2500 2850
 	1    0    0    -1
 $EndComp
@@
 L Device:R R1401
 U 1 1 5F420CA2
-P 2400 2850
-F 0 "R1401" H 2300 2900 50  0000 R CNN
-F 1 "10kR" H 2300 2850 50  0000 R CNN
-F 2 "Resistor_SMD:R_0603_1608Metric" V 2330 2850 50  0001 C CNN
-F 3 "~" H 2400 2850 50  0001 C CNN
-F 4 "CR0603-JW-103ELF" H 2400 2850 50  0001 C CNN "Mfg Part Num"
-F 5 "Bourns" H 2400 2850 50  0001 C CNN "Mfg"
-F 6 "232-00024" H 2400 2850 50  0001 C CNN "CPN"
-F 7 "300uW" H 2400 2850 50  0001 C CNN "R_P"
-	1    2400 2850
-	1    0    0    -1
-$EndComp
-Wire Wire Line
-	2400 3000 2400 3300
-Connection ~ 2400 3300
-Wire Wire Line
-	2600 3000 2600 3500
-Connection ~ 2600 3800
-Wire Wire Line
-	2600 3800 3100 3800
-Wire Wire Line
-	2400 2700 2500 2700
+P 2300 2850
+F 0 "R1401" H 2200 2900 50  0000 R CNN
+F 1 "10kR" H 2200 2850 50  0000 R CNN
+F 2 "Resistor_SMD:R_0603_1608Metric" V 2230 2850 50  0001 C CNN
+F 3 "~" H 2300 2850 50  0001 C CNN
+F 4 "CR0603-JW-103ELF" H 2300 2850 50  0001 C CNN "Mfg Part Num"
+F 5 "Bourns" H 2300 2850 50  0001 C CNN "Mfg"
+F 6 "232-00024" H 2300 2850 50  0001 C CNN "CPN"
+F 7 "300uW" H 2300 2850 50  0001 C CNN "R_P"
+	1    2300 2850
+	1    0    0    -1
+$EndComp
+Wire Wire Line
+	2300 3000 2300 3300
+Connection ~ 2300 3300
+Connection ~ 2500 3800
+Wire Wire Line
+	2500 3800 3100 3800
+Wire Wire Line
+	2300 2700 2400 2700
 $Comp
 L power:+3V3 #PWR0106
 U 1 1 5F422974
-P 2500 2700
-F 0 "#PWR0106" H 2500 2550 50  0001 C CNN
-F 1 "+3V3" H 2515 2873 50  0000 C CNN
-F 2 "" H 2500 2700 50  0001 C CNN
-F 3 "" H 2500 2700 50  0001 C CNN
-	1    2500 2700
-	1    0    0    -1
-$EndComp
-Connection ~ 2500 2700
-Wire Wire Line
-	2500 2700 2600 2700
+P 2400 2700
+F 0 "#PWR0106" H 2400 2550 50  0001 C CNN
+F 1 "+3V3" H 2415 2873 50  0000 C CNN
+F 2 "" H 2400 2700 50  0001 C CNN
+F 3 "" H 2400 2700 50  0001 C CNN
+	1    2400 2700
+	1    0    0    -1
+$EndComp
+Connection ~ 2400 2700
+Wire Wire Line
+	2400 2700 2500 2700
 $Comp
 L power:PWR_FLAG #FLG0101
@@
 Connection ~ 5450 3400
 Wire Wire Line
-	2250 3300 2400 3300
-Wire Wire Line
-	2250 3600 3100 3600
-Wire Wire Line
-	2250 3700 3100 3700
-Wire Wire Line
-	2250 3800 2600 3800
-Wire Wire Line
-	3100 3500 2900 3500
-Wire Wire Line
-	2600 3500 2250 3500
+	2150 3300 2300 3300
+Wire Wire Line
+	2150 3600 3100 3600
+Wire Wire Line
+	2150 3700 3100 3700
+Wire Wire Line
+	2150 3800 2500 3800
 $Comp
 L Device:R R1404
@@
 	1    0    0    -1
 $EndComp
-Connection ~ 2600 3500
-Wire Wire Line
-	2600 3500 2600 3800
+Wire Wire Line
+	3100 3500 2850 3500
 $Comp
 L Device:R R1403
 U 1 1 5F683FBE
-P 2750 3500
-F 0 "R1403" V 2650 3500 50  0000 C CNN
-F 1 "22R" V 2750 3500 50  0000 C CNN
-F 2 "Resistor_SMD:R_0603_1608Metric" V 2680 3500 50  0001 C CNN
-F 3 "~" H 2750 3500 50  0001 C CNN
-F 4 "CR0603-JW-220ELF" H 2750 3500 50  0001 C CNN "Mfg Part Num"
-F 5 "Bourns" H 2750 3500 50  0001 C CNN "Mfg"
-F 6 "232-00019" H 2750 3500 50  0001 C CNN "CPN"
-	1    2750 3500
+P 2700 3500
+F 0 "R1403" V 2600 3500 50  0000 C CNN
+F 1 "22R" V 2700 3500 50  0000 C CNN
+F 2 "Resistor_SMD:R_0603_1608Metric" V 2630 3500 50  0001 C CNN
+F 3 "~" H 2700 3500 50  0001 C CNN
+F 4 "CR0603-JW-220ELF" H 2700 3500 50  0001 C CNN "Mfg Part Num"
+F 5 "Bourns" H 2700 3500 50  0001 C CNN "Mfg"
+F 6 "232-00019" H 2700 3500 50  0001 C CNN "CPN"
+	1    2700 3500
 	0    1    1    0
 $EndComp
+Wire Wire Line
+	2500 3000 2500 3800
+Wire Wire Line
+	2150 3500 2550 3500
 $EndSCHEMATC
