File: i2c-gpio.sch (KiCad schematic (older format))
At the start: 3 parts, among them J1501 I2CGPIO1, J1502 I2CGPIO0, U1501 PCA9555PW

Commit message: Route rest of local I2C bus, GPIO expander
Parts:
- J1501, J1502: footprint Connector_PinHeader_2.54mm:PinHeader_1x10_P2.54mm_Vertical -> Connector_PinHeader_2.54mm:PinHeader_2x05_P2.54mm_Vertical_SMD
Changed lines of the file:
@@
 F 0 "J1502" H 7380 2842 50  0000 L CNN
 F 1 "I2CGPIO0" H 7380 2751 50  0000 L CNN
-F 2 "Connector_PinHeader_2.54mm:PinHeader_1x10_P2.54mm_Vertical" H 7300 2850 50  0001 C CNN
+F 2 "Connector_PinHeader_2.54mm:PinHeader_2x05_P2.54mm_Vertical_SMD" H 7300 2850 50  0001 C CNN
 F 3 "~" H 7300 2850 50  0001 C CNN
 	1    7300 2850
@@
 F 0 "J1501" H 6880 3742 50  0000 L CNN
 F 1 "I2CGPIO1" H 6880 3651 50  0000 L CNN
-F 2 "Connector_PinHeader_2.54mm:PinHeader_1x10_P2.54mm_Vertical" H 6800 3750 50  0001 C CNN
+F 2 "Connector_PinHeader_2.54mm:PinHeader_2x05_P2.54mm_Vertical_SMD" H 6800 3750 50  0001 C CNN
 F 3 "~" H 6800 3750 50  0001 C CNN
 	1    6800 3750

Commit message: MB: annotate everything with mfg/MPN
Parts:
- J1501, J1502: Mfg (none) -> Amphenol ICC; Mfg Part Num (none) -> 10129383-910001ALF
- U1501: Mfg (none) -> NXP; Mfg Part Num (none) -> PCA9555PW
Changed lines of the file:
@@
 F 2 "Package_SO:TSSOP-24_4.4x7.8mm_P0.65mm" H 5550 3350 50  0001 C CNN
 F 3 "https://www.nxp.com/docs/en/data-sheet/PCA9555.pdf" H 5550 3350 50  0001 C CNN
+F 4 "NXP" H 5550 3350 50  0001 C CNN "Mfg"
+F 5 "PCA9555PW" H 5550 3350 50  0001 C CNN "Mfg Part Num"
 	1    5550 3350
 	1    0    0    -1
@@
 F 2 "Connector_PinHeader_2.54mm:PinHeader_2x05_P2.54mm_Vertical_SMD" H 7300 2850 50  0001 C CNN
 F 3 "~" H 7300 2850 50  0001 C CNN
+F 4 "Amphenol ICC" H 7300 2850 50  0001 C CNN "Mfg"
+F 5 "10129383-910001ALF" H 7300 2850 50  0001 C CNN "Mfg Part Num"
 	1    7300 2850
 	1    0    0    -1
@@
 F 2 "Connector_PinHeader_2.54mm:PinHeader_2x05_P2.54mm_Vertical_SMD" H 6800 3750 50  0001 C CNN
 F 3 "~" H 6800 3750 50  0001 C CNN
+F 4 "Amphenol ICC" H 6800 3750 50  0001 C CNN "Mfg"
+F 5 "10129383-910001ALF" H 6800 3750 50  0001 C CNN "Mfg Part Num"
 	1    6800 3750
 	1    0    0    -1

Commit message: MB: add caps suggested in review
Parts:
- added C?: 0µ1, Capacitor_SMD:C_0603_1608Metric, symbol Device:C_Small
Connections:
- net +3V3: now also C?.1
- net GND: now also C?.2
Changed lines of the file:
@@
+	1    0    0    -1
+$EndComp
+$Comp
+L Device:C_Small C?
+U 1 1 5F6DEC9D
+P 4550 3450
+F 0 "C?" H 4642 3496 50  0000 L CNN
+F 1 "0µ1" H 4642 3405 50  0000 L CNN
+F 2 "Capacitor_SMD:C_0603_1608Metric" H 4550 3450 50  0001 C CNN
+F 3 "~" H 4550 3450 50  0001 C CNN
+F 4 "CL10B104KB8NNWC" H 4550 3450 50  0001 C CNN "Mfg Part Num"
+F 5 "Samsung Electro-Mechanics" H 4550 3450 50  0001 C CNN "Mfg"
+	1    4550 3450
+	1    0    0    -1
+$EndComp
+$Comp
+L power:+3V3 #PWR?
+U 1 1 5F6DEF02
+P 4550 3350
+F 0 "#PWR?" H 4550 3200 50  0001 C CNN
+F 1 "+3V3" H 4565 3523 50  0000 C CNN
+F 2 "" H 4550 3350 50  0001 C CNN
+F 3 "" H 4550 3350 50  0001 C CNN
+	1    4550 3350
+	1    0    0    -1
+$EndComp
+$Comp
+L power:GND #PWR?
+U 1 1 5F6DF3E1
+P 4550 3550
+F 0 "#PWR?" H 4550 3300 50  0001 C CNN
+F 1 "GND" H 4555 3377 50  0000 C CNN
+F 2 "" H 4550 3550 50  0001 C CNN
+F 3 "" H 4550 3550 50  0001 C CNN
+	1    4550 3550
 	1    0    0    -1
 $EndComp

Commit message: MB: finish routing
This finalizes layout and routing around the RoT carrier connector. I
have managed to avoid the layout gaffes that Mark pointed out in his
review -- clocks don't change layer, and when signals must change layer,
I put vias in the slower speed signals first.
Parts:
- gave numbers to parts that had none: 1
Changed lines of the file:
@@
 $EndComp
 $Comp
-L Device:C_Small C?
+L Device:C_Small C1501
 U 1 1 5F6DEC9D
 P 4550 3450
-F 0 "C?" H 4642 3496 50  0000 L CNN
+F 0 "C1501" H 4642 3496 50  0000 L CNN
 F 1 "0µ1" H 4642 3405 50  0000 L CNN
 F 2 "Capacitor_SMD:C_0603_1608Metric" H 4550 3450 50  0001 C CNN
@@
 $EndComp
 $Comp
-L power:+3V3 #PWR?
+L power:+3V3 #PWR0121
 U 1 1 5F6DEF02
 P 4550 3350
-F 0 "#PWR?" H 4550 3200 50  0001 C CNN
+F 0 "#PWR0121" H 4550 3200 50  0001 C CNN
 F 1 "+3V3" H 4565 3523 50  0000 C CNN
 F 2 "" H 4550 3350 50  0001 C CNN
@@
 $EndComp
 $Comp
-L power:GND #PWR?
+L power:GND #PWR0122
 U 1 1 5F6DF3E1
 P 4550 3550
-F 0 "#PWR?" H 4550 3300 50  0001 C CNN
+F 0 "#PWR0122" H 4550 3300 50  0001 C CNN
 F 1 "GND" H 4555 3377 50  0000 C CNN
 F 2 "" H 4550 3550 50  0001 C CNN

Commit message: gemini-bringup: Add CPNs for all components
Parts:
- C1501: CPN (none) -> 212-00011
- J1501, J1502: CPN (none) -> 215-00035
- U1501: CPN (none) -> 221-00023
Changed lines of the file:
@@
 F 4 "NXP" H 5550 3350 50  0001 C CNN "Mfg"
 F 5 "PCA9555PW" H 5550 3350 50  0001 C CNN "Mfg Part Num"
+F 6 "221-00023" H 5550 3350 50  0001 C CNN "CPN"
 	1    5550 3350
 	1    0    0    -1
@@
 F 4 "Amphenol ICC" H 7300 2850 50  0001 C CNN "Mfg"
 F 5 "10129383-910001ALF" H 7300 2850 50  0001 C CNN "Mfg Part Num"
+F 6 "215-00035" H 7300 2850 50  0001 C CNN "CPN"
 	1    7300 2850
 	1    0    0    -1
@@
 F 4 "Amphenol ICC" H 6800 3750 50  0001 C CNN "Mfg"
 F 5 "10129383-910001ALF" H 6800 3750 50  0001 C CNN "Mfg Part Num"
+F 6 "215-00035" H 6800 3750 50  0001 C CNN "CPN"
 	1    6800 3750
 	1    0    0    -1
@@
 F 4 "CL10B104KB8NNWC" H 4550 3450 50  0001 C CNN "Mfg Part Num"
 F 5 "Samsung Electro-Mechanics" H 4550 3450 50  0001 C CNN "Mfg"
+F 6 "212-00011" H 4550 3450 50  0001 C CNN "CPN"
 	1    4550 3450
 	1    0    0    -1

Commit message: i2c-gpio: specify rating constraints on passives
Parts:
- C1501: value 0µ1 -> 0.1uF 3.3VDCbias
Other:
- moved on the sheet: C1501
Changed lines of the file:
@@
 L Device:C_Small C1501
 U 1 1 5F6DEC9D
-P 4550 3450
-F 0 "C1501" H 4642 3496 50  0000 L CNN
-F 1 "0µ1" H 4642 3405 50  0000 L CNN
-F 2 "Capacitor_SMD:C_0603_1608Metric" H 4550 3450 50  0001 C CNN
-F 3 "~" H 4550 3450 50  0001 C CNN
-F 4 "CL10B104KB8NNWC" H 4550 3450 50  0001 C CNN "Mfg Part Num"
-F 5 "Samsung Electro-Mechanics" H 4550 3450 50  0001 C CNN "Mfg"
-F 6 "212-00011" H 4550 3450 50  0001 C CNN "CPN"
-	1    4550 3450
+P 4150 3450
+F 0 "C1501" H 4242 3496 50  0000 L CNN
+F 1 "0.1uF 3.3VDCbias" H 4242 3405 50  0000 L CNN
+F 2 "Capacitor_SMD:C_0603_1608Metric" H 4150 3450 50  0001 C CNN
+F 3 "~" H 4150 3450 50  0001 C CNN
+F 4 "CL10B104KB8NNWC" H 4150 3450 50  0001 C CNN "Mfg Part Num"
+F 5 "Samsung Electro-Mechanics" H 4150 3450 50  0001 C CNN "Mfg"
+F 6 "212-00011" H 4150 3450 50  0001 C CNN "CPN"
+	1    4150 3450
 	1    0    0    -1
 $EndComp
@@
 L power:+3V3 #PWR0121
 U 1 1 5F6DEF02
-P 4550 3350
-F 0 "#PWR0121" H 4550 3200 50  0001 C CNN
-F 1 "+3V3" H 4565 3523 50  0000 C CNN
-F 2 "" H 4550 3350 50  0001 C CNN
-F 3 "" H 4550 3350 50  0001 C CNN
-	1    4550 3350
+P 4150 3350
+F 0 "#PWR0121" H 4150 3200 50  0001 C CNN
+F 1 "+3V3" H 4165 3523 50  0000 C CNN
+F 2 "" H 4150 3350 50  0001 C CNN
+F 3 "" H 4150 3350 50  0001 C CNN
+	1    4150 3350
 	1    0    0    -1
 $EndComp
@@
 L power:GND #PWR0122
 U 1 1 5F6DF3E1
-P 4550 3550
-F 0 "#PWR0122" H 4550 3300 50  0001 C CNN
-F 1 "GND" H 4555 3377 50  0000 C CNN
-F 2 "" H 4550 3550 50  0001 C CNN
-F 3 "" H 4550 3550 50  0001 C CNN
-	1    4550 3550
+P 4150 3550
+F 0 "#PWR0122" H 4150 3300 50  0001 C CNN
+F 1 "GND" H 4155 3377 50  0000 C CNN
+F 2 "" H 4150 3550 50  0001 C CNN
+F 3 "" H 4150 3550 50  0001 C CNN
+	1    4150 3550
 	1    0    0    -1
 $EndComp

Commit message: gemini-bringup: custom fields for rating constraints on passives
Instead of packing tons of detail into a single "Value" field, limit
"Value" to the primary characteristic of the device (i.e. capacitance
for capacitors, resistance for resistors, current for fuses, impedence
at frequency for ferrite beads). For all other rating constraints, use
custom fields of the form <component-refdes-prefix>_<constraint>. For
example, R_P contains the power a resistor must dissipate.  Use
calculated values when possible rather than standard values as the
intent is to capture the constraint, not a specific device choice.
Parts:
- C1501: value 0.1uF 3.3VDCbias -> 0.1uF; C_Vbias (none) -> 3.3V
Other:
- moved on the sheet: C1501
Changed lines of the file:
@@
 L Device:C_Small C1501
 U 1 1 5F6DEC9D
-P 4150 3450
-F 0 "C1501" H 4242 3496 50  0000 L CNN
-F 1 "0.1uF 3.3VDCbias" H 4242 3405 50  0000 L CNN
-F 2 "Capacitor_SMD:C_0603_1608Metric" H 4150 3450 50  0001 C CNN
-F 3 "~" H 4150 3450 50  0001 C CNN
-F 4 "CL10B104KB8NNWC" H 4150 3450 50  0001 C CNN "Mfg Part Num"
-F 5 "Samsung Electro-Mechanics" H 4150 3450 50  0001 C CNN "Mfg"
-F 6 "212-00011" H 4150 3450 50  0001 C CNN "CPN"
-	1    4150 3450
+P 4550 3450
+F 0 "C1501" H 4642 3496 50  0000 L CNN
+F 1 "0.1uF" H 4642 3405 50  0000 L CNN
+F 2 "Capacitor_SMD:C_0603_1608Metric" H 4550 3450 50  0001 C CNN
+F 3 "~" H 4550 3450 50  0001 C CNN
+F 4 "CL10B104KB8NNWC" H 4550 3450 50  0001 C CNN "Mfg Part Num"
+F 5 "Samsung Electro-Mechanics" H 4550 3450 50  0001 C CNN "Mfg"
+F 6 "212-00011" H 4550 3450 50  0001 C CNN "CPN"
+F 7 "3.3V" H 4550 3450 50  0001 C CNN "C_Vbias"
+	1    4550 3450
 	1    0    0    -1
 $EndComp
@@
 L power:+3V3 #PWR0121
 U 1 1 5F6DEF02
-P 4150 3350
-F 0 "#PWR0121" H 4150 3200 50  0001 C CNN
-F 1 "+3V3" H 4165 3523 50  0000 C CNN
-F 2 "" H 4150 3350 50  0001 C CNN
-F 3 "" H 4150 3350 50  0001 C CNN
-	1    4150 3350
+P 4550 3350
+F 0 "#PWR0121" H 4550 3200 50  0001 C CNN
+F 1 "+3V3" H 4565 3523 50  0000 C CNN
+F 2 "" H 4550 3350 50  0001 C CNN
+F 3 "" H 4550 3350 50  0001 C CNN
+	1    4550 3350
 	1    0    0    -1
 $EndComp
@@
 L power:GND #PWR0122
 U 1 1 5F6DF3E1
-P 4150 3550
-F 0 "#PWR0122" H 4150 3300 50  0001 C CNN
-F 1 "GND" H 4155 3377 50  0000 C CNN
-F 2 "" H 4150 3550 50  0001 C CNN
-F 3 "" H 4150 3550 50  0001 C CNN
-	1    4150 3550
+P 4550 3550
+F 0 "#PWR0122" H 4550 3300 50  0001 C CNN
+F 1 "GND" H 4555 3377 50  0000 C CNN
+F 2 "" H 4550 3550 50  0001 C CNN
+F 3 "" H 4550 3550 50  0001 C CNN
+	1    4550 3550
 	1    0    0    -1
 $EndComp

Commit message: gemini-bringup: reselect all caps respecting C/V derating
Parts:
- C1501: Mfg Samsung Electro-Mechanics -> Kemet; Mfg Part Num CL10B104KB8NNWC -> C0603C104M4RACTU
Changed lines of the file:
@@
 F 2 "Capacitor_SMD:C_0603_1608Metric" H 4550 3450 50  0001 C CNN
 F 3 "~" H 4550 3450 50  0001 C CNN
-F 4 "CL10B104KB8NNWC" H 4550 3450 50  0001 C CNN "Mfg Part Num"
-F 5 "Samsung Electro-Mechanics" H 4550 3450 50  0001 C CNN "Mfg"
+F 4 "C0603C104M4RACTU" H 4550 3450 50  0001 C CNN "Mfg Part Num"
+F 5 "Kemet" H 4550 3450 50  0001 C CNN "Mfg"
 F 6 "212-00011" H 4550 3450 50  0001 C CNN "CPN"
 F 7 "3.3V" H 4550 3450 50  0001 C CNN "C_Vbias"
