File: i2c-gpio.sch (KiCad schematic (older format))
At the start: 4 parts, among them J1501 I2CGPIO1, J1502 I2CGPIO0, U1501 PCA9555PW

Commit message: Change column "Mfg Part Num" to "MPN" to align with manufacturer guidelines
Parts:
- C1501: MPN (none) -> C0603C104M4RACTU; Mfg Part Num C0603C104M4RACTU -> (none)
- J1501, J1502: MPN (none) -> 10129383-910001ALF; Mfg Part Num 10129383-910001ALF -> (none)
- U1501: MPN (none) -> PCA9555PW; Mfg Part Num PCA9555PW -> (none)
Changed lines of the file:
@@
 F 3 "https://www.nxp.com/docs/en/data-sheet/PCA9555.pdf" H 5550 3350 50  0001 C CNN
 F 4 "NXP" H 5550 3350 50  0001 C CNN "Mfg"
-F 5 "PCA9555PW" H 5550 3350 50  0001 C CNN "Mfg Part Num"
+F 5 "PCA9555PW" H 5550 3350 50  0001 C CNN "MPN"
 F 6 "221-00023" H 5550 3350 50  0001 C CNN "CPN"
 	1    5550 3350
@@
 F 3 "~" H 7300 2850 50  0001 C CNN
 F 4 "Amphenol ICC" H 7300 2850 50  0001 C CNN "Mfg"
-F 5 "10129383-910001ALF" H 7300 2850 50  0001 C CNN "Mfg Part Num"
+F 5 "10129383-910001ALF" H 7300 2850 50  0001 C CNN "MPN"
 F 6 "215-00035" H 7300 2850 50  0001 C CNN "CPN"
 	1    7300 2850
@@
 F 3 "~" H 6800 3750 50  0001 C CNN
 F 4 "Amphenol ICC" H 6800 3750 50  0001 C CNN "Mfg"
-F 5 "10129383-910001ALF" H 6800 3750 50  0001 C CNN "Mfg Part Num"
+F 5 "10129383-910001ALF" H 6800 3750 50  0001 C CNN "MPN"
 F 6 "215-00035" H 6800 3750 50  0001 C CNN "CPN"
 	1    6800 3750
@@
 F 2 "Capacitor_SMD:C_0603_1608Metric" H 4550 3450 50  0001 C CNN
 F 3 "~" H 4550 3450 50  0001 C CNN
-F 4 "C0603C104M4RACTU" H 4550 3450 50  0001 C CNN "Mfg Part Num"
+F 4 "C0603C104M4RACTU" H 4550 3450 50  0001 C CNN "MPN"
 F 5 "Kemet" H 4550 3450 50  0001 C CNN "Mfg"
 F 6 "212-00011" H 4550 3450 50  0001 C CNN "CPN"
