File: gimletlet.kicad_pcb (KiCad board)
At the start: 4 copper layers, 99.7 x 103.5 mm, 131 parts, among them J1 12V, J10 I2C3, J11 I2C4, J12 USART1, J13 USART2, J14 UART7, J15 SWD, J16 GPIO1, J17 Conn_01x07, J2 QSPI, J3 SPI3, J4 SPI4, J5 SPI6, J6 NIC, J7 12V, J8 3V3, J9 I2C2, SW1 RESET, U1 OKI-78SR-3.3_1.5-W36-C, U2 STM32H753ZITx, Y1 8MHz

Commit message: Add PNs to Gimletlet for easier Circuithub import (#39)
* Add PNs to Gimletlet for easier Circuithub import

* Move part-specific details to 'Comment' field for better import
Parts:
- J1: value 12V -> BarrelJack
- J10: value I2C3 -> Conn6x1
- J11: value I2C4 -> Conn6x1
- J12: value USART1 -> Conn6x1
- J13: value USART2 -> Conn6x1
- J14: value UART7 -> Conn6x1
- J16: value GPIO1 -> Conn9x1
- J2: value QSPI -> Conn6x2
- J3: value SPI3 -> Conn6x2
- J4: value SPI4 -> Conn6x2
- J5: value SPI6 -> Conn6x2
- J6: value NIC -> Conn41x2
- J7: value 12V -> Conn3x2
- J8: value 3V3 -> Conn3x2
- J9: value I2C2 -> Conn6x1
- JP1: value JACK -> Conn2x1
- JP2: value REG -> Conn2x1
- JP3: value ROM -> Conn2x1
- SW1: value RESET -> Button
- TP12, TP13, TP14, TP15, TP16, TP17, TP18, TP19, TP20, TP21, TP22, TP23: value GND -> TestPoint
