File: ignitionlet-config.sch (KiCad schematic (older format))
At the start: 23 parts

Commit message: Various, mostly documentation/style
Parts:
- gave numbers to parts that had none: 3
Changed lines of the file:
@@
 Sheet 3 3
 Title "Programming & Configuration"
-Date ""
-Rev ""
+Date "2021-06-17"
+Rev "1"
 Comp ""
 Comment1 ""
@@
 P 12100 5000
 AR Path="/6171A8C5" Ref="U?"  Part="3"
-AR Path="/61701F79/6171A8C5" Ref="U?"  Part="3"
-F 0 "U?" H 12100 5965 50  0000 C CNN
+AR Path="/61701F79/6171A8C5" Ref="U1"  Part="3"
+F 0 "U1" H 12100 5965 50  0000 C CNN
 F 1 "IGNITION001-QFN" H 12100 5874 50  0000 C CNN
 F 2 "" H 13000 6000 50  0001 C CNN
@@
 	10100 6600 10100 7100
 $Comp
-L Ignition:MT25QL128ABB8E12-0AUT U?
+L Ignition:MT25QL128ABB8E12-0AUT U5
 U 1 1 618573CD
 P 9200 6500
-F 0 "U?" H 9200 7065 50  0000 C CNN
+F 0 "U5" H 9200 7065 50  0000 C CNN
 F 1 "MT25QL128ABB8E12-0AUT" H 9200 6974 50  0000 C CNN
 F 2 "" H 9200 5800 50  0001 C CNN
@@
 	9700 6400 9900 6400
 $Comp
-L Ignition:AT25PE80-SSHN-B U?
+L Ignition:AT25PE80-SSHN-B U6
 U 1 1 618594E5
 P 9200 7800
-F 0 "U?" H 9200 8365 50  0000 C CNN
+F 0 "U6" H 9200 8365 50  0000 C CNN
 F 1 "AT25PE80-SSHN-B" H 9200 8274 50  0000 C CNN
 F 2 "" H 9200 7100 50  0001 C CNN

Commit message: Various
- Simplify power, assume always powered via barrel jack or J2
- Add operating mode descriptions
- Rename IGNITION_TARGET_HDR
- Small visual improvements
Parts:
- removed J?: IGNITION_HDR_TARGET, symbol Ignition:IGNITION_HDR_TARGET
- added J?: IGNITION_TARGET_HDR, symbol Ignition:IGNITION_TARGET_HDR
Connections:
- net labels removed: VIN_VBUS
- wire segments 138 -> 135
- no-connect marks 2 -> 3
Other:
- note added: "- FPGA as SPI master (default)\n\nThe default operating mode for this board is with the FPGA acting as SPI master.\nWithout anything driving SPI_SS this signal is pulled high. On init (after PoR\nor asserting CRESET) the FPGA will sample this pin. With the pin pulled high it\nwill resume its init sequence as SPI master. Consequently it will then assert\nSPI_SS and drive SPI_SCK, allowing it to re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"
- note added: "ColdBoot Header/Test Points"
- note added: "Header/Jumper/Test Points"
- note added: "If the SPI flash is programmed with an appropriate\nColdBoot applet these headers can be used to select\none of four bitstreams.\n\nSee Lattice FPGA-TN-02001-3.2 for details."
- note added: "Ignition Program/Debug Header"
- note added: "Intended for hacking and/or\nforced reset/write protect."
- note added: "Intended to allow a Gimletlet\nto program either SPI flash\nor the FPGA."
- note added: "Intended to make with Adafruit\nFT232H + adapter to allow\nsoftware compatibility with both\nLattice and open source\nprogramming tools.\n\nThe pinout is compatible with a\nstraight PMOD 2A connector to\nallow for alternative adapters if\ndesired.\n\nWhatever connects to this header\nis expected to bring slew limiting\nresistors."
- note added: "Operating Modes"
- note added: "PMOD 2A Peripheral (optional)"
- note removed: "Coldboot header/test points\n\nIf the SPI flash is programmed with an appropriate\nColdBoot applet these headers can be used to select\none of four bitstreams.\n\nSee Lattice FPGA-TN-02001-3.2 for details."
- note removed: "Header/jumper/testpoints\n\nIntended for hacking and/or\nforced reset/write protect."
- note removed: "Ignition Program/Debug Header\n\nIntended to make with Adafruit\nFT232H + adapter to allow\nsoftware compatibility with both\nLattice and open source\nprogramming tools.\n\nThe pinout is compatible with a\nstraight PMOD 2A connector to\nallow for alternative adapters if\ndesired.\n\nWhatever connects to this header\nis expected to bring slew limiting\nresistors."
- note removed: "PMOD 2A Peripheral (optional)\n\nIntended to allow a Gimletlet\nto program either SPI flash\nor the FPGA."
- moved on the sheet: C?, J?, R?, U1C, U5, U6

Commit message: LED picked, fixed cap/resistor values, make RX hackable, improve readability
Parts:
- added R?: 10K, Resistor_SMD:R_0603_1608Metric, symbol Device:R_Small_US
- R?: value 10K -> 100K
Connections:
- net labels added: FLASH_HOLD_L
- wire segments 135 -> 137
Other:
- note added: "Fit one of two SPI flash\noptions."
- note removed: "One of two SPI flash\noptions. Not intended\nto be fitted simultanously."
- moved on the sheet: C?, J?, R?, U1C, U5, U6

Commit message: Annotate schematic, pass ERC
Parts:
- gave numbers to parts that had none: 21
Connections:
- no-connect marks 3 -> 4
Other:
- moved on the sheet: J203, J204, J205, R208, R211, R212, R213, R214, U5, U6

Commit message: Make use of ~/_L more consistent
Connections:
- net FLASH_HOLD_L renamed ~FLASH_HOLD
- net FLASH_RESET_L renamed ~FLASH_RESET
- net FLASH_WP_L renamed ~FLASH_WP
- net FPGA_RESET_L renamed ~FPGA_RESET
Changed lines of the file:
@@
 CBSEL0
 Text Label 6600 7800 0    50   ~ 0
-FLASH_RESET_L
+~FLASH_RESET
 Text Label 6600 7700 0    50   ~ 0
-FPGA_RESET_L
+~FPGA_RESET
 Text Label 6600 7900 0    50   ~ 0
-FLASH_WP_L
+~FLASH_WP
 Wire Wire Line
 	12300 6400 12300 5200
@@
 	8100 4200 8400 4200
 Text Label 9700 6400 0    50   ~ 0
-FLASH_RESET_L
+~FLASH_RESET
 Text Label 9700 6500 0    50   ~ 0
 ~SPI_SS
@@
 SPI_SCK
 Text Label 9700 7800 0    50   ~ 0
-FLASH_HOLD_L
+~FLASH_HOLD
 Text Label 9700 7900 0    50   ~ 0
-FLASH_WP_L
+~FLASH_WP
 Wire Wire Line
 	9000 7900 12000 7900
@@
 NoConn ~ 6000 8000
 Text Label 9700 8700 0    50   ~ 0
-FLASH_WP_L
+~FLASH_WP
 Text Label 9700 8800 0    50   ~ 0
 SPI_SCK
@@
 ~SPI_SS
 Text Label 9700 8500 0    50   ~ 0
-FLASH_RESET_L
+~FLASH_RESET
 Wire Wire Line
 	8900 8700 10700 8700
