File: ignitionlet-config.sch (KiCad schematic (older format))
At the start: 24 parts, among them J201 PMOD_2A_PERIPHERAL, J202 IGNITION_TARGET_HDR, J203 Conn_02x04_Odd_Even, J204 Conn_01x03, J205 Conn_01x03, U1 IGNITION001-QFN, U5 MT25QL128ABB8E12-0AUT, U6 AT25PE80-SSHN-B

Commit message: Finish first pass of layout, lots of small fixes
Parts:
- added SW1: FPGA_RST, c-and-k-pts851:PTS815, symbol Switch:SW_Push
- J201: footprint (none) -> pmod:PMOD_12pin_peripheral_horizontal
- J202: footprint (none) -> samtec-tfc:TFC-105-02-F-D-A-K
- J203: footprint (none) -> Connector_PinHeader_2.54mm:PinHeader_2x04_P2.54mm_Vertical
- J204, J205: footprint (none) -> Connector_PinHeader_2.54mm:PinHeader_1x03_P2.54mm_Vertical
- U5: footprint (none) -> micron-sop2:Micron_SOP2-16_7.5x10.3mm_P1.27mm
- U6: footprint (none) -> Package_SO:SOIC-8_3.9x4.9mm_P1.27mm
Connections:
- net labels added: FLASH_DO
- wire segments 137 -> 141
Other:
- note added: "Intended to mate with Adafruit\nFT232H + adapter to allow\nsoftware compatibility with both\nLattice and open source\nprogramming tools.\n\nThe pinout is compatible with a\nstraight PMOD 2A connector to\nallow for alternative adapters if\ndesired.\n\nWhatever connects to this header\nis expected to bring slew limiting\nresistors."
- note removed: "Intended to make with Adafruit\nFT232H + adapter to allow\nsoftware compatibility with both\nLattice and open source\nprogramming tools.\n\nThe pinout is compatible with a\nstraight PMOD 2A connector to\nallow for alternative adapters if\ndesired.\n\nWhatever connects to this header\nis expected to bring slew limiting\nresistors."
Changed lines of the file:
@@
 L power:GND #PWR0152
 U 1 1 619276BD
-P 5900 8000
-F 0 "#PWR0152" H 5900 7750 50  0001 C CNN
-F 1 "GND" H 5905 7827 50  0000 C CNN
-F 2 "" H 5900 8000 50  0001 C CNN
-F 3 "" H 5900 8000 50  0001 C CNN
-	1    5900 8000
+P 5900 8500
+F 0 "#PWR0152" H 5900 8250 50  0001 C CNN
+F 1 "GND" H 5905 8327 50  0000 C CNN
+F 2 "" H 5900 8500 50  0001 C CNN
+F 3 "" H 5900 8500 50  0001 C CNN
+	1    5900 8500
 	1    0    0    -1
 $EndComp
@@
 	6000 7900 5900 7900
 Connection ~ 5900 7900
-Wire Wire Line
-	5900 7900 5900 8000
 Text Label 13900 7400 0    50   ~ 0
 CBSEL1
@@
 F 0 "J201" H 6200 4167 50  0000 C CNN
 F 1 "PMOD_2A_PERIPHERAL" H 6200 4076 50  0000 C CNN
-F 2 "" H 6200 3500 50  0001 C CNN
+F 2 "pmod:PMOD_12pin_peripheral_horizontal" H 6200 3500 50  0001 C CNN
 F 3 "https://www.digilentinc.com/Pmods/Digilent-Pmod_%20Interface_Specification.pdf" V 5850 2250 50  0001 C CNN
 	1    6200 3500
@@
 NoConn ~ 5700 3200
 NoConn ~ 5700 3100
-Text Label 10300 4700 0    50   ~ 0
+Text Label 9700 4700 0    50   ~ 0
 ~SPI_RESET
-Text Label 10300 4900 0    50   ~ 0
+Text Label 9700 4900 0    50   ~ 0
 SPI_SCK
-Text Label 10300 5000 0    50   ~ 0
+Text Label 9700 5000 0    50   ~ 0
 ~SPI_SS
-Text Label 10300 5100 0    50   ~ 0
+Text Label 9700 5100 0    50   ~ 0
 SPI_MISO
-Text Label 10300 5200 0    50   ~ 0
+Text Label 9700 5200 0    50   ~ 0
 SPI_MOSI
 Wire Notes Line
@@
 Intended for hacking and/or\nforced reset/write protect.
 Wire Notes Line
-	5500 6900 5500 8300
-Wire Notes Line
-	5500 8300 7400 8300
-Wire Notes Line
-	7400 8300 7400 6900
+	5500 6900 5500 8800
+Wire Notes Line
+	5500 8800 7400 8800
+Wire Notes Line
+	7400 8800 7400 6900
 Wire Notes Line
 	7400 6900 5500 6900
@@
 	5200 2300 5200 2400
 Text Notes 3700 5700 0    50   ~ 0
-Intended to make with Adafruit\nFT232H + adapter to allow\nsoftware compatibility with both\nLattice and open source\nprogramming tools.\n\nThe pinout is compatible with a\nstraight PMOD 2A connector to\nallow for alternative adapters if\ndesired.\n\nWhatever connects to this header\nis expected to bring slew limiting\nresistors.
+Intended to mate with Adafruit\nFT232H + adapter to allow\nsoftware compatibility with both\nLattice and open source\nprogramming tools.\n\nThe pinout is compatible with a\nstraight PMOD 2A connector to\nallow for alternative adapters if\ndesired.\n\nWhatever connects to this header\nis expected to bring slew limiting\nresistors.
 Wire Notes Line
 	3600 4300 3600 5800
@@
 F 0 "J203" H 6250 8117 50  0000 C CNN
 F 1 "Conn_02x04_Odd_Even" H 6250 8026 50  0000 C CNN
-F 2 "" H 6200 7800 50  0001 C CNN
+F 2 "Connector_PinHeader_2.54mm:PinHeader_2x04_P2.54mm_Vertical" H 6200 7800 50  0001 C CNN
 F 3 "~" H 6200 7800 50  0001 C CNN
 	1    6200 7800
@@
 F 0 "J204" H 13380 7442 50  0000 L CNN
 F 1 "Conn_01x03" H 13380 7351 50  0000 L CNN
-F 2 "" H 13300 7400 50  0001 C CNN
+F 2 "Connector_PinHeader_2.54mm:PinHeader_1x03_P2.54mm_Vertical" H 13300 7400 50  0001 C CNN
 F 3 "~" H 13300 7400 50  0001 C CNN
 	1    13300 7400
@@
 F 0 "J205" H 14580 7442 50  0000 L CNN
 F 1 "Conn_01x03" H 14580 7351 50  0000 L CNN
-F 2 "" H 14500 7400 50  0001 C CNN
+F 2 "Connector_PinHeader_2.54mm:PinHeader_1x03_P2.54mm_Vertical" H 14500 7400 50  0001 C CNN
 F 3 "~" H 14500 7400 50  0001 C CNN
 	1    14500 7400
@@
 F 0 "J202" H 6200 5767 50  0000 C CNN
 F 1 "IGNITION_TARGET_HDR" H 6200 5676 50  0000 C CNN
-F 2 "" H 6200 5100 50  0001 C CNN
-F 3 "" V 5850 3850 50  0001 C CNN
+F 2 "samtec-tfc:TFC-105-02-F-D-A-K" H 6200 5100 50  0001 C CNN
+F 3 "https://www.samtec.com/products/tfc-105-02-f-d-a-k" V 5850 3850 50  0001 C CNN
 	1    6200 5100
 	1    0    0    -1
@@
 	7400 4700 8100 4700
 Wire Wire Line
-	6500 7700 8100 7700
+	6500 7700 7200 7700
 Wire Wire Line
 	7200 5000 8700 5000
@@
 Wire Wire Line
 	9000 7900 12000 7900
-Text Label 11900 8600 0    50   ~ 0
-SPI_MISO
-Text Label 11900 8500 0    50   ~ 0
-SPI_MOSI
-Text Label 11900 6400 0    50   ~ 0
-SPI_MOSI
 NoConn ~ 6000 8000
 Text Label 9700 8700 0    50   ~ 0
@@
 F 0 "U6" H 11200 9165 50  0000 C CNN
 F 1 "AT25PE80-SSHN-B" H 11200 9074 50  0000 C CNN
-F 2 "" H 11200 7900 50  0001 C CNN
+F 2 "Package_SO:SOIC-8_3.9x4.9mm_P1.27mm" H 11200 7900 50  0001 C CNN
 F 3 "" H 11200 7800 50  0001 C CNN
 	1    11200 8600
@@
 Wire Wire Line
 	12400 6500 12400 5600
-Text Label 11900 6500 0    50   ~ 0
-SPI_MISO
 Connection ~ 12400 6500
 $Comp
@@
 F 0 "U5" H 11200 7675 50  0000 C CNN
 F 1 "MT25QL128ABB8E12-0AUT" H 11200 7575 50  0000 C CNN
-F 2 "" H 11200 6100 50  0001 C CNN
+F 2 "micron-sop2:Micron_SOP2-16_7.5x10.3mm_P1.27mm" H 11200 6100 50  0001 C CNN
 F 3 "" H 11200 5900 50  0001 C CNN
 	1    11200 6800
@@
 Wire Wire Line
 	11700 6500 12400 6500
+$Comp
+L Switch:SW_Push SW?
+U 1 1 60D8ACEC
+P 6300 8500
+AR Path="/60D8ACEC" Ref="SW?"  Part="1"
+AR Path="/61701F79/60D8ACEC" Ref="SW1"  Part="1"
+F 0 "SW1" H 6300 8785 50  0000 C CNN
+F 1 "FPGA_RST" H 6300 8694 50  0000 C CNN
+F 2 "c-and-k-pts851:PTS815" H 6300 8700 50  0001 C CNN
+F 3 "~" H 6300 8700 50  0001 C CNN
+	1    6300 8500
+	1    0    0    -1
+$EndComp
+Wire Wire Line
+	5900 8500 6100 8500
+Wire Wire Line
+	6500 8500 7200 8500
+Connection ~ 7200 7700
+Wire Wire Line
+	7200 7700 8100 7700
+Wire Wire Line
+	7200 8500 7200 7700
+Wire Wire Line
+	5900 7900 5900 8500
+Connection ~ 5900 8500
+Text Label 11900 8600 0    50   ~ 0
+FLASH_DO
+Text Label 11900 8500 0    50   ~ 0
+SPI_MOSI
+Text Label 11900 6500 0    50   ~ 0
+FLASH_DO
+Text Label 11900 6400 0    50   ~ 0
+SPI_MOSI
 $EndSCHEMATC

Commit message: Ignitionlet rev 2, first pass
Parts:
- removed J203: Conn_02x04_Odd_Even, Connector_PinHeader_2.54mm:PinHeader_2x04_P2.54mm_Vertical, symbol Connector_Generic:Conn_02x04_Odd_Even
- added C203, C204: GCM188R71E105KA64D, Capacitor_SMD:C_0603_1608Metric, symbol Ignition:GCM188R71E105KA64D
- added J203: Conn_02x05_Odd_Even, Connector_PinHeader_2.54mm:PinHeader_2x05_P2.54mm_Vertical, symbol Connector_Generic:Conn_02x05_Odd_Even
- added R215, R216, R217: 10K, Resistor_SMD:R_0603_1608Metric, symbol Device:R_Small_US
- added SW202: FLASH_RST, c-and-k-pts851:PTS815, symbol Switch:SW_Push
- added U7: SN74CBTLV3257RSV, Package_DFN_QFN_0x:Texas_RSV_S-UQFN-16_2.4x1.6mm, symbol Ignition:SN74CBTLV3257RSV
- added U8: SN74AUP1G08DBVR, Package_TO_SOT_SMD:SOT-23-5, symbol 74xGxx:74AUP1G08
- U5: footprint micron-sop2:Micron_SOP2-16_7.5x10.3mm_P1.27mm -> Package_BGA_0x:T-PBGA-24_6x8mm_Layout5x5_P1.0mm
- renumbered SW1 to SW201
Connections:
- net labels added: FLASH_HOLD_L, FLASH_MISO, FLASH_RESET_JP_L, FLASH_RESET_L, FLASH_WP_L, FPGA_CDONE, FPGA_MISO, FPGA_MODE, FPGA_MOSI, MUX_OE_L, SPI_RESET_L, SPI_SS_L
- net labels removed: CDONE, FLASH_DO, ~FLASH_HOLD, ~FLASH_RESET, ~FLASH_WP, ~FPGA_RESET, ~SPI_RESET, ~SPI_SS
- wire segments 141 -> 157
- no-connect marks 4 -> 8
Other:
- note added: "- FPGA as SPI Master (default)\n\nThe default operating mode for this board is with the FPGA acting as SPI master.\nWithout anything driving SPI_SS this signal is pulled high. On init (after PoR\nor asserting CRESET) the FPGA will sample this pin. With the pin pulled high it\nwill resume its init sequence as SPI master. Consequently it will then assert\nSPI_SS and drive SPI_SCK, allowing it to re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"
- note added: "- Program the FPGA SRAM from IGNITION_TARGET_HDR\n\nThe FTDI programmer can program the FPGA SRAM (or NVCM) directly if the user\ninstalls a jumper on the FPGA_MODE signal. This will cause the SPI flash to\nremain in reset and ignore any SPI traffic while mux beteen the header and FPGA\nSPI port will switch the SDO/SDI lines appropriately. The programmer then asserts\nSPI_SS while toggling SPI_RE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"
- note added: "1A\nSPI_MOSI\nSPI_MISO\n"
- note added: "2A\nSPI_MISO\nSPI_MOSI\n"
- note added: "FPGA SPI Mode MUX"
- note added: "FPGA_MODE\nH: SPI Master (default)\nL: SPI Slave"
- note added: "Header/Jumpers/Test Points"
- note added: "If the SPI flash is programmed with an appropriate\nColdBoot applet and the FPGA boots in SPI Master\nmode, these headers can be used to select one of\nfour bitstreams as defined in the applet.\n\nSee Lattice FPGA-TN-02001-3.2 for details."
- note added: "The SDI/SDO signals of the FPGA SPI port switch direction\ndepending on whether the FPGA acts as controller or\nperipheral. U7 handles this reversal of the signals allowing\nthe FPGA to be programmed by reading from the SPI flash,\nor by another controller. The logic is as follows:"
- note removed: "- FPGA as SPI master (default)\n\nThe default operating mode for this board is with the FPGA acting as SPI master.\nWithout anything driving SPI_SS this signal is pulled high. On init (after PoR\nor asserting CRESET) the FPGA will sample this pin. With the pin pulled high it\nwill resume its init sequence as SPI master. Consequently it will then assert\nSPI_SS and drive SPI_SCK, allowing it to re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"
- note removed: "Header/Jumper/Test Points"
- note removed: "If the SPI flash is programmed with an appropriate\nColdBoot applet these headers can be used to select\none of four bitstreams.\n\nSee Lattice FPGA-TN-02001-3.2 for details."
- moved on the sheet: C201, C202, J201, J202, J204, J205, R201, R202, R203, R204, R205, R206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
