File: ignitionlet-power.sch (KiCad schematic (older format))
At the start: 37 parts, among them J101 Barrel_Jack_MountingPin, J102 Conn_01x02, J103 Conn_01x03, U101 LT3013EFE#PBF, U102 LT3013EFE#PBF, U103 TPS7A0525PDBVR, U104 IGNITION001-QFN

Commit message: Finish first pass of layout, lots of small fixes
Parts:
- removed F101: Polyfuse_Small, symbol Device:Polyfuse_Small
- J101: footprint (none) -> Connector_BarrelJack:BarrelJack_Horizontal
- J102: footprint (none) -> Connector_PinHeader_2.54mm:PinHeader_1x02_P2.54mm_Vertical
- J103: footprint (none) -> Connector_PinHeader_2.54mm:PinHeader_1x03_P2.54mm_Vertical
- R101, R102, R103, R104, R105, R106: footprint (none) -> Resistor_SMD:R_0603_1608Metric
- U101, U102: footprint (none) -> Package_SO:TSSOP-16-1EP_4.4x5mm_P0.65mm
- renumbered U104 to U1
Connections:
- net labels added: VCCIO_3
- wire segments 185 -> 182
- no-connect marks 1 -> 3
Other:
- note added: "I_hold: 100mA\nI_trip: 300mA\n\nV_max: 30V\nI_max: 10A"
- moved on the sheet: J101, J102
Changed lines of the file:
@@
 F 0 "U102" H 7400 7765 50  0000 C CNN
 F 1 "LT3013EFE#PBF" H 7400 7674 50  0000 C CNN
-F 2 "" H 7400 6200 50  0001 C CNN
+F 2 "Package_SO:TSSOP-16-1EP_4.4x5mm_P0.65mm" H 7400 6200 50  0001 C CNN
 F 3 "https://www.analog.com/media/en/technical-documentation/data-sheets/3013fe.pdf" H 7400 6100 50  0001 C CNN
 	1    7400 6700
@@
 F 0 "U101" H 7400 5465 50  0000 C CNN
 F 1 "LT3013EFE#PBF" H 7400 5374 50  0000 C CNN
-F 2 "" H 7400 3900 50  0001 C CNN
+F 2 "Package_SO:TSSOP-16-1EP_4.4x5mm_P0.65mm" H 7400 3900 50  0001 C CNN
 F 3 "https://www.analog.com/media/en/technical-documentation/data-sheets/3013fe.pdf" H 7400 3800 50  0001 C CNN
 	1    7400 4400
@@
 $EndComp
 Wire Wire Line
-	13400 6800 13300 6800
-Wire Wire Line
-	13300 6800 13300 6900
-Wire Wire Line
 	13400 6900 13300 6900
-Connection ~ 13300 6900
 Wire Wire Line
 	13300 6900 13300 7000
@@
 F 0 "R103" H 8168 3891 50  0000 L CNN
 F 1 "1K" H 8168 3800 50  0000 L CNN
-F 2 "" H 8100 3800 50  0001 C CNN
+F 2 "Resistor_SMD:R_0603_1608Metric" H 8100 3800 50  0001 C CNN
 F 3 "~" H 8100 3800 50  0001 C CNN
 F 4 "1%" H 8168 3709 50  0000 L CNN "Tolerance"
@@
 F 0 "R104" H 8168 4291 50  0000 L CNN
 F 1 "147K" H 8168 4200 50  0000 L CNN
-F 2 "" H 8100 4200 50  0001 C CNN
+F 2 "Resistor_SMD:R_0603_1608Metric" H 8100 4200 50  0001 C CNN
 F 3 "~" H 8100 4200 50  0001 C CNN
 F 4 "1%" H 8168 4109 50  0000 L CNN "Tolerance"
@@
 F 0 "R102" H 6468 4191 50  0000 L CNN
 F 1 "100K" H 6468 4100 50  0000 L CNN
-F 2 "" H 6400 4100 50  0001 C CNN
+F 2 "Resistor_SMD:R_0603_1608Metric" H 6400 4100 50  0001 C CNN
 F 3 "~" H 6400 4100 50  0001 C CNN
 F 4 "1%" H 6468 4009 50  0000 L CNN "Tolerance"
@@
 F 0 "R105" H 8168 6191 50  0000 L CNN
 F 1 "147K" H 8168 6100 50  0000 L CNN
-F 2 "" H 8100 6100 50  0001 C CNN
+F 2 "Resistor_SMD:R_0603_1608Metric" H 8100 6100 50  0001 C CNN
 F 3 "~" H 8100 6100 50  0001 C CNN
 F 4 "1%" H 8168 6009 50  0000 L CNN "Tolerance"
@@
 F 0 "R106" H 8168 6591 50  0000 L CNN
 F 1 "88K7" H 8168 6500 50  0000 L CNN
-F 2 "" H 8100 6500 50  0001 C CNN
+F 2 "Resistor_SMD:R_0603_1608Metric" H 8100 6500 50  0001 C CNN
 F 3 "~" H 8100 6500 50  0001 C CNN
 F 4 "1%" H 8168 6409 50  0000 L CNN "Tolerance"
@@
 P 14200 5900
 AR Path="/6127169A" Ref="U?"  Part="2"
-AR Path="/61252D76/6127169A" Ref="U104"  Part="2"
-F 0 "U104" H 14100 7500 50  0000 L CNN
+AR Path="/61252D76/6127169A" Ref="U1"  Part="2"
+F 0 "U1" H 14100 7500 50  0000 L CNN
 F 1 "IGNITION001-QFN" H 13900 4400 50  0000 L CNN
 F 2 "" H 15100 6900 50  0001 C CNN
@@
 F 0 "J103" H 11318 5875 50  0000 C CNN
 F 1 "Conn_01x03" H 11318 5966 50  0000 C CNN
-F 2 "" H 11400 6200 50  0001 C CNN
+F 2 "Connector_PinHeader_2.54mm:PinHeader_1x03_P2.54mm_Vertical" H 11400 6200 50  0001 C CNN
 F 3 "~" H 11400 6200 50  0001 C CNN
 	1    11400 6200
@@
 F 0 "R101" H 5668 6491 50  0000 L CNN
 F 1 "100K" H 5668 6400 50  0000 L CNN
-F 2 "" H 5600 6400 50  0001 C CNN
+F 2 "Resistor_SMD:R_0603_1608Metric" H 5600 6400 50  0001 C CNN
 F 3 "~" H 5600 6400 50  0001 C CNN
 F 4 "1%" H 5668 6309 50  0000 L CNN "Tolerance"
@@
 2.5V: pins 1-2 \n3.3V: pins 2-3
 Wire Wire Line
-	2800 3800 2900 3800
+	2500 3800 2600 3800
 $Comp
 L power:GND #PWR?
 U 1 1 61E843B3
-P 2900 3800
+P 2600 3800
 AR Path="/61E843B3" Ref="#PWR?"  Part="1"
 AR Path="/61252D76/61E843B3" Ref="#PWR0147"  Part="1"
-F 0 "#PWR0147" H 2900 3550 50  0001 C CNN
-F 1 "GND" H 2905 3627 50  0000 C CNN
-F 2 "" H 2900 3800 50  0001 C CNN
-F 3 "" H 2900 3800 50  0001 C CNN
-	1    2900 3800
+F 0 "#PWR0147" H 2600 3550 50  0001 C CNN
+F 1 "GND" H 2605 3627 50  0000 C CNN
+F 2 "" H 2600 3800 50  0001 C CNN
+F 3 "" H 2600 3800 50  0001 C CNN
+	1    2600 3800
 	1    0    0    -1
 $EndComp
@@
 L Connector:Barrel_Jack_MountingPin J101
 U 1 1 61E83C2F
-P 2500 3700
-F 0 "J101" H 2557 4017 50  0000 C CNN
-F 1 "Barrel_Jack_MountingPin" H 2557 3926 50  0000 C CNN
-F 2 "" H 2550 3660 50  0001 C CNN
-F 3 "~" H 2550 3660 50  0001 C CNN
-	1    2500 3700
+P 2200 3700
+F 0 "J101" H 2257 4017 50  0000 C CNN
+F 1 "Barrel_Jack_MountingPin" H 2257 3926 50  0000 C CNN
+F 2 "Connector_BarrelJack:BarrelJack_Horizontal" H 2250 3660 50  0001 C CNN
+F 3 "~" H 2250 3660 50  0001 C CNN
+	1    2200 3700
 	1    0    0    -1
 $EndComp
@@
 VIN_12V
 $Comp
-L Device:Polyfuse_Small F101
-U 1 1 61EAD4BD
-P 3900 3600
-F 0 "F101" V 3695 3600 50  0000 C CNN
-F 1 "Polyfuse_Small" V 3786 3600 50  0000 C CNN
-F 2 "" H 3950 3400 50  0001 L CNN
-F 3 "~" H 3900 3600 50  0001 C CNN
-	1    3900 3600
-	0    1    1    0
-$EndComp
-Wire Wire Line
-	4000 3600 4400 3600
-$Comp
 L power:PWR_FLAG #FLG0101
 U 1 1 61F2FBE3
@@
 	1    0    0    -1
 $EndComp
-Text Notes 2100 4400 0    50   ~ 0
+Text Notes 1800 4400 0    50   ~ 0
 The Fake Bus Bar can take 5-12V from the barrel jack\nor J2 can be used to injecting 12V from the Gimletlet\nusing short Dupont wires. This allows both boards to\nbe powered by a single supply.
 Text Notes 2100 3200 0    50   ~ 10
 Fake Bus Bar
 Wire Notes Line
-	2000 3000 2000 4500
+	1700 3000 1700 4500
 Wire Notes Line
-	2000 4500 5400 4500
+	1700 4500 5400 4500
 Wire Notes Line
 	5400 4500 5400 3000
 Wire Notes Line
-	5400 3000 2000 3000
+	5400 3000 1700 3000
 Text Notes 8600 4700 0    50   ~ 0
 The number of input/output capacitors was copied from\nthe Gimlet implementation, which assumes a 54V input\nvoltage. Given a smaller difference between VIN of this\nboard and the output less may be required. The footprints\nare here to adjust/fix if needed.
@@
 L Connector_Generic:Conn_01x02 J102
 U 1 1 60DD6D36
-P 3600 3700
-F 0 "J102" H 3680 3692 50  0000 L CNN
-F 1 "Conn_01x02" H 3680 3601 50  0000 L CNN
-F 2 "" H 3600 3700 50  0001 C CNN
-F 3 "~" H 3600 3700 50  0001 C CNN
-	1    3600 3700
-	1    0    0    -1
-$EndComp
-Wire Wire Line
-	3400 3800 3300 3800
-Connection ~ 2900 3800
-Wire Wire Line
-	3400 3700 3400 3600
-Wire Wire Line
-	2800 3600 3400 3600
-Wire Wire Line
-	3400 3600 3800 3600
-Connection ~ 3400 3600
+P 3300 3700
+F 0 "J102" H 3380 3692 50  0000 L CNN
+F 1 "Conn_01x02" H 3380 3601 50  0000 L CNN
+F 2 "Connector_PinHeader_2.54mm:PinHeader_1x02_P2.54mm_Vertical" H 3300 3700 50  0001 C CNN
+F 3 "~" H 3300 3700 50  0001 C CNN
+	1    3300 3700
+	1    0    0    -1
+$EndComp
+Wire Wire Line
+	3100 3800 3000 3800
+Connection ~ 2600 3800
+Wire Wire Line
+	3100 3700 3100 3600
+Wire Wire Line
+	2500 3600 3100 3600
+Connection ~ 3100 3600
 Wire Wire Line
 	7800 8500 8100 8500
@@
 L power:PWR_FLAG #FLG0103
 U 1 1 61AA36E8
-P 3300 3800
-F 0 "#FLG0103" H 3300 3875 50  0001 C CNN
-F 1 "PWR_FLAG" H 3300 3973 50  0000 C CNN
-F 2 "" H 3300 3800 50  0001 C CNN
-F 3 "~" H 3300 3800 50  0001 C CNN
-	1    3300 3800
+P 3000 3800
+F 0 "#FLG0103" H 3000 3875 50  0001 C CNN
+F 1 "PWR_FLAG" H 3000 3973 50  0000 C CNN
+F 2 "" H 3000 3800 50  0001 C CNN
+F 3 "~" H 3000 3800 50  0001 C CNN
+	1    3000 3800
 	-1   0    0    1
 $EndComp
-Connection ~ 3300 3800
-Wire Wire Line
-	3300 3800 2900 3800
-NoConn ~ 2500 4000
+Connection ~ 3000 3800
+Wire Wire Line
+	3000 3800 2600 3800
+NoConn ~ 2200 4000
 Connection ~ 9300 3600
+NoConn ~ 13400 6800
+NoConn ~ 13600 8200
+Text Notes 4300 4300 0    50   ~ 0
+I_hold: 100mA\nI_trip: 300mA\n\nV_max: 30V\nI_max: 10A
+Text Label 12200 6200 0    50   ~ 0
+VCCIO_3
+Wire Wire Line
+	3100 3600 4400 3600
 $EndSCHEMATC

Commit message: Add chokes on TX SerDes
Changed lines of the file:
@@
 L Ignition:VIN_12V #PWR0148
 U 1 1 61E4983E
-P 4400 3600
-F 0 "#PWR0148" H 4400 3450 50  0001 C CNN
-F 1 "VIN_12V" H 4400 3800 50  0000 C CNN
-F 2 "" H 4400 3600 50  0001 C CNN
-F 3 "" H 4400 3600 50  0001 C CNN
-	1    4400 3600
+P 4000 3600
+F 0 "#PWR0148" H 4000 3450 50  0001 C CNN
+F 1 "VIN_12V" H 4000 3800 50  0000 C CNN
+F 2 "" H 4000 3600 50  0001 C CNN
+F 3 "" H 4000 3600 50  0001 C CNN
+	1    4000 3600
 	1    0    0    -1
 $EndComp
-Text Label 4900 3600 0    50   ~ 0
+Text Label 4800 3600 0    50   ~ 0
 VIN_12V
 $Comp
 L power:PWR_FLAG #FLG0101
 U 1 1 61F2FBE3
-P 4800 3600
-F 0 "#FLG0101" H 4800 3675 50  0001 C CNN
-F 1 "PWR_FLAG" H 4800 3773 50  0000 C CNN
-F 2 "" H 4800 3600 50  0001 C CNN
-F 3 "~" H 4800 3600 50  0001 C CNN
-	1    4800 3600
+P 4600 3600
+F 0 "#FLG0101" H 4600 3675 50  0001 C CNN
+F 1 "PWR_FLAG" H 4600 3773 50  0000 C CNN
+F 2 "" H 4600 3600 50  0001 C CNN
+F 3 "~" H 4600 3600 50  0001 C CNN
+	1    4600 3600
 	1    0    0    -1
 $EndComp
@@
 Connection ~ 6800 5100
 Wire Wire Line
-	5200 3600 4800 3600
+	5200 3600 4600 3600
 Connection ~ 5200 3600
-Connection ~ 4400 3600
-Connection ~ 4800 3600
+Connection ~ 4000 3600
+Connection ~ 4600 3600
 Wire Wire Line
-	4800 3600 4400 3600
+	4600 3600 4000 3600
 $Comp
 L power:PWR_FLAG #FLG0102
@@
 VCCIO_3
 Wire Wire Line
-	3100 3600 4400 3600
+	3100 3600 4000 3600
 $EndSCHEMATC

Commit message: Add TPs, routing tweaks, stitch top ground, add CMD1 LED
Parts:
- added TP101, TP102, TP103: TestPoint, TestPoint:TestPoint_THTPad_D1.0mm_Drill0.5mm, symbol Connector:TestPoint
- added TP104, TP105: TestPoint, TestPoint:TestPoint_Keystone_5015_Micro-Minature, symbol Connector:TestPoint
Connections:
- net GND: now also TP104.1, TP105.1
- net V1P2: now also TP101.1
- net V2P5: now also TP103.1
- net V3P3: now also TP102.1
Other:
- note added: "Keystone 5015s for easier probe access."
Changed lines of the file:
@@
 Sheet 2 3
 Title "Power"
-Date "2021-07-01"
+Date "2021-07-02"
 Rev "1"
 Comp ""
@@
 P 11800 4500
 AR Path="/61271727" Ref="#PWR?"  Part="1"
-AR Path="/61252D76/61271727" Ref="#PWR0121"  Part="1"
-F 0 "#PWR0121" H 11800 4350 50  0001 C CNN
+AR Path="/61252D76/61271727" Ref="#PWR0165"  Part="1"
+F 0 "#PWR0165" H 11800 4350 50  0001 C CNN
 F 1 "V1P2" H 11800 4675 50  0000 C CNN
 F 2 "" H 11800 4500 50  0001 C CNN
@@
 Connection ~ 3100 3600
 Wire Wire Line
-	7800 8500 8100 8500
+	7800 8500 7900 8500
 Connection ~ 8100 8500
 Wire Wire Line
-	8500 5900 8900 5900
-Wire Wire Line
-	8500 3600 8900 3600
+	8500 5900 8700 5900
+Wire Wire Line
+	8500 3600 8700 3600
 Wire Wire Line
 	6900 5100 6800 5100
@@
 Wire Wire Line
 	3100 3600 4000 3600
+$Comp
+L Connector:TestPoint TP101
+U 1 1 61D4307F
+P 8700 3600
+F 0 "TP101" H 8643 3672 50  0000 R CNN
+F 1 "TestPoint" H 8758 3627 50  0001 L CNN
+F 2 "TestPoint:TestPoint_THTPad_D1.0mm_Drill0.5mm" H 8900 3600 50  0001 C CNN
+F 3 "~" H 8900 3600 50  0001 C CNN
+	1    8700 3600
+	1    0    0    -1
+$EndComp
+Connection ~ 8700 3600
+Wire Wire Line
+	8700 3600 8900 3600
+$Comp
+L Connector:TestPoint TP102
+U 1 1 61D43B3D
+P 8700 5900
+F 0 "TP102" H 8643 5972 50  0000 R CNN
+F 1 "TestPoint" H 8758 5927 50  0001 L CNN
+F 2 "TestPoint:TestPoint_THTPad_D1.0mm_Drill0.5mm" H 8900 5900 50  0001 C CNN
+F 3 "~" H 8900 5900 50  0001 C CNN
+	1    8700 5900
+	1    0    0    -1
+$EndComp
+Connection ~ 8700 5900
+Wire Wire Line
+	8700 5900 8900 5900
+$Comp
+L Connector:TestPoint TP103
+U 1 1 61D46D51
+P 7900 8500
+F 0 "TP103" H 7750 8750 50  0000 L CNN
+F 1 "TestPoint" H 7958 8527 50  0001 L CNN
+F 2 "TestPoint:TestPoint_THTPad_D1.0mm_Drill0.5mm" H 8100 8500 50  0001 C CNN
+F 3 "~" H 8100 8500 50  0001 C CNN
+	1    7900 8500
+	1    0    0    -1
+$EndComp
+Connection ~ 7900 8500
+Wire Wire Line
+	7900 8500 8100 8500
+$Comp
+L Connector:TestPoint TP104
+U 1 1 61D47B76
+P 8700 7750
+F 0 "TP104" H 8700 7983 50  0000 C CNN
+F 1 "TestPoint" H 8758 7777 50  0001 L CNN
+F 2 "TestPoint:TestPoint_Keystone_5015_Micro-Minature" H 8900 7750 50  0001 C CNN
+F 3 "~" H 8900 7750 50  0001 C CNN
+	1    8700 7750
+	1    0    0    -1
+$EndComp
+$Comp
+L power:GND #PWR?
+U 1 1 61D4831A
+P 8700 7750
+AR Path="/61D4831A" Ref="#PWR?"  Part="1"
+AR Path="/61252D76/61D4831A" Ref="#PWR05"  Part="1"
+F 0 "#PWR05" H 8700 7500 50  0001 C CNN
+F 1 "GND" H 8705 7577 50  0000 C CNN
+F 2 "" H 8700 7750 50  0001 C CNN
+F 3 "" H 8700 7750 50  0001 C CNN
+	1    8700 7750
+	1    0    0    -1
+$EndComp
+$Comp
+L Connector:TestPoint TP105
+U 1 1 61D64422
+P 9000 7750
+F 0 "TP105" H 9000 7983 50  0000 C CNN
+F 1 "TestPoint" H 9058 7777 50  0001 L CNN
+F 2 "TestPoint:TestPoint_Keystone_5015_Micro-Minature" H 9200 7750 50  0001 C CNN
+F 3 "~" H 9200 7750 50  0001 C CNN
+	1    9000 7750
+	1    0    0    -1
+$EndComp
+$Comp
+L power:GND #PWR?
+U 1 1 61D64428
+P 9000 7750
+AR Path="/61D64428" Ref="#PWR?"  Part="1"
+AR Path="/61252D76/61D64428" Ref="#PWR0164"  Part="1"
+F 0 "#PWR0164" H 9000 7500 50  0001 C CNN
+F 1 "GND" H 9005 7577 50  0000 C CNN
+F 2 "" H 9000 7750 50  0001 C CNN
+F 3 "" H 9000 7750 50  0001 C CNN
+	1    9000 7750
+	1    0    0    -1
+$EndComp
+Text Notes 8600 8100 0    50   ~ 0
+Keystone 5015s for easier probe access.
 $EndSCHEMATC

Commit message: Ignitionlet rev 2, first pass
Parts:
- TP103: footprint TestPoint:TestPoint_THTPad_D1.0mm_Drill0.5mm -> test-point:TestPoint_Pad_D0.6mm
Changed lines of the file:
@@
 Sheet 2 3
 Title "Power"
-Date "2021-07-02"
-Rev "1"
+Date "2021-07-21"
+Rev "2"
 Comp ""
 Comment1 ""
@@
 L Ignition:V3P3 #PWR?
 U 1 1 6127172E
-P 11900 5400
+P 11700 5400
 AR Path="/6127172E" Ref="#PWR?"  Part="1"
 AR Path="/61252D76/6127172E" Ref="#PWR0123"  Part="1"
-F 0 "#PWR0123" H 11900 5250 50  0001 C CNN
-F 1 "V3P3" H 11915 5573 50  0000 C CNN
-F 2 "" H 11900 5400 50  0001 C CNN
-F 3 "" H 11900 5400 50  0001 C CNN
-	1    11900 5400
+F 0 "#PWR0123" H 11700 5250 50  0001 C CNN
+F 1 "V3P3" H 11715 5573 50  0000 C CNN
+F 2 "" H 11700 5400 50  0001 C CNN
+F 3 "" H 11700 5400 50  0001 C CNN
+	1    11700 5400
 	1    0    0    -1
 $EndComp
@@
 U 1 1 61D74AC0
 P 11400 6200
-F 0 "J103" H 11318 5875 50  0000 C CNN
-F 1 "Conn_01x03" H 11318 5966 50  0000 C CNN
+F 0 "J103" H 11400 5850 50  0000 C CNN
+F 1 "Conn_01x03" H 11400 5950 50  0000 C CNN
 F 2 "Connector_PinHeader_2.54mm:PinHeader_1x03_P2.54mm_Vertical" H 11400 6200 50  0001 C CNN
 F 3 "~" H 11400 6200 50  0001 C CNN
@@
 $EndComp
 Wire Wire Line
-	11600 6100 11900 6100
-Wire Wire Line
-	11900 6100 11900 5400
-Wire Wire Line
-	11900 5400 12200 5400
-Connection ~ 11900 5400
-Wire Wire Line
-	11600 6200 12600 6200
+	11600 6100 11700 6100
+Wire Wire Line
+	11700 6100 11700 5400
+Wire Wire Line
+	11700 5400 12200 5400
+Connection ~ 11700 5400
+Wire Wire Line
+	11600 6200 11900 6200
 Wire Wire Line
 	11600 6300 11700 6300
@@
 Wire Wire Line
 	13000 6600 13000 6700
-$Comp
-L Ignition:V2P5 #PWR?
-U 1 1 61271789
-P 11900 6500
-AR Path="/61271789" Ref="#PWR?"  Part="1"
-AR Path="/61252D76/61271789" Ref="#PWR0124"  Part="1"
-F 0 "#PWR0124" H 11900 6350 50  0001 C CNN
-F 1 "V2P5" H 11900 6675 50  0000 C CNN
-F 2 "" H 11900 6500 50  0001 C CNN
-F 3 "" H 11900 6500 50  0001 C CNN
-	1    11900 6500
-	1    0    0    -1
-$EndComp
 Wire Wire Line
 	11900 6500 12200 6500
@@
 Connection ~ 13000 6300
 Wire Notes Line
-	10500 5150 12100 5150
+	10400 5150 12100 5150
 Wire Notes Line
 	12100 5150 12100 6600
 Wire Notes Line
-	12100 6600 10500 6600
+	12100 6600 10400 6600
 Wire Notes Line
-	10500 6600 10500 5150
-Text Notes 10600 5800 0    50   ~ 0
+	10400 6600 10400 5150
+Text Notes 10500 5800 0    50   ~ 0
 JP3 allows VCCIO_3 to be\nconfigurable as 2.5V/3.3V.\n\nIf configured as 3.3V the\nLVDS TX resistors need\nto be adjusted for compliant\ndiff swing.
 Wire Wire Line
@@
 	5200 3600 5600 3600
 Connection ~ 6000 5900
-Text Notes 10600 6200 0    50   ~ 0
+Text Notes 10500 6200 0    50   ~ 0
 2.5V: pins 1-2 \n3.3V: pins 2-3
 Wire Wire Line
@@
 Text Notes 4300 4300 0    50   ~ 0
 I_hold: 100mA\nI_trip: 300mA\n\nV_max: 30V\nI_max: 10A
-Text Label 12200 6200 0    50   ~ 0
-VCCIO_3
 Wire Wire Line
 	3100 3600 4000 3600
@@
 F 0 "TP103" H 7750 8750 50  0000 L CNN
 F 1 "TestPoint" H 7958 8527 50  0001 L CNN
-F 2 "TestPoint:TestPoint_THTPad_D1.0mm_Drill0.5mm" H 8100 8500 50  0001 C CNN
+F 2 "test-point:TestPoint_Pad_D0.6mm" H 8100 8500 50  0001 C CNN
 F 3 "~" H 8100 8500 50  0001 C CNN
 	1    7900 8500
@@
 Text Notes 8600 8100 0    50   ~ 0
 Keystone 5015s for easier probe access.
+$Comp
+L Ignition:VCCIO_3 #PWR0103
+U 1 1 6113E3B2
+P 11900 6200
+F 0 "#PWR0103" H 11900 6050 50  0001 C CNN
+F 1 "VCCIO_3" H 11900 6350 50  0000 C CNN
+F 2 "" H 11900 6200 50  0001 C CNN
+F 3 "" H 11900 6200 50  0001 C CNN
+	1    11900 6200
+	1    0    0    -1
+$EndComp
+Connection ~ 11900 6200
+Wire Wire Line
+	11900 6200 12600 6200
+$Comp
+L Ignition:V2P5 #PWR?
+U 1 1 61271789
+P 11900 6500
+AR Path="/61271789" Ref="#PWR?"  Part="1"
+AR Path="/61252D76/61271789" Ref="#PWR0124"  Part="1"
+F 0 "#PWR0124" H 11900 6350 50  0001 C CNN
+F 1 "V2P5" H 11900 6675 50  0000 C CNN
+F 2 "" H 11900 6500 50  0001 C CNN
+F 3 "" H 11900 6500 50  0001 C CNN
+	1    11900 6500
+	1    0    0    -1
+$EndComp
 $EndSCHEMATC
