File: ignitionlet.sch (KiCad schematic (older format))
At the start: 25 parts

Commit message: Implement most of the board
Parts:
- removed C?: C_Small, symbol Device:C_Small
- removed C? (x8): C0603C106M8PACTU, Capacitor_SMD:C_0603_1608Metric, symbol Ignition:C0603C106M8PACTU
- removed C? (x4): GRM21BR61E106KA73K, Capacitor_SMD:C_0805_2012Metric, symbol Ignition:GRM21BR61E106KA73K
- removed R?: 1K, symbol Device:R_Small_US
- removed R? (x2): 147K, symbol Device:R_Small_US
- removed R? (x2): 100K, symbol Device:R_Small_US
- removed R?: 88K7, symbol Device:R_Small_US
- removed U? (x2): IGNITION001-QFN, symbol Ignition:IGNITION001-QFN
- removed U? (x2): LT3013EFE#PBF, symbol Ignition:LT3013EFE#PBF
- removed U?: TPS7A0525PDBVR, Package_TO_SOT_SMD:SOT-23-5, symbol Ignition:TPS7A0525PDBVR
- added C? (x7): GCM188R71E105KA64D, Capacitor_SMD:C_0603_1608Metric, symbol Ignition:GCM188R71E105KA64D
- added D?: LED, symbol Device:LED
- added J? (x2): Conn_02x06_Odd_Even, symbol Connector_Generic:Conn_02x06_Odd_Even
- added J?: Conn_01x04, symbol Connector_Generic:Conn_01x04
- added R? (x18): 10K, Resistor_SMD:R_0603_1608Metric, symbol Device:R_Small_US
- added R? (x4): 50, Resistor_SMD:R_0603_1608Metric, symbol Device:R_Small_US
- added R? (x4): 150, Resistor_SMD:R_0603_1608Metric, symbol Device:R_Small_US
- added R? (x2): 140, Resistor_SMD:R_0603_1608Metric, symbol Device:R_Small_US
- added SW?: SYS_RST, symbol Switch:SW_Push
- added SW?: FLT, symbol Switch:SW_Push
- added U?: AMPMGFB-50.0000T, symbol Ignition:AMPMGFB-50.0000T
Connections:
- net labels added: CMD1, CMD2, ID0, ID1, ID2, ID3, ID4, ID5, PWR_EN_L, PWR_FLT0_L, PWR_FLT1_L, PWR_FLT2_L, PWR_FLT3_L, PWR_FLT4_L, ROT_FLT_L, SYS_RST_L, V2P5
- net labels removed: PGOOD_V1P2, PGOOD_V3P3
- wire segments 106 -> 183
Other:
- note added: "CMD Bits Header"
- note added: "Command bits are exposed on a header\nfor easy test probing and alternative\nprototyping."
- note added: "Fault Pin Straps"
- note added: "Fault pin straps allow setting fixed fault values. The switch\nattached to ROT_FLT provides a convenient way to cause\nfault interrupts during integration tests. The header allows\nreuse of these pins for alternative prototyping."
- note added: "ID Straps"
- note added: "ID straps allow setting the desired value. The header\nallows reuse of these pins for alternative prototyping\n\nSee RFD 142 for currently allocated ID values."
- note added: "Power"
- note added: "Power Enable LED"
- note added: "Programming & Configuration"
- note added: "TODO: pick LED and limit resisitor"
- note added: "TODO:\n\n- SMA connectors\n- Explain TX resistor values"
- moved on the sheet: U?A

Commit message: Various, mostly documentation/style
Parts:
- added J? (x8): Conn_Coaxial, symbol Connector:Conn_Coaxial
- added J? (x2): Conn_01x04, symbol Connector_Generic:Conn_01x04
- added R? (x4): 75, Resistor_SMD:R_0603_1608Metric, symbol Device:R_Small_US
- R? (x4): value 150 -> 75
- gave numbers to parts that had none: 1
Connections:
- net labels added: AUX0_RX_N, AUX0_TX_P, AUX1_TX_N, AUX1_TX_P
- wire segments 183 -> 209
Other:
- note added: "Ignition Target"
- note added: "LVDS TX"
- note added: "TODO:\n\n- Document program/configuration modes\n- Rework AUX_RX for alternative prototyping\n- Pick LED and limit resisitor"
- note added: "The LVDS transmitter pair is implemented as per Lattice\nFPGA-TN-1253 using PIO pin pairs in Bank 3. The resistor\nvalues above were derived using the equations on p. 4\nand the following assumptions:\n\nZ0 = 50 ohm\nVCCIO = 2.5V\nV_OD = 0.35V\nR_OUTPUT = 30 ohm\n\nR_P = 2 * ((Z0 * VCCIO) / (VCCIO - (2 * V_OD)))\n = 2 * (165 / 1.8)\n = 139 ohm\n\nR_S = ((Z0 * R_P / 2) / ((R_P / 2) - Z0) - R_OUTPU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"
- note removed: "TODO: pick LED and limit resisitor"
- note removed: "TODO:\n\n- SMA connectors\n- Explain TX resistor values"
- moved on the sheet: C?, R?, SW?, U1A, U?

Commit message: Various
- Simplify power, assume always powered via barrel jack or J2
- Add operating mode descriptions
- Rename IGNITION_TARGET_HDR
- Small visual improvements
Other:
- note added: "TODO:\n\n- Rework AUX_RX for alternative prototyping\n- Pick LED and limit resisitor"
- note removed: "TODO:\n\n- Document program/configuration modes\n- Rework AUX_RX for alternative prototyping\n- Pick LED and limit resisitor"
Changed lines of the file:
@@
 Sheet 1 3
 Title "Ignition Application"
-Date "2021-06-17"
+Date "2021-06-18"
 Rev "1"
 Comp ""
@@
 $EndDescr
 $Sheet
-S 11300 7200 2300 2500
+S 11300 7200 2200 2500
 U 61252D76
 F0 "Power" 50
@@
 $EndComp
 $Sheet
-S 13800 7200 2100 2500
+S 13700 7200 2200 2500
 U 61701F79
 F0 "Config" 50
@@
 	15900 700  15900 7000
 Wire Notes Line
-	13700 5400 13700 7000
-Text Notes 12300 8500 0    79   ~ 16
+	13600 5400 13600 7000
+Text Notes 12200 8500 0    79   ~ 16
 Power
-Text Notes 13950 8500 0    79   ~ 16
+Text Notes 13900 8500 0    79   ~ 16
 Programming & Configuration
 Text Notes 8400 9500 0    50   ~ 0
@@
 $EndComp
 Text Notes 2000 7700 0    50   ~ 10
-TODO:\n\n- Document program/configuration modes\n- Rework AUX_RX for alternative prototyping\n- Pick LED and limit resisitor
+TODO:\n\n- Rework AUX_RX for alternative prototyping\n- Pick LED and limit resisitor
 Text Notes 1450 2450 0    79   ~ 16
 Ignition Target
@@
 Wire Wire Line
 	5600 4700 6100 4700
+Text Notes 11400 3400 0    79   ~ 16
+ID Straps
+Wire Wire Line
+	8400 4400 8400 4900
+Wire Wire Line
+	8400 3400 8400 3900
+Wire Wire Line
+	10700 3600 10700 4100
+Wire Wire Line
+	10700 4600 10700 5100
+Connection ~ 10700 4600
+Wire Wire Line
+	9800 4700 9800 4900
+Wire Wire Line
+	9800 3400 9800 3600
 $Comp
 L Ignition:IGNITION001-QFN U1
@@
 	1    0    0    -1
 $EndComp
-Text Notes 11400 3400 0    79   ~ 16
-ID Straps
-Wire Wire Line
-	8400 4400 8400 4900
-Wire Wire Line
-	8400 3400 8400 3900
-Wire Wire Line
-	10700 3600 10700 4100
-Wire Wire Line
-	10700 4600 10700 5100
-Connection ~ 10700 4600
-Wire Wire Line
-	9800 4700 9800 4900
-Wire Wire Line
-	9800 3400 9800 3600
 $EndSCHEMATC

Commit message: LED picked, fixed cap/resistor values, make RX hackable, improve readability
Parts:
- removed D?: LED, symbol Device:LED
- added C? (x4): GCM188R71E105KA64D, Capacitor_SMD:C_0603_1608Metric, symbol Ignition:GCM188R71E105KA64D
- added D?: LTST-C193KGKT-5A, symbol Ignition:LTST-C193KGKT-5A
- added J? (x2): Conn_01x04, symbol Connector_Generic:Conn_01x04
- added R? (x4): 0, Resistor_SMD:R_0603_1608Metric, symbol Device:R_Small_US
- R?: value 10K -> 280
Connections:
- net labels added: AUX0_RX_P, AUX0_RX_TAP_N, AUX0_RX_TAP_P, AUX0_TX_LVDS_N, AUX0_TX_LVDS_P, AUX0_TX_TAP_P, AUX1_RX_N, AUX1_RX_P, AUX1_RX_TAP_N, AUX1_RX_TAP_P, AUX1_TX_LVDS_N, AUX1_TX_LVDS_P, AUX1_TX_TAP_N, AUX1_TX_TAP_P, PWR_EN
- net labels removed: PWR_EN_L
- wire segments 209 -> 224
Other:
- note added: "If: 5mA\nVf: 1.9V\nRlim: 280ohm"
- note added: "LVDS RX"
- note added: "TODO:\n\n- Check TX/RX caps\n- Add TPs, mounting holes, fiducials, logo, P/N, S/N “parts”"
- note added: "The LVDS transmitter pair is implemented as per Lattice FPGA-TN-1253 using\nPIO pin pairs in Bank 3. The iCE40 inputs expect a proper LVDS signal so the\ninputs are biased after the AC-coupling cap. Resistor and capacitor values can\nbe tuned where required.\n\nAn optional header footprint/via is placed near the SMA connector allowing\nalternate prototyping, either using either single-ended or di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"
- note added: "The LVDS transmitter pair is implemented as per Lattice FPGA-TN-1253\nusing PIO pin pairs in Bank 3. The resistor values above were derived\nusing the equations on p. 4 and the following assumptions:\n\nZ0 = 50 ohm\nVCCIO = 2.5V\nV_OD = 0.35V\nR_OUTPUT = 30 ohm\n\nR_P = 2 * ((Z0 * VCCIO) / (VCCIO - (2 * V_OD)))\n = 2 * (165 / 1.8)\n = 139 ohm\n\nR_S = ((Z0 * R_P / 2) / ((R_P / 2) - Z0) - R_OUTPUT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"
- note removed: "TODO:\n\n- Rework AUX_RX for alternative prototyping\n- Pick LED and limit resisitor"
- note removed: "The LVDS transmitter pair is implemented as per Lattice\nFPGA-TN-1253 using PIO pin pairs in Bank 3. The resistor\nvalues above were derived using the equations on p. 4\nand the following assumptions:\n\nZ0 = 50 ohm\nVCCIO = 2.5V\nV_OD = 0.35V\nR_OUTPUT = 30 ohm\n\nR_P = 2 * ((Z0 * VCCIO) / (VCCIO - (2 * V_OD)))\n = 2 * (165 / 1.8)\n = 139 ohm\n\nR_S = ((Z0 * R_P / 2) / ((R_P / 2) - Z0) - R_OUTPU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"
- moved on the sheet: C?, J?, R?, SW?, U1A, U?

Commit message: Documentation fixes, add TODOs
Other:
- note added: "TODO:\n\n- Check TX/RX cap values againt bit rate\n- Add TPs, mounting holes, fiducials, logo, P/N, S/N “parts”"
- note added: "The LVDS transmitter pair is implemented as per Lattice FPGA-TN-1253 using\nPIO pin pairs in Bank 3. The iCE40 inputs expect a proper LVDS signal so the\ninputs are biased after the AC-coupling cap. Resistor and capacitor values can\nbe tuned where required.\n\nAn optional header footprint/via is placed near the SMA connector to allow for\nalternate prototyping, using either single-ended or diffe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"
- note removed: "TODO:\n\n- Check TX/RX caps\n- Add TPs, mounting holes, fiducials, logo, P/N, S/N “parts”"
- note removed: "The LVDS transmitter pair is implemented as per Lattice FPGA-TN-1253 using\nPIO pin pairs in Bank 3. The iCE40 inputs expect a proper LVDS signal so the\ninputs are biased after the AC-coupling cap. Resistor and capacitor values can\nbe tuned where required.\n\nAn optional header footprint/via is placed near the SMA connector allowing\nalternate prototyping, either using either single-ended or di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"
Changed lines of the file:
@@
 	8000 2400 11100 2400
 Wire Notes Line
-	11100 9300 11100 2400
+	11100 9700 11100 2400
 Wire Notes Line
-	8000 9300 11100 9300
+	8000 9700 11100 9700
 Wire Notes Line
-	8000 2400 8000 9300
+	8000 2400 8000 9700
 Wire Wire Line
 	8100 3300 8300 3300
@@
 $EndComp
 Text Notes 1000 10600 0    50   ~ 10
-TODO:\n\n- Check TX/RX caps\n- Add TPs, mounting holes, fiducials, logo, P/N, S/N “parts”
+TODO:\n\n- Check TX/RX cap values againt bit rate\n- Add TPs, mounting holes, fiducials, logo, P/N, S/N “parts”
 Text Notes 800  2200 0    79   ~ 16
 Ignition Target
@@
 	700  2400 700  8000
 Text Notes 800  7900 0    50   ~ 0
-The LVDS transmitter pair is implemented as per Lattice FPGA-TN-1253 using\nPIO pin pairs in Bank 3. The iCE40 inputs expect a proper LVDS signal so the\ninputs are biased after the AC-coupling cap. Resistor and capacitor values can\nbe tuned where required.\n\nAn optional header footprint/via is placed near the SMA connector allowing\nalternate prototyping, either using either single-ended or differential\nsignaling. The zero ohm resistor pads can be used for termination or slew\nlimiting resistors if desired.
+The LVDS transmitter pair is implemented as per Lattice FPGA-TN-1253 using\nPIO pin pairs in Bank 3. The iCE40 inputs expect a proper LVDS signal so the\ninputs are biased after the AC-coupling cap. Resistor and capacitor values can\nbe tuned where required.\n\nAn optional header footprint/via is placed near the SMA connector to allow for\nalternate prototyping, using either single-ended or differential signaling. The\nzero ohm resistor footprint can be used for termination or slew limiting\nresistors if desired.
 Wire Notes Line
 	4000 2400 4000 8000
@@
 Wire Wire Line
 	10400 5000 10500 5000
-Text Notes 8100 9200 0    50   ~ 0
-The LVDS transmitter pair is implemented as per Lattice FPGA-TN-1253\nusing PIO pin pairs in Bank 3. The resistor values above were derived\nusing the equations on p. 4 and the following assumptions:\n\nZ0 = 50 ohm\nVCCIO = 2.5V\nV_OD = 0.35V\nR_OUTPUT = 30 ohm\n\nR_P = 2 * ((Z0 * VCCIO) / (VCCIO - (2 * V_OD)))\n     = 2 * (165 / 1.8)\n     = 139 ohm\n\nR_S = ((Z0 * R_P / 2) / ((R_P / 2) - Z0) - R_OUTPUT\n     = (3472 / 19) - 30\n     = 149 ohm\n\nThe series resistor is broken into two pieces of 75 ohm each. The intend\nhere is that one pin of a 100 mil header/ footprint is inserted between the\ntwo resistors. If done using a tight layout this via should add minimal\ndisruption at the edge rates of these transmitters.\n\nInserting the via would allow for IO pin to be reused for alternative\nprototyping by not fitting the second series resistor, parallel resistor and\nSMA connector, while using the first resistor footprint as slew limiting\nresistor or for series termination.\n\nOne possible application of this alternative scheme is to allow the Ignition\nprotocol to be carried using single ended LVCMOS signaling at 3.3V\nbetween this broad and an ECP5 dev board without requiring SMA\nconnectors for the link partner. This would simplify initial prototyping work.
+Text Notes 8100 9600 0    50   ~ 0
+The LVDS transmitter pair is implemented as per Lattice FPGA-TN-1253\nusing PIO pin pairs in Bank 3. The resistor values above were derived\nusing the equations on p. 4 and the following assumptions:\n\nZ0 = 50 ohm\nVCCIO = 2.5V\nV_OD = 0.35V\nR_OUTPUT = 30 ohm\n\nR_P = 2 * ((Z0 * VCCIO) / (VCCIO - (2 * V_OD)))\n     = 2 * (165 / 1.8)\n     = 139 ohm\n\nR_S = ((Z0 * R_P / 2) / ((R_P / 2) - Z0) - R_OUTPUT\n     = (3472 / 19) - 30\n     = 149 ohm\n\nThe series resistor is broken into two pieces of 75 ohm each. The intend\nhere is that one pin of a 100 mil header/ footprint is inserted between the\ntwo resistors. If done using a tight layout this via should add minimal\ndisruption at the edge rates of these transmitters.\n\nInserting the via would allow for IO pin to be reused for alternative\nprototyping by not fitting the second series resistor, parallel resistor and\nSMA connector, while using the first resistor footprint as slew limiting\nresistor or for series termination.\n\nOne possible application of this alternative scheme is to allow the Ignition\nprotocol to be carried using single ended LVCMOS signaling at 3.3V\nbetween this broad and an ECP5 dev board without requiring SMA\nconnectors for the link partner. This would simplify initial prototyping work.\n\nThe AC couping capacitors near the SMA connector are optional in case\none wants to experiment. The layout should allow for some copper nearby\nconnected to ground so experiments with a choke are possible. If not in\nuse 0 ohm resistors should be fitted.
 $EndSCHEMATC

Commit message: Annotate schematic, pass ERC
Parts:
- gave numbers to parts that had none: 66
Connections:
- wire segments 224 -> 223
Other:
- note added: "If: 5mA\nVf: 1.9V\nRlim: 280Ω"
- note removed: "If: 5mA\nVf: 1.9V\nRlim: 280ohm"

Commit message: Make use of ~/_L more consistent
Connections:
- net labels added: ~PWR_FLT0, ~PWR_FLT1, ~PWR_FLT2, ~PWR_FLT3, ~PWR_FLT4, ~ROT_FLT, ~SYS_RST
- net labels removed: PWR_FLT0_L, PWR_FLT1_L, PWR_FLT2_L, PWR_FLT3_L, PWR_FLT4_L, ROT_FLT_L, SYS_RST_L
Changed lines of the file:
@@
 	11600 2200 11600 2300
 Text Label 12500 2200 0    50   ~ 0
-ROT_FLT_L
+~ROT_FLT
 Text Label 12500 2100 0    50   ~ 0
-PWR_FLT4_L
+~PWR_FLT4
 Text Label 12500 2000 0    50   ~ 0
-PWR_FLT3_L
+~PWR_FLT3
 Text Label 12500 1900 0    50   ~ 0
-PWR_FLT2_L
+~PWR_FLT2
 Text Label 12500 1800 0    50   ~ 0
-PWR_FLT1_L
+~PWR_FLT1
 Text Label 12500 1700 0    50   ~ 0
-PWR_FLT0_L
+~PWR_FLT0
 Wire Wire Line
 	12400 2200 15000 2200
@@
 $EndComp
 Text Label 5300 5500 0    50   ~ 0
-SYS_RST_L
+~SYS_RST
 Text Label 5300 5800 0    50   ~ 0
 ID0
@@
 $EndComp
 Text Label 5300 4700 0    50   ~ 0
-PWR_FLT0_L
+~PWR_FLT0
 Text Label 5300 4800 0    50   ~ 0
-PWR_FLT1_L
+~PWR_FLT1
 Text Label 5300 4900 0    50   ~ 0
-PWR_FLT2_L
+~PWR_FLT2
 Text Label 5300 5000 0    50   ~ 0
-PWR_FLT3_L
+~PWR_FLT3
 Text Label 5300 5100 0    50   ~ 0
-PWR_FLT4_L
+~PWR_FLT4
 Text Label 5300 5200 0    50   ~ 0
-ROT_FLT_L
+~ROT_FLT
 Wire Wire Line
 	5300 5200 5800 5200
