File: ignitionlet.sch (KiCad schematic (older format))
At the start: 67 parts, among them J1 Conn_Coaxial, J10 Conn_Coaxial, J11 Conn_Coaxial, J12 Conn_Coaxial, J13 Conn_02x06_Odd_Even, J14 Conn_02x06_Odd_Even, J15 Conn_01x04, J2 Conn_Coaxial, J3 Conn_Coaxial, J4 Conn_Coaxial, J5 Conn_01x04, J6 Conn_01x04, J7 Conn_01x04, J8 Conn_01x04, J9 Conn_Coaxial, SW1 SYS_RST, SW2 FLT, U1 IGNITION001-QFN, U2 AMPMGFB-50.0000T

Commit message: Finish first pass of layout, lots of small fixes
Parts:
- added FID1: IGNITIONLET, grumpy:Oxide_Board_Identifier_23x6mm, symbol Mechanical:Fiducial
- added FID2: Fiducial, Fiducial:Fiducial_1mm_Mask2mm, symbol Mechanical:Fiducial
- added H1, H2, H3, H4: MountingHole_Pad, MountingHole:MountingHole_3.2mm_M3_Pad_Via, symbol Mechanical:MountingHole_Pad
- added J16: Conn_02x06_Top_Bottom, pmod:PMOD_12pin_peripheral_horizontal, symbol Connector_Generic:Conn_02x06_Top_Bottom
- D1: footprint (none) -> LED_SMD:LED_0603_1608Metric
- J1, J11, J2, J3, J4, J9: footprint (none) -> Connector_Coaxial:SMA_Amphenol_132134-16_Vertical
- J10: renamed from J12; footprint (none) -> Connector_Coaxial:SMA_Amphenol_132134-16_Vertical
- J12: renamed from J10; footprint (none) -> Connector_Coaxial:SMA_Amphenol_132134-16_Vertical
- J13, J14: footprint (none) -> Connector_PinHeader_2.54mm:PinHeader_2x06_P2.54mm_Vertical
- J15: footprint (none) -> Connector_PinHeader_2.54mm:PinHeader_1x04_P2.54mm_Vertical
- J5, J6, J7, J8: footprint (none) -> Connector_PinHeader_2.54mm:PinHeader_1x04_P2.54mm_Vertical_SMD_Pin1Left
- SW2: renamed from SW1; footprint (none) -> c-and-k-pts851:PTS815
- SW3: renamed from SW2; footprint (none) -> c-and-k-pts851:PTS815
- U1: footprint (none) -> lattice-drqfn84:Lattice_DRQFN-84-1EP_7x7mm_P0.50mm_EP3.5x3.5mm_ThermalVias
- U2: footprint (none) -> Package_LGA_ABRACON:ABRACON_VFLGA-4_1.6x1.2mm
- renumbered C11 to C10, C10 to C11, R17 to R16, R16 to R17
Connections:
- net labels added: AUX0_TX_N, AUX0_TX_TAP_N, CLK_50M
- wire segments 223 -> 228
- no-connect marks 0 -> 10
Other:
- note added: "Mechanical"
- note added: "TODO:\n\n- Check TX/RX cap values againt bit rate"
- note added: "The board assumes the width of two standard\n0.80” PMOD boards. J16 is present only for\nadditional mechanical stability, but can be used\nfor prototyping."
- note removed: "TODO:\n\n- Check TX/RX cap values againt bit rate\n- Add TPs, mounting holes, fiducials, logo, P/N, S/N “parts”"
- moved on the sheet: C7, J15, U2

Commit message: Simplify copper pours, improve silkscreen, small fixes/improvements
Parts:
- FID1: value IGNITIONLET -> Ignitionlet
Other:
- note added: "TODO:\n\n- Check TX/RX cap values againt bit rate\n- Add chokes on SerDes"
- note removed: "TODO:\n\n- Check TX/RX cap values againt bit rate"
Changed lines of the file:
@@
 Sheet 1 3
 Title "Ignition Target"
-Date "2021-06-21"
+Date "2021-07-01"
 Rev "1"
-Comp ""
+Comp "Oxide Computer Co."
 Comment1 ""
 Comment2 ""
@@
 	-1   0    0    -1
 $EndComp
-Text Notes 9200 10600 0    50   ~ 10
-TODO:\n\n- Check TX/RX cap values againt bit rate
+Text Notes 5100 8000 0    50   ~ 10
+TODO:\n\n- Check TX/RX cap values againt bit rate\n- Add chokes on SerDes
 Text Notes 800  2200 0    79   ~ 16
 Ignition Target
@@
 P 3200 8700
 F 0 "FID1" H 3285 8746 50  0000 L CNN
-F 1 "IGNITIONLET" H 3285 8655 50  0000 L CNN
+F 1 "Ignitionlet" H 3285 8655 50  0000 L CNN
 F 2 "grumpy:Oxide_Board_Identifier_23x6mm" H 3200 8700 50  0001 C CNN
 F 3 "~" H 3200 8700 50  0001 C CNN
@@
 Text Notes 800  8300 0    79   ~ 16
 Mechanical
-Text Notes 2100 9800 0    50   ~ 0
+Text Notes 1900 9800 0    50   ~ 0
 The board assumes the width of two standard\n0.80” PMOD boards. J16 is present only for\nadditional mechanical stability, but can be used\nfor prototyping.
 NoConn ~ 2200 8700
@@
 Text Label 8500 6000 0    50   ~ 0
 AUX1_TX_TAP_N
+Wire Notes Line
+	700  8100 4000 8100
+Wire Notes Line
+	4000 8100 4000 10000
+Wire Notes Line
+	4000 10000 700  10000
+Wire Notes Line
+	700  10000 700  8100
 $EndSCHEMATC

Commit message: Add chokes on TX SerDes
Parts:
- added L1, L2: MCZ1210AH900L2TA0G, passives:L_Choke_MCZ1210AH, symbol Ignition:MCZ1210AH900L2TA0G
Connections:
- wire segments 228 -> 236
Other:
- note added: "TODO:\n\n- Check TX/RX cap values againt bit rate"
- note added: "The LVDS transmitter pair is implemented as per Lattice FPGA-TN-1253 using\nPIO pin pairs in Bank 3. The iCE40 inputs expect a proper LVDS signal so the\ninputs are biased after the AC-coupling cap. Resistor and capacitor values\ncan be tuned where required.\n\nAn optional header footprint/via is placed near the SMA connector to allow for\nalternate prototyping, using either single-ended or diffe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"
- note removed: "TODO:\n\n- Check TX/RX cap values againt bit rate\n- Add chokes on SerDes"
- note removed: "The LVDS transmitter pair is implemented as per Lattice FPGA-TN-1253 using\nPIO pin pairs in Bank 3. The iCE40 inputs expect a proper LVDS signal so the\ninputs are biased after the AC-coupling cap. Resistor and capacitor values can\nbe tuned where required.\n\nAn optional header footprint/via is placed near the SMA connector to allow for\nalternate prototyping, using either single-ended or diffe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"
- moved on the sheet: C1, C10, C11, C2, C3, C4, C5, C6, C7, C8, C9, D1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

Commit message: Add TPs, routing tweaks, stitch top ground, add CMD1 LED
Parts:
- added D2: LTST-C193KGKT-5A, LED_SMD:LED_0603_1608Metric, symbol Ignition:LTST-C193KGKT-5A
- added R37: 280, Resistor_SMD:R_0603_1608Metric, symbol Device:R_Small_US
- added TP1, TP2: TestPoint, test-point:TestPoint_THTPad_D0.6mm_Drill0.3mm, symbol Connector:TestPoint
Connections:
- wire segments 236 -> 241
Other:
- note added: "CMDx LEDs"
- note removed: "Power Enable LED"
Changed lines of the file:
@@
 Sheet 1 3
 Title "Ignition Target"
-Date "2021-07-01"
+Date "2021-07-02"
 Rev "1"
 Comp "Oxide Computer Co."
@@
 Wire Notes Line
 	11400 600  16000 600
-Text Notes 13900 5500 0    79   ~ 16
-Power Enable LED
 Text Notes 11500 5500 0    79   ~ 16
 CMD Bits Header
@@
 Connection ~ 4000 3300
 Wire Wire Line
-	4000 3300 4500 3300
+	4000 3300 4200 3300
 Wire Wire Line
 	5500 3100 5500 3300
@@
 	4000 2800 4400 2800
 Connection ~ 4000 2800
-Text Label 5200 3100 0    50   ~ 0
+Text Label 5100 3100 0    50   ~ 0
 CLK_50M
 $Comp
@@
 Wire Notes Line
 	11400 600  11400 9400
+Connection ~ 5500 3100
+$Comp
+L Connector:TestPoint TP1
+U 1 1 61CD52A4
+P 5500 3100
+F 0 "TP1" H 5558 3218 50  0000 L CNN
+F 1 "TestPoint" H 5558 3127 50  0000 L CNN
+F 2 "test-point:TestPoint_THTPad_D0.6mm_Drill0.3mm" H 5700 3100 50  0001 C CNN
+F 3 "~" H 5700 3100 50  0001 C CNN
+	1    5500 3100
+	1    0    0    -1
+$EndComp
+$Comp
+L Connector:TestPoint TP2
+U 1 1 61CF29FF
+P 4200 3300
+F 0 "TP2" H 4150 3400 50  0000 R CNN
+F 1 "TestPoint" H 4150 3500 50  0000 R CNN
+F 2 "test-point:TestPoint_THTPad_D0.6mm_Drill0.3mm" H 4400 3300 50  0001 C CNN
+F 3 "~" H 4400 3300 50  0001 C CNN
+	1    4200 3300
+	-1   0    0    1
+$EndComp
+Connection ~ 4200 3300
+Wire Wire Line
+	4200 3300 4500 3300
+Wire Wire Line
+	14700 6450 14750 6450
+Wire Wire Line
+	15100 6450 15100 6550
+Wire Wire Line
+	15050 6450 15100 6450
+$Comp
+L power:GND #PWR0121
+U 1 1 61D8CF1B
+P 15100 6550
+F 0 "#PWR0121" H 15100 6300 50  0001 C CNN
+F 1 "GND" H 15105 6377 50  0000 C CNN
+F 2 "" H 15100 6550 50  0001 C CNN
+F 3 "" H 15100 6550 50  0001 C CNN
+	1    15100 6550
+	1    0    0    -1
+$EndComp
+Wire Wire Line
+	14000 6450 14500 6450
+$Comp
+L Device:R_Small_US R37
+U 1 1 61D8CF23
+P 14600 6450
+F 0 "R37" V 14700 6450 50  0000 C CNN
+F 1 "280" V 14800 6450 50  0000 C CNN
+F 2 "Resistor_SMD:R_0603_1608Metric" H 14600 6450 50  0001 C CNN
+F 3 "~" H 14600 6450 50  0001 C CNN
+F 4 "1%" H 14668 6359 50  0001 L CNN "Tolerance"
+	1    14600 6450
+	0    1    1    0
+$EndComp
+Text Label 14000 6450 0    50   ~ 0
+CMD1
+$Comp
+L Ignition:LTST-C193KGKT-5A D2
+U 1 1 61D8CF2A
+P 14900 6450
+F 0 "D2" H 14893 6195 50  0000 C CNN
+F 1 "LTST-C193KGKT-5A" H 14893 6286 50  0000 C CNN
+F 2 "LED_SMD:LED_0603_1608Metric" H 14900 6450 50  0001 C CNN
+F 3 "~" H 14900 6450 50  0001 C CNN
+	1    14900 6450
+	-1   0    0    1
+$EndComp
+Text Notes 13900 5500 0    79   ~ 16
+CMDx LEDs
 $EndSCHEMATC

Commit message: Extend J16 to allow Type 1 GPIO interface
Parts:
- added J17: Conn_01x04, Connector_PinHeader_2.54mm:PinHeader_1x04_P2.54mm_Vertical, symbol Connector_Generic:Conn_01x04
Connections:
- wire segments 241 -> 245
- no-connect marks 10 -> 6
Other:
- note added: "The board assumes the width of two standard\n0.80” PMOD boards. J16 is intended for additional\nmechanical stability, but is connected to J17 as a\nType 1 interface, providing GPIOs for prototyping\nwhich for example can be wired to CDONE or\nFLASH_RESET when connected to an appropriate\nhost board."
- note removed: "The board assumes the width of two standard\n0.80” PMOD boards. J16 is present only for\nadditional mechanical stability, but can be used\nfor prototyping."
- moved on the sheet: FID1, FID2, H1, H2, H3, H4, J16
Changed lines of the file:
@@
 L Mechanical:MountingHole_Pad H1
 U 1 1 61186B02
-P 900 8300
-F 0 "H1" V 854 8450 50  0000 L CNN
-F 1 "MountingHole_Pad" V 945 8450 50  0000 L CNN
-F 2 "MountingHole:MountingHole_3.2mm_M3_Pad_Via" H 900 8300 50  0001 C CNN
-F 3 "~" H 900 8300 50  0001 C CNN
-	1    900  8300
+P 900 9500
+F 0 "H1" V 854 9650 50  0000 L CNN
+F 1 "MountingHole_Pad" V 945 9650 50  0000 L CNN
+F 2 "MountingHole:MountingHole_3.2mm_M3_Pad_Via" H 900 9500 50  0001 C CNN
+F 3 "~" H 900 9500 50  0001 C CNN
+	1    900  9500
 	0    1    1    0
 $EndComp
@@
 L Mechanical:MountingHole_Pad H2
 U 1 1 61197EFF
-P 900 8500
-F 0 "H2" V 854 8650 50  0000 L CNN
-F 1 "MountingHole_Pad" V 945 8650 50  0000 L CNN
-F 2 "MountingHole:MountingHole_3.2mm_M3_Pad_Via" H 900 8500 50  0001 C CNN
-F 3 "~" H 900 8500 50  0001 C CNN
-	1    900  8500
+P 900 9700
+F 0 "H2" V 854 9850 50  0000 L CNN
+F 1 "MountingHole_Pad" V 945 9850 50  0000 L CNN
+F 2 "MountingHole:MountingHole_3.2mm_M3_Pad_Via" H 900 9700 50  0001 C CNN
+F 3 "~" H 900 9700 50  0001 C CNN
+	1    900  9700
 	0    1    1    0
 $EndComp
@@
 L Mechanical:MountingHole_Pad H3
 U 1 1 611C8D25
-P 900 8700
-F 0 "H3" V 854 8850 50  0000 L CNN
-F 1 "MountingHole_Pad" V 945 8850 50  0000 L CNN
-F 2 "MountingHole:MountingHole_3.2mm_M3_Pad_Via" H 900 8700 50  0001 C CNN
-F 3 "~" H 900 8700 50  0001 C CNN
-	1    900  8700
+P 900 9900
+F 0 "H3" V 854 10050 50  0000 L CNN
+F 1 "MountingHole_Pad" V 945 10050 50  0000 L CNN
+F 2 "MountingHole:MountingHole_3.2mm_M3_Pad_Via" H 900 9900 50  0001 C CNN
+F 3 "~" H 900 9900 50  0001 C CNN
+	1    900  9900
 	0    1    1    0
 $EndComp
@@
 L Mechanical:MountingHole_Pad H4
 U 1 1 611D8E91
-P 900 8900
-F 0 "H4" V 854 9050 50  0000 L CNN
-F 1 "MountingHole_Pad" V 945 9050 50  0000 L CNN
-F 2 "MountingHole:MountingHole_3.2mm_M3_Pad_Via" H 900 8900 50  0001 C CNN
-F 3 "~" H 900 8900 50  0001 C CNN
-	1    900  8900
+P 900 10100
+F 0 "H4" V 854 10250 50  0000 L CNN
+F 1 "MountingHole_Pad" V 945 10250 50  0000 L CNN
+F 2 "MountingHole:MountingHole_3.2mm_M3_Pad_Via" H 900 10100 50  0001 C CNN
+F 3 "~" H 900 10100 50  0001 C CNN
+	1    900  10100
 	0    1    1    0
 $EndComp
@@
 L power:GND #PWR04
 U 1 1 611E8DC8
-P 800 9000
-F 0 "#PWR04" H 800 8750 50  0001 C CNN
-F 1 "GND" H 805 8827 50  0000 C CNN
-F 2 "" H 800 9000 50  0001 C CNN
-F 3 "" H 800 9000 50  0001 C CNN
-	1    800  9000
-	1    0    0    -1
-$EndComp
-Wire Wire Line
-	800  8300 800  8500
-Connection ~ 800  8500
-Wire Wire Line
-	800  8500 800  8700
-Connection ~ 800  8700
-Wire Wire Line
-	800  8700 800  8900
-Connection ~ 800  8900
-Wire Wire Line
-	800  8900 800  9000
+P 800 10200
+F 0 "#PWR04" H 800 9950 50  0001 C CNN
+F 1 "GND" H 805 10027 50  0000 C CNN
+F 2 "" H 800 10200 50  0001 C CNN
+F 3 "" H 800 10200 50  0001 C CNN
+	1    800  10200
+	1    0    0    -1
+$EndComp
+Wire Wire Line
+	800  9500 800  9700
+Connection ~ 800  9700
+Wire Wire Line
+	800  9700 800  9900
+Connection ~ 800  9900
+Wire Wire Line
+	800  9900 800  10100
+Connection ~ 800  10100
+Wire Wire Line
+	800  10100 800  10200
 $Comp
 L Mechanical:Fiducial FID1
 U 1 1 6120074B
-P 3100 8400
-F 0 "FID1" H 3185 8446 50  0000 L CNN
-F 1 "Ignitionlet" H 3185 8355 50  0000 L CNN
-F 2 "grumpy:Oxide_Board_Identifier_23x6mm" H 3100 8400 50  0001 C CNN
-F 3 "~" H 3100 8400 50  0001 C CNN
-	1    3100 8400
+P 3800 9400
+F 0 "FID1" H 3885 9446 50  0000 L CNN
+F 1 "Ignitionlet" H 3885 9355 50  0000 L CNN
+F 2 "grumpy:Oxide_Board_Identifier_23x6mm" H 3800 9400 50  0001 C CNN
+F 3 "~" H 3800 9400 50  0001 C CNN
+	1    3800 9400
 	1    0    0    -1
 $EndComp
@@
 L Mechanical:Fiducial FID2
 U 1 1 61202097
-P 3100 8700
-F 0 "FID2" H 3185 8746 50  0000 L CNN
-F 1 "Fiducial" H 3185 8655 50  0000 L CNN
-F 2 "Fiducial:Fiducial_1mm_Mask2mm" H 3100 8700 50  0001 C CNN
-F 3 "~" H 3100 8700 50  0001 C CNN
-	1    3100 8700
-	1    0    0    -1
-$EndComp
-Text Notes 700  8000 0    79   ~ 16
+P 3800 9700
+F 0 "FID2" H 3885 9746 50  0000 L CNN
+F 1 "Fiducial" H 3885 9655 50  0000 L CNN
+F 2 "Fiducial:Fiducial_1mm_Mask2mm" H 3800 9700 50  0001 C CNN
+F 3 "~" H 3800 9700 50  0001 C CNN
+	1    3800 9700
+	1    0    0    -1
+$EndComp
+Text Notes 700  9200 0    79   ~ 16
 Mechanical
-Text Notes 1800 9500 0    50   ~ 0
-The board assumes the width of two standard\n0.80” PMOD boards. J16 is present only for\nadditional mechanical stability, but can be used\nfor prototyping.
-NoConn ~ 2100 8400
-NoConn ~ 2100 8500
-NoConn ~ 2100 8600
-NoConn ~ 2100 8700
-NoConn ~ 2100 8900
-NoConn ~ 2600 8900
-NoConn ~ 2600 8700
-NoConn ~ 2600 8600
-NoConn ~ 2600 8500
-NoConn ~ 2600 8400
+Text Notes 1800 10900 0    50   ~ 0
+The board assumes the width of two standard\n0.80” PMOD boards. J16 is intended for additional\nmechanical stability, but is connected to J17 as a\nType 1 interface, providing GPIOs for prototyping\nwhich for example can be wired to CDONE or\nFLASH_RESET when connected to an appropriate\nhost board.
+NoConn ~ 2100 9600
+NoConn ~ 2100 9700
+NoConn ~ 2100 9800
+NoConn ~ 2100 9900
+NoConn ~ 2100 10100
+NoConn ~ 2600 10100
 $Comp
 L Connector_Generic:Conn_02x06_Top_Bottom J16
 U 1 1 6130518A
-P 2300 8600
-F 0 "J16" H 2350 9017 50  0000 C CNN
-F 1 "Conn_02x06_Top_Bottom" H 2350 8926 50  0000 C CNN
-F 2 "pmod:PMOD_12pin_peripheral_horizontal" H 2300 8600 50  0001 C CNN
-F 3 "~" H 2300 8600 50  0001 C CNN
-	1    2300 8600
+P 2300 9800
+F 0 "J16" H 2350 10217 50  0000 C CNN
+F 1 "Conn_02x06_Top_Bottom" H 2350 10126 50  0000 C CNN
+F 2 "pmod:PMOD_12pin_peripheral_horizontal" H 2300 9800 50  0001 C CNN
+F 3 "~" H 2300 9800 50  0001 C CNN
+	1    2300 9800
 	1    0    0    -1
 $EndComp
@@
 L power:GND #PWR0162
 U 1 1 61307B28
-P 2000 8800
-F 0 "#PWR0162" H 2000 8550 50  0001 C CNN
-F 1 "GND" H 2005 8627 50  0000 C CNN
-F 2 "" H 2000 8800 50  0001 C CNN
-F 3 "" H 2000 8800 50  0001 C CNN
-	1    2000 8800
+P 2000 10000
+F 0 "#PWR0162" H 2000 9750 50  0001 C CNN
+F 1 "GND" H 2005 9827 50  0000 C CNN
+F 2 "" H 2000 10000 50  0001 C CNN
+F 3 "" H 2000 10000 50  0001 C CNN
+	1    2000 10000
 	1    0    0    -1
 $EndComp
@@
 L power:GND #PWR0163
 U 1 1 61307EE4
-P 2700 8800
-F 0 "#PWR0163" H 2700 8550 50  0001 C CNN
-F 1 "GND" H 2705 8627 50  0000 C CNN
-F 2 "" H 2700 8800 50  0001 C CNN
-F 3 "" H 2700 8800 50  0001 C CNN
-	1    2700 8800
-	1    0    0    -1
-$EndComp
-Wire Wire Line
-	2000 8800 2100 8800
-Wire Wire Line
-	2600 8800 2700 8800
+P 2700 10000
+F 0 "#PWR0163" H 2700 9750 50  0001 C CNN
+F 1 "GND" H 2705 9827 50  0000 C CNN
+F 2 "" H 2700 10000 50  0001 C CNN
+F 3 "" H 2700 10000 50  0001 C CNN
+	1    2700 10000
+	1    0    0    -1
+$EndComp
+Wire Wire Line
+	2000 10000 2100 10000
+Wire Wire Line
+	2600 10000 2700 10000
 Wire Wire Line
 	11900 6100 12200 6100
@@
 AUX1_TX_TAP_N
 Wire Notes Line
-	600  7800 3900 7800
-Wire Notes Line
-	3900 7800 3900 9700
-Wire Notes Line
-	3900 9700 600  9700
-Wire Notes Line
-	600  9700 600  7800
+	600  9000 4400 9000
+Wire Notes Line
+	4400 9000 4400 11000
+Wire Notes Line
+	4400 11000 600  11000
+Wire Notes Line
+	600  11000 600  9000
 $Comp
 L Ignition:MCZ1210AH900L2TA0G L1
@@
 Text Notes 13900 5500 0    79   ~ 16
 CMDx LEDs
+$Comp
+L Connector_Generic:Conn_01x04 J17
+U 1 1 60E0E021
+P 3200 9700
+F 0 "J17" H 3200 10025 50  0000 C CNN
+F 1 "Conn_01x04" H 3200 9925 50  0000 C CNN
+F 2 "Connector_PinHeader_2.54mm:PinHeader_1x04_P2.54mm_Vertical" H 3200 9700 50  0001 C CNN
+F 3 "~" H 3200 9700 50  0001 C CNN
+	1    3200 9700
+	1    0    0    -1
+$EndComp
+Wire Wire Line
+	2600 9600 3000 9600
+Wire Wire Line
+	3000 9700 2600 9700
+Wire Wire Line
+	2600 9800 3000 9800
+Wire Wire Line
+	3000 9900 2600 9900
 $EndSCHEMATC

Commit message: Ignitionlet rev 2, first pass
Parts:
- removed R24, R25, R26, R27, R28, R29, R30, R31, R32, R33, R34, R35: 10K, Resistor_SMD:R_0603_1608Metric, symbol Device:R_Small_US
- added FID3: Fiducial, Fiducial:Fiducial_1mm_Mask2mm, symbol Mechanical:Fiducial
- FID1: footprint grumpy:Oxide_Board_Identifier_23x6mm -> grumpy:Oxide_Board_Identifier_23x6mm_PCBWay
- R36, R37: value 280 -> 309
- TP1: footprint test-point:TestPoint_THTPad_D0.6mm_Drill0.3mm -> test-point:TestPoint_Pad_D0.6mm
Connections:
- net labels added: VCCIO_3
- net labels removed: V2P5
- wire segments 245 -> 209
Other:
- note added: "Command bits are exposed on a header\nfor easy probing and/or alternative\nprototyping."
- note added: "Fault pin straps allow setting fixed fault values.\nThe switch attached to PWR_FLT0 provides a\nconvenient way to cause fault interrupts during\nintegration tests. The header allows reuse of\nthese pins for alternative prototyping.\n\nThe FPGA should use programmable\npull-up/pull-down on these poins if required."
- note added: "ID straps allow setting the desired value.\nThe header allows reuse of these pins\nfor alternative prototyping.\n\nSee RFD 142 for currently allocated ID\nvalues. The FPGA should use programmable\npull-up/pull-down on these pins if required."
- note added: "If: 5mA\nVf: 1.9V\nRlim: ~~300Ω"
- note added: "The LVDS transmitter pair is implemented as per Lattice FPGA-TN-1253 using PIO pin pairs in Bank 3.\nThe resistor values above were derived using the equations on p. 4 and the following assumptions:\n\nZ0 = 50 ohm\nVCCIO = 2.5V\nV_OD = 0.35V\nR_OUTPUT = 30 ohm\n\nR_P = 2 * ((Z0 * VCCIO) / (VCCIO - (2 * V_OD)))\n = 2 * (165 / 1.8)\n = 139 ohm\n\nR_S = ((Z0 * R_P / 2) / ((R_P / 2) - Z0) - R_OUTPUT\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"
- note removed: "Command bits are exposed on a header\nfor easy test probing and alternative\nprototyping."
- note removed: "Fault pin straps allow setting fixed fault values. The switch\nattached to ROT_FLT provides a convenient way to cause\nfault interrupts during integration tests. The header allows\nreuse of these pins for alternative prototyping."
- note removed: "ID straps allow setting the desired value. The header\nallows reuse of these pins for alternative prototyping\n\nSee RFD 142 for currently allocated ID values."
- note removed: "If: 5mA\nVf: 1.9V\nRlim: 280Ω"
- note removed: "The LVDS transmitter pair is implemented as per Lattice FPGA-TN-1253\nusing PIO pin pairs in Bank 3. The resistor values above were derived\nusing the equations on p. 4 and the following assumptions:\n\nZ0 = 50 ohm\nVCCIO = 2.5V\nV_OD = 0.35V\nR_OUTPUT = 30 ohm\n\nR_P = 2 * ((Z0 * VCCIO) / (VCCIO - (2 * V_OD)))\n = 2 * (165 / 1.8)\n = 139 ohm\n\nR_S = ((Z0 * R_P / 2) / ((R_P / 2) - Z0) - R_OUTPUT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"
- moved on the sheet: D1, D2, FID1, FID2, H1, H2, H3, H4, J13, J14, J15, J16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

Commit message: Ignitionlet rev 2, Gerbers out
Changed lines of the file:
@@
 Sheet 1 3
 Title "Ignition Target"
-Date "2021-07-21"
+Date "2021-07-22"
 Rev "2"
 Comp "Oxide Computer Co."
@@
 Wire Wire Line
 	14200 1800 14500 1800
-Connection ~ 14200 1300
-Wire Wire Line
-	14200 1200 14200 1300
 Wire Wire Line
 	14200 1400 14200 1500
@@
 Wire Wire Line
 	5000 6000 5500 6000
-$Comp
-L Ignition:V3P3 #PWR0120
-U 1 1 60E4E2D4
-P 14200 1200
-F 0 "#PWR0120" H 14200 1050 50  0001 C CNN
-F 1 "V3P3" H 14215 1373 50  0000 C CNN
-F 2 "" H 14200 1200 50  0001 C CNN
-F 3 "" H 14200 1200 50  0001 C CNN
-	1    14200 1200
-	1    0    0    -1
-$EndComp
 Text Label 5000 4400 0    50   ~ 0
 ~PWR_FLT0
@@
 	1    0    0    -1
 $EndComp
+$Comp
+L power:GND #PWR0120
+U 1 1 60FAAE32
+P 14200 1900
+F 0 "#PWR0120" H 14200 1650 50  0001 C CNN
+F 1 "GND" H 14205 1727 50  0000 C CNN
+F 2 "" H 14200 1900 50  0001 C CNN
+F 3 "" H 14200 1900 50  0001 C CNN
+	1    14200 1900
+	1    0    0    -1
+$EndComp
+Wire Wire Line
+	14200 1900 14200 1800
+Connection ~ 14200 1800
 $EndSCHEMATC
