File: ignitionlet.kicad_pcb (KiCad board)
At the start: 4 copper layers, 153.7 x 43.2 mm, 133 parts, among them J1 Conn_Coaxial, J10 Conn_Coaxial, J101 Barrel_Jack_MountingPin, J102 Conn_01x02, J103 Conn_01x03, J11 Conn_Coaxial, J12 Conn_Coaxial, J13 Conn_02x06_Odd_Even, J14 Conn_02x06_Odd_Even, J15 Conn_01x04, J16 Conn_02x06_Top_Bottom, J2 Conn_Coaxial, J201 PMOD_2A_PERIPHERAL, J202 IGNITION_TARGET_HDR, J203 Conn_02x04_Odd_Even, J204 Conn_01x03, J205 Conn_01x03, J3 Conn_Coaxial, J4 Conn_Coaxial, J5 Conn_01x04, J6 Conn_01x04, J7 Conn_01x04, J8 Conn_01x04, J9 Conn_Coaxial, SW1 FPGA_RST, SW2 SYS_RST, SW3 FLT, U1 IGNITION001-QFN, U101 LT3013EFE#PBF, U102 LT3013EFE#PBF, U103 TPS7A0525PDBVR, U2 AMPMGFB-50.0000T, U5 MT25QL128ABB8E12-0AUT, U6 AT25PE80-SSHN-B

Commit message: Simplify copper pours, improve silkscreen, small fixes/improvements
Parts:
- FID1: value IGNITIONLET -> Ignitionlet
- moved C103 70.2 mm to (107.3, 101.9)
- moved C115 70.2 mm to (134.5, 98.8)
- moved C116 70.2 mm to (138.3, 92.2)
- moved C120 70.2 mm to (137.9, 98.1)
- moved C121 70.2 mm to (140.2, 97.3)
- moved C122 70.2 mm to (134.1, 101.9)
- moved C202 70.2 mm to (132.1, 92.2)
- moved J10 70.2 mm to (193.8, 109.7)
- moved J15 70.2 mm to (155.7, 76.7)
- moved J3 70.2 mm to (168.4, 109.7)
- moved J4 70.2 mm to (206.5, 109.7)
- moved R104 70.2 mm to (117.9, 87.1)
- moved R2 70.2 mm to (148.2, 100.6)
- moved R20 70.2 mm to (178.5, 86.4)
- moved R201 70.2 mm to (140.2, 83.5)
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Routing:
- net GND: track 70.5 -> 78.3 mm

Commit message: Add chokes on TX SerDes
Parts:
- added L1: MCZ1210AH900L2TA0G, passives:L_Choke_MCZ1210AH, F.Cu at (180.5, 103.4)
- added L2: MCZ1210AH900L2TA0G, passives:L_Choke_MCZ1210AH, F.Cu at (193.2, 103.4)
- moved C10 3.05 mm to (190.0, 102.6)
- moved C11 3.05 mm to (190.0, 104.1)
- moved C8 2.74 mm to (177.6, 104.1)
- moved C9 2.74 mm to (177.6, 102.6)
Connections:
- J10 pad 1: Net-(C11-Pad2) -> Net-(J10-Pad1)
- J11 pad 1: Net-(C8-Pad2) -> Net-(J11-Pad1)
- J12 pad 1: Net-(C10-Pad2) -> Net-(J12-Pad1)
- J9 pad 1: Net-(C9-Pad2) -> Net-(J9-Pad1)
Routing:
- net Net-(J9-Pad1): track 0.00 -> 6.10 mm
- net Net-(J12-Pad1): track 0.00 -> 6.07 mm
- net Net-(J10-Pad1): track 0.00 -> 6.07 mm
- net Net-(J11-Pad1): track 0.00 -> 6.05 mm
- net GND: track 78.3 -> 82.8 mm
- net Net-(C8-Pad2): track 5.59 -> 1.74 mm
- net Net-(C9-Pad2): track 5.59 -> 1.75 mm
- net Net-(C11-Pad2): track 5.59 -> 2.05 mm
- net Net-(C10-Pad2): track 5.59 -> 2.05 mm
- net /AUX1_TX_LVDS_P: track 29.8 -> 26.7 mm
- net /AUX1_TX_LVDS_N: track 29.8 -> 26.7 mm
- net /AUX0_TX_LVDS_P: track 35.0 -> 32.3 mm
- net /AUX0_TX_LVDS_N: track 35.0 -> 32.3 mm

Commit message: Add TPs, routing tweaks, stitch top ground, add CMD1 LED
Parts:
- added D2: LTST-C193KGKT-5A, LED_SMD:LED_0603_1608Metric, F.Cu at (158.5, 77.5)
- added R37: 280, Resistor_SMD:R_0603_1608Metric, F.Cu at (158.5, 82.8)
- added TP1: TestPoint, test-point:TestPoint_THTPad_D0.6mm_Drill0.3mm, F.Cu at (136.1, 103.1)
- added TP101: TestPoint, TestPoint:TestPoint_THTPad_D1.0mm_Drill0.5mm, F.Cu at (122.8, 88.6)
- added TP102: TestPoint, TestPoint:TestPoint_THTPad_D1.0mm_Drill0.5mm, F.Cu at (141.9, 108.2)
- added TP103: TestPoint, TestPoint:TestPoint_THTPad_D1.0mm_Drill0.5mm, F.Cu at (145.0, 114.8)
- added TP104: TestPoint, TestPoint:TestPoint_Keystone_5015_Micro-Minature, F.Cu at (113.7, 94.4)
- added TP105: TestPoint, TestPoint:TestPoint_Keystone_5015_Micro-Minature, F.Cu at (217.9, 99.1)
- added TP2: TestPoint, test-point:TestPoint_THTPad_D0.6mm_Drill0.3mm, F.Cu at (138.2, 102.6)
- moved R36 2.65 mm to (160.5, 82.8)
- moved R209 1.32 mm to (131.3, 90.4), turned to 90 degrees
- moved D1 1.14 mm to (160.5, 77.4)
- moved C120 0.11 mm to (138.0, 98.0)
Routing:
- net Net-(D2-Pad2): track 0.00 -> 3.76 mm
- net /CMD1: track 26.8 -> 30.4 mm
- net GND: track 82.8 -> 79.5 mm, vias 113 -> 180
- net Net-(D1-Pad2): track 1.40 -> 3.78 mm
- net /Config/SPI_SCK: track 157.1 -> 155.0 mm, vias 3 -> 4
- net Net-(R209-Pad1): track 2.21 -> 3.72 mm
- net V2P5: track 81.9 -> 82.6 mm, vias 8 -> 9
- net /Config/~FPGA_RESET: track 123.2 -> 123.8 mm
- net V3P3: vias 29 -> 31
- net V1P2: vias 7 -> 6
Other:
- outline, holes or cut-outs redrawn
- board text added: "2.5V"
- board text added: "3.3V"
- board text added: "CDONE"
- board text added: "CRESET"
- board text added: "FLASH RST"
- board text added: "FLASH WP"
- board text added: "FLT"
- board text added: "ID: 0 1 2 3 4 5"
- board text added: "RST"
- board text added: "RoT 4 FLT: 3 2 1 0"

Commit message: Add SerDes silkscreen labels
Other:
- board text added: "AUX0 RX+"
- board text added: "AUX0 RX-"
- board text added: "AUX0 TX+"
- board text added: "AUX0 TX-"
- board text added: "AUX1 RX+"
- board text added: "AUX1 RX-"
- board text added: "AUX1 TX+"
- board text added: "AUX1 TX-"
Changed lines of the file:
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@@
   (general
     (thickness 1.6)
-    (drawings 18)
+    (drawings 26)
     (tracks 1258)
     (zones 0)
@@
     )
   )
+  (gr_text "AUX1 RX+" (at 201.93 96.774 90) (layer F.SilkS)
+    (effects (font (size 1 1) (thickness 0.15)))
+  )
+  (gr_text "AUX1 RX-" (at 201.93 109.601 90) (layer F.SilkS)
+    (effects (font (size 1 1) (thickness 0.15)))
+  )
+  (gr_text "AUX1 TX-" (at 189.23 96.901 90) (layer F.SilkS)
+    (effects (font (size 1 1) (thickness 0.15)))
+  )
+  (gr_text "AUX1 TX+" (at 189.23 109.728 90) (layer F.SilkS)
+    (effects (font (size 1 1) (thickness 0.15)))
+  )
+  (gr_text "AUX0 TX-" (at 176.53 96.901 90) (layer F.SilkS)
+    (effects (font (size 1 1) (thickness 0.15)))
+  )
+  (gr_text "AUX0 TX+" (at 176.53 109.728 90) (layer F.SilkS)
+    (effects (font (size 1 1) (thickness 0.15)))
+  )
+  (gr_text "AUX0 RX-" (at 163.83 109.728 90) (layer F.SilkS)
+    (effects (font (size 1 1) (thickness 0.15)))
+  )
+  (gr_text "AUX0 RX+" (at 163.83 96.901 90) (layer F.SilkS)
+    (effects (font (size 1 1) (thickness 0.15)))
+  )
   (gr_arc (start 74.168 75.184) (end 74.168 74.168) (angle -90) (layer Edge.Cuts) (width 0.05))

Commit message: Small top pour/signal tweaks
Parts:
- moved R210 0.13 mm to (134.0, 88.7)
Routing:
- net /Config/SPI_MISO: track 121.1 -> 124.0 mm
- net GND: vias 180 -> 183

Commit message: Extend J16 to allow Type 1 GPIO interface
Parts:
- added J17: Conn_01x04, Connector_PinHeader_2.54mm:PinHeader_1x04_P2.54mm_Vertical, F.Cu at (73.7, 76.2)
- moved TP102 9.44 mm to (132.6, 106.4)
- moved R30 8.57 mm to (124.5, 107.2)
- moved C117 8.57 mm to (124.6, 94.5)
- moved J13 8.57 mm to (124.5, 74.9)
- moved R210 8.57 mm to (125.6, 86.9)
- moved C1 8.57 mm to (159.2, 100.8)
- moved C10 8.57 mm to (181.6, 100.8)
- moved C105 8.57 mm to (111.6, 93.5)
- moved C106 8.57 mm to (100.1, 85.3)
- moved C108 8.57 mm to (111.0, 88.6)
- moved C11 8.57 mm to (181.6, 102.4)
- moved C110 8.57 mm to (117.0, 93.8)
- moved C111 8.57 mm to (109.5, 88.6)
- moved C113 8.57 mm to (112.4, 88.6)
- moved C120 8.57 mm to (129.6, 96.2)
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Routing:
- net Net-(J16-Pad8): track 0.00 -> 6.13 mm
- net Net-(J16-Pad10): track 0.00 -> 6.13 mm
- net Net-(J16-Pad9): track 0.00 -> 6.13 mm
- net Net-(J16-Pad7): track 0.00 -> 6.13 mm
- net GND: vias 183 -> 181
