File: ignition_adafruit_ft232h_rD_adapter.kicad_pcb (KiCad board)
At the start: 4 copper layers, 48.3 x 22.9 mm, 11 parts, among them J1 ADAFRUIT_FT232H_REV_D, J2 IGNITION_TARGET_HDR

Commit message: Add LVDS SMA adapter, finish programming adapter, Ignitionlet nits
- Add LVDS SMA adapter for ULX3S/ECP5 EVN boards
- Finish Ignition Target programming adapter
- Small nit fixes in Ignitionlet found after tapeout
Parts:
- added FID3: Fiducial, Fiducial:Fiducial_0.5mm_Mask1mm, F.Cu at (123.2, 99.1)
- moved FID1 1.27 mm to (163.8, 90.2)
