File: ignition_adafruit_ft232h_rD_adapter.sch (KiCad schematic (older format))
At the start: 11 parts, among them J1 ADAFRUIT_FT232H_REV_D, J2 IGNITION_TARGET_HDR

Commit message: Add LVDS SMA adapter, finish programming adapter, Ignitionlet nits
- Add LVDS SMA adapter for ULX3S/ECP5 EVN boards
- Finish Ignition Target programming adapter
- Small nit fixes in Ignitionlet found after tapeout
Parts:
- added FID3: Fiducial, Fiducial:Fiducial_0.5mm_Mask1mm, symbol Mechanical:Fiducial
Changed lines of the file:
@@
 Sheet 1 1
 Title "Ignition Header Adapter for Adafruit FT232H rev D"
-Date "2021-07-06"
-Rev ""
-Comp ""
+Date "2021-07-12"
+Rev "1"
+Comp "Oxide Computer Co."
 Comment1 ""
 Comment2 ""
@@
 Wire Wire Line
 	7000 4200 7100 4200
+$Comp
+L Mechanical:Fiducial FID3
+U 1 1 60E8A50C
+P 7900 5500
+F 0 "FID3" H 7985 5500 50  0000 L CNN
+F 1 "Fiducial" H 7985 5455 50  0001 L CNN
+F 2 "Fiducial:Fiducial_0.5mm_Mask1mm" H 7900 5500 50  0001 C CNN
+F 3 "~" H 7900 5500 50  0001 C CNN
+	1    7900 5500
+	1    0    0    -1
+$EndComp
 $EndSCHEMATC
