File: gimletlet.sch (KiCad schematic (older format))
At the start: 59 parts, among them J1 Conn_02x16_Odd_Even, J2 Conn_02x15_Odd_Even, J3 Conn_01x04, J4 SWD, J5 I2C, SW1 RESET, U1 STM32H753IITx, Y1 8MHz

Commit message: gimletlet: revamp into useful board
Parts:
- removed C6, C7, C8, C9: 0µ1, Capacitor_SMD:C_0603_1608Metric, symbol Device:C
- removed H1: MountingHole, MountingHole:MountingHole_3.2mm_M3, symbol Mechanical:MountingHole
- removed J1: Conn_02x16_Odd_Even, Connector_PinSocket_2.54mm:PinSocket_2x02_P2.54mm_Vertical, symbol Connector_Generic:Conn_02x02_Odd_Even
- removed J2: Conn_02x15_Odd_Even, Connector_PinSocket_2.54mm:PinSocket_2x15_P2.54mm_Vertical, symbol Connector_Generic:Conn_02x15_Odd_Even
- removed J3: Conn_01x04, Connector_PinHeader_2.54mm:PinHeader_1x04_P2.54mm_Horizontal, symbol Connector_Generic:Conn_01x04
- removed J5: I2C, Connector_PinHeader_2.54mm:PinHeader_1x04_P2.54mm_Vertical_SMD_Pin1Left, symbol Connector_Generic:Conn_01x04
- removed R8: 22, Resistor_SMD:R_0603_1608Metric, symbol Device:R
- added C1, C2: 22µ, Capacitor_Tantalum_SMD:CP_EIA-7343-31_Kemet-D, symbol Device:CP_Small
- added F1: Polyfuse, Fuse:Fuse_1812_4532Metric, symbol Device:Polyfuse
- added H1, H2, H3, H4: MountingHole, MountingHole:MountingHole_3.2mm_M3_Pad_Via, symbol Mechanical:MountingHole_Pad
- added H5, H6: MountingHole, MountingHole:MountingHole_3.2mm_M3, symbol Mechanical:MountingHole
- added J1: 12V, Connector_BarrelJack:BarrelJack_CUI_PJ-036AH-SMT_Horizontal, symbol Connector:Barrel_Jack_Switch
- added J10: I2C3, pmod:PMOD_6pin_host_horizontal, symbol Connector_Generic:Conn_01x06
- added J11: I2C4, pmod:PMOD_6pin_host_horizontal, symbol Connector_Generic:Conn_01x06
- added J12: USART1, pmod:PMOD_6pin_host_horizontal, symbol Connector_Generic:Conn_01x06
- added J13: USART2, pmod:PMOD_6pin_host_horizontal, symbol Connector_Generic:Conn_01x06
- added J14: UART7, pmod:PMOD_6pin_host_horizontal, symbol Connector_Generic:Conn_01x06
- added J16: GPIO1, Connector_PinSocket_2.54mm:PinSocket_1x09_P2.54mm_Vertical, symbol Connector_Generic:Conn_01x09
- added J17: Conn_01x07, Connector_PinSocket_2.54mm:PinSocket_1x07_P2.54mm_Vertical, symbol Connector_Generic:Conn_01x07
- added J2: QSPI, pmod:PMOD_12pin_host_horizontal, symbol Connector_Generic:Conn_02x06_Top_Bottom
- added J3: SPI3, pmod:PMOD_12pin_host_horizontal, symbol Connector_Generic:Conn_02x06_Top_Bottom
- added J4: SPI4, pmod:PMOD_12pin_host_horizontal, symbol Connector_Generic:Conn_02x06_Top_Bottom
- added J5: SPI6, pmod:PMOD_12pin_host_horizontal, symbol Connector_Generic:Conn_02x06_Top_Bottom
- added J6: NIC, hirose-df9:Hirose_DF9-41S-1V(69)_2Rows_41Pin-2MP_P1.0mm_Vertical, symbol Connector_Generic:Conn_2Rows-41Pins
- added J7: 12V, Connector_PinSocket_2.54mm:PinSocket_2x03_P2.54mm_Vertical, symbol Connector_Generic:Conn_02x03_Odd_Even
- added J8: 3V3, Connector_PinSocket_2.54mm:PinSocket_2x03_P2.54mm_Vertical, symbol Connector_Generic:Conn_02x03_Odd_Even
- added J9: I2C2, pmod:PMOD_6pin_host_horizontal, symbol Connector_Generic:Conn_01x06
- added JP1: JACK, Connector_PinHeader_2.54mm:PinHeader_1x02_P2.54mm_Vertical, symbol Device:Jumper
- added JP2: REG, Connector_PinHeader_2.54mm:PinHeader_1x02_P2.54mm_Vertical, symbol Device:Jumper
- added R1, R10, R12, R13, R14, R16, R17, R18, R19, R20, R21, R22, R23, R24, R26, R27, R29, R30, R5, R7: 10k, Resistor_SMD:R_0603_1608Metric, symbol Device:R
- added R31, R32, R33, R34, R35, R36, R37, R39, R40, R45, R46: 22, Resistor_SMD:R_0603_1608Metric, symbol Device:R
- added TP1, TP10, TP11, TP2, TP3, TP4, TP5, TP6, TP7, TP8, TP9: TestPoint_Small, TestPoint:TestPoint_THTPad_D2.0mm_Drill1.0mm, symbol Connector:TestPoint_Small
- added TP12, TP13, TP14, TP15, TP16, TP17, TP18, TP19, TP20, TP21, TP22, TP23: GND, TestPoint:TestPoint_Loop_D3.50mm_Drill1.4mm_Beaded, symbol Connector:TestPoint
- added U1: OKI-78SR-3.3_1.5-W36-C, Converter_DCDC:Converter_DCDC_muRata_OKI-78SR_Vertical, symbol Converter_DCDC:OKI-78SR-3.3_1.5-W36-C
- JP3: renamed from JP1; footprint Jumper:SolderJumper-2_P1.3mm_Open_RoundedPad1.0x1.5mm -> Connector_PinHeader_2.54mm:PinHeader_2x01_P2.54mm_Vertical; symbol Jumper:SolderJumper_2_Open -> Jumper:Jumper_2_Open
- R11, R2, R3, R6, R9: value 22 -> 10k
- R15: value 100k -> 10k
- U2: renamed from U1; value STM32H753IITx -> STM32H753ZITx; footprint Package_QFP:LQFP-176_24x24mm_P0.5mm -> Package_QFP:LQFP-144_20x20mm_P0.5mm; symbol MCU_ST_STM32H7:STM32H753IITx -> MCU_ST_STM32H7:STM32H753ZITx
- renumbered C12 to C10, C13 to C11, C14 to C12, C15 to C13, C16 to C14, C17 to C15, C18 to C16, C19 to C17, C20 to C18, C21 to C19, C22 to C20, C2 to C3, C1 to C4, C3 to C5, C4 to C6, C5 to C7, C10 to C8, C11 to C9, J4 to J15, R21 to R25, R22 to R28, R12 to R38, R14 to R4, R7 to R41, R5 to R42, R10 to R43, R1 to R44, R4 to R47, R16 to R48, R17 to R49, R18 to R50, R19 to R51, R20 to R52, R13 to R8
Connections:
- net labels added: +12V, 12V_IN, I2C2_SCL, I2C2_SDA, I2C3_SCL, I2C3_SDA, I2C4_SCL, I2C4_SDA, JACK_12V, PB0, PB1, PB14, PB15, PB2, PD10, PD11, PD12, PD8, PD9, PE2, PE3, PE4, PE5, PE6, PF11, PF12, QSPI_CLK, QSPI_IO0, QSPI_IO1, QSPI_IO2, QSPI_IO3, QSPI_XTRA10, QSPI_XTRA7, REG_3V3, SPI3_MISO, SPI3_MOSI, SPI3_SCK, SPI4_MISO, SPI4_MOSI, SPI4_SCK, SPI6_MISO, SPI6_MOSI, SPI6_SCK, UART7_CTS, UART7_RTS, UART7_RX, UART7_TX, USART1_CTS, USART1_RTS, USART2_CTS, USART2_RTS, USART2_RX, USART2_TX, ~I2C2_RESET, ~I2C2_SMBA, ~I2C3_RESET, ~I2C3_SMBA, ~I2C4_RESET, ~I2C4_SMBA, ~QSPI_CS, ~SMI_RESET, ~SPI3_CS, ~SPI3_INT, ~SPI3_RESET, ~SPI4_CS, ~SPI4_INT, ~SPI4_RESET, ~SPI6_CS, ~SPI6_INT, ~SPI6_RESET
- net labels removed: SCL, SDA, SPI2_MISO, SPI2_MOSI, SPI2_SCK, X_MDC, X_MDIO, X_RMII_CRS_DV, X_RMII_REFCLK, X_RMII_RXD0, X_RMII_RXD1, X_RMII_TXD0, X_RMII_TXD1, X_RMII_TXEN, X_SPI_MISO, X_SPI_MOSI, X_SPI_SCK, ~SPI2_CS0, ~SW_IRQ, ~X_SMI_INTR, ~X_SPI_CS, ~X_SW_INTR
- wire segments 145 -> 313
- no-connect marks 115 -> 35
Other:
- note added: "ALL I/O 3.3V."
- note added: "For dupont wires →"
- note added: "General notes:"
- note added: "HACKING"
- note added: "I2C2: SDA=F0 SCL=F1 ~SMBA=F2"
- note added: "I2C3: SDA=C9 SCL=A8 ~SMBA=A9"
- note added: "I2C4: SDA=F15, SCL=F14, ~SMBA=F13"
- note added: "INT and RESET lines can also act as extra chip selects."
- note added: "Interfaces routed:"
- note added: "I²C (PMOD type 6)"
- note added: "JP1 allows power injection\nupstream from fuse."
- note added: "JP2 allows disconnection of\npower supply or 3v3 injection."
- note added: "NIC RMII+SPI+I2C"
- note added: "POWER"
- note added: "PROGRAM/DEBUG"
- note added: "Probing I²C?\nUse J11."
- note added: "Probing SPI?\nUse J4."
- note added: "Pull resistors provided and placed near primary\nconnector."
- note added: "QSPI: CLK=F10 IO{3,2,0,1}=F6-9 ~CS=G6"
- note added: "QUADSPI"
- note added: "Qwiic/Grove/Stemma/QT connectors can be\njumpered to the 100mil PMOD headers."
- note added: "REMOVE DEVICE PULLUP JUMPERS"
- note added: "SHARED\nWITH NIC!"
- note added: "SPI (PMOD type 2A)"
- note added: "SPI3: MISO=C11 MOSI=C12 SCK=C10 ~CS=A15"
- note added: "SPI4: MISO=E13 MOSI=E14 SCK=E12 ~CS=E11"
- note added: "SPI6: MISO=G12 MOSI=G14 SCK=G13 CS=G8"
- note added: "Slew-limiting resistors placed near the driver."
- note added: "Test points placed near primary connector."
- note added: "UART (PMOD type 3)"
- note added: "UART7: TX=E8 RX=E7 RTS=E9 CTS=E10"
- note added: "USART1: TX=B6 RX=B7 RTS=A12 CTS=A11"
- note added: "USART2: TX=D5 RX=D6 CTS=D3 RTS=D4"
- note removed: "NOTE: mgmt board does *not* have\nslew limiting resistors on outputs"
- moved on the sheet: C10, C11, C12, C13, C14, C15, C16, C17, C18, C19, C20, C3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

Commit message: gimletlet: fork stm32h7 symbol to fix ERC
Parts:
- U2: symbol MCU_ST_STM32H7:STM32H753ZITx -> stm32h7:STM32H753ZITx
Changed lines of the file:
@@
 Connection ~ 8700 850
 $Comp
-L MCU_ST_STM32H7:STM32H753ZITx U2
+L stm32h7:STM32H753ZITx U2
 U 1 1 607C1E77
 P 8600 4450

Commit message: Add PNs to Gimletlet for easier Circuithub import
Parts:
- C1, C2: MPN (none) -> T491D226K020AT7280; Mfg (none) -> Kemet
- C10, C11, C12, C13, C14, C15, C16, C17, C18, C19, C20, C8, C9: MPN (none) -> C0603C104M4RACTU; Mfg (none) -> Kemet
- C3, C4: MPN (none) -> C0603C110J5GACTU; Mfg (none) -> Kemet
- C5, C6: MPN (none) -> C0603C225K4PACTU; Mfg (none) -> Kemet
- C7: MPN (none) -> CL10A475KQ8NNNC; Mfg (none) -> Samsung Electro-Mechanics
- D1: MPN (none) -> 150060RS75000; Mfg (none) -> Würth Elektronik
- D2: MPN (none) -> 150060AS75000; Mfg (none) -> Würth Elektronik
- D3: MPN (none) -> 150060GS75000; Mfg (none) -> Würth Elektronik
- D4: MPN (none) -> 150060BS75000; Mfg (none) -> Würth Elektronik
- F1: MPN (none) -> 1812L200/16DR; Mfg (none) -> Littelfuse Inc.
- J1: MPN (none) -> PJ-036AH-SMT-TR; Mfg (none) -> CUI Devices
- J10, J11, J12, J13, J14, J9: MPN (none) -> FR20206HBNN; Mfg (none) -> Metz Connect USA Inc.
- J15: MPN (none) -> FTSH-105-01-F-DV-K; Mfg (none) -> Samtec Inc.
- J16: MPN (none) -> RS1-09-G; Mfg (none) -> Adam Tech
- J17: MPN (none) -> RS1-07-G; Mfg (none) -> Adam Tech
- J2, J3, J4, J5: MPN (none) -> PPTC062LJBN-RC; Mfg (none) -> Sullins Connector Solutions
- J6: MPN (none) -> DF9-41S-1V(32); Mfg (none) -> Hirose Electric Co Ltd
- J7, J8: MPN (none) -> RS2-06-G; Mfg (none) -> Adam Tech
- JP1, JP2, JP3: MPN (none) -> PH1-02-UA; Mfg (none) -> Adam Tech
- R1, R10, R11, R12, R13, R14, R15, R16, R17, R18, R19, R2, R20, R21, R22, R23, R24, R25, R26, R27, R28, R29, R3, R30, R38, R5, R52, R6, R7, R9: MPN (none) -> CR0603-JW-103ELF; Mfg (none) -> Bourns Inc.
- R31, R32, R33, R34, R35, R36, R37, R39, R40, R41, R42, R43, R44, R45, R46, R47: MPN (none) -> CR0603-JW-220ELF; Mfg (none) -> Bourns Inc.
- R4, R8: MPN (none) -> CR0603-JW-104ELF; Mfg (none) -> Bourns Inc.
- R48, R49, R50, R51: MPN (none) -> CR0603-JW-680ELF; Mfg (none) -> Bourns Inc.
- SW1: MPN (none) -> PTS815 SJM 250 SMTR LFS; Mfg (none) -> C&K
- TP12, TP13, TP14, TP15, TP16, TP17, TP18, TP19, TP20, TP21, TP22, TP23: MPN (none) -> 5006; Mfg (none) -> Keystone Electronics
- U1: MPN (none) -> OKI-78SR-3.3/1.5-W36-C; Mfg (none) -> Murata Power Solutions Inc.
- U2: MPN (none) -> STM32H753ZIT6; Mfg (none) -> STMicroelectronics
- Y1: MPN (none) -> ECS-80-12-30Q-DS-TR; Mfg (none) -> ECS Inc.

Commit message: Move part-specific details to 'Comment' field for better import
Parts:
- J1: value 12V -> BarrelJack; Comment (none) -> 12V
- J10: value I2C3 -> Conn6x1; Comment (none) -> I2C3
- J11: value I2C4 -> Conn6x1; Comment (none) -> I2C4
- J12: value USART1 -> Conn6x1; Comment (none) -> USART1
- J13: value USART2 -> Conn6x1; Comment (none) -> USART2
- J14: value UART7 -> Conn6x1; Comment (none) -> UART7
- J15: Comment (none) -> SWD
- J16: value GPIO1 -> Conn9x1; Comment (none) -> GPIO1
- J17: Comment (none) -> GPIO2
- J2: value QSPI -> Conn6x2; Comment (none) -> QSPI
- J3: value SPI3 -> Conn6x2; Comment (none) -> SPI3
- J4: value SPI4 -> Conn6x2; Comment (none) -> SPI4
- J5: value SPI6 -> Conn6x2; Comment (none) -> SPI6
- J6: value NIC -> Conn41x2; Comment (none) -> NIC
- J7: value 12V -> Conn3x2; Comment (none) -> 12V
- J8: value 3V3 -> Conn3x2; Comment (none) -> 3V3
- J9: value I2C2 -> Conn6x1; Comment (none) -> I2C2
- JP1: value JACK -> Conn2x1; Comment (none) -> JACK
- JP2: value REG -> Conn2x1; Comment (none) -> REG
- JP3: value ROM -> Conn2x1; Comment (none) -> ROM
- SW1: value RESET -> Button; Comment (none) -> RESET
- TP12, TP13, TP14, TP15, TP16, TP17, TP18, TP19, TP20, TP21, TP22, TP23: value GND -> TestPoint; Comment (none) -> GND
