File: gimletlet.sch (KiCad schematic (older format))
At the start: 131 parts, among them J1 12V, J10 I2C3, J11 I2C4, J12 USART1, J13 USART2, J14 UART7, J15 SWD, J16 GPIO1, J17 Conn_01x07, J2 QSPI, J3 SPI3, J4 SPI4, J5 SPI6, J6 NIC, J7 12V, J8 3V3, J9 I2C2, SW1 RESET, U1 OKI-78SR-3.3_1.5-W36-C, U2 STM32H753ZITx, Y1 8MHz

Commit message: Add PNs to Gimletlet for easier Circuithub import (#39)
* Add PNs to Gimletlet for easier Circuithub import

* Move part-specific details to 'Comment' field for better import
Parts:
- C1, C2: MPN (none) -> T491D226K020AT7280; Mfg (none) -> Kemet
- C10, C11, C12, C13, C14, C15, C16, C17, C18, C19, C20, C8, C9: MPN (none) -> C0603C104M4RACTU; Mfg (none) -> Kemet
- C3, C4: MPN (none) -> C0603C110J5GACTU; Mfg (none) -> Kemet
- C5, C6: MPN (none) -> C0603C225K4PACTU; Mfg (none) -> Kemet
- C7: MPN (none) -> CL10A475KQ8NNNC; Mfg (none) -> Samsung Electro-Mechanics
- D1: MPN (none) -> 150060RS75000; Mfg (none) -> Würth Elektronik
- D2: MPN (none) -> 150060AS75000; Mfg (none) -> Würth Elektronik
- D3: MPN (none) -> 150060GS75000; Mfg (none) -> Würth Elektronik
- D4: MPN (none) -> 150060BS75000; Mfg (none) -> Würth Elektronik
- F1: MPN (none) -> 1812L200/16DR; Mfg (none) -> Littelfuse Inc.
- J1: value 12V -> BarrelJack; Comment (none) -> 12V; MPN (none) -> PJ-036AH-SMT-TR; Mfg (none) -> CUI Devices
- J10: value I2C3 -> Conn6x1; Comment (none) -> I2C3; MPN (none) -> FR20206HBNN; Mfg (none) -> Metz Connect USA Inc.
- J11: value I2C4 -> Conn6x1; Comment (none) -> I2C4; MPN (none) -> FR20206HBNN; Mfg (none) -> Metz Connect USA Inc.
- J12: value USART1 -> Conn6x1; Comment (none) -> USART1; MPN (none) -> FR20206HBNN; Mfg (none) -> Metz Connect USA Inc.
- J13: value USART2 -> Conn6x1; Comment (none) -> USART2; MPN (none) -> FR20206HBNN; Mfg (none) -> Metz Connect USA Inc.
- J14: value UART7 -> Conn6x1; Comment (none) -> UART7; MPN (none) -> FR20206HBNN; Mfg (none) -> Metz Connect USA Inc.
- J15: Comment (none) -> SWD; MPN (none) -> FTSH-105-01-F-DV-K; Mfg (none) -> Samtec Inc.
- J16: value GPIO1 -> Conn9x1; Comment (none) -> GPIO1; MPN (none) -> RS1-09-G; Mfg (none) -> Adam Tech
- J17: Comment (none) -> GPIO2; MPN (none) -> RS1-07-G; Mfg (none) -> Adam Tech
- J2: value QSPI -> Conn6x2; Comment (none) -> QSPI; MPN (none) -> PPTC062LJBN-RC; Mfg (none) -> Sullins Connector Solutions
- J3: value SPI3 -> Conn6x2; Comment (none) -> SPI3; MPN (none) -> PPTC062LJBN-RC; Mfg (none) -> Sullins Connector Solutions
- J4: value SPI4 -> Conn6x2; Comment (none) -> SPI4; MPN (none) -> PPTC062LJBN-RC; Mfg (none) -> Sullins Connector Solutions
- J5: value SPI6 -> Conn6x2; Comment (none) -> SPI6; MPN (none) -> PPTC062LJBN-RC; Mfg (none) -> Sullins Connector Solutions
- J6: value NIC -> Conn41x2; Comment (none) -> NIC; MPN (none) -> DF9-41S-1V(32); Mfg (none) -> Hirose Electric Co Ltd
- J7: value 12V -> Conn3x2; Comment (none) -> 12V; MPN (none) -> RS2-06-G; Mfg (none) -> Adam Tech
- J8: value 3V3 -> Conn3x2; Comment (none) -> 3V3; MPN (none) -> RS2-06-G; Mfg (none) -> Adam Tech
- J9: value I2C2 -> Conn6x1; Comment (none) -> I2C2; MPN (none) -> FR20206HBNN; Mfg (none) -> Metz Connect USA Inc.
- JP1: value JACK -> Conn2x1; Comment (none) -> JACK; MPN (none) -> PH1-02-UA; Mfg (none) -> Adam Tech
- JP2: value REG -> Conn2x1; Comment (none) -> REG; MPN (none) -> PH1-02-UA; Mfg (none) -> Adam Tech
- JP3: value ROM -> Conn2x1; Comment (none) -> ROM; MPN (none) -> PH1-02-UA; Mfg (none) -> Adam Tech
- R1, R10, R11, R12, R13, R14, R15, R16, R17, R18, R19, R2, R20, R21, R22, R23, R24, R25, R26, R27, R28, R29, R3, R30, R38, R5, R52, R6, R7, R9: MPN (none) -> CR0603-JW-103ELF; Mfg (none) -> Bourns Inc.
- R31, R32, R33, R34, R35, R36, R37, R39, R40, R41, R42, R43, R44, R45, R46, R47: MPN (none) -> CR0603-JW-220ELF; Mfg (none) -> Bourns Inc.
- R4, R8: MPN (none) -> CR0603-JW-104ELF; Mfg (none) -> Bourns Inc.
- R48, R49, R50, R51: MPN (none) -> CR0603-JW-680ELF; Mfg (none) -> Bourns Inc.
- SW1: value RESET -> Button; Comment (none) -> RESET; MPN (none) -> PTS815 SJM 250 SMTR LFS; Mfg (none) -> C&K
- TP12, TP13, TP14, TP15, TP16, TP17, TP18, TP19, TP20, TP21, TP22, TP23: value GND -> TestPoint; Comment (none) -> GND; MPN (none) -> 5006; Mfg (none) -> Keystone Electronics
- U1: MPN (none) -> OKI-78SR-3.3/1.5-W36-C; Mfg (none) -> Murata Power Solutions Inc.
- U2: MPN (none) -> STM32H753ZIT6; Mfg (none) -> STMicroelectronics
- Y1: MPN (none) -> ECS-80-12-30Q-DS-TR; Mfg (none) -> ECS Inc.
