File: dimmlet/dimmlet/dimmlet.sch (KiCad schematic (older format))
At the start: 9 parts, among them J4 Conn_01x06, U1 ‎TXB0102, U2 ‎MIC5365-2.5YC5-TR

Commit message: Incorporate rev2 changes due to rework on dimmlet. add gerbers for both spi-mux and dimmlet rev2
Parts:
- U1: value ‎TXB0102 -> ‎TXS0102; symbol dimmlet:‎TXB0102 -> dimmlet:‎TXS0102
Connections:
- net +2V5: now also U1.3 (Vcca), U1.6 (OE); no longer U1.7 (Vccb)
- net +3V3: now also U1.7 (Vccb); no longer U1.3 (Vcca), U1.6 (OE)
- net SCL: now also U1.1 (B2); no longer U1.5 (A1)
- net SCL_2V5: now also U1.4 (A2); no longer U1.8 (B1)
- net SDA: now also U1.8 (B1); no longer U1.4 (A2)
- net SDA_2V5: now also U1.5 (A1); no longer U1.1 (B2)
Other:
- note added: "The swaps here and on the other side \nmake layout easier (and match the \nreworked rev1 boards with U1 \ninstalled upside-down"
- note added: "This chip *DOES NOT WORK* unless Vcca is <= Vccb"
