File: dimmlet/dimmlet/dimmlet.kicad_pcb (KiCad board)
At the start: 2 copper layers, 204 x 20 mm, 23 parts, among them J1 Conn_01x02, J2 Conn_01x02, J3 2-2308107-0, J4 Conn_01x06, J5 Conn_01x02, J6 Conn_01x02, J7 2-2308107-0, U1 ‎TXB0102, U2 ‎MIC5365-2.5YC5-TR

Commit message: Incorporate rev2 changes due to rework on dimmlet. add gerbers for both spi-mux and dimmlet rev2
Parts:
- U1: value ‎TXB0102 -> ‎TXS0102
- turned U1 to 180 degrees
Connections:
- U1 pad 1: /SDA_2V5 -> /SCL
- U1 pad 3: +3V3 -> +2V5
- U1 pad 4: /SDA -> /SCL_2V5
- U1 pad 5: /SCL -> /SDA_2V5
- U1 pad 6: +3V3 -> +2V5
- U1 pad 7: +2V5 -> +3V3
- U1 pad 8: /SCL_2V5 -> /SDA
Routing:
- net +2V5: track 6.34 -> 9.59 mm
- net +3V3: track 11.6 -> 8.45 mm
- net GNDREF: track 11.1 -> 11.0 mm, vias 6 -> 7

Commit message: clean up commit
Parts:
- J3, J7: value 2-2308107-0 -> CONN288_2-2308107-0_TEC
