File: dimmlet/dimmlet/dimms.sch (KiCad schematic (older format))
At the start: 6 parts, among them J1 Conn_01x02, J2 Conn_01x02, J3 2-2308107-0

Commit message: Incorporate rev2 changes due to rework on dimmlet. add gerbers for both spi-mux and dimmlet rev2
Changed lines of the file:
@@
 AR Path="/6107DF6E/61278AE3" Ref="J3"  Part="6"
 AR Path="/612A90FD/61278AE3" Ref="J7"  Part="6"
-F 0 "J7" H 9450 1450 60  0000 L CNN
+F 0 "J3" H 9450 1450 60  0000 L CNN
 F 1 "2-2308107-0" H 9450 1350 60  0000 L CNN
 F 2 "footprints:2-2308107-0" H 9650 -1260 60  0001 C CNN
@@
 AR Path="/6107DF6E/61278AE9" Ref="J3"  Part="5"
 AR Path="/612A90FD/61278AE9" Ref="J7"  Part="5"
-F 0 "J7" H 8200 1450 60  0000 L CNN
+F 0 "J3" H 8200 1450 60  0000 L CNN
 F 1 "2-2308107-0" H 8200 1350 60  0000 L CNN
 F 2 "footprints:2-2308107-0" H 8400 -1260 60  0001 C CNN
@@
 AR Path="/6107DF6E/61278AEF" Ref="J3"  Part="4"
 AR Path="/612A90FD/61278AEF" Ref="J7"  Part="4"
-F 0 "J7" H 7150 1450 60  0000 L CNN
+F 0 "J3" H 7150 1450 60  0000 L CNN
 F 1 "2-2308107-0" H 7150 1350 60  0000 L CNN
 F 2 "footprints:2-2308107-0" H 7350 -1260 60  0001 C CNN
@@
 AR Path="/6107DF6E/61278AFB" Ref="J3"  Part="2"
 AR Path="/612A90FD/61278AFB" Ref="J7"  Part="2"
-F 0 "J7" H 4950 1450 60  0000 L CNN
+F 0 "J3" H 4950 1450 60  0000 L CNN
 F 1 "2-2308107-0" H 4950 1350 60  0000 L CNN
 F 2 "footprints:2-2308107-0" H 5150 -1260 60  0001 C CNN
@@
 AR Path="/6107DF6E/61278B01" Ref="J3"  Part="1"
 AR Path="/612A90FD/61278B01" Ref="J7"  Part="1"
-F 0 "J7" H 3950 1450 60  0000 L CNN
+F 0 "J3" H 3950 1450 60  0000 L CNN
 F 1 "2-2308107-0" H 3950 1350 60  0000 L CNN
 F 2 "footprints:2-2308107-0" H 4150 -1260 60  0001 C CNN
@@
 AR Path="/6107DF6E/61298937" Ref="J1"  Part="1"
 AR Path="/612A90FD/61298937" Ref="J5"  Part="1"
-F 0 "J5" H 2868 1717 50  0000 C CNN
+F 0 "J1" H 2868 1717 50  0000 C CNN
 F 1 "Conn_01x02" H 2868 1626 50  0000 C CNN
 F 2 "Connector_PinHeader_2.54mm:PinHeader_1x02_P2.54mm_Vertical" H 2950 1500 50  0001 C CNN
@@
 AR Path="/6107DF6E/61298943" Ref="R1"  Part="1"
 AR Path="/612A90FD/61298943" Ref="R3"  Part="1"
-F 0 "R3" H 2668 1346 50  0000 L CNN
+F 0 "R1" H 2668 1346 50  0000 L CNN
 F 1 "R_US" H 2668 1255 50  0000 L CNN
 F 2 "Resistor_SMD:R_0402_1005Metric_Pad0.72x0.64mm_HandSolder" V 2640 1290 50  0001 C CNN
@@
 AR Path="/6107DF6E/61298957" Ref="J2"  Part="1"
 AR Path="/612A90FD/61298957" Ref="J6"  Part="1"
-F 0 "J6" H 2868 2917 50  0000 C CNN
+F 0 "J2" H 2868 2917 50  0000 C CNN
 F 1 "Conn_01x02" H 2868 2826 50  0000 C CNN
 F 2 "Connector_PinHeader_2.54mm:PinHeader_1x02_P2.54mm_Vertical" H 2950 2700 50  0001 C CNN
@@
 AR Path="/6107DF6E/61298963" Ref="R2"  Part="1"
 AR Path="/612A90FD/61298963" Ref="R4"  Part="1"
-F 0 "R4" H 2668 2546 50  0000 L CNN
+F 0 "R2" H 2668 2546 50  0000 L CNN
 F 1 "R_US" H 2668 2455 50  0000 L CNN
 F 2 "Resistor_SMD:R_0402_1005Metric_Pad0.72x0.64mm_HandSolder" V 2640 2490 50  0001 C CNN
@@
 AR Path="/6107DF6E/61298979" Ref="C1"  Part="1"
 AR Path="/612A90FD/61298979" Ref="C2"  Part="1"
-F 0 "C2" H 2465 3746 50  0000 L CNN
+F 0 "C1" H 2465 3746 50  0000 L CNN
 F 1 "C" H 2465 3655 50  0000 L CNN
 F 2 "Capacitor_SMD:C_0402_1005Metric_Pad0.74x0.62mm_HandSolder" H 2388 3550 50  0001 C CNN
@@
 AR Path="/6107DF6E/61278AF5" Ref="J3"  Part="3"
 AR Path="/612A90FD/61278AF5" Ref="J7"  Part="3"
-F 0 "J7" H 6100 1450 60  0000 L CNN
+F 0 "J3" H 6100 1450 60  0000 L CNN
 F 1 "2-2308107-0" H 6100 1350 60  0000 L CNN
 F 2 "footprints:2-2308107-0" H 6300 -1260 60  0001 C CNN
