File: spimux/spimux.kicad_pcb (KiCad board)
At the start: 2 copper layers, 70 x 20 mm, 23 parts, among them J1 Conn_01x02, J2 Conn_01x02, J3 QSPI PMOD, J4 Connector_Generic_Conn_02x06_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, J5 Conn_01x02, J6 Conn_01x03, U1 LM1117-1.8, U2 ADG3308BCPZ, U3 TS3A27518EPW, U4 MT25QU256ABA8E12

Commit message: Add dimmlet schematic pdf that matches reworked boards. Updated spi-mux with fixed U2 pinout
Parts:
- C4: moved to B.Cu
- U2: value ADG3308BCPZ -> ADG3308BRUZ
- U4: footprint spimux:BGA-25_5x5_6.0x6.0mm -> spimux:BGA-25_5x5_6.0x8.0mm
- moved C4 13.7 mm to (137.2, 95.2), turned to 270 degrees
- moved C3 12.1 mm to (113.4, 99.2)
- moved C5 7.84 mm to (118.1, 99.1)
- moved U2 1.32 mm to (116.7, 95.1), turned to 180 degrees
Connections:
- U2 pad 1: /SP_QSPI_IO2 -> +1V8
- U2 pad 10: Net-(U2-Pad10) -> /SP_TRANS_EN
- U2 pad 11: /~SP_FLASH_RESET_L_1V8 -> GNDREF
- U2 pad 12: /SP_FLASH_CLK_1V8 -> Net-(U2-Pad12)
- U2 pad 13: /~SP_FLASH_CS_L_1V8 -> /SP_QSPI_IO3
- U2 pad 14: /SP_FLASH_DQ0_1V8 -> /SP_QSPI_IO2
- U2 pad 15: /SP_FLASH_DQ1_1V8 -> /SP_QSPI_IO1
- U2 pad 16: /SP_FLASH_DQ2_1V8 -> /SP_QSPI_IO0
- U2 pad 17: /SP_FLASH_DQ3_1V8 -> /~SP_QSPI_CS
- U2 pad 18: +1V8 -> /SP_QSPI_XTRA7
- U2 pad 19: +3V3 -> /SP_QSPI_CLK
- U2 pad 2: /SP_QSPI_IO1 -> /SP_FLASH_CLK_1V8
- U2 pad 20: /SP_QSPI_IO3 -> +3V3
- U2 pad 3: /SP_QSPI_IO0 -> /~SP_FLASH_RESET_L_1V8
- U2 pad 4: /~SP_QSPI_CS -> /~SP_FLASH_CS_L_1V8
- U2 pad 5: /SP_QSPI_CLK -> /SP_FLASH_DQ0_1V8
- U2 pad 6: /SP_QSPI_XTRA7 -> /SP_FLASH_DQ1_1V8
- U2 pad 7: Net-(U2-Pad7) -> /SP_FLASH_DQ2_1V8
- U2 pad 8: /SP_TRANS_EN -> /SP_FLASH_DQ3_1V8
- U2 pad 9: GNDREF -> Net-(U2-Pad9)
Routing:
- net /SP_QSPI_IO1: track 27.3 -> 10.5 mm
- net /SP_QSPI_IO3: track 29.9 -> 13.1 mm
- net /SP_TRANS_EN: track 92.4 -> 105.9 mm, vias 0 -> 2
- net /SP_QSPI_XTRA7: track 31.7 -> 18.4 mm, vias 0 -> 1
- net /SP_QSPI_IO0: track 14.4 -> 7.84 mm, vias 0 -> 1
- net /SP_QSPI_CLK: track 14.6 -> 9.14 mm
- net +3V3: track 68.8 -> 64.2 mm
- net /SP_QSPI_IO2: track 14.9 -> 10.9 mm, vias 0 -> 1
- net /~SP_QSPI_CS: track 9.09 -> 12.4 mm, vias 0 -> 1
- net /SP_FLASH_DQ1_1V8: track 13.1 -> 14.8 mm
- net /SP_FLASH_DQ0_1V8: track 11.1 -> 12.8 mm
- net /SP_FLASH_DQ3_1V8: track 12.4 -> 14.1 mm
- net /~SP_FLASH_CS_L_1V8: track 9.40 -> 11.1 mm
- net /~SP_FLASH_RESET_L_1V8: track 21.5 -> 23.1 mm
- net /SP_FLASH_DQ2_1V8: track 13.5 -> 15.2 mm
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Other:
- net class Default: trace_width 0.15 -> 0.16
- rule trace_min: 0.1 -> 0.16

Commit message: Adding rev2 spimux stuff
Parts:
- H1: footprint MountingHole:MountingHole_2.2mm_M2_DIN965_Pad -> MountingHole:MountingHole_3.2mm_M3_Pad
- moved H1 3.94 mm to (170.4, 99.8)
Routing:
- net /~SP_QSPI_CS: track 12.4 -> 11.5 mm
- net +1V8: track 72.5 -> 71.8 mm
- net /SP_TRANS_EN: track 105.9 -> 105.3 mm
Other:
- board size 70 x 20 mm -> 75 x 20 mm
- net class Default: clearance 0.1 -> 0.153
- rule trace_clearance: 0.1 -> 0.153
- board text added: "Jumper section: Hold my beer I got this!"
- board text removed: "Hold my beer I got this!"
