File: spimux/spimux.sch (KiCad schematic (older format))
At the start: 21 parts, among them J1 Conn_01x02, J2 Conn_01x02, J3 Connector_Generic_Conn_02x06_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, J4 Connector_Generic_Conn_02x06_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, J5 Conn_01x02, J6 Conn_01x03, U1 LM1117-1.8, U2 ADG3308BCPZ, U3 TS3A27518EPW, U4 MT25QU256ABA8E12

Commit message: Add spimux files sent out for production. Add dimmlet files
Parts:
- added H1: MountingHole_Pad, MountingHole:MountingHole_2.2mm_M2_DIN965_Pad, symbol Mechanical:MountingHole_Pad
- C1, C2: footprint (none) -> Capacitor_SMD:CP_Elec_5x5.3; MPN (none) -> EDK106M050A9DAA; Source (none) -> Digikey
- C3, C4, C5, C6: footprint (none) -> Capacitor_SMD:C_0402_1005Metric
- J1, J2, J5: footprint (none) -> Connector_PinHeader_2.54mm:PinHeader_1x02_P2.54mm_Vertical; MPN (none) -> PRPC024SAAN-RC
- J3: value Connector_Generic_Conn_02x06_Top_Bottom -> QSPI PMOD; footprint (none) -> pmod:PMOD_12pin_peripheral_horizontal
- J4: footprint (none) -> Connector_PinHeader_2.54mm:PinHeader_2x06_P2.54mm_Vertical
- J6: footprint (none) -> Connector_PinHeader_2.54mm:PinHeader_1x03_P2.54mm_Vertical; MPN (none) -> PRPC024SAAN-RC
- R1, R2, R3, R4, R5: footprint (none) -> Resistor_SMD:R_0402_1005Metric
- U1: footprint (none) -> Package_TO_SOT_SMD:SOT-223; MPN (none) -> LM1117MPX-18NOPB
- U2: footprint (none) -> Package_SO:TSSOP-20_4.4x6.5mm_P0.65mm; MPN (none) -> ADG3308BRUZ; Source (none) -> Digikey
- U3: MPN (none) -> TS3A27518EPWR; Source (none) -> Mouser
- U4: footprint (none) -> spimux:BGA-25_5x5_6.0x6.0mm
Connections:
- wire segments 130 -> 131
Changed lines of the file:
@@
 F 0 "U4" H 14100 3600 50  0000 L CNN
 F 1 "MT25QU256ABA8E12" H 14150 2000 50  0000 L CNN
-F 2 "" H 14000 3350 50  0001 C CNN
+F 2 "spimux:BGA-25_5x5_6.0x6.0mm" H 14000 3350 50  0001 C CNN
 F 3 "" H 14000 3350 50  0001 C CNN
 	1    14000 3350
@@
 F 0 "R5" H 13668 3246 50  0000 L CNN
 F 1 "10k" H 13668 3155 50  0000 L CNN
-F 2 "" V 13640 3190 50  0001 C CNN
+F 2 "Resistor_SMD:R_0402_1005Metric" V 13640 3190 50  0001 C CNN
 F 3 "~" H 13600 3200 50  0001 C CNN
 	1    13600 3200
@@
 F 0 "R4" H 13418 3246 50  0000 L CNN
 F 1 "10k" H 13418 3155 50  0000 L CNN
-F 2 "" V 13390 3190 50  0001 C CNN
+F 2 "Resistor_SMD:R_0402_1005Metric" V 13390 3190 50  0001 C CNN
 F 3 "~" H 13350 3200 50  0001 C CNN
 	1    13350 3200
@@
 F 0 "C5" H 12515 5446 50  0000 L CNN
 F 1 "1uF" H 12515 5355 50  0000 L CNN
-F 2 "" H 12438 5250 50  0001 C CNN
+F 2 "Capacitor_SMD:C_0402_1005Metric" H 12438 5250 50  0001 C CNN
 F 3 "~" H 12400 5400 50  0001 C CNN
 	1    12400 5400
@@
 F 0 "C6" H 12915 5446 50  0000 L CNN
 F 1 "1uF" H 12915 5355 50  0000 L CNN
-F 2 "" H 12838 5250 50  0001 C CNN
+F 2 "Capacitor_SMD:C_0402_1005Metric" H 12838 5250 50  0001 C CNN
 F 3 "~" H 12800 5400 50  0001 C CNN
 	1    12800 5400
@@
 P 1650 4450
 F 0 "J3" H 1700 4867 50  0000 C CNN
-F 1 "Connector_Generic_Conn_02x06_Top_Bottom" H 1700 4776 50  0000 C CNN
-F 2 "" H 1650 4450 50  0001 C CNN
+F 1 "QSPI PMOD" H 1700 4776 50  0000 C CNN
+F 2 "pmod:PMOD_12pin_peripheral_horizontal" H 1650 4450 50  0001 C CNN
 F 3 "" H 1650 4450 50  0001 C CNN
 	1    1650 4450
@@
 F 0 "U2" H 7150 3765 50  0000 C CNN
 F 1 "ADG3308BCPZ" H 7150 3674 50  0000 C CNN
-F 2 "" H 6700 3500 50  0001 C CNN
+F 2 "Package_SO:TSSOP-20_4.4x6.5mm_P0.65mm" H 6700 3500 50  0001 C CNN
 F 3 "" H 6700 3500 50  0001 C CNN
+F 4 "ADG3308BRUZ" H 6700 3500 50  0001 C CNN "MPN"
+F 5 "Digikey" H 6700 3500 50  0001 C CNN "Source"
 	1    6700 3500
 	-1   0    0    -1
@@
 F 0 "C3" H 6165 5296 50  0000 L CNN
 F 1 "1uF" H 6165 5205 50  0000 L CNN
-F 2 "" H 6088 5100 50  0001 C CNN
+F 2 "Capacitor_SMD:C_0402_1005Metric" H 6088 5100 50  0001 C CNN
 F 3 "~" H 6050 5250 50  0001 C CNN
 	1    6050 5250
@@
 F 0 "C4" H 6565 5296 50  0000 L CNN
 F 1 "1uF" H 6565 5205 50  0000 L CNN
-F 2 "" H 6488 5100 50  0001 C CNN
+F 2 "Capacitor_SMD:C_0402_1005Metric" H 6488 5100 50  0001 C CNN
 F 3 "~" H 6450 5250 50  0001 C CNN
 	1    6450 5250
@@
 F 2 "Package_SO:TSSOP-24_4.4x7.8mm_P0.65mm" H 10500 5250 50  0001 C CNN
 F 3 "http://www.ti.com/lit/ds/symlink/ts3a27518e.pdf" H 10500 4150 50  0001 C CNN
+F 4 "TS3A27518EPWR" H 10500 4250 50  0001 C CNN "MPN"
+F 5 "Mouser" H 10500 4250 50  0001 C CNN "Source"
 	1    10500 4250
 	-1   0    0    -1
@@
 F 0 "J1" H 718 8767 50  0000 C CNN
 F 1 "Conn_01x02" H 718 8676 50  0000 C CNN
-F 2 "" H 800 8550 50  0001 C CNN
+F 2 "Connector_PinHeader_2.54mm:PinHeader_1x02_P2.54mm_Vertical" H 800 8550 50  0001 C CNN
 F 3 "~" H 800 8550 50  0001 C CNN
+F 4 "PRPC024SAAN-RC" H 800 8550 50  0001 C CNN "MPN"
 	1    800  8550
 	-1   0    0    -1
@@
 F 0 "R1" H 1218 8896 50  0000 L CNN
 F 1 "10k" H 1218 8805 50  0000 L CNN
-F 2 "" V 1190 8840 50  0001 C CNN
+F 2 "Resistor_SMD:R_0402_1005Metric" V 1190 8840 50  0001 C CNN
 F 3 "~" H 1150 8850 50  0001 C CNN
 	1    1150 8850
@@
 F 0 "R2" H 1968 9346 50  0000 L CNN
 F 1 "10k" H 1968 9255 50  0000 L CNN
-F 2 "" V 1940 9290 50  0001 C CNN
+F 2 "Resistor_SMD:R_0402_1005Metric" V 1940 9290 50  0001 C CNN
 F 3 "~" H 1900 9300 50  0001 C CNN
 	1    1900 9300
@@
 F 0 "J2" H 1468 9767 50  0000 C CNN
 F 1 "Conn_01x02" H 1468 9676 50  0000 C CNN
-F 2 "" H 1550 9550 50  0001 C CNN
+F 2 "Connector_PinHeader_2.54mm:PinHeader_1x02_P2.54mm_Vertical" H 1550 9550 50  0001 C CNN
 F 3 "~" H 1550 9550 50  0001 C CNN
+F 4 "PRPC024SAAN-RC" H 1550 9550 50  0001 C CNN "MPN"
 	1    1550 9550
 	-1   0    0    -1
@@
 F 0 "J4" H 1700 6817 50  0000 C CNN
 F 1 "Connector_Generic_Conn_02x06_Top_Bottom" H 1700 6726 50  0000 C CNN
-F 2 "" H 1650 6400 50  0001 C CNN
+F 2 "Connector_PinHeader_2.54mm:PinHeader_2x06_P2.54mm_Vertical" H 1650 6400 50  0001 C CNN
 F 3 "" H 1650 6400 50  0001 C CNN
 	1    1650 6400
@@
 F 0 "U1" H 3550 2442 50  0000 C CNN
 F 1 "LM1117-1.8" H 3550 2351 50  0000 C CNN
-F 2 "" H 3550 2200 50  0001 C CNN
+F 2 "Package_TO_SOT_SMD:SOT-223" H 3550 2200 50  0001 C CNN
 F 3 "http://www.ti.com/lit/ds/symlink/lm1117.pdf" H 3550 2200 50  0001 C CNN
+F 4 "LM1117MPX-18NOPB" H 3550 2200 50  0001 C CNN "MPN"
 	1    3550 2200
 	1    0    0    -1
@@
 F 0 "C1" H 2991 2446 50  0000 L CNN
 F 1 "10uF" H 2991 2355 50  0000 L CNN
-F 2 "" H 2900 2400 50  0001 C CNN
+F 2 "Capacitor_SMD:CP_Elec_5x5.3" H 2900 2400 50  0001 C CNN
 F 3 "~" H 2900 2400 50  0001 C CNN
+F 4 "EDK106M050A9DAA" H 2900 2400 50  0001 C CNN "MPN"
+F 5 "Digikey" H 2900 2400 50  0001 C CNN "Source"
 	1    2900 2400
 	1    0    0    -1
@@
 F 0 "C2" H 4241 2446 50  0000 L CNN
 F 1 "10uF" H 4241 2355 50  0000 L CNN
-F 2 "" H 4150 2400 50  0001 C CNN
+F 2 "Capacitor_SMD:CP_Elec_5x5.3" H 4150 2400 50  0001 C CNN
 F 3 "~" H 4150 2400 50  0001 C CNN
+F 4 "EDK106M050A9DAA" H 4150 2400 50  0001 C CNN "MPN"
+F 5 "Digikey" H 4150 2400 50  0001 C CNN "Source"
 	1    4150 2400
 	1    0    0    -1
@@
 F 0 "J5" H 4968 8717 50  0000 C CNN
 F 1 "Conn_01x02" H 4968 8626 50  0000 C CNN
-F 2 "" H 5050 8500 50  0001 C CNN
+F 2 "Connector_PinHeader_2.54mm:PinHeader_1x02_P2.54mm_Vertical" H 5050 8500 50  0001 C CNN
 F 3 "~" H 5050 8500 50  0001 C CNN
+F 4 "PRPC024SAAN-RC" H 5050 8500 50  0001 C CNN "MPN"
 	1    5050 8500
 	-1   0    0    -1
@@
 F 0 "R3" H 5468 8846 50  0000 L CNN
 F 1 "10k" H 5468 8755 50  0000 L CNN
-F 2 "" V 5440 8790 50  0001 C CNN
+F 2 "Resistor_SMD:R_0402_1005Metric" V 5440 8790 50  0001 C CNN
 F 3 "~" H 5400 8800 50  0001 C CNN
 	1    5400 8800
@@
 F 0 "J6" H 6780 8542 50  0000 L CNN
 F 1 "Conn_01x03" H 6780 8451 50  0000 L CNN
-F 2 "" H 6700 8500 50  0001 C CNN
+F 2 "Connector_PinHeader_2.54mm:PinHeader_1x03_P2.54mm_Vertical" H 6700 8500 50  0001 C CNN
 F 3 "~" H 6700 8500 50  0001 C CNN
+F 4 "PRPC024SAAN-RC" H 6700 8500 50  0001 C CNN "MPN"
 	1    6700 8500
 	1    0    0    -1
@@
 Text Notes 3350 4250 0    50   ~ 0
 (~SP_FLASH_RESET_L)
+$Comp
+L Mechanical:MountingHole_Pad H1
+U 1 1 60F345F9
+P 9050 6500
+F 0 "H1" H 9150 6549 50  0000 L CNN
+F 1 "MountingHole_Pad" H 9150 6458 50  0000 L CNN
+F 2 "MountingHole:MountingHole_2.2mm_M2_DIN965_Pad" H 9050 6500 50  0001 C CNN
+F 3 "~" H 9050 6500 50  0001 C CNN
+	1    9050 6500
+	1    0    0    -1
+$EndComp
+$Comp
+L power:GNDREF #PWR0101
+U 1 1 60F35A7B
+P 9050 6700
+F 0 "#PWR0101" H 9050 6450 50  0001 C CNN
+F 1 "GNDREF" H 9055 6527 50  0000 C CNN
+F 2 "" H 9050 6700 50  0001 C CNN
+F 3 "" H 9050 6700 50  0001 C CNN
+	1    9050 6700
+	1    0    0    -1
+$EndComp
+Wire Wire Line
+	9050 6700 9050 6600
 $EndSCHEMATC

Commit message: Add dimmlet schematic pdf that matches reworked boards. Updated spi-mux with fixed U2 pinout
Parts:
- removed U2: ADG3308BCPZ, Package_SO:TSSOP-20_4.4x6.5mm_P0.65mm, symbol oxide_spimux:ADG3308BCPZ
- added U2: ADG3308BRUZ, Package_SO:TSSOP-20_4.4x6.5mm_P0.65mm, symbol oxide_spimux:ADG3308BRUZ
- U4: footprint spimux:BGA-25_5x5_6.0x6.0mm -> spimux:BGA-25_5x5_6.0x8.0mm
Connections:
- wire segments 131 -> 139
Changed lines of the file:
@@
 F 0 "U4" H 14100 3600 50  0000 L CNN
 F 1 "MT25QU256ABA8E12" H 14150 2000 50  0000 L CNN
-F 2 "spimux:BGA-25_5x5_6.0x6.0mm" H 14000 3350 50  0001 C CNN
+F 2 "spimux:BGA-25_5x5_6.0x8.0mm" H 14000 3350 50  0001 C CNN
 F 3 "" H 14000 3350 50  0001 C CNN
 	1    14000 3350
@@
 	1950 4750 2800 4750
 Wire Wire Line
+	5100 4250 5700 4250
+Wire Wire Line
+	5100 4150 5700 4150
+Wire Wire Line
+	5100 4050 5700 4050
+Wire Wire Line
+	5100 3950 5700 3950
+Wire Wire Line
+	5100 3850 5700 3850
+Wire Wire Line
 	5100 3650 5700 3650
-Wire Wire Line
-	5100 3750 5700 3750
-Wire Wire Line
-	5100 3850 5700 3850
-Wire Wire Line
-	5100 3950 5700 3950
-Wire Wire Line
-	5100 4050 5700 4050
-Wire Wire Line
-	5100 4150 5700 4150
-Text Label 5150 3650 0    50   ~ 0
+Text Label 5150 4250 0    50   ~ 0
 SP_QSPI_IO3
-Text Label 5150 3750 0    50   ~ 0
+Text Label 5150 4150 0    50   ~ 0
 SP_QSPI_IO2
-Text Label 5150 3850 0    50   ~ 0
+Text Label 5150 4050 0    50   ~ 0
 SP_QSPI_IO1
 Text Label 5150 3950 0    50   ~ 0
 SP_QSPI_IO0
-Text Label 5150 4050 0    50   ~ 0
+Text Label 5150 3850 0    50   ~ 0
 ~SP_QSPI_CS
-Text Label 5150 4150 0    50   ~ 0
+Text Label 5150 3650 0    50   ~ 0
 SP_QSPI_CLK
 Wire Wire Line
@@
 Text Label 11300 4350 0    50   ~ 0
 ~SPI_MUX_EN_L
-$Comp
-L oxide_spimux:ADG3308BCPZ U2
-U 1 1 60F6D145
-P 6700 3500
-F 0 "U2" H 7150 3765 50  0000 C CNN
-F 1 "ADG3308BCPZ" H 7150 3674 50  0000 C CNN
-F 2 "Package_SO:TSSOP-20_4.4x6.5mm_P0.65mm" H 6700 3500 50  0001 C CNN
-F 3 "" H 6700 3500 50  0001 C CNN
-F 4 "ADG3308BRUZ" H 6700 3500 50  0001 C CNN "MPN"
-F 5 "Digikey" H 6700 3500 50  0001 C CNN "Source"
-	1    6700 3500
-	-1   0    0    -1
-$EndComp
 $Comp
 L power:+1V8 #PWR020
@@
 Wire Wire Line
 	6950 3500 6950 3400
-Wire Wire Line
-	5700 3500 5500 3500
-Wire Wire Line
-	5500 3500 5500 3400
 $Comp
 L power:GNDREF #PWR021
@@
 $EndComp
 Wire Wire Line
-	6800 4600 6950 4600
-Wire Wire Line
-	6950 4600 6950 4700
-Wire Wire Line
 	6800 4500 6950 4500
-Wire Wire Line
-	6950 4500 6950 4600
-Connection ~ 6950 4600
 $Comp
 L power:+3.3V #PWR017
@@
 Wire Wire Line
 	6050 5400 6050 5450
-Text Label 7900 3650 0    50   ~ 0
+Text Label 8400 3650 0    50   ~ 0
 SP_FLASH_DQ3_1V8
-Text Label 7900 3750 0    50   ~ 0
+Text Label 8400 3750 0    50   ~ 0
 SP_FLASH_DQ2_1V8
-Text Label 7900 3850 0    50   ~ 0
+Text Label 8400 3850 0    50   ~ 0
 SP_FLASH_DQ1_1V8
-Text Label 7900 3950 0    50   ~ 0
+Text Label 8400 3950 0    50   ~ 0
 SP_FLASH_DQ0_1V8
-Text Label 7900 4050 0    50   ~ 0
+Text Label 6800 3850 0    50   ~ 0
 ~SP_FLASH_CS_L_1V8
-Text Label 7900 4150 0    50   ~ 0
+Text Label 8400 4150 0    50   ~ 0
 SP_FLASH_CLK_1V8
-Text Label 6900 4250 0    50   ~ 0
-~SP_FLASH_RESET_L_1V8
-Wire Wire Line
-	6800 4250 7800 4250
 Wire Wire Line
 	13600 3350 13600 3550
@@
 	11200 4550 11250 4550
 Wire Wire Line
-	6800 3850 9800 3850
-Wire Wire Line
-	9800 4150 6800 4150
-Wire Wire Line
-	9800 3950 6800 3950
-Wire Wire Line
 	11200 4350 11900 4350
 Wire Wire Line
-	6800 3650 9800 3650
-Wire Wire Line
-	6800 4050 9800 4050
-Wire Wire Line
 	11250 4650 11200 4650
 Wire Wire Line
@@
 Wire Wire Line
 	11200 4050 14000 4050
-Wire Wire Line
-	9800 3750 6800 3750
 $Comp
 L Analog_Switch:TS3A27518EPW U3
@@
 	1150 8350 1150 8550
 Wire Wire Line
-	1950 4250 5700 4250
+	1950 4250 4500 4250
 Text Notes 1200 3800 0    50   ~ 0
 Matches gimletlet QSPI Header.\nXTRA7 is ~FLASH_RESET_L\nXTRA10 is SP_FLASH_MUX_SELECT
@@
 Wire Wire Line
 	9050 6700 9050 6600
+$Comp
+L oxide_spimux:ADG3308BRUZ U2
+U 1 1 610B68DB
+P 5800 3500
+F 0 "U2" H 6250 3765 50  0000 C CNN
+F 1 "ADG3308BRUZ" H 6250 3674 50  0000 C CNN
+F 2 "Package_SO:TSSOP-20_4.4x6.5mm_P0.65mm" H 5800 3500 50  0001 C CNN
+F 3 "" H 5800 3500 50  0001 C CNN
+	1    5800 3500
+	1    0    0    -1
+$EndComp
+Wire Wire Line
+	6950 4500 6950 4700
+Wire Wire Line
+	6800 4250 7850 4250
+Wire Wire Line
+	7850 3650 9800 3650
+Wire Wire Line
+	7750 3750 7750 4150
+Wire Wire Line
+	7750 4150 6800 4150
+Wire Wire Line
+	7650 3850 9800 3850
+Wire Wire Line
+	7750 3750 9800 3750
+Wire Wire Line
+	7650 3850 7650 4050
+Wire Wire Line
+	7650 4050 6800 4050
+Wire Wire Line
+	7850 3650 7850 4250
+Wire Wire Line
+	9800 3950 6800 3950
+Text Label 8400 4050 0    50   ~ 0
+~SP_FLASH_CS_L_1V8
+Wire Wire Line
+	8400 4050 9800 4050
+Wire Wire Line
+	8400 4150 9800 4150
+Wire Wire Line
+	6800 3850 7550 3850
+Wire Wire Line
+	6800 3650 7550 3650
+Text Label 6800 3650 0    50   ~ 0
+SP_FLASH_CLK_1V8
+Wire Wire Line
+	7550 3750 6800 3750
+Text Label 6800 3750 0    50   ~ 0
+~SP_FLASH_RESET_L_1V8
+Wire Wire Line
+	5700 3500 5500 3500
+Wire Wire Line
+	5500 3500 5500 3400
+Wire Wire Line
+	5700 3750 4500 3750
+Wire Wire Line
+	4500 3750 4500 4250
 $EndSCHEMATC

Commit message: Adding rev2 spimux stuff
Parts:
- H1: footprint MountingHole:MountingHole_2.2mm_M2_DIN965_Pad -> MountingHole:MountingHole_3.2mm_M3_Pad
Changed lines of the file:
@@
 F 0 "H1" H 9150 6549 50  0000 L CNN
 F 1 "MountingHole_Pad" H 9150 6458 50  0000 L CNN
-F 2 "MountingHole:MountingHole_2.2mm_M2_DIN965_Pad" H 9050 6500 50  0001 C CNN
+F 2 "MountingHole:MountingHole_3.2mm_M3_Pad" H 9050 6500 50  0001 C CNN
 F 3 "~" H 9050 6500 50  0001 C CNN
 	1    9050 6500
