File: nic2/nic2.kicad_pcb (KiCad board)
At the start: 4 copper layers, 70.8 x 47 mm, 37 parts, among them J1 Conn_2Rows-41Pins, J2 Wuerth_74980111211, J3 Wuerth_74980111211, U1 KSZ8463FRLI, X1 ASE-25.000MHZ-LC

Commit message: Tweaks to NIC before review
Parts:
- added C14: 10 µF, Capacitor_SMD:C_0805_2012Metric, F.Cu at (178.5, 80.0)
- added D3: LED, LED_SMD:LED_0402_1005Metric, F.Cu at (169.2, 60.0)
- added R12: 143Ω, Resistor_SMD:R_0402_1005Metric, F.Cu at (169.2, 61.2)
- added TP1: TestPoint, TestPoint:TestPoint_Pad_2.5x2.5mm, F.Cu at (165.8, 60.5)
- added TP2: TestPoint, TestPoint:TestPoint_Pad_2.5x2.5mm, F.Cu at (160.6, 60.5)
- C2: footprint Capacitor_SMD:C_0402_1005Metric -> Capacitor_SMD:C_0805_2012Metric
- moved C2 1.77 mm to (157.8, 68.8), turned to 90 degrees
Routing:
- net GND: track 45.9 -> 50.6 mm, vias 29 -> 32
- net +3V3: track 31.4 -> 36.1 mm, vias 19 -> 21
- net Net-(C2-Pad2): track 12.7 -> 14.8 mm
- net Net-(D3-Pad1): track 0.00 -> 1.26 mm
Other:
- board text added: "+3V3"
- board text added: "GND"

Commit message: Update NIC2 per review
Parts:
- removed C2: 10 µF, Capacitor_SMD:C_0805_2012Metric
- removed D1, D2: 1N4148W, Diode_SMD:D_SOD-123
- added TP3: TestPoint, TestPoint:TestPoint_Keystone_5015_Micro-Minature, F.Cu at (164.5, 62.8)
- added TP5: TestPoint, TestPoint:TestPoint_Keystone_5015_Micro-Minature, F.Cu at (169.2, 65.8)
- added TP6: TestPoint, TestPoint:TestPoint_Keystone_5015_Micro-Minature, F.Cu at (164.5, 65.8)
- added TP7: TestPoint, TestPoint:TestPoint_Keystone_5015_Micro-Minature, F.Cu at (169.2, 59.8)
- added TP8: TestPoint, TestPoint:TestPoint_Keystone_5015_Micro-Minature, F.Cu at (169.2, 62.8)
- added U2: TPD4S010DQAR, Package_SON:USON-10_2.5x1.0mm_P0.5mm, F.Cu at (149.0, 68.5)
- added U3: TPD4S010DQAR, Package_SON:USON-10_2.5x1.0mm_P0.5mm, F.Cu at (149.0, 90.8)
- TP2: footprint TestPoint:TestPoint_Pad_2.5x2.5mm -> TestPoint:TestPoint_Keystone_5015_Micro-Minature
- moved D3 12.6 mm to (157.2, 63.8)
- moved R12 12.6 mm to (157.2, 65.0)
- moved TP1 12.6 mm to (153.8, 64.2)
- moved R2 4.37 mm to (159.0, 70.0)
- moved TP2 4.05 mm to (164.5, 59.8)
Connections:
- R2 pad 1: Net-(C2-Pad2) -> GND
- R2 pad 2: +3V3 -> /~{SPI4_RESET}
- U1 pad 63: Net-(C2-Pad2) -> /~{SPI4_RESET}
Routing:
- net /SPI4_MISO: track 21.3 -> 43.8 mm, vias 3 -> 4
- net /~{SPI4_CS}: track 17.0 -> 39.1 mm, vias 1 -> 3
- net /SPI4_MOSI: track 23.7 -> 38.6 mm
- net Net-(C2-Pad2): track 14.8 -> 0.00 mm
- net /~{SPI4_RESET}: track 27.6 -> 40.7 mm
- net /SPI4_SCK: track 22.5 -> 34.3 mm, vias 3 -> 4
- net GND: track 50.6 -> 55.4 mm, vias 32 -> 34
- net +3V3: track 36.1 -> 39.5 mm, vias 21 -> 19
- net /RX2_P: track 22.0 -> 24.8 mm
- net /RX2_N: track 22.0 -> 24.8 mm
- net /TX1_P: track 16.9 -> 19.5 mm
- net /TX1_N: track 16.8 -> 19.4 mm
- net /RX1_N: track 17.5 -> 20.0 mm
- net /RX1_P: track 17.5 -> 19.9 mm
- net /P1LED0: track 22.8 -> 24.7 mm
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Other:
- board text added: "CS"
- board text added: "MISO"
- board text added: "MOSI"
- board text added: "RST"
- board text added: "SCK"

Commit message: Add Oxide wordmark
Parts:
- added LOGO1: LOGO, Logos_0x:OXIDE_Wordmark, F.Cu at (165.0, 89.6)
Other:
- board text added: "Gimletlet NIC 2 Rev A MJK 1/2022"
- board text removed: "Gimletlet NIC 2 Rev A MJK 12/2021"

Commit message: Exporting gerbers for NIC2 order
Parts:
- moved FID3 11.6 mm to (184.2, 93.0)
- moved FID2 11.2 mm to (184.2, 63.8)
- moved D3 2.30 mm to (155.8, 62.0)
- moved R12 2.30 mm to (155.8, 63.2)
- moved TP1 2.30 mm to (152.2, 62.5)
- moved TP2 1.36 mm to (164.0, 58.5)
- moved TP7 1.26 mm to (169.4, 58.5)
- moved TP3 0.92 mm to (164.0, 62.0)
- moved TP8 0.76 mm to (169.4, 62.0)
- moved TP6 0.50 mm to (164.0, 65.8)
- moved TP5 0.25 mm to (169.5, 65.8)
Routing:
- net /SPI4_MISO: track 43.8 -> 45.1 mm
- net /~{SPI4_CS}: track 39.1 -> 40.0 mm
- net /SPI4_MOSI: track 38.6 -> 39.3 mm
- net /SPI4_SCK: track 34.3 -> 34.8 mm

Commit message: Updates to NIC
Parts:
- removed TP1: TestPoint, TestPoint:TestPoint_Pad_2.5x2.5mm
- removed TP2, TP3, TP5, TP6, TP7, TP8: TestPoint, TestPoint:TestPoint_Keystone_5015_Micro-Minature
- added D1: LED, LED_SMD:LED_0402_1005Metric, F.Cu at (169.2, 95.7)
- added D2: LED, LED_SMD:LED_0402_1005Metric, F.Cu at (169.2, 94.5)
- added D4: LED, LED_SMD:LED_0402_1005Metric, F.Cu at (169.2, 92.0)
- added D5: LED, LED_SMD:LED_0402_1005Metric, F.Cu at (149.2, 56.8)
- added H3: MountingHole_Pad, MountingHole:MountingHole_3.2mm_M3_DIN965_Pad, F.Cu at (122.0, 51.0)
- added H4: MountingHole_Pad, MountingHole:MountingHole_3.2mm_M3_DIN965_Pad, F.Cu at (122.0, 106.2)
- added J4: Conn_01x07_Male, Connector_PinHeader_2.54mm:PinHeader_1x07_P2.54mm_Vertical, F.Cu at (167.4, 57.5)
- added R13: 143Ω, Resistor_SMD:R_0402_1005Metric, F.Cu at (171.2, 95.7)
- added R14: 143Ω, Resistor_SMD:R_0402_1005Metric, F.Cu at (171.2, 94.5)
- added R15: 143Ω, Resistor_SMD:R_0402_1005Metric, F.Cu at (171.2, 93.2)
- added R16: 143Ω, Resistor_SMD:R_0402_1005Metric, F.Cu at (171.2, 92.0)
- C13, R11: moved to B.Cu
- FB1: footprint Resistor_SMD:R_0603_1608Metric -> Resistor_SMD:R_0402_1005Metric
- moved D3 34.0 mm to (169.2, 93.2)
- moved R12 8.36 mm to (149.2, 58.0)
- moved LOGO1 7.32 mm to (157.7, 90.6)
- moved C13 3.14 mm to (140.6, 77.8)
- moved R11 3.14 mm to (140.6, 79.0)
- moved FID1 1.75 mm to (143.2, 57.5)
Connections:
- D3 pad 2: +3V3 -> Net-(D3-Pad2)
- R12 pad 2: Net-(D3-Pad1) -> Net-(D5-Pad1)
- U1 pad 52: unconnected-(U1-Pad52) -> Net-(D4-Pad2)
- U1 pad 53: unconnected-(U1-Pad53) -> Net-(D3-Pad2)
- U1 pad 54: unconnected-(U1-Pad54) -> Net-(D2-Pad2)
- U1 pad 55: unconnected-(U1-Pad55) -> Net-(D1-Pad2)
Routing:
- net Net-(D1-Pad2): track 0.00 -> 30.9 mm, vias 0 -> 2
- net Net-(D2-Pad2): track 0.00 -> 28.5 mm, vias 0 -> 2
- net Net-(D3-Pad2): track 0.00 -> 25.6 mm, vias 0 -> 2
- net Net-(D4-Pad2): track 0.00 -> 24.0 mm, vias 0 -> 2
- net /SPI4_SCK: track 34.8 -> 48.7 mm
- net /SPI4_MOSI: track 39.3 -> 50.2 mm, vias 3 -> 5
- net Earth: track 3.80 -> 11.3 mm, vias 0 -> 23
- net /SPI4_MISO: track 45.1 -> 50.3 mm
- net /~{SPI4_RESET}: track 40.7 -> 45.7 mm, vias 1 -> 2
- net /~{SPI4_CS}: track 40.0 -> 42.7 mm, vias 3 -> 1
- net +3V3: track 39.5 -> 37.5 mm, vias 19 -> 18
- net /P1LED0: track 24.7 -> 22.8 mm
- net Net-(D5-Pad1): track 0.00 -> 1.26 mm
- net GND: track 55.4 -> 56.4 mm, vias 34 -> 37
- net Net-(D2-Pad1): track 0.00 -> 1.01 mm
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- added copper zone on B.Cu, net Earth
- added copper zone on In1.Cu, net Earth
- added copper zone on In2.Cu, net Earth
Other:
- board size 70.8 x 47 mm -> 70.8 x 66.5 mm
- board text added: "3V3"
- board text added: "Gimletlet NIC 2 Rev B MJK 4/2022"
- board text added: "PORT 1"
- board text added: "PORT 2"
- board text removed: "+3V3"
- board text removed: "Gimletlet NIC 2 Rev A MJK 1/2022"

Commit message: Add NRST LED
Parts:
- added D6: LED, LED_SMD:LED_0402_1005Metric, F.Cu at (170.5, 60.5)
- added R17: 143Ω, Resistor_SMD:R_0402_1005Metric, F.Cu at (170.5, 61.5)
- moved D5 4.23 mm to (152.2, 59.8)
- moved R12 4.23 mm to (152.2, 61.0)
Routing:
- net /~{SPI4_RESET}: track 45.7 -> 50.8 mm
- net +3V3: track 37.5 -> 39.2 mm, vias 18 -> 17
- net Net-(D6-Pad1): track 0.00 -> 1.01 mm
- net GND: track 56.4 -> 57.2 mm, vias 37 -> 38
Other:
- board text added: "~{RST}"
- board text removed: "RST"

Commit message: Fix LED colors in BOM
Parts:
- D1: value LED -> LED_RED
- D2: value LED -> LED_ORANGE
- D3, D5, D6: value LED -> LED_GREEN
- D4: value LED -> LED_BLUE
Changed lines of the file:
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@@
     (tags "LED")
     (property "MFG" "SunLed")
-    (property "MPN" "XZVGR68W-3")
+    (property "MPN" "XZVG68W-2")
     (property "Sheetfile" "nic2.kicad_sch")
     (property "Sheetname" "")
@@
       (effects (font (size 1 1) (thickness 0.15)))
     )
-    (fp_text value "LED" (at 0 1.17) (layer "F.Fab")
+    (fp_text value "LED_GREEN" (at 0 1.17) (layer "F.Fab")
       (effects (font (size 1 1) (thickness 0.15)))
     )
@@
       (effects (font (size 1 1) (thickness 0.15)))
     )
-    (fp_text value "LED" (at 0 1.17) (layer "F.Fab")
+    (fp_text value "LED_ORANGE" (at 0 1.17) (layer "F.Fab")
       (effects (font (size 1 1) (thickness 0.15)))
     )
@@
       (effects (font (size 1 1) (thickness 0.15)))
     )
-    (fp_text value "LED" (at 0 1.17) (layer "F.Fab")
+    (fp_text value "LED_GREEN" (at 0 1.17) (layer "F.Fab")
       (effects (font (size 1 1) (thickness 0.15)))
     )
@@
     (tags "LED")
     (property "MFG" "SunLed")
-    (property "MPN" "XZVGR68W-3")
+    (property "MPN" "XZVG68W-2")
     (property "Sheetfile" "nic2.kicad_sch")
     (property "Sheetname" "")
@@
       (effects (font (size 1 1) (thickness 0.15)))
     )
-    (fp_text value "LED" (at 0 1.17) (layer "F.Fab")
+    (fp_text value "LED_GREEN" (at 0 1.17) (layer "F.Fab")
       (effects (font (size 1 1) (thickness 0.15)))
     )
@@
       (effects (font (size 1 1) (thickness 0.15)))
     )
-    (fp_text value "LED" (at 0 1.17) (layer "F.Fab")
+    (fp_text value "LED_RED" (at 0 1.17) (layer "F.Fab")
       (effects (font (size 1 1) (thickness 0.15)))
     )
@@
       (effects (font (size 1 1) (thickness 0.15)))
     )
-    (fp_text value "LED" (at 0 1.17) (layer "F.Fab")
-      (effects (font (size 1 1) (thickness 0.15)))
-    )
+    (fp_text value "LED_BLUE" (at 0 1.17) (layer "F.Fab")
+      (effects (font (size 1 1) (thickness 0.15)))
+    )
