File: nic2/nic2.kicad_pcb (KiCad board)
At the start: 4 copper layers, 70.8 x 47 mm, 47 parts, among them J1 Conn_2Rows-41Pins, J2 Wuerth_74980111211, J3 Wuerth_74980111211, U1 KSZ8463FRLI, U2 TPD4S010DQAR, U3 TPD4S010DQAR, X1 ASE-25.000MHZ-LC

Commit message: Updates to NIC (#44)
* Updates to NIC

* Add NRST LED

* Fix LED colors in BOM
Parts:
- removed TP1: TestPoint, TestPoint:TestPoint_Pad_2.5x2.5mm
- removed TP2, TP3, TP5, TP6, TP7, TP8: TestPoint, TestPoint:TestPoint_Keystone_5015_Micro-Minature
- added D1: LED_RED, LED_SMD:LED_0402_1005Metric, F.Cu at (169.2, 95.7)
- added D2: LED_ORANGE, LED_SMD:LED_0402_1005Metric, F.Cu at (169.2, 94.5)
- added D4: LED_BLUE, LED_SMD:LED_0402_1005Metric, F.Cu at (169.2, 92.0)
- added D5: LED_GREEN, LED_SMD:LED_0402_1005Metric, F.Cu at (152.2, 59.8)
- added D6: LED_GREEN, LED_SMD:LED_0402_1005Metric, F.Cu at (170.5, 60.5)
- added H3: MountingHole_Pad, MountingHole:MountingHole_3.2mm_M3_DIN965_Pad, F.Cu at (122.0, 51.0)
- added H4: MountingHole_Pad, MountingHole:MountingHole_3.2mm_M3_DIN965_Pad, F.Cu at (122.0, 106.2)
- added J4: Conn_01x07_Male, Connector_PinHeader_2.54mm:PinHeader_1x07_P2.54mm_Vertical, F.Cu at (167.4, 57.5)
- added R13: 143Ω, Resistor_SMD:R_0402_1005Metric, F.Cu at (171.2, 95.7)
- added R14: 143Ω, Resistor_SMD:R_0402_1005Metric, F.Cu at (171.2, 94.5)
- added R15: 143Ω, Resistor_SMD:R_0402_1005Metric, F.Cu at (171.2, 93.2)
- added R16: 143Ω, Resistor_SMD:R_0402_1005Metric, F.Cu at (171.2, 92.0)
- added R17: 143Ω, Resistor_SMD:R_0402_1005Metric, F.Cu at (170.5, 61.5)
- C13, R11: moved to B.Cu
- D3: value LED -> LED_GREEN
- FB1: footprint Resistor_SMD:R_0603_1608Metric -> Resistor_SMD:R_0402_1005Metric
- moved D3 34.0 mm to (169.2, 93.2)
- moved LOGO1 7.32 mm to (157.7, 90.6)
- moved R12 4.17 mm to (152.2, 61.0)
- moved C13 3.14 mm to (140.6, 77.8)
- moved R11 3.14 mm to (140.6, 79.0)
- moved FID1 1.75 mm to (143.2, 57.5)
Connections:
- D3 pad 2: +3V3 -> Net-(D3-Pad2)
- R12 pad 2: Net-(D3-Pad1) -> Net-(D5-Pad1)
- U1 pad 52: unconnected-(U1-Pad52) -> Net-(D4-Pad2)
- U1 pad 53: unconnected-(U1-Pad53) -> Net-(D3-Pad2)
- U1 pad 54: unconnected-(U1-Pad54) -> Net-(D2-Pad2)
- U1 pad 55: unconnected-(U1-Pad55) -> Net-(D1-Pad2)
Routing:
- net Net-(D1-Pad2): track 0.00 -> 30.9 mm, vias 0 -> 2
- net Net-(D2-Pad2): track 0.00 -> 28.5 mm, vias 0 -> 2
- net Net-(D3-Pad2): track 0.00 -> 25.6 mm, vias 0 -> 2
- net Net-(D4-Pad2): track 0.00 -> 24.0 mm, vias 0 -> 2
- net /SPI4_SCK: track 34.8 -> 48.7 mm
- net /SPI4_MOSI: track 39.3 -> 50.2 mm, vias 3 -> 5
- net /~{SPI4_RESET}: track 40.7 -> 50.8 mm, vias 1 -> 2
- net Earth: track 3.80 -> 11.3 mm, vias 0 -> 23
- net /SPI4_MISO: track 45.1 -> 50.3 mm
- net /~{SPI4_CS}: track 40.0 -> 42.7 mm, vias 3 -> 1
- net /P1LED0: track 24.7 -> 22.8 mm
- net GND: track 55.4 -> 57.2 mm, vias 34 -> 38
- net Net-(D5-Pad1): track 0.00 -> 1.26 mm
- net Net-(D6-Pad1): track 0.00 -> 1.01 mm
- net Net-(D2-Pad1): track 0.00 -> 1.01 mm
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- added copper zone on B.Cu, net Earth
- added copper zone on In1.Cu, net Earth
- added copper zone on In2.Cu, net Earth
Other:
- board size 70.8 x 47 mm -> 70.8 x 66.5 mm
- board text added: "3V3"
- board text added: "Gimletlet NIC 2 Rev B MJK 4/2022"
- board text added: "PORT 1"
- board text added: "PORT 2"
- board text added: "~{RST}"
- board text removed: "+3V3"
- board text removed: "Gimletlet NIC 2 Rev A MJK 1/2022"
- board text removed: "RST"
