File: nic2/nic2.kicad_sch (KiCad schematic)
At the start: 37 parts, among them J1 Conn_2Rows-41Pins, J2 Wuerth_74980111211, J3 Wuerth_74980111211, U1 KSZ8463FRLI, X1 ASE-25.000MHZ-LC

Commit message: Tweaks to NIC before review
Parts:
- added C14: 10 µF, Capacitor_SMD:C_0805_2012Metric, symbol Device:C
- added D3: LED, LED_SMD:LED_0402_1005Metric, symbol Device:LED
- added R12: 143Ω, Resistor_SMD:R_0402_1005Metric, symbol Device:R
- added TP1, TP2: TestPoint, TestPoint:TestPoint_Pad_2.5x2.5mm, symbol Connector:TestPoint
- C1, C3, C4, C5, C6, C7, C8: MFG (none) -> KEMET; MPN (none) -> C0402C105K9PAC7800
- C10, C11, C12, C9: MFG (none) -> KEMET; MPN (none) -> C0402C104K9RAC7867
- C13: MFG (none) -> KEMET; MPN (none) -> C0402C472K3RAC7867
- C2: footprint Capacitor_SMD:C_0402_1005Metric -> Capacitor_SMD:C_0805_2012Metric; MFG (none) -> KEMET; MPN (none) -> C0805C106K9RAC7800
- D1, D2: MFG (none) -> Vishay; MPN (none) -> 1N4148W-G3-18
- FB1: MFG (none) -> Murata Electronics
- J2, J3: MFG (none) -> Würth Elektronik; MPN (none) -> 74980111211
- R1, R2, R5: MFG (none) -> TE Connectivity; MPN (none) -> CRG0402F10K
- R10, R7, R8, R9: MFG (none) -> YAGEO; MPN (none) -> RC0402FR-07143RL
- R11: MFG (none) -> TE Connectivity; MPN (none) -> CRG0402F1M0
- R3, R6: MFG (none) -> TE Connectivity; MPN (none) -> CRG0402F4K7
- R4: MFG (none) -> YAGEO; MPN (none) -> RC0402FR-076K49L
- U1: MFG (none) -> Microchip Technology; MPN (none) -> KSZ8463FRLI
- X1: MFG (none) -> Abracon LLC; MPN (none) -> ASE-25.000MHZ-LC-T
Connections:
- net +3V3: now also C14.2, D3.2 (A), TP1.1
- net GND: now also C14.1, R12.1, TP2.1
- new net: D3.1 (K), R12.2
Other:
- note added: "Power LED and bulk capacitance"

Commit message: Update NIC2 per review
Parts:
- removed C2: 10 µF, Capacitor_SMD:C_0805_2012Metric, symbol Device:C
- removed D1, D2: 1N4148W, Diode_SMD:D_SOD-123, symbol Diode:1N4148W
- added TP3, TP5, TP6, TP7, TP8: TestPoint, TestPoint:TestPoint_Keystone_5015_Micro-Minature, symbol Connector:TestPoint
- added U2, U3: TPD4S010DQAR, Package_SON:USON-10_2.5x1.0mm_P0.5mm, symbol Power protection (Oxide):TPD4S010DQAR
- TP2: footprint TestPoint:TestPoint_Pad_2.5x2.5mm -> TestPoint:TestPoint_Keystone_5015_Micro-Minature
Connections:
- net +3V3: no longer R2.2
- net GND: now also R2.1, U2.3 (GND), U2.8 (GND), U3.3 (GND), U3.8 (GND)
- net RX1_N: now also U2.5 (D2-), U2.6 (NC)
- net RX1_P: now also U2.4 (D2+), U2.7 (NC)
- net RX2_N: now also U3.5 (D2-), U3.6 (NC)
- net RX2_P: now also U3.4 (D2+), U3.7 (NC)
- net SPI4_MISO: now also TP7.1
- net SPI4_MOSI: now also TP8.1
- net SPI4_SCK: now also TP6.1
- net TX1_N: now also U2.2 (D1-), U2.9 (NC)
- net TX1_P: now also U2.1 (D1+), U2.10 (NC)
- net TX2_N: now also U3.2 (D1-), U3.9 (NC)
- net TX2_P: now also U3.1 (D1+), U3.10 (NC)
- net ~{SPI4_CS}: now also TP3.1
- net ~{SPI4_RESET}: now also R2.2, U1.63 (~{RST}), TP5.1
Other:
- note added: "The datasheet has a more complicated reset circuit (to do a delayed reset at power on), but we can handle that sequencing from the SP."
- note removed: "RC reset circuit from datasheet"
- company: (none) -> Oxide Computer Company
- title: (none) -> Gimletlet NIC 2
- moved on the sheet: C10, C11, C12, C13, C9, J2, J3, R10, R11, R2, R7, R8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

Commit message: Add Oxide wordmark
Parts:
- added LOGO1: LOGO, Logos_0x:OXIDE_Wordmark, symbol Logos_0x:LOGO
Changed lines of the file:
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@@
     (pin "1")
+  )
+  (symbol (lib_id "Logos_0x:LOGO") (at 314.96 194.31 0) (unit 1)
+    (in_bom no) (on_board yes) (fields_autoplaced)
+    (property "Reference" "LOGO1" (id 0) (at 320.04 192.4049 0)
+      (effects (font (size 1.27 1.27)) (justify left))
+    )
+    (property "Value" "LOGO" (id 1) (at 313.69 189.23 0)
+      (effects (font (size 1.27 1.27)) hide)
+    )
+    (property "Footprint" "Logos_0x:OXIDE_Wordmark" (id 2) (at 314.96 194.31 0)
+      (effects (font (size 1.27 1.27)) hide)
+    )
+    (property "Datasheet" "" (id 3) (at 314.96 194.31 0)
+      (effects (font (size 1.27 1.27)) hide)
+    )
   )
   (symbol (lib_id "power:GND") (at 93.98 128.27 90) (unit 1)
@@
       (reference "J3") (unit 1) (value "Wuerth_74980111211") (footprint "Connector_RJ:RJ45_Wuerth_74980111211_Horizontal")
     )
+    (path "/9e9e764f-20c0-4905-9d52-5781906b4576"
+      (reference "LOGO1") (unit 1) (value "LOGO") (footprint "Logos_0x:OXIDE_Wordmark")
+    )
     (path "/8a8ecf43-d848-404e-9132-8b8e8fc31a3b"

Commit message: Add MFG and MPN for remaining parts
Parts:
- TP2, TP3, TP5, TP6, TP7, TP8: MFG (none) -> Keystone Electronics; MPN (none) -> 5015
- U2, U3: MFG (none) -> Texas Instruments; MPN (none) -> TPD4S010DQAR
Changed lines of the file:
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@@
+      (effects (font (size 1.27 1.27)) hide)
+    )
+    (property "MFG" "Keystone Electronics" (id 4) (at 67.31 120.65 0)
+      (effects (font (size 1.27 1.27)) hide)
+    )
+    (property "MPN" "5015" (id 5) (at 67.31 120.65 0)
       (effects (font (size 1.27 1.27)) hide)
     )
@@
     )
     (property "Datasheet" "~" (id 3) (at 67.31 120.65 0)
+      (effects (font (size 1.27 1.27)) hide)
+    )
+    (property "MFG" "Keystone Electronics" (id 4) (at 67.31 125.73 0)
+      (effects (font (size 1.27 1.27)) hide)
+    )
+    (property "MPN" "5015" (id 5) (at 67.31 125.73 0)
       (effects (font (size 1.27 1.27)) hide)
     )
@@
     )
     (property "Datasheet" "https://www.ti.com/lit/ds/symlink/tpd4s010.pdf" (id 3) (at 311.15 124.46 0)
+      (effects (font (size 1.27 1.27)) hide)
+    )
+    (property "MFG" "Texas Instruments" (id 4) (at 311.15 124.46 0)
+      (effects (font (size 1.27 1.27)) hide)
+    )
+    (property "MPN" "TPD4S010DQAR" (id 5) (at 311.15 124.46 0)
       (effects (font (size 1.27 1.27)) hide)
     )
@@
       (effects (font (size 1.27 1.27)) hide)
     )
+    (property "MFG" "Keystone Electronics" (id 4) (at 109.22 120.65 0)
+      (effects (font (size 1.27 1.27)) hide)
+    )
+    (property "MPN" "5015" (id 5) (at 109.22 120.65 0)
+      (effects (font (size 1.27 1.27)) hide)
+    )
     (pin "1")
   )
@@
     )
     (property "Datasheet" "https://www.ti.com/lit/ds/symlink/tpd4s010.pdf" (id 3) (at 311.15 71.12 0)
+      (effects (font (size 1.27 1.27)) hide)
+    )
+    (property "MFG" "Texas Instruments" (id 4) (at 311.15 71.12 0)
+      (effects (font (size 1.27 1.27)) hide)
+    )
+    (property "MPN" "TPD4S010DQAR" (id 5) (at 311.15 71.12 0)
       (effects (font (size 1.27 1.27)) hide)
     )
@@
       (effects (font (size 1.27 1.27)) hide)
     )
+    (property "MFG" "Keystone Electronics" (id 4) (at 99.06 57.15 0)
+      (effects (font (size 1.27 1.27)) hide)
+    )
+    (property "MPN" "5015" (id 5) (at 99.06 57.15 0)
+      (effects (font (size 1.27 1.27)) hide)
+    )
     (pin "1")
   )
@@
     )
     (property "Datasheet" "~" (id 3) (at 109.22 128.27 0)
+      (effects (font (size 1.27 1.27)) hide)
+    )
+    (property "MFG" "Keystone Electronics" (id 4) (at 109.22 123.19 0)
+      (effects (font (size 1.27 1.27)) hide)
+    )
+    (property "MPN" "5015" (id 5) (at 109.22 123.19 0)
       (effects (font (size 1.27 1.27)) hide)
     )
@@
       (effects (font (size 1.27 1.27)) hide)
     )
+    (property "MFG" "Keystone Electronics" (id 4) (at 109.22 125.73 0)
+      (effects (font (size 1.27 1.27)) hide)
+    )
+    (property "MPN" "5015" (id 5) (at 109.22 125.73 0)
+      (effects (font (size 1.27 1.27)) hide)
+    )

Commit message: Updates to NIC
Parts:
- removed TP1: TestPoint, TestPoint:TestPoint_Pad_2.5x2.5mm, symbol Connector:TestPoint
- removed TP2, TP3, TP5, TP6, TP7, TP8: TestPoint, TestPoint:TestPoint_Keystone_5015_Micro-Minature, symbol Connector:TestPoint
- added D1, D2, D3: LED, LED_SMD:LED_0402_1005Metric, symbol Device:LED
- added D4: (no value), symbol Device:LED
- added H3, H4: MountingHole_Pad, MountingHole:MountingHole_3.2mm_M3_DIN965_Pad, symbol Mechanical:MountingHole_Pad
- added J4: Conn_01x07_Male, Connector_PinHeader_2.54mm:PinHeader_1x07_P2.54mm_Vertical, symbol Connector:Conn_01x07_Male
- added R13, R14, R15, R16: 143Ω, Resistor_SMD:R_0402_1005Metric, symbol Device:R
- FB1: footprint Resistor_SMD:R_0603_1608Metric -> Resistor_SMD:R_0402_1005Metric
- renumbered D3 to D5
Connections:
- net +3V3: now also J4.7 (Pin_7)
- net Earth: now also H3.1, H4.1
- net GND: now also J4.1 (Pin_1), R13.1, R14.1, R15.1, R16.1
- net SPI4_MISO: now also J4.5 (Pin_5)
- net SPI4_MOSI: now also J4.4 (Pin_4)
- net SPI4_SCK: now also J4.6 (Pin_6)
- net ~{SPI4_CS}: now also J4.3 (Pin_3)
- net ~{SPI4_RESET}: now also J4.2 (Pin_2)
- net at U1.52 (GPIO2): now also D4.2 (A)
- net at U1.53 (GPIO3): now also D3.2 (A)
- net at U1.54 (GPIO4): now also D2.2 (A)
- net at U1.55 (GPIO5): now also D1.2 (A)
- new net: D4.1 (K), R16.2
- new net: D3.1 (K), R15.2
- new net: D1.1 (K), R13.2
- new net: D2.1 (K), R14.2
Other:
- note added: "Debug header"

Commit message: Add NRST LED
Parts:
- added D6: LED, LED_SMD:LED_0402_1005Metric, symbol Device:LED
- added R17: 143Ω, Resistor_SMD:R_0402_1005Metric, symbol Device:R
Connections:
- net GND: now also R17.1
- net ~{SPI4_RESET}: now also D6.2 (A)
- new net: D6.1 (K), R17.2
Changed lines of the file:
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@@
   (junction (at 372.11 154.94) (diameter 0) (color 0 0 0 0)
   )
+  (junction (at 124.46 158.75) (diameter 0) (color 0 0 0 0)
+  )
   (junction (at 173.99 217.17) (diameter 0) (color 0 0 0 0)
   )
@@
     (stroke (width 0) (type default) (color 0 0 0 0))
   )
-  (wire (pts (xy 109.22 158.75) (xy 137.16 158.75))
+  (wire (pts (xy 109.22 158.75) (xy 124.46 158.75))
     (stroke (width 0) (type default) (color 0 0 0 0))
   )
@@
     (stroke (width 0) (type default) (color 0 0 0 0))
   )
+  (wire (pts (xy 124.46 168.91) (xy 124.46 166.37))
+    (stroke (width 0) (type default) (color 0 0 0 0))
+  )
   (wire (pts (xy 93.98 95.25) (xy 109.22 95.25))
     (stroke (width 0) (type default) (color 0 0 0 0))
@@
     (stroke (width 0) (type default) (color 0 0 0 0))
   )
+  (wire (pts (xy 124.46 158.75) (xy 137.16 158.75))
+    (stroke (width 0) (type default) (color 0 0 0 0))
+  )
   (wire (pts (xy 158.75 130.81) (xy 173.99 130.81))
     (stroke (width 0) (type default) (color 0 0 0 0))
@@
     (pin "2")
   )
+  (symbol (lib_id "Device:R") (at 124.46 172.72 180) (unit 1)
+    (in_bom yes) (on_board yes)
+    (property "Reference" "R17" (id 0) (at 121.92 172.72 90))
+    (property "Value" "143Ω" (id 1) (at 127 172.72 90))
+    (property "Footprint" "Resistor_SMD:R_0402_1005Metric" (id 2) (at 126.238 172.72 90)
+      (effects (font (size 1.27 1.27)) hide)
+    )
+    (property "Datasheet" "~" (id 3) (at 124.46 172.72 0)
+      (effects (font (size 1.27 1.27)) hide)
+    )
+    (property "MFG" "YAGEO" (id 4) (at 124.46 172.72 0)
+      (effects (font (size 1.27 1.27)) hide)
+    )
+    (property "MPN" "RC0402FR-07143RL" (id 5) (at 124.46 172.72 0)
+      (effects (font (size 1.27 1.27)) hide)
+    )
+    (pin "1")
+    (pin "2")
+  )
   (symbol (lib_id "power:GND") (at 137.16 166.37 0) (unit 1)
     (in_bom yes) (on_board yes)
@@
     (pin "1")
   )
+  (symbol (lib_id "power:GND") (at 124.46 176.53 0) (unit 1)
+    (in_bom yes) (on_board yes)
+    (property "Reference" "#PWR045" (id 0) (at 124.46 182.88 0)
+      (effects (font (size 1.27 1.27)) hide)
+    )
+    (property "Value" "GND" (id 1) (at 121.92 180.34 0)
+      (effects (font (size 1.27 1.27)) (justify left))
+    )
+    (property "Footprint" "" (id 2) (at 124.46 176.53 0)
+      (effects (font (size 1.27 1.27)) hide)
+    )
+    (property "Datasheet" "" (id 3) (at 124.46 176.53 0)
+      (effects (font (size 1.27 1.27)) hide)
+    )
+    (pin "1")
+  )
   (symbol (lib_id "power:GND") (at 93.98 107.95 90) (unit 1)
     (in_bom yes) (on_board yes)
@@
     (pin "2")
   )
+  (symbol (lib_id "Device:LED") (at 124.46 162.56 90) (unit 1)
+    (in_bom yes) (on_board yes) (fields_autoplaced)
+    (property "Reference" "D6" (id 0) (at 128.27 162.8774 90)
+      (effects (font (size 1.27 1.27)) (justify right))
+    )
+    (property "Value" "LED" (id 1) (at 128.27 165.4174 90)
+      (effects (font (size 1.27 1.27)) (justify right))
+    )
+    (property "Footprint" "LED_SMD:LED_0402_1005Metric" (id 2) (at 124.46 162.56 0)
+      (effects (font (size 1.27 1.27)) hide)
+    )
+    (property "Datasheet" "~" (id 3) (at 124.46 162.56 0)
+      (effects (font (size 1.27 1.27)) hide)
+    )
+    (property "MFG" "SunLed" (id 4) (at 124.46 162.56 0)
+      (effects (font (size 1.27 1.27)) hide)
+    )
+    (property "MPN" "XZVGR68W-3" (id 5) (at 124.46 162.56 0)
+      (effects (font (size 1.27 1.27)) hide)
+    )
+    (pin "1")
+    (pin "2")
+  )
   (symbol (lib_id "power:GND") (at 264.16 214.63 0) (unit 1)
     (in_bom yes) (on_board yes) (fields_autoplaced)
@@
       (reference "#PWR044") (unit 1) (value "GND") (footprint "")
     )
+    (path "/d18df553-9af1-44a0-a914-ea3192f344ac"
+      (reference "#PWR045") (unit 1) (value "GND") (footprint "")
+    )
     (path "/32b5234c-818b-49f1-a2b7-7d2751860c55"
       (reference "#PWR0101") (unit 1) (value "Earth") (footprint "")
@@
       (reference "D5") (unit 1) (value "LED") (footprint "LED_SMD:LED_0402_1005Metric")
     )
+    (path "/de975495-8370-449e-a7b1-45b734f1373e"
+      (reference "D6") (unit 1) (value "LED") (footprint "LED_SMD:LED_0402_1005Metric")
+    )
     (path "/bcebba2f-e391-44fb-b605-8e293bf73adb"
       (reference "FB1") (unit 1) (value "FerriteBead") (footprint "Resistor_SMD:R_0402_1005Metric")
@@
       (reference "R16") (unit 1) (value "143Ω") (footprint "Resistor_SMD:R_0402_1005Metric")
     )
+    (path "/4e1e01e0-bf25-4182-98aa-c2435302bac7"
+      (reference "R17") (unit 1) (value "143Ω") (footprint "Resistor_SMD:R_0402_1005Metric")
+    )
     (path "/bd370485-a322-4122-9614-51f744a64f3e"

Commit message: Fix LED colors in BOM
Parts:
- C1, C3, C4, C5, C6, C7, C8: value 1 µF -> (none); footprint Capacitor_SMD:C_0402_1005Metric -> (none)
- C10, C11, C12, C9: value 0.1 µF -> (none); footprint Capacitor_SMD:C_0402_1005Metric -> (none)
- C13: value 4700 pF -> (none); footprint Capacitor_SMD:C_0402_1005Metric -> (none)
- C14: value 10 µF -> (none); footprint Capacitor_SMD:C_0805_2012Metric -> (none)
- D1, D2, D5: value LED -> (none); footprint LED_SMD:LED_0402_1005Metric -> (none)
- D3, D6: value LED -> (none); footprint LED_SMD:LED_0402_1005Metric -> (none); MPN XZVGR68W-3 -> XZVG68W-2
- FB1: value FerriteBead -> (none); footprint Resistor_SMD:R_0402_1005Metric -> (none)
- FID1, FID2, FID3: value Fiducial -> (none); footprint Fiducial:Fiducial_0.75mm_Mask1.5mm -> (none)
- H1, H2: value MountingHole -> (none); footprint MountingHole:MountingHole_3.2mm_M3 -> (none)
- H3, H4: value MountingHole_Pad -> (none); footprint MountingHole:MountingHole_3.2mm_M3_DIN965_Pad -> (none)
- J1: value Conn_2Rows-41Pins -> (none); footprint Connectors_0x:DF9-41P-1V -> (none)
- J2, J3: value Wuerth_74980111211 -> (none); footprint Connector_RJ:RJ45_Wuerth_74980111211_Horizontal -> (none)
- J4: value Conn_01x07_Male -> (none); footprint Connector_PinHeader_2.54mm:PinHeader_1x07_P2.54mm_Vertical -> (none)
- LOGO1: value LOGO -> (none); footprint Logos_0x:OXIDE_Wordmark -> (none)
- R1, R2, R5: value 10KΩ -> (none); footprint Resistor_SMD:R_0402_1005Metric -> (none)
- R10, R12, R13, R14, R15, R16, R17, R7, R8, R9: value 143Ω -> (none); footprint Resistor_SMD:R_0402_1005Metric -> (none)
- R11: value 1 MΩ -> (none); footprint Resistor_SMD:R_0402_1005Metric -> (none)
- R3, R6: value 4.7 KΩ -> (none); footprint Resistor_SMD:R_0402_1005Metric -> (none)
- R4: value 6.49 KΩ -> (none); footprint Resistor_SMD:R_0402_1005Metric -> (none)
- U1: value KSZ8463FRLI -> (none); footprint Package_QFP:LQFP-64_10x10mm_P0.5mm -> (none)
- U2, U3: value TPD4S010DQAR -> (none); footprint Package_SON:USON-10_2.5x1.0mm_P0.5mm -> (none)
- X1: value ASE-25.000MHZ-LC -> (none); footprint Oscillator:Oscillator_SMD_Abracon_ASE-4Pin_3.2x2.5mm -> (none)
