File: nic2/nic2.kicad_sch (KiCad schematic)
At the start: 47 parts, among them J1 Conn_2Rows-41Pins, J2 Wuerth_74980111211, J3 Wuerth_74980111211, U1 KSZ8463FRLI, U2 TPD4S010DQAR, U3 TPD4S010DQAR, X1 ASE-25.000MHZ-LC

Commit message: Updates to NIC (#44)
* Updates to NIC

* Add NRST LED

* Fix LED colors in BOM
Parts:
- removed TP1: TestPoint, TestPoint:TestPoint_Pad_2.5x2.5mm, symbol Connector:TestPoint
- removed TP2, TP3, TP5, TP6, TP7, TP8: TestPoint, TestPoint:TestPoint_Keystone_5015_Micro-Minature, symbol Connector:TestPoint
- added D1, D2, D3, D4, D6: (no value), symbol Device:LED
- added H3, H4: (no value), symbol Mechanical:MountingHole_Pad
- added J4: (no value), symbol Connector:Conn_01x07_Male
- added R13, R14, R15, R16, R17: (no value), symbol Device:R
- C1, C3, C4, C5, C6, C7, C8: value 1 µF -> (none); footprint Capacitor_SMD:C_0402_1005Metric -> (none)
- C10, C11, C12, C9: value 0.1 µF -> (none); footprint Capacitor_SMD:C_0402_1005Metric -> (none)
- C13: value 4700 pF -> (none); footprint Capacitor_SMD:C_0402_1005Metric -> (none)
- C14: value 10 µF -> (none); footprint Capacitor_SMD:C_0805_2012Metric -> (none)
- D5: renamed from D3; value LED -> (none); footprint LED_SMD:LED_0402_1005Metric -> (none)
- FB1: value FerriteBead -> (none); footprint Resistor_SMD:R_0603_1608Metric -> (none)
- FID1, FID2, FID3: value Fiducial -> (none); footprint Fiducial:Fiducial_0.75mm_Mask1.5mm -> (none)
- H1, H2: value MountingHole -> (none); footprint MountingHole:MountingHole_3.2mm_M3 -> (none)
- J1: value Conn_2Rows-41Pins -> (none); footprint Connectors_0x:DF9-41P-1V -> (none)
- J2, J3: value Wuerth_74980111211 -> (none); footprint Connector_RJ:RJ45_Wuerth_74980111211_Horizontal -> (none)
- LOGO1: value LOGO -> (none); footprint Logos_0x:OXIDE_Wordmark -> (none)
- R1, R2, R5: value 10KΩ -> (none); footprint Resistor_SMD:R_0402_1005Metric -> (none)
- R10, R12, R7, R8, R9: value 143Ω -> (none); footprint Resistor_SMD:R_0402_1005Metric -> (none)
- R11: value 1 MΩ -> (none); footprint Resistor_SMD:R_0402_1005Metric -> (none)
- R3, R6: value 4.7 KΩ -> (none); footprint Resistor_SMD:R_0402_1005Metric -> (none)
- R4: value 6.49 KΩ -> (none); footprint Resistor_SMD:R_0402_1005Metric -> (none)
- U1: value KSZ8463FRLI -> (none); footprint Package_QFP:LQFP-64_10x10mm_P0.5mm -> (none)
- U2, U3: value TPD4S010DQAR -> (none); footprint Package_SON:USON-10_2.5x1.0mm_P0.5mm -> (none)
- X1: value ASE-25.000MHZ-LC -> (none); footprint Oscillator:Oscillator_SMD_Abracon_ASE-4Pin_3.2x2.5mm -> (none)
Connections:
- net +3V3: now also J4.7 (Pin_7)
- net Earth: now also H3.1, H4.1
- net GND: now also J4.1 (Pin_1), R13.1, R14.1, R15.1, R16.1, R17.1
- net SPI4_MISO: now also J4.5 (Pin_5)
- net SPI4_MOSI: now also J4.4 (Pin_4)
- net SPI4_SCK: now also J4.6 (Pin_6)
- net ~{SPI4_CS}: now also J4.3 (Pin_3)
- net ~{SPI4_RESET}: now also D6.2 (A), J4.2 (Pin_2)
- net at U1.52 (GPIO2): now also D4.2 (A)
- net at U1.53 (GPIO3): now also D3.2 (A)
- net at U1.54 (GPIO4): now also D2.2 (A)
- net at U1.55 (GPIO5): now also D1.2 (A)
- new net: D4.1 (K), R16.2
- new net: D3.1 (K), R15.2
- new net: D6.1 (K), R17.2
- new net: D1.1 (K), R13.2
- new net: D2.1 (K), R14.2
Other:
- note added: "Debug header"
