File: gimletlet-lpc55-adapter/gimletlet-lpc55-adapter.kicad_pcb (KiCad board)
At the start: 4 copper layers, 55 x 75 mm, 26 parts, among them J1 Conn_02x06_Odd_Even, J2 Conn_ARM_JTAG_SWD_10, J3 Conn_2Rows-51Pins, J4 USART, J5 Conn_01x06, J6 SPI, SW1 SW_SPST, SW2 SW_SPDT

Commit message: Update BOM
Parts:
- removed H111: GRAPHIC PLACEHOLDER, grumpy:newt_of_trust
- added C2: 1µF, Capacitor_SMD:C_0603_1608Metric, F.Cu at (80.1, 98.4)
- added C3: 1µF, Capacitor_SMD:C_0603_1608Metric, F.Cu at (103.0, 92.2)
- added H3: GRAPHIC PLACEHOLDER, grumpy:newt_of_trust, F.Cu at (79.8, 67.2)
- added R4: 22Ω, Resistor_SMD:R_0603_1608Metric, F.Cu at (109.0, 88.2)
- added R5: 22Ω, Resistor_SMD:R_0603_1608Metric, F.Cu at (114.2, 88.2)
- C1: value 0.1uF -> 1µF
- R1, R2, R3: value 68R -> 143Ω
- moved SW1 2.50 mm to (86.5, 40.0)
- moved C1 2.00 mm to (99.0, 36.0)
- moved J2 0.50 mm to (94.2, 40.0)
Connections:
- J3 pad 12: /FC3_RXD_DSA_MOSI -> Net-(J3-Pad12)
- J3 pad 4: /FC3_SCK -> Net-(J3-Pad4)
- J5 pad 1: GND -> +3V3
- J5 pad 2: +3V3 -> GND
- J6 pad 1: /FC3_CTS_SDAX_SSEL0 -> +3V3
- J6 pad 2: /FC3_RXD_DSA_MOSI -> GND
- J6 pad 3: /FC3_TXD_SCL_MISO -> /FC3_SCK
- J6 pad 4: /FC3_SCK -> /FC3_TXD_SCL_MISO
- J6 pad 5: GND -> /FC3_RXD_DSA_MOSI
- J6 pad 6: +3V3 -> /FC3_CTS_SDAX_SSEL0
Routing:
- net /FC3_RXD_DSA_MOSI: track 29.0 -> 7.72 mm, vias 0 -> 1
- net Net-(J3-Pad12): track 0.00 -> 15.3 mm
- net /FC3_SCK: track 20.1 -> 7.11 mm, vias 1 -> 0
- net Net-(J3-Pad4): track 0.00 -> 12.1 mm
- net /FC3_CTS_SDAX_SSEL0: track 45.3 -> 34.4 mm, vias 2 -> 0
- net GND: track 47.1 -> 52.9 mm
- net +3V3: track 19.1 -> 24.7 mm
- net /SPI_MOSI: track 46.2 -> 51.7 mm
- net /~{SWD_RESET}: track 38.8 -> 41.8 mm
- net /PIO0_4: track 53.4 -> 52.7 mm
- net /SWD_TRACESWO: track 35.6 -> 35.0 mm
- net /SWD_CLK: track 31.6 -> 32.1 mm
Other:
- board text added: "HS_SPI"
