File: gimletlet-lpc55-adapter/gimletlet-lpc55-adapter.kicad_pcb (KiCad board)
At the start: 4 copper layers, 55 x 75 mm, 30 parts, among them J1 Conn_02x06_Odd_Even, J2 Conn_ARM_JTAG_SWD_10, J3 Conn_2Rows-51Pins, J4 USART, J5 Conn_01x06, J6 SPI, SW1 SW_SPST, SW2 SW_SPDT

Commit message: Updates from review (adding test points)
Parts:
- added R6: 10KΩ, Resistor_SMD:R_0603_1608Metric, F.Cu at (114.2, 48.8)
- added R7: 143Ω, Resistor_SMD:R_0603_1608Metric, F.Cu at (115.0, 92.0)
- added TP10: TestPoint, TestPoint:TestPoint_Pad_1.5x1.5mm, F.Cu at (76.2, 94.5)
- added TP11: TestPoint, TestPoint:TestPoint_Pad_1.5x1.5mm, F.Cu at (109.8, 92.2)
- added TP12: TestPoint, TestPoint:TestPoint_Pad_1.5x1.5mm, F.Cu at (73.7, 94.5)
- added TP13: TestPoint, TestPoint:TestPoint_Pad_1.5x1.5mm, F.Cu at (71.1, 94.5)
- added TP14: TestPoint, TestPoint:TestPoint_Pad_1.5x1.5mm, F.Cu at (73.7, 107.2)
- added TP15: TestPoint, TestPoint:TestPoint_Pad_1.5x1.5mm, F.Cu at (71.1, 107.2)
- added TP9: TestPoint, TestPoint:TestPoint_Pad_1.5x1.5mm, F.Cu at (68.6, 94.5)
- D1: value Red -> Green
- moved R4 4.14 mm to (107.2, 92.0), turned to 90 degrees
- moved R5 4.14 mm to (112.5, 92.0), turned to 90 degrees
- moved C3 4.00 mm to (103.0, 96.2)
- moved J6 4.00 mm to (102.2, 99.0)
- moved SW2 3.76 mm to (91.8, 106.8)
- moved C2 3.43 mm to (80.0, 95.0)
- moved J5 1.99 mm to (81.3, 97.7)
- moved J4 0.89 mm to (81.3, 104.1)
Connections:
- J3 pad 32: /FC3_CTS_SDAX_SSEL0 -> Net-(J3-Pad32)
Routing:
- net Net-(J3-Pad32): track 0.00 -> 30.6 mm
- net /FC3_CTS_SDAX_SSEL0: track 34.4 -> 6.20 mm
- net /PIO0_25: track 57.8 -> 62.5 mm
- net /PIO0_4: track 52.7 -> 57.3 mm
- net /PIO0_22: track 59.0 -> 63.5 mm
- net /FC3_RTS_SCLX_SSEL1: track 62.6 -> 66.9 mm
- net Net-(J3-Pad12): track 15.3 -> 19.4 mm, vias 0 -> 2
- net Net-(J3-Pad4): track 12.1 -> 15.9 mm
- net /FC0_TXD: track 73.8 -> 77.2 mm
- net /FC0_RXD: track 70.8 -> 74.1 mm
- net /ISP0: track 28.3 -> 31.4 mm
- net /FC3_TXD_SCL_MISO: track 28.9 -> 31.5 mm
- net /FC3_RXD_DSA_MOSI: track 7.72 -> 6.22 mm, vias 1 -> 0
- net /~{SPI_CS}: track 47.0 -> 48.1 mm
- net +3V3: track 24.7 -> 25.7 mm, vias 10 -> 11
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Other:
- board size 55 x 75 mm -> 55 x 79 mm
