File: gimletlet-lpc55-adapter/gimletlet-lpc55-adapter.kicad_sch (KiCad schematic)
At the start: 25 parts, among them J2 Conn_ARM_JTAG_SWD_10, J3 Conn_2Rows-51Pins, J4 USART, SW1 SW_SPST, SW2 SW_SPDT

Commit message: Add title block
Other:
- company: (none) -> Oxide Computer Company
- title: (none) -> Gimletlet-LPC55 Adapter
Changed lines of the file:
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@@
 (kicad_sch (version 20211123) (generator eeschema)
   (paper "A4")
+  (title_block
+    (title "Gimletlet-LPC55 Adapter")
+    (date "2022-04-06")
+    (rev "A")
+    (company "Oxide Computer Company")
+    (comment 1 "matt@oxide.computer")
+    (comment 2 "Matt Keeter")
+  )
   (junction (at 175.26 53.975) (diameter 0) (color 0 0 0 0)
   )

Commit message: Update BOM
Parts:
- added C2, C3: (no value), symbol Device:C_Small
- added H3: (no value), symbol Mechanical:MountingHole
- added R4, R5: (no value), symbol Device:R
- C1: value 0.1uF -> (none); footprint Capacitor_SMD:C_0603_1608Metric -> (none); MPN C0603C104M4RACTU -> C0603C105K4RAC7867
- D1: value Red -> (none); footprint LED_SMD:LED_0603_1608Metric -> (none); MPN 150060RS75000 -> 150060GS75000
- D2: value Red -> (none); footprint LED_SMD:LED_0603_1608Metric -> (none)
- D3: value Amber -> (none); footprint LED_SMD:LED_0603_1608Metric -> (none)
- H1, H2: value M3 -> (none); footprint MountingHole:MountingHole_3.2mm_M3 -> (none)
- J1: MPN (none) -> PEC06DGBN; Mfg (none) -> Sullins Connector Solutions
- J2: value Conn_ARM_JTAG_SWD_10 -> (none); footprint Connector_PinHeader_1.27mm:PinHeader_2x05_P1.27mm_Vertical_SMD -> (none)
- J3: value Conn_2Rows-51Pins -> (none); footprint Oxide Connectors:DF9-51P-1V -> (none)
- J4: value USART -> (none); MPN (none) -> PR20206VBNN; Mfg (none) -> METZ CONNECT USA Inc.
- J5: MPN (none) -> PPTC061LFBN-RC; Mfg (none) -> Sullins Connector Solutions
- J6: MPN (none) -> PPPC061LGBN-RC; Mfg (none) -> Sullins Connector Solutions
- R1, R2, R3: value 68R -> (none); footprint Resistor_SMD:R_0603_1608Metric -> (none); MPN CR0603-JW-680ELF -> RC0603FR-07143RL; Mfg Bourns -> YAGEO; R_P 27mW -> (none)
- SW1: value SW_SPST -> (none); footprint Button_Switch_SMD:SW_SPST_PTS810 -> (none)
- SW2: value SW_SPDT -> (none); footprint Button_Switch_SMD:SW_SPDT_CK-JS102011SAQN -> (none)
- TP1: MPN (none) -> 5015; Mfg (none) -> Keystone Electronics
- TP2, TP3, TP4, TP5, TP6, TP7, TP8: value TestPoint -> (none); footprint TestPoint:TestPoint_Keystone_5015_Micro-Minature -> (none); MPN (none) -> 5015; Mfg (none) -> Keystone Electronics
Connections:
- net +3V3: now also J5.1 (Pin_1), J6.1 (Pin_1), C2.1, C3.1; no longer J5.2 (Pin_2), J6.6 (Pin_6)
- net FC3_CTS_SDAX_SSEL0: now also J6.6 (Pin_6); no longer J6.1 (Pin_1)
- net FC3_RXD_DSA_MOSI: now also J6.5 (Pin_5), R5.1; no longer J3.12 (Pin_12), J6.2 (Pin_2)
- net FC3_SCK: now also J6.3 (Pin_3), R4.1; no longer J3.4 (Pin_4), J6.4 (Pin_4)
- net FC3_TXD_SCL_MISO: now also J6.4 (Pin_4); no longer J6.3 (Pin_3)
- net GND: now also J5.2 (Pin_2), J6.2 (Pin_2), C2.2, C3.2; no longer J5.1 (Pin_1), J6.5 (Pin_5)
- new net: J3.4 (Pin_4), R4.2
- new net: J3.12 (Pin_12), R5.2
Other:
- note added: "Newt of Trust"

Commit message: Updates from review (adding test points)
Parts:
- added R6: (no value), symbol Device:R
- added R7: 143Ω, Resistor_SMD:R_0603_1608Metric, symbol Device:R
- added TP10, TP11, TP12, TP13, TP14, TP15: TestPoint, TestPoint:TestPoint_Pad_1.5x1.5mm, symbol Connector:TestPoint
- added TP9: TestPoint, symbol Connector:TestPoint
- C1, C2, C3: value (none) -> 1µF; footprint (none) -> Capacitor_SMD:C_0603_1608Metric
- D1: value (none) -> Green; footprint (none) -> LED_SMD:LED_0603_1608Metric
- D2: value (none) -> Red; footprint (none) -> LED_SMD:LED_0603_1608Metric
- D3: value (none) -> Amber; footprint (none) -> LED_SMD:LED_0603_1608Metric
- H1, H2: value (none) -> M3; footprint (none) -> MountingHole:MountingHole_3.2mm_M3
- H3: value (none) -> GRAPHIC PLACEHOLDER; footprint (none) -> grumpy:newt_of_trust
- J1: value (none) -> Conn_02x06_Odd_Even; footprint (none) -> Connector_PinHeader_2.54mm:PinHeader_2x06_P2.54mm_Horizontal
- J2: value (none) -> Conn_ARM_JTAG_SWD_10; footprint (none) -> Connector_PinHeader_1.27mm:PinHeader_2x05_P1.27mm_Vertical_SMD
- J3: value (none) -> Conn_2Rows-51Pins; footprint (none) -> Oxide Connectors:DF9-51P-1V
- J4: value (none) -> USART; footprint (none) -> Connector_PinHeader_2.54mm:PinHeader_1x06_P2.54mm_Vertical
- J5: value (none) -> Conn_01x06; footprint (none) -> Connector_PinSocket_2.54mm:PinSocket_1x06_P2.54mm_Vertical
- J6: value (none) -> SPI; footprint (none) -> Connector_PinSocket_2.54mm:PinSocket_1x06_P2.54mm_Horizontal
- R1, R2, R3: value (none) -> 143Ω; footprint (none) -> Resistor_SMD:R_0603_1608Metric
- R4, R5: value (none) -> 22Ω; footprint (none) -> Resistor_SMD:R_0603_1608Metric
- SW1: value (none) -> SW_SPST; footprint (none) -> Button_Switch_SMD:SW_SPST_PTS810
- SW2: value (none) -> SW_SPDT; footprint (none) -> Button_Switch_SMD:SW_SPDT_CK-JS102011SAQN
- TP1, TP2, TP3, TP4, TP5, TP6, TP7, TP8: value (none) -> TestPoint; footprint (none) -> TestPoint:TestPoint_Keystone_5015_Micro-Minature
Connections:
- net +3V3: now also R6.2
- net FC0_RXD: now also TP14.1
- net FC0_TXD: now also TP15.1
- net FC3_CTS_SDAX_SSEL0: now also R7.1; no longer J3.32 (Pin_32)
- net FC3_RTS_SCLX_SSEL1: now also TP9.1
- net FC3_TXD_SCL_MISO: now also TP11.1
- net PIO0_22: now also TP13.1
- net PIO0_25: now also TP12.1
- net PIO0_4: now also TP10.1
- net ~{SPI_CS}: now also R6.1
- new net: J3.32 (Pin_32), R7.2
Other:
- moved on the sheet: C3, J3, J6, R4, R5
